Commit message: update urdf.

File: pr2_defs/robots/hca.urdf.xacro (robot description, xacro)
@@ -19,5 +19,5 @@
     <inertial>
       <mass value="100" />
-      <com xyz=" 0 0 0 " />
+      <origin xyz=" 0 0 0 " />
       <inertia ixx="100"  ixy="0"  ixz="0" iyy="100" iyz="0" izz="100" />
     </inertial>
@@ -25,9 +25,6 @@
       <!-- 1.06m above ground -->
       <origin xyz="0 0 0" rpy="0 0 0 " />
-      <map name="gazebo_material" flag="gazebo">
-        <elem key="material">Gazebo/White</elem>
-      </map>
       <geometry name="unit_box">
-	<mesh scale=".6 0.45 1.06" />
+	<box size=".6 0.45 1.06" />
       </geometry>
     </visual>
@@ -39,4 +36,7 @@
     </collision>
   </link>
+  <gazebo reference="base_link">
+    <material>Gazebo/White</material>
+  </gazebo>
   <pr2_head_alpha2b name="head" parent="base_link">
     <!-- 213mm above tilt plate. Pan/tilt intersect is origin. -->

File: pr2_defs/robots/hcb.urdf.xacro (robot description, xacro)
@@ -19,5 +19,5 @@
     <inertial>
       <mass value="100" />
-      <com xyz=" 0 0 0 " />
+      <origin xyz=" 0 0 0 " />
       <inertia ixx="100"  ixy="0"  ixz="0" iyy="100" iyz="0" izz="100" />
     </inertial>
@@ -25,9 +25,6 @@
       <!-- 1.06m above ground -->
       <origin xyz="0 0 0" rpy="0 0 0 " />
-      <map name="gazebo_material" flag="gazebo">
-        <elem key="material">Gazebo/White</elem>
-      </map>
       <geometry name="unit_box">
-	<mesh scale=".6 0.45 1.06" />
+	<box size=".6 0.45 1.06" />
       </geometry>
     </visual>
@@ -39,4 +36,7 @@
     </collision>
   </link>
+  <gazebo reference="base_link">
+    <material>Gazebo/White</material>
+  </gazebo>
   <!-- These dimensions need to be checked -->
   <pr2_head name="head" parent="base_link">

File: pr2_defs/robots/hcc.urdf.xacro (robot description, xacro)
@@ -20,5 +20,5 @@
     <inertial>
       <mass value="100" />
-      <com xyz=" 0 0 0 " />
+      <origin xyz=" 0 0 0 " />
       <inertia ixx="100"  ixy="0"  ixz="0" iyy="100" iyz="0" izz="100" />
     </inertial>
@@ -26,9 +26,6 @@
       <!-- 1.06m above ground -->
       <origin xyz="0 0 0" rpy="0 0 0 " />
-      <map name="gazebo_material" flag="gazebo">
-        <elem key="material">Gazebo/White</elem>
-      </map>
       <geometry name="unit_box">
-	<mesh scale=".6 0.45 1.06" />
+	<box size=".6 0.45 1.06" />
       </geometry>
     </visual>
@@ -40,4 +37,7 @@
     </collision>
   </link>
+  <gazebo reference="base_link">
+    <material>Gazebo/White</material>
+  </gazebo>
   <!-- These dimensions need to be checked -->
   <pr2_head name="head" parent="base_link">

File: pr2_defs/robots/l_arm.urdf.xacro (robot description, xacro)
@@ -32,19 +32,16 @@
     <origin xyz="0 0 0" rpy="0 0 0" />
     <parent link="world" />
-    <child link="base_link" />
+    <child link="torso_lift_link" />
   </joint>
   <link name="torso_lift_link">
     <inertial>
       <mass value="1000" />
-      <com xyz="0 0 0" />
+      <origin xyz="0 0 0" />
       <inertia ixx="1000"  ixy="0"  ixz="0" iyy="1000" iyz="0" izz="1000" />
     </inertial>
     <visual>
       <origin xyz="0 0 0" rpy="0 0 0 " />
-      <map name="gazebo_material" flag="gazebo">
-        <elem key="material">PR2/White</elem>
-      </map>
       <geometry name="pr2_base_mesh_file">
-        <box scale="0.01 0.01 0.01" />
+        <box size="0.01 0.01 0.01" />
       </geometry>
     </visual>
@@ -52,13 +49,14 @@
       <origin xyz="0 0 0" rpy="0.0 0.0 0.0 " />
       <geometry name="base_collision_geom">
-        <box scale="0.01 0.01 0.01" />
+        <box size="0.01 0.01 0.01" />
       </geometry>
-      <map name="base_collision" flag="gazebo">
-        <elem key="mu1" value="10.0" />
-        <elem key="mu2" value="10.0" />
-        <elem key="kp"  value="10000000.0" />
-        <elem key="kd"  value="1.0" />
-      </map>
     </collision>
   </link>
+  <gazebo reference="torso_lift_link">
+    <material>PR2/White</material>
+    <mu1>10.0</mu1>
+    <mu2>10.0</mu2>
+    <kp>10000000.0</kp>
+    <kd>1.0</kd>
+  </gazebo>
 </robot>

File: pr2_defs/robots/l_gripper.urdf.xacro (robot description, xacro)
@@ -32,14 +32,11 @@
     <inertial>
       <mass value="1000" />
-      <com xyz="0 0 1" />
+      <origin xyz="0 0 1" />
       <inertia ixx="1000"  ixy="0"  ixz="0" iyy="1000" iyz="0" izz="1000" />
     </inertial>
     <visual>
       <origin xyz="0 0 0" rpy="0 0 0 " />
-      <map name="gazebo_material" flag="gazebo">
-        <elem key="material">PR2/White</elem>
-      </map>
       <geometry name="pr2_base_mesh_file">
-        <box scale="0.01 0.01 0.01" />
+        <box size="0.01 0.01 0.01" />
       </geometry>
     </visual>
@@ -47,10 +44,12 @@
       <origin xyz="0 0 0" rpy="0.0 0.0 0.0" />
       <geometry name="base_collision_geom">
-        <box scale="0.01 0.01 0.01" />
+        <box size="0.01 0.01 0.01" />
       </geometry>
     </collision>
   </link>
-  <map name="gazebo_material" flag="gazebo">
-  <verbatim>
+  <gazebo reference="base_link">
+    <material>PR2/White</material>
+  </gazebo>
+  <gazebo>
     <!-- ros_p3d for position groundtruth -->
     <controller:ros_p3d name="p3d_l_gripper_palm_controller" plugin="libros_p3d.so">
@@ -62,5 +61,4 @@
       <interface:position name="p3d_l_gripper_palm_position"/>
     </controller:ros_p3d>
-  </verbatim>
-  </map>
+  </gazebo>
 </robot>

File: pr2_defs/robots/r_arm.urdf.xacro (robot description, xacro)
@@ -37,14 +37,11 @@
     <inertial>
       <mass value="1000" />
-      <com xyz="0 0 0" />
+      <origin xyz="0 0 0" />
       <inertia ixx="1000"  ixy="0"  ixz="0" iyy="1000" iyz="0" izz="1000" />
     </inertial>
     <visual>
       <origin xyz="0 0 0" rpy="0 0 0 " />
-      <map name="gazebo_material" flag="gazebo">
-        <elem key="material">PR2/White</elem>
-      </map>
       <geometry name="pr2_base_mesh_file">
-        <box scale="0.01 0.01 0.01" />
+        <box size="0.01 0.01 0.01" />
       </geometry>
     </visual>
@@ -52,13 +49,14 @@
       <origin xyz="0 0 0" rpy="0.0 0.0 0.0 " />
       <geometry name="base_collision_geom">
-        <box scale="0.01 0.01 0.01" />
+        <box size="0.01 0.01 0.01" />
       </geometry>
-      <map name="base_collision" flag="gazebo">
-        <elem key="mu1" value="10.0" />
-        <elem key="mu2" value="10.0" />
-        <elem key="kp"  value="10000000.0" />
-        <elem key="kd"  value="1.0" />
-      </map>
     </collision>
   </link>
+  <gazebo reference="base_link">
+    <material>PR2/White</material>
+    <mu1>10.0</mu1>
+    <mu2>10.0</mu2>
+    <kp>10000000.0</kp>
+    <kd>1.0</kd>
+  </gazebo>
 </robot>

File: pr2_defs/robots/r_forearm_gripper.urdf.xacro (robot description, xacro)
@@ -29,5 +29,5 @@
   <joint name="base_joint" type="planar">
     <origin xyz="0 0 1.002" rpy=" 0 0 0" />
-    <parent link=" world" />
+    <parent link="world" />
     <!-- rotation of a local coordinate frame attached to the link with respect to a global coordinate frame -->
     <!-- position of a local coordinate frame attached to the link with respect to the parent link's coordinate frame -->
@@ -37,5 +37,5 @@
     <inertial>
       <mass value="1000" />
-      <com xyz=" 0 0 0 " /> <!-- position of the center of mass with respect to the link's own anchor in a local coordinate frame -->
+      <origin xyz=" 0 0 0 " /> <!-- position of the center of mass with respect to the link's own anchor in a local coordinate frame -->
       <inertia ixx="1000"  ixy="0"  ixz="0" iyy="1000" iyz="0" izz="1000" />
     </inertial>
@@ -43,9 +43,6 @@
       <origin xyz="0 0 -1" rpy="0 0 0 " /> <!-- location defined with respect to the link origin in a local coordinate frame -->
       <!-- All angles always in radians, yaw about Z axis, pitch about the Y axis and roll about the X axis -->
-      <map name="gazebo_material" flag="gazebo">
-        <elem key="material">PR2/White</elem>
-      </map>
       <geometry name="pr2_base_mesh_file">
-        <mesh scale="20 20 0.01" />
+        <box size="20 20 0.01" />
       </geometry>
     </visual>
@@ -58,6 +55,8 @@
     </collision>
   </link>
-  <map name="gazebo_material" flag="gazebo">
-  <verbatim>
+  <gazebo reference="base_link">
+    <material>PR2/White</material>
+  </gazebo>
+  <gazebo>
     <!-- ros_p3d for position groundtruth -->
     <controller:ros_p3d name="p3d_r_gripper_palm_controller" plugin="libros_p3d.so">
@@ -69,5 +68,4 @@
       <interface:position name="p3d_r_gripper_palm_position"/>
     </controller:ros_p3d>
-  </verbatim>
-  </map>
+  </gazebo>
 </robot>

File: pr2_defs/robots/r_gripper.urdf.xacro (robot description, xacro)
@@ -25,5 +25,5 @@
   <!-- Solid Base -->
   <joint name="base_joint" type="fixed">
-    <parent link=" world" />
+    <parent link="world" />
     <origin xyz="0 0 0" rpy="0 0 0" />
     <child link="base_link" />
@@ -32,14 +32,11 @@
     <inertial>
       <mass value="1000" />
-      <com xyz="0 0 1" />
+      <origin xyz="0 0 1" />
       <inertia ixx="1000"  ixy="0"  ixz="0" iyy="1000" iyz="0" izz="1000" />
     </inertial>
     <visual>
       <origin xyz="0 0 0" rpy="0 0 0 " />
-      <map name="gazebo_material" flag="gazebo">
-        <elem key="material">PR2/White</elem>
-      </map>
       <geometry name="pr2_base_mesh_file">
-        <box scale="0.01 0.01 0.01" />
+        <box size="0.01 0.01 0.01" />
       </geometry>
     </visual>
@@ -47,10 +44,12 @@
       <origin xyz="0 0 0" rpy="0.0 0.0 0.0" />
       <geometry name="base_collision_geom">
-        <box scale="0.01 0.01 0.01" />
+        <box size="0.01 0.01 0.01" />
       </geometry>
     </collision>
   </link>
-  <map name="gazebo_material" flag="gazebo">
-  <verbatim>
+  <gazebo reference="base_link">
+    <material>PR2/White</material>
+  </gazebo>
+  <gazebo>
     <!-- ros_p3d for position groundtruth -->
     <controller:ros_p3d name="p3d_r_gripper_palm_controller" plugin="libros_p3d.so">
@@ -62,5 +61,4 @@
       <interface:position name="p3d_r_gripper_palm_position"/>
     </controller:ros_p3d>
-  </verbatim>
-  </map>
+  </gazebo>
 </robot>
