Commit message: adding forearm cameras.

File: pr2_defs/robots/pr2.urdf.xacro (robot description, xacro)
@@ -15,4 +15,5 @@
   <include filename="$(find pr2_defs)/defs/head/prosilica_defs.urdf.xacro" />
   <include filename="$(find pr2_defs)/defs/gazebo/gazebo_defs.urdf.xacro" />
+  <include filename="$(find pr2_defs)/defs/arm/mono_cam_defs.urdf.xacro" />
   <include filename="$(find pr2_defs)/defs/materials.urdf.xacro" />
   <!-- Now we can start using the macros included above to define the actual PR2 -->

File: pr2_defs/robots/pre.urdf.xacro (robot description, xacro)
@@ -13,4 +13,5 @@
   <include filename="$(find pr2_defs)/defs/head/prosilica_defs.urdf.xacro" />
   <include filename="$(find pr2_defs)/defs/gazebo/gazebo_defs.urdf.xacro" />
+  <include filename="$(find pr2_defs)/defs/arm/mono_cam_defs.urdf.xacro" />
   <include filename="$(find pr2_defs)/defs/materials.urdf.xacro" />
   <!-- New casters have different encoder ticks, gear ratios -->
@@ -55,4 +56,13 @@
     <origin xyz="0 0 0" rpy="0 0 0" />
   </pr2_gripper>
+  <!-- Forearm Cam (Hand approximated values) -->
+  <mono_cam name="l_forearm_cam" parent="l_forearm_roll_link">
+    <origin xyz=".15 0 .07"
+            rpy="${ M_PI/2} ${-45*M_PI/180} 0" />
+  </mono_cam>
+  <mono_cam name="r_forearm_cam" parent="r_forearm_roll_link">
+    <origin xyz=".15 0 .07"
+            rpy="${-M_PI/2} ${-45*M_PI/180} 0" />
+  </mono_cam>
   <!-- Kinematic chains -->
   <chain root="torso_lift_link" tip="l_wrist_roll_link" />
