Commit message: fix gazebo extensions and fix gripper origin.

File: pr2_defs/defs/arm/arm_gazebo.xacro (robot description, xacro)
@@ -7,5 +7,5 @@
     <gazebo reference="${side}_shoulder_pan_link">
       <sensor:contact name="${side}_shoulder_pan_contact_sensor">
-        <geom>${side}_shoulder_pan_collision</geom>
+        <geom>${side}_shoulder_pan_link_geom</geom>
         <updateRate>100.0</updateRate>
         <controller:ros_bumper name="${side}_shoulder_pan_ros_bumper_controller" plugin="libros_bumper.so">
@@ -18,4 +18,6 @@
       <material value="PR2/Blue" />
       <turnGravityOff>true</turnGravityOff>
+    </gazebo>
+    <gazebo reference="${side}_shoulder_pan_joint">
       <stopKd value="1.0" />
       <stopKp value="1000000.0" />
@@ -24,5 +26,5 @@
     <gazebo reference="${side}_shoulder_lift_link">
       <sensor:contact name="${side}_shoulder_lift_contact_sensor">
-        <geom>${side}_shoulder_lift_collision_geom</geom>
+        <geom>${side}_shoulder_lift_link_geom</geom>
         <updateRate>100.0</updateRate>
         <controller:ros_bumper name="${side}_shoulder_lift_ros_bumper_controller" plugin="libros_bumper.so">
@@ -34,4 +36,6 @@
       </sensor:contact>
       <turnGravityOff>true</turnGravityOff>
+    </gazebo>
+    <gazebo reference="${side}_shoulder_lift_joint">
       <stopKd value="1.0" />
       <stopKp value="1000000.0" />
@@ -42,4 +46,6 @@
       <material value="PR2/RollLinks" />
       <turnGravityOff>true</turnGravityOff>
+    </gazebo>
+    <gazebo reference="${side}_upper_arm_roll_joint">
       <stopKd value="1.0" />
       <stopKp value="1000000.0" />
@@ -51,5 +57,5 @@
     <gazebo reference="${side}_upper_arm_link">
       <sensor:contact name="${side}_upper_arm_contact_sensor">
-        <geom>${side}_upper_arm_collision_geom</geom><!-- TODO -->
+        <geom>${side}_upper_arm_link_geom</geom><!-- TODO -->
         <updateRate>100.0</updateRate>
         <controller:ros_bumper name="${side}_upper_arm_ros_bumper_controller" plugin="libros_bumper.so">
@@ -66,5 +72,5 @@
     <gazebo reference="${side}_elbow_flex_link">
       <sensor:contact name="${side}_elbow_flex_contact_sensor">
-        <geom>${side}_elbow_flex_collision_geom</geom>
+        <geom>${side}_elbow_flex_link_geom</geom>
         <updateRate>100.0</updateRate>
         <controller:ros_bumper name="${side}_elbow_flex_ros_bumper_controller" plugin="libros_bumper.so">
@@ -76,13 +82,17 @@
       </sensor:contact>
       <material value="PR2/Grey" />
+      <turnGravityOff>true</turnGravityOff>
+    </gazebo>
+    <gazebo reference="${side}_elbow_flex_joint">
       <stopKd value="1.0" />
       <stopKp value="1000000.0" />
-      <turnGravityOff>true</turnGravityOff>
     </gazebo>
     <!-- Forearm roll -->
     <gazebo reference="${side}_forearm_roll_link">
       <material value="PR2/RollLinks" />
+      <turnGravityOff>true</turnGravityOff>
+    </gazebo>
+    <gazebo reference="${side}_forearm_roll_joint">
       <fudgeFactor value="0.5" />
-      <turnGravityOff>true</turnGravityOff>
     </gazebo>
   </macro>
@@ -92,5 +102,5 @@
       <turnGravityOff>true</turnGravityOff>
       <sensor:contact name="${side}_forearm_contact_sensor">
-        <geom>${side}_forearm_collision</geom>
+        <geom>${side}_forearm_link_geom</geom>
         <updateRate>100.0</updateRate>
         <controller:ros_bumper name="${side}_forearm_ros_bumper_controller" plugin="libros_bumper.so">
@@ -107,5 +117,5 @@
       <turnGravityOff>true</turnGravityOff>
       <sensor:contact name="${side}_wrist_flex_contact_sensor">
-        <geom>${side}_wrist_flex_collision</geom>
+        <geom>${side}_wrist_flex_link_geom</geom>
         <updateRate>100.0</updateRate>
         <controller:ros_bumper name="${side}_wrist_flex_ros_bumper_controller" plugin="libros_bumper.so">
@@ -117,4 +127,6 @@
       </sensor:contact>
       <material value="PR2/Grey" />
+    </gazebo>
+    <gazebo reference="${side}_wrist_flex_joint">
       <stopKd value="1.0" />
       <stopKp value="1000000.0" />
@@ -124,5 +136,5 @@
       <turnGravityOff>true</turnGravityOff>
       <sensor:contact name="${side}_wrist_roll_contact_sensor">
-        <geom>${side}_wrist_roll_collision</geom>
+        <geom>${side}_wrist_roll_link_geom</geom>
         <updateRate>100.0</updateRate>
         <controller:ros_bumper name="${side}_wrist_roll_ros_bumper_controller" plugin="libros_bumper.so">
@@ -134,4 +146,6 @@
       </sensor:contact>
       <material value="PR2/RollLinks" />
+    </gazebo>
+    <gazebo reference="${side}_wrist_roll_joint">
       <fudgeFactor value="0.5" />
     </gazebo>

File: pr2_defs/defs/base/alpha2_base_gazebo.xacro (robot description, xacro)
@@ -17,5 +17,5 @@
     <gazebo reference="${parent}_${suffix}_wheel_link">
       <sensor:contact name="${parent}_${suffix}_wheel_contact_sensor">
-        <geom>${parent}_${suffix}_wheel_collision</geom>
+        <geom>${parent}_${suffix}_wheel_link_geom</geom>
         <updateRate>100.0</updateRate>
         <controller:ros_bumper name="${parent}_${suffix}_wheel_ros_bumper_controller" plugin="libros_bumper.so">
@@ -35,5 +35,5 @@
     <gazebo reference="${name}_link">
       <sensor:contact name="${name}_contact_sensor">
-        <geom>${name}_collision</geom>
+        <geom>${name}_link_geom</geom>
         <updateRate>100.0</updateRate>
         <controller:ros_bumper name="${name}_ros_bumper_controller" plugin="libros_bumper.so">

File: pr2_defs/defs/base/base_gazebo.xacro (robot description, xacro)
@@ -14,5 +14,5 @@
     <gazebo reference="${parent}_${suffix}_wheel_link">
       <sensor:contact name="${parent}_${suffix}_wheel_contact_sensor">
-        <geom>${parent}_${suffix}_wheel_collision</geom>
+        <geom>${parent}_${suffix}_wheel_link_geom</geom>
         <updateRate>100.0</updateRate>
         <controller:ros_bumper name="${parent}_${suffix}_wheel_ros_bumper_controller" plugin="libros_bumper.so">
@@ -32,5 +32,5 @@
     <gazebo reference="${name}_link">
       <sensor:contact name="${name}_contact_sensor">
-        <geom>${name}_collision</geom>
+        <geom>${name}_link_geom</geom>
         <updateRate>100.0</updateRate>
         <controller:ros_bumper name="${name}_ros_bumper_controller" plugin="libros_bumper.so">

File: pr2_defs/defs/body/body_gazebo.xacro (robot description, xacro)
@@ -6,5 +6,5 @@
     <gazebo reference="${name}_link">
       <sensor:contact name="${name}_contact_sensor">
-        <geom>${name}_collision</geom>
+        <geom>${name}_link_geom</geom>
         <updateRate>100.0</updateRate>
         <controller:ros_bumper name="${name}_ros_bumper_controller" plugin="libros_bumper.so">

File: pr2_defs/defs/gripper/gripper_defs.urdf.xacro (robot description, xacro)
@@ -57,9 +57,8 @@
     <joint name="${prefix}_r_finger_joint" type="revolute">
       <axis xyz="0 0 -1" />
-      <origin xyz="0 0 0" rpy="0 0 0" />
+      <origin xyz="0.07691 -0.01 0" rpy="0 0 0" />
       <pr2_finger_limits reflect="1" />
       <dynamics damping="${finger_damping}" />
       <mimic name="${prefix}_l_finger_joint" mult="1" offset="0"/>
-      <origin xyz="0.07691 -0.01 0" rpy="0 0 0" />
       <parent link="${parent}"/>
       <child link="${prefix}_r_finger_link"/>
@@ -94,9 +93,8 @@
     <joint name="${prefix}_l_finger_tip_joint" type="revolute">
       <axis xyz="0 0 -1" />
-      <origin xyz="0 0 0" rpy="0 0 0" />
+      <origin xyz="0.09137 0.00495 0" rpy="0 0 0" />
       <pr2_finger_limits reflect="1" />
       <dynamics damping="${finger_tip_damping}" />
       <mimic name="${prefix}_l_finger_joint" mult="1" offset="0"/>
-      <origin xyz="0.09137 0.00495 0" rpy="0 0 0" />
       <parent link="${prefix}_l_finger_link"/>
       <child link="${prefix}_l_finger_tip_link"/>
@@ -128,9 +126,8 @@
     <joint name="${prefix}_r_finger_tip_joint" type="revolute">
       <axis xyz="0 0 1" />
-      <origin xyz="0 0 0" rpy="0 0 0" />
+      <origin xyz="${0.09137} ${-0.00495} 0" rpy="0 0 0" />
       <pr2_finger_limits reflect="1" />
       <dynamics damping="${finger_tip_damping}" />
       <mimic name="${prefix}_l_finger_joint" mult="1" offset="0"/>
-      <origin xyz="${0.09137} ${-0.00495} 0" rpy="0 0 0" />
       <parent link="${prefix}_r_finger_link"/>
       <child link="${prefix}_r_finger_tip_link"/>

File: pr2_defs/defs/gripper/gripper_gazebo.xacro (robot description, xacro)
@@ -20,5 +20,5 @@
       <turnGravityOff>true</turnGravityOff>
       <sensor:contact name="${prefix}_l_finger_contact_sensor">
-        <geom>${prefix}_l_finger_collision</geom>
+        <geom>${prefix}_l_finger_link_geom</geom>
         <updateRate>100.0</updateRate>
         <controller:ros_bumper name="${prefix}_l_finger_ros_bumper_controller" plugin="libros_bumper.so">
@@ -35,4 +35,6 @@
       <material value="PR2/Grey" />
       <!-- for "${prefix}_l_finger_joint"-->
+    </gazebo>
+    <gazebo reference="${prefix}_l_finger_joint">
       <stopKd value="${finger_stop_kd}" />
       <stopKp value="${finger_stop_kp}" />
@@ -44,5 +46,5 @@
       <turnGravityOff>true</turnGravityOff>
       <sensor:contact name="${prefix}_r_finger_contact_sensor">
-        <geom>${prefix}_r_finger_collision</geom>
+        <geom>${prefix}_r_finger_link_geom</geom>
         <updateRate>100.0</updateRate>
         <controller:ros_bumper name="${prefix}_r_finger_ros_bumper_controller" plugin="libros_bumper.so">
@@ -58,12 +60,10 @@
       <kd value="1.0" />
       <material value="PR2/Grey" />
-      <stopKd value="${finger_stop_kd}" />
-      <stopKp value="${finger_stop_kp}" />
-      <fudgeFactor value="${finger_fudge_factor}" />
-      <provideFeedback value="true"/>
-      <!-- for "${prefix}_r_finger_joint"-->
-      <mimicKp   value="${finger_kp}" />
-      <mimicKd   value="${finger_kd}" />
-      <mimicFMax value="${finger_fm}" />
+    </gazebo>
+    <gazebo reference="${prefix}_r_finger_joint">
+      <stopKd value="${finger_stop_kd}" />
+      <stopKp value="${finger_stop_kp}" />
+      <fudgeFactor value="${finger_fudge_factor}" />
+      <provideFeedback value="true"/>
     </gazebo>
     <!-- Finger tip -->
@@ -72,5 +72,5 @@
       <selfCollide value="false" />
       <sensor:contact name="${prefix}_l_finger_tip_contact_sensor">
-        <geom>${prefix}_l_finger_tip_collision</geom>
+        <geom>${prefix}_l_finger_tip_link_geom</geom>
         <updateRate>100.0</updateRate>
         <controller:ros_bumper name="${prefix}_l_finger_tip_ros_bumper_controller" plugin="libros_bumper.so">
@@ -86,11 +86,10 @@
       <kd  value="1.0" />
       <material value="PR2/Green" />
-      <stopKd value="${finger_stop_kd}" />
-      <stopKp value="${finger_stop_kp}" />
-      <fudgeFactor value="${finger_fudge_factor}" />
-      <provideFeedback value="true"/>
-      <mimicKp   value="${finger_tip_kp}" />
-      <mimicKd   value="${finger_tip_kd}" />
-      <mimicFMax value="${finger_tip_fm}" />
+    </gazebo>
+    <gazebo reference="${prefix}_l_finger_tip_joint">
+      <stopKd value="${finger_stop_kd}" />
+      <stopKp value="${finger_stop_kp}" />
+      <fudgeFactor value="${finger_fudge_factor}" />
+      <provideFeedback value="true"/>
     </gazebo>
     <!-- Finger tip -->
@@ -99,5 +98,5 @@
       <selfCollide value="false" />
       <sensor:contact name="${prefix}_r_finger_tip_contact_sensor">
-        <geom>${prefix}_r_finger_tip_collision</geom>
+        <geom>${prefix}_r_finger_tip_link_geom</geom>
         <updateRate>100.0</updateRate>
         <controller:ros_bumper name="${prefix}_r_finger_tip_ros_bumper_controller" plugin="libros_bumper.so">
@@ -113,11 +112,4 @@
       <kd  value="1.0" />
       <material value="PR2/Green" />
-      <stopKd value="${finger_stop_kd}" />
-      <stopKp value="${finger_stop_kp}" />
-      <fudgeFactor value="${finger_fudge_factor}" />
-      <mimicKp   value="${finger_tip_kp}" />
-      <mimicKd   value="${finger_tip_kd}" />
-      <mimicFMax value="${finger_tip_fm}" />
-      <provideFeedback value="true"/>
       <controller:ros_p3d name="p3d_${prefix}_l_finger_controller" plugin="libros_p3d.so">
         <alwaysOn>true</alwaysOn>
@@ -138,4 +130,10 @@
       </controller:ros_f3d>
     </gazebo>
+    <gazebo reference="${prefix}_r_finger_tip_joint">
+      <stopKd value="${finger_stop_kd}" />
+      <stopKp value="${finger_stop_kp}" />
+      <fudgeFactor value="${finger_fudge_factor}" />
+      <provideFeedback value="true"/>
+    </gazebo>
   </macro>
   <macro name="pr2_gripper_gazebo" params="side">
@@ -143,5 +141,5 @@
       <turnGravityOff>true</turnGravityOff>
       <sensor:contact name="${side}_gripper_palm_contact_sensor">
-        <geom>${side}_gripper_palm_collision</geom>
+        <geom>${side}_gripper_palm_link_geom</geom>
         <updateRate>100.0</updateRate>
         <controller:ros_bumper name="${side}_gripper_palm_ros_bumper_controller" plugin="libros_bumper.so">

Commit message: unused line in urdf.

File: pr2_defs/defs/arm/arm_gazebo.xacro (robot description, xacro)
@@ -43,5 +43,4 @@
     <!-- Upperarm roll: internal fixed attchment point for upper arm -->
     <gazebo reference="${side}_upper_arm_roll_link">
-      <mesh value="$(find pr2_ogre)/Media/models/upper_arm_roll.mesh" />
       <material value="PR2/RollLinks" />
       <turnGravityOff>true</turnGravityOff>
