Commit message: adding forearm cameras to pr2 robot as well.

File: pr2_defs/defs/arm/mono_cam_gazebo.xacro (robot description, xacro)
@@ -23,4 +23,7 @@
       <material>PR2/Blue</material>
     </gazebo>
+    <gazebo reference="${name}_optical_frame">
+      <turnGravityOff>true</turnGravityOff>
+    </gazebo>
   </macro>
 </robot>

File: pr2_defs/robots/pr2.urdf.xacro (robot description, xacro)
@@ -47,4 +47,13 @@
     <origin xyz="0 0 0" rpy="0 0 0" />
   </pr2_gripper>
+  <!-- Forearm Cam (Hand approximated values) -->
+  <mono_cam name="l_forearm_cam" parent="l_forearm_roll_link">
+    <origin xyz=".15 0 .07"
+            rpy="${ M_PI/2} ${-45*M_PI/180} 0" />
+  </mono_cam>
+  <mono_cam name="r_forearm_cam" parent="r_forearm_roll_link">
+    <origin xyz=".15 0 .07"
+            rpy="${-M_PI/2} ${-45*M_PI/180} 0" />
+  </mono_cam>
   <!-- Kinematic chains -->
   <chain root="torso_lift_link" tip="l_wrist_roll_link" />
