Commit message: fix urdf style for safety_controller

File: pr2_defs/defs/arm/arm_defs.urdf.xacro (robot description, xacro)
@@ -305,5 +305,6 @@
     <joint name="${side}_wrist_roll_joint" type="continuous">
       <axis xyz="1 0 0" />
-      <limit effort="10" velocity="${VELOCITY_LIMIT_SCALE*6}" k_velocity="2" />
+      <limit effort="10" velocity="${VELOCITY_LIMIT_SCALE*6}" />
+      <safety_controller k_velocity="2" />
       <dynamics damping="0.1" />
       <calibration reference_position="${1.27+cal_r_wrist_roll_flag}" values="1.5 -1" />

Commit message: flip forearm_roll and wrist_flex per ticket #3123

File: pr2_defs/defs/arm/arm_defs.urdf.xacro (robot description, xacro)
@@ -212,5 +212,5 @@
     <!-- Forearm roll -->
     <joint name="${side}_forearm_roll_joint" type="continuous">
-      <axis xyz="-1 0 0" />
+      <axis xyz="1 0 0" />
       <limit effort="30" velocity="${VELOCITY_LIMIT_SCALE*6}" />
       <safety_controller k_velocity="1" />
@@ -276,5 +276,5 @@
     <!-- Wrist flex -->
     <joint name="${side}_wrist_flex_joint" type="revolute">
-      <axis xyz="0 -1 0" />
+      <axis xyz="0 1 0" />
       <limit lower="-0.1" upper="2.2" effort="200" velocity="${VELOCITY_LIMIT_SCALE*5.13}" />
       <safety_controller k_position="20" k_velocity="4" soft_lower_limit="${-0.1+0.2}" soft_upper_limit="${2.2-0.2}" />

Commit message: Adding more config params to wrist transmission: Trac #3204. Finalizing swapping of forearm roll and wrist flex: Trac #3123

File: pr2_defs/defs/arm/arm_defs.urdf.xacro (robot description, xacro)
@@ -277,8 +277,8 @@
     <joint name="${side}_wrist_flex_joint" type="revolute">
       <axis xyz="0 1 0" />
-      <limit lower="-0.1" upper="2.2" effort="200" velocity="${VELOCITY_LIMIT_SCALE*5.13}" />
-      <safety_controller k_position="20" k_velocity="4" soft_lower_limit="${-0.1+0.2}" soft_upper_limit="${2.2-0.2}" />
+      <limit lower="-2.2" upper="0.1" effort="200" velocity="${VELOCITY_LIMIT_SCALE*5.13}" />
+      <safety_controller k_position="20" k_velocity="4" soft_lower_limit="${-2.2+0.2}" soft_upper_limit="${0.1-0.2}" />
       <dynamics damping="0.1" />
-      <calibration reference_position="${0.4363+cal_r_wrist_flex_flag}" />
+      <calibration reference_position="${-0.4363-cal_r_wrist_flex_flag}" />
       <origin xyz="0.32025 0 0" rpy="0 0 0" />
       <parent link="${side}_forearm_link"/>

File: pr2_defs/defs/arm/arm_transmission.xacro (robot description, xacro)
@@ -35,5 +35,5 @@
       <actuator name="${side}_forearm_roll_motor" />
       <joint name="${side}_forearm_roll_joint" />
-      <mechanicalReduction>${576/25*55/14}</mechanicalReduction>
+      <mechanicalReduction>-${576/25*55/14}</mechanicalReduction>
     </transmission>
   </macro>
@@ -42,8 +42,8 @@
     <!-- Wrist flex , Wrist roll -->
     <transmission type="WristTransmission" name="${side}_wrist_trans">
-      <rightActuator name="${side}_wrist_r_motor" />
-      <leftActuator name="${side}_wrist_l_motor" />
-      <flexJoint name="${side}_wrist_flex_joint" mechanicalReduction="${624/35*54/16}" />
-      <rollJoint name="${side}_wrist_roll_joint" mechanicalReduction="${624/35*54/16}"  />
+      <rightActuator name="${side}_wrist_r_motor" mechanicalReduction="${624/35*54/16}" />
+      <leftActuator name="${side}_wrist_l_motor"  mechanicalReduction="${624/35*54/16}" />
+      <flexJoint name="${side}_wrist_flex_joint"  mechanicalReduction="-1.0" />
+      <rollJoint name="${side}_wrist_roll_joint"  mechanicalReduction="1.0" />
     </transmission>
   </macro>

File: pr2_defs/robots/prf.urdf.xacro (robot description, xacro)
@@ -2,5 +2,5 @@
 <robot name="pr2">
   <!-- Include file with calibration parameters -->
-  <include filename="$(find pr2_defs)/calibration/prf_cal.xml" />
+  <include filename="$(find pr2_defs)/calibration/prf_cal_zeroed.xml" />
   <!-- declare the path where all models/textures/materials are stored -->
   <resource type="stl_meshes" location="$(find pr2_defs)/meshes"/>

File: pr2_description/urdf/forearm_v0/forearm.transmission.xacro (robot description, xacro)
@@ -7,8 +7,8 @@
     <!-- Wrist flex , Wrist roll -->
     <transmission type="WristTransmission" name="${side}_wrist_trans">
-      <rightActuator name="${side}_wrist_r_motor" />
-      <leftActuator name="${side}_wrist_l_motor" />
-      <flexJoint name="${side}_wrist_flex_joint" mechanicalReduction="${624/35*54/16}" />
-      <rollJoint name="${side}_wrist_roll_joint" mechanicalReduction="${624/35*54/16}"  />
+      <rightActuator name="${side}_wrist_r_motor" mechanicalReduction="${624/35*54/16}"/>
+      <leftActuator name="${side}_wrist_l_motor"  mechanicalReduction="${624/35*54/16}"/>
+      <flexJoint name="${side}_wrist_flex_joint"  mechanicalReduction="1.0" />
+      <rollJoint name="${side}_wrist_roll_joint"  mechanicalReduction="1.0" />
     </transmission>
   </xacro:macro>
