Commit message: fix stereo fhov for narrow stereo in sim

File: pr2_defs/defs/head/head_sensor_package_defs.urdf.xacro (robot description, xacro)
@@ -166,4 +166,7 @@
     <!-- extensions -->
     <double_stereo_camera_gazebo name="${name}" />
+    <!-- extensions -->
+    <stereo_camera_gazebo_wide name="wide_stereo" />
+    <stereo_camera_gazebo_narrow name="narrow_stereo" />
   </macro>
   <macro name="stereo_camera" params="name parent *origin">
@@ -275,6 +278,4 @@
       </collision>
     </link>
-    <!-- extensions -->
-    <stereo_camera_gazebo name="${name}" />
   </macro>
 </robot>

File: pr2_defs/defs/head/head_sensor_package_gazebo.xacro (robot description, xacro)
@@ -114,3 +114,135 @@
     </gazebo>
   </macro>
+  <macro name="stereo_camera_gazebo_wide" params="name">
+    <gazebo reference="${name}_link">
+      <material value="PR2/Blue" />
+    </gazebo>
+    <gazebo reference="${name}_optical_frame">
+      <material value="PR2/Blue" />
+    </gazebo>
+    <gazebo reference="${name}_l_stereo_camera_frame">
+      <sensor:camera name="${name}_l_sensor">
+        <imageSize>640 480</imageSize>
+        <imageFormat>L8</imageFormat>
+        <hfov>90</hfov>
+        <nearClip>0.1</nearClip>
+        <farClip>100</farClip>
+        <updateRate>20.0</updateRate>
+        <controller:ros_camera name="${name}_l_controller" plugin="libros_camera.so">
+          <alwaysOn>true</alwaysOn>
+          <updateRate>20.0</updateRate>
+          <topicName>${name}/left_image</topicName>
+          <frameName>${name}_l_stereo_camera_frame</frameName>
+          <interface:camera name="${name}_l_iface" />
+        </controller:ros_camera>
+      </sensor:camera>
+      <material value="PR2/Blue" />
+    </gazebo>
+    <gazebo reference="${name}_r_stereo_camera_frame">
+      <sensor:camera name="${name}_r_sensor">
+        <imageSize>640 480</imageSize>
+        <imageFormat>L8</imageFormat>
+        <hfov>90</hfov>
+        <nearClip>0.1</nearClip>
+        <farClip>100</farClip>
+        <updateRate>20.0</updateRate>
+        <controller:ros_camera name="${name}_r_controller" plugin="libros_camera.so">
+          <alwaysOn>true</alwaysOn>
+          <updateRate>20.0</updateRate>
+          <topicName>${name}/right_image</topicName>
+          <frameName>${name}_r_stereo_camera_frame</frameName>
+          <interface:camera name="${name}_r_iface" />
+        </controller:ros_camera>
+      </sensor:camera>
+      <material value="PR2/Blue" />
+    </gazebo>
+    <!-- stereo plugin that produces a raw_stereo message -->
+    <gazebo> <!-- this is not attached to any link!!!, there no reference -->
+      <controller:ros_stereo_camera name="${name}_controller" plugin="libros_stereo_camera.so">
+        <alwaysOn>true</alwaysOn>
+        <updateRate>20.0</updateRate>
+        <leftCamera>${name}_l_sensor</leftCamera>
+        <rightCamera>${name}_r_sensor</rightCamera>
+        <topicName>${name}/raw_stereo</topicName>
+        <frameName>${name}_optical_frame</frameName>
+        <CxPrime>320</CxPrime>
+        <Cx>320</Cx>
+        <Cy>240</Cy>
+        <focal_length>320</focal_length> <!-- image_width / (2*tan(hfov_radian /2)) -->
+        <distortion_k1>0</distortion_k1>
+        <distortion_k2>0</distortion_k2>
+        <distortion_k3>0</distortion_k3>
+        <distortion_t1>0</distortion_t1>
+        <distortion_t2>0</distortion_t2>
+        <baseline>${stereo_dy}</baseline> <!-- home pos. of robot has +x forward, +y left -->
+        <interface:stereocamera name="${name}_iface" />
+      </controller:ros_stereo_camera>
+    </gazebo>
+  </macro>
+  <macro name="stereo_camera_gazebo_narrow" params="name">
+    <gazebo reference="${name}_link">
+      <material value="PR2/Blue" />
+    </gazebo>
+    <gazebo reference="${name}_optical_frame">
+      <material value="PR2/Blue" />
+    </gazebo>
+    <gazebo reference="${name}_l_stereo_camera_frame">
+      <sensor:camera name="${name}_l_sensor">
+        <imageSize>640 480</imageSize>
+        <imageFormat>L8</imageFormat>
+        <hfov>45</hfov>
+        <nearClip>0.1</nearClip>
+        <farClip>100</farClip>
+        <updateRate>20.0</updateRate>
+        <controller:ros_camera name="${name}_l_controller" plugin="libros_camera.so">
+          <alwaysOn>true</alwaysOn>
+          <updateRate>20.0</updateRate>
+          <topicName>${name}/left_image</topicName>
+          <frameName>${name}_l_stereo_camera_frame</frameName>
+          <interface:camera name="${name}_l_iface" />
+        </controller:ros_camera>
+      </sensor:camera>
+      <material value="PR2/Blue" />
+    </gazebo>
+    <gazebo reference="${name}_r_stereo_camera_frame">
+      <sensor:camera name="${name}_r_sensor">
+        <imageSize>640 480</imageSize>
+        <imageFormat>L8</imageFormat>
+        <hfov>90</hfov>
+        <nearClip>0.1</nearClip>
+        <farClip>100</farClip>
+        <updateRate>20.0</updateRate>
+        <controller:ros_camera name="${name}_r_controller" plugin="libros_camera.so">
+          <alwaysOn>true</alwaysOn>
+          <updateRate>20.0</updateRate>
+          <topicName>${name}/right_image</topicName>
+          <frameName>${name}_r_stereo_camera_frame</frameName>
+          <interface:camera name="${name}_r_iface" />
+        </controller:ros_camera>
+      </sensor:camera>
+      <material value="PR2/Blue" />
+    </gazebo>
+    <!-- stereo plugin that produces a raw_stereo message -->
+    <gazebo> <!-- this is not attached to any link!!!, there no reference -->
+      <controller:ros_stereo_camera name="${name}_controller" plugin="libros_stereo_camera.so">
+        <alwaysOn>true</alwaysOn>
+        <updateRate>20.0</updateRate>
+        <leftCamera>${name}_l_sensor</leftCamera>
+        <rightCamera>${name}_r_sensor</rightCamera>
+        <topicName>${name}/raw_stereo</topicName>
+        <frameName>${name}_optical_frame</frameName>
+        <CxPrime>320</CxPrime>
+        <Cx>320</Cx>
+        <Cy>240</Cy>
+        <focal_length>320</focal_length> <!-- image_width / (2*tan(hfov_radian /2)) -->
+        <distortion_k1>0</distortion_k1>
+        <distortion_k2>0</distortion_k2>
+        <distortion_k3>0</distortion_k3>
+        <distortion_t1>0</distortion_t1>
+        <distortion_t2>0</distortion_t2>
+        <baseline>${stereo_dy}</baseline> <!-- home pos. of robot has +x forward, +y left -->
+        <interface:stereocamera name="${name}_iface" />
+      </controller:ros_stereo_camera>
+    </gazebo>
+  </macro>
 </robot>
