Commit message: * alpha2_head_defs.urdf.xacro and head_defs.urdf.xacro shares the same head_sensor_package_defs.urdf.xacro.  * removed alpha2_head_sensor_package

File: pr2_defs/defs/head/alpha2_head_defs.urdf.xacro (robot description, xacro)
@@ -3,5 +3,5 @@
        xmlns:controller="http://playerstage.sourceforge.net/gazebo/xmlschema/#controller"
        xmlns:interface="http://playerstage.sourceforge.net/gazebo/xmlschema/#interface">
-  <include filename="$(find pr2_defs)/defs/head/alpha2_head_sensor_package_defs.urdf.xacro" />
+  <include filename="$(find pr2_defs)/defs/head/head_sensor_package_defs.urdf.xacro" />
   <include filename="$(find pr2_defs)/defs/head/alpha2_head_gazebo.xacro" />
   <include filename="$(find pr2_defs)/defs/head/alpha2_head_transmission.xacro" />

File: pr2_defs/defs/head/head_sensor_package_defs.urdf.xacro (robot description, xacro)
@@ -19,5 +19,5 @@
     <joint name="${name}_mount_joint" type="revolute">
       <axis xyz="0 1 0" />
-      <limit lower="-0.785" upper="1.57" effort="0.5292" velocity="100" />
+      <limit lower="-0.785" upper="1.57" effort="0.5292" velocity="10.0" />
       <safety_controller k_position="100" k_velocity="0.05" soft_lower_limit="${-0.785+0.0}" soft_upper_limit="${1.57-0.0}" />
       <calibration reference_position="-0.35" />

File: pr2_defs/robots/hca.urdf.xacro (robot description, xacro)
@@ -44,9 +44,9 @@
             rpy="${cal_head_roll} ${cal_head_pitch} ${cal_head_yaw}" />
   </pr2_head_alpha2b>
-  <pr2_tilting_laser_alpha2 name="laser_tilt" parent="base_link">
+  <pr2_tilting_laser name="laser_tilt" parent="base_link">
     <!-- Was 0.11m forward of head pan, now 125 mm on head carts -->
     <!-- 66.5mm above head tilt plate -->
     <origin xyz="${0.125 + 0.13} 0 ${0.0665 + .53}" rpy="0 0 0" />
-  </pr2_tilting_laser_alpha2>
+  </pr2_tilting_laser>
   <!-- Camera package: double stereo, prosilica -->
   <pr2_head_sensor_package name="sensor_mount" hd_name="high_def"

File: pr2_defs/robots/hcc.urdf.xacro (robot description, xacro)
@@ -46,9 +46,9 @@
             rpy="${cal_head_roll} ${cal_head_pitch} ${cal_head_yaw}" />
   </pr2_head>
-  <pr2_tilting_laser_alpha2 name="laser_tilt" parent="base_link">
+  <pr2_tilting_laser name="laser_tilt" parent="base_link">
     <!-- Was 0.11m forward of head pan, now 115 mm on HCC -->
     <!-- 66.5mm above head tilt plate -->
     <origin xyz="${0.115 + 0.13} 0 ${0.0665 + .53}" rpy="0 0 0" />
-  </pr2_tilting_laser_alpha2>
+  </pr2_tilting_laser>
   <!-- Camera package: double stereo, prosilica -->
   <pr2_head_sensor_package name="sensor_mount" hd_name="high_def"

File: pr2_defs/robots/pre.urdf.xacro (robot description, xacro)
@@ -33,8 +33,8 @@
   </pr2_head_alpha2>
   <!-- Alpha 2.0 laser tilt installed 4/3/09 -->
-  <pr2_tilting_laser_alpha2 name="laser_tilt" parent="torso_lift_link">
+  <pr2_tilting_laser name="laser_tilt" parent="torso_lift_link">
     <!--origin xyz="0.1 0 0.19525" rpy="0 0 0" /-->
     <origin xyz="0.1 0 0.235" rpy="0 0 0" />
-  </pr2_tilting_laser_alpha2>
+  </pr2_tilting_laser>
   <!-- Camera package: double stereo, prosilica -->
   <pr2_head_sensor_package name="sensor_mount" hd_name="high_def"
