Commit message: remove unused visual, collision and geometry names in urdf for prosilica.

File: pr2_defs/defs/head/prosilica_defs.urdf.xacro (robot description, xacro)
@@ -18,14 +18,14 @@
                  izz="0.001" />
       </inertial>
-      <visual name="${name}_visual">
+      <visual>
         <origin xyz="0 0 0" rpy="0 0 0" />
-        <geometry name="${name}_visual_geom">
+        <geometry>
           <box size="0.01 0.01 0.01" />
         </geometry>
         <material name="Blue" />
       </visual>
-      <collision name="${name}_collision">
+      <collision>
         <origin xyz="0 0 0" rpy="0 0 0"/>
-        <geometry name="${name}_collision_geom">
+        <geometry>
           <box size="0.01 0.01 0.01" />
         </geometry>
@@ -46,14 +46,14 @@
                  izz="0.001" />
       </inertial>
-      <visual name="${name}_optical_visual">
+      <visual>
         <origin xyz="0 0 0" rpy="0 0 0"/>
-        <geometry name="${name}_optical_visual_geom">
+        <geometry>
           <box size="0.01 0.01 0.01" />
         </geometry>
         <material name="Blue" />
       </visual>
-      <collision name="${name}_optical_collision">
+      <collision>
         <origin xyz="0 0 0" rpy="0 0 0"/>
-        <geometry name="${name}_optical_collision_geom">
+        <geometry>
           <box size="0.01 0.01 0.01" />
         </geometry>
