Commit message: update wheel texture in sim.

File: pr2_defs/defs/base/base_gazebo.xacro (robot description, xacro)
@@ -23,4 +23,5 @@
         </controller:ros_bumper>
       </sensor:contact>
+      <material value="PR2/wheel_${suffix}" />
       <mu1 value="100.0" />
       <mu2 value="100.0" />

Commit message: * <geometry> has no name  * set canonicalBody for gazebo when base_link is present

File: pr2_defs/defs/base/base_gazebo.xacro (robot description, xacro)
@@ -49,4 +49,5 @@
     </gazebo>
     <gazebo>
+      <canonicalBody>${name}_link</canonicalBody>
       <controller:ros_p3d name="p3d_base_controller" plugin="libros_p3d.so">
         <alwaysOn>true</alwaysOn>

File: pr2_defs/robots/hca.urdf.xacro (robot description, xacro)
@@ -25,5 +25,5 @@
       <!-- 1.06m above ground -->
       <origin xyz="0 0 0" rpy="0 0 0 " />
-      <geometry name="unit_box">
+      <geometry>
 	<box size=".6 0.45 1.06" />
       </geometry>
@@ -31,5 +31,5 @@
     <collision>
       <origin xyz="0 0 0" rpy="0.0 0.0 0.0 " />
-      <geometry name="box_link_collision_geom">
+      <geometry>
         <box size="0.6 0.45 1.06" />
       </geometry>

File: pr2_defs/robots/hcb.urdf.xacro (robot description, xacro)
@@ -25,5 +25,5 @@
       <!-- 1.06m above ground -->
       <origin xyz="0 0 0" rpy="0 0 0 " />
-      <geometry name="unit_box">
+      <geometry>
 	<box size=".6 0.45 1.06" />
       </geometry>
@@ -31,5 +31,5 @@
     <collision>
       <origin xyz="0 0 0" rpy="0.0 0.0 0.0 " />
-      <geometry name="box_link_collision_geom">
+      <geometry>
         <box size="0.6 0.45 1.06" />
       </geometry>

File: pr2_defs/robots/hcc.urdf.xacro (robot description, xacro)
@@ -26,5 +26,5 @@
       <!-- 1.06m above ground -->
       <origin xyz="0 0 0" rpy="0 0 0 " />
-      <geometry name="unit_box">
+      <geometry>
 	<box size=".6 0.45 1.06" />
       </geometry>
@@ -32,5 +32,5 @@
     <collision>
       <origin xyz="0 0 0" rpy="0.0 0.0 0.0 " />
-      <geometry name="box_link_collision_geom">
+      <geometry>
         <box size="0.6 0.45 1.06" />
       </geometry>

File: pr2_defs/robots/l_arm.urdf.xacro (robot description, xacro)
@@ -42,5 +42,5 @@
     <visual>
       <origin xyz="0 0 0" rpy="0 0 0 " />
-      <geometry name="pr2_base_mesh_file">
+      <geometry>
         <box size="0.01 0.01 0.01" />
       </geometry>
@@ -48,5 +48,5 @@
     <collision>
       <origin xyz="0 0 0" rpy="0.0 0.0 0.0 " />
-      <geometry name="base_collision_geom">
+      <geometry>
         <box size="0.01 0.01 0.01" />
       </geometry>

File: pr2_defs/robots/l_gripper.urdf.xacro (robot description, xacro)
@@ -37,5 +37,5 @@
     <visual>
       <origin xyz="0 0 0" rpy="0 0 0 " />
-      <geometry name="pr2_base_mesh_file">
+      <geometry>
         <box size="0.01 0.01 0.01" />
       </geometry>
@@ -43,5 +43,5 @@
     <collision>
       <origin xyz="0 0 0" rpy="0.0 0.0 0.0" />
-      <geometry name="base_collision_geom">
+      <geometry>
         <box size="0.01 0.01 0.01" />
       </geometry>

File: pr2_defs/robots/r_arm.urdf.xacro (robot description, xacro)
@@ -42,5 +42,5 @@
     <visual>
       <origin xyz="0 0 0" rpy="0 0 0 " />
-      <geometry name="pr2_base_mesh_file">
+      <geometry>
         <box size="0.01 0.01 0.01" />
       </geometry>
@@ -48,10 +48,10 @@
     <collision>
       <origin xyz="0 0 0" rpy="0.0 0.0 0.0 " />
-      <geometry name="base_collision_geom">
+      <geometry>
         <box size="0.01 0.01 0.01" />
       </geometry>
     </collision>
   </link>
-  <gazebo reference="base_link">
+  <gazebo reference="torso_lift_link">
     <material>PR2/White</material>
     <mu1>10.0</mu1>

File: pr2_defs/robots/r_forearm_gripper.urdf.xacro (robot description, xacro)
@@ -43,5 +43,5 @@
       <origin xyz="0 0 -1" rpy="0 0 0 " /> <!-- location defined with respect to the link origin in a local coordinate frame -->
       <!-- All angles always in radians, yaw about Z axis, pitch about the Y axis and roll about the X axis -->
-      <geometry name="pr2_base_mesh_file">
+      <geometry>
         <box size="20 20 0.01" />
       </geometry>
@@ -50,5 +50,5 @@
       <origin xyz="0 0 -1" rpy="0.0 0.0 0.0 " /> <!-- default box is centered at the origin -->
       <!-- All angles always in radians, yaw about Z axis, pitch about the Y axis and roll about the X axis -->
-      <geometry name="base_collision_geom"> <!-- think about putting mesh here as well -->
+      <geometry>
         <box size="20 20 0.01" />
       </geometry>

File: pr2_defs/robots/r_gripper.urdf.xacro (robot description, xacro)
@@ -37,5 +37,5 @@
     <visual>
       <origin xyz="0 0 0" rpy="0 0 0 " />
-      <geometry name="pr2_base_mesh_file">
+      <geometry>
         <box size="0.01 0.01 0.01" />
       </geometry>
@@ -43,5 +43,5 @@
     <collision>
       <origin xyz="0 0 0" rpy="0.0 0.0 0.0" />
-      <geometry name="base_collision_geom">
+      <geometry>
         <box size="0.01 0.01 0.01" />
       </geometry>
