Commit message: minor urdf cleanup

File: pr2_defs/defs/base/base_defs.urdf.xacro (robot description, xacro)
@@ -133,5 +133,4 @@
     <!-- base laser -->
     <joint name="base_laser_joint" type="fixed">
-      <axis xyz="0 1 0" />
       <origin xyz="${base_laser_x} ${base_laser_y} ${base_height_offset+base_laser_z}" rpy="0 0 0" />
       <parent link="${name}_link"/>
@@ -160,6 +159,4 @@
     <!-- modeling plug on base holder magnet location -->
     <joint name="plug_magnet_joint" type="fixed">
-      <axis xyz="0 1 0" />
-      <anchor xyz="0 0 0" />
       <origin xyz="0.18 0 ${base_height_offset+0.235}" rpy="0 0 0" />
       <parent link="${name}_link"/>

Commit message: update base hokuyo collision, update mimics in gripper.

File: pr2_defs/defs/base/base_defs.urdf.xacro (robot description, xacro)
@@ -24,8 +24,8 @@
   <property name="base_laser_y" value="0.0" />
   <property name="base_laser_z" value="0.252" />
-  <property name="base_laser_size_x" value="0.08" />
-  <property name="base_laser_size_y" value="0.08" />
+  <property name="base_laser_size_x" value="0.06" />
+  <property name="base_laser_size_y" value="0.06" />
   <property name="base_laser_size_z" value="0.03" />
-  <property name="base_laser_collision_offset_z" value="0.03" />
+  <property name="base_laser_collision_offset_z" value="0.02" />
   <macro name="pr2_wheel" params="suffix parent reflect">
     <joint name="${parent}_${suffix}_wheel_joint" type="continuous">

File: pr2_defs/defs/gripper/gripper_defs.urdf.xacro (robot description, xacro)
@@ -60,5 +60,5 @@
       <pr2_finger_limits reflect="1" />
       <dynamics damping="${finger_damping}" />
-      <mimic name="${prefix}_l_finger_joint" mult="1" offset="0"/>
+      <mimic joint="${prefix}_l_finger_joint" multiplier="1" offset="0"/>
       <parent link="${parent}"/>
       <child link="${prefix}_r_finger_link"/>
@@ -96,5 +96,5 @@
       <pr2_finger_limits reflect="1" />
       <dynamics damping="${finger_tip_damping}" />
-      <mimic name="${prefix}_l_finger_joint" mult="1" offset="0"/>
+      <mimic joint="${prefix}_l_finger_joint" multiplier="1" offset="0"/>
       <parent link="${prefix}_l_finger_link"/>
       <child link="${prefix}_l_finger_tip_link"/>
@@ -129,5 +129,5 @@
       <pr2_finger_limits reflect="1" />
       <dynamics damping="${finger_tip_damping}" />
-      <mimic name="${prefix}_l_finger_joint" mult="1" offset="0"/>
+      <mimic joint="${prefix}_l_finger_joint" multiplier="1" offset="0"/>
       <parent link="${prefix}_r_finger_link"/>
       <child link="${prefix}_r_finger_tip_link"/>

Commit message: update plug demo in sim.

File: pr2_defs/defs/base/base_defs.urdf.xacro (robot description, xacro)
@@ -157,29 +157,4 @@
       </collision>
     </link>
-    <!-- modeling plug on base holder magnet location -->
-    <joint name="plug_magnet_joint" type="fixed">
-      <origin xyz="0.18 0 ${base_height_offset+0.235}" rpy="0 0 0" />
-      <parent link="${name}_link"/>
-      <child link="plug_magnet"/>
-    </joint>
-    <link name="plug_magnet" type="laser">
-      <inertial>
-        <mass value="0.1" />
-        <origin xyz="0 0 0.0" />
-        <inertia ixx="0.1" ixy="0" ixz="0" iyy="0.1" iyz="0" izz="0.1" />
-      </inertial>
-      <visual name="plug_mavisual">
-        <origin xyz="0 0 0" rpy="0 0 0" />
-        <geometry name="plug_magnet_visual_geom">
-          <box size="0.001 0.001 0.001"/>
-        </geometry>
-      </visual>
-      <collision name="plug_macollision">
-        <origin xyz="0 0 0.0" rpy="0 0 0" />
-        <geometry name="plug_magnet_collision_geom">
-          <box size=".001 .001 .001" />
-        </geometry>
-      </collision>
-    </link>
     <pr2_caster suffix="fl" parent="${name}_link">
       <origin xyz="${caster_offset_x} ${caster_offset_y} ${caster_offset_z}" rpy="0 0 0" />
@@ -196,4 +171,104 @@
     <!-- gazebo extensions -->
     <pr2_base_gazebo name="${name}" />
+    <!-- modeling plug on base holder magnet location -->
+    <pr2_plug_holder name="${name}"/>
+  </macro>
+  <macro name="pr2_plug_holder" params="name">
+    <joint name="plug_holder_1_joint" type="fixed">
+      <origin xyz="0.18 0 ${base_height_offset+0.235}" rpy="0 0 0" />
+      <parent link="${name}_link"/>
+      <child link="plug_holder_1"/>
+    </joint>
+    <link name="plug_holder_1">
+      <inertial>
+        <mass value="0.1" />
+        <origin xyz="0 0 0.0" />
+        <inertia ixx="0.1" ixy="0" ixz="0" iyy="0.1" iyz="0" izz="0.1" />
+      </inertial>
+      <visual>
+        <origin xyz="0 0 0" rpy="0 0 0" />
+        <geometry>
+          <box size="0.001 0.001 0.001"/>
+        </geometry>
+      </visual>
+      <collision>
+        <origin xyz="0 0 0.0" rpy="0 0 0" />
+        <geometry>
+          <box size=".001 .001 .001" />
+        </geometry>
+      </collision>
+    </link>
+    <joint name="plug_holder_2_joint" type="fixed">
+      <origin xyz="0.21 0 ${base_height_offset+0.235}" rpy="0 0 0" />
+      <parent link="${name}_link"/>
+      <child link="plug_holder_2"/>
+    </joint>
+    <link name="plug_holder_2">
+      <inertial>
+        <mass value="0.1" />
+        <origin xyz="0 0 0.0" />
+        <inertia ixx="0.1" ixy="0" ixz="0" iyy="0.1" iyz="0" izz="0.1" />
+      </inertial>
+      <visual>
+        <origin xyz="0 0 0" rpy="0 0 0" />
+        <geometry>
+          <box size="0.001 0.001 0.001"/>
+        </geometry>
+      </visual>
+      <collision>
+        <origin xyz="0 0 0.0" rpy="0 0 0" />
+        <geometry>
+          <box size=".001 .001 .001" />
+        </geometry>
+      </collision>
+    </link>
+    <joint name="plug_holder_3_joint" type="fixed">
+      <origin xyz="0.20 -.04 ${base_height_offset+0.235}" rpy="0 0 0" />
+      <parent link="${name}_link"/>
+      <child link="plug_holder_3"/>
+    </joint>
+    <link name="plug_holder_3">
+      <inertial>
+        <mass value="0.1" />
+        <origin xyz="0 0 0.0" />
+        <inertia ixx="0.1" ixy="0" ixz="0" iyy="0.1" iyz="0" izz="0.1" />
+      </inertial>
+      <visual>
+        <origin xyz="0 0 0" rpy="0 0 0" />
+        <geometry>
+          <box size="0.001 0.001 0.001"/>
+        </geometry>
+      </visual>
+      <collision>
+        <origin xyz="0 0 0.0" rpy="0 0 0" />
+        <geometry>
+          <box size=".001 .001 .001" />
+        </geometry>
+      </collision>
+    </link>
+    <joint name="plug_holder_4_joint" type="fixed">
+      <origin xyz="0.20 0.04 ${base_height_offset+0.235}" rpy="0 0 0" />
+      <parent link="${name}_link"/>
+      <child link="plug_holder_4"/>
+    </joint>
+    <link name="plug_holder_4">
+      <inertial>
+        <mass value="0.1" />
+        <origin xyz="0 0 0.0" />
+        <inertia ixx="0.1" ixy="0" ixz="0" iyy="0.1" iyz="0" izz="0.1" />
+      </inertial>
+      <visual>
+        <origin xyz="0 0 0" rpy="0 0 0" />
+        <geometry>
+          <box size="0.001 0.001 0.001"/>
+        </geometry>
+      </visual>
+      <collision>
+        <origin xyz="0 0 0.0" rpy="0 0 0" />
+        <geometry>
+          <box size=".001 .001 .001" />
+        </geometry>
+      </collision>
+    </link>
   </macro>
 </robot>

File: pr2_defs/defs/base/base_gazebo.xacro (robot description, xacro)
@@ -60,14 +60,14 @@
         <interface:position name="p3d_base_position"/>
       </controller:ros_p3d>
-      <controller:ros_p3d name="p3d_plug_magnet_controller" plugin="libros_p3d.so">
+      <controller:ros_p3d name="p3d_plug_holder_1_controller" plugin="libros_p3d.so">
         <alwaysOn>true</alwaysOn>
         <updateRate>100.0</updateRate>
-        <bodyName>plug_magnet</bodyName>
-        <topicName>plug_magnet_pose_ground_truth</topicName>
+        <bodyName>plug_holder_1</bodyName>
+        <topicName>plug_holder_1_pose_ground_truth</topicName>
         <gaussianNoise>0.01</gaussianNoise>
         <frameName>map</frameName>
         <xyzOffsets>0 0 0</xyzOffsets> <!-- initialize odometry for fake localization-->
         <rpyOffsets>0 0 0</rpyOffsets>
-        <interface:position name="p3d_plug_magnet_position"/>
+        <interface:position name="p3d_plug_holder_1_position"/>
       </controller:ros_p3d>
     </gazebo>
@@ -98,5 +98,14 @@
     </gazebo>
     <!-- modeling plug on base holder magnet location -->
-    <gazebo reference="plug_magnet">
+    <gazebo reference="plug_holder_1">
+      <material value="PR2/Red" />
+    </gazebo>
+    <gazebo reference="plug_holder_2">
+      <material value="PR2/Red" />
+    </gazebo>
+    <gazebo reference="plug_holder_3">
+      <material value="PR2/Red" />
+    </gazebo>
+    <gazebo reference="plug_holder_4">
       <material value="PR2/Red" />
     </gazebo>

Commit message: * update finger tip to use tip pads only for collision.  * turn on selfCollide for finger tip (needed for plug_in finger_tip collision with base_link).  * added some finger tip meshes for testing.  * update base plug holder.  * give mass to gripper_tool_frame so it's not ignored by simulator.  * set base_link friction to 0.

File: pr2_defs/defs/base/base_defs.urdf.xacro (robot description, xacro)
@@ -175,10 +175,10 @@
   </macro>
   <macro name="pr2_plug_holder" params="name">
-    <joint name="plug_holder_1_joint" type="fixed">
-      <origin xyz="0.18 0 ${base_height_offset+0.235}" rpy="0 0 0" />
+    <joint name="plug_holder_joint" type="fixed">
+      <origin xyz="0.18 0 ${base_height_offset+base_size_z - 0.001/2}" rpy="0 0 0" />
       <parent link="${name}_link"/>
-      <child link="plug_holder_1"/>
-    </joint>
-    <link name="plug_holder_1">
+      <child link="plug_holder"/>
+    </joint>
+    <link name="plug_holder">
       <inertial>
         <mass value="0.1" />
@@ -199,76 +199,4 @@
       </collision>
     </link>
-    <joint name="plug_holder_2_joint" type="fixed">
-      <origin xyz="0.21 0 ${base_height_offset+0.235}" rpy="0 0 0" />
-      <parent link="${name}_link"/>
-      <child link="plug_holder_2"/>
-    </joint>
-    <link name="plug_holder_2">
-      <inertial>
-        <mass value="0.1" />
-        <origin xyz="0 0 0.0" />
-        <inertia ixx="0.1" ixy="0" ixz="0" iyy="0.1" iyz="0" izz="0.1" />
-      </inertial>
-      <visual>
-        <origin xyz="0 0 0" rpy="0 0 0" />
-        <geometry>
-          <box size="0.001 0.001 0.001"/>
-        </geometry>
-      </visual>
-      <collision>
-        <origin xyz="0 0 0.0" rpy="0 0 0" />
-        <geometry>
-          <box size=".001 .001 .001" />
-        </geometry>
-      </collision>
-    </link>
-    <joint name="plug_holder_3_joint" type="fixed">
-      <origin xyz="0.20 -.04 ${base_height_offset+0.235}" rpy="0 0 0" />
-      <parent link="${name}_link"/>
-      <child link="plug_holder_3"/>
-    </joint>
-    <link name="plug_holder_3">
-      <inertial>
-        <mass value="0.1" />
-        <origin xyz="0 0 0.0" />
-        <inertia ixx="0.1" ixy="0" ixz="0" iyy="0.1" iyz="0" izz="0.1" />
-      </inertial>
-      <visual>
-        <origin xyz="0 0 0" rpy="0 0 0" />
-        <geometry>
-          <box size="0.001 0.001 0.001"/>
-        </geometry>
-      </visual>
-      <collision>
-        <origin xyz="0 0 0.0" rpy="0 0 0" />
-        <geometry>
-          <box size=".001 .001 .001" />
-        </geometry>
-      </collision>
-    </link>
-    <joint name="plug_holder_4_joint" type="fixed">
-      <origin xyz="0.20 0.04 ${base_height_offset+0.235}" rpy="0 0 0" />
-      <parent link="${name}_link"/>
-      <child link="plug_holder_4"/>
-    </joint>
-    <link name="plug_holder_4">
-      <inertial>
-        <mass value="0.1" />
-        <origin xyz="0 0 0.0" />
-        <inertia ixx="0.1" ixy="0" ixz="0" iyy="0.1" iyz="0" izz="0.1" />
-      </inertial>
-      <visual>
-        <origin xyz="0 0 0" rpy="0 0 0" />
-        <geometry>
-          <box size="0.001 0.001 0.001"/>
-        </geometry>
-      </visual>
-      <collision>
-        <origin xyz="0 0 0.0" rpy="0 0 0" />
-        <geometry>
-          <box size=".001 .001 .001" />
-        </geometry>
-      </collision>
-    </link>
   </macro>
 </robot>

File: pr2_defs/defs/base/base_gazebo.xacro (robot description, xacro)
@@ -42,7 +42,7 @@
         </controller:ros_bumper>
       </sensor:contact>
-      <mu1 value="500.0" />
-      <mu2 value="500.0" />
-      <kp  value="100000000.0" />
+      <mu1 value="0.0" />
+      <mu2 value="0.0" />
+      <kp  value="1000000.0" />
       <kd  value="1.0" />
       <material value="PR2/Green" />
@@ -60,14 +60,14 @@
         <interface:position name="p3d_base_position"/>
       </controller:ros_p3d>
-      <controller:ros_p3d name="p3d_plug_holder_1_controller" plugin="libros_p3d.so">
+      <controller:ros_p3d name="p3d_plug_holder_controller" plugin="libros_p3d.so">
         <alwaysOn>true</alwaysOn>
         <updateRate>100.0</updateRate>
-        <bodyName>plug_holder_1</bodyName>
-        <topicName>plug_holder_1_pose_ground_truth</topicName>
+        <bodyName>plug_holder</bodyName>
+        <topicName>plug_holder_pose_ground_truth</topicName>
         <gaussianNoise>0.01</gaussianNoise>
         <frameName>map</frameName>
         <xyzOffsets>0 0 0</xyzOffsets> <!-- initialize odometry for fake localization-->
         <rpyOffsets>0 0 0</rpyOffsets>
-        <interface:position name="p3d_plug_holder_1_position"/>
+        <interface:position name="p3d_plug_holder_position"/>
       </controller:ros_p3d>
     </gazebo>
@@ -98,5 +98,5 @@
     </gazebo>
     <!-- modeling plug on base holder magnet location -->
-    <gazebo reference="plug_holder_1">
+    <gazebo reference="plug_holder">
       <material value="PR2/Red" />
     </gazebo>

File: pr2_defs/defs/gripper/gripper_defs.urdf.xacro (robot description, xacro)
@@ -118,5 +118,5 @@
         <origin xyz="0 0 0" rpy="0 0 0" />
         <geometry name="${prefix}_l_finger_tip_collision_geom">
-          <mesh filename="package://pr2_defs/meshes/convex/finger_tip_l_convex.stlb" />
+          <mesh filename="package://pr2_defs/meshes/finger_tip_pad2_l.stlb" />
         </geometry>
         <verbose value="Yes" />
@@ -151,5 +151,5 @@
         <origin xyz="0 0 0" rpy="0 0 0" />
         <geometry name="${prefix}_r_finger_tip_collision_geom">
-          <mesh filename="package://pr2_defs/meshes/convex/finger_tip_r_convex.stlb" />
+          <mesh filename="package://pr2_defs/meshes/finger_tip_pad2_r.stlb" />
         </geometry>
         <verbose value="Yes" />
@@ -229,9 +229,9 @@
       <!-- TODO: all that follows is made-up and useless, but the old parser crashes without it -->
       <inertial>
-        <mass value="0" />
-        <origin xyz="0 0 0" rpy="0 0 0" />
-        <inertia ixx="0" ixy="0" ixz="0" iyy="0" iyz="0" izz="0" />
-      </inertial>
-      <visual name="${side}_gripper_tool_visual">
+        <mass value="0.01" />
+        <origin xyz="0 0 0" rpy="0 0 0" />
+        <inertia ixx="0.001" ixy="0" ixz="0" iyy="0.001" iyz="0" izz="0.001" />
+      </inertial>
+      <visual>
         <origin xyz="0 0 0" rpy="0 0 0" />
         <geometry name="${side}_gripper_tool_visual_geom">
@@ -240,5 +240,5 @@
         <material name="Grey" />
       </visual>
-      <collision name="${side}_gripper_tool_collision">
+      <collision>
         <origin xyz="-0.1 0 0" rpy="0 0 0" /> <!-- move it out of the way -->
         <geometry name="${side}_gripper_tool_collision_geom">

File: pr2_defs/defs/gripper/gripper_gazebo.xacro (robot description, xacro)
@@ -70,5 +70,5 @@
     <gazebo reference="${prefix}_l_finger_tip_link">
       <turnGravityOff>true</turnGravityOff>
-      <selfCollide value="false" />
+      <selfCollide value="true" />
       <sensor:contact name="${prefix}_l_finger_tip_contact_sensor">
         <geom>${prefix}_l_finger_tip_link_geom</geom>
@@ -85,5 +85,5 @@
       <kp  value="10000000.0" />
       <kd  value="1.0" />
-      <material value="PR2/Green" />
+      <material value="PR2/Red" />
     </gazebo>
     <gazebo reference="${prefix}_l_finger_tip_joint">
@@ -96,5 +96,5 @@
     <gazebo reference="${prefix}_r_finger_tip_link">
       <turnGravityOff>true</turnGravityOff>
-      <selfCollide value="false" />
+      <selfCollide value="true" />
       <sensor:contact name="${prefix}_r_finger_tip_contact_sensor">
         <geom>${prefix}_r_finger_tip_link_geom</geom>
@@ -111,5 +111,5 @@
       <kp  value="10000000.0" />
       <kd  value="1.0" />
-      <material value="PR2/Green" />
+      <material value="PR2/Red" />
     </gazebo>
     <gazebo>
@@ -198,6 +198,17 @@
         <interface:position name="p3d_${side}_gripper_palm_position_iface" />
       </controller:ros_p3d>
-    </gazebo>
-    <gazebo reference="${side}_gripper_tool_link">
+      <controller:ros_p3d name="p3d_${side}_gripper_tool_frame" plugin="libros_p3d.so">
+        <alwaysOn>true</alwaysOn>
+        <updateRate>100.0</updateRate>
+        <bodyName>${side}_gripper_tool_frame</bodyName>
+        <topicName>${side}_gripper_tool_frame_pose_ground_truth</topicName>
+        <xyzOffsets>0 0 0</xyzOffsets>
+        <rpyOffsets>0 0 0</rpyOffsets>
+        <gaussianNoise>0.0</gaussianNoise>
+        <frameName>/map</frameName>
+        <interface:position name="p3d_${side}_gripper_tool_frame_position_iface" />
+      </controller:ros_p3d>
+    </gazebo>
+    <gazebo reference="${side}_gripper_tool_frame">
       <turnGravityOff>true</turnGravityOff>
       <material value="PR2/Grey" />

Commit message: fix visualization scale, in the wrong place.

File: pr2_defs/defs/base/base_defs.urdf.xacro (robot description, xacro)
@@ -48,5 +48,5 @@
         <origin xyz="0 0 0" rpy="0 0 0" />
         <geometry>
-          <mesh filename="package://pr2_defs/meshes/pr2_wheel.stl" />
+          <mesh filename="package://pr2_defs/meshes/pr2_wheel.stl" scale="0.65 1.0 0.65"/>
         </geometry>
         <material name="Caster_${suffix}" />
@@ -120,5 +120,5 @@
         <origin xyz="0 0 ${base_height_offset}" rpy="0 0 0" />
         <geometry>
-          <mesh filename="package://pr2_defs/meshes/base.stl" scale="0.65 1.0 0.65"/>
+          <mesh filename="package://pr2_defs/meshes/base.stl"/>
         </geometry>
         <material name="Green" />
