Commit message: * turn off gripper finger tips selfCollide in sim.  enable base_link selfCollide.  selfCollide is needed for plug in to work.  * removed artificial height offset for base_link collision body. The offset was added because detecting plug on base was off by this amount, but measurement of the actual base does not reflect the height offset.  The offset must be introduced else where.

File: pr2_defs/defs/base/base_defs.urdf.xacro (robot description, xacro)
@@ -14,10 +14,9 @@
   <property name="base_cg_z" value="0.293" />
   <property name="base_mass" value="116.0" />
-  <!-- base appears "raised" from our initial geom def from function -->
-  <property name="base_height_offset" value="0.05" />
   <!-- simplified box collision geometry for base -->
   <property name="base_size_x" value="0.65" />
   <property name="base_size_y" value="0.65" />
   <property name="base_size_z" value="0.23" />
+  <property name="base_collision_size_z" value="0.04" />
   <!-- simplified box collision geometry for hokuyo laser -->
   <property name="base_laser_x" value="0.275" />
@@ -27,5 +26,5 @@
   <property name="base_laser_size_y" value="0.06" />
   <property name="base_laser_size_z" value="0.03" />
-  <property name="base_laser_collision_offset_z" value="0.02" />
+  <property name="base_laser_collision_offset_z" value="0.023" />
   <macro name="pr2_wheel" params="suffix parent reflect">
     <joint name="${parent}_${suffix}_wheel_joint" type="continuous">
@@ -48,5 +47,5 @@
         <origin xyz="0 0 0" rpy="0 0 0" />
         <geometry>
-          <mesh filename="package://pr2_defs/meshes/pr2_wheel.stl" scale="0.65 1.0 0.65"/>
+          <mesh filename="package://pr2_defs/meshes/pr2_wheel.stl" />
         </geometry>
         <material name="Caster_${suffix}" />
@@ -118,5 +117,5 @@
       </inertial>
       <visual>
-        <origin xyz="0 0 ${base_height_offset}" rpy="0 0 0" />
+        <origin xyz="0 0 0" rpy="0 0 0" />
         <geometry>
           <mesh filename="package://pr2_defs/meshes/base.stl"/>
@@ -125,7 +124,9 @@
       </visual>
       <collision>
-        <origin xyz="0 0 ${base_height_offset+base_size_z/2}" rpy="0 0 0" />
-        <geometry>
-          <box size="${base_size_x} ${base_size_y} ${base_size_z}" />
+        <!-- represent base collision with a simple rectangular model, positioned by base_size_z s.t. top
+             surface of the collision box matches the top surface of the PR2 base -->
+        <origin xyz="0 0 ${base_size_z-base_collision_size_z/2}" rpy="0 0 0" />
+        <geometry>
+          <box size="${base_size_x} ${base_size_y} ${base_collision_size_z}" />
         </geometry>
       </collision>
@@ -133,5 +134,5 @@
     <!-- base laser -->
     <joint name="base_laser_joint" type="fixed">
-      <origin xyz="${base_laser_x} ${base_laser_y} ${base_height_offset+base_laser_z}" rpy="0 0 0" />
+      <origin xyz="${base_laser_x} ${base_laser_y} ${base_laser_z}" rpy="0 0 0" />
       <parent link="${name}_link"/>
       <child link="base_laser"/>
@@ -176,5 +177,5 @@
   <macro name="pr2_plug_holder" params="name">
     <joint name="plug_holder_joint" type="fixed">
-      <origin xyz="0.18 0 ${base_height_offset+base_size_z - 0.001/2}" rpy="0 0 0" />
+      <origin xyz="0.18 0 ${base_size_z+0.001/2}" rpy="0 0 0" />
       <parent link="${name}_link"/>
       <child link="plug_holder"/>

File: pr2_defs/defs/base/base_gazebo.xacro (robot description, xacro)
@@ -32,4 +32,5 @@
   <macro name="pr2_base_gazebo" params="name">
     <gazebo reference="${name}_link">
+      <selfCollide value="true" />
       <sensor:contact name="${name}_contact_sensor">
         <geom>${name}_link_geom</geom>

File: pr2_defs/defs/gripper/gripper_defs.urdf.xacro (robot description, xacro)
@@ -9,4 +9,5 @@
   <property name="gripper_upper_angle" value="0.548" />
   <property name="gripper_lower_angle" value="0.00" />
+  <property name="gripper_margin"      value="0.0" />
   <property name="finger_damping"             value="0.2" />
   <property name="finger_tip_damping"         value="0.01" />
@@ -16,5 +17,5 @@
            lower="${gripper_lower_angle}" upper="${gripper_upper_angle}" />
     <safety_controller k_velocity="100.0" k_position="100.0"
-                       soft_lower_limit="${gripper_lower_angle+0.0}" soft_upper_limit="${gripper_upper_angle-0.0}" />
+                       soft_lower_limit="${gripper_lower_angle+gripper_margin}" soft_upper_limit="${gripper_upper_angle-gripper_margin}" />
   </macro>
   <macro name="pr2_finger" params="prefix parent">

File: pr2_defs/defs/gripper/gripper_gazebo.xacro (robot description, xacro)
@@ -5,12 +5,10 @@
        xmlns:interface="http://playerstage.sourceforge.net/gazebo/xmlschema/#interface">
   <property name="finger_stop_kd"             value="1.0" />
-  <property name="finger_stop_kp"             value="10000000.0" />
+  <property name="finger_stop_kp"             value="1000000.0" />
   <property name="finger_fudge_factor"        value="1.0" />
-  <property name="finger_kp"                  value="0.0" />
-  <property name="finger_kd"                  value="0.0" />
-  <property name="finger_fm"                  value="0.0" />
-  <property name="finger_tip_kp"              value="0.0" />
-  <property name="finger_tip_kd"              value="0.0" />
-  <property name="finger_tip_fm"              value="0.0" />
+  <property name="finger_kp"                  value="1000000.0" />
+  <property name="finger_kd"                  value="1.0" />
+  <property name="finger_tip_kp"              value="1000000.0" />
+  <property name="finger_tip_kd"              value="1.0" />
   <property name="finger_tip_mu"              value="500.0" />
   <property name="finger_mu"                  value="500.0" />
@@ -31,6 +29,6 @@
       <mu1 value="${finger_mu}" />
       <mu2 value="${finger_mu}" />
-      <kp value="1000000.0" />
-      <kd value="1.0" />
+      <kp value="${finger_kp}" />
+      <kd value="${finger_kd}" />
       <material value="PR2/Grey" />
       <!-- for "${prefix}_l_finger_joint"-->
@@ -57,6 +55,6 @@
       <mu1 value="${finger_mu}" />
       <mu2 value="${finger_mu}" />
-      <kp value="1000000.0" />
-      <kd value="1.0" />
+      <kp value="${finger_kp}" />
+      <kd value="${finger_kd}" />
       <material value="PR2/Grey" />
     </gazebo>
@@ -70,5 +68,5 @@
     <gazebo reference="${prefix}_l_finger_tip_link">
       <turnGravityOff>true</turnGravityOff>
-      <selfCollide value="true" />
+      <selfCollide value="false" />
       <sensor:contact name="${prefix}_l_finger_tip_contact_sensor">
         <geom>${prefix}_l_finger_tip_link_geom</geom>
@@ -83,6 +81,6 @@
       <mu1 value="${finger_tip_mu}" />
       <mu2 value="${finger_tip_mu}" />
-      <kp  value="10000000.0" />
-      <kd  value="1.0" />
+      <kp value="${finger_tip_kp}" />
+      <kd value="${finger_tip_kd}" />
       <material value="PR2/Red" />
     </gazebo>
@@ -96,5 +94,5 @@
     <gazebo reference="${prefix}_r_finger_tip_link">
       <turnGravityOff>true</turnGravityOff>
-      <selfCollide value="true" />
+      <selfCollide value="false" />
       <sensor:contact name="${prefix}_r_finger_tip_contact_sensor">
         <geom>${prefix}_r_finger_tip_link_geom</geom>
@@ -109,6 +107,6 @@
       <mu1 value="${finger_tip_mu}" />
       <mu2 value="${finger_tip_mu}" />
-      <kp  value="10000000.0" />
-      <kd  value="1.0" />
+      <kp value="${finger_tip_kp}" />
+      <kd value="${finger_tip_kd}" />
       <material value="PR2/Red" />
     </gazebo>
