Commit message: clean up urdf, visual/inertial/collision/geometry elements should not have names

File: pr2_defs/defs/base/alpha2_base_defs.urdf.xacro (robot description, xacro)
@@ -51,14 +51,14 @@
                   iyy="0.015218160428" iyz="-0.000004273467" izz="0.011763977943" />
       </inertial>
-      <visual name="${parent}_${suffix}_wheel_visual">
+      <visual>
         <origin xyz="0 0 0" rpy="0 0 0" />
-        <geometry name="${parent}_${suffix}_wheel_visual_geom">
-          <mesh filename="package://pr2_defs/meshes/pr2_wheel.stl" />
+        <geometry>
+          <mesh filename="package://pr2_defs/meshes/pr2_wheel.stl" scale="0.65 1.0 0.65"/>
         </geometry>
         <material name="Caster_${suffix}" />
       </visual>
-      <collision name="${parent}_${suffix}_wheel_collision">
+      <collision>
         <origin xyz="0 0 0" rpy="${M_PI/2} 0 0" />
-        <geometry name="${parent}_${suffix}_wheel_collision_geom">
+        <geometry>
           <cylinder radius="${wheel_radius}" length="${wheel_length}" />
         </geometry>
@@ -87,14 +87,14 @@
                   iyy="0.015218160428" iyz="-0.000004273467" izz="0.011763977943" />
       </inertial>
-      <visual name="${suffix}_caster_rotation_visual">
+      <visual>
         <origin xyz="0 0 0" rpy="0 0 0" />
-        <geometry name="${suffix}_caster_rotation_visual_geom">
+        <geometry>
           <mesh filename="package://pr2_defs/meshes/caster.stl" />
         </geometry>
         <material name="Green" />
       </visual>
-      <collision name="${suffix}_caster_rotation_collision">
+      <collision>
         <origin xyz="0 0 0.07" rpy="0.0 0.0 0.0" />
-        <geometry name="${suffix}_caster_rotation_collision_geom">
+        <geometry>
           <box size="0.192 0.164 0.013" />
         </geometry>
@@ -120,14 +120,14 @@
                  iyy="5.669473158652" iyz="-0.007379583694" izz="3.683196351726" />
       </inertial>
-      <visual name="${name}_visual">
+      <visual>
         <origin xyz="0 0 ${base_height_offset}" rpy="0 0 0" />
-        <geometry name="${name}_visual_geom">
+        <geometry>
           <mesh filename="package://pr2_defs/meshes/base.stl" />
         </geometry>
         <material name="Green" />
       </visual>
-      <collision name="${name}_collision">
+      <collision>
         <origin xyz="0 0 ${base_height_offset+base_size_z/2}" rpy="0 0 0" />
-        <geometry name="${name}_collision_geom">
+        <geometry>
           <box size="${base_size_x} ${base_size_y} ${base_size_z}" />
         </geometry>
@@ -147,14 +147,14 @@
         <inertia ixx="0.1" ixy="0" ixz="0" iyy="0.1" iyz="0" izz="0.1" />
       </inertial>
-      <visual name="base_lvisual">
+      <visual>
         <origin xyz="0 0 ${base_laser_collision_offset_z}" rpy="0 0 0" />
-        <geometry name="base_laser_visual_geom">
+        <geometry>
           <box size="${base_laser_size_x} ${base_laser_size_y} ${base_laser_size_z}"/>
         </geometry>
         <material name="Red" />
       </visual>
-      <collision name="base_lcollision">
+      <collision>
         <origin xyz="0 0 ${base_laser_collision_offset_z}" rpy="0 0 0" />
-        <geometry name="base_laser_collision_geom">
+        <geometry>
           <box size="${base_laser_size_x} ${base_laser_size_y} ${base_laser_size_z}"/>
         </geometry>

File: pr2_defs/defs/base/base_defs.urdf.xacro (robot description, xacro)
@@ -45,14 +45,14 @@
                   iyy="0.015218160428" iyz="-0.000004273467" izz="0.011763977943" />
       </inertial>
-      <visual name="${parent}_${suffix}_wheel_visual">
+      <visual>
         <origin xyz="0 0 0" rpy="0 0 0" />
-        <geometry name="${parent}_${suffix}_wheel_visual_geom">
+        <geometry>
           <mesh filename="package://pr2_defs/meshes/pr2_wheel.stl" />
         </geometry>
         <material name="Caster_${suffix}" />
       </visual>
-      <collision name="${parent}_${suffix}_wheel_collision">
+      <collision>
         <origin xyz="0 0 0" rpy="${M_PI/2} 0 0" />
-        <geometry name="${parent}_${suffix}_wheel_collision_geom">
+        <geometry>
           <cylinder radius="${wheel_radius}" length="${wheel_length}" />
         </geometry>
@@ -81,14 +81,14 @@
                   iyy="0.015218160428" iyz="-0.000004273467" izz="0.011763977943" />
       </inertial>
-      <visual name="${suffix}_caster_rotation_visual">
+      <visual>
         <origin xyz="0 0 0" rpy="0 0 0" />
-        <geometry name="${suffix}_caster_rotation_visual_geom">
+        <geometry>
           <mesh filename="package://pr2_defs/meshes/caster.stl" />
         </geometry>
         <material name="Green" />
       </visual>
-      <collision name="${suffix}_caster_rotation_collision">
+      <collision>
         <origin xyz="0 0 0.07" rpy="0.0 0.0 0.0" />
-        <geometry name="${suffix}_caster_rotation_collision_geom">
+        <geometry>
           <box size="0.192 0.164 0.013" />
         </geometry>
@@ -117,14 +117,14 @@
                  iyy="5.669473158652" iyz="-0.007379583694" izz="3.683196351726" />
       </inertial>
-      <visual name="${name}_visual">
+      <visual>
         <origin xyz="0 0 ${base_height_offset}" rpy="0 0 0" />
-        <geometry name="${name}_visual_geom">
-          <mesh filename="package://pr2_defs/meshes/base.stl" />
+        <geometry>
+          <mesh filename="package://pr2_defs/meshes/base.stl" scale="0.65 1.0 0.65"/>
         </geometry>
         <material name="Green" />
       </visual>
-      <collision name="${name}_collision">
+      <collision>
         <origin xyz="0 0 ${base_height_offset+base_size_z/2}" rpy="0 0 0" />
-        <geometry name="${name}_collision_geom">
+        <geometry>
           <box size="${base_size_x} ${base_size_y} ${base_size_z}" />
         </geometry>
@@ -143,14 +143,14 @@
         <inertia ixx="0.1" ixy="0" ixz="0" iyy="0.1" iyz="0" izz="0.1" />
       </inertial>
-      <visual name="base_lvisual">
+      <visual>
         <origin xyz="0 0 ${base_laser_collision_offset_z}" rpy="0 0 0" />
-        <geometry name="base_laser_visual_geom">
+        <geometry>
           <box size="${base_laser_size_x} ${base_laser_size_y} ${base_laser_size_z}"/>
         </geometry>
         <material name="Red" />
       </visual>
-      <collision name="base_lcollision">
+      <collision>
         <origin xyz="0 0 ${base_laser_collision_offset_z}" rpy="0 0 0" />
-        <geometry name="base_laser_collision_geom">
+        <geometry>
           <box size="${base_laser_size_x} ${base_laser_size_y} ${base_laser_size_z}"/>
         </geometry>

Commit message: URDF Link rename: base_laser --> base_laser_link.  Staying consistent with suffixed *_link naming convention (e.g. tilt_laser_link).  This change will not work with pre simulator_stage-0.10.0 stack release.

File: pr2_defs/defs/base/alpha2_base_defs.urdf.xacro (robot description, xacro)
@@ -139,7 +139,7 @@
       <origin xyz="${base_laser_x} ${base_laser_y} ${base_height_offset+base_laser_z}" rpy="0 0 0" />
       <parent link="${name}_link"/>
-      <child link="base_laser" />
+      <child link="base_laser_link" />
     </joint>
-    <link name="base_laser" type="laser">
+    <link name="base_laser_link" type="laser">
       <inertial>
         <mass value="1.0" />

File: pr2_defs/defs/base/alpha2_base_gazebo.xacro (robot description, xacro)
@@ -60,6 +60,6 @@
     </gazebo>
     <!-- base laser -->
-    <gazebo reference="base_laser">
-      <sensor:ray name="base_laser">
+    <gazebo reference="base_laser_link">
+      <sensor:ray name="base_laser_link">
         <rayCount>640</rayCount>
         <rangeCount>640</rangeCount>
@@ -73,11 +73,11 @@
         <resRange>0.01</resRange>
         <updateRate>20.0</updateRate>
-        <controller:gazebo_ros_laser name="gazebo_ros_base_laser_controller" plugin="libgazebo_ros_laser.so">
+        <controller:gazebo_ros_laser name="gazebo_ros_base_laser_link_controller" plugin="libgazebo_ros_laser.so">
           <gaussianNoise>0.005</gaussianNoise>
           <alwaysOn>true</alwaysOn>
           <updateRate>20.0</updateRate>
           <topicName>base_scan</topicName>
-          <frameName>base_laser</frameName>
-          <interface:laser name="gazebo_ros_base_laser_iface" />
+          <frameName>base_laser_link</frameName>
+          <interface:laser name="gazebo_ros_base_laser_link_iface" />
         </controller:gazebo_ros_laser>
       </sensor:ray>

File: pr2_defs/defs/base/base_defs.urdf.xacro (robot description, xacro)
@@ -136,7 +136,7 @@
       <origin xyz="${base_laser_x} ${base_laser_y} ${base_laser_z}" rpy="0 0 0" />
       <parent link="${name}_link"/>
-      <child link="base_laser"/>
-    </joint>
-    <link name="base_laser" type="laser">
+      <child link="base_laser_link"/>
+    </joint>
+    <link name="base_laser_link" type="laser">
       <inertial>
         <mass value="1.0" />

File: pr2_defs/defs/base/base_gazebo.xacro (robot description, xacro)
@@ -75,6 +75,6 @@
     </gazebo>
     <!-- base laser -->
-    <gazebo reference="base_laser">
-      <sensor:ray name="base_laser">
+    <gazebo reference="base_laser_link">
+      <sensor:ray name="base_laser_link">
         <rayCount>640</rayCount>
         <rangeCount>640</rangeCount>
@@ -88,11 +88,11 @@
         <resRange>0.01</resRange>
         <updateRate>20.0</updateRate>
-        <controller:gazebo_ros_laser name="gazebo_ros_base_laser_controller" plugin="libgazebo_ros_laser.so">
+        <controller:gazebo_ros_laser name="gazebo_ros_base_laser_link_controller" plugin="libgazebo_ros_laser.so">
           <gaussianNoise>0.005</gaussianNoise>
           <alwaysOn>true</alwaysOn>
           <updateRate>20.0</updateRate>
           <topicName>base_scan</topicName>
-          <frameName>base_laser</frameName>
-          <interface:laser name="gazebo_ros_base_laser_iface" />
+          <frameName>base_laser_link</frameName>
+          <interface:laser name="gazebo_ros_base_laser_link_iface" />
         </controller:gazebo_ros_laser>
       </sensor:ray>
