Commit message: update urdf, launch scripts to remove world links.

File: pr2_defs/defs/base/alpha2_base_defs.urdf.xacro (robot description, xacro)
@@ -107,10 +107,5 @@
     <pr2_caster_alpha2_transmission suffix="${suffix}" />
   </macro>
-  <macro name="pr2_base_alpha2" params="name *origin">
-    <joint name="${name}_joint" type="planar">
-      <insert_block name="origin" />
-      <parent link="world"/>
-      <child link="${name}_link" />
-    </joint>
+  <macro name="pr2_base_alpha2" params="name">
     <link name="${name}_link">
       <inertial>

File: pr2_defs/defs/base/base_defs.urdf.xacro (robot description, xacro)
@@ -103,10 +103,5 @@
   <property name="caster_offset_y" value="0.2225" />
   <property name="caster_offset_z" value="0.0282" />
-  <macro name="pr2_base" params="name *origin">
-    <joint name="${name}_joint" type="planar">
-      <insert_block name="origin" />
-      <parent link="world"/>
-      <child link="${name}_link"/>
-    </joint>
+  <macro name="pr2_base" params="name">
     <link name="${name}_link">
       <inertial>

File: pr2_defs/robots/hca.urdf.xacro (robot description, xacro)
@@ -1,4 +1,5 @@
 <?xml version="1.0"?>
-<robot name="hca">
+<robot name="hca"
+       xmlns:joint="http://playerstage.sourceforge.net/gazebo/xmlschema/#joint">
   <!-- Include file with calibration parameters -->
   <include filename="$(find pr2_defs)/calibration/default_cal.xml" />
@@ -11,18 +12,13 @@
   <include filename="$(find pr2_defs)/defs/materials.urdf.xacro" />
   <!-- Make base joint for visualization -->
-  <joint name="base_joint" type="fixed">
-    <origin xyz=" 0 0 0.53 " rpy=" 0 0 0" />
-    <parent link="world" />
-    <child link="base_link" />
-  </joint>
   <link name="base_link">
     <inertial>
       <mass value="100" />
-      <origin xyz=" 0 0 0 " />
+      <origin xyz="0 0 0" />
       <inertia ixx="100"  ixy="0"  ixz="0" iyy="100" iyz="0" izz="100" />
     </inertial>
     <visual>
       <!-- 1.06m above ground -->
-      <origin xyz="0 0 0" rpy="0 0 0 " />
+      <origin xyz="0 0 0" rpy="0 0 0" />
       <geometry>
 	<box size=".6 0.45 1.06" />
@@ -30,5 +26,5 @@
     </visual>
     <collision>
-      <origin xyz="0 0 0" rpy="0.0 0.0 0.0 " />
+      <origin xyz="0 0 0" rpy="0.0 0.0 0.0" />
       <geometry>
         <box size="0.6 0.45 1.06" />

File: pr2_defs/robots/hcb.urdf.xacro (robot description, xacro)
@@ -1,4 +1,5 @@
 <?xml version="1.0"?>
-<robot name="hcb">
+<robot name="hcb"
+       xmlns:joint="http://playerstage.sourceforge.net/gazebo/xmlschema/#joint">
   <!-- Include file with calibration parameters -->
   <include filename="$(find pr2_defs)/calibration/default_cal.xml" />
@@ -12,18 +13,13 @@
   <include filename="$(find pr2_defs)/defs/materials.urdf.xacro" />
   <!-- Make base joint for visualization -->
-  <joint name="base_joint" type="fixed">
-    <origin xyz="0 0 0.53" rpy="0 0 0" />
-    <parent link="world" />
-    <child link="base_link" />
-  </joint>
   <link name="base_link">
     <inertial>
       <mass value="100" />
-      <origin xyz=" 0 0 0 " />
+      <origin xyz="0 0 0" />
       <inertia ixx="100"  ixy="0"  ixz="0" iyy="100" iyz="0" izz="100" />
     </inertial>
     <visual>
       <!-- 1.06m above ground -->
-      <origin xyz="0 0 0" rpy="0 0 0 " />
+      <origin xyz="0 0 0" rpy="0 0 0" />
       <geometry>
 	<box size=".6 0.45 1.06" />
@@ -31,5 +27,5 @@
     </visual>
     <collision>
-      <origin xyz="0 0 0" rpy="0.0 0.0 0.0 " />
+      <origin xyz="0 0 0" rpy="0.0 0.0 0.0" />
       <geometry>
         <box size="0.6 0.45 1.06" />

File: pr2_defs/robots/hcc.urdf.xacro (robot description, xacro)
@@ -1,4 +1,5 @@
 <?xml version="1.0"?>
-<robot name="hcb">
+<robot name="hcb"
+       xmlns:joint="http://playerstage.sourceforge.net/gazebo/xmlschema/#joint">
   <!-- Include file with calibration parameters -->
   <include filename="$(find pr2_defs)/calibration/default_cal.xml" />
@@ -12,18 +13,13 @@
   <include filename="$(find pr2_defs)/defs/materials.urdf.xacro" />
   <!-- Make base joint for visualization -->
-  <joint name="base_joint" type="fixed">
-    <origin xyz="0 0 0.53" rpy="0 0 0" />
-    <parent link="world" />
-    <child link="base_link" />
-  </joint>
   <link name="base_link">
     <inertial>
       <mass value="100" />
-      <origin xyz=" 0 0 0 " />
+      <origin xyz="0 0 0" />
       <inertia ixx="100"  ixy="0"  ixz="0" iyy="100" iyz="0" izz="100" />
     </inertial>
     <visual>
       <!-- 1.06m above ground -->
-      <origin xyz="0 0 0" rpy="0 0 0 " />
+      <origin xyz="0 0 0" rpy="0 0 0" />
       <geometry>
 	<box size=".6 0.45 1.06" />
@@ -31,5 +27,5 @@
     </visual>
     <collision>
-      <origin xyz="0 0 0" rpy="0.0 0.0 0.0 " />
+      <origin xyz="0 0 0" rpy="0.0 0.0 0.0" />
       <geometry>
         <box size="0.6 0.45 1.06" />

File: pr2_defs/robots/l_arm.urdf.xacro (robot description, xacro)
@@ -29,9 +29,4 @@
   </pr2_gripper>
   <!-- Solid Base -->
-  <joint name="base_joint" type="fixed">
-    <origin xyz="0 0 0" rpy="0 0 0" />
-    <parent link="world" />
-    <child link="torso_lift_link" />
-  </joint>
   <link name="torso_lift_link">
     <inertial>
@@ -60,3 +55,14 @@
     <kd>1.0</kd>
   </gazebo>
+  <!-- fixed joint to the world for simulation -->
+  <gazebo>
+    <joint:hinge name="base_fixed_joint">
+      <body1>world</body1>
+      <body2>torso_lift_link</body2>
+      <anchor>torso_lift_link</anchor>
+      <lowStop>0</lowStop>
+      <highStop>0</highStop>
+      <axis>0 0 1</axis>
+    </joint:hinge>
+  </gazebo>
 </robot>

File: pr2_defs/robots/l_gripper.urdf.xacro (robot description, xacro)
@@ -23,10 +23,5 @@
     <origin xyz="0 0 1" rpy="0 0 0" />
   </pr2_gripper>
-  <!-- Solid Base -->
-  <joint name="base_joint" type="fixed">
-    <origin xyz="0 0 0" rpy="0 0 0" />
-    <parent link="world" />
-    <child link="base_link" />
-  </joint>
+  <!-- Base -->
   <link name="base_link">
     <inertial>
@@ -36,7 +31,7 @@
     </inertial>
     <visual>
-      <origin xyz="0 0 0" rpy="0 0 0 " />
+      <origin xyz="0 0 0" rpy="0 0 0" />
       <geometry>
-        <box size="0.01 0.01 0.01" />
+        <box size="0.0 0.0 0.0" />
       </geometry>
     </visual>
@@ -44,5 +39,5 @@
       <origin xyz="0 0 0" rpy="0.0 0.0 0.0" />
       <geometry>
-        <box size="0.01 0.01 0.01" />
+        <box size="1.0 1.0 0.001" />
       </geometry>
     </collision>
@@ -61,4 +56,13 @@
       <interface:position name="p3d_l_gripper_palm_position"/>
     </controller:gazebo_ros_p3d>
+    <!-- fixed joint to the world for simulation -->
+    <joint:hinge name="base_fixed_joint">
+      <body1>world</body1>
+      <body2>base_link</body2>
+      <anchor>base_link</anchor>
+      <lowStop>0</lowStop>
+      <highStop>0</highStop>
+      <axis>0 0 1</axis>
+    </joint:hinge>
   </gazebo>
 </robot>

File: pr2_defs/robots/laser_tilt.urdf.xacro (robot description, xacro)
@@ -1,7 +1,8 @@
- <robot name="laser_tilt_test">
+ <robot name="laser_tilt_test"
+        xmlns:joint="http://playerstage.sourceforge.net/gazebo/xmlschema/#joint">
   <include filename="$(find pr2_defs)/defs/materials.urdf.xacro" />
   <include filename="$(find pr2_defs)/defs/head/head_defs.urdf.xacro" />
   <include filename="$(find pr2_defs)/defs/body/body_defs.urdf.xacro" />
-  <pr2_torso name="torso_lift" parent="world">
+  <pr2_torso name="torso_lift" parent="base_link">
     <origin xyz="0 0 0" rpy="0 0 0" />
   </pr2_torso>
@@ -9,3 +10,34 @@
     <origin xyz="0 0 0.03" rpy="0 0 0" />
   </pr2_tilting_laser>
+  <!-- Base -->
+  <link name="base_link">
+    <inertial>
+      <mass value="100" />
+      <origin xyz="0 0 1" />
+      <inertia ixx="100"  ixy="0"  ixz="0" iyy="1000" iyz="0" izz="1000" />
+    </inertial>
+    <visual>
+      <origin xyz="0 0 0" rpy="0 0 0 " />
+      <geometry>
+        <box size="0.01 0.01 0.01" />
+      </geometry>
+    </visual>
+    <collision>
+      <origin xyz="0 0 0" rpy="0.0 0.0 0.0" />
+      <geometry>
+        <box size="0.01 0.01 0.01" />
+      </geometry>
+    </collision>
+  </link>
+  <gazebo>
+    <!-- fixed joint to the world for simulation -->
+    <joint:hinge name="base_fixed_joint">
+      <body1>world</body1>
+      <body2>base_link</body2>
+      <anchor>base_link</anchor>
+      <lowStop>0</lowStop>
+      <highStop>0</highStop>
+      <axis>0 1 0</axis>
+    </joint:hinge>
+  </gazebo>
 </robot>

File: pr2_defs/robots/pr2.urdf.xacro (robot description, xacro)
@@ -25,7 +25,5 @@
        the origin block defines where the component is w.r.t its parent (in this case the parent
        is the world frame). For more, see http://www.ros.org/wiki/xacro -->
-  <pr2_base name="base" >
-    <origin xyz="0 0 0.051" rpy="0 0 0" /> <!-- 5.1cm is the height of the base when wheels contact ground -->
-  </pr2_base>
+  <pr2_base name="base"/>
   <pr2_torso name="torso_lift" parent="base_link">
     <origin xyz="-0.05 0 0.739675" rpy="0 0 0" />

File: pr2_defs/robots/pr2_armless.urdf.xacro (robot description, xacro)
@@ -11,7 +11,5 @@
   <include filename="$(find pr2_defs)/defs/gazebo/gazebo_defs.urdf.xacro" />
   <include filename="$(find pr2_defs)/defs/materials.urdf.xacro" />
-  <pr2_base name="base" >
-    <origin xyz="0 0 0.051" rpy="0 0 0" />
-  </pr2_base>
+  <pr2_base name="base"/>
   <pr2_torso name="torso_lift" parent="base_link">
     <origin xyz="-0.05 0 0.739675" rpy="0 0 0" />

File: pr2_defs/robots/r_arm.urdf.xacro (robot description, xacro)
@@ -28,10 +28,5 @@
     <origin xyz="0 0 0" rpy="0 0 0" />
   </pr2_gripper>
-  <!-- Solid Base -->
-  <joint name="base_joint" type="fixed">
-    <origin xyz="0 0 0" rpy="0 0 0" />
-    <parent link="world" />
-    <child link="torso_lift_link" />
-  </joint>
+  <!-- Base -->
   <link name="torso_lift_link">
     <inertial>
@@ -60,3 +55,14 @@
     <kd>1.0</kd>
   </gazebo>
+  <gazebo>
+    <!-- fixed joint to the world for simulation -->
+    <joint:hinge name="base_fixed_joint">
+      <body1>world</body1>
+      <body2>torso_lift_link</body2>
+      <anchor>torso_lift_link</anchor>
+      <lowStop>0</lowStop>
+      <highStop>0</highStop>
+      <axis>0 0 1</axis>
+    </joint:hinge>
+  </gazebo>
 </robot>

File: pr2_defs/robots/r_forearm_gripper.urdf.xacro (robot description, xacro)
@@ -26,20 +26,13 @@
     <origin xyz="0 0 0" rpy="0 0 0" />
   </pr2_gripper>
-  <!-- Solid Base -->
-  <joint name="base_joint" type="planar">
-    <origin xyz="0 0 1.002" rpy=" 0 0 0" />
-    <parent link="world" />
-    <!-- rotation of a local coordinate frame attached to the link with respect to a global coordinate frame -->
-    <!-- position of a local coordinate frame attached to the link with respect to the parent link's coordinate frame -->
-    <child link="base_link" />
-  </joint>
+  <!-- Base -->
   <link name="base_link"><!-- link specifying the base of the robot -->
     <inertial>
       <mass value="1000" />
-      <origin xyz=" 0 0 0 " /> <!-- position of the center of mass with respect to the link's own anchor in a local coordinate frame -->
+      <origin xyz="0 0 0" /> <!-- position of the center of mass with respect to the link's own anchor in a local coordinate frame -->
       <inertia ixx="1000"  ixy="0"  ixz="0" iyy="1000" iyz="0" izz="1000" />
     </inertial>
     <visual>
-      <origin xyz="0 0 -1" rpy="0 0 0 " /> <!-- location defined with respect to the link origin in a local coordinate frame -->
+      <origin xyz="0 0 -1" rpy="0 0 0" /> <!-- location defined with respect to the link origin in a local coordinate frame -->
       <!-- All angles always in radians, yaw about Z axis, pitch about the Y axis and roll about the X axis -->
       <geometry>
@@ -48,5 +41,5 @@
     </visual>
     <collision>
-      <origin xyz="0 0 -1" rpy="0.0 0.0 0.0 " /> <!-- default box is centered at the origin -->
+      <origin xyz="0 0 -1" rpy="0.0 0.0 0.0" /> <!-- default box is centered at the origin -->
       <!-- All angles always in radians, yaw about Z axis, pitch about the Y axis and roll about the X axis -->
       <geometry>

File: pr2_defs/robots/r_gripper.urdf.xacro (robot description, xacro)
@@ -23,10 +23,5 @@
     <origin xyz="0 0 1" rpy="0 0 0" />
   </pr2_gripper>
-  <!-- Solid Base -->
-  <joint name="base_joint" type="fixed">
-    <parent link="world" />
-    <origin xyz="0 0 0" rpy="0 0 0" />
-    <child link="base_link" />
-  </joint>
+  <!-- Base -->
   <link name="base_link">
     <inertial>
@@ -36,7 +31,7 @@
     </inertial>
     <visual>
-      <origin xyz="0 0 0" rpy="0 0 0 " />
+      <origin xyz="0 0 0" rpy="0 0 0" />
       <geometry>
-        <box size="0.01 0.01 0.01" />
+        <box size="0.0 0.0 0.0" />
       </geometry>
     </visual>
@@ -44,5 +39,5 @@
       <origin xyz="0 0 0" rpy="0.0 0.0 0.0" />
       <geometry>
-        <box size="0.01 0.01 0.01" />
+        <box size="1.0 1.0 0.001" />
       </geometry>
     </collision>
@@ -61,4 +56,13 @@
       <interface:position name="p3d_r_gripper_palm_position"/>
     </controller:gazebo_ros_p3d>
+    <!-- fixed joint to the world for simulation -->
+    <joint:hinge name="base_fixed_joint">
+      <body1>world</body1>
+      <body2>base_link</body2>
+      <anchor>base_link</anchor>
+      <lowStop>0</lowStop>
+      <highStop>0</highStop>
+      <axis>0 0 1</axis>
+    </joint:hinge>
   </gazebo>
 </robot>

File: pr2_description/robots/pr2.urdf.xacro (robot description, xacro)
@@ -38,7 +38,5 @@
        the origin block defines where the component is w.r.t its parent (in this case the parent
        is the world frame). For more, see http://www.ros.org/wiki/xacro -->
-  <xacro:pr2_base_v0 name="base" >
-    <origin xyz="0 0 0.051" rpy="0 0 0" /> <!-- 5.1cm is the height of the base when wheels contact ground -->
-  </xacro:pr2_base_v0>
+  <xacro:pr2_base_v0 name="base"/>
   <xacro:pr2_torso_v0 name="torso_lift" parent="base_link">
     <origin xyz="-0.05 0 0.739675" rpy="0 0 0" />

File: pr2_description/urdf/base_v0/base.urdf.xacro (robot description, xacro)
@@ -120,10 +120,5 @@
   </xacro:macro>
   <!-- The xacro macro xacro:pr2_base contains: base, casters and wheels -->
-  <xacro:macro name="pr2_base_v0" params="name *origin">
-    <joint name="${name}_joint" type="planar">
-      <insert_block name="origin" />
-      <parent link="world"/>
-      <child link="${name}_link" />
-    </joint>
+  <xacro:macro name="pr2_base_v0" params="name">
     <link name="${name}_link">
       <inertial>
