Commit message: reset collision geom for torso to the shoulder plate

File: pr2_defs/defs/body/body_defs.urdf.xacro (robot description, xacro)
@@ -20,4 +20,5 @@
     <link name="${name}_link">
       <inertial>
+        <!-- from function 090224_link_data.xls -->
         <mass value="36.248046" />
         <origin xyz="-0.1 0 -0.0885" />
@@ -33,7 +34,8 @@
       </visual>
       <collision name="${name}_collision">
-        <origin xyz="-0.1 0 -0.0885" rpy="0 0 0" />
+        <origin xyz="0 0 0.16" rpy="0 0 0" />
         <geometry name="${name}_collision_geom">
-          <box size="0.30 0.620 0.823" />
+          <!-- arbitrarily chosen collision box by JH, torso collision is not important for now -->
+          <box size="0.30 0.620 0.02" />
         </geometry>
       </collision>
