Commit message: minor fix.

File: pr2_description/urdf/sensors/prosilica_gc2450_camera.urdf.xacro (robot description, xacro)
@@ -20,7 +20,8 @@
       </inertial>
       <visual>
-        <origin xyz="0 0 0" rpy="0 0 0" />
+        <!-- bogus values for visual aesthetics -->
+        <origin xyz="-0.02 0 0" rpy="0 0 0"/>
         <geometry>
-          <box size="0.01 0.01 0.01" />
+          <box size="0.04 0.04 0.04" />
         </geometry>
         <material name="Blue" />
@@ -48,7 +49,8 @@
       </inertial>
       <visual>
-        <origin xyz="0 0 0" rpy="0 0 0"/>
+        <!-- bogus values for visual aesthetics -->
+        <origin xyz="0 0 0" rpy="0 0 ${M_PI/2}" />
         <geometry>
-          <box size="0.01 0.01 0.01" />
+          <cylinder radius="0.02" length="0.05" />
         </geometry>
         <material name="Blue" />
