Commit message: typo.

File: pr2_description/urdf/sensors/hokuyo_lx30_laser.gazebo.xacro (robot description, xacro)
@@ -4,5 +4,5 @@
        xmlns:interface="http://playerstage.sourceforge.net/gazebo/xmlschema/#interface"
        xmlns:xacro="http://ros.org/wiki/xacro">
-  <xacro:macro name="hokuyo_lx30_laser_gazebo_v0" params="name gazebo_ros_topic update_rate">
+  <xacro:macro name="hokuyo_lx30_laser_gazebo_v0" params="name ros_topic update_rate">
     <gazebo reference="${name}_link">
       <sensor:ray name="${name}">
@@ -22,5 +22,5 @@
           <alwaysOn>true</alwaysOn>
           <updateRate>${update_rate}</updateRate>
-          <topicName>${gazebo_ros_topic}</topicName>
+          <topicName>${ros_topic}</topicName>
           <frameName>${name}_link</frameName>
           <interface:laser name="gazebo_ros_${name}_iface" />
