Commit message: * make camera collision geometry 0-sized.  * fix frame_id of stereo cameras: [narrow|wide]_stere_optical_frame.

File: pr2_description/urdf/sensors/stereo_camera.urdf.xacro (robot description, xacro)
@@ -62,5 +62,5 @@
         <origin xyz="0 0 0" rpy="0 0 0" />
         <geometry>
-          <box size="0.01 0.01 0.01" />
+          <box size="0.001 0.001 0.001" />
         </geometry>
         <material name="Blue" />
@@ -69,5 +69,5 @@
         <origin xyz="0 0 0" rpy="0 0 0" />
         <geometry>
-          <box size="0.01 0.01 0.01" />
+          <box size="0.0 0.0 0.0" />
         </geometry>
       </collision>
@@ -77,5 +77,5 @@
                             camera_info_topic_name="${name}/left/camera_info" parent="${name}_optical_frame"
                             hfov="${hfov}" focal_length="${focal_length}"
-                            frame_id="${name}_l_stereo_camera_frame" hack_baseline="0"
+                            frame_id="${name}_optical_frame" hack_baseline="0"
                             image_width="${image_width}" image_height="${image_height}">
       <origin xyz="0 0 0" rpy="0 ${-M_PI/2} ${M_PI/2}" />
@@ -85,5 +85,5 @@
                             camera_info_topic_name="${name}/right/camera_info" parent="${name}_l_stereo_camera_frame"
                             hfov="${hfov}" focal_length="${focal_length}"
-                            frame_id="${name}_l_stereo_camera_frame" hack_baseline="${stereo_dy}"
+                            frame_id="${name}_optical_frame" hack_baseline="${stereo_dy}"
                             image_width="${image_width}" image_height="${image_height}">
       <origin xyz="${stereo_dx} ${stereo_dy} ${stereo_dz}" rpy="${stereo_rx} ${stereo_ry} ${stereo_rz}" />

Commit message: removing inertial, visual and collision for stereo and wge100 camera optical frames.

File: pr2_description/urdf/sensors/stereo_camera.urdf.xacro (robot description, xacro)
@@ -51,26 +51,5 @@
       <child link="${name}_optical_frame"/>
     </joint>
-    <link name="${name}_optical_frame" type="camera">
-      <inertial>
-        <mass value="0.01" />
-        <origin xyz="0 0 0" rpy="0 0 0" />
-        <inertia ixx="0.001"  ixy="0.0"  ixz="0.0"
-                 iyy="0.001"  iyz="0.0"
-                 izz="0.001" />
-      </inertial>
-      <visual>
-        <origin xyz="0 0 0" rpy="0 0 0" />
-        <geometry>
-          <box size="0.001 0.001 0.001" />
-        </geometry>
-        <material name="Blue" />
-      </visual>
-      <collision>
-        <origin xyz="0 0 0" rpy="0 0 0" />
-        <geometry>
-          <box size="0.0 0.0 0.0" />
-        </geometry>
-      </collision>
-    </link>
+    <link name="${name}_optical_frame" type="camera"/>
     <!-- stereo left camera -->
     <xacro:wge100_camera_v0 name="${name}_l_stereo_camera" image_format="${image_format}" image_topic_name="${name}/left/image_raw"

File: pr2_description/urdf/sensors/wge100_camera.urdf.xacro (robot description, xacro)
@@ -40,25 +40,5 @@
       <child link="${name}_optical_frame"/>
     </joint>
-    <link name="${name}_optical_frame">
-      <inertial>
-        <mass value="0.01" />
-        <origin xyz="0 0 0" />
-        <inertia ixx="0.001"  ixy="0.0"  ixz="0.0"
-                 iyy="0.001"  iyz="0.0"
-                 izz="0.001" />
-      </inertial>
-      <visual>
-        <origin xyz="0 0 0" rpy="0 0 0"/>
-        <geometry>
-          <box size="0.01 0.01 0.01" />
-        </geometry>
-      </visual>
-      <collision>
-        <origin xyz="0 0 0" rpy="0 0 0"/>
-        <geometry>
-          <box size="0.01 0.01 0.01" />
-        </geometry>
-      </collision>
-    </link>
+    <link name="${name}_optical_frame"/>
     <!-- extensions -->
     <xacro:wge100_camera_gazebo_v0 name="${name}" image_format="${image_format}" image_topic_name="${image_topic_name}"
