Commit message: HACK for stereo_image_proc making prosilica distortion 1e-8 for now.
removed material for optical frame.

File: pr2_description/urdf/sensors/prosilica_gc2450_camera.gazebo.xacro (robot description, xacro)
@@ -26,9 +26,9 @@
         <Cy>1025.5</Cy>
         <focal_length>2955</focal_length> <!-- image_width / (2*tan(hfov_radian /2)) -->
-        <distortion_k1>0</distortion_k1>
-        <distortion_k2>0</distortion_k2>
-        <distortion_k3>0</distortion_k3>
-        <distortion_t1>0</distortion_t1>
-        <distortion_t2>0</distortion_t2>
+        <distortion_k1>0.00000001</distortion_k1>
+        <distortion_k2>0.00000001</distortion_k2>
+        <distortion_k3>0.00000001</distortion_k3>
+        <distortion_t1>0.00000001</distortion_t1>
+        <distortion_t2>0.00000001</distortion_t2>
         <interface:camera name="${name}_iface" />
       </controller:gazebo_ros_prosilica>
@@ -36,7 +36,4 @@
     <material value="PR2/Blue" />
   </gazebo>
-  <gazebo reference="${name}_optical_frame">
-    <material value="PR2/Blue" />
-  </gazebo>
 </xacro:macro>
 </root>

Commit message: fix stereo simulation gazebo extension parent/child link error.

File: pr2_description/urdf/sensors/prosilica_gc2450_camera.gazebo.xacro (robot description, xacro)
@@ -16,10 +16,8 @@
         <alwaysOn>true</alwaysOn>
         <updateRate>20.0</updateRate>
-        <camInfoTopicName>/prosilica/cam_info</camInfoTopicName>
-        <imageTopicName>/prosilica/image</imageTopicName>
-        <imageRectTopicName>/prosilica/image_rect</imageRectTopicName>
-        <camInfoServiceName>/prosilica/cam_info_service</camInfoServiceName>
-        <pollServiceName>/prosilica/poll</pollServiceName>
-        <frameName>hight_def_optical_frame</frameName>
+        <imageTopicName>/prosilica/image_raw</imageTopicName>
+        <cameraInfoTopicName>/prosilica/camera_info</cameraInfoTopicName>
+        <pollServiceName>/prosilica/request_image</pollServiceName>
+        <frameName>${name}_frame</frameName>
         <CxPrime>1224.5</CxPrime>
         <Cx>1224.5</Cx>

File: pr2_description/urdf/sensors/stereo_camera.urdf.xacro (robot description, xacro)
@@ -54,9 +54,9 @@
     <!-- stereo left camera -->
     <xacro:wge100_camera_v0 name="${name}_l_stereo_camera" image_format="${image_format}" image_topic_name="${name}/left/image_raw"
-                            camera_info_topic_name="${name}/left/camera_info" parent="${name}_optical_frame"
+                            camera_info_topic_name="${name}/left/camera_info" parent="${name}_link"
                             hfov="${hfov}" focal_length="${focal_length}"
                             frame_id="${name}_optical_frame" hack_baseline="0"
                             image_width="${image_width}" image_height="${image_height}">
-      <origin xyz="0 0 0" rpy="0 ${-M_PI/2} ${M_PI/2}" />
+      <origin xyz="0 0 0" rpy="0 0 0" />
     </xacro:wge100_camera_v0>
     <!-- stereo right camera -->
