Commit message: adding link for imu.

File: pr2_description/urdf/sensors/microstrain_3dmgx2_imu.gazebo.xacro (robot description, xacro)
@@ -3,6 +3,6 @@
        xmlns:interface="http://playerstage.sourceforge.net/gazebo/xmlschema/#interface"
        xmlns:xacro="http://ros.org/wiki/xacro">
-  <xacro:macro name="microstrain_3dmgx2_imu_gazebo_v0" params="name ros_topic deprecated_ros_topic update_rate">
-    <gazebo reference="${name}_link">
+  <xacro:macro name="microstrain_3dmgx2_imu_gazebo_v0" params="name ros_topic update_rate">
+    <gazebo>
       <controller:gazebo_ros_imu name="imu_controller" plugin="libgazebo_ros_imu.so">
         <alwaysOn>true</alwaysOn>
@@ -10,5 +10,4 @@
         <bodyName>${name}_link</bodyName>
         <topicName>${ros_topic}</topicName>
-        <deprecatedTopicName>${deprecated_ros_topic}</deprecatedTopicName>
         <gaussianNoise>0.01</gaussianNoise>
         <frameName>map</frameName>

File: pr2_description/urdf/sensors/microstrain_3dmgx2_imu.urdf.xacro (robot description, xacro)
@@ -2,5 +2,5 @@
 <robot xmlns:xacro="http://ros.org/wiki/xacro">
   <include filename="$(find pr2_description)/urdf/sensors/microstrain_3dmgx2_imu.gazebo.xacro" />
-  <xacro:macro name="microstrain_3dmgx2_imu_v0" params="name parent *origin ros_topic deprecated_ros_topic update_rate">
+  <xacro:macro name="microstrain_3dmgx2_imu_v0" params="name parent *origin ros_topic update_rate">
     <joint name="${name}_joint" type="fixed">
       <axis xyz="0 1 0" />
@@ -9,5 +9,5 @@
       <child link="${name}_link"/>
     </joint>
-    <link name="${name}_link" type="laser">
+    <link name="${name}_link">
       <inertial>
         <mass value="0.001" />
@@ -30,5 +30,5 @@
     </link>
     <!-- gazebo extensions -->
-    <xacro:microstrain_3dmgx2_imu_gazebo_v0 name="${name}" ros_topic="${ros_topic}" deprecated_ros_topic="${deprecated_ros_topic}" update_rate="${update_rate}" />
+    <xacro:microstrain_3dmgx2_imu_gazebo_v0 name="${name}" ros_topic="${ros_topic}" update_rate="${update_rate}" />
   </xacro:macro>
 </robot>

File: pr2_description/urdf/torso_v0/torso.urdf.xacro (robot description, xacro)
@@ -6,4 +6,5 @@
   <include filename="$(find pr2_description)/urdf/torso_v0/torso.gazebo.xacro" />
   <include filename="$(find pr2_description)/urdf/torso_v0/torso.transmission.xacro" />
+  <include filename="$(find pr2_description)/urdf/sensors/microstrain_3dmgx2_imu.urdf.xacro" />
   <xacro:macro name="pr2_torso_v0" params="name parent *origin">
     <joint name="${name}_joint" type="prismatic">
@@ -12,5 +13,5 @@
       <safety_controller  k_velocity="400000" soft_lower_limit="${0.0+0.003}" soft_upper_limit="${0.31-0.005}" k_position="1000" />
       <calibration reference_position="0.00536" />
-      <dynamics damping="10.0" />
+      <dynamics damping="5000.0" />
       <insert_block name="origin" />
       <parent link="${parent}"/>
@@ -42,4 +43,8 @@
     <xacro:pr2_torso_gazebo_v0 name="${name}" />
     <xacro:pr2_torso_transmission_v0 name="${name}" />
+    <!-- imu -->
+    <xacro:microstrain_3dmgx2_imu_v0 name="imu" parent="${name}" ros_topic="imu_data" update_rate="100.0">
+        <origin xyz="0 0 0" rpy="0 0 0" />
+    </xacro:microstrain_3dmgx2_imu_v0>
   </xacro:macro>
 </robot>

Commit message: renaming imu/data to torso_lift_imu/data per ticket #3451

File: pr2_description/urdf/sensors/microstrain_3dmgx2_imu.gazebo.xacro (robot description, xacro)
@@ -3,5 +3,5 @@
        xmlns:interface="http://playerstage.sourceforge.net/gazebo/xmlschema/#interface"
        xmlns:xacro="http://ros.org/wiki/xacro">
-  <xacro:macro name="microstrain_3dmgx2_imu_gazebo_v0" params="name ros_topic update_rate">
+  <xacro:macro name="microstrain_3dmgx2_imu_gazebo_v0" params="name imu_topic update_rate">
     <gazebo>
       <controller:gazebo_ros_imu name="imu_controller" plugin="libgazebo_ros_imu.so">
@@ -9,5 +9,5 @@
         <updateRate>${update_rate}</updateRate>
         <bodyName>${name}_link</bodyName>
-        <topicName>${ros_topic}</topicName>
+        <topicName>${imu_topic}</topicName>
         <gaussianNoise>0.01</gaussianNoise>
         <frameName>map</frameName>

File: pr2_description/urdf/sensors/microstrain_3dmgx2_imu.urdf.xacro (robot description, xacro)
@@ -2,5 +2,5 @@
 <robot xmlns:xacro="http://ros.org/wiki/xacro">
   <include filename="$(find pr2_description)/urdf/sensors/microstrain_3dmgx2_imu.gazebo.xacro" />
-  <xacro:macro name="microstrain_3dmgx2_imu_v0" params="name parent *origin ros_topic update_rate">
+  <xacro:macro name="microstrain_3dmgx2_imu_v0" params="name parent *origin imu_topic update_rate">
     <joint name="${name}_joint" type="fixed">
       <axis xyz="0 1 0" />
@@ -30,5 +30,5 @@
     </link>
     <!-- gazebo extensions -->
-    <xacro:microstrain_3dmgx2_imu_gazebo_v0 name="${name}" ros_topic="${ros_topic}" update_rate="${update_rate}" />
+    <xacro:microstrain_3dmgx2_imu_gazebo_v0 name="${name}" imu_topic="${imu_topic}" update_rate="${update_rate}" />
   </xacro:macro>
 </robot>

File: pr2_description/urdf/torso_v0/torso.urdf.xacro (robot description, xacro)
@@ -14,5 +14,5 @@
       <!-- hold both reference_position and upper/lower for tick-tock, remove reference_positiion after verifying upper/lower works with calibration controllers.  if search velocity in pr2_calibration_controllers.yaml is +, the reference_position is rising, if - then it is falling -->
       <calibration reference_position="0.00536" falling="0.00536" />
-      <dynamics damping="5000.0" />
+      <dynamics damping="5000.0" /> <!-- strictly tuned for sim only right now -->
       <insert_block name="origin" />
       <parent link="${parent}"/>
@@ -45,5 +45,5 @@
     <xacro:pr2_torso_transmission_v0 name="${name}" />
     <!-- imu -->
-    <xacro:microstrain_3dmgx2_imu_v0 name="imu" parent="${name}" ros_topic="imu_data" update_rate="100.0">
+    <xacro:microstrain_3dmgx2_imu_v0 name="imu" parent="${name}" imu_topic="torso_lift_imu/data" update_rate="100.0">
         <origin xyz="-0.02977 -0.1497 0.164" rpy="0 0 0" />
     </xacro:microstrain_3dmgx2_imu_v0>
