Commit message: updated imu orientation

File: pr2_description/urdf/sensors/microstrain_3dmgx2_imu.urdf.xacro (robot description, xacro)
@@ -12,5 +12,5 @@
       <inertial>
         <mass value="0.001" />
-        <origin xyz="0 0 0" rpy="0 0 0" />
+        <origin xyz="0 0 0" rpy="0 ${M_PI} 0" />
         <inertia ixx="0.0001" ixy="0" ixz="0" iyy="0.000001" iyz="0" izz="0.0001" />
       </inertial>

Commit message: correction for imu orientation #3364

File: pr2_description/urdf/sensors/microstrain_3dmgx2_imu.urdf.xacro (robot description, xacro)
@@ -12,5 +12,5 @@
       <inertial>
         <mass value="0.001" />
-        <origin xyz="0 0 0" rpy="0 ${M_PI} 0" />
+        <origin xyz="0 0 0" rpy="0 0 0" />
         <inertia ixx="0.0001" ixy="0" ixz="0" iyy="0.000001" iyz="0" izz="0.0001" />
       </inertial>

File: pr2_description/urdf/torso_v0/torso.urdf.xacro (robot description, xacro)
@@ -46,5 +46,5 @@
     <!-- imu -->
     <xacro:microstrain_3dmgx2_imu_v0 name="imu" parent="${name}" imu_topic="torso_lift_imu/data" update_rate="100.0" stdev="0.00017" >
-        <origin xyz="-0.02977 -0.1497 0.164" rpy="0 0 0" />
+        <origin xyz="-0.02977 -0.1497 0.164" rpy="0 ${M_PI} 0" />
     </xacro:microstrain_3dmgx2_imu_v0>
   </xacro:macro>
