Commit message: correction for kinect optical frame

File: pr2_description/urdf/sensors/kinect_camera.gazebo.xacro (robot description, xacro)
@@ -6,5 +6,5 @@
 <xacro:macro name="kinect_camera_gazebo_v0" params="name">
   <gazebo reference="${name}_frame">
-    <sensor:stereocamera name="${name}_sensor">
+    <sensor:camera name="${name}_frame_sensor">
       <imageFormat>R8G8B8</imageFormat>
       <imageSize>640 480</imageSize>
@@ -14,5 +14,5 @@
       <updateRate>20.0</updateRate>
       <baseline>0.2</baseline>
-      <controller:gazebo_ros_stereo_camera name="${name}_controller" plugin="libgazebo_ros_stereo_camera.so">
+      <controller:gazebo_ros_camera name="${name}_frame_controller" plugin="libgazebo_ros_camera.so">
         <alwaysOn>true</alwaysOn>
         <updateRate>20.0</updateRate>
@@ -20,5 +20,5 @@
         <pointCloudTopicName>/kinect_camera/points</pointCloudTopicName>
         <cameraInfoTopicName>/kinect_camera/camera_info</cameraInfoTopicName>
-        <frameName>${name}_frame</frameName>
+        <frameName>${name}_optical_frame</frameName>
         <distortion_k1>0.00000001</distortion_k1>
         <distortion_k2>0.00000001</distortion_k2>
@@ -26,7 +26,6 @@
         <distortion_t1>0.00000001</distortion_t1>
         <distortion_t2>0.00000001</distortion_t2>
-      </controller:gazebo_ros_stereo_camera>
-    </sensor:stereocamera>
-    <material value="Gazebo/Black" />
+      </controller:gazebo_ros_camera>
+    </sensor:camera>
   </gazebo>
 </xacro:macro>

File: pr2_description/urdf/sensors/kinect_camera.urdf.xacro (robot description, xacro)
@@ -32,5 +32,5 @@
       </collision>
     </link>
-    <joint name="${name}_optical_frame_joint" type="fixed">
+    <joint name="${name}_optical_joint" type="fixed">
       <origin xyz="${cal_kinect_x}            ${cal_kinect_y}         ${cal_kinect_z}"
                 rpy="${-M_PI/2+cal_kinect_roll} ${0.0+cal_kinect_pitch} ${-M_PI/2+cal_kinect_yaw}" />
@@ -40,5 +40,5 @@
     <link name="${name}_optical_frame"/>
     <!-- extensions -->
-    <xacro:kinect_camera_gazebo_v0 name="${name}"/>
+    <xacro:kinect_camera_gazebo_v0 name="${name}" />
   </xacro:macro>
 </root>

Commit message: move kinect center over to center on middle camera on the front plate.

File: pr2_description/urdf/sensors/kinect_camera.gazebo.xacro (robot description, xacro)
@@ -10,5 +10,5 @@
       <imageSize>640 480</imageSize>
       <hfov>60</hfov>
-      <nearClip>0.5</nearClip>
+      <nearClip>0.01</nearClip>
       <farClip>5</farClip>
       <updateRate>20.0</updateRate>
@@ -21,4 +21,5 @@
         <cameraInfoTopicName>/kinect_camera/camera_info</cameraInfoTopicName>
         <frameName>${name}_optical_frame</frameName>
+        <pointCloudCutoff>0.5</pointCloudCutoff>
         <distortion_k1>0.00000001</distortion_k1>
         <distortion_k2>0.00000001</distortion_k2>

File: pr2_description/urdf/sensors/kinect_camera.urdf.xacro (robot description, xacro)
@@ -20,5 +20,5 @@
       </inertial>
       <visual>
-        <origin xyz="0.0 0 0" rpy="0 0 0"/>
+        <origin xyz="0.0 0.012 0" rpy="0 0 0"/>
         <geometry>
           <mesh filename="package://pr2_description/meshes/kinect/kinect.dae" />
@@ -26,5 +26,5 @@
       </visual>
       <collision>
-        <origin xyz="0.0 0 0" rpy="0 0 0"/>
+        <origin xyz="0.0 0.012 0" rpy="0 0 0"/>
         <geometry>
           <mesh filename="package://pr2_description/meshes/kinect/kinect.dae" />
