Commit message: removing unnecessary collision and visual geometries for cameras.

File: pr2_description/urdf/sensors/head_sensor_package.urdf.xacro (robot description, xacro)
@@ -36,10 +36,4 @@
         <material name="Blue" />
       </visual>
-      <collision name="${name}_sensor_collision">
-        <origin xyz="0 0 0" rpy="0 0 0" />
-        <geometry>
-          <box size="0.01 0.01 0.01" />
-        </geometry>
-      </collision>
     </link>
     <!-- Prosilica Camera -->

File: pr2_description/urdf/sensors/hokuyo_lx30_laser.urdf.xacro (robot description, xacro)
@@ -18,17 +18,4 @@
         <inertia ixx="0.0001" ixy="0" ixz="0" iyy="0.000001" iyz="0" izz="0.0001" />
       </inertial>
-      <visual>
-        <origin xyz="0 0 0" rpy="0 0 0" />
-        <geometry>
-          <box size="0.001 0.001 0.001" />
-        </geometry>
-        <material name="Red" />
-      </visual>
-      <collision>
-        <origin xyz="0 0 0" rpy="0 0 0" />
-        <geometry>
-          <box size=".001 .001 .001" />
-        </geometry>
-      </collision>
     </link>
     <!-- gazebo extensions -->

File: pr2_description/urdf/sensors/microstrain_3dmgx2_imu.urdf.xacro (robot description, xacro)
@@ -15,17 +15,4 @@
         <inertia ixx="0.0001" ixy="0" ixz="0" iyy="0.000001" iyz="0" izz="0.0001" />
       </inertial>
-      <visual>
-        <origin xyz="0 0 0" rpy="0 0 0" />
-        <geometry>
-          <box size="0.001 0.001 0.001" />
-        </geometry>
-        <material name="Red" />
-      </visual>
-      <collision>
-        <origin xyz="0 0 0" rpy="0 0 0" />
-        <geometry>
-          <box size=".001 .001 .001" />
-        </geometry>
-      </collision>
     </link>
     <!-- gazebo extensions -->

File: pr2_description/urdf/sensors/projector_wg6802418.urdf.xacro (robot description, xacro)
@@ -27,10 +27,4 @@
         <material name="Blue" />
       </visual>
-      <collision>
-        <origin xyz="0 0 0" rpy="0 0 0"/>
-        <geometry>
-          <box size="0.01 0.01 0.01" />
-        </geometry>
-      </collision>
     </link>
     <joint name="${name}_child_frame_joint" type="fixed">
@@ -54,10 +48,4 @@
         <material name="Red" />
       </visual>
-      <collision>
-        <origin xyz="0 0 0" rpy="0 0 0"/>
-        <geometry>
-          <box size="0.01 0.01 0.01" />
-        </geometry>
-      </collision>
     </link>
     <!-- extensions -->

File: pr2_description/urdf/sensors/stereo_camera.urdf.xacro (robot description, xacro)
@@ -27,17 +27,4 @@
         <inertia ixx="0.01"  ixy="0"  ixz="0" iyy="0.01"  iyz="0"  izz="0.01" /> <!-- this inertia is made up for now. -->
       </inertial>
-      <visual>
-        <origin xyz="0 0 0" rpy="0 0 0" />
-        <geometry>
-          <box size="0.001 0.001 0.001" />
-        </geometry>
-        <material name="Blue" />
-      </visual>
-      <collision>
-        <origin xyz="0 0 0" rpy="0 0 0" />
-        <geometry>
-          <box size="0.001 0.001 0.001" />
-        </geometry>
-      </collision>
     </link>
     <!-- attach optical frame to the camera link -->

File: pr2_description/urdf/sensors/wge100_camera.urdf.xacro (robot description, xacro)
@@ -22,10 +22,4 @@
                  izz="0.001" />
       </inertial>
-      <visual>
-        <origin xyz="0 0 0" rpy="0 0 0" />
-        <geometry>
-          <box size="0.01 0.01 0.01" />
-        </geometry>
-      </visual>
     </link>
     <joint name="${name}_optical_frame_joint" type="fixed">

Commit message: updated 5mp prosilica focal point from s. stanford (called kowa from prosilica)

File: pr2_description/urdf/sensors/head_sensor_package.urdf.xacro (robot description, xacro)
@@ -39,7 +39,6 @@
     <!-- Prosilica Camera -->
     <xacro:prosilica_cam_v0 frame_name="${hd_frame_name}" camera_name="${hd_camera_name}" parent="${name}_link" >
-      <!-- Center of camera is 109mm right of center screw, 35mm up -->
-      <!-- Camera is slightly recessed from front, where is camera origin? Lens? -->
-      <origin xyz="0 -0.109 0.035" rpy="0 0 0" />
+      <!-- camera focal point update from S. Stanford (called Kowa from Prosilica) 2011-08-18 -->
+      <origin xyz="0.046457 -0.110 0.054600" rpy="0 0 0" />
     </xacro:prosilica_cam_v0>
     <!-- construct wide and narrow double stereo camera -->
