Commit message: fix kinect urdf (frame should not have children)

File: pr2_description/urdf/sensors/kinect_prosilica_camera.gazebo.xacro (robot description, xacro)
@@ -4,9 +4,37 @@
       xmlns:interface="http://playerstage.sourceforge.net/gazebo/xmlschema/#interface"
       xmlns:xacro="http://ros.org/wiki/xacro">
-<xacro:macro name="kinect_camera_gazebo_v0" params="link_name frame_name camera_name">
+<xacro:macro name="kinect_ir_gazebo_v0" params="link_name frame_name camera_name">
+  <gazebo reference="${link_name}">
+    <sensor:camera name="${name}_sensor">
+      <imageFormat>L8</imageFormat>
+      <imageSize>640 480</imageSize>
+      <hfov>57</hfov>
+      <nearClip>0.01</nearClip>
+      <farClip>5</farClip>
+      <updateRate>1.0</updateRate>
+      <baseline>0.2</baseline>
+      <controller:gazebo_ros_camera name="${link_name}_controller" plugin="libgazebo_ros_camera.so">
+        <alwaysOn>true</alwaysOn>
+        <updateRate>1.0</updateRate>
+        <imageTopicName>/${camera_name}/image_raw</imageTopicName>
+        <pointCloudTopicName>/${camera_name}/points</pointCloudTopicName>
+        <cameraInfoTopicName>/${camera_name}/camera_info</cameraInfoTopicName>
+        <frameName>${frame_name}</frameName>
+        <pointCloudCutoff>0.5</pointCloudCutoff>
+        <distortion_k1>0.00000001</distortion_k1>
+        <distortion_k2>0.00000001</distortion_k2>
+        <distortion_k3>0.00000001</distortion_k3>
+        <distortion_t1>0.00000001</distortion_t1>
+        <distortion_t2>0.00000001</distortion_t2>
+      </controller:gazebo_ros_camera>
+    </sensor:camera>
+    <material value="Gazebo/Red" />
+  </gazebo>
+</xacro:macro>
+<xacro:macro name="kinect_rgb_gazebo_v0" params="link_name frame_name camera_name">
   <gazebo reference="${link_name}">
     <sensor:camera name="${name}_sensor">
       <imageFormat>R8G8B8</imageFormat>
-      <imageSize>320 240</imageSize>
+      <imageSize>640 480</imageSize>
       <hfov>57</hfov>
       <nearClip>0.01</nearClip>

File: pr2_description/urdf/sensors/kinect_prosilica_camera.urdf.xacro (robot description, xacro)
@@ -43,18 +43,11 @@
                                    link_name="${name}_kinect_prosilica_link" />
     -->
-    <!-- kinect housing physical attachment -->
-    <joint name="${name}_kinect_joint" type="fixed">
+    <!-- kinect ir sensor physical attachment -->
+    <joint name="${name}_kinect_ir_joint" type="fixed">
       <origin xyz="-0.032267 0.0125 0.136453" rpy="0 0 0"/>
       <parent link="${name}_link"/>
-      <child link="${name}_kinect_frame"/>
+      <child link="${name}_kinect_ir_link"/>
     </joint>
-    <link name="${name}_kinect_frame"/>
-    <!-- kinect ir sensor physical attachment -->
-    <joint name="${name}_kinect_ir_frame_joint" type="fixed">
-      <origin xyz="0 0 0" rpy="0 0 0"/>
-      <parent link="${name}_kinect_frame"/>
-      <child link="${name}_kinect_ir_frame"/>
-    </joint>
-    <link name="${name}_kinect_ir_frame" >
+    <link name="${name}_kinect_ir_link">
       <inertial>
         <mass value="0.1" />
@@ -81,17 +74,17 @@
       <origin xyz="${cal_kinect_x}            ${cal_kinect_y}         ${cal_kinect_z}"
                 rpy="${-M_PI/2+cal_kinect_roll} ${0.0+cal_kinect_pitch} ${-M_PI/2+cal_kinect_yaw}" />
-      <parent link="${name}_kinect_ir_frame"/>
+      <parent link="${name}_kinect_ir_link"/>
       <child link="${name}_kinect_ir_optical_frame"/>
     </joint>
     <link name="${name}_kinect_ir_optical_frame"/>
     <!-- gazebo extensions -->
-    <xacro:kinect_camera_gazebo_v0 link_name="${name}_kinect_ir_link" frame_name="${name}_kinect_ir_optical_frame" camera_name="kinect_camera" />
+    <xacro:kinect_ir_gazebo_v0 link_name="${name}_kinect_ir_link" frame_name="${name}_kinect_ir_optical_frame" camera_name="kinect_ir" />
     <!-- kinect rgb sensor physical attachment -->
-    <joint name="${name}_kinect_rgb_frame_joint" type="fixed">
+    <joint name="${name}_kinect_rgb_joint" type="fixed">
       <origin xyz="0 -0.03 0" rpy="0 0 0"/>
-      <parent link="${name}_kinect_frame"/>
-      <child link="${name}_kinect_rgb_frame"/>
+      <parent link="${name}_kinect_ir_link"/>
+      <child link="${name}_kinect_rgb_link"/>
     </joint>
-    <link name="${name}_kinect_rgb_frame" >
+    <link name="${name}_kinect_rgb_link" >
       <inertial>
         <mass value="0.1" />
@@ -118,8 +111,10 @@
       <origin xyz="${cal_kinect_x}            ${cal_kinect_y}         ${cal_kinect_z}"
                 rpy="${-M_PI/2+cal_kinect_roll} ${0.0+cal_kinect_pitch} ${-M_PI/2+cal_kinect_yaw}" />
-      <parent link="${name}_kinect_rgb_frame"/>
+      <parent link="${name}_kinect_rgb_link"/>
       <child link="${name}_kinect_rgb_optical_frame"/>
     </joint>
     <link name="${name}_kinect_rgb_optical_frame"/>
+    <!-- gazebo extensions -->
+    <xacro:kinect_rgb_gazebo_v0 link_name="${name}_kinect_ir_link" frame_name="${name}_kinect_ir_optical_frame" camera_name="kinect_rgb" />
     <!-- prosilica sensor physical attachment -->
     <joint name="${name}_prosilica_joint" type="fixed">
