Commit message: remove bogus visuals for projector and prosilica

File: pr2_description/urdf/sensors/projector_wg6802418.urdf.xacro (robot description, xacro)
@@ -19,12 +19,4 @@
                  izz="0.001" />
       </inertial>
-      <visual>
-        <!-- bogus values for visual aesthetics -->
-        <origin xyz="-0.02 0 0" rpy="0 0 0"/>
-        <geometry>
-          <box size="0.04 0.04 0.04" />
-        </geometry>
-        <material name="Blue" />
-      </visual>
     </link>
     <joint name="${name}_child_frame_joint" type="fixed">
@@ -41,11 +33,4 @@
                  izz="0.001" />
       </inertial>
-      <visual>
-        <origin xyz="0 0 0" rpy="0 0 ${M_PI/2}" />
-        <geometry>
-          <cylinder radius="0.02" length="0.05" />
-        </geometry>
-        <material name="Red" />
-      </visual>
     </link>
     <!-- extensions -->

File: pr2_description/urdf/sensors/prosilica_gc2450_camera.urdf.xacro (robot description, xacro)
@@ -19,12 +19,4 @@
                  izz="0.001" />
       </inertial>
-      <visual>
-        <!-- bogus values for visual aesthetics -->
-        <origin xyz="-0.02 0 0" rpy="0 0 0"/>
-        <geometry>
-          <box size="0.04 0.04 0.04" />
-        </geometry>
-        <material name="Blue" />
-      </visual>
     </link>
     <joint name="${frame_name}_optical_frame_joint" type="fixed">
@@ -42,12 +34,4 @@
                  izz="0.001" />
       </inertial>
-      <visual>
-        <!-- bogus values for visual aesthetics -->
-        <origin xyz="0 0 0" rpy="0 0 ${M_PI/2}" />
-        <geometry>
-          <cylinder radius="0.02" length="0.05" />
-        </geometry>
-        <material name="Blue" />
-      </visual>
     </link>
     <!-- extensions -->
