Commit message: moving kinect meshes to a better location

File: pr2_description/urdf/sensors/kinect_camera.urdf.xacro (robot description, xacro)
@@ -22,5 +22,5 @@
         <origin xyz="0.0 0.012 0" rpy="0 0 0"/>
         <geometry>
-          <mesh filename="package://pr2_description/meshes/kinect/kinect.dae" />
+          <mesh filename="package://pr2_description/meshes/sensors/kinect_v0/kinect.dae" />
         </geometry>
       </visual>
@@ -28,5 +28,5 @@
         <origin xyz="0.0 0.012 0" rpy="0 0 0"/>
         <geometry>
-          <mesh filename="package://pr2_description/meshes/kinect/kinect.dae" />
+          <mesh filename="package://pr2_description/meshes/sensors/kinect_v0/kinect.dae" />
         </geometry>
       </collision>

Commit message: fix scale for kinect model mesh

File: pr2_description/urdf/sensors/kinect_camera.urdf.xacro (robot description, xacro)
@@ -22,5 +22,5 @@
         <origin xyz="0.0 0.012 0" rpy="0 0 0"/>
         <geometry>
-          <mesh filename="package://pr2_description/meshes/sensors/kinect_v0/kinect.dae" />
+          <mesh filename="package://pr2_description/meshes/sensors/kinect_v0/kinect.dae" scale="0.001 0.001 0.001" />
         </geometry>
       </visual>
@@ -28,5 +28,5 @@
         <origin xyz="0.0 0.012 0" rpy="0 0 0"/>
         <geometry>
-          <mesh filename="package://pr2_description/meshes/sensors/kinect_v0/kinect.dae" />
+          <mesh filename="package://pr2_description/meshes/sensors/kinect_v0/kinect.dae" scale="0.001 0.001 0.001" />
         </geometry>
       </collision>
