Commit message: adding offset between kinect ir and rgb frame, need to find the right value for the offset.

File: pr2_description/urdf/sensors/kinect_prosilica_camera.urdf.xacro (robot description, xacro)
@@ -5,4 +5,5 @@
       xmlns:xacro="http://ros.org/wiki/xacro">
   <include filename="$(find pr2_description)/urdf/sensors/kinect_prosilica_camera.gazebo.xacro" />
+  <property name="ir_depth_rgb_offset_y" value="0.01"/> <!-- FIXME: what is this offset? -->
   <!-- kinect and prosilica combo -->
   <xacro:macro name="kinect_prosilica_camera_swept_back_v0" params="name parent *origin">
@@ -72,5 +73,5 @@
     <!-- kinect ir sensor frame -->
     <joint name="${name}_kinect_ir_optical_frame_joint" type="fixed">
-      <origin xyz="${cal_kinect_x}            ${cal_kinect_y}         ${cal_kinect_z}"
+      <origin xyz="${cal_kinect_x}            ${cal_kinect_y + ir_depth_rgb_offset_y}         ${cal_kinect_z}"
                 rpy="${-M_PI/2+cal_kinect_roll} ${0.0+cal_kinect_pitch} ${-M_PI/2+cal_kinect_yaw}" />
       <parent link="${name}_kinect_ir_link"/>

Commit message: Changed mesh collision sizes for kinect2 apparatus.

File: pr2_description/urdf/sensors/kinect_prosilica_camera.urdf.xacro (robot description, xacro)
@@ -9,5 +9,5 @@
       <!-- <limit lower="0.1" upper="0.1" effort="10000" velocity="100.0"/> -->
       <!-- <insert_block name="origin" /> -->
-      <origin xyz="-0.228 -0.148 0.091" rpy="${M_PI/2} 0 ${M_PI/2}"/> <!-- 0.0905 -->
+      <origin xyz="-0.228 -0.148 0.091" rpy="${M_PI/2} 0 ${M_PI/2}"/>
       <parent link="${parent}"/>
       <child link="${name}_link"/>
@@ -59,5 +59,5 @@
         <origin xyz="0 0 0" rpy="0 0 0"/>
         <geometry>
-          <box size="0.15 0.08 0.06" />
+          <sphere radius="0.0005"/>
         </geometry>
       </collision>
@@ -168,5 +168,5 @@
         <origin xyz="0 0 0" rpy="0 0 0"/>
         <geometry>
-          <box size="0.25 0.043 0.067"/>
+          <sphere radius="0.0005"/>
         </geometry>
       </collision>
