Commit message: * stereo_camera.urdf.xacro: change inertia to round numbers.  previously copied from arm components incorrectly.  removed offset between camera_link and camera_optical_frame (should contain only two 90deg rotations to make z-forward).  per disc with vijay, add "gazebo" to names of wge100 cameras in double stereo, since we want to hide them as actual individual cameras to end users.  * stereo_camera.gazebo.xacro: minor color change  * double_stereo_camera.urdf.xacro: moved calibration offset and translational offset between _link and _optical_frame here, into pose transform from double_stereo_link to narrow/wide_stereo_link (ticket #3337).

File: pr2_description/urdf/sensors/double_stereo_camera.urdf.xacro (robot description, xacro)
@@ -6,4 +6,9 @@
   <include filename="$(find pr2_description)/urdf/sensors/double_stereo_camera.gazebo.xacro" />
   <include filename="$(find pr2_description)/urdf/sensors/stereo_camera.urdf.xacro" />
+  <property name="stereo_size_x" value="0.02" />
+  <property name="stereo_size_y" value="0.12" />
+  <property name="stereo_size_z" value="0.05" />
+  <property name="stereo_center_box_center_offset_x" value="-0.01" />
+  <property name="stereo_center_box_center_offset_z" value="0.025" />
   <!-- Made by Kevin for double stereo camera for PR-2 Beta. -->
   <!-- Needs calibration verification, and CAD check. -->
@@ -25,14 +30,14 @@
       <!-- Should probably get real visuals here at some point -->
       <visual>
-        <origin xyz="0 0 0" rpy="0 0 0" />
+        <origin xyz="${stereo_center_box_center_offset_x} 0 ${stereo_center_box_center_offset_z}" rpy="0 0 0" />
         <geometry>
-          <box size="0.01 0.01 0.01" />
+          <box size="${stereo_size_x} ${stereo_size_y} ${stereo_size_z}" />
         </geometry>
         <material name="Blue" />
       </visual>
       <collision>
-        <origin xyz="0 0 0" rpy="0 0 0" />
+        <origin xyz="${stereo_center_box_center_offset_x} 0 ${stereo_center_box_center_offset_z}" rpy="0 0 0" />
         <geometry>
-          <box size="0.01 0.01 0.01" />
+          <box size="${stereo_size_x} ${stereo_size_y} ${stereo_size_z}" />
         </geometry>
       </collision>
@@ -41,8 +46,8 @@
     <!-- 15mm offset from center needs check with CAD -->
     <xacro:stereo_camera_v0 parent="${name}_link" name="wide_stereo" focal_length="320" hfov="90" image_format="BAYER_BGGR8" image_width="640" image_height="480" >
-      <origin xyz="0 -0.015 0" rpy="0 0 0" />
+      <origin xyz="${cal_stereo_x} ${0.045+cal_stereo_y-0.015} ${0.0305+cal_stereo_z}" rpy="${cal_stereo_roll} ${cal_stereo_pitch} ${cal_stereo_yaw}" />
     </xacro:stereo_camera_v0>
     <xacro:stereo_camera_v0 parent="${name}_link" name="narrow_stereo" focal_length="772.55" hfov="45" image_format="L8" image_width="640" image_height="480" >
-      <origin xyz="0 0.015 0" rpy="0 0 0" />
+      <origin xyz="${cal_stereo_x} ${0.045+cal_stereo_y+0.015} ${0.0305+cal_stereo_z}" rpy="${cal_stereo_roll} ${cal_stereo_pitch} ${cal_stereo_yaw}" />
     </xacro:stereo_camera_v0>
     <!-- extensions -->

File: pr2_description/urdf/sensors/stereo_camera.gazebo.xacro (robot description, xacro)
@@ -11,5 +11,5 @@
     </gazebo>
     <gazebo reference="${name}_optical_frame">
-      <material value="PR2/Blue" />
+      <material value="PR2/Green" />
       <turnGravityOff value="true" />
     </gazebo>

File: pr2_description/urdf/sensors/stereo_camera.urdf.xacro (robot description, xacro)
@@ -7,9 +7,4 @@
   <include filename="$(find pr2_description)/urdf/sensors/wge100_camera.urdf.xacro" />
   <include filename="$(find pr2_description)/urdf/sensors/stereo_camera.gazebo.xacro" />
-  <property name="stereo_size_x" value="0.005" />
-  <property name="stereo_size_y" value="0.010" />
-  <property name="stereo_size_z" value="0.005" />
-  <property name="stereo_center_box_center_offset_x" value="0.00" />
-  <property name="stereo_center_box_center_offset_z" value="0.05" />
   <property name="stereo_dx" value="0.00" />
   <property name="stereo_dy" value="-0.09" /> <!-- +y to the left -->
@@ -25,33 +20,35 @@
       <child link="${name}_link"/>
     </joint>
+    <!-- camera link is at center of the optical frame, but in x-forward notation -->
     <link name="${name}_link">
       <inertial>
         <mass value="0.1" />
         <origin xyz="0 0 0" rpy="0 0 0" />
-        <inertia ixx="0.00482611007"  ixy="-0.000144683999"  ixz="0.000110076136"
-                 iyy="0.005218991412"  iyz="-0.000314239509"  izz="0.008618784925" />
+        <inertia ixx="0.01"  ixy="0"  ixz="0" iyy="0.01"  iyz="0"  izz="0.01" /> <!-- this inertia is made up for now. -->
       </inertial>
       <visual>
-        <origin xyz="${stereo_center_box_center_offset_x} 0 ${stereo_center_box_center_offset_z}" rpy="0 0 0" />
+        <origin xyz="0 0 0" rpy="0 0 0" />
         <geometry>
-          <box size="${stereo_size_x} ${stereo_size_y} ${stereo_size_z}" />
+          <box size="0.001 0.001 0.001" />
         </geometry>
         <material name="Blue" />
       </visual>
       <collision>
-        <origin xyz="${stereo_center_box_center_offset_x} 0 ${stereo_center_box_center_offset_z}" rpy="0 0 0" />
+        <origin xyz="0 0 0" rpy="0 0 0" />
         <geometry>
-          <box size="${stereo_size_x} ${stereo_size_y} ${stereo_size_z}" />
+          <box size="0.001 0.001 0.001" />
         </geometry>
       </collision>
     </link>
+    <!-- attach optical frame to the camera link -->
     <joint name="${name}_optical_frame_joint" type="fixed">
-      <origin xyz="${cal_stereo_x}            ${0.045+cal_stereo_y}   ${.0305+cal_stereo_z}" rpy="${-M_PI/2+cal_stereo_roll} ${0.0+cal_stereo_pitch} ${-M_PI/2+cal_stereo_yaw}" />
+      <origin xyz="0 0 0" rpy="${-M_PI/2} 0.0 ${-M_PI/2}" /> <!-- rotate frame from x-forward to z-forward camera coords -->
       <parent link="${name}_link"/>
       <child link="${name}_optical_frame"/>
     </joint>
+    <!-- optical frame for the stereo camera, with z-forward notation, this is the frame stereo camera images users should refer to -->
     <link name="${name}_optical_frame" type="camera"/>
     <!-- stereo left camera -->
-    <xacro:wge100_camera_v0 name="${name}_l_stereo_camera" image_format="${image_format}" image_topic_name="${name}/left/image_raw"
+    <xacro:wge100_camera_v0 name="${name}_gazebo_l_stereo_camera" image_format="${image_format}" image_topic_name="${name}/left/image_raw"
                             camera_info_topic_name="${name}/left/camera_info" parent="${name}_link"
                             hfov="${hfov}" focal_length="${focal_length}"
@@ -61,6 +58,6 @@
     </xacro:wge100_camera_v0>
     <!-- stereo right camera -->
-    <xacro:wge100_camera_v0 name="${name}_r_stereo_camera" image_format="${image_format}" image_topic_name="${name}/right/image_raw"
-                            camera_info_topic_name="${name}/right/camera_info" parent="${name}_l_stereo_camera_frame"
+    <xacro:wge100_camera_v0 name="${name}_gazebo_r_stereo_camera" image_format="${image_format}" image_topic_name="${name}/right/image_raw"
+                            camera_info_topic_name="${name}/right/camera_info" parent="${name}_gazebo_l_stereo_camera_frame"
                             hfov="${hfov}" focal_length="${focal_length}"
                             frame_id="${name}_optical_frame" hack_baseline="${-stereo_dy}"

Commit message: Removing old/unused calibration offset variables

File: pr2_description/urdf/sensors/double_stereo_camera.urdf.xacro (robot description, xacro)
@@ -46,8 +46,8 @@
     <!-- 15mm offset from center needs check with CAD -->
     <xacro:stereo_camera_v0 parent="${name}_link" name="wide_stereo" focal_length="320" hfov="90" image_format="BAYER_BGGR8" image_width="640" image_height="480" >
-      <origin xyz="${cal_stereo_x} ${0.045+cal_stereo_y-0.015} ${0.0305+cal_stereo_z}" rpy="${cal_stereo_roll} ${cal_stereo_pitch} ${cal_stereo_yaw}" />
+      <origin xyz="0.0 ${0.045-0.015} 0.0305" rpy="0.0   0.0   0.0" />
     </xacro:stereo_camera_v0>
     <xacro:stereo_camera_v0 parent="${name}_link" name="narrow_stereo" focal_length="772.55" hfov="45" image_format="L8" image_width="640" image_height="480" >
-      <origin xyz="${cal_stereo_x} ${0.045+cal_stereo_y+0.015} ${0.0305+cal_stereo_z}" rpy="${cal_stereo_roll} ${cal_stereo_pitch} ${cal_stereo_yaw}" />
+      <origin xyz="0.0 ${0.045+0.015} 0.0305" rpy="0.0   0.0   0.0" />
     </xacro:stereo_camera_v0>
     <!-- extensions -->

Commit message: removing collision geometries per #4631, given camera sensor bodies have no child links

File: pr2_description/urdf/sensors/double_stereo_camera.urdf.xacro (robot description, xacro)
@@ -36,10 +36,4 @@
         <material name="Blue" />
       </visual>
-      <collision>
-        <origin xyz="${stereo_center_box_center_offset_x} 0 ${stereo_center_box_center_offset_z}" rpy="0 0 0" />
-        <geometry>
-          <box size="${stereo_size_x} ${stereo_size_y} ${stereo_size_z}" />
-        </geometry>
-      </collision>
     </link>
     <!-- Wide camera is on robot right (hca1), narrow on left (hca2)? -->

File: pr2_description/urdf/sensors/prosilica_gc2450_camera.urdf.xacro (robot description, xacro)
@@ -27,10 +27,4 @@
         <material name="Blue" />
       </visual>
-      <collision>
-        <origin xyz="0 0 0" rpy="0 0 0"/>
-        <geometry>
-          <box size="0.01 0.01 0.01" />
-        </geometry>
-      </collision>
     </link>
     <joint name="${name}_optical_frame_joint" type="fixed">
@@ -56,10 +50,4 @@
         <material name="Blue" />
       </visual>
-      <collision>
-        <origin xyz="0 0 0" rpy="0 0 0"/>
-        <geometry>
-          <box size="0.01 0.01 0.01" />
-        </geometry>
-      </collision>
     </link>
     <!-- extensions -->

File: pr2_description/urdf/sensors/wge100_camera.urdf.xacro (robot description, xacro)
@@ -28,10 +28,4 @@
         </geometry>
       </visual>
-      <collision>
-        <origin xyz="0 0 0" rpy="0 0 0"/>
-        <geometry>
-          <box size="0.01 0.01 0.01" />
-        </geometry>
-      </collision>
     </link>
     <joint name="${name}_optical_frame_joint" type="fixed">

Commit message: remove useless visual geometry
MoveIt master recently changed its policy w.r.t. empty collision geometries.
The current version complains:

ros.moveit_core.robot_model.empty_collision_geometry: Link sensor_mount_link has visual geometry but no collision geometry. Collision geometry will be left empty. Fix your URDF file by explicitly specifying collision
geometry.
ros.moveit_core.robot_model.empty_collision_geometry: Link double_stereo_link has visual geometry but no collision geometry. Collision geometry will be left empty. Fix your URDF file by explicitly specifying collision geometry.

As these visuals are not helpful and do not add anything to the description, I just remove them.

File: pr2_description/urdf/sensors/double_stereo_camera.urdf.xacro (robot description, xacro)
@@ -25,12 +25,4 @@
                  iyy="0.001" iyz="0.0" izz="0.01" />
       </inertial>
-      <!-- Should probably get real visuals here at some point -->
-      <visual>
-        <origin xyz="${stereo_center_box_center_offset_x} 0 ${stereo_center_box_center_offset_z}" rpy="0 0 0" />
-        <geometry>
-          <box size="${stereo_size_x} ${stereo_size_y} ${stereo_size_z}" />
-        </geometry>
-        <material name="Blue" />
-      </visual>
     </link>
     <!-- Wide camera is on robot right (hca1), narrow on left (hca2)? -->

File: pr2_description/urdf/sensors/head_sensor_package.urdf.xacro (robot description, xacro)
@@ -25,12 +25,4 @@
                  iyy="0.001" iyz="0.0" izz="0.01" />
       </inertial>
-      <!-- Should probably get real visuals here at some point -->
-      <visual>
-        <origin xyz="0 0 0" rpy="0 0 0" />
-        <geometry>
-          <box size="0.01 0.01 0.01" />
-        </geometry>
-        <material name="Blue" />
-      </visual>
     </link>
     <!-- Prosilica Camera -->
