Commit message: Changed name of link from head_mount_frame to head_mount_kinect2_frame to keep naming scheme consistent

File: pr2_description/urdf/sensors/kinect2.urdf.xacro (robot description, xacro)
@@ -5,10 +5,10 @@
   <!-- Kinect2 and mount assembly -->
   <xacro:macro name="kinect2_v0" params="name parent *origin">
-    <joint name="${name}_joint" type="fixed">
+    <joint name="${name}_kinect2_joint" type="fixed">
       <insert_block name="origin" />
       <parent link="${parent}"/>
-      <child link="${name}_link"/>
+      <child link="${name}_kinect2_link"/>
     </joint>
-    <link name="${name}_link">
+    <link name="${name}_kinect2_link">
       <inertial>
         <mass value="0.1"/>
@@ -37,5 +37,5 @@
     <joint name="${name}_kinect2_ir_joint" type="fixed">
       <origin xyz="-0.032267 -0.0475 0.155" rpy="0 0 0"/>
-      <parent link="${name}_link"/>
+      <parent link="${name}_kinect2_link"/>
       <child link="${name}_kinect2_ir_link"/>
     </joint>

Commit message: use collada to store kinect mesh
The STL produced the following warning with RViz:

[ WARN]: The STL file 'package://pr2_description/meshes/sensors/kinect2_v0/kinect2_assembly.STL' is malformed. It starts with the word 'solid', indicating that it's an ASCII STL file, but it does not contain the word 'endsolid' so it is either a malformed ASCII STL file or it is actually a binary STL file. Trying to interpret it as a binary STL file instead.

File: pr2_description/urdf/sensors/kinect2.urdf.xacro (robot description, xacro)
@@ -21,5 +21,5 @@
         <origin xyz="-0.102 -0.148 0" rpy="0 0 0"/>
         <geometry>
-          <mesh filename="package://pr2_description/meshes/sensors/kinect2_v0/kinect2_assembly.STL" scale="0.001 0.001 0.001" />
+          <mesh filename="package://pr2_description/meshes/sensors/kinect2_v0/kinect2_assembly.dae" scale="0.001 0.001 0.001" />
         </geometry>
         <material name="gray">

Commit message: provide bounding box for kinect2 spoiler
to enable *some* collision checking.

It was not enabled at all before and it's barely in the workspace of the arms at all (without tool use).
So a rough bounding box is fine.

File: pr2_description/urdf/sensors/kinect2.urdf.xacro (robot description, xacro)
@@ -28,7 +28,7 @@
       </visual>
       <collision>
-        <origin xyz="0 0 0" rpy="0 0 0"/>
+        <origin xyz="-0.042 0 0.1" rpy="0 0 0"/>
         <geometry>
-          <sphere radius="0.0005"/>
+          <box size="0.12 0.3 0.2"/>
         </geometry>
       </collision>

Commit message: remove auxiliary shapes from kinect2 links
If one wants to see the frames, just enable the frame in RViz.
There is no need whatsoever to keep these in the description.

File: pr2_description/urdf/sensors/kinect2.urdf.xacro (robot description, xacro)
@@ -48,16 +48,4 @@
                  izz="0.01" />
       </inertial>
-      <visual>
-        <origin xyz="0.0 0.0 0" rpy="0 0 0"/>
-        <geometry>
-          <sphere radius="0.0005"/>
-        </geometry>
-      </visual>
-      <collision>
-        <origin xyz="0.0 0.0 0" rpy="0 0 0"/>
-        <geometry>
-          <sphere radius="0.0005"/>
-        </geometry>
-      </collision>
     </link>
     <!-- kinect2 ir sensor frame -->
@@ -85,17 +73,4 @@
                  izz="0.01" />
       </inertial>
-      <visual>
-        <origin xyz="${cal_kinect_x}            ${cal_kinect_y}                 ${cal_kinect_z}"
-                rpy="${-M_PI/2+cal_kinect_roll} ${0.0+cal_kinect_pitch}         ${-M_PI/2+cal_kinect_yaw}" />
-        <geometry>
-          <sphere radius="0.0005"/>
-        </geometry>
-      </visual>
-      <collision>
-        <origin xyz="0.0 0.0 0" rpy="0 0 0"/>
-        <geometry>
-          <sphere radius="0.0005"/>
-        </geometry>
-      </collision>
     </link>
     <!-- kinect2 rgb sensor frame -->
