Commit message: Adding laser tilt limits from Fx for laser tilt. Transmission was verified empirically on A2 unit by moving it to limit stops. New ratio is 6.05:1

File: pr2_description/urdf/tilting_laser_v0/tilting_laser.transmission.xacro (robot description, xacro)
@@ -8,5 +8,5 @@
       <actuator name="${name}_mount_motor" />
       <joint name="${name}_mount_joint" />
-      <mechanicalReduction>6.0</mechanicalReduction>
+      <mechanicalReduction>6.05</mechanicalReduction>
     </transmission>
   </xacro:macro>

File: pr2_description/urdf/tilting_laser_v0/tilting_laser.urdf.xacro (robot description, xacro)
@@ -10,6 +10,6 @@
     <joint name="${name}_mount_joint" type="revolute">
       <axis xyz="0 1 0" />
-      <limit lower="-0.7854" upper="1.48353" effort="0.5292" velocity="10.0" />
-      <safety_controller k_position="100" k_velocity="0.05" soft_lower_limit="${-0.785+0.0}" soft_upper_limit="${1.57-0.0}" />
+      <limit lower="-0.7854" upper="1.48353" effort="0.65" velocity="10.0" />
+      <safety_controller k_position="100" k_velocity="0.05" soft_lower_limit="${-0.7854+0.05}" soft_upper_limit="${1.48353-0.05}" />
       <calibration reference_position="${laser_calib_ref}" />
       <dynamics damping="0.008" />
