Commit message: cleanup meshes in pr2_description.  new beta meshes.  delete unused meshes.  renaming shoulder_yaw to shoulder_pan.  renaming hok_tilt.stl to tilting_hokuyo.stl

File: pr2_description/urdf/tilting_laser_v0/tilting_laser.urdf.xacro (robot description, xacro)
@@ -30,5 +30,5 @@
         <origin xyz="0 0 0" rpy="0 0 0" />
         <geometry>
-          <mesh filename="package://pr2_description/meshes/tilting_laser_v0/hok_tilt.stl" />
+          <mesh filename="package://pr2_description/meshes/tilting_laser_v0/tilting_hokuyo.stl" />
         </geometry>
         <material name="Red" />

File: pr2_description/urdf/torso_v0/torso.urdf.xacro (robot description, xacro)
@@ -29,5 +29,5 @@
         <origin xyz="0 0 0" rpy="0 0 0" />
         <geometry>
-          <mesh filename="package://pr2_description/meshes/torso_v0/torso_lift_2k.stl"  />
+          <mesh filename="package://pr2_description/meshes/torso_v0/torso_lift.stl"  />
         </geometry>
         <material name="Grey2" />

Commit message: #5028 update mass / inertia values from 090224_link_data.xls.

File: pr2_description/urdf/tilting_laser_v0/tilting_laser.urdf.xacro (robot description, xacro)
@@ -20,9 +20,9 @@
     <link name="${name}_mount_link">
       <inertial>
-        <mass value="0.05" />
-        <origin xyz="-0.03 0 -0.03" rpy="0 0 0" />
-        <inertia ixx="0.0001" ixy="0" ixz="0"
-                 iyy="0.00001" iyz="0"
-                 izz="0.0001" />
+        <mass value="0.591" />
+        <origin xyz="-0.001136 0.00167 -0.00713" rpy="0 0 0" />
+        <inertia ixx="0.001195273" ixy="0.000023087" ixz="0.000037467"
+                 iyy="0.001083956" iyz="0.000034906"
+                 izz="0.000795014" />
       </inertial>
       <visual>
