Commit message: Changed motor name to remove _v0 suffix for caster. Corrected typo

File: pr2_description/urdf/base_v0/base.transmission.xacro (robot description, xacro)
@@ -7,14 +7,14 @@
   <!-- Alpha 2.0 hardware                                   -->
   <!--                                                      -->
-  <xacro:macro name="pr2_wheel_transmission_v0" params="suffix parent reflect">
+  <xacro:macro name="pr2_wheel_transmission" params="suffix parent reflect">
     <transmission type="SimpleTransmission" name="${parent}_${suffix}_wheel_trans">
-      <actuator name="${parent}_${suffix}_wheel_motor_v0" />
+      <actuator name="${parent}_${suffix}_wheel_motor" />
       <joint name="${parent}_${suffix}_wheel_joint" />
       <mechanicalReduction>${-1 * reflect * 624/35 * 80/18}</mechanicalReduction>
     </transmission>
   </xacro:macro>
-  <xacro:macro name="pr2_caster_transmission_v0" params="suffix">
+  <xacro:macro name="pr2_caster_transmission" params="suffix">
     <transmission type="SimpleTransmission" name="${suffix}_caster_rotation_trans">
-      <actuator name="${suffix}_caster_rotation_motor_v0" />
+      <actuator name="${suffix}_caster_rotation_motor" />
       <joint name="${suffix}_caster_rotation_joint" />
       <mechanicalReduction>${624/35 * 80/18}</mechanicalReduction>

Commit message: Changes to Beta caster defs for reflection, tilting laser reflection, added separate 'robot' for caster hub

File: pr2_description/urdf/base_v0/base.transmission.xacro (robot description, xacro)
@@ -4,19 +4,18 @@
        xmlns:interface="http://playerstage.sourceforge.net/gazebo/xmlschema/#interface"
        xmlns:xacro="http://ros.org/wiki/xacro">
-  <!--                                                      -->
-  <!-- Alpha 2.0 hardware                                   -->
-  <!--                                                      -->
+  <!--  Caster wheel transmission   -->
   <xacro:macro name="pr2_wheel_transmission_v0" params="suffix parent reflect">
     <transmission type="SimpleTransmission" name="${parent}_${suffix}_wheel_trans">
       <actuator name="${parent}_${suffix}_wheel_motor" />
       <joint name="${parent}_${suffix}_wheel_joint" />
-      <mechanicalReduction>${-1 * reflect * 624/35 * 80/18}</mechanicalReduction>
+      <mechanicalReduction>${reflect * 624/35 * 80/18}</mechanicalReduction>
     </transmission>
   </xacro:macro>
+  <!-- Hub transmission only -->
   <xacro:macro name="pr2_caster_transmission_v0" params="suffix">
-    <transmission type="SimpleTransmission" name="${suffix}_caster_rotation_trans">
-      <actuator name="${suffix}_caster_rotation_motor" />
-      <joint name="${suffix}_caster_rotation_joint" />
-      <mechanicalReduction>${624/35 * 80/18}</mechanicalReduction>
+    <transmission type="SimpleTransmission" name="${suffix}_rotation_trans">
+      <actuator name="${suffix}_rotation_motor" />
+      <joint name="${suffix}_rotation_joint" />
+      <mechanicalReduction>${-1 * 624/35 * 80/18}</mechanicalReduction>
     </transmission>
   </xacro:macro>

File: pr2_description/urdf/base_v0/base.urdf.xacro (robot description, xacro)
@@ -72,6 +72,7 @@
     <xacro:pr2_wheel_transmission_v0 parent="${parent}" suffix="${suffix}" reflect="${reflect}" />
   </xacro:macro>
-  <xacro:macro name="pr2_caster_v0" params="suffix parent *origin ref_position">
-    <joint name="${suffix}_caster_rotation_joint" type="continuous">
+  <!-- Macro for PR2 Caster hub only -->
+  <xacro:macro name="pr2_caster_hub_v0" params="suffix parent *origin ref_position" >
+    <joint name="${suffix}_rotation_joint" type="continuous">
       <axis xyz="0 0 1" />
       <limit effort="100" velocity="100"/>
@@ -81,7 +82,7 @@
       <insert_block name="origin" />
       <parent link="${parent}"/>
-      <child link="${suffix}_caster_rotation_link" />
+      <child link="${suffix}_rotation_link" />
     </joint>
-    <link name="${suffix}_caster_rotation_link">
+    <link name="${suffix}_rotation_link">
       <inertial>
         <mass value="3.473082"/>
@@ -104,4 +105,12 @@
       </collision>
     </link>
+    <!-- extensions -->
+    <xacro:pr2_caster_transmission_v0 suffix="${suffix}" />
+  </xacro:macro>
+  <xacro:macro name="pr2_caster_v0" params="suffix parent *origin ref_position">
+    <xacro:pr2_caster_hub_v0 parent="${parent}" suffix="${suffix}_caster"
+                             ref_position="${ref_position}" >
+      <insert_block name="origin" />
+    </xacro:pr2_caster_hub_v0>
     <!-- wheel macros -->
     <xacro:pr2_wheel_v0 parent="${suffix}_caster" suffix="l" reflect="1" />
@@ -109,5 +118,4 @@
     <!-- extensions -->
     <xacro:pr2_caster_gazebo_v0 suffix="${suffix}" />
-    <xacro:pr2_caster_transmission_v0 suffix="${suffix}" />
   </xacro:macro>
   <!-- The xacro macro xacro:pr2_base contains: base, casters and wheels -->

File: pr2_description/urdf/tilting_laser_v0/tilting_laser.transmission.xacro (robot description, xacro)
@@ -8,5 +8,5 @@
       <actuator name="${name}_mount_motor" />
       <joint name="${name}_mount_joint" />
-      <mechanicalReduction>6.05</mechanicalReduction>
+      <mechanicalReduction>-6.05</mechanicalReduction>
     </transmission>
   </xacro:macro>
