Commit message: update urdf for base

File: pr2_description/urdf/base_v0/base.gazebo.xacro (robot description, xacro)
@@ -11,4 +11,7 @@
   <property name="base_laser_size_z" value="0.03" />
   <property name="base_laser_collision_offset_z" value="0.03" />
+  <!--                                                      -->
+  <!-- Alpha 2.0 hardware                                   -->
+  <!--                                                      -->
   <macro name="pr2_wheel_gazebo" params="suffix parent">
     <gazebo reference="${parent}_${suffix}_wheel_link">
@@ -23,5 +26,4 @@
         </controller:ros_bumper>
       </sensor:contact>
-      <material value="PR2/wheel_${suffix}" />
       <mu1 value="100.0" />
       <mu2 value="100.0" />
@@ -42,8 +44,4 @@
         </controller:ros_bumper>
       </sensor:contact>
-      <mu1 value="0.0" />
-      <mu2 value="0.0" />
-      <kp  value="1000000.0" />
-      <kd  value="1.0" />
       <material value="PR2/Green" />
     </gazebo>
@@ -59,15 +57,4 @@
         <rpyOffsets>0 0 0</rpyOffsets>
         <interface:position name="p3d_base_position"/>
-      </controller:ros_p3d>
-      <controller:ros_p3d name="p3d_plug_holder_controller" plugin="libros_p3d.so">
-        <alwaysOn>true</alwaysOn>
-        <updateRate>100.0</updateRate>
-        <bodyName>plug_holder</bodyName>
-        <topicName>plug_holder_pose_ground_truth</topicName>
-        <gaussianNoise>0.01</gaussianNoise>
-        <frameName>map</frameName>
-        <xyzOffsets>0 0 0</xyzOffsets> <!-- initialize odometry for fake localization-->
-        <rpyOffsets>0 0 0</rpyOffsets>
-        <interface:position name="p3d_plug_holder_position"/>
       </controller:ros_p3d>
     </gazebo>
@@ -97,17 +84,4 @@
       <material value="PR2/Red" />
     </gazebo>
-    <!-- modeling plug on base holder magnet location -->
-    <gazebo reference="plug_holder">
-      <material value="PR2/Red" />
-    </gazebo>
-    <gazebo reference="plug_holder_2">
-      <material value="PR2/Red" />
-    </gazebo>
-    <gazebo reference="plug_holder_3">
-      <material value="PR2/Red" />
-    </gazebo>
-    <gazebo reference="plug_holder_4">
-      <material value="PR2/Red" />
-    </gazebo>
   </macro>
 </robot>

File: pr2_description/urdf/base_v0/base.transmission.xacro (robot description, xacro)
@@ -3,16 +3,19 @@
        xmlns:controller="http://playerstage.sourceforge.net/gazebo/xmlschema/#controller"
        xmlns:interface="http://playerstage.sourceforge.net/gazebo/xmlschema/#interface">
+  <!--                                                      -->
+  <!-- Alpha 2.0 hardware                                   -->
+  <!--                                                      -->
   <macro name="pr2_wheel_transmission" params="suffix parent reflect">
     <transmission type="SimpleTransmission" name="${parent}_${suffix}_wheel_trans">
-      <actuator name="${parent}_${suffix}_wheel_motor" />
+      <actuator name="${parent}_${suffix}_wheel_motor_v0" />
       <joint name="${parent}_${suffix}_wheel_joint" />
-      <mechanicalReduction>${reflect * 624/35 * 80/19}</mechanicalReduction>
+      <mechanicalReduction>${-1 * reflect * 624/35 * 80/18}</mechanicalReduction>
     </transmission>
   </macro>
   <macro name="pr2_caster_transmission" params="suffix">
     <transmission type="SimpleTransmission" name="${suffix}_caster_rotation_trans">
-      <actuator name="${suffix}_caster_rotation_motor" />
+      <actuator name="${suffix}_caster_rotation_motor_v0" />
       <joint name="${suffix}_caster_rotation_joint" />
-      <mechanicalReduction>${-1 * 624/35 * 80/19}</mechanicalReduction>
+      <mechanicalReduction>${624/35 * 80/18}</mechanicalReduction>
     </transmission>
   </macro>

File: pr2_description/urdf/base_v0/base.urdf.xacro (robot description, xacro)
@@ -3,7 +3,10 @@
        xmlns:controller="http://playerstage.sourceforge.net/gazebo/xmlschema/#controller"
        xmlns:interface="http://playerstage.sourceforge.net/gazebo/xmlschema/#interface">
-  <include filename="$(find pr2_defs)/defs/base/base_gazebo.xacro" />
-  <include filename="$(find pr2_defs)/defs/base/base_transmission.xacro" />
+  <include filename="$(find pr2_description)/urdf/base_v0/base.gazebo.xacro" />
+  <include filename="$(find pr2_description)/urdf/base/base.transmission.xacro" />
   <property name="M_PI" value="3.1415926535897931" />
+  <property name="caster_offset_x" value="0.2225" />
+  <property name="caster_offset_y" value="0.2225" />
+  <property name="caster_offset_z" value="0.0282" />
   <property name="caster_wheel_offset_y" value="0.049" /> <!-- from function spreadsheet -->
   <property name="wheel_length" value="0.03" />  <!-- FIXME -->
@@ -24,13 +27,16 @@
   <property name="base_laser_y" value="0.0" />
   <property name="base_laser_z" value="0.252" />
-  <property name="base_laser_size_x" value="0.06" />
-  <property name="base_laser_size_y" value="0.06" />
+  <property name="base_laser_size_x" value="0.08" />
+  <property name="base_laser_size_y" value="0.08" />
   <property name="base_laser_size_z" value="0.03" />
-  <property name="base_laser_collision_offset_z" value="0.02" />
+  <property name="base_laser_collision_offset_z" value="0.03" />
+  <!--                                                      -->
+  <!-- Alpha 2.0 hardware                                   -->
+  <!--                                                      -->
   <macro name="pr2_wheel" params="suffix parent reflect">
     <joint name="${parent}_${suffix}_wheel_joint" type="continuous">
       <axis xyz="0 1 0" />
       <limit effort="100" velocity="100"/>
-      <safety_controller k_velocity="10" />
+      <safety_controller  k_velocity="10" />
       <dynamics damping="0.0" friction="0.0" />
       <origin xyz="0 ${reflect*caster_wheel_offset_y} 0" rpy="0 0 0" />
@@ -41,5 +47,5 @@
       <inertial>
         <mass value="0.44036" /> <!-- check jmh 20081205 -->
-        <origin xyz=" 0 0 0 " />
+        <origin xyz="0 0 0" />
         <inertia  ixx="0.012411765597" ixy="-0.000711733678" ixz="0.00050272983"
                   iyy="0.015218160428" iyz="-0.000004273467" izz="0.011763977943" />
@@ -48,5 +54,5 @@
         <origin xyz="0 0 0" rpy="0 0 0" />
         <geometry name="${parent}_${suffix}_wheel_visual_geom">
-          <mesh filename="package://pr2_defs/meshes/pr2_wheel.stl" />
+          <mesh filename="package://pre_description/meshes/base_v0/pr2_wheel.stl" />
         </geometry>
         <material name="Caster_${suffix}" />
@@ -63,18 +69,18 @@
     <pr2_wheel_transmission parent="${parent}" suffix="${suffix}" reflect="${reflect}" />
   </macro>
-  <macro name="pr2_caster" params="suffix parent *origin">
+  <macro name="pr2_caster" params="suffix parent *origin ref_position">
     <joint name="${suffix}_caster_rotation_joint" type="continuous">
       <axis xyz="0 0 1" />
       <limit effort="100" velocity="100"/>
-      <safety_controller k_velocity="10" />
-      <calibration reference_position="0.0" />
+      <safety_controller  k_velocity="10" />
+      <calibration reference_position="${ref_position}" />
       <dynamics damping="0.0" friction="0.0" />
-      <insert_block name="origin"/>
+      <insert_block name="origin" />
       <parent link="${parent}"/>
-      <child link="${suffix}_caster_rotation_link"/>
+      <child link="${suffix}_caster_rotation_link" />
     </joint>
     <link name="${suffix}_caster_rotation_link">
       <inertial>
-        <mass value="3.473082" />
+        <mass value="3.473082"/>
         <origin xyz="0 0 0.07" />
         <inertia  ixx="0.012411765597" ixy="-0.000711733678" ixz="0.00050272983"
@@ -84,5 +90,5 @@
         <origin xyz="0 0 0" rpy="0 0 0" />
         <geometry name="${suffix}_caster_rotation_visual_geom">
-          <mesh filename="package://pr2_defs/meshes/caster.stl" />
+          <mesh filename="package://pr2_description/meshes/base_v0/caster.stl" />
         </geometry>
         <material name="Green" />
@@ -95,18 +101,15 @@
       </collision>
     </link>
+    <!-- Double check these are right for the Alpha 2.0's -->
+    <pr2_wheel_alpha2 parent="${suffix}_caster" suffix="l" reflect="1" />
+    <pr2_wheel_alpha2 parent="${suffix}_caster" suffix="r" reflect="-1" />
     <!-- extensions -->
-    <pr2_caster_transmission suffix="${suffix}" />
-    <!-- wheel macros -->
-    <pr2_wheel parent="${suffix}_caster" suffix="l" reflect="1" />
-    <pr2_wheel parent="${suffix}_caster" suffix="r" reflect="-1" />
+    <pr2_caster_alpha2_transmission suffix="${suffix}" />
   </macro>
-  <property name="caster_offset_x" value="0.2225" />
-  <property name="caster_offset_y" value="0.2225" />
-  <property name="caster_offset_z" value="0.0282" />
   <macro name="pr2_base" params="name *origin">
     <joint name="${name}_joint" type="planar">
       <insert_block name="origin" />
       <parent link="world"/>
-      <child link="${name}_link"/>
+      <child link="${name}_link" />
     </joint>
     <link name="${name}_link">
@@ -120,5 +123,5 @@
         <origin xyz="0 0 ${base_height_offset}" rpy="0 0 0" />
         <geometry name="${name}_visual_geom">
-          <mesh filename="package://pr2_defs/meshes/base.stl" />
+          <mesh filename="package://pr2_description/meshes/base_v0/base.stl" />
         </geometry>
         <material name="Green" />
@@ -133,7 +136,8 @@
     <!-- base laser -->
     <joint name="base_laser_joint" type="fixed">
+      <axis xyz="0 1 0" />
       <origin xyz="${base_laser_x} ${base_laser_y} ${base_height_offset+base_laser_z}" rpy="0 0 0" />
       <parent link="${name}_link"/>
-      <child link="base_laser"/>
+      <child link="base_laser" />
     </joint>
     <link name="base_laser" type="laser">
@@ -157,46 +161,19 @@
       </collision>
     </link>
-    <pr2_caster suffix="fl" parent="${name}_link">
+    <!-- all four caster macros -->
+    <pr2_caster suffix="fl" parent="${name}_link" ref_position="${cal_caster_fl}" >
       <origin xyz="${caster_offset_x} ${caster_offset_y} ${caster_offset_z}" rpy="0 0 0" />
     </pr2_caster>
-    <pr2_caster suffix="fr" parent="${name}_link">
+    <pr2_caster suffix="fr" parent="${name}_link" ref_position="${cal_caster_fr}" >
       <origin xyz="${caster_offset_x} ${-caster_offset_y} ${caster_offset_z}" rpy="0 0 0" />
     </pr2_caster>
-    <pr2_caster suffix="bl" parent="${name}_link">
+    <pr2_caster suffix="bl" parent="${name}_link" ref_position="${cal_caster_bl}" >
       <origin xyz="${-caster_offset_x} ${caster_offset_y} ${caster_offset_z}" rpy="0 0 0" />
     </pr2_caster>
-    <pr2_caster suffix="br" parent="${name}_link">
+    <pr2_caster suffix="br" parent="${name}_link" ref_position="${cal_caster_br}"  >
       <origin xyz="${-caster_offset_x} ${-caster_offset_y} ${caster_offset_z}" rpy="0 0 0" />
     </pr2_caster>
     <!-- gazebo extensions -->
     <pr2_base_gazebo name="${name}" />
-    <!-- modeling plug on base holder magnet location -->
-    <pr2_plug_holder name="${name}"/>
-  </macro>
-  <macro name="pr2_plug_holder" params="name">
-    <joint name="plug_holder_joint" type="fixed">
-      <origin xyz="0.18 0 ${base_height_offset+base_size_z - 0.001/2}" rpy="0 0 0" />
-      <parent link="${name}_link"/>
-      <child link="plug_holder"/>
-    </joint>
-    <link name="plug_holder">
-      <inertial>
-        <mass value="0.1" />
-        <origin xyz="0 0 0.0" />
-        <inertia ixx="0.1" ixy="0" ixz="0" iyy="0.1" iyz="0" izz="0.1" />
-      </inertial>
-      <visual>
-        <origin xyz="0 0 0" rpy="0 0 0" />
-        <geometry>
-          <box size="0.001 0.001 0.001"/>
-        </geometry>
-      </visual>
-      <collision>
-        <origin xyz="0 0 0.0" rpy="0 0 0" />
-        <geometry>
-          <box size=".001 .001 .001" />
-        </geometry>
-      </collision>
-    </link>
   </macro>
 </robot>
