Commit message: Update urdf, further clean up and breakdown of current pr2_defs. This is still pending more discussion on how to handle multiple versions of the same components on a single robot.

File: pr2_description/urdf/base_v0/base.gazebo.xacro (robot description, xacro)
@@ -3,16 +3,8 @@
        xmlns:controller="http://playerstage.sourceforge.net/gazebo/xmlschema/#controller"
        xmlns:interface="http://playerstage.sourceforge.net/gazebo/xmlschema/#interface">
-  <!-- simplified box collision geometry for hokuyo laser -->
-  <property name="base_laser_x" value="0.275" />
-  <property name="base_laser_y" value="0.0" />
-  <property name="base_laser_z" value="0.252" />
-  <property name="base_laser_size_x" value="0.08" />
-  <property name="base_laser_size_y" value="0.08" />
-  <property name="base_laser_size_z" value="0.03" />
-  <property name="base_laser_collision_offset_z" value="0.03" />
   <!--                                                      -->
   <!-- Alpha 2.0 hardware                                   -->
   <!--                                                      -->
-  <macro name="pr2_wheel_gazebo" params="suffix parent">
+  <xacro:macro name="pr2_wheel_gazebo" params="suffix parent">
     <gazebo reference="${parent}_${suffix}_wheel_link">
       <sensor:contact name="${parent}_${suffix}_wheel_contact_sensor">
@@ -31,6 +23,6 @@
       <kd  value="1.0" />
     </gazebo>
-  </macro>
-  <macro name="pr2_base_gazebo" params="name">
+  </xacro:macro>
+  <xacro:macro name="pr2_base_gazebo" params="name">
     <gazebo reference="${name}_link">
       <sensor:contact name="${name}_contact_sensor">
@@ -59,29 +51,4 @@
       </controller:ros_p3d>
     </gazebo>
-    <!-- base laser -->
-    <gazebo reference="base_laser">
-      <sensor:ray name="base_laser">
-        <rayCount>640</rayCount>
-        <rangeCount>640</rangeCount>
-        <laserCount>1</laserCount>
-        <origin>0.0 0.0 0.0</origin>
-        <displayRays>false</displayRays>
-        <minAngle>-100</minAngle> <!-- scans own arms if -135~+135 -->
-        <maxAngle>100</maxAngle>
-        <minRange>0.05</minRange>
-        <maxRange>10.0</maxRange>
-        <resRange>0.01</resRange>
-        <updateRate>20.0</updateRate>
-        <controller:ros_laser name="ros_base_laser_controller" plugin="libros_laser.so">
-          <gaussianNoise>0.005</gaussianNoise>
-          <alwaysOn>true</alwaysOn>
-          <updateRate>20.0</updateRate>
-          <topicName>base_scan</topicName>
-          <frameName>base_laser</frameName>
-          <interface:laser name="ros_base_laser_iface" />
-        </controller:ros_laser>
-      </sensor:ray>
-      <material value="PR2/Red" />
-    </gazebo>
-  </macro>
+  </xacro:macro>
 </robot>

File: pr2_description/urdf/base_v0/base.transmission.xacro (robot description, xacro)
@@ -6,5 +6,5 @@
   <!-- Alpha 2.0 hardware                                   -->
   <!--                                                      -->
-  <macro name="pr2_wheel_transmission" params="suffix parent reflect">
+  <xacro:macro name="pr2_wheel_transmission" params="suffix parent reflect">
     <transmission type="SimpleTransmission" name="${parent}_${suffix}_wheel_trans">
       <actuator name="${parent}_${suffix}_wheel_motor_v0" />
@@ -12,6 +12,6 @@
       <mechanicalReduction>${-1 * reflect * 624/35 * 80/18}</mechanicalReduction>
     </transmission>
-  </macro>
-  <macro name="pr2_caster_transmission" params="suffix">
+  </xacro:macro>
+  <xacro:macro name="pr2_caster_transmission" params="suffix">
     <transmission type="SimpleTransmission" name="${suffix}_caster_rotation_trans">
       <actuator name="${suffix}_caster_rotation_motor_v0" />
@@ -19,4 +19,4 @@
       <mechanicalReduction>${624/35 * 80/18}</mechanicalReduction>
     </transmission>
-  </macro>
+  </xacro:macro>
 </robot>

File: pr2_description/urdf/base_v0/base.urdf.xacro (robot description, xacro)
@@ -4,5 +4,5 @@
        xmlns:interface="http://playerstage.sourceforge.net/gazebo/xmlschema/#interface">
   <include filename="$(find pr2_description)/urdf/base_v0/base.gazebo.xacro" />
-  <include filename="$(find pr2_description)/urdf/base/base.transmission.xacro" />
+  <include filename="$(find pr2_description)/urdf/base_v0/base.transmission.xacro" />
   <property name="M_PI" value="3.1415926535897931" />
   <property name="caster_offset_x" value="0.2225" />
@@ -30,9 +30,8 @@
   <property name="base_laser_size_y" value="0.08" />
   <property name="base_laser_size_z" value="0.03" />
-  <property name="base_laser_collision_offset_z" value="0.03" />
   <!--                                                      -->
   <!-- Alpha 2.0 hardware                                   -->
   <!--                                                      -->
-  <macro name="pr2_wheel" params="suffix parent reflect">
+  <xacro:macro name="pr2_wheel" params="suffix parent reflect">
     <joint name="${parent}_${suffix}_wheel_joint" type="continuous">
       <axis xyz="0 1 0" />
@@ -66,8 +65,8 @@
     </link>
     <!-- extensions -->
-    <pr2_wheel_gazebo parent="${parent}" suffix="${suffix}" />
-    <pr2_wheel_transmission parent="${parent}" suffix="${suffix}" reflect="${reflect}" />
-  </macro>
-  <macro name="pr2_caster" params="suffix parent *origin ref_position">
+    <xacro:pr2_wheel_gazebo parent="${parent}" suffix="${suffix}" />
+    <xacro:pr2_wheel_transmission parent="${parent}" suffix="${suffix}" reflect="${reflect}" />
+  </xacro:macro>
+  <xacro:macro name="pr2_caster" params="suffix parent *origin ref_position">
     <joint name="${suffix}_caster_rotation_joint" type="continuous">
       <axis xyz="0 0 1" />
@@ -102,10 +101,10 @@
     </link>
     <!-- Double check these are right for the Alpha 2.0's -->
-    <pr2_wheel_alpha2 parent="${suffix}_caster" suffix="l" reflect="1" />
-    <pr2_wheel_alpha2 parent="${suffix}_caster" suffix="r" reflect="-1" />
+    <xacro:pr2_wheel_alpha2 parent="${suffix}_caster" suffix="l" reflect="1" />
+    <xacro:pr2_wheel_alpha2 parent="${suffix}_caster" suffix="r" reflect="-1" />
     <!-- extensions -->
-    <pr2_caster_alpha2_transmission suffix="${suffix}" />
-  </macro>
-  <macro name="pr2_base" params="name *origin">
+    <xacro:pr2_caster_alpha2_transmission suffix="${suffix}" />
+  </xacro:macro>
+  <xacro:macro name="pr2_base" params="name *origin">
     <joint name="${name}_joint" type="planar">
       <insert_block name="origin" />
@@ -135,45 +134,22 @@
     </link>
     <!-- base laser -->
-    <joint name="base_laser_joint" type="fixed">
-      <axis xyz="0 1 0" />
+    <xacro:hokuyo_lx30_laser name="${name}_laser" parent="${name}" ros_topic="base_scan" >
       <origin xyz="${base_laser_x} ${base_laser_y} ${base_height_offset+base_laser_z}" rpy="0 0 0" />
-      <parent link="${name}_link"/>
-      <child link="base_laser" />
-    </joint>
-    <link name="base_laser" type="laser">
-      <inertial>
-        <mass value="1.0" />
-        <origin xyz="0 0 0" />
-        <inertia ixx="0.1" ixy="0" ixz="0" iyy="0.1" iyz="0" izz="0.1" />
-      </inertial>
-      <visual name="base_lvisual">
-        <origin xyz="0 0 ${base_laser_collision_offset_z}" rpy="0 0 0" />
-        <geometry name="base_laser_visual_geom">
-          <box size="${base_laser_size_x} ${base_laser_size_y} ${base_laser_size_z}"/>
-        </geometry>
-        <material name="Red" />
-      </visual>
-      <collision name="base_lcollision">
-        <origin xyz="0 0 ${base_laser_collision_offset_z}" rpy="0 0 0" />
-        <geometry name="base_laser_collision_geom">
-          <box size="${base_laser_size_x} ${base_laser_size_y} ${base_laser_size_z}"/>
-        </geometry>
-      </collision>
-    </link>
+    </xacro:hokuyo_lx30_laser>
     <!-- all four caster macros -->
-    <pr2_caster suffix="fl" parent="${name}_link" ref_position="${cal_caster_fl}" >
+    <xacro:pr2_caster suffix="fl" parent="${name}_link" ref_position="${cal_caster_fl}" >
       <origin xyz="${caster_offset_x} ${caster_offset_y} ${caster_offset_z}" rpy="0 0 0" />
-    </pr2_caster>
-    <pr2_caster suffix="fr" parent="${name}_link" ref_position="${cal_caster_fr}" >
+    </xacro:pr2_caster>
+    <xacro:pr2_caster suffix="fr" parent="${name}_link" ref_position="${cal_caster_fr}" >
       <origin xyz="${caster_offset_x} ${-caster_offset_y} ${caster_offset_z}" rpy="0 0 0" />
-    </pr2_caster>
-    <pr2_caster suffix="bl" parent="${name}_link" ref_position="${cal_caster_bl}" >
+    </xacro:pr2_caster>
+    <xacro:pr2_caster suffix="bl" parent="${name}_link" ref_position="${cal_caster_bl}" >
       <origin xyz="${-caster_offset_x} ${caster_offset_y} ${caster_offset_z}" rpy="0 0 0" />
-    </pr2_caster>
-    <pr2_caster suffix="br" parent="${name}_link" ref_position="${cal_caster_br}"  >
+    </xacro:pr2_caster>
+    <xacro:pr2_caster suffix="br" parent="${name}_link" ref_position="${cal_caster_br}"  >
       <origin xyz="${-caster_offset_x} ${-caster_offset_y} ${caster_offset_z}" rpy="0 0 0" />
-    </pr2_caster>
+    </xacro:pr2_caster>
     <!-- gazebo extensions -->
-    <pr2_base_gazebo name="${name}" />
-  </macro>
+    <xacro:pr2_base_gazebo name="${name}" />
+  </xacro:macro>
 </robot>

File: pr2_description/urdf/forearm_v0/forearm.gazebo.xacro (robot description, xacro)
@@ -3,5 +3,5 @@
        xmlns:controller="http://playerstage.sourceforge.net/gazebo/xmlschema/#controller"
        xmlns:interface="http://playerstage.sourceforge.net/gazebo/xmlschema/#interface">
-  <macro name="pr2_forearm_gazebo" params="side">
+  <xacro:macro name="pr2_forearm_gazebo" params="side">
     <gazebo reference="${side}_forearm_link">
       <turnGravityOff>true</turnGravityOff>
@@ -55,4 +55,4 @@
       <fudgeFactor value="0.5" />
     </gazebo>
-  </macro>
+  </xacro:macro>
 </robot>

File: pr2_description/urdf/forearm_v0/forearm.transmission.xacro (robot description, xacro)
@@ -3,5 +3,5 @@
        xmlns:controller="http://playerstage.sourceforge.net/gazebo/xmlschema/#controller"
        xmlns:interface="http://playerstage.sourceforge.net/gazebo/xmlschema/#interface">
-  <macro name="pr2_forearm_transmission" params="side">
+  <xacro:macro name="pr2_forearm_transmission" params="side">
     <!-- Wrist flex , Wrist roll -->
     <transmission type="WristTransmission" name="${side}_wrist_trans">
@@ -11,4 +11,4 @@
       <rollJoint name="${side}_wrist_roll_joint" mechanicalReduction="${624/35*54/16}"  />
     </transmission>
-  </macro>
+  </xacro:macro>
 </robot>

File: pr2_description/urdf/forearm_v0/forearm.urdf.xacro (robot description, xacro)
@@ -10,5 +10,5 @@
   <include filename="$(find pr2_description)/urdf/common.xacro" />
   <!-- ============================   Forearm   ============================ -->
-  <macro name="pr2_forearm" params="side parent reflect">
+  <xacro:macro name="pr2_forearm" params="side parent reflect">
     <joint name="${side}_forearm_joint" type="fixed">
       <origin xyz="0 0 0" rpy="0 0 0" />
@@ -106,4 +106,7 @@
       </collision>
     </link>
-  </macro>
+    <!-- extensions-->
+    <xacro:pr2_forearm_gazebo side="${side}" />
+    <xacro:pr2_forearm_transmission side="${side}" />
+  </xacro:macro>
 </robot>

File: pr2_description/urdf/gripper_v0/gripper.transmission.xacro (robot description, xacro)
@@ -4,5 +4,5 @@
        xmlns:joint="http://playerstage.sourceforge.net/gazebo/xmlschema/#slider"
        xmlns:interface="http://playerstage.sourceforge.net/gazebo/xmlschema/#interface">
-  <macro name="pr2_gripper_transmission" params="side">
+  <xacro:macro name="pr2_gripper_transmission" params="side">
     <!-- [lr]_gripper_joint is a fictitious joint, used by transmission for controller gap   -->
     <!-- [lr]_gripper_joint is not attached to any link                                      -->
@@ -22,4 +22,4 @@
       <passive_joint  name="${side}_gripper_l_finger_tip_joint" />
     </transmission>
-  </macro>
+  </xacro:macro>
 </robot>

File: pr2_description/urdf/head_v0/head.gazebo.xacro (robot description, xacro)
@@ -3,18 +3,18 @@
        xmlns:controller="http://playerstage.sourceforge.net/gazebo/xmlschema/#controller"
        xmlns:interface="http://playerstage.sourceforge.net/gazebo/xmlschema/#interface">
-  <macro name="pr2_head_pan_gazebo" params="name">
+  <xacro:macro name="pr2_head_pan_gazebo" params="name">
     <gazebo reference="${name}_link">
       <material value="PR2/Blue" />
     </gazebo>
-  </macro>
-  <macro name="pr2_head_tilt_gazebo" params="name">
+  </xacro:macro>
+  <xacro:macro name="pr2_head_tilt_gazebo" params="name">
     <gazebo reference="${name}_link">
       <material value="PR2/Green" />
     </gazebo>
-  </macro>
-  <macro name="pr2_head_gazebo" params="name">
+  </xacro:macro>
+  <xacro:macro name="pr2_head_gazebo" params="name">
     <gazebo reference="${name}_plate_frame">
       <material value="PR2/Blue" />
     </gazebo>
-  </macro>
+  </xacro:macro>
 </robot>

File: pr2_description/urdf/head_v0/head.transmission.xacro (robot description, xacro)
@@ -3,5 +3,5 @@
        xmlns:controller="http://playerstage.sourceforge.net/gazebo/xmlschema/#controller"
        xmlns:interface="http://playerstage.sourceforge.net/gazebo/xmlschema/#interface">
-  <macro name="pr2_head_pan_transmission" params="name">
+  <xacro:macro name="pr2_head_pan_transmission" params="name">
     <transmission type="SimpleTransmission" name="${name}_trans">
       <actuator name="${name}_motor" />
@@ -9,6 +9,6 @@
       <mechanicalReduction>6.0</mechanicalReduction>
     </transmission>
-  </macro>
-  <macro name="pr2_head_tilt_transmission" params="name">
+  </xacro:macro>
+  <xacro:macro name="pr2_head_tilt_transmission" params="name">
     <transmission type="SimpleTransmission" name="${name}_trans">
       <actuator name="${name}_motor" />
@@ -16,4 +16,4 @@
       <mechanicalReduction>6.0</mechanicalReduction>
     </transmission>
-  </macro>
+  </xacro:macro>
 </robot>

File: pr2_description/urdf/head_v0/head.urdf.xacro (robot description, xacro)
@@ -3,9 +3,8 @@
        xmlns:controller="http://playerstage.sourceforge.net/gazebo/xmlschema/#controller"
        xmlns:interface="http://playerstage.sourceforge.net/gazebo/xmlschema/#interface">
-  <include filename="$(find pr2_defs)/defs/head/head_sensor_package_defs.urdf.xacro" />
-  <include filename="$(find pr2_defs)/defs/head/head_gazebo.xacro" />
-  <include filename="$(find pr2_defs)/defs/head/head_transmission.xacro" />
+  <include filename="$(find pr2_description)/urdf/head_v0/head.gazebo.xacro" />
+  <include filename="$(find pr2_description)/urdf/head_v0/head.transmission.xacro" />
   <property name="M_PI" value="3.1415926535897931" />
-  <macro name="pr2_head_pan" params="name parent *origin">
+  <xacro:macro name="pr2_head_pan" params="name parent *origin">
     <joint name="${name}_joint" type="revolute">
       <axis xyz="0 0 1" />
@@ -40,8 +39,8 @@
     </link>
     <!-- extensions -->
-    <pr2_head_pan_gazebo name="${name}" />
-    <pr2_head_pan_transmission name="${name}" />
-  </macro>
-  <macro name="pr2_head_tilt" params="name parent *origin">
+    <xacro:pr2_head_pan_gazebo name="${name}" />
+    <xacro:pr2_head_pan_transmission name="${name}" />
+  </xacro:macro>
+  <xacro:macro name="pr2_head_tilt" params="name parent *origin">
     <joint name="${name}_joint" type="revolute">
       <axis xyz="0 1 0" />
@@ -77,14 +76,14 @@
     </link>
     <!-- extensions -->
-    <pr2_head_tilt_gazebo name="${name}" />
-    <pr2_head_tilt_transmission name="${name}" />
-  </macro>
-  <macro name="pr2_head" params="name parent *origin">
-    <pr2_head_pan name="${name}_pan" parent="${parent}">
+    <xacro:pr2_head_tilt_gazebo name="${name}" />
+    <xacro:pr2_head_tilt_transmission name="${name}" />
+  </xacro:macro>
+  <xacro:macro name="pr2_head" params="name parent *origin">
+    <xacro:pr2_head_pan name="${name}_pan" parent="${parent}">
       <insert_block name="origin" />
-    </pr2_head_pan>
-    <pr2_head_tilt name="${name}_tilt" parent="${name}_pan_link">
+    </xacro:pr2_head_pan>
+    <xacro:pr2_head_tilt name="${name}_tilt" parent="${name}_pan_link">
       <origin xyz="0.058 0 0" rpy="0 0 0" />
-    </pr2_head_tilt>
+    </xacro:pr2_head_tilt>
     <!-- Head plate frame -->
     <joint name="${name}_plate_frame_joint" type="fixed">
@@ -116,5 +115,5 @@
     </link>
     <!-- extensions -->
-    <pr2_head_gazebo name="${name}" />
-  </macro>
+    <xacro:pr2_head_gazebo name="${name}" />
+  </xacro:macro>
 </robot>

File: pr2_description/urdf/sensors/prosilica_gc2450_camera.gazebo.xacro (robot description, xacro)
@@ -3,5 +3,5 @@
       xmlns:controller="http://playerstage.sourceforge.net/gazebo/xmlschema/#controller"
       xmlns:interface="http://playerstage.sourceforge.net/gazebo/xmlschema/#interface">
-<macro name="prosilica_cam_gazebo" params="name">
+<xacro:macro name="prosilica_cam_gazebo" params="name">
   <gazebo reference="${name}_frame">
     <sensor:camera name="${name}_sensor">
@@ -38,4 +38,4 @@
     <material value="PR2/Blue" />
   </gazebo>
-</macro>
+</xacro:macro>
 </root>

File: pr2_description/urdf/sensors/prosilica_gc2450_camera.urdf.xacro (robot description, xacro)
@@ -3,6 +3,6 @@
       xmlns:controller="http://playerstage.sourceforge.net/gazebo/xmlschema/#controller"
       xmlns:interface="http://playerstage.sourceforge.net/gazebo/xmlschema/#interface">
-  <include filename="$(find pr2_defs)/defs/head/prosilica_gazebo.xacro" />
-  <macro name="prosilica_cam" params="name parent *origin">
+  <include filename="$(find pr2_description)/urdf/sensors/prosilica_gc2450_camera.gazebo.xacro" />
+  <xacro:macro name="prosilica_cam" params="name parent *origin">
     <joint name="${name}_frame_joint" type="fixed">
       <insert_block name="origin" />
@@ -61,5 +61,5 @@
     </link>
     <!-- extensions -->
-    <prosilica_cam_gazebo name="${name}"/>
-  </macro>
+    <xacro:prosilica_cam_gazebo name="${name}"/>
+  </xacro:macro>
 </root>

File: pr2_description/urdf/sensors/wge100_camera.gazebo.xacro (robot description, xacro)
@@ -3,5 +3,5 @@
        xmlns:controller="http://playerstage.sourceforge.net/gazebo/xmlschema/#controller"
        xmlns:interface="http://playerstage.sourceforge.net/gazebo/xmlschema/#interface">
-  <macro name="wge100_camera_gazebo" params="name">
+  <xacro:macro name="wge100_camera_gazebo" params="name">
     <gazebo reference="${name}_frame">
       <sensor:camera name="${name}_sensor">
@@ -26,4 +26,4 @@
       <turnGravityOff>true</turnGravityOff>
     </gazebo>
-  </macro>
+  </xacro:macro>
 </robot>

File: pr2_description/urdf/sensors/wge100_camera.urdf.xacro (robot description, xacro)
@@ -1,6 +1,6 @@
 <?xml version="1.0"?>
 <robot>
-  <include filename="$(find pr2_description)/urdf/sensors/wge100_gazebo.xacro" />
-  <macro name="wge100_camera" params="name parent *origin">
+  <include filename="$(find pr2_description)/urdf/sensors/wge100.gazebo.xacro" />
+  <xacro:macro name="wge100_camera" params="name parent *origin">
     <joint name="${name}_frame_joint" type="fixed">
       <insert_block name="origin" />
@@ -56,5 +56,5 @@
     </link>
     <!-- extensions -->
-    <mono_cam_gazebo name="${name}" />
-  </macro>
+    <xacro:wge100_camera_gazebo name="${name}" />
+  </xacro:macro>
 </robot>

File: pr2_description/urdf/shoulder_v0/shoulder.gazebo.xacro (robot description, xacro)
@@ -3,5 +3,5 @@
        xmlns:controller="http://playerstage.sourceforge.net/gazebo/xmlschema/#controller"
        xmlns:interface="http://playerstage.sourceforge.net/gazebo/xmlschema/#interface">
-  <macro name="pr2_shoulder_gazebo" params="side">
+  <xacro:macro name="pr2_shoulder_gazebo" params="side">
     <!-- Shoulder pan -->
     <gazebo reference="${side}_shoulder_pan_link">
@@ -51,4 +51,4 @@
       <fudgeFactor value="0.5" />
     </gazebo>
-  </macro>
+  </xacro:macro>
 </robot>

File: pr2_description/urdf/shoulder_v0/shoulder.transmission.xacro (robot description, xacro)
@@ -3,5 +3,5 @@
        xmlns:controller="http://playerstage.sourceforge.net/gazebo/xmlschema/#controller"
        xmlns:interface="http://playerstage.sourceforge.net/gazebo/xmlschema/#interface">
-  <macro name="pr2_shoulder_transmission" params="side">
+  <xacro:macro name="pr2_shoulder_transmission" params="side">
     <!-- Shoulder pan -->
     <transmission type="SimpleTransmission" name="${side}_shoulder_pan_trans">
@@ -22,4 +22,4 @@
       <mechanicalReduction>${32.65/cal_r_upper_arm_roll_gearing}</mechanicalReduction>
     </transmission>
-  </macro>
+  </xacro:macro>
 </robot>

File: pr2_description/urdf/shoulder_v0/shoulder.urdf.xacro (robot description, xacro)
@@ -12,5 +12,5 @@
   <property name="shoulder_lift_radius" value="0.12" />  <!--TODO Define and give source-->
  <!-- ============================   Shoulder   ============================ -->
-  <macro name="pr2_shoulder" params="side parent reflect *origin">
+  <xacro:macro name="pr2_shoulder" params="side parent reflect *origin">
     <!-- Shoulder pan -->
     <joint name="${side}_shoulder_pan_joint" type="revolute">
@@ -122,4 +122,7 @@
       </collision>
     </link>
-  </macro>
+    <!-- extensions -->
+    <xacro:pr2_shoulder_gazebo side="${side}" />
+    <xacro:pr2_shoulder_transmission side="${side}" />
+  </xacro:macro>
 </robot>

File: pr2_description/urdf/tilting_laser_v0/tilting_laser.gazebo.xacro (robot description, xacro)
@@ -3,10 +3,8 @@
        xmlns:controller="http://playerstage.sourceforge.net/gazebo/xmlschema/#controller"
        xmlns:interface="http://playerstage.sourceforge.net/gazebo/xmlschema/#interface">
-  <macro name="pr2_torso_transmission" params="name">
-    <transmission type="SimpleTransmission" name="${name}_trans">
-      <actuator name="${name}_motor" />
-      <joint name="${name}_joint" />
-      <mechanicalReduction>-52143.33</mechanicalReduction>
-    </transmission>
-  </macro>
+  <xacro:macro name="pr2_tilting_laser_gazebo" params="name">
+    <gazebo reference="${name}_mount_link">
+      <material value="PR2/Red" />
+    </gazebo>
+  </xacro:macro>
 </robot>

File: pr2_description/urdf/torso_v0/torso.gazebo.xacro (robot description, xacro)
@@ -3,5 +3,5 @@
        xmlns:controller="http://playerstage.sourceforge.net/gazebo/xmlschema/#controller"
        xmlns:interface="http://playerstage.sourceforge.net/gazebo/xmlschema/#interface">
-  <macro name="pr2_torso_ext" params="name">
+  <xacro:macro name="pr2_torso_ext" params="name">
     <gazebo reference="${name}_link">
       <sensor:contact name="${name}_contact_sensor">
@@ -17,4 +17,4 @@
       <material value="PR2/Grey2" />
     </gazebo>
-  </macro>
+  </xacro:macro>
 </robot>
