Commit message: Update urdf, further clean up and breakdown of current pr2_defs. This is still pending more discussion on how to handle multiple versions of the same components on a single robot.

File: pr2_description/urdf/torso_v0/torso.transmission.xacro (robot description, xacro)
@@ -3,10 +3,10 @@
        xmlns:controller="http://playerstage.sourceforge.net/gazebo/xmlschema/#controller"
        xmlns:interface="http://playerstage.sourceforge.net/gazebo/xmlschema/#interface">
-  <macro name="pr2_tilting_laser_transmission" params="name">
-    <transmission type="SimpleTransmission" name="${name}_mount_trans">
-      <actuator name="${name}_mount_motor" />
-      <joint name="${name}_mount_joint" />
-      <mechanicalReduction>6.0</mechanicalReduction>
+  <xacro:macro name="pr2_torso_transmission" params="name">
+    <transmission type="SimpleTransmission" name="${name}_trans">
+      <actuator name="${name}_motor" />
+      <joint name="${name}_joint" />
+      <mechanicalReduction>-52143.33</mechanicalReduction>
     </transmission>
-  </macro>
+  </xacro:macro>
 </robot>

Commit message: update base collision according to last measured values, switch selfCollide(for plug_in-sim) from gripper to base

File: pr2_description/urdf/base_v0/base.gazebo.xacro (robot description, xacro)
@@ -17,4 +17,5 @@
   <xacro:macro name="pr2_base_gazebo" params="name">
     <gazebo reference="${name}_link">
+      <selfCollide>true</selfCollide>
       <sensor:contact name="${name}_contact_sensor">
         <geom>${name}_link_geom</geom>

File: pr2_description/urdf/base_v0/base.urdf.xacro (robot description, xacro)
@@ -25,13 +25,15 @@
   <property name="base_size_y" value="0.65" />
   <property name="base_size_z" value="0.23" />
+  <property name="base_collision_size_z" value="0.04" />
   <!-- simplified box collision geometry for hokuyo laser -->
   <property name="base_laser_x" value="0.275" />
   <property name="base_laser_y" value="0.0" />
   <property name="base_laser_z" value="0.252" />
-  <property name="base_laser_size_x" value="0.08" />
-  <property name="base_laser_size_y" value="0.08" />
+  <property name="base_laser_size_x" value="0.06" />
+  <property name="base_laser_size_y" value="0.06" />
   <property name="base_laser_size_z" value="0.03" />
+  <property name="base_laser_collision_offset_z" value="0.023" />
   <!--                                                      -->
-  <!-- Alpha 2.0 hardware                                   -->
+  <!--           wheel                                      -->
   <!--                                                      -->
   <xacro:macro name="pr2_wheel" params="suffix parent reflect">
@@ -52,14 +54,14 @@
                   iyy="0.015218160428" iyz="-0.000004273467" izz="0.011763977943" />
       </inertial>
-      <visual name="${parent}_${suffix}_wheel_visual">
+      <visual>
         <origin xyz="0 0 0" rpy="0 0 0" />
-        <geometry name="${parent}_${suffix}_wheel_visual_geom">
+        <geometry>
           <mesh filename="package://pr2_description/meshes/base_v0/pr2_wheel.stl" />
         </geometry>
         <material name="Caster_${suffix}" />
       </visual>
-      <collision name="${parent}_${suffix}_wheel_collision">
+      <collision>
         <origin xyz="0 0 0" rpy="${M_PI/2} 0 0" /> <!-- rotation because cyl. geom primitive has symmetry axis in +x direction -->
-        <geometry name="${parent}_${suffix}_wheel_collision_geom">
+        <geometry>
           <cylinder radius="${wheel_radius}" length="${wheel_length}" />
         </geometry>
@@ -88,19 +90,19 @@
                   iyy="0.015218160428" iyz="-0.000004273467" izz="0.011763977943" />
       </inertial>
-      <visual name="${suffix}_caster_rotation_visual">
+      <visual>
         <origin xyz="0 0 0" rpy="0 0 0" />
-        <geometry name="${suffix}_caster_rotation_visual_geom">
+        <geometry>
           <mesh filename="package://pr2_description/meshes/base_v0/caster.stl" />
         </geometry>
         <material name="Green" />
       </visual>
-      <collision name="${suffix}_caster_rotation_collision">
+      <collision>
         <origin xyz="0 0 0.07" rpy="0.0 0.0 0.0" />
-        <geometry name="${suffix}_caster_rotation_collision_geom">
+        <geometry>
           <box size="0.192 0.164 0.013" />
         </geometry>
       </collision>
     </link>
-    <!-- Double check these are right for the Alpha 2.0's -->
+    <!-- wheel macros -->
     <xacro:pr2_wheel parent="${suffix}_caster" suffix="l" reflect="1" />
     <xacro:pr2_wheel parent="${suffix}_caster" suffix="r" reflect="-1" />
@@ -122,15 +124,17 @@
                  iyy="5.669473158652" iyz="-0.007379583694" izz="3.683196351726" />
       </inertial>
-      <visual name="${name}_visual">
+      <visual>
         <origin xyz="0 0 0" rpy="0 0 0" />
-        <geometry name="${name}_visual_geom">
+        <geometry>
           <mesh filename="package://pr2_description/meshes/base_v0/base.stl" />
         </geometry>
         <material name="Green" />
       </visual>
-      <collision name="${name}_collision">
-        <origin xyz="0 0 ${base_size_z/2}" rpy="0 0 0" />
-        <geometry name="${name}_collision_geom">
-          <box size="${base_size_x} ${base_size_y} ${base_size_z}" />
+      <collision>
+        <!-- represent base collision with a simple rectangular model, positioned by base_size_z s.t. top
+             surface of the collision box matches the top surface of the PR2 base -->
+        <origin xyz="0 0 ${base_size_z-base_collision_size_z/2}" rpy="0 0 0" />
+        <geometry>
+          <box size="${base_size_x} ${base_size_y} ${base_collision_size_z}" />
         </geometry>
       </collision>

File: pr2_description/urdf/gripper_v0/gripper.gazebo.xacro (robot description, xacro)
@@ -71,5 +71,5 @@
     <gazebo reference="${prefix}_l_finger_tip_link">
       <turnGravityOff>true</turnGravityOff>
-      <selfCollide value="true" />
+      <selfCollide>false</selfCollide>
       <sensor:contact name="${prefix}_l_finger_tip_contact_sensor">
         <geom>${prefix}_l_finger_tip_link_geom</geom>
@@ -97,5 +97,5 @@
     <gazebo reference="${prefix}_r_finger_tip_link">
       <turnGravityOff>true</turnGravityOff>
-      <selfCollide value="true" />
+      <selfCollide>false</selfCollide>
       <sensor:contact name="${prefix}_r_finger_tip_contact_sensor">
         <geom>${prefix}_r_finger_tip_link_geom</geom>

Commit message: add texture for caster

File: pr2_description/urdf/base_v0/base.gazebo.xacro (robot description, xacro)
@@ -13,4 +13,10 @@
       <kp  value="1000000.0" />
       <kd  value="1.0" />
+      <material value="PR2/wheel_${suffix}" />
+    </gazebo>
+  </xacro:macro>
+  <xacro:macro name="pr2_caster_gazebo_v0" params="suffix">
+    <gazebo reference="${suffix}_caster_rotation_link">
+      <material value="PR2/caster_texture" />
     </gazebo>
   </xacro:macro>

File: pr2_description/urdf/base_v0/base.urdf.xacro (robot description, xacro)
@@ -108,4 +108,5 @@
     <xacro:pr2_wheel_v0 parent="${suffix}_caster" suffix="r" reflect="-1" />
     <!-- extensions -->
+    <xacro:pr2_caster_gazebo_v0 suffix="${suffix}" />
     <xacro:pr2_caster_transmission_v0 suffix="${suffix}" />
   </xacro:macro>

Commit message: make base_footprint parent of base_link. added tag for gazebo specikfying base_link as the canonicalBody.  Does not seem to be registered by gazebo yet.

File: pr2_description/urdf/base_v0/base.gazebo.xacro (robot description, xacro)
@@ -45,4 +45,5 @@
         <interface:position name="p3d_base_position"/>
       </controller:gazebo_ros_p3d>
+      <canonicalBody>${name}_link</canonicalBody>
     </gazebo>
   </xacro:macro>

File: pr2_description/urdf/base_v0/base.urdf.xacro (robot description, xacro)
@@ -146,9 +146,31 @@
     <!-- base_footprint is a fictitious link(frame) that is on the ground right below base_link origin,
          navigation stack dedpends on this frame -->
-    <link name="${name}_footprint"/>
+    <link name="${name}_footprint">
+      <inertial>
+        <mass value="1.0" />
+        <origin xyz="0 0 0" />
+        <inertia ixx="0.01" ixy="0.0" ixz="0.0"
+                 iyy="0.01" iyz="0.0" izz="0.01" />
+      </inertial>
+      <visual>
+        <origin xyz="0 0 0" rpy="0 0 0" />
+        <geometry>
+          <box size="0.01 0.01 0.01" />
+        </geometry>
+        <material name="Green" />
+      </visual>
+      <collision>
+        <!-- represent base collision with a simple rectangular model, positioned by base_size_z s.t. top
+             surface of the collision box matches the top surface of the PR2 base -->
+        <origin xyz="0 0 ${0.051+base_collision_size_z/2}" rpy="0 0 0" />
+        <geometry>
+          <box size="0.001 0.001 0.001" />
+        </geometry>
+      </collision>
+    </link>
     <joint name="${name}_footprint_joint" type="fixed">
-      <origin xyz="0 0 -0.051" rpy="0 0 0" />
-      <parent link="${name}_link" />
-      <child link="${name}_footprint"/>
+      <origin xyz="0 0 0.051" rpy="0 0 0" />
+      <child link="${name}_link" />
+      <parent link="${name}_footprint"/>
     </joint>
     <!-- base laser -->

Commit message: Updated the colors for the PR2

File: pr2_description/urdf/base_v0/base.gazebo.xacro (robot description, xacro)
@@ -31,5 +31,5 @@
         </controller:gazebo_ros_bumper>
       </sensor:contact>
-      <material value="PR2/Green" />
+      <material value="Gazebo/White" />
     </gazebo>
     <gazebo>

File: pr2_description/urdf/base_v0/base.urdf.xacro (robot description, xacro)
@@ -96,5 +96,5 @@
           <mesh filename="package://pr2_description/meshes/base_v0/caster.stl" />
         </geometry>
-        <material name="Green" />
+        <material name="White" />
       </visual>
       <collision>
@@ -133,5 +133,5 @@
           <mesh filename="package://pr2_description/meshes/base_v0/base.stl" />
         </geometry>
-        <material name="Green" />
+        <material name="White" />
       </visual>
       <collision>
@@ -158,5 +158,5 @@
           <box size="0.01 0.01 0.01" />
         </geometry>
-        <material name="Green" />
+        <material name="White" />
       </visual>
       <collision>

File: pr2_description/urdf/forearm_v0/forearm.gazebo.xacro (robot description, xacro)
@@ -17,5 +17,5 @@
         </controller:gazebo_ros_bumper>
       </sensor:contact>
-      <material value="PR2/Blue" />
+      <material value="PR2/Grey" />
     </gazebo>
     <!-- Wrist flex -->

File: pr2_description/urdf/forearm_v0/forearm.urdf.xacro (robot description, xacro)
@@ -30,5 +30,5 @@
           <mesh filename="package://pr2_description/meshes/forearm_v0/forearm.stl" />
         </geometry>
-        <material name="Blue" />
+        <material name="Grey" />
       </visual>
       <collision name="${side}_forearm_collision">

File: pr2_description/urdf/gripper_v0/gripper.gazebo.xacro (robot description, xacro)
@@ -88,5 +88,5 @@
       <kp  value="10000000.0" />
       <kd  value="1.0" />
-      <material value="PR2/Red" />
+      <material value="PR2/Grey" />
     </gazebo>
     <gazebo reference="${prefix}_l_finger_tip_joint">
@@ -114,5 +114,5 @@
       <kp  value="10000000.0" />
       <kd  value="1.0" />
-      <material value="PR2/Red" />
+      <material value="PR2/Grey" />
     </gazebo>
     <gazebo>
@@ -155,5 +155,5 @@
         </controller:gazebo_ros_bumper>
       </sensor:contact>
-      <material value="PR2/Red" />
+      <material value="PR2/Grey" />
     </gazebo>
     <!-- floating link for simulating gripper constraints -->

File: pr2_description/urdf/upper_arm_v0/upper_arm.gazebo.xacro (robot description, xacro)
@@ -17,5 +17,5 @@
       </sensor:contact>
       <turnGravityOff>true</turnGravityOff>
-      <material value="PR2/Green" />
+      <material value="Gazebo/Grey" />
     </gazebo>
   </xacro:macro>
