Commit message: using low res stl for collision

File: pr2_description/urdf/base_v0/base.gazebo.xacro (robot description, xacro)
@@ -31,5 +31,5 @@
         </controller:gazebo_ros_bumper>
       </sensor:contact>
-      <material value="Gazebo/White" />
+      <material value="PR2/caster_texture" />
     </gazebo>
     <gazebo>

File: pr2_description/urdf/base_v0/base.urdf.xacro (robot description, xacro)
@@ -97,10 +97,10 @@
           <mesh filename="package://pr2_description/meshes/base_v0/caster.stl" />
         </geometry>
-        <material name="White" />
+        <material name="Caster" />
       </visual>
       <collision>
-        <origin xyz="0 0 0.07" rpy="0.0 0.0 0.0" />
+        <origin xyz="0 0 0" rpy="0 0 0" />
         <geometry>
-          <box size="0.192 0.164 0.013" />
+          <mesh filename="package://pr2_description/meshes/base_v0/caster_L.stl" />
         </geometry>
       </collision>
@@ -137,9 +137,7 @@
       </visual>
       <collision>
-        <!-- represent base collision with a simple rectangular model, positioned by base_size_z s.t. top
-             surface of the collision box matches the top surface of the PR2 base -->
-        <origin xyz="0 0 ${base_size_z-base_collision_size_z/2}" rpy="0 0 0" />
+        <origin xyz="0 0 0" rpy="0 0 0" />
         <geometry>
-          <box size="${base_size_x} ${base_size_y} ${base_collision_size_z}" />
+          <mesh filename="package://pr2_description/meshes/base_v0/base_L.stl" />
         </geometry>
       </collision>

File: pr2_description/urdf/base_v1/base.urdf.xacro (robot description, xacro)
@@ -97,10 +97,10 @@
           <mesh filename="package://pr2_description/meshes/base_v1/caster.stl" />
         </geometry>
-        <material name="White" />
+        <material name="Caster" />
       </visual>
       <collision>
-        <origin xyz="0 0 0.07" rpy="0.0 0.0 0.0" />
+        <origin xyz="0 0 0" rpy="0 0 0" />
         <geometry>
-          <box size="0.192 0.164 0.013" />
+          <mesh filename="package://pr2_description/meshes/base_v0/caster_L.stl" />
         </geometry>
       </collision>
@@ -137,9 +137,7 @@
       </visual>
       <collision>
-        <!-- represent base collision with a simple rectangular model, positioned by base_size_z s.t. top
-             surface of the collision box matches the top surface of the PR2 base -->
-        <origin xyz="0 0 ${base_size_z-base_collision_size_z/2}" rpy="0 0 0" />
+        <origin xyz="0 0 0" rpy="0 0 0" />
         <geometry>
-          <box size="${base_size_x} ${base_size_y} ${base_collision_size_z}" />
+          <mesh filename="package://pr2_description/meshes/base_v0/base_L.stl" />
         </geometry>
       </collision>

File: pr2_description/urdf/forearm_v0/forearm.urdf.xacro (robot description, xacro)
@@ -59,14 +59,14 @@
                  izz="0.00064450498" />
       </inertial>
-      <visual name="${side}_wrist_flex_visual">
+      <visual>
         <origin xyz="0 0 0" rpy="0 0 0" />
-        <geometry name="${side}_wrist_flex_visual_geom">
+        <geometry>
           <mesh filename="package://pr2_description/meshes/forearm_v0/wrist_flex.stl" />
         </geometry>
         <material name="Grey" />
       </visual>
-      <collision name="${side}_wrist_flex_collision">
+      <collision>
         <origin xyz="0 0 0" rpy="0 0 0" />
-        <geometry name="${side}_wrist_flex_collision_geom">
+        <geometry>
           <mesh filename="package://pr2_description/meshes/forearm_v0/wrist_flex.stl" />
         </geometry>
@@ -94,15 +94,15 @@
                  izz="0.01" />
       </inertial>
-      <visual name="${side}_wrist_roll_visual">
+      <visual>
         <origin xyz="0 0 0" rpy="0 0 0" />
-        <geometry name="${side}_wrist_roll_visual_geom">
+        <geometry>
           <mesh filename="package://pr2_description/meshes/forearm_v0/wrist_roll.stl" />
         </geometry>
         <material name="RollLinks" />
       </visual>
-      <collision name="${side}_wrist_roll_collision">
-        <origin xyz="0.0 0 0" rpy="0 0 0" />
-        <geometry name="${side}_wrist_roll_collision_geom">
-          <box size="0.01 0.01 0.01" />
+      <collision>
+        <origin xyz="0 0 0" rpy="0 0 0" />
+        <geometry>
+          <mesh filename="package://pr2_description/meshes/forearm_v0/wrist_roll_L.stl" />
         </geometry>
         <verbose value="Yes" />

File: pr2_description/urdf/forearm_v1/forearm.urdf.xacro (robot description, xacro)
@@ -59,15 +59,15 @@
                  izz="0.00064450498" />
       </inertial>
-      <visual name="${side}_wrist_flex_visual">
+      <visual>
         <origin xyz="0 0 0" rpy="0 0 0" />
-        <geometry name="${side}_wrist_flex_visual_geom">
+        <geometry>
           <mesh filename="package://pr2_description/meshes/forearm_v1/wrist_flex.dae" />
         </geometry>
         <material name="Grey" />
       </visual>
-      <collision name="${side}_wrist_flex_collision">
+      <collision>
         <origin xyz="0 0 0" rpy="0 0 0" />
-        <geometry name="${side}_wrist_flex_collision_geom">
-          <mesh filename="package://pr2_description/meshes/forearm_v1/wrist_flex.dae" />
+        <geometry>
+          <mesh filename="package://pr2_description/meshes/forearm_v0/wrist_flex.stl" />
         </geometry>
       </collision>
@@ -94,15 +94,15 @@
                  izz="0.01" />
       </inertial>
-      <visual name="${side}_wrist_roll_visual">
+      <visual>
         <origin xyz="0 0 0" rpy="0 0 0" />
-        <geometry name="${side}_wrist_roll_visual_geom">
+        <geometry>
           <mesh filename="package://pr2_description/meshes/forearm_v1/wrist_roll.stl" />
         </geometry>
         <material name="RollLinks" />
       </visual>
-      <collision name="${side}_wrist_roll_collision">
-        <origin xyz="0.0 0 0" rpy="0 0 0" />
-        <geometry name="${side}_wrist_roll_collision_geom">
-          <box size="0.01 0.01 0.01" />
+      <collision>
+        <origin xyz="0 0 0" rpy="0 0 0" />
+        <geometry>
+          <mesh filename="package://pr2_description/meshes/forearm_v0/wrist_roll_L.stl" />
         </geometry>
         <verbose value="Yes" />

File: pr2_description/urdf/head_v0/head.urdf.xacro (robot description, xacro)
@@ -34,7 +34,7 @@
       </visual>
       <collision>
-        <origin xyz="-0.005717  0.010312 -0.029649" rpy="0.0 0.0 0.0 " />
+        <origin xyz="0 0 0.0" rpy="0 0 0 " />
         <geometry>
-          <box size="0.188 0.219 0.137" />
+          <mesh filename="package://pr2_description/meshes/head_v0/head_pan_L.stl"  />
         </geometry>
       </collision>
@@ -72,7 +72,7 @@
       </visual>
       <collision>
-        <origin xyz="0.041935 0.003569 0.028143" rpy="0 0 0" />
+        <origin xyz="0 0 0" rpy="0.0 0.0 0.0" />
         <geometry>
-          <box size="0.064 0.253 0.181" />
+          <mesh filename="package://pr2_description/meshes/head_v0/head_tilt_L.stl"  />
         </geometry>
       </collision>

File: pr2_description/urdf/head_v1/head.urdf.xacro (robot description, xacro)
@@ -34,7 +34,6 @@
       </visual>
       <collision>
-        <origin xyz="-0.005717  0.010312 -0.029649" rpy="0.0 0.0 0.0 " />
         <geometry>
-          <box size="0.188 0.219 0.137" />
+          <mesh filename="package://pr2_description/meshes/head_v0/head_pan_L.stl"  />
         </geometry>
       </collision>
@@ -72,7 +71,7 @@
       </visual>
       <collision>
-        <origin xyz="0.041935 0.003569 0.028143" rpy="0 0 0" />
+        <origin xyz="0 0 0" rpy="0.0 0.0 0.0" />
         <geometry>
-          <box size="0.064 0.253 0.181" />
+          <mesh filename="package://pr2_description/meshes/head_v0/head_tilt_L.stl"  />
         </geometry>
       </collision>

File: pr2_description/urdf/shoulder_v0/shoulder.urdf.xacro (robot description, xacro)
@@ -45,5 +45,5 @@
         <material name="Blue" />
       </visual>
-      <collision name="${side}_shoulder_pan_collision">
+      <collision>
         <origin xyz="0.0 0 0.0" rpy="0 0 0" />
         <geometry>
@@ -82,5 +82,5 @@
         <material name="Grey" />
       </visual>
-      <collision name="${side}_shoulder_lift_collision">
+      <collision>
         <origin xyz="0 0 0" rpy="0 0 0" />
         <geometry>
@@ -127,9 +127,8 @@
         <material name="RollLinks" />
       </visual>
-      <collision name="${side}_upper_arm_roll_collision">
-        <!-- TODO: collision tag should be optional -->
-        <origin xyz="0.0 0 0" rpy="0 0 0" />
+      <collision>
+        <origin xyz="0 0 0" rpy="0 0 0" />
         <geometry>
-          <box size="0.1 0.1 0.1" />
+          <mesh filename="package://pr2_description/meshes/shoulder_v0/upper_arm_roll_L.stl"  />
         </geometry>
       </collision>

File: pr2_description/urdf/shoulder_v1/shoulder.urdf.xacro (robot description, xacro)
@@ -45,5 +45,5 @@
         <material name="Blue" />
       </visual>
-      <collision name="${side}_shoulder_pan_collision">
+      <collision>
         <origin xyz="0.0 0 0.0" rpy="0 0 0" />
         <geometry>
@@ -82,5 +82,5 @@
         <material name="Grey" />
       </visual>
-      <collision name="${side}_shoulder_lift_collision">
+      <collision>
         <origin xyz="0 0 0" rpy="0 0 0" />
         <geometry>
@@ -123,13 +123,12 @@
         <origin xyz="0 0 0" rpy="0 0 0" />
         <geometry>
-          <mesh filename="package://pr2_description/meshes/shoulder_v1/upper_arm_roll.dae"  />
+          <mesh filename="package://pr2_description/meshes/shoulder_v0/upper_arm_roll.stl"  />
         </geometry>
         <material name="RollLinks" />
       </visual>
-      <collision name="${side}_upper_arm_roll_collision">
-        <!-- TODO: collision tag should be optional -->
-        <origin xyz="0.0 0 0" rpy="0 0 0" />
+      <collision>
+        <origin xyz="0 0 0" rpy="0 0 0" />
         <geometry>
-          <box size="0.1 0.1 0.1" />
+          <mesh filename="package://pr2_description/meshes/shoulder_v0/upper_arm_roll_L.stl"  />
         </geometry>
       </collision>

File: pr2_description/urdf/tilting_laser_v0/tilting_laser.urdf.xacro (robot description, xacro)
@@ -34,8 +34,8 @@
         <material name="Red" />
       </visual>
-      <collision name="${name}_mount_collision">
+      <collision>
         <origin xyz="0 0 0" rpy="0 0 0" />
         <geometry>
-          <box size=".001 .001 .001" />
+          <mesh filename="package://pr2_description/meshes/tilting_laser_v0/tilting_hokuyo_L.stl" />
         </geometry>
       </collision>

File: pr2_description/urdf/tilting_laser_v1/tilting_laser.urdf.xacro (robot description, xacro)
@@ -34,8 +34,8 @@
         <material name="Red" />
       </visual>
-      <collision name="${name}_mount_collision">
+      <collision>
         <origin xyz="0 0 0" rpy="0 0 0" />
         <geometry>
-          <box size=".001 .001 .001" />
+          <mesh filename="package://pr2_description/meshes/tilting_laser_v0/tilting_hokuyo_L.stl" />
         </geometry>
       </collision>

File: pr2_description/urdf/torso_v0/torso.urdf.xacro (robot description, xacro)
@@ -34,8 +34,7 @@
       </visual>
       <collision name="${name}_collision">
-        <origin xyz="0 0 0.16" rpy="0 0 0" />
+        <origin xyz="0 0 0" rpy="0 0 0" />
         <geometry>
-          <!-- arbitrarily chosen collision box by JH, torso collision is not important for now -->
-          <box size="0.30 0.620 0.02" />
+          <mesh filename="package://pr2_description/meshes/torso_v0/torso_lift_L.stl"  />
         </geometry>
       </collision>

File: pr2_description/urdf/torso_v1/torso.urdf.xacro (robot description, xacro)
@@ -34,8 +34,7 @@
       </visual>
       <collision name="${name}_collision">
-        <origin xyz="0 0 0.16" rpy="0 0 0" />
+        <origin xyz="0 0 0" rpy="0 0 0" />
         <geometry>
-          <!-- arbitrarily chosen collision box by JH, torso collision is not important for now -->
-          <box size="0.30 0.620 0.02" />
+          <mesh filename="package://pr2_description/meshes/torso_v0/torso_lift_L.stl"  />
         </geometry>
       </collision>

File: pr2_description/urdf/upper_arm_v0/upper_arm.urdf.xacro (robot description, xacro)
@@ -99,5 +99,5 @@
         <material name="Grey" />
       </visual>
-      <collision name="${side}_elbow_flex_collision">
+      <collision>
         <origin xyz="0 0 0" rpy="0 0 0" />
         <geometry>
@@ -141,9 +141,8 @@
       </visual>
       <!-- TODO: collision tag should be optional -->
-      <collision name="${side}_forearm_roll_collision">
-        <!-- dummy geom, to be removed -->
+      <collision>
         <origin xyz="0 0 0" rpy="0 0 0" />
         <geometry>
-          <box size="0.1 0.1 0.1" />
+          <mesh filename="package://pr2_description/meshes/upper_arm_v0/forearm_roll_L.stl"  />
         </geometry>
       </collision>

File: pr2_description/urdf/upper_arm_v1/upper_arm.urdf.xacro (robot description, xacro)
@@ -99,5 +99,5 @@
         <material name="Grey" />
       </visual>
-      <collision name="${side}_elbow_flex_collision">
+      <collision>
         <origin xyz="0 0 0" rpy="0 0 0" />
         <geometry>
@@ -141,9 +141,8 @@
       </visual>
       <!-- TODO: collision tag should be optional -->
-      <collision name="${side}_forearm_roll_collision">
-        <!-- dummy geom, to be removed -->
+      <collision>
         <origin xyz="0 0 0" rpy="0 0 0" />
         <geometry>
-          <box size="0.1 0.1 0.1" />
+          <mesh filename="package://pr2_description/meshes/upper_arm_v0/forearm_roll_L.stl"  />
         </geometry>
       </collision>
