Commit message: switched default to collada (dae) visual meshes and removed collada test urdf's.

File: pr2_description/urdf/base_v0/base.gazebo.xacro (robot description, xacro)
@@ -10,5 +10,4 @@
       <kp  value="1000000.0" />
       <kd  value="1.0" />
-      <material value="PR2/wheel_${suffix}" />
     </gazebo>
   </xacro:macro>
@@ -31,5 +30,4 @@
         </controller:gazebo_ros_bumper>
       </sensor:contact>
-      <material value="PR2/caster_texture" />
     </gazebo>
     <gazebo>

File: pr2_description/urdf/base_v0/base.urdf.xacro (robot description, xacro)
@@ -58,5 +58,5 @@
         <origin xyz="0 0 0" rpy="0 0 0" />
         <geometry>
-          <mesh filename="package://pr2_description/meshes/base_v0/wheel.stl" />
+          <mesh filename="package://pr2_description/meshes/base_v0/wheel.dae" />
         </geometry>
         <material name="Wheel_${suffix}" />
@@ -132,5 +132,5 @@
         <origin xyz="0 0 0" rpy="0 0 0" />
         <geometry>
-          <mesh filename="package://pr2_description/meshes/base_v0/base.stl" />
+          <mesh filename="package://pr2_description/meshes/base_v0/base.dae" />
         </geometry>
         <material name="White" />

File: pr2_description/urdf/forearm_v0/forearm.gazebo.xacro (robot description, xacro)
@@ -31,5 +31,4 @@
         </controller:gazebo_ros_bumper>
       </sensor:contact>
-      <material value="PR2/Grey" />
     </gazebo>
     <gazebo reference="${side}_wrist_flex_joint">

File: pr2_description/urdf/forearm_v0/forearm.urdf.xacro (robot description, xacro)
@@ -28,5 +28,5 @@
         <origin xyz="0 0 0" rpy="0 0 0" />
         <geometry>
-          <mesh filename="package://pr2_description/meshes/forearm_v0/forearm.stl" />
+          <mesh filename="package://pr2_description/meshes/forearm_v0/forearm.dae" />
        </geometry>
         <material name="Grey" />
@@ -62,5 +62,5 @@
         <origin xyz="0 0 0" rpy="0 0 0" />
         <geometry>
-          <mesh filename="package://pr2_description/meshes/forearm_v0/wrist_flex.stl" />
+          <mesh filename="package://pr2_description/meshes/forearm_v0/wrist_flex.dae" />
         </geometry>
         <material name="Grey" />

File: pr2_description/urdf/gripper_v0/gripper.gazebo.xacro (robot description, xacro)
@@ -36,5 +36,4 @@
       <kp value="1000000.0" />
       <kd value="1.0" />
-      <material value="PR2/Grey" />
       <!-- for "${prefix}_l_finger_joint"-->
     </gazebo>
@@ -62,5 +61,4 @@
       <kp value="1000000.0" />
       <kd value="1.0" />
-      <material value="PR2/Grey" />
     </gazebo>
     <gazebo reference="${prefix}_r_finger_joint">
@@ -88,5 +86,4 @@
       <kp  value="10000000.0" />
       <kd  value="1.0" />
-      <material value="PR2/Grey" />
     </gazebo>
     <gazebo reference="${prefix}_l_finger_tip_joint">
@@ -114,5 +111,4 @@
       <kp  value="10000000.0" />
       <kd  value="1.0" />
-      <material value="PR2/Grey" />
     </gazebo>
     <gazebo>
@@ -186,5 +182,4 @@
         </controller:gazebo_ros_bumper>
       </sensor:contact>
-      <material value="PR2/Grey" />
     </gazebo>
     <gazebo>

File: pr2_description/urdf/gripper_v0/gripper.urdf.xacro (robot description, xacro)
@@ -49,5 +49,5 @@
         <origin xyz="0 0 0" rpy="0 0 0" />
         <geometry>
-          <mesh filename="package://pr2_description/meshes/gripper_v0/l_finger.stl" />
+          <mesh filename="package://pr2_description/meshes/gripper_v0/l_finger.dae" />
         </geometry>
         <material name="Grey" />
@@ -85,5 +85,5 @@
         <origin xyz="0 0 0" rpy="${M_PI} 0 0" />
         <geometry>
-          <mesh filename="package://pr2_description/meshes/gripper_v0/l_finger.stl" />
+          <mesh filename="package://pr2_description/meshes/gripper_v0/l_finger.dae" />
         </geometry>
         <material name="Grey" />
@@ -193,5 +193,5 @@
         <origin xyz="0 0 0" rpy="0 0 0" />
         <geometry>
-          <mesh filename="package://pr2_description/meshes/gripper_v0/l_finger_tip.stl" />
+          <mesh filename="package://pr2_description/meshes/gripper_v0/l_finger_tip.dae" />
         </geometry>
         <material name="Green" />
@@ -226,5 +226,5 @@
         <origin xyz="0 0 0" rpy="${M_PI} 0 0" />
         <geometry>
-          <mesh filename="package://pr2_description/meshes/gripper_v0/l_finger_tip.stl"  />
+          <mesh filename="package://pr2_description/meshes/gripper_v0/l_finger_tip.dae"  />
         </geometry>
         <material name="Green" />
@@ -258,5 +258,5 @@
         <origin xyz="0 0 0" rpy="0 0 0" />
         <geometry>
-          <mesh filename="package://pr2_description/meshes/gripper_v0/gripper_palm.stl"  />
+          <mesh filename="package://pr2_description/meshes/gripper_v0/gripper_palm.dae"  />
         </geometry>
         <material name="Red" />

File: pr2_description/urdf/head_v0/head.gazebo.xacro (robot description, xacro)
@@ -4,14 +4,4 @@
        xmlns:interface="http://playerstage.sourceforge.net/gazebo/xmlschema/#interface"
        xmlns:xacro="http://ros.org/wiki/xacro">
-  <xacro:macro name="pr2_head_pan_gazebo_v0" params="name">
-    <gazebo reference="${name}_link">
-      <material value="Gazebo/Black" />
-    </gazebo>
-  </xacro:macro>
-  <xacro:macro name="pr2_head_tilt_gazebo_v0" params="name">
-    <gazebo reference="${name}_link">
-      <material value="Gazebo/White" />
-    </gazebo>
-  </xacro:macro>
   <xacro:macro name="pr2_head_gazebo_v0" params="name">
     <gazebo reference="${name}_plate_frame">

File: pr2_description/urdf/head_v0/head.urdf.xacro (robot description, xacro)
@@ -29,10 +29,9 @@
         <origin xyz="0 0 0.0" rpy="0 0 0 " />
         <geometry>
-          <mesh filename="package://pr2_description/meshes/head_v0/head_pan.stl"  />
+          <mesh filename="package://pr2_description/meshes/head_v0/head_pan.dae"  />
         </geometry>
         <material name="Blue" />
       </visual>
       <collision>
-        <origin xyz="0 0 0.0" rpy="0 0 0 " />
         <geometry>
           <mesh filename="package://pr2_description/meshes/head_v0/head_pan_L.stl"  />
@@ -67,5 +66,5 @@
         <origin xyz="0 0 0" rpy="0.0 0.0 0.0" />
         <geometry>
-          <mesh filename="package://pr2_description/meshes/head_v0/head_tilt.stl"  />
+          <mesh filename="package://pr2_description/meshes/head_v0/head_tilt.dae"  />
         </geometry>
         <material name="Green" />

File: pr2_description/urdf/shoulder_v0/shoulder.gazebo.xacro (robot description, xacro)
@@ -17,5 +17,4 @@
         </controller:gazebo_ros_bumper>
       </sensor:contact>
-      <material value="PR2/Grey" />
       <turnGravityOff>true</turnGravityOff>
     </gazebo>

File: pr2_description/urdf/shoulder_v0/shoulder.urdf.xacro (robot description, xacro)
@@ -41,5 +41,5 @@
         <origin xyz="0 0 0" rpy="0 0 0" />
         <geometry>
-          <mesh filename="package://pr2_description/meshes/shoulder_v0/shoulder_pan.stl"  />
+          <mesh filename="package://pr2_description/meshes/shoulder_v0/shoulder_pan.dae"  />
         </geometry>
         <material name="Blue" />
@@ -78,5 +78,5 @@
         <origin xyz="0 0 0" rpy="0 0 0" />
         <geometry>
-          <mesh filename="package://pr2_description/meshes/shoulder_v0/shoulder_lift.stl"  />
+          <mesh filename="package://pr2_description/meshes/shoulder_v0/shoulder_lift.dae"  />
         </geometry>
         <material name="Grey" />

File: pr2_description/urdf/tilting_laser_v0/tilting_laser.gazebo.xacro (robot description, xacro)
@@ -6,5 +6,4 @@
   <xacro:macro name="pr2_tilting_laser_gazebo_v0" params="name">
     <gazebo reference="${name}_mount_link">
-      <material value="Gazebo/Grey" />
     </gazebo>
   </xacro:macro>

File: pr2_description/urdf/tilting_laser_v0/tilting_laser.urdf.xacro (robot description, xacro)
@@ -30,5 +30,5 @@
         <origin xyz="0 0 0" rpy="0 0 0" />
         <geometry>
-          <mesh filename="package://pr2_description/meshes/tilting_laser_v0/tilting_hokuyo.stl" />
+          <mesh filename="package://pr2_description/meshes/tilting_laser_v0/tilting_hokuyo.dae" />
         </geometry>
         <material name="Red" />

File: pr2_description/urdf/torso_v0/torso.gazebo.xacro (robot description, xacro)
@@ -16,5 +16,4 @@
         </controller:gazebo_ros_bumper>
       </sensor:contact>
-      <material value="PR2/Grey2" />
     </gazebo>
   </xacro:macro>

File: pr2_description/urdf/torso_v0/torso.urdf.xacro (robot description, xacro)
@@ -29,5 +29,5 @@
         <origin xyz="0 0 0" rpy="0 0 0" />
         <geometry>
-          <mesh filename="package://pr2_description/meshes/torso_v0/torso_lift.stl"  />
+          <mesh filename="package://pr2_description/meshes/torso_v0/torso_lift.dae"  />
         </geometry>
         <material name="Grey2" />

File: pr2_description/urdf/upper_arm_v0/upper_arm.gazebo.xacro (robot description, xacro)
@@ -36,5 +36,4 @@
         </controller:gazebo_ros_bumper>
       </sensor:contact>
-      <material value="PR2/Grey" />
       <turnGravityOff>true</turnGravityOff>
     </gazebo>

File: pr2_description/urdf/upper_arm_v0/upper_arm.urdf.xacro (robot description, xacro)
@@ -52,5 +52,5 @@
         <origin xyz="0 0 0" rpy="0 0 0" />
         <geometry>
-          <mesh filename="package://pr2_description/meshes/upper_arm_v0/upper_arm.stl"  />
+          <mesh filename="package://pr2_description/meshes/upper_arm_v0/upper_arm.dae"  />
         </geometry>
         <material name="Green" />
@@ -95,5 +95,5 @@
         <origin xyz="0 0 0" rpy="0 0 0" />
         <geometry>
-          <mesh filename="package://pr2_description/meshes/upper_arm_v0/elbow_flex.stl"  />
+          <mesh filename="package://pr2_description/meshes/upper_arm_v0/elbow_flex.dae"  />
         </geometry>
         <material name="Grey" />

Commit message: added bellow, turned off self collide.  At highest torso_lift position, there's a small gap, need to add overlapping bellow from the top down.

File: pr2_description/urdf/base_v0/base.gazebo.xacro (robot description, xacro)
@@ -19,5 +19,5 @@
   <xacro:macro name="pr2_base_gazebo_v0" params="name">
     <gazebo reference="${name}_link">
-      <selfCollide>true</selfCollide>
+      <selfCollide>false</selfCollide>
       <sensor:contact name="${name}_contact_sensor">
         <geom>${name}_link_geom</geom>
@@ -30,4 +30,7 @@
         </controller:gazebo_ros_bumper>
       </sensor:contact>
+    </gazebo>
+    <gazebo reference="${name}_bellow_link">
+      <material value="PR2/Black" />
     </gazebo>
     <gazebo>

File: pr2_description/urdf/base_v0/base.urdf.xacro (robot description, xacro)
@@ -173,4 +173,32 @@
       <parent link="${name}_footprint"/>
     </joint>
+    <!-- visualize bellow -->
+    <link name="${name}_bellow_link">
+      <inertial>
+        <mass value="1.0" />
+        <origin xyz="0 0 0" />
+        <inertia ixx="0.01" ixy="0.0" ixz="0.0"
+                 iyy="0.01" iyz="0.0" izz="0.01" />
+      </inertial>
+      <visual>
+        <origin xyz="0 0 0" rpy="0 0 0" />
+        <geometry>
+          <box size="0.05 0.37 0.3" />
+        </geometry>
+        <material name="Black" />
+      </visual>
+      <collision>
+        <origin xyz="0 0 0" rpy="0 0 0" />
+        <geometry>
+          <box size="0.05 0.37 0.3" />
+        </geometry>
+        <material name="Black" />
+      </collision>
+    </link>
+    <joint name="${name}_bellow_joint" type="fixed">
+      <origin xyz="-0.29 0 0.8" rpy="0 0 0" />
+      <parent link="${name}_link" />
+      <child link="${name}_bellow_link"/>
+    </joint>
     <!-- base laser -->
     <xacro:hokuyo_lx30_laser_v0 name="${name}_laser" parent="${name}" ros_topic="base_scan" update_rate="20" min_angle="-2.2689" max_angle="2.2689" >

Commit message: changed default collision name suffix from _geom to _collision

File: pr2_description/urdf/base_v0/base.gazebo.xacro (robot description, xacro)
@@ -23,5 +23,5 @@
         <update_rate>100.0</update_rate>
         <contact>
-          <collision>${name}_link_geom</collision>
+          <collision>${name}_link_collision</collision>
         </contact>
         <plugin name="${name}_gazebo_ros_bumper_controller" filename="libgazebo_ros_bumper.so">

File: pr2_description/urdf/gripper_v0/gripper.gazebo.xacro (robot description, xacro)
@@ -57,5 +57,5 @@
         <update_rate>100.0</update_rate>
         <contact>
-          <collision>${prefix}_l_finger_tip_link_geom</collision>
+          <collision>${prefix}_l_finger_tip_link_collision</collision>
         </contact>
         <plugin name="${prefix}_l_finger_tip_gazebo_ros_bumper_controller" filename="libgazebo_ros_bumper.so">
@@ -84,5 +84,5 @@
         <update_rate>100.0</update_rate>
         <contact>
-          <collision>${prefix}_r_finger_tip_link_geom</collision>
+          <collision>${prefix}_r_finger_tip_link_collision</collision>
         </contact>
         <plugin name="${prefix}_r_finger_tip_gazebo_ros_bumper_controller" filename="libgazebo_ros_bumper.so">

File: pr2_description/urdf/torso_v0/torso.gazebo.xacro (robot description, xacro)
@@ -10,5 +10,5 @@
         <update_rate>100.0</update_rate>
         <contact>
-          <collision>${name}_link_geom</collision>
+          <collision>${name}_link_collision</collision>
         </contact>
         <plugin name="${name}_gazebo_ros_bumper_controller" filename="libgazebo_ros_bumper.so">

Commit message: update gripper joint gazebo extensions (got parent child reversed)

File: pr2_description/urdf/base_v0/base.gazebo.xacro (robot description, xacro)
@@ -10,4 +10,5 @@
       <kp  value="1000000.0" />
       <kd  value="1.0" />
+      <maxVel  value="1000.0" />
     </gazebo>
   </xacro:macro>

File: pr2_description/urdf/gripper_v0/gripper.gazebo.xacro (robot description, xacro)
@@ -7,6 +7,6 @@
        xmlns:geom="http://playerstage.sourceforge.net/gazebo/xmlschema/#geom"
        xmlns:xacro="http://ros.org/wiki/xacro">
-  <property name="finger_stop_kd"             value="1.0" />
-  <property name="finger_stop_kp"             value="0.001" />
+  <property name="finger_stop_erp"             value="0.0" />
+  <property name="finger_stop_cfm"             value="0.1" />
   <property name="finger_fudge_factor"        value="1.0" />
   <property name="finger_kp"                  value="0.0" />
@@ -31,6 +31,6 @@
     </gazebo>
     <gazebo reference="${prefix}_l_finger_joint">
-      <stop_erp value="${finger_stop_kd}" />
-      <stop_cfm value="${finger_stop_kp}" />
+      <stop_erp value="${finger_stop_erp}" />
+      <stop_cfm value="${finger_stop_cfm}" />
       <fudge_factor value="${finger_fudge_factor}" />
       <provideFeedback value="true"/>
@@ -45,6 +45,6 @@
     </gazebo>
     <gazebo reference="${prefix}_r_finger_joint">
-      <stop_erp value="${finger_stop_kd}" />
-      <stop_cfm value="${finger_stop_kp}" />
+      <stop_erp value="${finger_stop_erp}" />
+      <stop_cfm value="${finger_stop_cfm}" />
       <fudge_factor value="${finger_fudge_factor}" />
       <provideFeedback value="true"/>
@@ -72,6 +72,6 @@
     </gazebo>
     <gazebo reference="${prefix}_l_finger_tip_joint">
-      <stop_erp value="${finger_stop_kd}" />
-      <stop_cfm value="${finger_stop_kp}" />
+      <stop_erp value="${finger_stop_erp}" />
+      <stop_cfm value="${finger_stop_cfm}" />
       <fudge_factor value="${finger_fudge_factor}" />
       <provideFeedback value="true"/>
@@ -116,6 +116,6 @@
     </gazebo>
     <gazebo reference="${prefix}_r_finger_tip_joint">
-      <stop_erp value="${finger_stop_kd}" />
-      <stop_cfm value="${finger_stop_kp}" />
+      <stop_erp value="${finger_stop_erp}" />
+      <stop_cfm value="${finger_stop_cfm}" />
       <fudge_factor value="${finger_fudge_factor}" />
       <provideFeedback value="true"/>
@@ -160,6 +160,6 @@
     <gazebo>
       <joint type="screw" name="${prefix}_r_screw_screw_joint">
-          <parent>${prefix}_motor_screw_link</parent>
-          <child>${prefix}_r_finger_tip_link</child>
+          <child>${prefix}_motor_screw_link</child>
+          <parent>${prefix}_r_finger_tip_link</parent>
           <pose>0 0 0 0 0 0</pose>
           <axis>
@@ -169,6 +169,6 @@
       </joint>
       <joint type="screw" name="${prefix}_l_screw_screw_joint">
-          <parent>${prefix}_motor_screw_link</parent>
-          <child>${prefix}_l_finger_tip_link</child>
+          <child>${prefix}_motor_screw_link</child>
+          <parent>${prefix}_l_finger_tip_link</parent>
           <pose>0 0 0 0 0 0</pose>
           <axis>
@@ -180,6 +180,6 @@
     <gazebo>
       <joint type="revolute" name="${prefix}_r_parallel_root_joint">
-          <child>${prefix}_r_parallel_link</child>
-          <parent>${prefix}_palm_link</parent>
+          <parent>${prefix}_r_parallel_link</parent>
+          <child>${prefix}_palm_link</child>
           <axis>
             <xyz>0 0 -1</xyz>
@@ -191,6 +191,6 @@
       </joint>
       <joint type="revolute" name="${prefix}_l_parallel_root_joint">
-          <child>${prefix}_l_parallel_link</child>
-          <parent>${prefix}_palm_link</parent>
+          <parent>${prefix}_l_parallel_link</parent>
+          <child>${prefix}_palm_link</child>
           <axis>
             <xyz>0 0 1</xyz>
@@ -202,22 +202,22 @@
       </joint>
       <joint type="revolute" name="${prefix}_r_parallel_tip_joint">
-          <child>${prefix}_r_parallel_link</child>
+          <parent>${prefix}_r_parallel_link</parent>
+          <child>${prefix}_r_finger_tip_link</child>
+          <axis>
+            <xyz>0 0 1</xyz>
+          </axis>
+          <pose>${parallel_link_x_offset} ${-parallel_link_y_offset} 0 0 0 0</pose>
+      </joint>
+      <joint type="revolute" name="${prefix}_l_parallel_tip_joint">
+          <parent>${prefix}_l_parallel_link</parent>
+          <child>${prefix}_l_finger_tip_link</child>
+          <axis>
+            <xyz>0 0 1</xyz>
+          </axis>
+          <pose>${parallel_link_x_offset} ${parallel_link_y_offset} 0 0 0 0</pose>
+      </joint>
+      <joint type="prismatic" name="${prefix}_joint">
+          <child>${prefix}_l_finger_tip_link</child>
           <parent>${prefix}_r_finger_tip_link</parent>
-          <axis>
-            <xyz>0 0 1</xyz>
-          </axis>
-          <pose>${parallel_link_x_offset} ${-parallel_link_y_offset} 0 0 0 0</pose>
-      </joint>
-      <joint type="revolute" name="${prefix}_l_parallel_tip_joint">
-          <child>${prefix}_l_parallel_link</child>
-          <parent>${prefix}_l_finger_tip_link</parent>
-          <axis>
-            <xyz>0 0 1</xyz>
-          </axis>
-          <pose>${parallel_link_x_offset} ${parallel_link_y_offset} 0 0 0 0</pose>
-      </joint>
-      <joint type="prismatic" name="${prefix}_joint">
-          <parent>${prefix}_l_finger_tip_link</parent>
-          <child>${prefix}_r_finger_tip_link</child>
           <axis>
             <xyz>0 1 0</xyz>

Commit message: when using ROS Indigo and Gazebo 2.2.3, the name specified here must be <link_name>_collision

File: pr2_description/urdf/base_v0/base.gazebo.xacro (robot description, xacro)
@@ -23,5 +23,5 @@
         <update_rate>100.0</update_rate>
         <contact>
-          <collision>${name}_link_geom</collision>
+          <collision>${name}_link_collision</collision>
         </contact>
         <plugin name="${name}_gazebo_ros_bumper_controller" filename="libgazebo_ros_bumper.so">

File: pr2_description/urdf/gripper_v0/gripper.gazebo.xacro (robot description, xacro)
@@ -51,5 +51,5 @@
         <update_rate>100.0</update_rate>
         <contact>
-          <collision>${prefix}_l_finger_tip_link_geom</collision>
+          <collision>${prefix}_l_finger_tip_link_collision</collision>
         </contact>
         <plugin name="${prefix}_l_finger_tip_gazebo_ros_bumper_controller" filename="libgazebo_ros_bumper.so">
@@ -78,5 +78,5 @@
         <update_rate>100.0</update_rate>
         <contact>
-          <collision>${prefix}_r_finger_tip_link_geom</collision>
+          <collision>${prefix}_r_finger_tip_link_collision</collision>
         </contact>
         <plugin name="${prefix}_r_finger_tip_gazebo_ros_bumper_controller" filename="libgazebo_ros_bumper.so">

File: pr2_description/urdf/torso_v0/torso.gazebo.xacro (robot description, xacro)
@@ -5,5 +5,5 @@
       <sensor type="contact" name="${name}_contact_sensor">
         <contact>
-          <collision>${name}_link_geom</collision>
+          <collision>${name}_link_collision</collision>
         </contact>
         <update_rate>100.0</update_rate>
