Commit message: minor fixes for mesh and arm parent.

File: pr2_description/urdf/base_v0/base.urdf.xacro (robot description, xacro)
@@ -54,5 +54,5 @@
         <origin xyz="0 0 0" rpy="0 0 0" />
         <geometry name="${parent}_${suffix}_wheel_visual_geom">
-          <mesh filename="package://pre_description/meshes/base_v0/pr2_wheel.stl" />
+          <mesh filename="package://pr2_defs/meshes/pr2_wheel.stl" />
         </geometry>
         <material name="Caster_${suffix}" />
@@ -90,5 +90,5 @@
         <origin xyz="0 0 0" rpy="0 0 0" />
         <geometry name="${suffix}_caster_rotation_visual_geom">
-          <mesh filename="package://pr2_description/meshes/base_v0/caster.stl" />
+          <mesh filename="package://pr2_defs/meshes/caster.stl" />
         </geometry>
         <material name="Green" />
@@ -123,5 +123,5 @@
         <origin xyz="0 0 ${base_height_offset}" rpy="0 0 0" />
         <geometry name="${name}_visual_geom">
-          <mesh filename="package://pr2_description/meshes/base_v0/base.stl" />
+          <mesh filename="package://pr2_defs/meshes/base.stl" />
         </geometry>
         <material name="Green" />

File: pr2_description/urdf/materials.urdf.xacro (robot description, xacro)
@@ -1,3 +1,30 @@
 <?xml version="1.0"?>
 <robot>
+  <material name="Blue">
+    <color rgba="0.0 0.0 0.8 1.0"/>
+  </material>
+  <material name="Green">
+    <color rgba="0.0 0.8 0.0 1.0"/>
+  </material>
+  <material name="Grey">
+    <color rgba="0.7 0.7 0.7 1.0"/>
+  </material>
+  <material name="Grey2">
+    <color rgba="0.9 0.9 0.9 1.0"/>
+  </material>
+  <material name="Red">
+    <color rgba="0.8 0.0 0.0 1.0"/>
+  </material>
+  <material name="White">
+    <color rgba="1.0 1.0 1.0 1.0"/>
+  </material>
+  <material name="Caster_l">
+    <texture filename="package://pr2_ogre/Media/materials/textures/pr2_wheel_left.png" />
+  </material>
+  <material name="Caster_r">
+    <texture filename="package://pr2_ogre/Media/materials/textures/pr2_wheel_right.png" />
+  </material>
+  <material name="RollLinks">
+    <texture filename="package://pr2_ogre/Media/materials/textures/pr2_wheel_left.png" />
+  </material>
 </robot>

Commit message: adding caster material

File: pr2_description/urdf/base_v0/base.urdf.xacro (robot description, xacro)
@@ -59,5 +59,5 @@
           <mesh filename="package://pr2_description/meshes/base_v0/pr2_wheel.stl" />
         </geometry>
-        <material name="Caster_${suffix}" />
+        <material name="Wheel_${suffix}" />
       </visual>
       <collision>
@@ -96,5 +96,5 @@
           <mesh filename="package://pr2_description/meshes/base_v0/caster.stl" />
         </geometry>
-        <material name="Green" />
+        <material name="Caster" />
       </visual>
       <collision>

File: pr2_description/urdf/materials.urdf.xacro (robot description, xacro)
@@ -19,8 +19,11 @@
     <color rgba="1.0 1.0 1.0 1.0"/>
   </material>
-  <material name="Caster_l">
+  <material name="Caster">
     <texture filename="package://pr2_ogre/Media/materials/textures/pr2_wheel_left.png" />
   </material>
-  <material name="Caster_r">
+  <material name="Wheel_l">
+    <texture filename="package://pr2_ogre/Media/materials/textures/pr2_wheel_left.png" />
+  </material>
+  <material name="Wheel_r">
     <texture filename="package://pr2_ogre/Media/materials/textures/pr2_wheel_right.png" />
   </material>

Commit message: added comments for velocity and effort limits (alpha tested) and for gripper passive joint limits.

File: pr2_description/urdf/base_v0/base.urdf.xacro (robot description, xacro)
@@ -40,5 +40,5 @@
     <joint name="${parent}_${suffix}_wheel_joint" type="continuous">
       <axis xyz="0 1 0" />
-      <limit effort="100" velocity="100"/>
+      <limit effort="100" velocity="100"/> <!-- alpha tested effort and velocity limits -->
       <safety_controller  k_velocity="10" />
       <dynamics damping="0.0" friction="0.0" />
@@ -76,5 +76,5 @@
     <joint name="${suffix}_rotation_joint" type="continuous">
       <axis xyz="0 0 1" />
-      <limit effort="100" velocity="100"/>
+      <limit effort="100" velocity="100"/> <!-- alpha tested velocity and effort limits -->
       <safety_controller  k_velocity="10" />
       <calibration reference_position="${ref_position}" />

File: pr2_description/urdf/forearm_v0/forearm.urdf.xacro (robot description, xacro)
@@ -42,5 +42,5 @@
     <joint name="${side}_wrist_flex_joint" type="revolute">
       <axis xyz="0 1 0" />
-      <limit upper="0.0" lower="-2.094" effort="10" velocity="${VELOCITY_LIMIT_SCALE*5.13}" />
+      <limit upper="0.0" lower="-2.094" effort="10" velocity="${VELOCITY_LIMIT_SCALE*5.13}" /> <!-- alpha tested velocity and effort limits -->
       <safety_controller k_position="20" k_velocity="4" soft_upper_limit="${0.0 - 0.10}" soft_lower_limit="${-2.094 + 0.10}" />
       <dynamics damping="0.1" />
@@ -75,5 +75,5 @@
     <joint name="${side}_wrist_roll_joint" type="continuous">
       <axis xyz="1 0 0" />
-      <limit effort="10" velocity="${VELOCITY_LIMIT_SCALE*6}" />
+      <limit effort="10" velocity="${VELOCITY_LIMIT_SCALE*6}" /> <!-- alpha tested velocity and effort limits -->
       <safety_controller k_velocity="2" />
       <dynamics damping="0.1" />

File: pr2_description/urdf/gripper_v0/gripper.urdf.xacro (robot description, xacro)
@@ -14,4 +14,9 @@
   <property name="finger_joint_effort_limit"  value="100.0" />
   <xacro:macro name="pr2_finger_limits_v0" params="reflect">
+    <!-- limits on passive finger and finger top joints without
+         transmission are not enforced by safety controllers.
+         The lower/upper limits and are enforced in PR2 simulation and
+         effort and velocity limits are ignored. This is also needed because
+         these joints are declared revolute rather than continuous.-->
     <limit effort="${finger_joint_effort_limit}" velocity="0.5"
            lower="${gripper_lower_angle}" upper="${gripper_upper_angle}" />
@@ -245,4 +250,5 @@
          velocity limit is the linear velocity limit at the gripper gap
          try and introduce a very stiff spring
+         The velocity and effort limits are alpha tested.
     -->
     <joint name="${side}_gripper_joint" type="prismatic">

File: pr2_description/urdf/head_v0/head.urdf.xacro (robot description, xacro)
@@ -10,5 +10,5 @@
     <joint name="${name}_joint" type="revolute">
       <axis xyz="0 0 1" />
-      <limit lower="-3.007" upper="3.007" effort="2.645" velocity="6" />
+      <limit lower="-3.007" upper="3.007" effort="2.645" velocity="6" /> <!-- alpha tested velocity and effort limits -->
       <safety_controller k_velocity="1.5" soft_lower_limit="${-3.007+0.15}" soft_upper_limit="${3.007-0.15}" k_position="100" />
       <calibration reference_position="${0.0+cal_head_pan_flag}" />
@@ -46,5 +46,5 @@
     <joint name="${name}_joint" type="revolute">
       <axis xyz="0 1 0" />
-      <limit lower="-0.471238" upper="1.39626" effort="15" velocity="5" />
+      <limit lower="-0.471238" upper="1.39626" effort="15" velocity="5" /> <!-- alpha tested velocity and effort limits -->
       <safety_controller k_velocity="1.5" soft_lower_limit="${-0.4712 + 0.1}" soft_upper_limit="${1.39626 - 0.1}" k_position="100" />
       <calibration reference_position="${0.0+cal_head_tilt_flag}" />

File: pr2_description/urdf/shoulder_v0/shoulder.urdf.xacro (robot description, xacro)
@@ -21,5 +21,5 @@
       <child link="${side}_shoulder_pan_link"/>
       <limit lower="${reflect*M_PI/4-1.5}"  upper="${reflect*M_PI/4+1.5}"
-             effort="30" velocity="${VELOCITY_LIMIT_SCALE*3.48}" />
+             effort="30" velocity="${VELOCITY_LIMIT_SCALE*3.48}" /> <!-- alpha tested velocity and effort limits -->
       <dynamics damping="10.0" />
       <safety_controller k_position="100" k_velocity="10"
@@ -56,5 +56,5 @@
       <!-- Limits updated from Function's CAD values as of 2009_02_24 (link_data.xls) -->
       <limit lower="-0.5236" upper="1.3963"
-             effort="30" velocity="${VELOCITY_LIMIT_SCALE*3.47}" />
+             effort="30" velocity="${VELOCITY_LIMIT_SCALE*3.47}" /> <!-- alpha tested velocity and effort limits -->
       <safety_controller k_position="100" k_velocity="10"
                          soft_lower_limit="${-0.5236+0.17}" soft_upper_limit="${1.3963-0.10}" />
@@ -93,5 +93,5 @@
       <parent link="${side}_shoulder_lift_link" />
       <child link="${side}_upper_arm_roll_link"/>
-      <limit lower="${reflect*1.55-2.35}" upper="${reflect*1.55+2.35}" effort="30" velocity="${VELOCITY_LIMIT_SCALE*5.45}" />
+      <limit lower="${reflect*1.55-2.35}" upper="${reflect*1.55+2.35}" effort="30" velocity="${VELOCITY_LIMIT_SCALE*5.45}" /> <!-- alpha tested velocity and effort limits -->
       <safety_controller k_position="100" k_velocity="2" soft_lower_limit="${reflect*1.55-2.35+0.15}" soft_upper_limit="${reflect*1.55+2.35-0.15}" />
       <calibration reference_position="${(reflect*M_PI/2)*cal_r_upper_arm_roll_gearing + cal_r_upper_arm_roll_flag}" />

File: pr2_description/urdf/tilting_laser_v0/tilting_laser.urdf.xacro (robot description, xacro)
@@ -10,5 +10,5 @@
     <joint name="${name}_mount_joint" type="revolute">
       <axis xyz="0 1 0" />
-      <limit lower="-0.7854" upper="1.48353" effort="0.65" velocity="10.0" />
+      <limit lower="-0.7854" upper="1.48353" effort="0.65" velocity="10.0" /> <!-- alpha tested velocity and effort limits -->
       <safety_controller k_position="100" k_velocity="0.05" soft_lower_limit="${-0.7854+0.05}" soft_upper_limit="${1.48353-0.05}" />
       <calibration reference_position="${laser_calib_ref}" />

File: pr2_description/urdf/torso_v0/torso.urdf.xacro (robot description, xacro)
@@ -10,5 +10,5 @@
     <joint name="${name}_joint" type="prismatic">
       <axis xyz="0 0 1" />
-      <limit lower="0.0" upper="0.31" effort="10000" velocity="0.013"/>
+      <limit lower="0.0" upper="0.31" effort="10000" velocity="0.013"/> <!-- alpha tested velocity and effort limits -->
       <safety_controller  k_velocity="400000" soft_lower_limit="${0.0+0.003}" soft_upper_limit="${0.31-0.005}" k_position="1000" />
       <calibration reference_position="0.00536" />

File: pr2_description/urdf/upper_arm_v0/upper_arm.urdf.xacro (robot description, xacro)
@@ -75,5 +75,5 @@
       <axis xyz="0 1 0" />
       <!-- Note: Overtravel limits are 140, -7 degrees instead of 133, 0 -->
-      <limit lower="-2.3213" upper="0.00" effort="30" velocity="${VELOCITY_LIMIT_SCALE*5.5}" />
+      <limit lower="-2.3213" upper="0.00" effort="30" velocity="${VELOCITY_LIMIT_SCALE*5.5}" /> <!-- alpha tested velocity and effort limits -->
       <safety_controller k_position="100" k_velocity="3" soft_lower_limit="${-2.3213+0.2}" soft_upper_limit="${0.00-0.15}" />
       <calibration reference_position="${-1.1606 + cal_r_elbow_flex_flag}"/>
@@ -113,5 +113,5 @@
     <joint name="${side}_forearm_roll_joint" type="continuous">
       <axis xyz="1 0 0" />
-      <limit effort="30" velocity="${VELOCITY_LIMIT_SCALE*6}" />
+      <limit effort="30" velocity="${VELOCITY_LIMIT_SCALE*6}" /> <!-- alpha tested velocity and effort limits -->
       <safety_controller k_velocity="1" />
       <calibration reference_position="${0.0 + cal_r_forearm_roll_flag}" />

Commit message: adding base_footprint link as a frame, for navigation usage.  see ticket #3428

File: pr2_description/urdf/base_v0/base.urdf.xacro (robot description, xacro)
@@ -144,4 +144,12 @@
       </collision>
     </link>
+    <!-- base_footprint is a fictitious link(frame) that is on the ground right below base_link origin,
+         navigation stack dedpends on this frame -->
+    <link name="${name}_footprint"/>
+    <joint name="${name}_footprint_joint" type="fixed">
+      <origin xyz="0 0 0.051" rpy="0 0 0" />
+      <parent link="${name}_link" />
+      <child link="${name}_footprint"/>
+    </joint>
     <!-- base laser -->
     <xacro:hokuyo_lx30_laser_v0 name="${name}_laser" parent="${name}" ros_topic="base_scan" update_rate="20" >

Commit message: oops, base_footprint offset wrong sign

File: pr2_description/urdf/base_v0/base.urdf.xacro (robot description, xacro)
@@ -148,5 +148,5 @@
     <link name="${name}_footprint"/>
     <joint name="${name}_footprint_joint" type="fixed">
-      <origin xyz="0 0 0.051" rpy="0 0 0" />
+      <origin xyz="0 0 -0.051" rpy="0 0 0" />
       <parent link="${name}_link" />
       <child link="${name}_footprint"/>

Commit message: gazebo updates for laser (add min/max angles) and imu (add standard deviation)

File: pr2_description/urdf/base_v0/base.urdf.xacro (robot description, xacro)
@@ -175,5 +175,5 @@
     </joint>
     <!-- base laser -->
-    <xacro:hokuyo_lx30_laser_v0 name="${name}_laser" parent="${name}" ros_topic="base_scan" update_rate="20" >
+    <xacro:hokuyo_lx30_laser_v0 name="${name}_laser" parent="${name}" ros_topic="base_scan" update_rate="20" min_angle="-2.2689" max_angle="2.2689" >
       <origin xyz="${base_laser_x} ${base_laser_y} ${base_laser_z}" rpy="0 0 0" />
     </xacro:hokuyo_lx30_laser_v0>

File: pr2_description/urdf/sensors/hokuyo_lx30_laser.gazebo.xacro (robot description, xacro)
@@ -4,5 +4,5 @@
        xmlns:interface="http://playerstage.sourceforge.net/gazebo/xmlschema/#interface"
        xmlns:xacro="http://ros.org/wiki/xacro">
-  <xacro:macro name="hokuyo_lx30_laser_gazebo_v0" params="name ros_topic update_rate">
+  <xacro:macro name="hokuyo_lx30_laser_gazebo_v0" params="name ros_topic update_rate min_angle max_angle">
     <gazebo reference="${name}_link">
       <sensor:ray name="${name}">
@@ -12,6 +12,6 @@
         <origin>0.0 0.0 0.0</origin>
         <displayRays>false</displayRays>
-        <minAngle>-80</minAngle>
-        <maxAngle> 80</maxAngle>
+        <minAngle>${min_angle*180.0/M_PI}</minAngle>
+        <maxAngle>${max_angle*180.0/M_PI}</maxAngle>
         <minRange>0.05</minRange>
         <maxRange>10.0</maxRange>

File: pr2_description/urdf/sensors/hokuyo_lx30_laser.urdf.xacro (robot description, xacro)
@@ -5,5 +5,5 @@
        xmlns:xacro="http://ros.org/wiki/xacro">
   <include filename="$(find pr2_description)/urdf/sensors/hokuyo_lx30_laser.gazebo.xacro" />
-  <xacro:macro name="hokuyo_lx30_laser_v0" params="name parent *origin ros_topic update_rate">
+  <xacro:macro name="hokuyo_lx30_laser_v0" params="name parent *origin ros_topic update_rate min_angle max_angle">
     <joint name="${name}_joint" type="fixed">
       <axis xyz="0 1 0" />
@@ -33,5 +33,5 @@
     </link>
     <!-- gazebo extensions -->
-    <xacro:hokuyo_lx30_laser_gazebo_v0 name="${name}" ros_topic="${ros_topic}" update_rate="${update_rate}" />
+    <xacro:hokuyo_lx30_laser_gazebo_v0 name="${name}" ros_topic="${ros_topic}" update_rate="${update_rate}" min_angle="${min_angle}" max_angle="${max_angle}" />
   </xacro:macro>
 </robot>

File: pr2_description/urdf/sensors/microstrain_3dmgx2_imu.gazebo.xacro (robot description, xacro)
@@ -3,5 +3,5 @@
        xmlns:interface="http://playerstage.sourceforge.net/gazebo/xmlschema/#interface"
        xmlns:xacro="http://ros.org/wiki/xacro">
-  <xacro:macro name="microstrain_3dmgx2_imu_gazebo_v0" params="name imu_topic update_rate">
+  <xacro:macro name="microstrain_3dmgx2_imu_gazebo_v0" params="name imu_topic update_rate stdev">
     <gazebo>
       <controller:gazebo_ros_imu name="imu_controller" plugin="libgazebo_ros_imu.so">
@@ -10,5 +10,5 @@
         <bodyName>${name}_link</bodyName>
         <topicName>${imu_topic}</topicName>
-        <gaussianNoise>0.01</gaussianNoise>
+        <gaussianNoise>${stdev*stdev}</gaussianNoise>
         <frameName>map</frameName>
         <xyzOffsets>0 0 0</xyzOffsets>

File: pr2_description/urdf/sensors/microstrain_3dmgx2_imu.urdf.xacro (robot description, xacro)
@@ -2,5 +2,5 @@
 <robot xmlns:xacro="http://ros.org/wiki/xacro">
   <include filename="$(find pr2_description)/urdf/sensors/microstrain_3dmgx2_imu.gazebo.xacro" />
-  <xacro:macro name="microstrain_3dmgx2_imu_v0" params="name parent *origin imu_topic update_rate">
+  <xacro:macro name="microstrain_3dmgx2_imu_v0" params="name parent *origin imu_topic update_rate stdev">
     <joint name="${name}_joint" type="fixed">
       <axis xyz="0 1 0" />
@@ -30,5 +30,5 @@
     </link>
     <!-- gazebo extensions -->
-    <xacro:microstrain_3dmgx2_imu_gazebo_v0 name="${name}" imu_topic="${imu_topic}" update_rate="${update_rate}" />
+    <xacro:microstrain_3dmgx2_imu_gazebo_v0 name="${name}" imu_topic="${imu_topic}" update_rate="${update_rate}" stdev="${stdev}" />
   </xacro:macro>
 </robot>

File: pr2_description/urdf/tilting_laser_v0/tilting_laser.urdf.xacro (robot description, xacro)
@@ -41,5 +41,5 @@
       </collision>
     </link>
-    <xacro:hokuyo_lx30_laser_v0 name="${name}" parent="${name}_mount" ros_topic="tilt_scan" update_rate="40" >
+    <xacro:hokuyo_lx30_laser_v0 name="${name}" parent="${name}_mount" ros_topic="tilt_scan" update_rate="20" min_angle="-1.3962634" max_angle="1.3962634" >
       <origin xyz="0 0 0.03" rpy="0 0 0" />
     </xacro:hokuyo_lx30_laser_v0>

File: pr2_description/urdf/torso_v0/torso.urdf.xacro (robot description, xacro)
@@ -45,5 +45,5 @@
     <xacro:pr2_torso_transmission_v0 name="${name}" />
     <!-- imu -->
-    <xacro:microstrain_3dmgx2_imu_v0 name="imu" parent="${name}" imu_topic="torso_lift_imu/data" update_rate="100.0">
+    <xacro:microstrain_3dmgx2_imu_v0 name="imu" parent="${name}" imu_topic="torso_lift_imu/data" update_rate="100.0" stdev="0.00017" >
         <origin xyz="-0.02977 -0.1497 0.164" rpy="0 0 0" />
     </xacro:microstrain_3dmgx2_imu_v0>
