Commit message: new beta meshes

File: pr2_description/urdf/base_v0/base.urdf.xacro (robot description, xacro)
@@ -57,5 +57,5 @@
         <origin xyz="0 0 0" rpy="0 0 0" />
         <geometry>
-          <mesh filename="package://pr2_description/meshes/base_v0/pr2_wheel.stl" />
+          <mesh filename="package://pr2_description/meshes/base_v0/wheel.stl" scale=".001 .001 .001"/>
         </geometry>
         <material name="Wheel_${suffix}" />
@@ -131,5 +131,5 @@
         <origin xyz="0 0 0" rpy="0 0 0" />
         <geometry>
-          <mesh filename="package://pr2_description/meshes/base_v0/base.stl" />
+          <mesh filename="package://pr2_description/meshes/base_v0/base.stl" scale=".001 .001 .001"/>
         </geometry>
         <material name="Green" />

File: pr2_description/urdf/forearm_v0/forearm.urdf.xacro (robot description, xacro)
@@ -28,5 +28,5 @@
         <origin xyz="0 0 0" rpy="0 0 0" />
         <geometry name="${side}_forearm_visual_geom">
-          <mesh filename="package://pr2_description/meshes/forearm_v0/forearm.stl" />
+          <mesh filename="package://pr2_description/meshes/forearm_v0/forearm.stl" scale=".001 .001 .001"/>
         </geometry>
         <material name="Blue" />
@@ -35,5 +35,5 @@
         <origin xyz="0 0 0" rpy="0 0 0" />
         <geometry name="${side}_forearm_collision_geom">
-          <mesh filename="package://pr2_description/meshes/forearm_v0/convex/forearm_convex.stlb" />
+          <mesh filename="package://pr2_description/meshes/forearm_v0/forearm.stl" scale=".001 .001 .001"/>
         </geometry>
       </collision>
@@ -62,5 +62,5 @@
         <origin xyz="0 0 0" rpy="0 0 0" />
         <geometry name="${side}_wrist_flex_visual_geom">
-          <mesh filename="package://pr2_description/meshes/forearm_v0/wrist_flex.stl" />
+          <mesh filename="package://pr2_description/meshes/forearm_v0/wrist_flex.stl" scale=".001 .001 .001"/>
         </geometry>
         <material name="Grey" />
@@ -69,5 +69,5 @@
         <origin xyz="0 0 0" rpy="0 0 0" />
         <geometry name="${side}_wrist_flex_collision_geom">
-          <mesh filename="package://pr2_description/meshes/forearm_v0/convex/wrist_flex_convex.stlb" />
+          <mesh filename="package://pr2_description/meshes/forearm_v0/wrist_flex.stl" scale=".001 .001 .001"/>
         </geometry>
       </collision>
@@ -97,5 +97,5 @@
         <origin xyz="0 0 0" rpy="0 0 0" />
         <geometry name="${side}_wrist_roll_visual_geom">
-          <mesh filename="package://pr2_description/meshes/forearm_v0/wrist_roll.stl" />
+          <mesh filename="package://pr2_description/meshes/forearm_v0/wrist_roll.stl" scale=".001 .001 .001"/>
         </geometry>
         <material name="RollLinks" />

File: pr2_description/urdf/gripper_v0/gripper.urdf.xacro (robot description, xacro)
@@ -46,8 +46,8 @@
                   izz= "0.00018105446" />
       </inertial>
-      <visual name="${prefix}_l_finger_visual">
-        <origin xyz="0 0 0" rpy="0 0 0" />
-        <geometry name="${prefix}_l_finger_visual_geom">
-          <mesh filename="package://pr2_description/meshes/gripper_v0/upper_finger_l.stl" />
+      <visual>
+        <origin xyz="0 0 0" rpy="0 0 0" />
+        <geometry>
+          <mesh filename="package://pr2_description/meshes/gripper_v0/l_finger.stl" scale=".001 .001 .001"/>
         </geometry>
         <material name="Grey" />
@@ -55,6 +55,6 @@
       <collision name="${prefix}_l_finger_collision">
         <origin xyz="0 0 0" rpy="0 0 0" />
-        <geometry name="${prefix}_l_finger_collision_geom">
-          <mesh filename="package://pr2_description/meshes/gripper_v0/upper_finger_l.stl" />
+        <geometry>
+          <mesh filename="package://pr2_description/meshes/gripper_v0/l_finger.stl" scale=".001 .001 .001"/>
         </geometry>
         <verbose value="Yes" />
@@ -82,15 +82,15 @@
                   izz= "0.00018106988" />
       </inertial>
-      <visual name="${prefix}_r_finger_visual">
-        <origin xyz="0 0 0" rpy="0 0 0" />
-        <geometry name="${prefix}_r_finger_visual_geom">
-          <mesh filename="package://pr2_description/meshes/gripper_v0/upper_finger_r.stl" />
+      <visual>
+        <origin xyz="0 0 0" rpy="${M_PI} 0 0" />
+        <geometry>
+          <mesh filename="package://pr2_description/meshes/gripper_v0/l_finger.stl" scale=".001 .001 .001"/>
         </geometry>
         <material name="Grey" />
       </visual>
       <collision name="${prefix}_r_finger_collision">
-        <origin xyz="0 0 0" rpy="0 0 0" />
-        <geometry name="${prefix}_r_finger_collision_geom">
-          <mesh filename="package://pr2_description/meshes/gripper_v0/upper_finger_r.stl" />
+        <origin xyz="0 0 0" rpy="${M_PI} 0 0" />
+        <geometry>
+          <mesh filename="package://pr2_description/meshes/gripper_v0/l_finger.stl" scale=".001 .001 .001"/>
         </geometry>
         <verbose value="Yes" />
@@ -186,8 +186,8 @@
                   izz="0.00001541768" />
       </inertial>
-      <visual name="${prefix}_l_finger_tip_visual">
-        <origin xyz="0 0 0" rpy="0 0 0" />
-        <geometry name="${prefix}_l_finger_tip_visual_geom">
-          <mesh filename="package://pr2_description/meshes/gripper_v0/finger_tip_l.stl" />
+      <visual>
+        <origin xyz="0 0 0" rpy="0 0 0" />
+        <geometry>
+          <mesh filename="package://pr2_description/meshes/gripper_v0/l_finger_tip.stl" scale=".001 .001 .001"/>
         </geometry>
         <material name="Green" />
@@ -195,6 +195,6 @@
       <collision name="${prefix}_l_finger_tip_collision">
         <origin xyz="0 0 0" rpy="0 0 0" />
-        <geometry name="${prefix}_l_finger_tip_collision_geom">
-          <mesh filename="package://pr2_description/meshes/gripper_v0/finger_tip_pad2_l.stl" />
+        <geometry>
+          <mesh filename="package://pr2_description/meshes/gripper_v0/l_finger_tip.stl" scale=".001 .001 .001"/>
         </geometry>
         <verbose value="Yes" />
@@ -219,15 +219,15 @@
                   izz="0.00001541768" />
       </inertial>
-      <visual name="${prefix}_r_finger_tip_visual">
-        <origin xyz="0 0 0" rpy="0 0 0" />
-        <geometry name="${prefix}_r_finger_tip_visual_geom">
-          <mesh filename="package://pr2_description/meshes/gripper_v0/finger_tip_r.stl" />
+      <visual>
+        <origin xyz="0 0 0" rpy="${M_PI} 0 0" />
+        <geometry>
+          <mesh filename="package://pr2_description/meshes/gripper_v0/l_finger_tip.stl" scale=".001 .001 .001" />
         </geometry>
         <material name="Green" />
       </visual>
       <collision name="${prefix}_r_finger_tip_collision">
-        <origin xyz="0 0 0" rpy="0 0 0" />
-        <geometry name="${prefix}_r_finger_tip_collision_geom">
-          <mesh filename="package://pr2_description/meshes/gripper_v0/finger_tip_pad2_r.stl" />
+        <origin xyz="0 0 0" rpy="${M_PI} 0 0" />
+        <geometry>
+          <mesh filename="package://pr2_description/meshes/gripper_v0/l_finger_tip.stl" scale=".001 .001 .001" />
         </geometry>
         <verbose value="Yes" />
@@ -251,8 +251,8 @@
                   izz="0.00086563316" />
       </inertial>
-      <visual name="${side}_gripper_palm_visual">
-        <origin xyz="0 0 0" rpy="0 0 0" />
-        <geometry name="${side}_gripper_palm_visual_geom">
-          <mesh filename="package://pr2_description/meshes/gripper_v0/gripper_palm.stl" />
+      <visual>
+        <origin xyz="0 0 0" rpy="0 0 0" />
+        <geometry>
+          <mesh filename="package://pr2_description/meshes/gripper_v0/gripper_palm.stl" scale=".001 .001 .001" />
         </geometry>
         <material name="Red" />
@@ -260,6 +260,6 @@
       <collision name="${side}_gripper_palm_collision">
         <origin xyz="0 0 0" rpy="0 0 0" />
-        <geometry name="${side}_gripper_palm_collision_geom">
-          <mesh filename="package://pr2_description/meshes/gripper_v0/gripper_palm.stl" />
+        <geometry>
+          <mesh filename="package://pr2_description/meshes/gripper_v0/gripper_palm.stl" scale=".001 .001 .001" />
         </geometry>
         <verbose value="Yes" />

File: pr2_description/urdf/head_v0/head.urdf.xacro (robot description, xacro)
@@ -29,5 +29,5 @@
         <origin xyz="0 0 0.0" rpy="0 0 0 " />
         <geometry>
-          <mesh filename="package://pr2_description/meshes/head_v0/head_pan.stl" />
+          <mesh filename="package://pr2_description/meshes/head_v0/head_pan.stl" scale=".001 .001 .001" />
         </geometry>
         <material name="Blue" />
@@ -67,5 +67,5 @@
         <origin xyz="0 0 0" rpy="0.0 0.0 0.0" />
         <geometry>
-          <mesh filename="package://pr2_description/meshes/head_v0/head_tilt.stl" />
+          <mesh filename="package://pr2_description/meshes/head_v0/head_tilt.stl" scale=".001 .001 .001" />
         </geometry>
         <material name="Green" />

File: pr2_description/urdf/shoulder_v0/shoulder.urdf.xacro (robot description, xacro)
@@ -38,8 +38,8 @@
                  izz="0.27353821674" />
       </inertial>
-      <visual name="${side}_shoulder_pan_visual">
+      <visual>
         <origin xyz="0 0 0" rpy="0 0 0" />
-        <geometry name="${side}_shoulder_pan_visual_geom">
-          <mesh filename="package://pr2_description/meshes/shoulder_v0/shoulder_yaw.stl" />
+        <geometry>
+          <mesh filename="package://pr2_description/meshes/shoulder_v0/shoulder_pan.stl" scale=".001 .001 .001" />
         </geometry>
         <material name="Blue" />
@@ -47,6 +47,6 @@
       <collision name="${side}_shoulder_pan_collision">
         <origin xyz="0.0 0 0.0" rpy="0 0 0" />
-        <geometry name="${side}_shoulder_pan_collision_geom">
-          <mesh filename="package://pr2_description/meshes/shoulder_v0/convex/shoulder_yaw_convex.stlb" />
+        <geometry>
+          <mesh filename="package://pr2_description/meshes/shoulder_v0/shoulder_pan.stl" scale=".001 .001 .001" />
         </geometry>
       </collision>
@@ -75,8 +75,8 @@
                  izz="0.01975753814" />
       </inertial>
-      <visual name="${side}_shoulder_lift_visual">
+      <visual>
         <origin xyz="0 0 0" rpy="0 0 0" />
-        <geometry name="${side}_shoulder_lift_visual_geom">
-          <mesh filename="package://pr2_description/meshes/shoulder_v0/shoulder_lift.stl" />
+        <geometry>
+          <mesh filename="package://pr2_description/meshes/shoulder_v0/shoulder_lift.stl" scale=".001 .001 .001" />
         </geometry>
         <material name="Grey" />
@@ -84,6 +84,6 @@
       <collision name="${side}_shoulder_lift_collision">
         <origin xyz="0 0 0" rpy="0 0 0" />
-        <geometry name="${side}_shoulder_lift_collision_geom">
-          <mesh filename="package://pr2_description/meshes/shoulder_v0/convex/shoulder_lift_convex.stlb" />
+        <geometry>
+          <mesh filename="package://pr2_description/meshes/shoulder_v0/shoulder_lift.stl" scale=".001 .001 .001" />
         </geometry>
       </collision>
@@ -119,9 +119,9 @@
                   izz="0.01" />
       </inertial>
-      <visual name="${side}_upper_arm_roll_visual">
+      <visual>
         <!-- TODO: This component doesn't actually have a mesh -->
         <origin xyz="0 0 0" rpy="0 0 0" />
-        <geometry name="${side}_upper_arm_roll_visual_geom">
-          <mesh filename="package://pr2_description/meshes/shoulder_v0/upper_arm_roll.stl" />
+        <geometry>
+          <mesh filename="package://pr2_description/meshes/shoulder_v0/upper_arm_roll.stl" scale=".001 .001 .001" />
         </geometry>
         <material name="RollLinks" />
@@ -130,5 +130,5 @@
         <!-- TODO: collision tag should be optional -->
         <origin xyz="0.0 0 0" rpy="0 0 0" />
-        <geometry name="${side}_upper_arm_roll_collision_geom">
+        <geometry>
           <box size="0.1 0.1 0.1" />
         </geometry>

File: pr2_description/urdf/tilting_laser_v0/tilting_laser.urdf.xacro (robot description, xacro)
@@ -27,7 +27,7 @@
                  izz="0.0001" />
       </inertial>
-      <visual name="${name}_mount_visual">
+      <visual>
         <origin xyz="0 0 0" rpy="0 0 0" />
-        <geometry name="${name}_mount_visual_geom">
+        <geometry>
           <mesh filename="package://pr2_description/meshes/tilting_laser_v0/hok_tilt.stl" />
         </geometry>
@@ -36,5 +36,5 @@
       <collision name="${name}_mount_collision">
         <origin xyz="0 0 0" rpy="0 0 0" />
-        <geometry name="${name}_mount_collision_geom" >
+        <geometry>
           <box size=".001 .001 .001" />
         </geometry>

File: pr2_description/urdf/torso_v0/torso.urdf.xacro (robot description, xacro)
@@ -26,8 +26,8 @@
                  iyy="2.510019507959" iyz="0.029664468704" izz="0.526432355569" />
       </inertial>
-      <visual name="${name}_visual">
+      <visual>
         <origin xyz="0 0 0" rpy="0 0 0" />
-        <geometry name="${name}_visual_geom">
-          <mesh filename="package://pr2_description/meshes/torso_v0/torso.stl" />
+        <geometry>
+          <mesh filename="package://pr2_description/meshes/torso_v0/torso_lift_2k.stl" scale=".001 .001 .001" />
         </geometry>
         <material name="Grey2" />
@@ -35,5 +35,5 @@
       <collision name="${name}_collision">
         <origin xyz="0 0 0.16" rpy="0 0 0" />
-        <geometry name="${name}_collision_geom">
+        <geometry>
           <!-- arbitrarily chosen collision box by JH, torso collision is not important for now -->
           <box size="0.30 0.620 0.02" />

File: pr2_description/urdf/upper_arm_v0/upper_arm.urdf.xacro (robot description, xacro)
@@ -49,8 +49,8 @@
                   izz="${0.5*((reflect+1)*ual_izz+(1-reflect)*uar_izz)}" />
       </inertial>
-      <visual name="{side}_upper_arm_visual">
+      <visual>
         <origin xyz="0 0 0" rpy="0 0 0" />
-        <geometry name="${side}_upper_arm_visual_geom">
-          <mesh filename="package://pr2_description/meshes/upper_arm_v0/upper_arm.stl" />
+        <geometry>
+          <mesh filename="package://pr2_description/meshes/upper_arm_v0/upper_arm.stl" scale=".001 .001 .001" />
         </geometry>
         <material name="Green" />
@@ -58,6 +58,6 @@
       <collision name="${side}_upper_arm_collision">
         <origin xyz="0 0 0" rpy="0 0 0" />
-        <geometry name="${side}_upper_arm_collision_geom">
-          <mesh filename="package://pr2_description/meshes/upper_arm_v0/convex/upper_arm_convex.stlb" />
+        <geometry>
+          <mesh filename="package://pr2_description/meshes/upper_arm_v0/upper_arm.stl" scale=".001 .001 .001" />
         </geometry>
       </collision>
@@ -92,8 +92,8 @@
                   izz="0.00359156824" />
       </inertial>
-      <visual name="${side}_elbow_flex_visual">
+      <visual>
         <origin xyz="0 0 0" rpy="0 0 0" />
-        <geometry name="${side}_elbow_flex_visual_geom">
-          <mesh filename="package://pr2_description/meshes/upper_arm_v0/elbow_flex.stl" />
+        <geometry>
+          <mesh filename="package://pr2_description/meshes/upper_arm_v0/elbow_flex.stl" scale=".001 .001 .001" />
         </geometry>
         <material name="Grey" />
@@ -101,6 +101,6 @@
       <collision name="${side}_elbow_flex_collision">
         <origin xyz="0 0 0" rpy="0 0 0" />
-        <geometry name="${side}_elbow_flex_collision_geom">
-          <mesh filename="package://pr2_description/meshes/upper_arm_v0/convex/elbow_flex_convex.stlb" />
+        <geometry>
+          <mesh filename="package://pr2_description/meshes/upper_arm_v0/elbow_flex.stl" scale=".001 .001 .001" />
         </geometry>
       </collision>
@@ -133,8 +133,8 @@
                   izz="0.01" />
       </inertial>
-      <visual name="${side}_forearm_roll_visual">
+      <visual>
         <origin xyz="0 0 0" rpy="0 0 0" />
-        <geometry name="${side}_forearm_roll_visual_geom">
-          <mesh filename="package://pr2_description/meshes/upper_arm_v0/forearm_roll.stl" />
+        <geometry>
+          <mesh filename="package://pr2_description/meshes/upper_arm_v0/forearm_roll.stl" scale=".001 .001 .001" />
         </geometry>
         <material name="RollLinks" />
@@ -144,5 +144,5 @@
         <!-- dummy geom, to be removed -->
         <origin xyz="0 0 0" rpy="0 0 0" />
-        <geometry name="${side}_forearm_roll_collision_geom">
+        <geometry>
           <box size="0.1 0.1 0.1" />
         </geometry>

Commit message: scale caster

File: pr2_description/urdf/base_v0/base.urdf.xacro (robot description, xacro)
@@ -94,5 +94,5 @@
         <origin xyz="0 0 0" rpy="0 0 0" />
         <geometry>
-          <mesh filename="package://pr2_description/meshes/base_v0/caster.stl" />
+          <mesh filename="package://pr2_description/meshes/base_v0/caster.stl" scale=".001 .001 .001"/>
         </geometry>
         <material name="Green" />
