Commit message: meshes in meters

File: pr2_description/urdf/base_v0/base.urdf.xacro (robot description, xacro)
@@ -57,5 +57,5 @@
         <origin xyz="0 0 0" rpy="0 0 0" />
         <geometry>
-          <mesh filename="package://pr2_description/meshes/base_v0/wheel.stl" scale=".001 .001 .001"/>
+          <mesh filename="package://pr2_description/meshes/base_v0/wheel.stl" />
         </geometry>
         <material name="Wheel_${suffix}" />
@@ -94,5 +94,5 @@
         <origin xyz="0 0 0" rpy="0 0 0" />
         <geometry>
-          <mesh filename="package://pr2_description/meshes/base_v0/caster.stl" scale=".001 .001 .001"/>
+          <mesh filename="package://pr2_description/meshes/base_v0/caster.stl" />
         </geometry>
         <material name="Green" />
@@ -131,5 +131,5 @@
         <origin xyz="0 0 0" rpy="0 0 0" />
         <geometry>
-          <mesh filename="package://pr2_description/meshes/base_v0/base.stl" scale=".001 .001 .001"/>
+          <mesh filename="package://pr2_description/meshes/base_v0/base.stl" />
         </geometry>
         <material name="Green" />

File: pr2_description/urdf/forearm_v0/forearm.urdf.xacro (robot description, xacro)
@@ -28,5 +28,5 @@
         <origin xyz="0 0 0" rpy="0 0 0" />
         <geometry name="${side}_forearm_visual_geom">
-          <mesh filename="package://pr2_description/meshes/forearm_v0/forearm.stl" scale=".001 .001 .001"/>
+          <mesh filename="package://pr2_description/meshes/forearm_v0/forearm.stl" />
         </geometry>
         <material name="Blue" />
@@ -35,5 +35,5 @@
         <origin xyz="0 0 0" rpy="0 0 0" />
         <geometry name="${side}_forearm_collision_geom">
-          <mesh filename="package://pr2_description/meshes/forearm_v0/forearm.stl" scale=".001 .001 .001"/>
+          <mesh filename="package://pr2_description/meshes/forearm_v0/forearm.stl" />
         </geometry>
       </collision>
@@ -62,5 +62,5 @@
         <origin xyz="0 0 0" rpy="0 0 0" />
         <geometry name="${side}_wrist_flex_visual_geom">
-          <mesh filename="package://pr2_description/meshes/forearm_v0/wrist_flex.stl" scale=".001 .001 .001"/>
+          <mesh filename="package://pr2_description/meshes/forearm_v0/wrist_flex.stl" />
         </geometry>
         <material name="Grey" />
@@ -69,5 +69,5 @@
         <origin xyz="0 0 0" rpy="0 0 0" />
         <geometry name="${side}_wrist_flex_collision_geom">
-          <mesh filename="package://pr2_description/meshes/forearm_v0/wrist_flex.stl" scale=".001 .001 .001"/>
+          <mesh filename="package://pr2_description/meshes/forearm_v0/wrist_flex.stl" />
         </geometry>
       </collision>
@@ -97,5 +97,5 @@
         <origin xyz="0 0 0" rpy="0 0 0" />
         <geometry name="${side}_wrist_roll_visual_geom">
-          <mesh filename="package://pr2_description/meshes/forearm_v0/wrist_roll.stl" scale=".001 .001 .001"/>
+          <mesh filename="package://pr2_description/meshes/forearm_v0/wrist_roll.stl" />
         </geometry>
         <material name="RollLinks" />

File: pr2_description/urdf/gripper_v0/gripper.urdf.xacro (robot description, xacro)
@@ -49,5 +49,5 @@
         <origin xyz="0 0 0" rpy="0 0 0" />
         <geometry>
-          <mesh filename="package://pr2_description/meshes/gripper_v0/l_finger.stl" scale=".001 .001 .001"/>
+          <mesh filename="package://pr2_description/meshes/gripper_v0/l_finger.stl" />
         </geometry>
         <material name="Grey" />
@@ -56,5 +56,5 @@
         <origin xyz="0 0 0" rpy="0 0 0" />
         <geometry>
-          <mesh filename="package://pr2_description/meshes/gripper_v0/l_finger.stl" scale=".001 .001 .001"/>
+          <mesh filename="package://pr2_description/meshes/gripper_v0/l_finger.stl" />
         </geometry>
         <verbose value="Yes" />
@@ -85,5 +85,5 @@
         <origin xyz="0 0 0" rpy="${M_PI} 0 0" />
         <geometry>
-          <mesh filename="package://pr2_description/meshes/gripper_v0/l_finger.stl" scale=".001 .001 .001"/>
+          <mesh filename="package://pr2_description/meshes/gripper_v0/l_finger.stl" />
         </geometry>
         <material name="Grey" />
@@ -92,5 +92,5 @@
         <origin xyz="0 0 0" rpy="${M_PI} 0 0" />
         <geometry>
-          <mesh filename="package://pr2_description/meshes/gripper_v0/l_finger.stl" scale=".001 .001 .001"/>
+          <mesh filename="package://pr2_description/meshes/gripper_v0/l_finger.stl" />
         </geometry>
         <verbose value="Yes" />
@@ -189,5 +189,5 @@
         <origin xyz="0 0 0" rpy="0 0 0" />
         <geometry>
-          <mesh filename="package://pr2_description/meshes/gripper_v0/l_finger_tip.stl" scale=".001 .001 .001"/>
+          <mesh filename="package://pr2_description/meshes/gripper_v0/l_finger_tip.stl" />
         </geometry>
         <material name="Green" />
@@ -196,5 +196,5 @@
         <origin xyz="0 0 0" rpy="0 0 0" />
         <geometry>
-          <mesh filename="package://pr2_description/meshes/gripper_v0/l_finger_tip.stl" scale=".001 .001 .001"/>
+          <mesh filename="package://pr2_description/meshes/gripper_v0/l_finger_tip.stl" />
         </geometry>
         <verbose value="Yes" />
@@ -222,5 +222,5 @@
         <origin xyz="0 0 0" rpy="${M_PI} 0 0" />
         <geometry>
-          <mesh filename="package://pr2_description/meshes/gripper_v0/l_finger_tip.stl" scale=".001 .001 .001" />
+          <mesh filename="package://pr2_description/meshes/gripper_v0/l_finger_tip.stl"  />
         </geometry>
         <material name="Green" />
@@ -229,5 +229,5 @@
         <origin xyz="0 0 0" rpy="${M_PI} 0 0" />
         <geometry>
-          <mesh filename="package://pr2_description/meshes/gripper_v0/l_finger_tip.stl" scale=".001 .001 .001" />
+          <mesh filename="package://pr2_description/meshes/gripper_v0/l_finger_tip.stl"  />
         </geometry>
         <verbose value="Yes" />
@@ -254,5 +254,5 @@
         <origin xyz="0 0 0" rpy="0 0 0" />
         <geometry>
-          <mesh filename="package://pr2_description/meshes/gripper_v0/gripper_palm.stl" scale=".001 .001 .001" />
+          <mesh filename="package://pr2_description/meshes/gripper_v0/gripper_palm.stl"  />
         </geometry>
         <material name="Red" />
@@ -261,5 +261,5 @@
         <origin xyz="0 0 0" rpy="0 0 0" />
         <geometry>
-          <mesh filename="package://pr2_description/meshes/gripper_v0/gripper_palm.stl" scale=".001 .001 .001" />
+          <mesh filename="package://pr2_description/meshes/gripper_v0/gripper_palm.stl"  />
         </geometry>
         <verbose value="Yes" />

File: pr2_description/urdf/head_v0/head.urdf.xacro (robot description, xacro)
@@ -29,5 +29,5 @@
         <origin xyz="0 0 0.0" rpy="0 0 0 " />
         <geometry>
-          <mesh filename="package://pr2_description/meshes/head_v0/head_pan.stl" scale=".001 .001 .001" />
+          <mesh filename="package://pr2_description/meshes/head_v0/head_pan.stl"  />
         </geometry>
         <material name="Blue" />
@@ -67,5 +67,5 @@
         <origin xyz="0 0 0" rpy="0.0 0.0 0.0" />
         <geometry>
-          <mesh filename="package://pr2_description/meshes/head_v0/head_tilt.stl" scale=".001 .001 .001" />
+          <mesh filename="package://pr2_description/meshes/head_v0/head_tilt.stl"  />
         </geometry>
         <material name="Green" />

File: pr2_description/urdf/shoulder_v0/shoulder.urdf.xacro (robot description, xacro)
@@ -41,5 +41,5 @@
         <origin xyz="0 0 0" rpy="0 0 0" />
         <geometry>
-          <mesh filename="package://pr2_description/meshes/shoulder_v0/shoulder_pan.stl" scale=".001 .001 .001" />
+          <mesh filename="package://pr2_description/meshes/shoulder_v0/shoulder_pan.stl"  />
         </geometry>
         <material name="Blue" />
@@ -48,5 +48,5 @@
         <origin xyz="0.0 0 0.0" rpy="0 0 0" />
         <geometry>
-          <mesh filename="package://pr2_description/meshes/shoulder_v0/shoulder_pan.stl" scale=".001 .001 .001" />
+          <mesh filename="package://pr2_description/meshes/shoulder_v0/shoulder_pan.stl"  />
         </geometry>
       </collision>
@@ -78,5 +78,5 @@
         <origin xyz="0 0 0" rpy="0 0 0" />
         <geometry>
-          <mesh filename="package://pr2_description/meshes/shoulder_v0/shoulder_lift.stl" scale=".001 .001 .001" />
+          <mesh filename="package://pr2_description/meshes/shoulder_v0/shoulder_lift.stl"  />
         </geometry>
         <material name="Grey" />
@@ -85,5 +85,5 @@
         <origin xyz="0 0 0" rpy="0 0 0" />
         <geometry>
-          <mesh filename="package://pr2_description/meshes/shoulder_v0/shoulder_lift.stl" scale=".001 .001 .001" />
+          <mesh filename="package://pr2_description/meshes/shoulder_v0/shoulder_lift.stl"  />
         </geometry>
       </collision>
@@ -123,5 +123,5 @@
         <origin xyz="0 0 0" rpy="0 0 0" />
         <geometry>
-          <mesh filename="package://pr2_description/meshes/shoulder_v0/upper_arm_roll.stl" scale=".001 .001 .001" />
+          <mesh filename="package://pr2_description/meshes/shoulder_v0/upper_arm_roll.stl"  />
         </geometry>
         <material name="RollLinks" />

File: pr2_description/urdf/torso_v0/torso.urdf.xacro (robot description, xacro)
@@ -29,5 +29,5 @@
         <origin xyz="0 0 0" rpy="0 0 0" />
         <geometry>
-          <mesh filename="package://pr2_description/meshes/torso_v0/torso_lift_2k.stl" scale=".001 .001 .001" />
+          <mesh filename="package://pr2_description/meshes/torso_v0/torso_lift_2k.stl"  />
         </geometry>
         <material name="Grey2" />

File: pr2_description/urdf/upper_arm_v0/upper_arm.urdf.xacro (robot description, xacro)
@@ -52,5 +52,5 @@
         <origin xyz="0 0 0" rpy="0 0 0" />
         <geometry>
-          <mesh filename="package://pr2_description/meshes/upper_arm_v0/upper_arm.stl" scale=".001 .001 .001" />
+          <mesh filename="package://pr2_description/meshes/upper_arm_v0/upper_arm.stl"  />
         </geometry>
         <material name="Green" />
@@ -59,5 +59,5 @@
         <origin xyz="0 0 0" rpy="0 0 0" />
         <geometry>
-          <mesh filename="package://pr2_description/meshes/upper_arm_v0/upper_arm.stl" scale=".001 .001 .001" />
+          <mesh filename="package://pr2_description/meshes/upper_arm_v0/upper_arm.stl"  />
         </geometry>
       </collision>
@@ -95,5 +95,5 @@
         <origin xyz="0 0 0" rpy="0 0 0" />
         <geometry>
-          <mesh filename="package://pr2_description/meshes/upper_arm_v0/elbow_flex.stl" scale=".001 .001 .001" />
+          <mesh filename="package://pr2_description/meshes/upper_arm_v0/elbow_flex.stl"  />
         </geometry>
         <material name="Grey" />
@@ -102,5 +102,5 @@
         <origin xyz="0 0 0" rpy="0 0 0" />
         <geometry>
-          <mesh filename="package://pr2_description/meshes/upper_arm_v0/elbow_flex.stl" scale=".001 .001 .001" />
+          <mesh filename="package://pr2_description/meshes/upper_arm_v0/elbow_flex.stl"  />
         </geometry>
       </collision>
@@ -136,5 +136,5 @@
         <origin xyz="0 0 0" rpy="0 0 0" />
         <geometry>
-          <mesh filename="package://pr2_description/meshes/upper_arm_v0/forearm_roll.stl" scale=".001 .001 .001" />
+          <mesh filename="package://pr2_description/meshes/upper_arm_v0/forearm_roll.stl"  />
         </geometry>
         <material name="RollLinks" />
