Commit message: update simulation gripper joint:  * removed old slider "floating link".  * added parallel links to enforce tips stay parallel.  * added slider between finger tips.  * added slider to gripper transmission.  this will be used by updated pr2 gripper transmission. * new beta meshes in meters

File: pr2_description/urdf/base_v0/base.urdf.xacro (robot description, xacro)
@@ -57,5 +57,5 @@
         <origin xyz="0 0 0" rpy="0 0 0" />
         <geometry>
-          <mesh filename="package://pr2_description/meshes/base_v0/pr2_wheel.stl" />
+          <mesh filename="package://pr2_description/meshes/base_v0/wheel.stl" />
         </geometry>
         <material name="Wheel_${suffix}" />

File: pr2_description/urdf/forearm_v0/forearm.urdf.xacro (robot description, xacro)
@@ -35,29 +35,5 @@
         <origin xyz="0 0 0" rpy="0 0 0" />
         <geometry>
-          <mesh filename="package://pr2_description/meshes/forearm_v0/convex/forearm_convex.stlb" />
-        </geometry>
-      </collision>
-    </link>
-    <joint name="${side}_forearm_sleeve_joint" type="fixed">
-      <insert_block name="origin" /> <!-- transform from parent link to this joint frame -->
-      <parent link="${parent}"/>
-      <child link="${side}_forearm_sleeve_link"/>
-    </joint>
-    <link name="${side}_forearm_sleeve_link">
-      <inertial>
-        <mass value="0.1" />
-        <origin xyz="0 0 0" />
-        <inertia ixx="0.01" ixy="0.00" ixz="0.00" iyy="0.01" iyz="0.00" izz="0.01" />
-      </inertial>
-      <visual>
-        <origin xyz="-0.03 0.009 0" rpy="0 1.5707 -0.04" />
-        <geometry>
-          <mesh filename="package://pr2_description/meshes/forearm_v0/forearm.dae" scale="0.001 0.001 0.001" />
-        </geometry>
-      </visual>
-      <collision>
-        <origin xyz="-0.03 0.009 0" rpy="0 1.5707 -0.04" />
-        <geometry>
-          <mesh filename="package://pr2_description/meshes/forearm_v0/forearm.dae" scale="0.001 0.001 0.001" />
+          <mesh filename="package://pr2_description/meshes/forearm_v0/forearm.stl" />
         </geometry>
       </collision>
@@ -93,5 +69,5 @@
         <origin xyz="0 0 0" rpy="0 0 0" />
         <geometry name="${side}_wrist_flex_collision_geom">
-          <mesh filename="package://pr2_description/meshes/forearm_v0/convex/wrist_flex_convex.stlb" />
+          <mesh filename="package://pr2_description/meshes/forearm_v0/wrist_flex.stl" />
         </geometry>
       </collision>

File: pr2_description/urdf/gripper_v0/gripper.gazebo.xacro (robot description, xacro)
@@ -18,5 +18,5 @@
   <property name="finger_tip_mu"              value="500.0" />
   <property name="finger_mu"                  value="500.0" />
-  <xacro:macro name="pr2_finger_gazebo_v0" params="prefix">
+  <xacro:macro name="pr2_finger_gazebo_v0" params="prefix parallel_link_x_offset parallel_link_y_offset">
     <!-- Finger proximal digit -->
     <gazebo reference="${prefix}_l_finger_link">
@@ -141,4 +141,35 @@
       <provideFeedback value="true"/>
     </gazebo>
+    <!-- parallel link for simulating gripper constraints -->
+    <gazebo>
+      <joint:hinge name="${prefix}_r_parallel_tip_joint">
+          <body1>${prefix}_r_parallel_link</body1>
+          <body2>${prefix}_r_finger_tip_link</body2>
+          <anchor>${prefix}_r_finger_tip_link</anchor>
+          <axis>0 0 1</axis>
+          <anchorOffset>${parallel_link_x_offset} ${-parallel_link_y_offset} 0</anchorOffset>
+      </joint:hinge>
+      <joint:hinge name="${prefix}_l_parallel_tip_joint">
+          <body1>${prefix}_l_parallel_link</body1>
+          <body2>${prefix}_l_finger_tip_link</body2>
+          <anchor>${prefix}_l_finger_tip_link</anchor>
+          <axis>0 0 1</axis>
+          <anchorOffset>${parallel_link_x_offset} ${parallel_link_y_offset} 0</anchorOffset>
+      </joint:hinge>
+      <joint:slider name="${prefix}_simulated_joint">
+          <body1>${prefix}_l_finger_tip_link</body1>
+          <body2>${prefix}_r_finger_tip_link</body2>
+          <anchor>${prefix}_r_finger_tip_link</anchor>
+          <axis>0 1 0</axis>
+      </joint:slider>
+    </gazebo>
+    <gazebo reference="${prefix}_l_parallel_link">
+      <turnGravityOff>true</turnGravityOff>
+      <material value="PR2/Red" />
+    </gazebo>
+    <gazebo reference="${prefix}_r_parallel_link">
+      <turnGravityOff>true</turnGravityOff>
+      <material value="PR2/Red" />
+    </gazebo>
   </xacro:macro>
   <xacro:macro name="pr2_gripper_gazebo_v0" params="side">
@@ -157,73 +188,16 @@
       <material value="PR2/Grey" />
     </gazebo>
-    <!-- floating link for simulating gripper constraints -->
-    <gazebo reference="${side}_gripper_float_link">
-      <turnGravityOff>true</turnGravityOff>
-      <material value="PR2/White" />
-    </gazebo>
     <gazebo>
-      <!-- floating link for enforcing gripper constraints -->
-      <body:box name="${side}_gripper_float_link">
-          <massMatrix>true</massMatrix>
-          <mass>0.01</mass>
-          <ixx>0.0001</ixx>
-          <ixy>0</ixy>
-          <ixz>0</ixz>
-          <iyy>0.0001</iyy>
-          <iyz>0</iyz>
-          <izz>0.0001</izz>
-          <cx>0</cx>
-          <cy>0</cy>
-          <cz>0</cz>
-          <xyz>0.82025 0.188 0.790675</xyz>
-          <rpy>0 -0 0</rpy>
-          <geom:box name="${side}_gripper_float_link_geom">
-              <xyz>0 0 0</xyz>
-              <rpy>0 -0 0</rpy>
-              <size>0.0 0.0 0.0</size>
-              <visual>
-                  <xyz>0 0 0</xyz>
-                  <rpy>0 -0 0</rpy>
-                  <scale>0.0 0.0 0.0</scale>
-                  <mesh>unit_box</mesh>
-                  <material>PR2/White</material>
-              </visual>
-          </geom:box>
-          <turnGravityOff>true</turnGravityOff>
-          <selfCollide>false</selfCollide>
-      </body:box>
-      <joint:slider name="${side}_gripper_float_joint">
-          <body1>${side}_gripper_float_link</body1>
-          <body2>${side}_gripper_palm_link</body2>
-          <anchor>${side}_gripper_float_link</anchor>
-          <axis>1 0 0</axis>
-          <lowStop>-0.05</lowStop>
-          <highStop>0.001</highStop>
-      </joint:slider>
-      <joint:slider name="${side}_gripper_l_finger_tip_slider_joint">
-          <body1>${side}_gripper_l_finger_tip_link</body1>
-          <body2>${side}_gripper_float_link</body2>
-          <anchor>${side}_gripper_l_finger_tip_link</anchor>
-          <axis>0 1 0</axis>
-          <anchorOffset>0 0 0</anchorOffset>
-      </joint:slider>
-      <joint:slider name="${side}_gripper_r_finger_tip_slider_joint">
-          <body1>${side}_gripper_r_finger_tip_link</body1>
-          <body2>${side}_gripper_float_link</body2>
-          <anchor>${side}_gripper_r_finger_tip_link</anchor>
-          <axis>0 1 0</axis>
-          <anchorOffset>0 0 0</anchorOffset>
-      </joint:slider>
-      <!--
-      <joint:slider name="${side}_gripper_finger_tip_slider_joint">
-          <body1>${side}_gripper_l_finger_tip_link</body1>
-          <body2>${side}_gripper_r_finger_tip_link</body2>
-          <anchor>${side}_gripper_l_finger_tip_link</anchor>
-          <axis>0 1 0</axis>
-          <anchorOffset>0 0 0</anchorOffset>
-          <lowStop>0.0</lowStop>
-          <highStop>0.08</highStop>
-      </joint:slider>
-      -->
+      <controller:gazebo_ros_p3d name="p3d_${side}_gripper_palm_controller" plugin="libgazebo_ros_p3d.so">
+        <alwaysOn>true</alwaysOn>
+        <updateRate>100.0</updateRate>
+        <bodyName>${side}_gripper_palm_link</bodyName>
+        <topicName>${side}_gripper_palm_pose_ground_truth</topicName>
+        <xyzOffsets>0 0 0</xyzOffsets>
+        <rpyOffsets>0 0 0</rpyOffsets>
+        <gaussianNoise>0.0</gaussianNoise>
+        <frameName>map</frameName>
+        <interface:position name="p3d_${side}_gripper_palm_position_iface" />
+      </controller:gazebo_ros_p3d>
     </gazebo>
   </xacro:macro>

File: pr2_description/urdf/gripper_v0/gripper.urdf.xacro (robot description, xacro)
@@ -11,5 +11,8 @@
   <property name="gripper_lower_angle" value="0.00" />
   <property name="finger_damping"             value="0.2" />
+  <property name="gripper_damping"            value="100.0" />
   <property name="finger_tip_damping"         value="0.01" />
+  <property name="parallel_link_x_offset"     value="-0.018" />
+  <property name="parallel_link_y_offset"     value="0.021" />
   <property name="finger_joint_effort_limit"  value="1000.0" />
   <xacro:macro name="pr2_finger_limits_v0" params="reflect">
@@ -43,8 +46,8 @@
                   izz= "0.00018105446" />
       </inertial>
-      <visual name="${prefix}_l_finger_visual">
-        <origin xyz="0 0 0" rpy="0 0 0" />
-        <geometry name="${prefix}_l_finger_visual_geom">
-          <mesh filename="package://pr2_description/meshes/gripper_v0/upper_finger_l.stl" />
+      <visual>
+        <origin xyz="0 0 0" rpy="0 0 0" />
+        <geometry>
+          <mesh filename="package://pr2_description/meshes/gripper_v0/l_finger.stl" />
         </geometry>
         <material name="Grey" />
@@ -52,6 +55,6 @@
       <collision name="${prefix}_l_finger_collision">
         <origin xyz="0 0 0" rpy="0 0 0" />
-        <geometry name="${prefix}_l_finger_collision_geom">
-          <mesh filename="package://pr2_description/meshes/gripper_v0/upper_finger_l.stl" />
+        <geometry>
+          <mesh filename="package://pr2_description/meshes/gripper_v0/l_finger.stl" />
         </geometry>
         <verbose value="Yes" />
@@ -79,15 +82,86 @@
                   izz= "0.00018106988" />
       </inertial>
-      <visual name="${prefix}_r_finger_visual">
-        <origin xyz="0 0 0" rpy="0 0 0" />
-        <geometry name="${prefix}_r_finger_visual_geom">
-          <mesh filename="package://pr2_description/meshes/gripper_v0/upper_finger_r.stl" />
+      <visual>
+        <origin xyz="0 0 0" rpy="${M_PI} 0 0" />
+        <geometry>
+          <mesh filename="package://pr2_description/meshes/gripper_v0/l_finger.stl" />
         </geometry>
         <material name="Grey" />
       </visual>
       <collision name="${prefix}_r_finger_collision">
-        <origin xyz="0 0 0" rpy="0 0 0" />
-        <geometry name="${prefix}_r_finger_collision_geom">
-          <mesh filename="package://pr2_description/meshes/gripper_v0/upper_finger_r.stl" />
+        <origin xyz="0 0 0" rpy="${M_PI} 0 0" />
+        <geometry>
+          <mesh filename="package://pr2_description/meshes/gripper_v0/l_finger.stl" />
+        </geometry>
+        <verbose value="Yes" />
+      </collision>
+    </link>
+    <!-- Floating Link -->
+    <joint name="${prefix}_l_parallel_root_joint" type="revolute">
+      <axis xyz="0 0 1" />
+      <origin xyz="${0.07691+parallel_link_x_offset} ${+0.01+parallel_link_y_offset} 0" rpy="0 0 0" />
+      <dynamics damping="${finger_damping}" />
+      <mimic joint="${prefix}_l_finger_joint" multiplier="1" offset="0"/>
+      <parent link="${parent}"/>
+      <child link="${prefix}_l_parallel_link"/>
+      <xacro:pr2_finger_limits_v0 reflect="1" />
+    </joint>
+    <joint name="${prefix}_r_parallel_root_joint" type="revolute">
+      <axis xyz="0 0 -1" />
+      <origin xyz="${0.07691+parallel_link_x_offset} ${-0.01-parallel_link_y_offset} 0" rpy="0 0 0" />
+      <dynamics damping="${finger_damping}" />
+      <mimic joint="${prefix}_l_finger_joint" multiplier="-1" offset="0"/>
+      <parent link="${parent}"/>
+      <child link="${prefix}_r_parallel_link"/>
+      <xacro:pr2_finger_limits_v0 reflect="1" />
+    </joint>
+    <link name="${prefix}_l_parallel_link">
+      <inertial>
+        <mass value="0.17126" />
+        <origin xyz="${0.03598} 0.01730 -0.00164" rpy="0 0 0" />
+        <inertia  ixx= "0.00007756198"
+                  ixy= "0.00000149095"
+                  ixz="-0.00000983385"
+                  iyy= "0.00019708305"
+                  iyz="-0.00000306125"
+                  izz= "0.00018105446" />
+      </inertial>
+      <visual>
+        <origin xyz="${0.0914942479/2.0} 0 0" rpy="0 0 0.0541224233" />
+        <geometry>
+          <box size="${0.0914942479} 0.005 0.005" />
+        </geometry>
+        <material name="Green" />
+      </visual>
+      <collision>
+        <origin xyz="${0.0914942479/2.0} 0 0" rpy="0 0 0.0541224233" />
+        <geometry>
+          <box size="${0.0914942479} 0.005 0.005" />
+        </geometry>
+        <verbose value="Yes" />
+      </collision>
+    </link>
+    <link name="${prefix}_r_parallel_link">
+      <inertial>
+        <mass value="0.17389" />
+        <origin xyz="${0.03576} -0.01736 -0.00095" rpy="0 0 0" />
+        <inertia  ixx= "0.00007738410"
+                  ixy="-0.00000209309"
+                  ixz="-0.00000836228"
+                  iyy= "0.00019847383"
+                  iyz= "0.00000246110"
+                  izz= "0.00018106988" />
+      </inertial>
+      <visual>
+        <origin xyz="${0.0914942479/2.0} 0 0" rpy="0 0 -0.0541224233" />
+        <geometry>
+          <box size="${0.0914942479} 0.005 0.005" />
+        </geometry>
+        <material name="Green" />
+      </visual>
+      <collision>
+        <origin xyz="${0.0914942479/2.0} 0 0" rpy="0 0 -0.0541224233" />
+        <geometry>
+          <box size="${0.0914942479} 0.005 0.005" />
         </geometry>
         <verbose value="Yes" />
@@ -112,8 +186,8 @@
                   izz="0.00001541768" />
       </inertial>
-      <visual name="${prefix}_l_finger_tip_visual">
-        <origin xyz="0 0 0" rpy="0 0 0" />
-        <geometry name="${prefix}_l_finger_tip_visual_geom">
-          <mesh filename="package://pr2_description/meshes/gripper_v0/finger_tip_l.stl" />
+      <visual>
+        <origin xyz="0 0 0" rpy="0 0 0" />
+        <geometry>
+          <mesh filename="package://pr2_description/meshes/gripper_v0/l_finger_tip.stl" />
         </geometry>
         <material name="Green" />
@@ -121,6 +195,6 @@
       <collision name="${prefix}_l_finger_tip_collision">
         <origin xyz="0 0 0" rpy="0 0 0" />
-        <geometry name="${prefix}_l_finger_tip_collision_geom">
-          <mesh filename="package://pr2_description/meshes/gripper_v0/finger_tip_pad2_l.stl" />
+        <geometry>
+          <mesh filename="package://pr2_description/meshes/gripper_v0/l_finger_tip.stl" />
         </geometry>
         <verbose value="Yes" />
@@ -145,15 +219,15 @@
                   izz="0.00001541768" />
       </inertial>
-      <visual name="${prefix}_r_finger_tip_visual">
-        <origin xyz="0 0 0" rpy="0 0 0" />
-        <geometry name="${prefix}_r_finger_tip_visual_geom">
-          <mesh filename="package://pr2_description/meshes/gripper_v0/finger_tip_r.stl" />
+      <visual>
+        <origin xyz="0 0 0" rpy="${M_PI} 0 0" />
+        <geometry>
+          <mesh filename="package://pr2_description/meshes/gripper_v0/l_finger_tip.stl"  />
         </geometry>
         <material name="Green" />
       </visual>
       <collision name="${prefix}_r_finger_tip_collision">
-        <origin xyz="0 0 0" rpy="0 0 0" />
-        <geometry name="${prefix}_r_finger_tip_collision_geom">
-          <mesh filename="package://pr2_description/meshes/gripper_v0/finger_tip_pad2_r.stl" />
+        <origin xyz="0 0 0" rpy="${M_PI} 0 0" />
+        <geometry>
+          <mesh filename="package://pr2_description/meshes/gripper_v0/l_finger_tip.stl"  />
         </geometry>
         <verbose value="Yes" />
@@ -161,5 +235,5 @@
     </link>
     <!-- extensions -->
-    <xacro:pr2_finger_gazebo_v0 prefix="${prefix}" />
+    <xacro:pr2_finger_gazebo_v0 prefix="${prefix}" parallel_link_x_offset="${parallel_link_x_offset}" parallel_link_y_offset="${parallel_link_y_offset}" />
   </xacro:macro>
   <xacro:macro name="pr2_gripper_v0" params="side parent *origin gear_ratio screw_reduction theta0 phi0 t0 L0 h a b r">
@@ -177,8 +251,8 @@
                   izz="0.00086563316" />
       </inertial>
-      <visual name="${side}_gripper_palm_visual">
-        <origin xyz="0 0 0" rpy="0 0 0" />
-        <geometry name="${side}_gripper_palm_visual_geom">
-          <mesh filename="package://pr2_description/meshes/gripper_v0/gripper_palm.stl" />
+      <visual>
+        <origin xyz="0 0 0" rpy="0 0 0" />
+        <geometry>
+          <mesh filename="package://pr2_description/meshes/gripper_v0/gripper_palm.stl"  />
         </geometry>
         <material name="Red" />
@@ -186,6 +260,6 @@
       <collision name="${side}_gripper_palm_collision">
         <origin xyz="0 0 0" rpy="0 0 0" />
-        <geometry name="${side}_gripper_palm_collision_geom">
-          <mesh filename="package://pr2_description/meshes/gripper_v0/gripper_palm.stl" />
+        <geometry>
+          <mesh filename="package://pr2_description/meshes/gripper_v0/gripper_palm.stl"  />
         </geometry>
         <verbose value="Yes" />
@@ -242,5 +316,13 @@
     -->
     <joint name="${side}_gripper_joint" type="prismatic">
-      <axis xyz="0 0 1" />
+      <axis xyz="0 1 0" />
+      <dynamics damping="${gripper_damping}" />
+      <limit effort="1000.0" velocity="0.2" lower="0.0" upper="0.09" />
+      <safety_controller k_velocity="5000.0" k_position="20.0" soft_lower_limit="${0.0-0.01}" soft_upper_limit="${0.09-0.002}" />
+    </joint>
+    <!-- simulated gripper joint between gripper tips -->
+    <joint name="${side}_gripper_simulated_joint" type="prismatic">
+      <axis xyz="0 1 0" />
+      <dynamics damping="${gripper_damping}" />
       <limit effort="1000.0" velocity="0.2" lower="0.0" upper="0.09" />
       <safety_controller k_velocity="5000.0" k_position="20.0" soft_lower_limit="${0.0-0.01}" soft_upper_limit="${0.09-0.002}" />

File: pr2_description/urdf/shoulder_v0/shoulder.urdf.xacro (robot description, xacro)
@@ -38,8 +38,8 @@
                  izz="0.27353821674" />
       </inertial>
-      <visual name="${side}_shoulder_pan_visual">
+      <visual>
         <origin xyz="0 0 0" rpy="0 0 0" />
-        <geometry name="${side}_shoulder_pan_visual_geom">
-          <mesh filename="package://pr2_description/meshes/shoulder_v0/shoulder_yaw.stl" />
+        <geometry>
+          <mesh filename="package://pr2_description/meshes/shoulder_v0/shoulder_pan.stl"  />
         </geometry>
         <material name="Blue" />
@@ -47,6 +47,6 @@
       <collision name="${side}_shoulder_pan_collision">
         <origin xyz="0.0 0 0.0" rpy="0 0 0" />
-        <geometry name="${side}_shoulder_pan_collision_geom">
-          <mesh filename="package://pr2_description/meshes/shoulder_v0/convex/shoulder_yaw_convex.stlb" />
+        <geometry>
+          <mesh filename="package://pr2_description/meshes/shoulder_v0/shoulder_pan.stl"  />
         </geometry>
       </collision>
@@ -75,8 +75,8 @@
                  izz="0.01975753814" />
       </inertial>
-      <visual name="${side}_shoulder_lift_visual">
+      <visual>
         <origin xyz="0 0 0" rpy="0 0 0" />
-        <geometry name="${side}_shoulder_lift_visual_geom">
-          <mesh filename="package://pr2_description/meshes/shoulder_v0/shoulder_lift.stl" />
+        <geometry>
+          <mesh filename="package://pr2_description/meshes/shoulder_v0/shoulder_lift.stl"  />
         </geometry>
         <material name="Grey" />
@@ -84,6 +84,6 @@
       <collision name="${side}_shoulder_lift_collision">
         <origin xyz="0 0 0" rpy="0 0 0" />
-        <geometry name="${side}_shoulder_lift_collision_geom">
-          <mesh filename="package://pr2_description/meshes/shoulder_v0/convex/shoulder_lift_convex.stlb" />
+        <geometry>
+          <mesh filename="package://pr2_description/meshes/shoulder_v0/shoulder_lift.stl"  />
         </geometry>
       </collision>
@@ -119,9 +119,9 @@
                   izz="0.01" />
       </inertial>
-      <visual name="${side}_upper_arm_roll_visual">
+      <visual>
         <!-- TODO: This component doesn't actually have a mesh -->
         <origin xyz="0 0 0" rpy="0 0 0" />
-        <geometry name="${side}_upper_arm_roll_visual_geom">
-          <mesh filename="package://pr2_description/meshes/shoulder_v0/upper_arm_roll.stl" />
+        <geometry>
+          <mesh filename="package://pr2_description/meshes/shoulder_v0/upper_arm_roll.stl"  />
         </geometry>
         <material name="RollLinks" />
@@ -130,5 +130,5 @@
         <!-- TODO: collision tag should be optional -->
         <origin xyz="0.0 0 0" rpy="0 0 0" />
-        <geometry name="${side}_upper_arm_roll_collision_geom">
+        <geometry>
           <box size="0.1 0.1 0.1" />
         </geometry>

File: pr2_description/urdf/torso_v0/torso.urdf.xacro (robot description, xacro)
@@ -26,8 +26,8 @@
                  iyy="2.510019507959" iyz="0.029664468704" izz="0.526432355569" />
       </inertial>
-      <visual name="${name}_visual">
+      <visual>
         <origin xyz="0 0 0" rpy="0 0 0" />
-        <geometry name="${name}_visual_geom">
-          <mesh filename="package://pr2_description/meshes/torso_v0/torso.stl" />
+        <geometry>
+          <mesh filename="package://pr2_description/meshes/torso_v0/torso_lift_2k.stl"  />
         </geometry>
         <material name="Grey2" />
@@ -35,5 +35,5 @@
       <collision name="${name}_collision">
         <origin xyz="0 0 0.16" rpy="0 0 0" />
-        <geometry name="${name}_collision_geom">
+        <geometry>
           <!-- arbitrarily chosen collision box by JH, torso collision is not important for now -->
           <box size="0.30 0.620 0.02" />
