Commit message: update simulation gripper joint:  * removed old slider "floating link".  * added parallel links to enforce tips stay parallel.  * added slider between finger tips.  * added slider to gripper transmission.  this will be used by updated pr2 gripper transmission. * new beta meshes in meters

File: pr2_description/urdf/upper_arm_v0/upper_arm.urdf.xacro (robot description, xacro)
@@ -52,5 +52,5 @@
         <origin xyz="0 0 0" rpy="0 0 0" />
         <geometry>
-          <mesh filename="package://pr2_description/meshes/upper_arm_v0/upper_arm.stl" scale="0.98 0.98 0.98" />
+          <mesh filename="package://pr2_description/meshes/upper_arm_v0/upper_arm.stl"  />
         </geometry>
         <material name="Green" />
@@ -59,31 +59,5 @@
         <origin xyz="0 0 0" rpy="0 0 0" />
         <geometry>
-          <mesh filename="package://pr2_description/meshes/upper_arm_v0/convex/upper_arm_convex.stlb" scale="0.98 0.98 0.98" />
-        </geometry>
-      </collision>
-    </link>
-    <joint name="${side}_upper_arm_sleeve_joint" type="fixed">
-      <origin xyz="0 0 0" rpy="0 0 0" />
-      <parent link="${parent}"/>
-      <child link="${side}_upper_arm_sleeve_link"/>
-    </joint>
-    <link name="${side}_upper_arm_sleeve_link">
-      <inertial>
-        <!-- NOTE:reflect==-1 for right side, reflect==1 for the left side -->
-        <mass value="0.1" />
-        <origin xyz="0 0 0" />
-        <inertia  ixx="0.01" ixy="0.00" ixz="0.00" iyy="0.01" iyz="0.00" izz="0.01" />
-      </inertial>
-      <visual>
-        <origin rpy="0 1.59 0.02" xyz="-0.015 0 0"/>
-        <geometry>
-          <mesh filename="package://pr2_description/meshes/upper_arm_v0/upper_arm.dae" scale="0.001 0.001 0.001"/>
-        </geometry>
-        <material name="Green" />
-      </visual>
-      <collision>
-        <origin rpy="0 1.59 0.02" xyz="-0.015 0 0"/>
-        <geometry>
-          <mesh filename="package://pr2_description/meshes/upper_arm_v0/upper_arm.dae" scale="0.001 0.001 0.001"/>
+          <mesh filename="package://pr2_description/meshes/upper_arm_v0/upper_arm.stl"  />
         </geometry>
       </collision>
@@ -118,8 +92,8 @@
                   izz="0.00359156824" />
       </inertial>
-      <visual name="${side}_elbow_flex_visual">
+      <visual>
         <origin xyz="0 0 0" rpy="0 0 0" />
-        <geometry name="${side}_elbow_flex_visual_geom">
-          <mesh filename="package://pr2_description/meshes/upper_arm_v0/elbow_flex.stl" />
+        <geometry>
+          <mesh filename="package://pr2_description/meshes/upper_arm_v0/elbow_flex.stl"  />
         </geometry>
         <material name="Grey" />
@@ -127,6 +101,6 @@
       <collision name="${side}_elbow_flex_collision">
         <origin xyz="0 0 0" rpy="0 0 0" />
-        <geometry name="${side}_elbow_flex_collision_geom">
-          <mesh filename="package://pr2_description/meshes/upper_arm_v0/convex/elbow_flex_convex.stlb" />
+        <geometry>
+          <mesh filename="package://pr2_description/meshes/upper_arm_v0/elbow_flex.stl"  />
         </geometry>
       </collision>
@@ -159,8 +133,8 @@
                   izz="0.01" />
       </inertial>
-      <visual name="${side}_forearm_roll_visual">
+      <visual>
         <origin xyz="0 0 0" rpy="0 0 0" />
-        <geometry name="${side}_forearm_roll_visual_geom">
-          <mesh filename="package://pr2_description/meshes/upper_arm_v0/forearm_roll.stl" />
+        <geometry>
+          <mesh filename="package://pr2_description/meshes/upper_arm_v0/forearm_roll.stl"  />
         </geometry>
         <material name="RollLinks" />
@@ -170,5 +144,5 @@
         <!-- dummy geom, to be removed -->
         <origin xyz="0 0 0" rpy="0 0 0" />
-        <geometry name="${side}_forearm_roll_collision_geom">
+        <geometry>
           <box size="0.1 0.1 0.1" />
         </geometry>

Commit message: switching collision to new beta meshes

File: pr2_description/urdf/base_v0/base.urdf.xacro (robot description, xacro)
@@ -100,7 +100,7 @@
       </visual>
       <collision>
-        <origin xyz="0 0 0.07" rpy="0.0 0.0 0.0" />
+        <origin xyz="0 0 0" rpy="0 0 0" />
         <geometry>
-          <box size="0.192 0.164 0.013" />
+          <mesh filename="package://pr2_description/meshes/base_v0/caster_L.stl" />
         </geometry>
       </collision>
@@ -137,9 +137,7 @@
       </visual>
       <collision>
-        <!-- represent base collision with a simple rectangular model, positioned by base_size_z s.t. top
-             surface of the collision box matches the top surface of the PR2 base -->
-        <origin xyz="0 0 ${base_size_z-base_collision_size_z/2}" rpy="0 0 0" />
+        <origin xyz="0 0 0" rpy="0 0 0" />
         <geometry>
-          <box size="${base_size_x} ${base_size_y} ${base_collision_size_z}" />
+          <mesh filename="package://pr2_description/meshes/base_v0/base_L.stl" />
         </geometry>
       </collision>

File: pr2_description/urdf/forearm_v0/forearm.urdf.xacro (robot description, xacro)
@@ -102,7 +102,7 @@
       </visual>
       <collision name="${side}_wrist_roll_collision">
-        <origin xyz="0.0 0 0" rpy="0 0 0" />
-        <geometry name="${side}_wrist_roll_collision_geom">
-          <box size="0.01 0.01 0.01" />
+        <origin xyz="0 0 0" rpy="0 0 0" />
+        <geometry name="${side}_wrist_roll_visual_geom">
+          <mesh filename="package://pr2_description/meshes/forearm_v0/wrist_roll_L.stl" />
         </geometry>
         <verbose value="Yes" />

File: pr2_description/urdf/shoulder_v0/shoulder.urdf.xacro (robot description, xacro)
@@ -128,8 +128,7 @@
       </visual>
       <collision name="${side}_upper_arm_roll_collision">
-        <!-- TODO: collision tag should be optional -->
-        <origin xyz="0.0 0 0" rpy="0 0 0" />
+        <origin xyz="0 0 0" rpy="0 0 0" />
         <geometry>
-          <box size="0.1 0.1 0.1" />
+          <mesh filename="package://pr2_description/meshes/shoulder_v0/upper_arm_roll_L.stl"  />
         </geometry>
       </collision>

File: pr2_description/urdf/tilting_laser_v0/tilting_laser.urdf.xacro (robot description, xacro)
@@ -35,7 +35,6 @@
       </visual>
       <collision name="${name}_mount_collision">
-        <origin xyz="0 0 0" rpy="0 0 0" />
         <geometry>
-          <box size=".001 .001 .001" />
+          <mesh filename="package://pr2_description/meshes/tilting_laser_v0/tilting_hokuyo_L.stl" />
         </geometry>
       </collision>

File: pr2_description/urdf/upper_arm_v0/upper_arm.urdf.xacro (robot description, xacro)
@@ -142,8 +142,7 @@
       <!-- TODO: collision tag should be optional -->
       <collision name="${side}_forearm_roll_collision">
-        <!-- dummy geom, to be removed -->
         <origin xyz="0 0 0" rpy="0 0 0" />
         <geometry>
-          <box size="0.1 0.1 0.1" />
+          <mesh filename="package://pr2_description/meshes/upper_arm_v0/forearm_roll_L.stl"  />
         </geometry>
       </collision>

Commit message: remove beta meshes

File: pr2_description/urdf/base_v0/base.urdf.xacro (robot description, xacro)
@@ -58,5 +58,5 @@
         <origin xyz="0 0 0" rpy="0 0 0" />
         <geometry>
-          <mesh filename="package://pr2_description/meshes/base_v0/wheel.stl" />
+          <mesh filename="package://pr2_description/meshes/base_v0/pr2_wheel.stl" />
         </geometry>
         <material name="Wheel_${suffix}" />
@@ -100,7 +100,7 @@
       </visual>
       <collision>
-        <origin xyz="0 0 0" rpy="0 0 0" />
+        <origin xyz="0 0 0.07" rpy="0.0 0.0 0.0" />
         <geometry>
-          <mesh filename="package://pr2_description/meshes/base_v0/caster_L.stl" />
+          <box size="0.192 0.164 0.013" />
         </geometry>
       </collision>
@@ -137,7 +137,9 @@
       </visual>
       <collision>
-        <origin xyz="0 0 0" rpy="0 0 0" />
+        <!-- represent base collision with a simple rectangular model, positioned by base_size_z s.t. top
+             surface of the collision box matches the top surface of the PR2 base -->
+        <origin xyz="0 0 ${base_size_z-base_collision_size_z/2}" rpy="0 0 0" />
         <geometry>
-          <mesh filename="package://pr2_description/meshes/base_v0/base_L.stl" />
+          <box size="${base_size_x} ${base_size_y} ${base_collision_size_z}" />
         </geometry>
       </collision>

File: pr2_description/urdf/forearm_v0/forearm.urdf.xacro (robot description, xacro)
@@ -25,15 +25,15 @@
                  izz="0.01659310749" />
       </inertial>
-      <visual name="${side}_forearm_visual">
+      <visual>
         <origin xyz="0 0 0" rpy="0 0 0" />
-        <geometry name="${side}_forearm_visual_geom">
+        <geometry>
           <mesh filename="package://pr2_description/meshes/forearm_v0/forearm.stl" />
         </geometry>
         <material name="Blue" />
       </visual>
-      <collision name="${side}_forearm_collision">
+      <collision>
         <origin xyz="0 0 0" rpy="0 0 0" />
-        <geometry name="${side}_forearm_collision_geom">
-          <mesh filename="package://pr2_description/meshes/forearm_v0/forearm.stl" />
+        <geometry>
+          <mesh filename="package://pr2_description/meshes/forearm_v0/convex/forearm_convex.stlb" />
         </geometry>
       </collision>
@@ -59,15 +59,15 @@
                  izz="0.00064450498" />
       </inertial>
-      <visual name="${side}_wrist_flex_visual">
+      <visual>
         <origin xyz="0 0 0" rpy="0 0 0" />
-        <geometry name="${side}_wrist_flex_visual_geom">
+        <geometry>
           <mesh filename="package://pr2_description/meshes/forearm_v0/wrist_flex.stl" />
         </geometry>
         <material name="Grey" />
       </visual>
-      <collision name="${side}_wrist_flex_collision">
+      <collision>
         <origin xyz="0 0 0" rpy="0 0 0" />
-        <geometry name="${side}_wrist_flex_collision_geom">
-          <mesh filename="package://pr2_description/meshes/forearm_v0/wrist_flex.stl" />
+        <geometry>
+          <mesh filename="package://pr2_description/meshes/forearm_v0/convex/wrist_flex_convex.stlb" />
         </geometry>
       </collision>
@@ -94,15 +94,15 @@
                  izz="0.01" />
       </inertial>
-      <visual name="${side}_wrist_roll_visual">
+      <visual>
         <origin xyz="0 0 0" rpy="0 0 0" />
-        <geometry name="${side}_wrist_roll_visual_geom">
+        <geometry>
           <mesh filename="package://pr2_description/meshes/forearm_v0/wrist_roll.stl" />
         </geometry>
         <material name="RollLinks" />
       </visual>
-      <collision name="${side}_wrist_roll_collision">
-        <origin xyz="0 0 0" rpy="0 0 0" />
-        <geometry name="${side}_wrist_roll_visual_geom">
-          <mesh filename="package://pr2_description/meshes/forearm_v0/wrist_roll_L.stl" />
+      <collision>
+        <origin xyz="0.0 0 0" rpy="0 0 0" />
+        <geometry>
+          <box size="0.01 0.01 0.01" />
         </geometry>
         <verbose value="Yes" />

File: pr2_description/urdf/gripper_v0/gripper.urdf.xacro (robot description, xacro)
@@ -49,12 +49,12 @@
         <origin xyz="0 0 0" rpy="0 0 0" />
         <geometry>
-          <mesh filename="package://pr2_description/meshes/gripper_v0/l_finger.stl" />
+          <mesh filename="package://pr2_description/meshes/gripper_v0/upper_finger_l.stl" />
         </geometry>
         <material name="Grey" />
       </visual>
-      <collision name="${prefix}_l_finger_collision">
-        <origin xyz="0 0 0" rpy="0 0 0" />
-        <geometry>
-          <mesh filename="package://pr2_description/meshes/gripper_v0/l_finger.stl" />
+      <collision>
+        <origin xyz="0 0 0" rpy="0 0 0" />
+        <geometry>
+          <mesh filename="package://pr2_description/meshes/gripper_v0/upper_finger_l.stl" />
         </geometry>
         <verbose value="Yes" />
@@ -83,14 +83,14 @@
       </inertial>
       <visual>
-        <origin xyz="0 0 0" rpy="${M_PI} 0 0" />
-        <geometry>
-          <mesh filename="package://pr2_description/meshes/gripper_v0/l_finger.stl" />
+        <origin xyz="0 0 0" rpy="0 0 0" />
+        <geometry>
+          <mesh filename="package://pr2_description/meshes/gripper_v0/upper_finger_r.stl" />
         </geometry>
         <material name="Grey" />
       </visual>
-      <collision name="${prefix}_r_finger_collision">
-        <origin xyz="0 0 0" rpy="${M_PI} 0 0" />
-        <geometry>
-          <mesh filename="package://pr2_description/meshes/gripper_v0/l_finger.stl" />
+      <collision>
+        <origin xyz="0 0 0" rpy="0 0 0" />
+        <geometry>
+          <mesh filename="package://pr2_description/meshes/gripper_v0/upper_finger_r.stl" />
         </geometry>
         <verbose value="Yes" />
@@ -189,12 +189,12 @@
         <origin xyz="0 0 0" rpy="0 0 0" />
         <geometry>
-          <mesh filename="package://pr2_description/meshes/gripper_v0/l_finger_tip.stl" />
+          <mesh filename="package://pr2_description/meshes/gripper_v0/finger_tip_l.stl" />
         </geometry>
         <material name="Green" />
       </visual>
-      <collision name="${prefix}_l_finger_tip_collision">
-        <origin xyz="0 0 0" rpy="0 0 0" />
-        <geometry>
-          <mesh filename="package://pr2_description/meshes/gripper_v0/l_finger_tip.stl" />
+      <collision>
+        <origin xyz="0 0 0" rpy="0 0 0" />
+        <geometry>
+          <mesh filename="package://pr2_description/meshes/gripper_v0/finger_tip_pad2_l.stl" />
         </geometry>
         <verbose value="Yes" />
@@ -220,14 +220,14 @@
       </inertial>
       <visual>
-        <origin xyz="0 0 0" rpy="${M_PI} 0 0" />
-        <geometry>
-          <mesh filename="package://pr2_description/meshes/gripper_v0/l_finger_tip.stl"  />
+        <origin xyz="0 0 0" rpy="0 0 0" />
+        <geometry>
+          <mesh filename="package://pr2_description/meshes/gripper_v0/finger_tip_r.stl" />
         </geometry>
         <material name="Green" />
       </visual>
-      <collision name="${prefix}_r_finger_tip_collision">
-        <origin xyz="0 0 0" rpy="${M_PI} 0 0" />
-        <geometry>
-          <mesh filename="package://pr2_description/meshes/gripper_v0/l_finger_tip.stl"  />
+      <collision>
+        <origin xyz="0 0 0" rpy="0 0 0" />
+        <geometry>
+          <mesh filename="package://pr2_description/meshes/gripper_v0/finger_tip_pad2_r.stl" />
         </geometry>
         <verbose value="Yes" />
@@ -258,5 +258,5 @@
         <material name="Red" />
       </visual>
-      <collision name="${side}_gripper_palm_collision">
+      <collision>
         <origin xyz="0 0 0" rpy="0 0 0" />
         <geometry>

File: pr2_description/urdf/head_v0/head.urdf.xacro (robot description, xacro)
@@ -34,7 +34,7 @@
       </visual>
       <collision>
-        <origin xyz="0 0 0.0" rpy="0 0 0 " />
+        <origin xyz="-0.005717  0.010312 -0.029649" rpy="0.0 0.0 0.0 " />
         <geometry>
-          <mesh filename="package://pr2_description/meshes/head_v0/head_pan_L.stl"  />
+          <box size="0.188 0.219 0.137" />
         </geometry>
       </collision>
@@ -72,7 +72,7 @@
       </visual>
       <collision>
-        <origin xyz="0 0 0" rpy="0.0 0.0 0.0" />
+        <origin xyz="0.041935 0.003569 0.028143" rpy="0 0 0" />
         <geometry>
-          <mesh filename="package://pr2_description/meshes/head_v0/head_tilt_L.stl"  />
+          <box size="0.064 0.253 0.181" />
         </geometry>
       </collision>

File: pr2_description/urdf/sensors/head_sensor_package.urdf.xacro (robot description, xacro)
@@ -36,5 +36,5 @@
         <material name="Blue" />
       </visual>
-      <collision name="${name}_sensor_collision">
+      <collision>
         <origin xyz="0 0 0" rpy="0 0 0" />
         <geometry>

File: pr2_description/urdf/shoulder_v0/shoulder.urdf.xacro (robot description, xacro)
@@ -41,12 +41,12 @@
         <origin xyz="0 0 0" rpy="0 0 0" />
         <geometry>
-          <mesh filename="package://pr2_description/meshes/shoulder_v0/shoulder_pan.stl"  />
+          <mesh filename="package://pr2_description/meshes/shoulder_v0/shoulder_yaw.stl"  />
         </geometry>
         <material name="Blue" />
       </visual>
-      <collision name="${side}_shoulder_pan_collision">
+      <collision>
         <origin xyz="0.0 0 0.0" rpy="0 0 0" />
         <geometry>
-          <mesh filename="package://pr2_description/meshes/shoulder_v0/shoulder_pan.stl"  />
+          <mesh filename="package://pr2_description/meshes/shoulder_v0/convex/shoulder_yaw_convex.stlb" />
         </geometry>
       </collision>
@@ -82,8 +82,8 @@
         <material name="Grey" />
       </visual>
-      <collision name="${side}_shoulder_lift_collision">
+      <collision>
         <origin xyz="0 0 0" rpy="0 0 0" />
         <geometry>
-          <mesh filename="package://pr2_description/meshes/shoulder_v0/shoulder_lift.stl"  />
+          <mesh filename="package://pr2_description/meshes/shoulder_v0/convex/shoulder_lift_convex.stlb" />
         </geometry>
       </collision>
@@ -127,8 +127,9 @@
         <material name="RollLinks" />
       </visual>
-      <collision name="${side}_upper_arm_roll_collision">
-        <origin xyz="0 0 0" rpy="0 0 0" />
+      <collision>
+        <!-- TODO: collision tag should be optional -->
+        <origin xyz="0.0 0 0" rpy="0 0 0" />
         <geometry>
-          <mesh filename="package://pr2_description/meshes/shoulder_v0/upper_arm_roll_L.stl"  />
+          <box size="0.1 0.1 0.1" />
         </geometry>
       </collision>

File: pr2_description/urdf/tilting_laser_v0/tilting_laser.urdf.xacro (robot description, xacro)
@@ -30,11 +30,12 @@
         <origin xyz="0 0 0" rpy="0 0 0" />
         <geometry>
-          <mesh filename="package://pr2_description/meshes/tilting_laser_v0/tilting_hokuyo.stl" />
+          <mesh filename="package://pr2_description/meshes/tilting_laser_v0/hok_tilt.stl" />
         </geometry>
         <material name="Red" />
       </visual>
-      <collision name="${name}_mount_collision">
+      <collision>
+        <origin xyz="0 0 0" rpy="0 0 0" />
         <geometry>
-          <mesh filename="package://pr2_description/meshes/tilting_laser_v0/tilting_hokuyo_L.stl" />
+          <box size=".001 .001 .001" />
         </geometry>
       </collision>

File: pr2_description/urdf/torso_v0/torso.urdf.xacro (robot description, xacro)
@@ -29,12 +29,13 @@
         <origin xyz="0 0 0" rpy="0 0 0" />
         <geometry>
-          <mesh filename="package://pr2_description/meshes/torso_v0/torso_lift.stl"  />
+          <mesh filename="package://pr2_description/meshes/torso_v0/torso.stl" />
         </geometry>
         <material name="Grey2" />
       </visual>
-      <collision name="${name}_collision">
-        <origin xyz="0 0 0" rpy="0 0 0" />
+      <collision>
+        <origin xyz="0 0 0.16" rpy="0 0 0" />
         <geometry>
-          <mesh filename="package://pr2_description/meshes/torso_v0/torso_lift_L.stl"  />
+          <!-- arbitrarily chosen collision box by JH, torso collision is not important for now -->
+          <box size="0.30 0.620 0.02" />
         </geometry>
       </collision>

File: pr2_description/urdf/upper_arm_v0/upper_arm.urdf.xacro (robot description, xacro)
@@ -56,8 +56,8 @@
         <material name="Green" />
       </visual>
-      <collision name="${side}_upper_arm_collision">
+      <collision>
         <origin xyz="0 0 0" rpy="0 0 0" />
         <geometry>
-          <mesh filename="package://pr2_description/meshes/upper_arm_v0/upper_arm.stl"  />
+          <mesh filename="package://pr2_description/meshes/upper_arm_v0/convex/upper_arm_convex.stlb" />
         </geometry>
       </collision>
@@ -99,8 +99,8 @@
         <material name="Grey" />
       </visual>
-      <collision name="${side}_elbow_flex_collision">
+      <collision>
         <origin xyz="0 0 0" rpy="0 0 0" />
         <geometry>
-          <mesh filename="package://pr2_description/meshes/upper_arm_v0/elbow_flex.stl"  />
+          <mesh filename="package://pr2_description/meshes/upper_arm_v0/convex/elbow_flex_convex.stlb" />
         </geometry>
       </collision>
@@ -141,8 +141,9 @@
       </visual>
       <!-- TODO: collision tag should be optional -->
-      <collision name="${side}_forearm_roll_collision">
+      <collision>
+        <!-- dummy geom, to be removed -->
         <origin xyz="0 0 0" rpy="0 0 0" />
         <geometry>
-          <mesh filename="package://pr2_description/meshes/upper_arm_v0/forearm_roll_L.stl"  />
+          <box size="0.1 0.1 0.1" />
         </geometry>
       </collision>

Commit message: #5126 removal of extra stuff in pr2 urdf

File: pr2_description/urdf/base_v0/base.urdf.xacro (robot description, xacro)
@@ -193,5 +193,4 @@
           <box size="0.05 0.37 0.3" />
         </geometry>
-        <material name="Black" />
       </collision>
     </link>

File: pr2_description/urdf/forearm_v0/forearm.urdf.xacro (robot description, xacro)
@@ -104,5 +104,4 @@
           <mesh filename="package://pr2_description/meshes/forearm_v0/wrist_roll_L.stl" />
         </geometry>
-        <verbose value="Yes" />
       </collision>
     </link>

File: pr2_description/urdf/gripper_v0/gripper.urdf.xacro (robot description, xacro)
@@ -58,5 +58,4 @@
           <mesh filename="package://pr2_description/meshes/gripper_v0/l_finger.stl" />
         </geometry>
-        <verbose value="Yes" />
       </collision>
     </link>
@@ -94,5 +93,4 @@
           <mesh filename="package://pr2_description/meshes/gripper_v0/l_finger.stl" />
         </geometry>
-        <verbose value="Yes" />
       </collision>
     </link>
@@ -127,5 +125,4 @@
           <mesh filename="package://pr2_description/meshes/gripper_v0/l_finger_tip.stl" />
         </geometry>
-        <verbose value="Yes" />
       </collision>
     </link>
@@ -160,5 +157,4 @@
           <mesh filename="package://pr2_description/meshes/gripper_v0/l_finger_tip.stl"  />
         </geometry>
-        <verbose value="Yes" />
       </collision>
     </link>
@@ -192,5 +188,4 @@
           <mesh filename="package://pr2_description/meshes/gripper_v0/gripper_palm.stl"  />
         </geometry>
-        <verbose value="Yes" />
       </collision>
     </link>

File: pr2_description/urdf/head_v0/head.urdf.xacro (robot description, xacro)
@@ -39,5 +39,4 @@
     </link>
     <!-- extensions -->
-    <xacro:pr2_head_pan_gazebo_v0 name="${name}" />
     <xacro:pr2_head_pan_transmission_v0 name="${name}" />
   </xacro:macro>
@@ -76,5 +75,4 @@
     </link>
     <!-- extensions -->
-    <xacro:pr2_head_tilt_gazebo_v0 name="${name}" />
     <xacro:pr2_head_tilt_transmission_v0 name="${name}" />
   </xacro:macro>
