Commit message: caster and wheel effort velocity limits #5031

File: pr2_description/urdf/base_v0/base.urdf.xacro (robot description, xacro)
@@ -41,7 +41,7 @@
     <joint name="${parent}_${suffix}_wheel_joint" type="continuous">
       <axis xyz="0 1 0" />
-      <limit effort="100" velocity="100"/> <!-- alpha tested effort and velocity limits -->
+      <limit effort="7" velocity="15"/> <!-- alpha tested effort and velocity limits -->
       <safety_controller  k_velocity="10" />
-      <dynamics damping="0.0" friction="0.0" />
+      <dynamics damping="1.0" friction="0.0" />
       <origin xyz="0 ${reflect*caster_wheel_offset_y} 0" rpy="0 0 0" />
       <parent link="${parent}_rotation_link"/>
@@ -77,8 +77,8 @@
     <joint name="${suffix}_rotation_joint" type="continuous">
       <axis xyz="0 0 1" />
-      <limit effort="100" velocity="100"/> <!-- alpha tested velocity and effort limits -->
+      <limit effort="6.5" velocity="10"/> <!-- alpha tested velocity and effort limits -->
       <safety_controller  k_velocity="10" />
       <calibration rising="${ref_position}" />
-      <dynamics damping="0.0" friction="0.0" />
+      <dynamics damping="1.0" friction="0.0" />
       <insert_block name="origin" />
       <parent link="${parent}"/>
