Commit message: Prepend xacro tags with xacro xml namespace

File: pr2_description/urdf/base_v0/base.urdf.xacro (robot description, xacro)
@@ -11,28 +11,28 @@
   <!-- all link geometry sizes are obtained from Function provided CAD model unless stated otherwise -->
   <!-- all simplified collision geometry are hand approximated from CAD model, sometimes from respective bounding boxes -->
-  <property name="M_PI" value="3.1415926535897931" />
-  <property name="caster_offset_x" value="0.2246" />
-  <property name="caster_offset_y" value="0.2246" />
-  <property name="caster_offset_z" value="0.0282" />
-  <property name="caster_wheel_offset_y" value="0.049" />
-  <property name="wheel_length" value="0.034" />
-  <property name="wheel_radius" value="0.074792" />   <!-- This is the 'effective' wheel radius. Wheel radius for uncompressed wheel is 0.079.  mp 20080801 -->
-  <property name="base_cg_x" value="-0.061" />
-  <property name="base_cg_y" value="0.0" />
-  <property name="base_cg_z" value="${0.5*0.293}" />
-  <property name="base_mass" value="116.0" />
+  <xacro:property name="M_PI" value="3.1415926535897931" />
+  <xacro:property name="caster_offset_x" value="0.2246" />
+  <xacro:property name="caster_offset_y" value="0.2246" />
+  <xacro:property name="caster_offset_z" value="0.0282" />
+  <xacro:property name="caster_wheel_offset_y" value="0.049" />
+  <xacro:property name="wheel_length" value="0.034" />
+  <xacro:property name="wheel_radius" value="0.074792" />   <!-- This is the 'effective' wheel radius. Wheel radius for uncompressed wheel is 0.079.  mp 20080801 -->
+  <xacro:property name="base_cg_x" value="-0.061" />
+  <xacro:property name="base_cg_y" value="0.0" />
+  <xacro:property name="base_cg_z" value="${0.5*0.293}" />
+  <xacro:property name="base_mass" value="116.0" />
   <!-- simplified box collision geometry for base -->
-  <property name="base_size_x" value="0.65" />
-  <property name="base_size_y" value="0.65" />
-  <property name="base_size_z" value="0.23" />
-  <property name="base_collision_size_z" value="0.04" />
+  <xacro:property name="base_size_x" value="0.65" />
+  <xacro:property name="base_size_y" value="0.65" />
+  <xacro:property name="base_size_z" value="0.23" />
+  <xacro:property name="base_collision_size_z" value="0.04" />
   <!-- simplified box collision geometry for hokuyo laser -->
-  <property name="base_laser_x" value="0.275" />
-  <property name="base_laser_y" value="0.0" />
-  <property name="base_laser_z" value="0.252" />
-  <property name="base_laser_size_x" value="0.06" />
-  <property name="base_laser_size_y" value="0.06" />
-  <property name="base_laser_size_z" value="0.03" />
-  <property name="base_laser_collision_offset_z" value="0.023" />
+  <xacro:property name="base_laser_x" value="0.275" />
+  <xacro:property name="base_laser_y" value="0.0" />
+  <xacro:property name="base_laser_z" value="0.252" />
+  <xacro:property name="base_laser_size_x" value="0.06" />
+  <xacro:property name="base_laser_size_y" value="0.06" />
+  <xacro:property name="base_laser_size_z" value="0.03" />
+  <xacro:property name="base_laser_collision_offset_z" value="0.023" />
   <!--                                                      -->
   <!--           wheel                                      -->
@@ -81,5 +81,5 @@
       <calibration rising="${ref_position}" />
       <dynamics damping="1.0" friction="0.0" />
-      <insert_block name="origin" />
+      <xacro:insert_block name="origin" />
       <parent link="${parent}"/>
       <child link="${suffix}_rotation_link" />
@@ -112,5 +112,5 @@
     <xacro:pr2_caster_hub_v0 parent="${parent}" suffix="${suffix}_caster"
                              ref_position="${ref_position}" >
-      <insert_block name="origin" />
+      <xacro:insert_block name="origin" />
     </xacro:pr2_caster_hub_v0>
     <!-- wheel macros -->

File: pr2_description/urdf/common.xacro (robot description, xacro)
@@ -1,60 +1,63 @@
 <?xml version="1.0"?>
-<robot>
-  <property name="M_PI" value="3.1415926535897931" />
-  <property name="VELOCITY_LIMIT_SCALE" value="0.6" />
+<robot xmlns:sensor="http://playerstage.sourceforge.net/gazebo/xmlschema/#sensor"
+       xmlns:controller="http://playerstage.sourceforge.net/gazebo/xmlschema/#controller"
+       xmlns:interface="http://playerstage.sourceforge.net/gazebo/xmlschema/#interface"
+       xmlns:xacro="http://ros.org/wiki/xacro">
+  <xacro:property name="M_PI" value="3.1415926535897931" />
+  <xacro:property name="VELOCITY_LIMIT_SCALE" value="0.6" />
   <!-- Gear Ratio Corrections: Divide transmission reductions by these factors (Nominally 1)-->
-  <property name="cal_r_shoulder_pan_gearing"   value="1.0" />
-  <property name="cal_r_shoulder_lift_gearing"  value="1.0" />
-  <property name="cal_r_upper_arm_roll_gearing" value="1.0" />
+  <xacro:property name="cal_r_shoulder_pan_gearing"   value="1.0" />
+  <xacro:property name="cal_r_shoulder_lift_gearing"  value="1.0" />
+  <xacro:property name="cal_r_upper_arm_roll_gearing" value="1.0" />
   <!-- ********** Right Arm ********** -->
   <!-- Flag offsets: Add to the optical flag locations (Nominally 0) -->
-  <property name="cal_r_shoulder_pan_flag"   value="0.0" />
-  <property name="cal_r_shoulder_lift_flag"  value="0.0" />
-  <property name="cal_r_upper_arm_roll_flag" value="0.0" />
-  <property name="cal_r_elbow_flex_flag"     value="0.0" />
-  <property name="cal_r_forearm_roll_flag"   value="0.0" />
-  <property name="cal_r_wrist_flex_flag"     value="0.0" />
-  <property name="cal_r_wrist_roll_flag"     value="0.0" />
+  <xacro:property name="cal_r_shoulder_pan_flag"   value="0.0" />
+  <xacro:property name="cal_r_shoulder_lift_flag"  value="0.0" />
+  <xacro:property name="cal_r_upper_arm_roll_flag" value="0.0" />
+  <xacro:property name="cal_r_elbow_flex_flag"     value="0.0" />
+  <xacro:property name="cal_r_forearm_roll_flag"   value="0.0" />
+  <xacro:property name="cal_r_wrist_flex_flag"     value="0.0" />
+  <xacro:property name="cal_r_wrist_roll_flag"     value="0.0" />
   <!-- ********** Head ********** -->
   <!-- Head Location: Add to the transform from torso to head_pan_link (Nominally 0) -->
-  <property name="cal_head_x" value="0.0" />
-  <property name="cal_head_y" value="0.0" />
-  <property name="cal_head_z" value="0.0" />
-  <property name="cal_head_roll" value="0.0" />
-  <property name="cal_head_pitch" value="0.0" />
-  <property name="cal_head_yaw" value="0.0" />
+  <xacro:property name="cal_head_x" value="0.0" />
+  <xacro:property name="cal_head_y" value="0.0" />
+  <xacro:property name="cal_head_z" value="0.0" />
+  <xacro:property name="cal_head_roll" value="0.0" />
+  <xacro:property name="cal_head_pitch" value="0.0" />
+  <xacro:property name="cal_head_yaw" value="0.0" />
   <!-- Flag Offsets -->
-  <property name="cal_head_pan_flag"  value="0.0" />
-  <property name="cal_head_tilt_flag" value="0.0" />
-  <property name="cal_head_pan_flag" value="0.0"/>
-  <property name="cal_head_tilt_flag" value="0.0"/>
+  <xacro:property name="cal_head_pan_flag"  value="0.0" />
+  <xacro:property name="cal_head_tilt_flag" value="0.0" />
+  <xacro:property name="cal_head_pan_flag" value="0.0"/>
+  <xacro:property name="cal_head_tilt_flag" value="0.0"/>
   <!-- Casters -->
-  <property name="cal_caster_fl" value="0.0" />
-  <property name="cal_caster_fr" value="0.0" />
-  <property name="cal_caster_bl" value="0.0" />
-  <property name="cal_caster_br" value="0.0" />
+  <xacro:property name="cal_caster_fl" value="0.0" />
+  <xacro:property name="cal_caster_fr" value="0.0" />
+  <xacro:property name="cal_caster_bl" value="0.0" />
+  <xacro:property name="cal_caster_br" value="0.0" />
   <!-- Stereo Camera Location (Nominally 0) -->
-  <property name="cal_stereo_x" value="0.0" />
-  <property name="cal_stereo_y" value="0.0" />
-  <property name="cal_stereo_z" value="0.0" />
-  <property name="cal_stereo_roll" value="0.0" />
-  <property name="cal_stereo_pitch" value="0.0" />
-  <property name="cal_stereo_yaw" value="0.0" />
+  <xacro:property name="cal_stereo_x" value="0.0" />
+  <xacro:property name="cal_stereo_y" value="0.0" />
+  <xacro:property name="cal_stereo_z" value="0.0" />
+  <xacro:property name="cal_stereo_roll" value="0.0" />
+  <xacro:property name="cal_stereo_pitch" value="0.0" />
+  <xacro:property name="cal_stereo_yaw" value="0.0" />
   <!-- Kinect Camera Location (Nominally 0) -->
-  <property name="cal_kinect_x" value="0.0" />
-  <property name="cal_kinect_y" value="0.0" />
-  <property name="cal_kinect_z" value="0.0" />
-  <property name="cal_kinect_roll" value="0.0" />
-  <property name="cal_kinect_pitch" value="0.0" />
-  <property name="cal_kinect_yaw" value="0.0" />
+  <xacro:property name="cal_kinect_x" value="0.0" />
+  <xacro:property name="cal_kinect_y" value="0.0" />
+  <xacro:property name="cal_kinect_z" value="0.0" />
+  <xacro:property name="cal_kinect_roll" value="0.0" />
+  <xacro:property name="cal_kinect_pitch" value="0.0" />
+  <xacro:property name="cal_kinect_yaw" value="0.0" />
   <!-- HighDef Camera Location (Nominally 0) -->
-  <property name="cal_high_def_x" value="0.0" />
-  <property name="cal_high_def_y" value="0.0" />
-  <property name="cal_high_def_z" value="0.0" />
-  <property name="cal_high_def_roll" value="0.0" />
-  <property name="cal_high_def_pitch" value="0.0" />
-  <property name="cal_high_def_yaw" value="0.0" />
+  <xacro:property name="cal_high_def_x" value="0.0" />
+  <xacro:property name="cal_high_def_y" value="0.0" />
+  <xacro:property name="cal_high_def_z" value="0.0" />
+  <xacro:property name="cal_high_def_roll" value="0.0" />
+  <xacro:property name="cal_high_def_pitch" value="0.0" />
+  <xacro:property name="cal_high_def_yaw" value="0.0" />
   <!-- Throwing in left arm constants to appease the xacro parser -->
-  <property name="cal_l_shoulder_pan_flag" value="0.000000" />
-  <property name="cal_l_wrist_roll_flag" value="0.0" />
+  <xacro:property name="cal_l_shoulder_pan_flag" value="0.000000" />
+  <xacro:property name="cal_l_wrist_roll_flag" value="0.0" />
 </robot>

File: pr2_description/urdf/forearm_v0/forearm.urdf.xacro (robot description, xacro)
@@ -13,5 +13,5 @@
   <xacro:macro name="pr2_forearm_v0" params="side parent reflect *origin">
     <joint name="${side}_forearm_joint" type="fixed">
-      <insert_block name="origin" /> <!-- transform from parent link to this joint frame -->
+      <xacro:insert_block name="origin" /> <!-- transform from parent link to this joint frame -->
       <parent link="${parent}"/>
       <child link="${side}_forearm_link"/>

File: pr2_description/urdf/gripper_v0/gripper.gazebo.xacro (robot description, xacro)
@@ -1,17 +1,17 @@
 <?xml version="1.0"?>
 <robot xmlns:xacro="http://ros.org/wiki/xacro">
-  <property name="finger_stop_kd"             value="1.0" />
-  <property name="finger_stop_kp"             value="10000000.0" />
-  <property name="finger_fudge_factor"        value="1.0" />
-  <property name="finger_kp"                  value="0.0" />
-  <property name="finger_kd"                  value="0.0" />
-  <property name="finger_fm"                  value="0.0" />
-  <property name="finger_tip_kp"              value="0.0" />
-  <property name="finger_tip_kd"              value="0.0" />
-  <property name="finger_tip_fm"              value="0.0" />
-  <property name="finger_tip_mu"              value="500.0" />
-  <property name="finger_mu"                  value="500.0" />
-  <property name="parallel_link_x_offset"     value="-0.018" />
-  <property name="parallel_link_y_offset"     value="0.021" />
+  <xacro:property name="finger_stop_kd"             value="1.0" />
+  <xacro:property name="finger_stop_kp"             value="10000000.0" />
+  <xacro:property name="finger_fudge_factor"        value="1.0" />
+  <xacro:property name="finger_kp"                  value="0.0" />
+  <xacro:property name="finger_kd"                  value="0.0" />
+  <xacro:property name="finger_fm"                  value="0.0" />
+  <xacro:property name="finger_tip_kp"              value="0.0" />
+  <xacro:property name="finger_tip_kd"              value="0.0" />
+  <xacro:property name="finger_tip_fm"              value="0.0" />
+  <xacro:property name="finger_tip_mu"              value="500.0" />
+  <xacro:property name="finger_mu"                  value="500.0" />
+  <xacro:property name="parallel_link_x_offset"     value="-0.018" />
+  <xacro:property name="parallel_link_y_offset"     value="0.021" />
   <xacro:macro name="pr2_finger_gazebo_v0" params="prefix reflect">
     <!-- Finger proximal digit -->

File: pr2_description/urdf/gripper_v0/gripper.urdf.xacro (robot description, xacro)
@@ -7,13 +7,13 @@
   <xacro:include filename="$(find pr2_description)/urdf/gripper_v0/gripper.gazebo.xacro" />
   <xacro:include filename="$(find pr2_description)/urdf/gripper_v0/gripper.transmission.xacro" />
-  <property name="M_PI" value="3.1415926535897931" />
-  <property name="gripper_upper_angle" value="0.548" />
-  <property name="gripper_lower_angle" value="0.00" />
-  <property name="finger_damping"             value="0.02" />
-  <property name="gripper_damping"            value="10.0" />
-  <property name="finger_tip_damping"         value="0.001" />
-  <property name="finger_joint_effort_limit"  value="1000.0" />
-  <property name="finger_to_finger_tip_x"     value="0.09137" />
-  <property name="palm_to_finger_x"           value="0.07691" />
+  <xacro:property name="M_PI" value="3.1415926535897931" />
+  <xacro:property name="gripper_upper_angle" value="0.548" />
+  <xacro:property name="gripper_lower_angle" value="0.00" />
+  <xacro:property name="finger_damping"             value="0.02" />
+  <xacro:property name="gripper_damping"            value="10.0" />
+  <xacro:property name="finger_tip_damping"         value="0.001" />
+  <xacro:property name="finger_joint_effort_limit"  value="1000.0" />
+  <xacro:property name="finger_to_finger_tip_x"     value="0.09137" />
+  <xacro:property name="palm_to_finger_x"           value="0.07691" />
   <xacro:macro name="pr2_finger_limits_v0">
     <!-- limits on passive finger and finger top joints without
@@ -164,5 +164,5 @@
   <xacro:macro name="pr2_gripper_v0" params="side reflect parent *origin gear_ratio screw_reduction theta0 phi0 t0 L0 h a b r">
     <joint name="${side}_gripper_palm_joint" type="fixed">
-      <insert_block name="origin"/>
+      <xacro:insert_block name="origin"/>
       <parent link="${parent}"/>
       <child link="${side}_gripper_palm_link"/>

File: pr2_description/urdf/head_v0/head.urdf.xacro (robot description, xacro)
@@ -6,5 +6,5 @@
   <xacro:include filename="$(find pr2_description)/urdf/head_v0/head.gazebo.xacro" />
   <xacro:include filename="$(find pr2_description)/urdf/head_v0/head.transmission.xacro" />
-  <property name="M_PI" value="3.1415926535897931" />
+  <xacro:property name="M_PI" value="3.1415926535897931" />
   <xacro:macro name="pr2_head_pan_v0" params="name parent *origin">
     <joint name="${name}_joint" type="revolute">
@@ -14,5 +14,5 @@
       <calibration rising="0.0" />
       <dynamics damping="0.5" />
-      <insert_block name="origin" />
+      <xacro:insert_block name="origin" />
       <parent link="${parent}"/>
       <child link="${name}_link"/>
@@ -48,5 +48,5 @@
       <calibration falling="${0.0+cal_head_tilt_flag}" />
       <dynamics damping="10.0" />
-      <insert_block name="origin" />
+      <xacro:insert_block name="origin" />
       <parent link="${parent}"/>
       <child link="${name}_link"/>
@@ -79,5 +79,5 @@
   <xacro:macro name="pr2_head_v0" params="name parent *origin">
     <xacro:pr2_head_pan_v0 name="${name}_pan" parent="${parent}">
-      <insert_block name="origin" />
+      <xacro:insert_block name="origin" />
     </xacro:pr2_head_pan_v0>
     <xacro:pr2_head_tilt_v0 name="${name}_tilt" parent="${name}_pan_link">

File: pr2_description/urdf/sensors/double_stereo_camera.urdf.xacro (robot description, xacro)
@@ -6,9 +6,9 @@
   <xacro:include filename="$(find pr2_description)/urdf/sensors/double_stereo_camera.gazebo.xacro" />
   <xacro:include filename="$(find pr2_description)/urdf/sensors/stereo_camera.urdf.xacro" />
-  <property name="stereo_size_x" value="0.02" />
-  <property name="stereo_size_y" value="0.12" />
-  <property name="stereo_size_z" value="0.05" />
-  <property name="stereo_center_box_center_offset_x" value="-0.01" />
-  <property name="stereo_center_box_center_offset_z" value="0.025" />
+  <xacro:property name="stereo_size_x" value="0.02" />
+  <xacro:property name="stereo_size_y" value="0.12" />
+  <xacro:property name="stereo_size_z" value="0.05" />
+  <xacro:property name="stereo_center_box_center_offset_x" value="-0.01" />
+  <xacro:property name="stereo_center_box_center_offset_z" value="0.025" />
   <!-- Made by Kevin for double stereo camera for PR-2 Beta. -->
   <!-- Needs calibration verification, and CAD check. -->
@@ -16,5 +16,5 @@
     <!-- Define link to stereo cameras, set origin relative to that -->
     <joint name="${name}_frame_joint" type="fixed">
-      <insert_block name="origin" />
+      <xacro:insert_block name="origin" />
       <parent link="${parent}"/>
       <child link="${name}_link"/>

File: pr2_description/urdf/sensors/head_sensor_package.gazebo.xacro (robot description, xacro)
@@ -4,5 +4,5 @@
        xmlns:interface="http://playerstage.sourceforge.net/gazebo/xmlschema/#interface"
        xmlns:xacro="http://ros.org/wiki/xacro">
-  <property name="M_PI" value="3.1415926535897931" />
+  <xacro:property name="M_PI" value="3.1415926535897931" />
   <!-- Made by Kevin for A2 sensor package -->
   <!-- Origin is center mount screw on sensor plate mount -->

File: pr2_description/urdf/sensors/head_sensor_package.urdf.xacro (robot description, xacro)
@@ -16,5 +16,5 @@
   <xacro:macro name="pr2_head_sensor_package_v0" params="name hd_frame_name hd_camera_name stereo_name parent *origin">
     <joint name="${name}_frame_joint" type="fixed">
-      <insert_block name="origin" />
+      <xacro:insert_block name="origin" />
       <parent link="${parent}"/>
       <child link="${name}_link"/>

File: pr2_description/urdf/sensors/hokuyo_lx30_laser.urdf.xacro (robot description, xacro)
@@ -8,5 +8,5 @@
     <joint name="${name}_joint" type="fixed">
       <axis xyz="0 1 0" />
-      <insert_block name="origin" />
+      <xacro:insert_block name="origin" />
       <parent link="${parent}_link"/>
       <child link="${name}_link"/>

File: pr2_description/urdf/sensors/kinect2.urdf.xacro (robot description, xacro)
@@ -2,9 +2,9 @@
 <robot xmlns:xacro="http://ros.org/wiki/xacro">
   <xacro:include filename="$(find pr2_description)/urdf/sensors/kinect2.gazebo.xacro" />
-  <property name="ir_depth_rgb_offset_y" value="0.01"/> <!-- FIXME: what is this offset? -->
+  <xacro:property name="ir_depth_rgb_offset_y" value="0.01"/> <!-- FIXME: what is this offset? -->
   <!-- Kinect2 and mount assembly -->
   <xacro:macro name="kinect2_v0" params="name parent *origin">
     <joint name="${name}_kinect2_joint" type="fixed">
-      <insert_block name="origin" />
+      <xacro:insert_block name="origin" />
       <parent link="${parent}"/>
       <child link="${name}_kinect2_link"/>

File: pr2_description/urdf/sensors/kinect_camera.urdf.xacro (robot description, xacro)
@@ -7,5 +7,5 @@
   <xacro:macro name="kinect_camera_v0" params="name parent *origin">
     <joint name="${name}_frame_joint" type="fixed">
-      <insert_block name="origin" />
+      <xacro:insert_block name="origin" />
       <parent link="${parent}"/>
       <child link="${name}_frame"/>

File: pr2_description/urdf/sensors/kinect_prosilica_camera.urdf.xacro (robot description, xacro)
@@ -5,5 +5,5 @@
       xmlns:xacro="http://ros.org/wiki/xacro">
   <xacro:include filename="$(find pr2_description)/urdf/sensors/kinect_prosilica_camera.gazebo.xacro" />
-  <property name="ir_depth_rgb_offset_y" value="0.01"/> <!-- FIXME: what is this offset? -->
+  <xacro:property name="ir_depth_rgb_offset_y" value="0.01"/> <!-- FIXME: what is this offset? -->
   <!-- kinect and prosilica combo -->
   <xacro:macro name="kinect_prosilica_camera_swept_back_v0" params="name parent *origin">
@@ -11,5 +11,5 @@
     <joint name="${name}_joint" type="fixed">
       <!-- <limit lower="0.1" upper="0.1" effort="10000" velocity="100.0"/> -->
-      <!-- <insert_block name="origin" /> -->
+      <!-- <xacro:insert_block name="origin" /> -->
       <origin xyz="-0.138 0 0.091" rpy="0 0 0"/>
       <parent link="${parent}"/>

File: pr2_description/urdf/sensors/microstrain_3dmgx2_imu.urdf.xacro (robot description, xacro)
@@ -5,5 +5,5 @@
     <joint name="${name}_joint" type="fixed">
       <axis xyz="0 1 0" />
-      <insert_block name="origin" />
+      <xacro:insert_block name="origin" />
       <parent link="${parent}_link"/>
       <child link="${name}_link"/>

File: pr2_description/urdf/sensors/projector_wg6802418.urdf.xacro (robot description, xacro)
@@ -7,5 +7,5 @@
   <xacro:macro name="projector_wg6802418_v0" params="name parent *origin">
     <joint name="${name}_frame_joint" type="fixed">
-      <insert_block name="origin" />
+      <xacro:insert_block name="origin" />
       <parent link="${parent}"/>
       <child link="${name}_frame"/>

File: pr2_description/urdf/sensors/prosilica_gc2450_camera.urdf.xacro (robot description, xacro)
@@ -7,5 +7,5 @@
   <xacro:macro name="prosilica_cam_v0" params="frame_name parent *origin camera_name">
     <joint name="${frame_name}_frame_joint" type="fixed">
-      <insert_block name="origin" />
+      <xacro:insert_block name="origin" />
       <parent link="${parent}"/>
       <child link="${frame_name}_frame"/>

File: pr2_description/urdf/sensors/stereo_camera.urdf.xacro (robot description, xacro)
@@ -7,14 +7,14 @@
   <xacro:include filename="$(find pr2_description)/urdf/sensors/wge100_camera.urdf.xacro" />
   <xacro:include filename="$(find pr2_description)/urdf/sensors/stereo_camera.gazebo.xacro" />
-  <property name="stereo_dx" value="0.00" />
-  <property name="stereo_dy" value="-0.09" /> <!-- +y to the left -->
-  <property name="stereo_dz" value="0.00" />
-  <property name="stereo_rx" value="0.00" />
-  <property name="stereo_ry" value="0.00" />
-  <property name="stereo_rz" value="0.00" />
+  <xacro:property name="stereo_dx" value="0.00" />
+  <xacro:property name="stereo_dy" value="-0.09" /> <!-- +y to the left -->
+  <xacro:property name="stereo_dz" value="0.00" />
+  <xacro:property name="stereo_rx" value="0.00" />
+  <xacro:property name="stereo_ry" value="0.00" />
+  <xacro:property name="stereo_rz" value="0.00" />
   <!-- this macro is used for creating wide and narrow double stereo camera links -->
   <xacro:macro name="stereo_camera_v0" params="name parent focal_length hfov image_format image_width image_height *origin">
     <joint name="${name}_frame_joint" type="fixed">
-      <insert_block name="origin" />
+      <xacro:insert_block name="origin" />
       <parent link="${parent}"/>
       <child link="${name}_link"/>
