Commit message: Prepend xacro tags with xacro xml namespace

File: pr2_description/urdf/sensors/wge100_camera.urdf.xacro (robot description, xacro)
@@ -10,5 +10,5 @@
   <xacro:macro name="wge100_camera_v0" params="name camera_name image_format image_topic_name camera_info_topic_name parent hfov focal_length frame_id hack_baseline image_width image_height *origin">
     <joint name="${name}_frame_joint" type="fixed">
-      <insert_block name="origin" />
+      <xacro:insert_block name="origin" />
       <parent link="${parent}"/>
       <child link="${name}_frame"/>

File: pr2_description/urdf/shoulder_v0/shoulder.urdf.xacro (robot description, xacro)
@@ -10,6 +10,6 @@
   <xacro:include filename="$(find pr2_description)/urdf/shoulder_v0/shoulder.transmission.xacro" />
   <xacro:include filename="$(find pr2_description)/urdf/common.xacro" />
-  <property name="shoulder_lift_length" value="0.10" />  <!--TODO Define and give source-->
-  <property name="shoulder_lift_radius" value="0.12" />  <!--TODO Define and give source-->
+  <xacro:property name="shoulder_lift_length" value="0.10" />  <!--TODO Define and give source-->
+  <xacro:property name="shoulder_lift_radius" value="0.12" />  <!--TODO Define and give source-->
  <!-- ============================   Shoulder   ============================ -->
   <xacro:macro name="pr2_shoulder_v0" params="side parent reflect *origin">
@@ -17,5 +17,5 @@
     <joint name="${side}_shoulder_pan_joint" type="revolute">
       <axis xyz="0 0 1" />
-      <insert_block name="origin" /> <!-- transform from parent link to this joint frame -->
+      <xacro:insert_block name="origin" /> <!-- transform from parent link to this joint frame -->
       <parent link="${parent}"/>
       <child link="${side}_shoulder_pan_link"/>
@@ -99,5 +99,5 @@
     <joint name="${side}_upper_arm_roll_joint" type="revolute">
       <axis xyz="1 0 0" />
-      <insert_block name="origin" />
+      <xacro:insert_block name="origin" />
       <parent link="${parent}" />
       <child link="${side}_upper_arm_roll_link"/>

File: pr2_description/urdf/tilting_laser_v0/tilting_laser.urdf.xacro (robot description, xacro)
@@ -14,5 +14,5 @@
       <calibration falling="${laser_calib_ref}" />
       <dynamics damping="0.008" />
-      <insert_block name="origin" />
+      <xacro:insert_block name="origin" />
       <parent link="${parent}"/>
       <child link="${name}_mount_link"/>

Commit message: remove guessed inertia on base_footprint
These values are obviously fictitious (the whole link is...)
Additionally, KDL datastructures have been complaining about this for ages
because KDL does not support inertials for the model root (whatever that means).

File: pr2_description/urdf/base_v0/base.urdf.xacro (robot description, xacro)
@@ -143,10 +143,4 @@
          navigation stack dedpends on this frame -->
     <link name="${name}_footprint">
-      <inertial>
-        <mass value="1.0" />
-        <origin xyz="0 0 0" />
-        <inertia ixx="0.01" ixy="0.0" ixz="0.0"
-                 iyy="0.01" iyz="0.0" izz="0.01" />
-      </inertial>
       <visual>
         <origin xyz="0 0 0" rpy="0 0 0" />

Commit message: Update base.urdf.xacro to clean up footprint link
The footprint link seems no need to contain visual and collision, so left it empty

File: pr2_description/urdf/base_v0/base.urdf.xacro (robot description, xacro)
@@ -142,21 +142,5 @@
     <!-- base_footprint is a fictitious link(frame) that is on the ground right below base_link origin,
          navigation stack dedpends on this frame -->
-    <link name="${name}_footprint">
-      <visual>
-        <origin xyz="0 0 0" rpy="0 0 0" />
-        <geometry>
-          <box size="0.01 0.01 0.01" />
-        </geometry>
-        <material name="White" />
-      </visual>
-      <collision>
-        <!-- represent base collision with a simple rectangular model, positioned by base_size_z s.t. top
-             surface of the collision box matches the top surface of the PR2 base -->
-        <origin xyz="0 0 ${0.051+base_collision_size_z/2}" rpy="0 0 0" />
-        <geometry>
-          <box size="0.001 0.001 0.001" />
-        </geometry>
-      </collision>
-    </link>
+    <link name="${name}_footprint" />
     <joint name="${name}_footprint_joint" type="fixed">
       <origin xyz="0 0 0.051" rpy="0 0 0" />
