Commit message: Adding URDF from all qual and burn in tests, adding unit test to check URDF

File: pr2_description/robots/caster.urdf.xacro (robot description, xacro)
@@ -11,31 +11,4 @@
     <origin xyz="0 0 0" rpy="0 0 0" />
   </xacro:pr2_caster_v0>
-  <!-- Solid Base for visualizer -->
-  <joint name="base_joint" type="fixed">
-    <parent link="world" />
-    <origin xyz="0 0 0" rpy="0 0 0" />
-    <child link="base_link" />
-  </joint>
-  <link name="base_link">
-    <inertial>
-      <mass value="1000" />
-      <origin xyz=" 0 0 0 " />
-      <inertia ixx="1000"  ixy="0"  ixz="0" iyy="1000" iyz="0" izz="1000" />
-    </inertial>
-    <visual>
-      <origin xyz="0 0 -1" rpy="0 0 0 " />
-      <geometry name="pr2_base_mesh_file">
-        <box size="20 20 0.01" />
-      </geometry>
-    </visual>
-    <collision>
-      <origin xyz="0 0 -1" rpy="0.0 0.0 0.0 " />
-      <geometry name="base_collision_geom">
-        <box size="20 20 0.01" />
-      </geometry>
-    </collision>
-  </link>
-  <gazebo reference="base_link" >
-    <material>Gazebo/White</material>
-  </gazebo>
+  <include filename="$(find pr2_description)/urdf/base_link.xacro" />
 </robot>

File: pr2_description/robots/gripper.urdf.xacro (robot description, xacro)
@@ -21,31 +21,4 @@
     <origin xyz="0 0 0" rpy="0 0 0" />
   </xacro:pr2_gripper_v0>
-  <!-- Solid Base for visualizer -->
-  <joint name="base_joint" type="fixed">
-    <parent link="world" />
-    <origin xyz="0 0 0" rpy="0 0 0" />
-    <child link="base_link" />
-  </joint>
-  <link name="base_link">
-    <inertial>
-      <mass value="1000" />
-      <origin xyz=" 0 0 0 " />
-      <inertia ixx="1000" ixy="0" ixz="0" iyy="1000" iyz="0" izz="1000" />
-    </inertial>
-    <visual>
-      <origin xyz="0 0 0" rpy="0 0 0 " />
-      <geometry name="pr2_base_mesh_file">
-        <box size="1 1 1" />
-      </geometry>
-    </visual>
-    <collision>
-      <origin xyz="0 0 0" rpy="0.0 0.0 0.0 " />
-      <geometry name="base_collision_geom">
-        <box size="1 1 1" />
-      </geometry>
-    </collision>
-  </link>
-  <gazebo reference="base_link" >
-    <material>Gazebo/White</material>
-  </gazebo>
+  <include filename="$(find pr2_description)/urdf/base_link.xacro" />
 </robot>

File: pr2_description/robots/head.urdf.xacro (robot description, xacro)
@@ -11,31 +11,4 @@
     <origin xyz="0 0 0" rpy="0 0 0" />
   </xacro:pr2_head_v0>
-  <!-- Solid Base for visualizer -->
-  <joint name="base_joint" type="fixed">
-    <parent link="world" />
-    <origin xyz="0 0 0" rpy="0 0 0" />
-    <child link="base_link" />
-  </joint>
-  <link name="base_link">
-    <inertial>
-      <mass value="1000" />
-      <origin xyz=" 0 0 0 " />
-      <inertia ixx="1000" ixy="0" ixz="0" iyy="1000" iyz="0" izz="1000" />
-    </inertial>
-    <visual>
-      <origin xyz="0 0 0" rpy="0 0 0 " />
-      <geometry name="pr2_base_mesh_file">
-        <box size=".01 .01 .01" />
-      </geometry>
-    </visual>
-    <collision>
-      <origin xyz="0 0 0" rpy="0.0 0.0 0.0 " />
-      <geometry name="base_collision_geom">
-        <box size=".01 .01 .01" />
-      </geometry>
-    </collision>
-  </link>
-  <gazebo reference="base_link" >
-    <material>Gazebo/White</material>
-  </gazebo>
+   <include filename="$(find pr2_description)/urdf/base_link.xacro" />
 </robot>

File: pr2_description/robots/laser_tilt.urdf.xacro (robot description, xacro)
@@ -11,31 +11,4 @@
     <origin xyz="0 0 0" rpy="0 0 0" />
   </xacro:pr2_tilting_laser_v0>
-  <!-- Solid Base for visualizer -->
-  <joint name="base_joint" type="fixed">
-    <parent link="world" />
-    <origin xyz="0 0 0" rpy="0 0 0" />
-    <child link="base_link" />
-  </joint>
-  <link name="base_link">
-    <inertial>
-      <mass value="1000" />
-      <origin xyz=" 0 0 0 " />
-      <inertia ixx="1000" ixy="0" ixz="0" iyy="1000" iyz="0" izz="1000" />
-    </inertial>
-    <visual>
-      <origin xyz="0 0 0" rpy="0 0 0 " />
-      <geometry name="pr2_base_mesh_file">
-        <box size="1 1 1" />
-      </geometry>
-    </visual>
-    <collision>
-      <origin xyz="0 0 0" rpy="0.0 0.0 0.0 " />
-      <geometry name="base_collision_geom">
-        <box size="1 1 1" />
-      </geometry>
-    </collision>
-  </link>
-  <gazebo reference="base_link" >
-    <material>Gazebo/White</material>
-  </gazebo>
+  <include filename="$(find pr2_description)/urdf/base_link.xacro" />
 </robot>

File: pr2_description/robots/shoulder.urdf.xacro (robot description, xacro)
@@ -8,34 +8,7 @@
   <include filename="$(find pr2_description)/urdf/materials.urdf.xacro" />
   <include filename="$(find pr2_description)/urdf/shoulder_v0/shoulder.urdf.xacro" />
+  <include filename="$(find pr2_description)/urdf/base_link.xacro" />
   <xacro:pr2_shoulder_v0 side="r" reflect="-1" parent="base_link">
     <origin xyz="0 0 0" rpy="0 0 0" />
   </xacro:pr2_shoulder_v0>
-  <!-- Solid Base for visualizer -->
-  <joint name="base_joint" type="fixed">
-    <parent link="world" />
-    <origin xyz="0 0 0" rpy="0 0 0" />
-    <child link="base_link" />
-  </joint>
-  <link name="base_link">
-    <inertial>
-      <mass value="1000" />
-      <origin xyz=" 0 0 0 " />
-      <inertia ixx="1000" ixy="0" ixz="0" iyy="1000" iyz="0" izz="1000" />
-    </inertial>
-    <visual>
-      <origin xyz="0 0 0" rpy="0 0 0 " />
-      <geometry name="pr2_base_mesh_file">
-        <box size="1 1 1" />
-      </geometry>
-    </visual>
-    <collision>
-      <origin xyz="0 0 0" rpy="0.0 0.0 0.0 " />
-      <geometry name="base_collision_geom">
-        <box size="1 1 1" />
-      </geometry>
-    </collision>
-  </link>
-  <gazebo reference="base_link" >
-    <material>Gazebo/White</material>
-  </gazebo>
 </robot>

File: pr2_description/robots/torso.urdf.xacro (robot description, xacro)
@@ -11,31 +11,4 @@
     <origin xyz="0 0 0" rpy="0 0 0" />
   </xacro:pr2_torso_v0>
-  <!-- Solid Base for visualizer -->
-  <joint name="base_joint" type="fixed">
-    <parent link="world" />
-    <origin xyz="0 0 0" rpy="0 0 0" />
-    <child link="base_link" />
-  </joint>
-  <link name="base_link">
-    <inertial>
-      <mass value="1000" />
-      <origin xyz=" 0 0 0 " />
-      <inertia ixx="1000" ixy="0" ixz="0" iyy="1000" iyz="0" izz="1000" />
-    </inertial>
-    <visual>
-      <origin xyz="0 0 0" rpy="0 0 0 " />
-      <geometry name="pr2_base_mesh_file">
-        <box size="1 1 1" />
-      </geometry>
-    </visual>
-    <collision>
-      <origin xyz="0 0 0" rpy="0.0 0.0 0.0 " />
-      <geometry name="base_collision_geom">
-        <box size="1 1 1" />
-      </geometry>
-    </collision>
-  </link>
-  <gazebo reference="base_link" >
-    <material>Gazebo/White</material>
-  </gazebo>
+  <include filename="$(find pr2_description)/urdf/base_link.xacro" />
 </robot>

File: pr2_description/robots/upperarm.urdf.xacro (robot description, xacro)
@@ -11,31 +11,4 @@
     <origin xyz="0 0 0" rpy="0 0 0" />
   </xacro:pr2_upper_arm_v0>
-  <!-- Solid Base for visualizer -->
-  <joint name="base_joint" type="fixed">
-    <parent link="world" />
-    <origin xyz="0 0 0" rpy="0 0 0" />
-    <child link="base_link" />
-  </joint>
-  <link name="base_link">
-    <inertial>
-      <mass value="1000" />
-      <origin xyz=" 0 0 0 " />
-      <inertia ixx="1000" ixy="0" ixz="0" iyy="1000" iyz="0" izz="1000" />
-    </inertial>
-    <visual>
-      <origin xyz="0 0 0" rpy="0 0 0 " />
-      <geometry name="pr2_base_mesh_file">
-        <box size="1 1 1" />
-      </geometry>
-    </visual>
-    <collision>
-      <origin xyz="0 0 0" rpy="0.0 0.0 0.0 " />
-      <geometry name="base_collision_geom">
-        <box size="1 1 1" />
-      </geometry>
-    </collision>
-  </link>
-  <gazebo reference="base_link" >
-    <material>Gazebo/White</material>
-  </gazebo>
+  <include filename="$(find pr2_description)/urdf/base_link.xacro" />
 </robot>

File: pr2_description/robots/upperarm_wrist.urdf.xacro (robot description, xacro)
@@ -1,4 +1,4 @@
 <?xml version="1.0"?>
-<robot name="forearm"
+<robot name="pr2_upper_arm"
        xmlns:sensor="http://playerstage.sourceforge.net/gazebo/xmlschema/#sensor"
        xmlns:controller="http://playerstage.sourceforge.net/gazebo/xmlschema/#controller"
@@ -7,6 +7,10 @@
   <include filename="$(find pr2_description)/urdf/common.xacro" />
   <include filename="$(find pr2_description)/urdf/materials.urdf.xacro" />
+  <include filename="$(find pr2_description)/urdf/upper_arm_v0/upper_arm.urdf.xacro" />
   <include filename="$(find pr2_description)/urdf/forearm_v0/forearm.urdf.xacro" />
-  <xacro:pr2_forearm_v0 side="r" reflect="-1" parent="base_link">
+  <xacro:pr2_upper_arm_v0 side="r" reflect="-1" parent="base_link">
+    <origin xyz="0 0 0" rpy="0 0 0" />
+  </xacro:pr2_upper_arm_v0>
+    <xacro:pr2_forearm_v0 side="r" reflect="-1" parent="r_forearm_roll_link">
     <origin xyz="0 0 0" rpy="0 0 0" />
   </xacro:pr2_forearm_v0>

File: pr2_description/robots/wrist_gripper.urdf.xacro (robot description, xacro)
@@ -8,7 +8,21 @@
   <include filename="$(find pr2_description)/urdf/materials.urdf.xacro" />
   <include filename="$(find pr2_description)/urdf/forearm_v0/forearm.urdf.xacro" />
+  <include filename="$(find pr2_description)/urdf/gripper_v0/gripper.urdf.xacro" />
   <xacro:pr2_forearm_v0 side="r" reflect="-1" parent="base_link">
     <origin xyz="0 0 0" rpy="0 0 0" />
   </xacro:pr2_forearm_v0>
+  <xacro:pr2_gripper_v0 side="r" parent="r_wrist_roll_link"
+                        screw_reduction="${4.0/1000.0}"
+                        gear_ratio="${(729.0/25.0)*(22.0/16.0)}"
+                        theta0="${3.6029*M_PI/180.0}"
+                        phi0="${29.7089*M_PI/180.0}"
+                        t0="${-0.1914/1000.0}"
+                        L0="${37.5528/1000.0}"
+                        h="${0.0/1000.0}"
+                        a="${68.3698/1000.0}"
+                        b="${43.3849/1000.0}"
+                        r="${91.5/1000.0}" >
+    <origin xyz="0 0 0" rpy="0 0 0" />
+  </xacro:pr2_gripper_v0>
   <include filename="$(find pr2_description)/urdf/base_link.xacro" />
 </robot>

File: pr2_description/urdf/common.xacro (robot description, xacro)
@@ -15,5 +15,5 @@
   <property name="cal_r_forearm_roll_flag"   value="0.0" />
   <property name="cal_r_wrist_flex_flag"     value="0.0" />
-  <property name="cal_r_wrist_roll_flag"     value="0.4" />
+  <property name="cal_r_wrist_roll_flag"     value="0.0" />
   <!-- ********** Head ********** -->
   <!-- Head Location: Add to the transform from torso to head_pan_link (Nominally 0) -->
@@ -31,5 +31,5 @@
   <!-- Casters -->
   <property name="cal_caster_fl" value="0.0" />
-  <property name="cal_caster_fr" value="0.025" />
+  <property name="cal_caster_fr" value="0.0" />
   <property name="cal_caster_bl" value="0.0" />
   <property name="cal_caster_br" value="0.0" />

File: pr2_description/urdf/forearm_v0/forearm.urdf.xacro (robot description, xacro)
@@ -42,8 +42,8 @@
     <joint name="${side}_wrist_flex_joint" type="revolute">
       <axis xyz="0 -1 0" />
-      <limit lower="-0.1" upper="2.2" effort="200" velocity="${VELOCITY_LIMIT_SCALE*5.13}" />
-      <safety_controller k_position="20" k_velocity="4" soft_lower_limit="${-0.1+0.2}" soft_upper_limit="${2.2-0.2}" />
+      <limit lower="0.0" upper="2.094" effort="10" velocity="${VELOCITY_LIMIT_SCALE*5.13}" />
+      <safety_controller k_position="20" k_velocity="4" soft_lower_limit="${0.0 + 0.15}" soft_upper_limit="${2.094 - 0.15}" />
       <dynamics damping="0.1" />
-      <calibration reference_position="${0.4363+cal_r_wrist_flex_flag}" />
+      <calibration reference_position="${0.5410521 + cal_r_wrist_flex_flag}" />
       <origin xyz="0.32025 0 0" rpy="0 0 0" />
       <parent link="${side}_forearm_link"/>
@@ -78,5 +78,5 @@
       <safety_controller k_velocity="2" />
       <dynamics damping="0.1" />
-      <calibration reference_position="${1.27+cal_r_wrist_roll_flag}" values="1.5 -1" />
+      <calibration reference_position="${M_PI / 2 + cal_r_wrist_roll_flag}" />
       <origin xyz="0 0 0" rpy="0 0 0" />
       <parent link="${side}_wrist_flex_link"/>

File: pr2_description/urdf/upper_arm_v0/upper_arm.urdf.xacro (robot description, xacro)
@@ -65,6 +65,7 @@
     <joint name="${side}_elbow_flex_joint" type="revolute">
       <axis xyz="0 1 0" />
-      <limit lower="-2.3" upper="0.1" effort="30" velocity="${VELOCITY_LIMIT_SCALE*5.5}" />
-      <safety_controller k_position="100" k_velocity="3" soft_lower_limit="${-2.3+0.25}" soft_upper_limit="${0.1-0.1}" />
+      <!-- Note: Overtravel limits are 140, -7 degrees instead of 133, 0 -->
+      <limit lower="-2.3213" upper="0.00" effort="30" velocity="${VELOCITY_LIMIT_SCALE*5.5}" />
+      <safety_controller k_position="100" k_velocity="3" soft_lower_limit="${-2.3213+0.2}" soft_upper_limit="${0.00-0.15}" />
       <calibration reference_position="${-1.1606 + cal_r_elbow_flex_flag}"/>
       <dynamics damping="1.0" />
@@ -100,5 +101,5 @@
       <limit effort="30" velocity="${VELOCITY_LIMIT_SCALE*6}" />
       <safety_controller k_velocity="1" />
-      <calibration reference_position="${cal_r_forearm_roll_flag}" />
+      <calibration reference_position="${0.0 + cal_r_forearm_roll_flag}" />
       <dynamics damping="0.1" />
       <origin xyz="0 0 0" rpy="0 0 0" />

Commit message: Minor def changes for Beta caster

File: pr2_description/robots/caster.urdf.xacro (robot description, xacro)
@@ -9,5 +9,5 @@
   <include filename="$(find pr2_description)/urdf/base_v0/base.urdf.xacro" />
   <xacro:pr2_caster_v0 suffix="fl" parent="base_link" ref_position="0.0" >
-    <origin xyz="0 0 0" rpy="0 0 0" />
+    <origin xyz="0 0 0" rpy="0 3.14 0" />
   </xacro:pr2_caster_v0>
   <include filename="$(find pr2_description)/urdf/base_link.xacro" />

File: pr2_description/urdf/base_v0/base.gazebo.xacro (robot description, xacro)
@@ -4,7 +4,4 @@
        xmlns:interface="http://playerstage.sourceforge.net/gazebo/xmlschema/#interface"
        xmlns:xacro="http://ros.org/wiki/xacro">
-  <!--                                                      -->
-  <!-- Alpha 2.0 hardware                                   -->
-  <!--                                                      -->
   <xacro:macro name="pr2_wheel_gazebo_v0" params="suffix parent">
     <gazebo reference="${parent}_${suffix}_wheel_link">

File: pr2_description/urdf/base_v0/base.urdf.xacro (robot description, xacro)
@@ -96,5 +96,5 @@
           <mesh filename="package://pr2_description/meshes/base_v0/caster.stl" />
         </geometry>
-        <material name="Caster" />
+        <material name="Green" />
       </visual>
       <collision>
