Commit message: Changed file organization by separating all Kinect2 files. May not compile if using Kinect2 files but Kinect1 urdf is fine.

File: pr2_description/robots/pr2_kinect2.urdf.xacro (robot description, xacro)
@@ -1,8 +1,4 @@
 <?xml version="1.0"?>
-<robot xmlns:sensor="http://playerstage.sourceforge.net/gazebo/xmlschema/#sensor"
-       xmlns:controller="http://playerstage.sourceforge.net/gazebo/xmlschema/#controller"
-       xmlns:interface="http://playerstage.sourceforge.net/gazebo/xmlschema/#interface"
-       xmlns:xacro="http://playerstage.sourceforge.net/gazebo/xmlschema/#interface"
-       name="pr2" >
+<robot name="pr2" xmlns:xacro="http://ros.org/wiki/xacro">
   <!-- The following included files set up definitions of parts of the robot body -->
   <!-- misc common stuff? -->
@@ -24,5 +20,5 @@
   <!-- Head sensors -->
   <xacro:include filename="$(find pr2_description)/urdf/sensors/head_sensor_package.urdf.xacro" />
-  <xacro:include filename="$(find pr2_description)/urdf/sensors/kinect_prosilica_camera.urdf.xacro" />
+  <xacro:include filename="$(find pr2_description)/urdf/sensors/kinect2.urdf.xacro" />
   <!-- Camera sensors -->
   <xacro:include filename="$(find pr2_description)/urdf/sensors/wge100_camera.urdf.xacro" />
@@ -64,5 +60,5 @@
   </xacro:projector_wg6802418_v0>
   <!-- Base of Kinect/Prosilica Mount -->
-  <xacro:kinect_prosilica_camera_swept_back_v0 name="head_mount" parent="head_plate_frame" >
+  <xacro:kinect2_v0 name="head_mount" parent="head_plate_frame" >
     <origin xyz="-0.137376 0 0.091746" rpy="0 0 0" />
     <!--
@@ -78,5 +74,5 @@
           Just need to roscd and svn up.
     -->
-  </xacro:kinect_prosilica_camera_swept_back_v0>
+  </xacro:kinect2_v0>
   <xacro:pr2_tilting_laser_v0 name="laser_tilt" parent="torso_lift_link" laser_calib_ref="0.0">
     <origin xyz="0.09893 0 0.227" rpy="0 0 0" />

File: pr2_description/urdf/sensors/kinect2.gazebo.xacro (robot description, xacro)
@@ -1,5 +1,5 @@
 <?xml version="1.0"?>
-<root xmlns:xacro="http://ros.org/wiki/xacro">
-<xacro:macro name="kinect_ir_gazebo_v0" params="link_name frame_name camera_name">
+<robot xmlns:xacro="http://ros.org/wiki/xacro">
+<xacro:macro name="kinect2_ir_gazebo_v0" params="link_name frame_name camera_name">
   <gazebo reference="${link_name}">
     <sensor type="depth" name="${name}_ir_sensor">
@@ -45,5 +45,5 @@
   </gazebo>
 </xacro:macro>
-<xacro:macro name="kinect_rgb_gazebo_v0" params="link_name frame_name camera_name">
+<xacro:macro name="kinect2_rgb_gazebo_v0" params="link_name frame_name camera_name">
   <gazebo reference="${link_name}">
     <sensor type="depth" name="${name}_rgb_sensor">
@@ -88,5 +88,5 @@
   </gazebo>
 </xacro:macro>
-<xacro:macro name="kinect_prosilica_gazebo" params="joint_name link_name">
+<xacro:macro name="kinect2_prosilica_gazebo" params="joint_name link_name">
   <gazebo>
     <plugin name="${link_name}_srp_controller" filename="libgazebo_ros_srp.so">
@@ -103,85 +103,3 @@
   </transmission>
 </xacro:macro>
-<xacro:macro name="prosilica_cam_gazebo_v1" params="link_name frame_name camera_name ">
-  <gazebo reference="${link_name}">
-    <sensor type="camera" name="${link_name}_sensor">
-      <always_on>true</always_on>
-      <update_rate>1.0</update_rate>
-      <camera>
-        <horizontal_fov>${64.2*M_PI/180.0}</horizontal_fov>
-        <image>
-          <format>R8G8B8</format>
-          <width>320</width>
-          <height>240</height>
-        </image>
-        <clip>
-          <near>0.1</near>
-          <far>100</far>
-        </clip>
-      </camera>
-      <plugin name="${link_name}_controller" filename="libgazebo_ros_prosilica.so">
-        <alwaysOn>true</alwaysOn>
-        <updateRate>1.0</updateRate>
-        <cameraName>${camera_name}_1mb</cameraName>
-        <imageTopicName>image_raw</imageTopicName>
-        <cameraInfoTopicName>camera_info</cameraInfoTopicName>
-        <depthImageTopicName>depth/image_raw</depthImageTopicName>
-        <depthImageCameraInfoTopicName>depth/camera_info</depthImageCameraInfoTopicName>
-        <pollServiceName>request_image</pollServiceName>
-        <pointCloudTopicName>points</pointCloudTopicName>
-        <frameName>${frame_name}</frameName>
-        <pointCloudCutoff>0.4</pointCloudCutoff>
-        <distortionK1>0.0</distortionK1>
-        <distortionK2>0.0</distortionK2>
-        <distortionK3>0.0</distortionK3>
-        <distortionT1>0.0</distortionT1>
-        <distortionT2>0.0</distortionT2>
-        <CxPrime>0</CxPrime>
-        <Cx>0</Cx>
-        <Cy>0</Cy>
-        <focalLength>0</focalLength>
-        <hackBaseline>0</hackBaseline>
-      </plugin>
-    </sensor>
-    <sensor type="depth" name="${link_name}_sim_pcd_sensor">
-      <always_on>true</always_on>
-      <update_rate>1.0</update_rate>
-      <camera>
-        <horizontal_fov>${64.2*M_PI/180.0}</horizontal_fov>
-        <image>
-          <format>R8G8B8</format>
-          <width>320</width>
-          <height>240</height>
-        </image>
-        <clip>
-          <near>0.1</near>
-          <far>100</far>
-        </clip>
-      </camera>
-      <plugin name="${link_name}_sim_pcd_controller" filename="libgazebo_ros_openni_kinect.so">
-        <alwaysOn>true</alwaysOn>
-        <updateRate>1.0</updateRate>
-        <cameraName>${camera_name}_1mb_sim_pcd</cameraName>
-        <imageTopicName>image_raw</imageTopicName>
-        <depthImageTopicName>depth/image_raw</depthImageTopicName>
-        <depthImageCameraInfoTopicName>depth/camera_info</depthImageCameraInfoTopicName>
-        <cameraInfoTopicName>camera_info</cameraInfoTopicName>
-        <pointCloudTopicName>points</pointCloudTopicName>
-        <frameName>${frame_name}</frameName>
-        <pointCloudCutoff>0.4</pointCloudCutoff>
-        <distortionK1>0.00000001</distortionK1>
-        <distortionK2>0.00000001</distortionK2>
-        <distortionK3>0.00000001</distortionK3>
-        <distortionT1>0.00000001</distortionT1>
-        <distortionT2>0.00000001</distortionT2>
-        <CxPrime>0</CxPrime>
-        <Cx>0</Cx>
-        <Cy>0</Cy>
-        <focalLength>0</focalLength>
-        <hackBaseline>0</hackBaseline>
-      </plugin>
-    </sensor>
-    <material value="Gazebo/Red" />
-  </gazebo>
-</xacro:macro>
-</root>
+</robot>

File: pr2_description/urdf/sensors/kinect_prosilica_camera.urdf.xacro (robot description, xacro)
@@ -1,13 +1,16 @@
 <?xml version="1.0"?>
-<robot xmlns:xacro="http://ros.org/wiki/xacro">
+<root xmlns:sensor="http://playerstage.sourceforge.net/gazebo/xmlschema/#sensor"
+      xmlns:controller="http://playerstage.sourceforge.net/gazebo/xmlschema/#controller"
+      xmlns:interface="http://playerstage.sourceforge.net/gazebo/xmlschema/#interface"
+      xmlns:xacro="http://ros.org/wiki/xacro">
   <xacro:include filename="$(find pr2_description)/urdf/sensors/kinect_prosilica_camera.gazebo.xacro" />
   <property name="ir_depth_rgb_offset_y" value="0.01"/> <!-- FIXME: what is this offset? -->
-  <!-- kinect2 combo -->
+  <!-- kinect and prosilica combo -->
   <xacro:macro name="kinect_prosilica_camera_swept_back_v0" params="name parent *origin">
-    <!-- stl contains structure + kinect2 bracket + kinect2 combo -->
+    <!-- stl contains structure + kinect + prosilica combo -->
     <joint name="${name}_joint" type="fixed">
       <!-- <limit lower="0.1" upper="0.1" effort="10000" velocity="100.0"/> -->
-      <insert_block name="origin" />
-      <!-- <origin xyz="-0.228 -0.148 0.091" rpy="${M_PI/2} 0 ${M_PI/2}"/> -->
+      <!-- <insert_block name="origin" /> -->
+      <origin xyz="-0.138 0 0.091" rpy="0 0 0"/>
       <parent link="${parent}"/>
       <child link="${name}_link"/>
@@ -15,5 +18,5 @@
     <link name="${name}_link">
       <inertial>
-        <mass value="0.1"/>
+        <mass value="0.1" />
         <origin xyz="0 0 0" rpy="0 0 0"/>
         <inertia ixx="0.01"  ixy="0.0"  ixz="0.0"
@@ -22,7 +25,7 @@
       </inertial>
       <visual>
-        <origin xyz="0 -0.138 0" rpy="${M_PI/2} 0 ${M_PI/2}"/>
+        <origin xyz="0.0 0.0 0" rpy="0 0 0"/>
         <geometry>
-          <mesh filename="package://pr2_description/meshes/sensors/kinect_prosilica_v0/kinect2_mount.STL" scale="0.001 0.001 0.001" />
+          <mesh filename="package://pr2_description/meshes/sensors/kinect_prosilica_v0/115x100_swept_back--coarse.STL" scale="0.001 0.001 0.001" />
         </geometry>
         <material name="gray">
@@ -31,31 +34,5 @@
       </visual>
       <collision>
-        <origin xyz="0 0 0" rpy="0 0 0"/>
-        <geometry>
-          <sphere radius="0.0005"/>
-        </geometry>
-      </collision>
-    </link>
-    <joint name="${name}_bracket_joint" type="fixed">
-      <origin xyz="0.148 0.128 0.0321" rpy="${M_PI} ${M_PI} ${M_PI}"/>
-      <parent link="${name}_link"/>
-      <child link="${name}_bracket_link"/>
-    </joint>
-    <link name="${name}_bracket_link">
-      <inertial>
-        <mass value="0.1"/>
-        <origin xyz="0 0 0" rpy="0 0 0"/>
-        <inertia ixx="0.01"  ixy="0.0"  ixz="0.0"
-                 iyy="0.01"  iyz="0.0"
-                 izz="0.01" />
-      </inertial>
-      <visual>
-        <origin xyz="0 0 0" rpy="0 0 0"/>
-        <geometry>
-          <mesh filename="package://pr2_description/meshes/sensors/kinect_prosilica_v0/kinect2_bracket.STL" />
-        </geometry>
-      </visual>
-      <collision>
-        <origin xyz="0 0 0" rpy="0 0 0"/>
+        <origin xyz="0.0 0.0 0" rpy="0 0 0"/>
         <geometry>
           <sphere radius="0.0005"/>
@@ -68,5 +45,5 @@
     -->
     <!-- kinect ir sensor physical attachment -->
-<!--    <joint name="${name}_kinect_ir_joint" type="fixed">
+    <joint name="${name}_kinect_ir_joint" type="fixed">
       <origin xyz="-0.032267 0.0125 0.136453" rpy="0 0 0"/>
       <parent link="${name}_link"/>
@@ -93,7 +70,7 @@
         </geometry>
       </collision>
-    </link> -->
+    </link>
     <!-- kinect ir sensor frame -->
-<!--    <joint name="${name}_kinect_ir_optical_frame_joint" type="fixed">
+    <joint name="${name}_kinect_ir_optical_frame_joint" type="fixed">
       <origin xyz="${cal_kinect_x}            ${cal_kinect_y + ir_depth_rgb_offset_y}         ${cal_kinect_z}"
                 rpy="${-M_PI/2+cal_kinect_roll} ${0.0+cal_kinect_pitch} ${-M_PI/2+cal_kinect_yaw}" />
@@ -101,11 +78,9 @@
       <child link="${name}_kinect_ir_optical_frame"/>
     </joint>
-    <link name="${name}_kinect_ir_optical_frame"/> -->
+    <link name="${name}_kinect_ir_optical_frame"/>
     <!-- gazebo extensions -->
-<!--     <xacro:kinect_ir_gazebo_v0 link_name="${name}_kinect_ir_link" frame_name="${name}_kinect_ir_optical_frame" camera_name="head_mount_kinect" />
- -->
-<!-- kinect2 -->
+    <xacro:kinect_ir_gazebo_v0 link_name="${name}_kinect_ir_link" frame_name="${name}_kinect_ir_optical_frame" camera_name="head_mount_kinect" />
     <!-- kinect rgb sensor physical attachment -->
-<!--     <joint name="${name}_kinect_rgb_joint" type="fixed">
+    <joint name="${name}_kinect_rgb_joint" type="fixed">
       <origin xyz="0 -0.03 0" rpy="0 0 0"/>
       <parent link="${name}_kinect_ir_link"/>
@@ -132,7 +107,7 @@
         </geometry>
       </collision>
-    </link> -->
+    </link>
     <!-- kinect rgb sensor frame -->
-<!--    <joint name="${name}_kinect_rgb_optical_frame_joint" type="fixed">
+    <joint name="${name}_kinect_rgb_optical_frame_joint" type="fixed">
       <origin xyz="${cal_kinect_x}            ${cal_kinect_y}         ${cal_kinect_z}"
                 rpy="${-M_PI/2+cal_kinect_roll} ${0.0+cal_kinect_pitch} ${-M_PI/2+cal_kinect_yaw}" />
@@ -140,31 +115,29 @@
       <child link="${name}_kinect_rgb_optical_frame"/>
     </joint>
-    <link name="${name}_kinect_rgb_optical_frame"/> -->
+    <link name="${name}_kinect_rgb_optical_frame"/>
     <!-- gazebo extensions -->
-<!--     <xacro:kinect_rgb_gazebo_v0 link_name="${name}_kinect_rgb_link" frame_name="${name}_kinect_rgb_optical_frame" camera_name="head_mount_kinect" /> -->
-    <joint name="${name}_kinect2_joint" type="fixed">
-      <origin xyz="0 0.0255 0.01" rpy="0 0 0"/>
-      <parent link="${name}_bracket_link"/>
-      <child link="${name}_kinect2_link"/>
+    <xacro:kinect_rgb_gazebo_v0 link_name="${name}_kinect_rgb_link" frame_name="${name}_kinect_rgb_optical_frame" camera_name="head_mount_kinect" />
+    <!-- prosilica sensor physical attachment -->
+    <joint name="${name}_prosilica_joint" type="fixed">
+      <origin xyz="-0.046457 0.0125 0.088921" rpy="0 0 0"/>
+      <parent link="${name}_link"/>
+      <child link="${name}_prosilica_link"/>
     </joint>
-    <link name="${name}_kinect2_link">
+    <link name="${name}_prosilica_link">
       <inertial>
-        <mass value="0.1"/>
+        <mass value="0.1" />
         <origin xyz="0 0 0" rpy="0 0 0"/>
         <inertia ixx="0.01"  ixy="0.0"  ixz="0.0"
                  iyy="0.01"  iyz="0.0"
-                 izz="0.01"/>
+                 izz="0.01" />
       </inertial>
       <visual>
-        <origin xyz="0 0 0" rpy="0 0 0"/>
+        <origin xyz="0.0 0.0 0" rpy="0 0 0"/>
         <geometry>
-          <box size="0.25 0.043 0.067"/>
-          <material name="black">
-            <color rgba="0.05 0.05 0.05 1"/>
-          </material>
+          <sphere radius="0.0005"/>
         </geometry>
       </visual>
       <collision>
-        <origin xyz="0 0 0" rpy="0 0 0"/>
+        <origin xyz="0.0 0.0 0" rpy="0 0 0"/>
         <geometry>
           <sphere radius="0.0005"/>
@@ -172,13 +145,14 @@
       </collision>
     </link>
-<!--
-    <joint name="${name}_optical_joint" type="fixed">
-      <origin xyz="${cal_kinect_x}            ${cal_kinect_y}         ${cal_kinect_z}"
-                rpy="${-M_PI/2+cal_kinect_roll} ${0.0+cal_kinect_pitch} ${-M_PI/2+cal_kinect_yaw}" />
-      <parent link="${name}_kinect_frame"/>
-      <child link="${name}_optical_frame"/>
+    <!-- prosilica sensor frame -->
+    <joint name="${name}_prosilica_optical_frame_joint" type="fixed">
+      <origin xyz="${cal_high_def_x}            ${cal_high_def_y}         ${cal_high_def_z}"
+                rpy="${-M_PI/2+cal_high_def_roll} ${0.0+cal_high_def_pitch} ${-M_PI/2+cal_high_def_yaw}" />
+      <parent link="${name}_prosilica_link"/>
+      <child link="${name}_prosilica_optical_frame"/>
     </joint>
-    <link name="${name}_optical_frame"/>
--->
+    <link name="${name}_prosilica_optical_frame"/>
+    <!-- gazebo extensions -->
+    <xacro:prosilica_cam_gazebo_v1 link_name="${name}_prosilica_link" camera_name="prosilica_camera" frame_name="${name}_prosilica_optical_frame" />
   </xacro:macro>
-</robot>
+</root>

Commit message: Added new files for Kinect2

File: pr2_description/robots/pr2_kinect2.urdf.xacro (robot description, xacro)
@@ -20,5 +20,5 @@
   <!-- Head sensors -->
   <xacro:include filename="$(find pr2_description)/urdf/sensors/head_sensor_package.urdf.xacro" />
-  <xacro:include filename="$(find pr2_description)/urdf/sensors/kinect2.urdf.xacro" />
+  <xacro:include filename="$(find pr2_description)/urdf/sensors/kinect2_v0/kinect2.urdf.xacro" />
   <!-- Camera sensors -->
   <xacro:include filename="$(find pr2_description)/urdf/sensors/wge100_camera.urdf.xacro" />

File: pr2_description/urdf/sensors/kinect2.urdf.xacro (robot description, xacro)
@@ -3,5 +3,4 @@
   <!-- Instead of making a xacro for each individual component, create one .STL for the frame, mount and the Kinect2 -->
   <!-- Multiple components is also likely the cause of the tf linking problem -->
-  <!-- Jeff is making the CAD file for the assembly -->
   <!-- Depending on where origin is for the mesh, a joint and link may be needed for the camera/ir sensor -->
   <xacro:include filename="$(find pr2_description)/urdf/sensors/kinect2.gazebo.xacro" />
@@ -27,5 +26,5 @@
         <origin xyz="0 -0.138 0" rpy="${M_PI/2} 0 ${M_PI/2}"/>
         <geometry>
-          <mesh filename="package://pr2_description/meshes/sensors/kinect2_v0/kinect2_mount.STL" scale="0.001 0.001 0.001" />
+          <mesh filename="package://pr2_description/meshes/sensors/kinect2_v0/KinectAssembly.stl" scale="0.001 0.001 0.001" />
         </geometry>
         <material name="gray">
@@ -90,5 +89,5 @@
             <color rgba="0.05 0.05 0.05 1"/>
           </material>
-        </geometry>
+        </geometry>  if [ $V \< 13.10 ]; then
       </visual>
       <collision>
