Commit message: now it runs in sim.  but you'll need the latest branch.

File: pr2_description/robots/pr2.urdf.xacro (robot description, xacro)
@@ -61,6 +61,6 @@
     <origin xyz="0.0 -0.188 0.0" rpy="0 0 0" />
   </xacro:pr2_shoulder>
-  <xacro:pr2_upper_arm side="r" reflect="-1" parent="torso_lift_link"/>
-  <xacro:pr2_forearm side="r" reflect="-1" parent="torso_lift_link"/>
+  <xacro:pr2_upper_arm side="r" reflect="-1" parent="r_upper_arm_roll_link"/>
+  <xacro:pr2_forearm side="r" reflect="-1" parent="r_forearm_roll_link"/>
   <xacro:pr2_gripper screw_reduction="${2.0/1000.0}" gear_ratio="${29.16}" side="r" parent="r_wrist_roll_link" >
     <origin xyz="0 0 0" rpy="0 0 0" />
@@ -69,6 +69,6 @@
     <origin xyz="0.0 0.188 0.0" rpy="0 0 0" />
   </xacro:pr2_shoulder>
-  <xacro:pr2_upper_arm side="l" reflect="1" parent="torso_lift_link"/>
-  <xacro:pr2_forearm side="l" reflect="1" parent="torso_lift_link"/>
+  <xacro:pr2_upper_arm side="l" reflect="1" parent="l_upper_arm_roll_link"/>
+  <xacro:pr2_forearm side="l" reflect="1" parent="l_forearm_roll_link"/>
   <xacro:pr2_gripper screw_reduction="${2.0/1000.0}" gear_ratio="${29.16}" side="l" parent="l_wrist_roll_link" >
     <origin xyz="0 0 0" rpy="0 0 0" />

File: pr2_description/urdf/base_v0/base.gazebo.xacro (robot description, xacro)
@@ -9,14 +9,4 @@
   <xacro:macro name="pr2_wheel_gazebo" params="suffix parent">
     <gazebo reference="${parent}_${suffix}_wheel_link">
-      <sensor:contact name="${parent}_${suffix}_wheel_contact_sensor">
-        <geom>${parent}_${suffix}_wheel_link_geom</geom>
-        <updateRate>100.0</updateRate>
-        <controller:ros_bumper name="${parent}_${suffix}_wheel_ros_bumper_controller" plugin="libros_bumper.so">
-          <alwaysOn>true</alwaysOn>
-          <updateRate>100.0</updateRate>
-          <bumperTopicName>${parent}_${suffix}_wheel_bumper</bumperTopicName>
-          <interface:bumper name="${parent}_${suffix}_wheel_ros_bumper_iface" />
-        </controller:ros_bumper>
-      </sensor:contact>
       <mu1 value="100.0" />
       <mu2 value="100.0" />

File: pr2_description/urdf/base_v0/base.urdf.xacro (robot description, xacro)
@@ -6,18 +6,19 @@
   <include filename="$(find pr2_description)/urdf/base_v0/base.gazebo.xacro" />
   <include filename="$(find pr2_description)/urdf/base_v0/base.transmission.xacro" />
+  <!-- DATA SOURCES -->
+  <!-- all link offsets, CG, limits are obtained from Function Engineering spreadsheet 090224_link_data.xls unless stated otherwise -->
+  <!-- all link geometry sizes are obtained from Function provided CAD model unless stated otherwise -->
+  <!-- all simplified collision geometry are hand approximated from CAD model, sometimes from respective bounding boxes -->
   <property name="M_PI" value="3.1415926535897931" />
   <property name="caster_offset_x" value="0.2225" />
   <property name="caster_offset_y" value="0.2225" />
   <property name="caster_offset_z" value="0.0282" />
-  <property name="caster_wheel_offset_y" value="0.049" /> <!-- from function spreadsheet -->
-  <property name="wheel_length" value="0.03" />  <!-- FIXME -->
+  <property name="caster_wheel_offset_y" value="0.049" />
+  <property name="wheel_length" value="0.034" />
   <property name="wheel_radius" value="0.074792" />   <!-- This is the 'effective' wheel radius. Wheel radius for uncompressed wheel is 0.079.  mp 20080801 -->
-  <!-- based on 090224_link_data from function engineering -->
   <property name="base_cg_x" value="-0.061" />
   <property name="base_cg_y" value="0.0" />
   <property name="base_cg_z" value="0.293" />
   <property name="base_mass" value="116.0" />
-  <!-- base appears "raised" from our initial geom def from function -->
-  <property name="base_height_offset" value="0.05" />
   <!-- simplified box collision geometry for base -->
   <property name="base_size_x" value="0.65" />
@@ -46,5 +47,5 @@
     <link name="${parent}_${suffix}_wheel_link">
       <inertial>
-        <mass value="0.44036" /> <!-- check jmh 20081205 -->
+        <mass value="0.44036" />
         <origin xyz="0 0 0" />
         <inertia  ixx="0.012411765597" ixy="-0.000711733678" ixz="0.00050272983"
@@ -54,10 +55,10 @@
         <origin xyz="0 0 0" rpy="0 0 0" />
         <geometry name="${parent}_${suffix}_wheel_visual_geom">
-          <mesh filename="package://pr2_defs/meshes/pr2_wheel.stl" />
+          <mesh filename="package://pr2_description/meshes/base_v0/pr2_wheel.stl" />
         </geometry>
         <material name="Caster_${suffix}" />
       </visual>
       <collision name="${parent}_${suffix}_wheel_collision">
-        <origin xyz="0 0 0" rpy="${M_PI/2} 0 0" />
+        <origin xyz="0 0 0" rpy="${M_PI/2} 0 0" /> <!-- rotation because cyl. geom primitive has symmetry axis in +x direction -->
         <geometry name="${parent}_${suffix}_wheel_collision_geom">
           <cylinder radius="${wheel_radius}" length="${wheel_length}" />
@@ -90,5 +91,5 @@
         <origin xyz="0 0 0" rpy="0 0 0" />
         <geometry name="${suffix}_caster_rotation_visual_geom">
-          <mesh filename="package://pr2_defs/meshes/caster.stl" />
+          <mesh filename="package://pr2_description/meshes/base_v0/caster.stl" />
         </geometry>
         <material name="Green" />
@@ -102,9 +103,10 @@
     </link>
     <!-- Double check these are right for the Alpha 2.0's -->
-    <xacro:pr2_wheel_alpha2 parent="${suffix}_caster" suffix="l" reflect="1" />
-    <xacro:pr2_wheel_alpha2 parent="${suffix}_caster" suffix="r" reflect="-1" />
+    <xacro:pr2_wheel parent="${suffix}_caster" suffix="l" reflect="1" />
+    <xacro:pr2_wheel parent="${suffix}_caster" suffix="r" reflect="-1" />
     <!-- extensions -->
-    <xacro:pr2_caster_alpha2_transmission suffix="${suffix}" />
+    <xacro:pr2_caster_transmission suffix="${suffix}" />
   </xacro:macro>
+  <!-- The xacro macro xacro:pr2_base contains: base, casters and wheels -->
   <xacro:macro name="pr2_base" params="name *origin">
     <joint name="${name}_joint" type="planar">
@@ -121,12 +123,12 @@
       </inertial>
       <visual name="${name}_visual">
-        <origin xyz="0 0 ${base_height_offset}" rpy="0 0 0" />
+        <origin xyz="0 0 0" rpy="0 0 0" />
         <geometry name="${name}_visual_geom">
-          <mesh filename="package://pr2_defs/meshes/base.stl" />
+          <mesh filename="package://pr2_description/meshes/base_v0/base.stl" />
         </geometry>
         <material name="Green" />
       </visual>
       <collision name="${name}_collision">
-        <origin xyz="0 0 ${base_height_offset+base_size_z/2}" rpy="0 0 0" />
+        <origin xyz="0 0 ${base_size_z/2}" rpy="0 0 0" />
         <geometry name="${name}_collision_geom">
           <box size="${base_size_x} ${base_size_y} ${base_size_z}" />
@@ -136,5 +138,5 @@
     <!-- base laser -->
     <xacro:hokuyo_lx30_laser name="${name}_laser" parent="${name}" ros_topic="base_scan" >
-      <origin xyz="${base_laser_x} ${base_laser_y} ${base_height_offset+base_laser_z}" rpy="0 0 0" />
+      <origin xyz="${base_laser_x} ${base_laser_y} ${base_laser_z}" rpy="0 0 0" />
     </xacro:hokuyo_lx30_laser>
     <!-- all four caster macros -->

File: pr2_description/urdf/common.xacro (robot description, xacro)
@@ -27,6 +27,6 @@
   <property name="cal_head_pan_flag"  value="0.0" />
   <property name="cal_head_tilt_flag" value="0.0" />
-  <property name="cal_head_pan_flag_alpha2" value="0.0"/>
-  <property name="cal_head_tilt_flag_alpha2" value="0.0"/>
+  <property name="cal_head_pan_flag" value="0.0"/>
+  <property name="cal_head_tilt_flag" value="0.0"/>
   <!-- Casters -->
   <property name="cal_caster_fl" value="0.0" />

File: pr2_description/urdf/forearm_v0/forearm.urdf.xacro (robot description, xacro)
@@ -28,5 +28,5 @@
         <origin xyz="0 0 0" rpy="0 0 0" />
         <geometry name="${side}_forearm_visual_geom">
-          <mesh filename="package://pr2_defs/meshes/forearm.stl" />
+          <mesh filename="package://pr2_description/meshes/forearm_v0/forearm.stl" />
         </geometry>
         <material name="Blue" />
@@ -35,5 +35,5 @@
         <origin xyz="0 0 0" rpy="0 0 0" />
         <geometry name="${side}_forearm_collision_geom">
-          <mesh filename="package://pr2_defs/meshes/convex/forearm_convex.stlb" />
+          <mesh filename="package://pr2_description/meshes/forearm_v0/convex/forearm_convex.stlb" />
         </geometry>
       </collision>
@@ -61,5 +61,5 @@
         <origin xyz="0 0 0" rpy="0 0 0" />
         <geometry name="${side}_wrist_flex_visual_geom">
-          <mesh filename="package://pr2_defs/meshes/wrist_flex.stl" />
+          <mesh filename="package://pr2_description/meshes/forearm_v0/wrist_flex.stl" />
         </geometry>
         <material name="Grey" />
@@ -68,5 +68,5 @@
         <origin xyz="0 0 0" rpy="0 0 0" />
         <geometry name="${side}_wrist_flex_collision_geom">
-          <mesh filename="package://pr2_defs/meshes/convex/wrist_flex_convex.stlb" />
+          <mesh filename="package://pr2_description/meshes/forearm_v0/convex/wrist_flex_convex.stlb" />
         </geometry>
       </collision>
@@ -95,5 +95,5 @@
         <origin xyz="0 0 0" rpy="0 0 0" />
         <geometry name="${side}_wrist_roll_visual_geom">
-          <mesh filename="package://pr2_defs/meshes/wrist_roll.stl" />
+          <mesh filename="package://pr2_description/meshes/forearm_v0/wrist_roll.stl" />
         </geometry>
         <material name="RollLinks" />

File: pr2_description/urdf/gripper_v0/gripper.urdf.xacro (robot description, xacro)
@@ -43,5 +43,5 @@
         <origin xyz="0 0 0" rpy="0 0 0" />
         <geometry name="${prefix}_l_finger_visual_geom">
-          <mesh filename="package://pr2_defs/meshes/upper_finger_l.stl" />
+          <mesh filename="package://pr2_description/meshes/gripper_v0/upper_finger_l.stl" />
         </geometry>
         <material name="Grey" />
@@ -50,5 +50,5 @@
         <origin xyz="0 0 0" rpy="0 0 0" />
         <geometry name="${prefix}_l_finger_collision_geom">
-          <mesh filename="package://pr2_defs/meshes/convex/upper_finger_l_convex.stlb" />
+          <mesh filename="package://pr2_description/meshes/gripper_v0/convex/upper_finger_l_convex.stlb" />
         </geometry>
         <verbose value="Yes" />
@@ -79,5 +79,5 @@
         <origin xyz="0 0 0" rpy="0 0 0" />
         <geometry name="${prefix}_r_finger_visual_geom">
-          <mesh filename="package://pr2_defs/meshes/upper_finger_r.stl" />
+          <mesh filename="package://pr2_description/meshes/gripper_v0/upper_finger_r.stl" />
         </geometry>
         <material name="Grey" />
@@ -86,5 +86,5 @@
         <origin xyz="0 0 0" rpy="0 0 0" />
         <geometry name="${prefix}_r_finger_collision_geom">
-          <mesh filename="package://pr2_defs/meshes/convex/upper_finger_r_convex.stlb" />
+          <mesh filename="package://pr2_description/meshes/gripper_v0/convex/upper_finger_r_convex.stlb" />
         </geometry>
         <verbose value="Yes" />
@@ -112,5 +112,5 @@
         <origin xyz="0 0 0" rpy="0 0 0" />
         <geometry name="${prefix}_l_finger_tip_visual_geom">
-          <mesh filename="package://pr2_defs/meshes/finger_tip_l.stl" />
+          <mesh filename="package://pr2_description/meshes/gripper_v0/finger_tip_l.stl" />
         </geometry>
         <material name="Green" />
@@ -119,5 +119,5 @@
         <origin xyz="0 0 0" rpy="0 0 0" />
         <geometry name="${prefix}_l_finger_tip_collision_geom">
-          <mesh filename="package://pr2_defs/meshes/finger_tip_pad2_l.stl" />
+          <mesh filename="package://pr2_description/meshes/gripper_v0/finger_tip_pad2_l.stl" />
         </geometry>
         <verbose value="Yes" />
@@ -145,5 +145,5 @@
         <origin xyz="0 0 0" rpy="0 0 0" />
         <geometry name="${prefix}_r_finger_tip_visual_geom">
-          <mesh filename="package://pr2_defs/meshes/finger_tip_r.stl" />
+          <mesh filename="package://pr2_description/meshes/gripper_v0/finger_tip_r.stl" />
         </geometry>
         <material name="Green" />
@@ -152,5 +152,5 @@
         <origin xyz="0 0 0" rpy="0 0 0" />
         <geometry name="${prefix}_r_finger_tip_collision_geom">
-          <mesh filename="package://pr2_defs/meshes/finger_tip_pad2_r.stl" />
+          <mesh filename="package://pr2_description/meshes/gripper_v0/finger_tip_pad2_r.stl" />
         </geometry>
         <verbose value="Yes" />
@@ -177,5 +177,5 @@
         <origin xyz="0 0 0" rpy="0 0 0" />
         <geometry name="${side}_gripper_palm_visual_geom">
-          <mesh filename="package://pr2_defs/meshes/gripper_palm.stl" />
+          <mesh filename="package://pr2_description/meshes/gripper_v0/gripper_palm.stl" />
         </geometry>
         <material name="Red" />
@@ -184,5 +184,5 @@
         <origin xyz="0 0 0" rpy="0 0 0" />
         <geometry name="${side}_gripper_palm_collision_geom">
-          <mesh filename="package://pr2_defs/meshes/convex/gripper_palm_convex.stlb" />
+          <mesh filename="package://pr2_description/meshes/gripper_v0/convex/gripper_palm_convex.stlb" />
         </geometry>
         <verbose value="Yes" />

File: pr2_description/urdf/head_v0/head.urdf.xacro (robot description, xacro)
@@ -28,5 +28,5 @@
         <origin xyz="0 0 0.0" rpy="0 0 0 " />
         <geometry name="${name}_visual_geom">
-          <mesh filename="package://pr2_defs/meshes/head_pan.stl" />
+          <mesh filename="package://pr2_description/head_v0/meshes/head_pan.stl" />
         </geometry>
         <material name="Blue" />
@@ -65,5 +65,5 @@
         <origin xyz="0 0 0" rpy="0.0 0.0 0.0 " />
         <geometry name="${name}_visual_geom">
-          <mesh filename="package://pr2_defs/meshes/head_tilt.stl" />
+          <mesh filename="package://pr2_description/head_v0/meshes/head_tilt.stl" />
         </geometry>
         <material name="Green" />

File: pr2_description/urdf/shoulder_v0/shoulder.urdf.xacro (robot description, xacro)
@@ -40,5 +40,5 @@
         <origin xyz="0 0 0" rpy="0 0 0" />
         <geometry name="${side}_shoulder_pan_visual_geom">
-          <mesh filename="package://pr2_defs/meshes/shoulder_yaw.stl" />
+          <mesh filename="package://pr2_description/meshes/shoulder_v0/shoulder_yaw.stl" />
         </geometry>
         <material name="Blue" />
@@ -47,5 +47,5 @@
         <origin xyz="0.0 0 0.0" rpy="0 0 0" />
         <geometry name="${side}_shoulder_pan_collision_geom">
-          <mesh filename="package://pr2_defs/meshes/convex/shoulder_yaw_convex.stlb" />
+          <mesh filename="package://pr2_description/meshes/shoulder_v0/convex/shoulder_yaw_convex.stlb" />
         </geometry>
       </collision>
@@ -76,5 +76,5 @@
         <origin xyz="0 0 0" rpy="0 0 0" />
         <geometry name="${side}_shoulder_lift_visual_geom">
-          <mesh filename="package://pr2_defs/meshes/shoulder_lift.stl" />
+          <mesh filename="package://pr2_description/meshes/shoulder_v0/shoulder_lift.stl" />
         </geometry>
         <material name="Grey" />
@@ -83,5 +83,5 @@
         <origin xyz="0 0 0" rpy="0 0 0" />
         <geometry name="${side}_shoulder_lift_collision_geom">
-          <mesh filename="package://pr2_defs/meshes/convex/shoulder_lift_convex.stlb" />
+          <mesh filename="package://pr2_description/meshes/shoulder_v0/convex/shoulder_lift_convex.stlb" />
         </geometry>
       </collision>
@@ -111,5 +111,5 @@
         <origin xyz="0 0 0" rpy="0 0 0" />
         <geometry name="${side}_upper_arm_roll_visual_geom">
-          <mesh filename="package://pr2_defs/meshes/upper_arm_roll.stl" />
+          <mesh filename="package://pr2_description/shoulder_v0/meshes/upper_arm_roll.stl" />
         </geometry>
         <material name="RollLinks" />

File: pr2_description/urdf/tilting_laser_v0/tilting_laser.urdf.xacro (robot description, xacro)
@@ -29,5 +29,5 @@
         <origin xyz="0 0 0" rpy="0 0 0" />
         <geometry name="${name}_mount_visual_geom">
-          <mesh filename="package://pr2_defs/meshes/hok_tilt.stl" />
+          <mesh filename="package://pr2_description/meshes/tilting_laser_v0/hok_tilt.stl" />
         </geometry>
         <material name="Red" />

File: pr2_description/urdf/torso_v0/torso.urdf.xacro (robot description, xacro)
@@ -29,12 +29,13 @@
         <origin xyz="0 0 0" rpy="0 0 0" />
         <geometry name="${name}_visual_geom">
-          <mesh filename="package://pr2_defs/meshes/torso.stl" />
+          <mesh filename="package://pr2_description/meshes/torso_v0/torso.stl" />
         </geometry>
         <material name="Grey2" />
       </visual>
       <collision name="${name}_collision">
-        <origin xyz="-0.1 0 -0.0885" rpy="0 0 0" />
+        <origin xyz="0 0 0.16" rpy="0 0 0" />
         <geometry name="${name}_collision_geom">
-          <box size="0.30 0.620 0.823" />
+          <!-- arbitrarily chosen collision box by JH, torso collision is not important for now -->
+          <box size="0.30 0.620 0.02" />
         </geometry>
       </collision>

File: pr2_description/urdf/upper_arm_v0/upper_arm.urdf.xacro (robot description, xacro)
@@ -51,5 +51,5 @@
         <origin xyz="0 0 0" rpy="0 0 0" />
         <geometry name="${side}_upper_arm_visual_geom">
-          <mesh filename="package://pr2_defs/meshes/upper_arm.stl" />
+          <mesh filename="package://pr2_description/meshes/upper_arm_v0/upper_arm.stl" />
         </geometry>
         <material name="Green" />
@@ -58,5 +58,5 @@
         <origin xyz="0 0 0" rpy="0 0 0" />
         <geometry name="${side}_upper_arm_collision_geom">
-          <mesh filename="package://pr2_defs/meshes/convex/upper_arm_convex.stlb" />
+          <mesh filename="package://pr2_description/meshes/upper_arm_v0/convex/upper_arm_convex.stlb" />
         </geometry>
       </collision>
@@ -84,5 +84,5 @@
         <origin xyz="0 0 0" rpy="0 0 0" />
         <geometry name="${side}_elbow_flex_visual_geom">
-          <mesh filename="package://pr2_defs/meshes/elbow_flex.stl" />
+          <mesh filename="package://pr2_description/meshes/upper_arm_v0/elbow_flex.stl" />
         </geometry>
         <material name="Grey" />
@@ -91,9 +91,9 @@
         <origin xyz="0 0 0" rpy="0 0 0" />
         <geometry name="${side}_elbow_flex_collision_geom">
-          <mesh filename="package://pr2_defs/meshes/convex/elbow_flex_convex.stlb" />
+          <mesh filename="package://pr2_description/meshes/upper_arm_v0/convex/elbow_flex_convex.stlb" />
         </geometry>
       </collision>
     </link>
-<!-- forearm roll -->
+    <!-- forearm_roll_link is a fictitious link internal to elbow_flex_link, provides an attachment point for the actual forearm -->
     <joint name="${side}_forearm_roll_joint" type="continuous">
       <axis xyz="-1 0 0" />
@@ -106,4 +106,5 @@
       <child link="${side}_forearm_roll_link"/>
     </joint>
+    <!-- TODO: inertial tag should be optional -->
     <link name="${side}_forearm_roll_link">
       <inertial>
@@ -115,12 +116,14 @@
                   izz="0.01" />
       </inertial>
-      <visual name="${side}_forearm_roll_visual"><!-- TODO: need a mesh for this -->
+      <visual name="${side}_forearm_roll_visual">
         <origin xyz="0 0 0" rpy="0 0 0" />
         <geometry name="${side}_forearm_roll_visual_geom">
-          <mesh filename="package://pr2_defs/meshes/forearm_roll.stl" />
+          <mesh filename="package://pr2_description/meshes/upper_arm_v0/forearm_roll.stl" />
         </geometry>
         <material name="RollLinks" />
       </visual>
-      <collision name="${side}_forearm_roll_collision"> <!-- TODO: collision tag should be optional -->
+      <!-- TODO: collision tag should be optional -->
+      <collision name="${side}_forearm_roll_collision">
+        <!-- dummy geom, to be removed -->
         <origin xyz="0 0 0" rpy="0 0 0" />
         <geometry name="${side}_forearm_roll_collision_geom">
