Commit message: migrated gripper_beta from pr2_defs into pr2_description/urdf/gripper_v0.

File: pr2_description/robots/pr2.urdf.xacro (robot description, xacro)
@@ -63,5 +63,15 @@
   <xacro:pr2_upper_arm side="r" reflect="-1" parent="r_upper_arm_roll_link"/>
   <xacro:pr2_forearm side="r" reflect="-1" parent="r_forearm_roll_link"/>
-  <xacro:pr2_gripper screw_reduction="${2.0/1000.0}" gear_ratio="${29.16}" side="r" parent="r_wrist_roll_link" >
+  <xacro:pr2_gripper side="r" parent="r_wrist_roll_link"
+               screw_reduction="${4.0/1000.0}"
+               gear_ratio="${(729.0/25.0)*(22.0/16.0)}"
+               theta0="${3.6029*M_PI/180.0}"
+               phi0="${29.7089*M_PI/180.0}"
+               t0="${-0.1914/1000.0}"
+               L0="${37.5528/1000.0}"
+               h="${0.0/1000.0}"
+               a="${68.3698/1000.0}"
+               b="${43.3849/1000.0}"
+               r="${91.5/1000.0}" >
     <origin xyz="0 0 0" rpy="0 0 0" />
   </xacro:pr2_gripper>
@@ -71,5 +81,15 @@
   <xacro:pr2_upper_arm side="l" reflect="1" parent="l_upper_arm_roll_link"/>
   <xacro:pr2_forearm side="l" reflect="1" parent="l_forearm_roll_link"/>
-  <xacro:pr2_gripper screw_reduction="${2.0/1000.0}" gear_ratio="${29.16}" side="l" parent="l_wrist_roll_link" >
+  <xacro:pr2_gripper side="l" parent="l_wrist_roll_link"
+               screw_reduction="${4.0/1000.0}"
+               gear_ratio="${(729.0/25.0)*(22.0/16.0)}"
+               theta0="${3.6029*M_PI/180.0}"
+               phi0="${29.7089*M_PI/180.0}"
+               t0="${-0.1914/1000.0}"
+               L0="${37.5528/1000.0}"
+               h="${0.0/1000.0}"
+               a="${68.3698/1000.0}"
+               b="${43.3849/1000.0}"
+               r="${91.5/1000.0}" >
     <origin xyz="0 0 0" rpy="0 0 0" />
   </xacro:pr2_gripper>

File: pr2_description/urdf/gripper_v0/gripper.transmission.xacro (robot description, xacro)
@@ -5,5 +5,5 @@
        xmlns:interface="http://playerstage.sourceforge.net/gazebo/xmlschema/#interface"
        xmlns:xacro="http://ros.org/wiki/xacro">
-  <xacro:macro name="pr2_gripper_transmission" params="side">
+  <xacro:macro name="pr2_gripper_transmission" params="side screw_reduction gear_ratio theta0 phi0 t0 L0 h a b r">
     <!-- [lr]_gripper_joint is a fictitious joint, used by transmission for controller gap   -->
     <!-- [lr]_gripper_joint is not attached to any link                                      -->
@@ -17,5 +17,17 @@
     <transmission type="PR2GripperTransmission" name="${side}_gripper_trans" >
       <actuator       name="${side}_gripper_motor" />
-      <gap_joint      name="${side}_gripper_joint" screw_reduction="${screw_reduction}" gear_ratio="${gear_ratio}" mechanical_reduction="1.0" />
+      <gap_joint      name="${side}_gripper_joint"
+                      mechanical_reduction="1.0"
+                      screw_reduction="${screw_reduction}"
+                      gear_ratio="${gear_ratio}"
+                      theta0="${theta0}"
+                      phi0="${phi0}"
+                      t0="${t0}"
+                      L0="${L0}"
+                      h="${h}"
+                      a="${a}"
+                      b="${b}"
+                      r="${r}"
+                      />
       <passive_joint  name="${side}_gripper_l_finger_joint"     />
       <passive_joint  name="${side}_gripper_r_finger_joint"     />

File: pr2_description/urdf/gripper_v0/gripper.urdf.xacro (robot description, xacro)
@@ -23,5 +23,5 @@
     <joint name="${prefix}_l_finger_joint" type="revolute">
       <axis xyz="0 0 1" />
-      <pr2_finger_limits reflect="1" />
+      <xacro:pr2_finger_limits reflect="1" />
       <dynamics damping="${finger_damping}" />
       <origin xyz="0.07691 0.01 0" rpy="0 0 0" />
@@ -43,5 +43,5 @@
         <origin xyz="0 0 0" rpy="0 0 0" />
         <geometry name="${prefix}_l_finger_visual_geom">
-          <mesh filename="package://pr2_description/meshes/gripper_v0/upper_finger_l.stl" />
+          <mesh filename="package://pr2_defs/meshes/upper_finger_l.stl" />
         </geometry>
         <material name="Grey" />
@@ -50,5 +50,5 @@
         <origin xyz="0 0 0" rpy="0 0 0" />
         <geometry name="${prefix}_l_finger_collision_geom">
-          <mesh filename="package://pr2_description/meshes/gripper_v0/convex/upper_finger_l_convex.stlb" />
+          <mesh filename="package://pr2_defs/meshes/convex/upper_finger_l_convex.stlb" />
         </geometry>
         <verbose value="Yes" />
@@ -59,5 +59,5 @@
       <axis xyz="0 0 -1" />
       <origin xyz="0.07691 -0.01 0" rpy="0 0 0" />
-      <pr2_finger_limits reflect="1" />
+      <xacro:pr2_finger_limits reflect="1" />
       <dynamics damping="${finger_damping}" />
       <mimic joint="${prefix}_l_finger_joint" multiplier="1" offset="0"/>
@@ -79,5 +79,5 @@
         <origin xyz="0 0 0" rpy="0 0 0" />
         <geometry name="${prefix}_r_finger_visual_geom">
-          <mesh filename="package://pr2_description/meshes/gripper_v0/upper_finger_r.stl" />
+          <mesh filename="package://pr2_defs/meshes/upper_finger_r.stl" />
         </geometry>
         <material name="Grey" />
@@ -86,5 +86,5 @@
         <origin xyz="0 0 0" rpy="0 0 0" />
         <geometry name="${prefix}_r_finger_collision_geom">
-          <mesh filename="package://pr2_description/meshes/gripper_v0/convex/upper_finger_r_convex.stlb" />
+          <mesh filename="package://pr2_defs/meshes/convex/upper_finger_r_convex.stlb" />
         </geometry>
         <verbose value="Yes" />
@@ -95,5 +95,5 @@
       <axis xyz="0 0 -1" />
       <origin xyz="0.09137 0.00495 0" rpy="0 0 0" />
-      <pr2_finger_limits reflect="1" />
+      <xacro:pr2_finger_limits reflect="1" />
       <dynamics damping="${finger_tip_damping}" />
       <mimic joint="${prefix}_l_finger_joint" multiplier="1" offset="0"/>
@@ -112,5 +112,5 @@
         <origin xyz="0 0 0" rpy="0 0 0" />
         <geometry name="${prefix}_l_finger_tip_visual_geom">
-          <mesh filename="package://pr2_description/meshes/gripper_v0/finger_tip_l.stl" />
+          <mesh filename="package://pr2_defs/meshes/finger_tip_l.stl" />
         </geometry>
         <material name="Green" />
@@ -119,5 +119,5 @@
         <origin xyz="0 0 0" rpy="0 0 0" />
         <geometry name="${prefix}_l_finger_tip_collision_geom">
-          <mesh filename="package://pr2_description/meshes/gripper_v0/finger_tip_pad2_l.stl" />
+          <mesh filename="package://pr2_defs/meshes/finger_tip_pad2_l.stl" />
         </geometry>
         <verbose value="Yes" />
@@ -128,5 +128,5 @@
       <axis xyz="0 0 1" />
       <origin xyz="${0.09137} ${-0.00495} 0" rpy="0 0 0" />
-      <pr2_finger_limits reflect="1" />
+      <xacro:pr2_finger_limits reflect="1" />
       <dynamics damping="${finger_tip_damping}" />
       <mimic joint="${prefix}_l_finger_joint" multiplier="1" offset="0"/>
@@ -145,5 +145,5 @@
         <origin xyz="0 0 0" rpy="0 0 0" />
         <geometry name="${prefix}_r_finger_tip_visual_geom">
-          <mesh filename="package://pr2_description/meshes/gripper_v0/finger_tip_r.stl" />
+          <mesh filename="package://pr2_defs/meshes/finger_tip_r.stl" />
         </geometry>
         <material name="Green" />
@@ -152,5 +152,5 @@
         <origin xyz="0 0 0" rpy="0 0 0" />
         <geometry name="${prefix}_r_finger_tip_collision_geom">
-          <mesh filename="package://pr2_description/meshes/gripper_v0/finger_tip_pad2_r.stl" />
+          <mesh filename="package://pr2_defs/meshes/finger_tip_pad2_r.stl" />
         </geometry>
         <verbose value="Yes" />
@@ -158,7 +158,7 @@
     </link>
     <!-- extensions -->
-    <pr2_finger_gazebo prefix="${prefix}" />
+    <xacro:pr2_finger_gazebo prefix="${prefix}" />
   </xacro:macro>
-  <xacro:macro name="pr2_gripper" params="side parent *origin gear_ratio screw_reduction">
+  <xacro:macro name="pr2_gripper" params="side parent *origin gear_ratio screw_reduction theta0 phi0 t0 L0 h a b r">
     <joint name="${side}_gripper_palm_joint" type="fixed">
       <insert_block name="origin"/>
@@ -177,5 +177,5 @@
         <origin xyz="0 0 0" rpy="0 0 0" />
         <geometry name="${side}_gripper_palm_visual_geom">
-          <mesh filename="package://pr2_description/meshes/gripper_v0/gripper_palm.stl" />
+          <mesh filename="package://pr2_defs/meshes/gripper_palm.stl" />
         </geometry>
         <material name="Red" />
@@ -184,5 +184,5 @@
         <origin xyz="0 0 0" rpy="0 0 0" />
         <geometry name="${side}_gripper_palm_collision_geom">
-          <mesh filename="package://pr2_description/meshes/gripper_v0/convex/gripper_palm_convex.stlb" />
+          <mesh filename="package://pr2_defs/meshes/convex/gripper_palm_convex.stlb" />
         </geometry>
         <verbose value="Yes" />
@@ -284,9 +284,19 @@
       <axis xyz="0 0 1" />
       <limit effort="100.0" velocity="0.2" lower="0.0" upper="0.09" />
-      <safety_controller k_velocity="500.0" k_position="20.0" soft_lower_limit="${0.0-0.01}" soft_upper_limit="${0.09-0.001}" />
+      <safety_controller k_velocity="500.0" k_position="20.0" soft_lower_limit="${0.0-0.01}" soft_upper_limit="${0.09-0.002}" />
     </joint>
     <!-- extensions -->
-    <pr2_gripper_gazebo side="${side}" />
-    <pr2_gripper_transmission side="${side}" />
+    <xacro:pr2_gripper_gazebo side="${side}" />
+    <xacro:pr2_gripper_transmission side="${side}"
+        screw_reduction="${screw_reduction}"
+        gear_ratio="${gear_ratio}"
+        theta0="${theta0}"
+        phi0="${phi0}"
+        t0="${t0}"
+        L0="${L0}"
+        h="${h}"
+        a="${a}"
+        b="${b}"
+        r="${r}" />
   </xacro:macro>
 </robot>
