Commit message: * adding _v0 suffix to all macros.  * reuse wge100_camera macros for stereo camera.

File: pr2_description/robots/pr2.urdf.xacro (robot description, xacro)
@@ -24,4 +24,6 @@
   <!-- Head sensors -->
   <include filename="$(find pr2_description)/urdf/sensors/head_sensor_package.urdf.xacro" />
+  <!-- Camera sensors -->
+  <include filename="$(find pr2_description)/urdf/sensors/wge100_camera.urdf.xacro" />
   <!-- generic simulator_gazebo plugins for starting mechanism control, ros time, ros battery -->
   <include filename="$(find pr2_description)/gazebo/gazebo.urdf.xacro" />
@@ -36,32 +38,32 @@
        the origin block defines where the component is w.r.t its parent (in this case the parent
        is the world frame). For more, see http://www.ros.org/wiki/xacro -->
-  <xacro:pr2_base name="base" >
+  <xacro:pr2_base_v0 name="base" >
     <origin xyz="0 0 0.051" rpy="0 0 0" /> <!-- 5.1cm is the height of the base when wheels contact ground -->
-  </xacro:pr2_base>
-  <xacro:pr2_torso name="torso_lift" parent="base_link">
+  </xacro:pr2_base_v0>
+  <xacro:pr2_torso_v0 name="torso_lift" parent="base_link">
     <origin xyz="-0.05 0 0.739675" rpy="0 0 0" />
-  </xacro:pr2_torso>
+  </xacro:pr2_torso_v0>
   <!-- The xacro preprocesser will replace the parameters below, such as ${cal_head_x}, with
        numerical values that were specified in default_cal.xml which was included above -->
-  <xacro:pr2_head name="head" parent="torso_lift_link">
+  <xacro:pr2_head_v0 name="head" parent="torso_lift_link">
     <origin xyz="${cal_head_x}    ${cal_head_y}     ${0.3915+cal_head_z}"
             rpy="${cal_head_roll} ${cal_head_pitch} ${cal_head_yaw}" />
-  </xacro:pr2_head>
+  </xacro:pr2_head_v0>
   <!-- Camera package: double stereo, prosilica -->
-  <xacro:pr2_head_sensor_package name="sensor_mount" hd_name="high_def"
+  <xacro:pr2_head_sensor_package_v0 name="sensor_mount" hd_name="high_def"
 			   stereo_name="double_stereo"
 			   parent="head_plate_frame">
     <origin xyz="0.0 0.0 0.0" rpy="0 0 0" />
-  </xacro:pr2_head_sensor_package>
-  <xacro:pr2_tilting_laser name="laser_tilt" parent="torso_lift_link" laser_calib_ref="-0.35">
+  </xacro:pr2_head_sensor_package_v0>
+  <xacro:pr2_tilting_laser_v0 name="laser_tilt" parent="torso_lift_link" laser_calib_ref="-0.35">
     <origin xyz="0.1 0 0.235" rpy="0 0 0" />
-  </xacro:pr2_tilting_laser>
+  </xacro:pr2_tilting_laser_v0>
   <!-- This is a common convention, to use a reflect parameter that equals +-1 to distinguish left from right -->
-  <xacro:pr2_shoulder side="r" reflect="-1" parent="torso_lift_link">
+  <xacro:pr2_shoulder_v0 side="r" reflect="-1" parent="torso_lift_link">
     <origin xyz="0.0 -0.188 0.0" rpy="0 0 0" />
-  </xacro:pr2_shoulder>
-  <xacro:pr2_upper_arm side="r" reflect="-1" parent="r_upper_arm_roll_link"/>
-  <xacro:pr2_forearm side="r" reflect="-1" parent="r_forearm_roll_link"/>
-  <xacro:pr2_gripper side="r" parent="r_wrist_roll_link"
+  </xacro:pr2_shoulder_v0>
+  <xacro:pr2_upper_arm_v0 side="r" reflect="-1" parent="r_upper_arm_roll_link"/>
+  <xacro:pr2_forearm_v0 side="r" reflect="-1" parent="r_forearm_roll_link"/>
+  <xacro:pr2_gripper_v0 side="r" parent="r_wrist_roll_link"
                screw_reduction="${4.0/1000.0}"
                gear_ratio="${(729.0/25.0)*(22.0/16.0)}"
@@ -75,11 +77,11 @@
                r="${91.5/1000.0}" >
     <origin xyz="0 0 0" rpy="0 0 0" />
-  </xacro:pr2_gripper>
-  <xacro:pr2_shoulder side="l" reflect="1" parent="torso_lift_link">
+  </xacro:pr2_gripper_v0>
+  <xacro:pr2_shoulder_v0 side="l" reflect="1" parent="torso_lift_link">
     <origin xyz="0.0 0.188 0.0" rpy="0 0 0" />
-  </xacro:pr2_shoulder>
-  <xacro:pr2_upper_arm side="l" reflect="1" parent="l_upper_arm_roll_link"/>
-  <xacro:pr2_forearm side="l" reflect="1" parent="l_forearm_roll_link"/>
-  <xacro:pr2_gripper side="l" parent="l_wrist_roll_link"
+  </xacro:pr2_shoulder_v0>
+  <xacro:pr2_upper_arm_v0 side="l" reflect="1" parent="l_upper_arm_roll_link"/>
+  <xacro:pr2_forearm_v0 side="l" reflect="1" parent="l_forearm_roll_link"/>
+  <xacro:pr2_gripper_v0 side="l" parent="l_wrist_roll_link"
                screw_reduction="${4.0/1000.0}"
                gear_ratio="${(729.0/25.0)*(22.0/16.0)}"
@@ -93,13 +95,13 @@
                r="${91.5/1000.0}" >
     <origin xyz="0 0 0" rpy="0 0 0" />
-  </xacro:pr2_gripper>
+  </xacro:pr2_gripper_v0>
   <!-- Forearm Cam (Hand approximated values) -->
-  <xacro:wge100_camera name="l_forearm_cam" parent="l_forearm_roll_link">
-    <origin xyz=".15 0 .07"
-            rpy="${ M_PI/2} ${-45*M_PI/180} 0" />
-  </xacro:wge100_camera>
-  <xacro:wge100_camera name="r_forearm_cam" parent="r_forearm_roll_link">
-    <origin xyz=".15 0 .07"
-            rpy="${-M_PI/2} ${-45*M_PI/180} 0" />
-  </xacro:wge100_camera>
+  <xacro:wge100_camera_v0 name="l_forearm_cam" topic_name="l_forearm_cam/image"
+                          parent="l_forearm_roll_link" hfov="90" focal_length="320">
+    <origin xyz=".15 0 .07" rpy="${ M_PI/2} ${-45*M_PI/180} 0" />
+  </xacro:wge100_camera_v0>
+  <xacro:wge100_camera_v0 name="r_forearm_cam" topic_name="r_forearm_cam/image"
+                          parent="r_forearm_roll_link" hfov="90" focal_length="320">
+    <origin xyz=".15 0 .07" rpy="${-M_PI/2} ${-45*M_PI/180} 0" />
+  </xacro:wge100_camera_v0>
 </robot>

File: pr2_description/urdf/base_v0/base.gazebo.xacro (robot description, xacro)
@@ -7,5 +7,5 @@
   <!-- Alpha 2.0 hardware                                   -->
   <!--                                                      -->
-  <xacro:macro name="pr2_wheel_gazebo" params="suffix parent">
+  <xacro:macro name="pr2_wheel_gazebo_v0" params="suffix parent">
     <gazebo reference="${parent}_${suffix}_wheel_link">
       <mu1 value="100.0" />
@@ -15,5 +15,5 @@
     </gazebo>
   </xacro:macro>
-  <xacro:macro name="pr2_base_gazebo" params="name">
+  <xacro:macro name="pr2_base_gazebo_v0" params="name">
     <gazebo reference="${name}_link">
       <selfCollide>true</selfCollide>

File: pr2_description/urdf/base_v0/base.transmission.xacro (robot description, xacro)
@@ -7,5 +7,5 @@
   <!-- Alpha 2.0 hardware                                   -->
   <!--                                                      -->
-  <xacro:macro name="pr2_wheel_transmission" params="suffix parent reflect">
+  <xacro:macro name="pr2_wheel_transmission_v0" params="suffix parent reflect">
     <transmission type="SimpleTransmission" name="${parent}_${suffix}_wheel_trans">
       <actuator name="${parent}_${suffix}_wheel_motor_v0" />
@@ -14,5 +14,5 @@
     </transmission>
   </xacro:macro>
-  <xacro:macro name="pr2_caster_transmission" params="suffix">
+  <xacro:macro name="pr2_caster_transmission_v0" params="suffix">
     <transmission type="SimpleTransmission" name="${suffix}_caster_rotation_trans">
       <actuator name="${suffix}_caster_rotation_motor_v0" />

File: pr2_description/urdf/base_v0/base.urdf.xacro (robot description, xacro)
@@ -37,5 +37,5 @@
   <!--           wheel                                      -->
   <!--                                                      -->
-  <xacro:macro name="pr2_wheel" params="suffix parent reflect">
+  <xacro:macro name="pr2_wheel_v0" params="suffix parent reflect">
     <joint name="${parent}_${suffix}_wheel_joint" type="continuous">
       <axis xyz="0 1 0" />
@@ -69,8 +69,8 @@
     </link>
     <!-- extensions -->
-    <xacro:pr2_wheel_gazebo parent="${parent}" suffix="${suffix}" />
-    <xacro:pr2_wheel_transmission parent="${parent}" suffix="${suffix}" reflect="${reflect}" />
+    <xacro:pr2_wheel_gazebo_v0 parent="${parent}" suffix="${suffix}" />
+    <xacro:pr2_wheel_transmission_v0 parent="${parent}" suffix="${suffix}" reflect="${reflect}" />
   </xacro:macro>
-  <xacro:macro name="pr2_caster" params="suffix parent *origin ref_position">
+  <xacro:macro name="pr2_caster_v0" params="suffix parent *origin ref_position">
     <joint name="${suffix}_caster_rotation_joint" type="continuous">
       <axis xyz="0 0 1" />
@@ -105,11 +105,11 @@
     </link>
     <!-- wheel macros -->
-    <xacro:pr2_wheel parent="${suffix}_caster" suffix="l" reflect="1" />
-    <xacro:pr2_wheel parent="${suffix}_caster" suffix="r" reflect="-1" />
+    <xacro:pr2_wheel_v0 parent="${suffix}_caster" suffix="l" reflect="1" />
+    <xacro:pr2_wheel_v0 parent="${suffix}_caster" suffix="r" reflect="-1" />
     <!-- extensions -->
-    <xacro:pr2_caster_transmission suffix="${suffix}" />
+    <xacro:pr2_caster_transmission_v0 suffix="${suffix}" />
   </xacro:macro>
   <!-- The xacro macro xacro:pr2_base contains: base, casters and wheels -->
-  <xacro:macro name="pr2_base" params="name *origin">
+  <xacro:macro name="pr2_base_v0" params="name *origin">
     <joint name="${name}_joint" type="planar">
       <insert_block name="origin" />
@@ -141,22 +141,22 @@
     </link>
     <!-- base laser -->
-    <xacro:hokuyo_lx30_laser name="${name}_laser" parent="${name}" ros_topic="base_scan" >
+    <xacro:hokuyo_lx30_laser_v0 name="${name}_laser" parent="${name}" ros_topic="base_scan" >
       <origin xyz="${base_laser_x} ${base_laser_y} ${base_laser_z}" rpy="0 0 0" />
-    </xacro:hokuyo_lx30_laser>
+    </xacro:hokuyo_lx30_laser_v0>
     <!-- all four caster macros -->
-    <xacro:pr2_caster suffix="fl" parent="${name}_link" ref_position="${cal_caster_fl}" >
+    <xacro:pr2_caster_v0 suffix="fl" parent="${name}_link" ref_position="${cal_caster_fl}" >
       <origin xyz="${caster_offset_x} ${caster_offset_y} ${caster_offset_z}" rpy="0 0 0" />
-    </xacro:pr2_caster>
-    <xacro:pr2_caster suffix="fr" parent="${name}_link" ref_position="${cal_caster_fr}" >
+    </xacro:pr2_caster_v0>
+    <xacro:pr2_caster_v0 suffix="fr" parent="${name}_link" ref_position="${cal_caster_fr}" >
       <origin xyz="${caster_offset_x} ${-caster_offset_y} ${caster_offset_z}" rpy="0 0 0" />
-    </xacro:pr2_caster>
-    <xacro:pr2_caster suffix="bl" parent="${name}_link" ref_position="${cal_caster_bl}" >
+    </xacro:pr2_caster_v0>
+    <xacro:pr2_caster_v0 suffix="bl" parent="${name}_link" ref_position="${cal_caster_bl}" >
       <origin xyz="${-caster_offset_x} ${caster_offset_y} ${caster_offset_z}" rpy="0 0 0" />
-    </xacro:pr2_caster>
-    <xacro:pr2_caster suffix="br" parent="${name}_link" ref_position="${cal_caster_br}"  >
+    </xacro:pr2_caster_v0>
+    <xacro:pr2_caster_v0 suffix="br" parent="${name}_link" ref_position="${cal_caster_br}"  >
       <origin xyz="${-caster_offset_x} ${-caster_offset_y} ${caster_offset_z}" rpy="0 0 0" />
-    </xacro:pr2_caster>
+    </xacro:pr2_caster_v0>
     <!-- gazebo extensions -->
-    <xacro:pr2_base_gazebo name="${name}" />
+    <xacro:pr2_base_gazebo_v0 name="${name}" />
   </xacro:macro>
 </robot>

File: pr2_description/urdf/forearm_v0/forearm.gazebo.xacro (robot description, xacro)
@@ -4,5 +4,5 @@
        xmlns:interface="http://playerstage.sourceforge.net/gazebo/xmlschema/#interface"
        xmlns:xacro="http://ros.org/wiki/xacro">
-  <xacro:macro name="pr2_forearm_gazebo" params="side">
+  <xacro:macro name="pr2_forearm_gazebo_v0" params="side">
     <gazebo reference="${side}_forearm_link">
       <turnGravityOff>true</turnGravityOff>

File: pr2_description/urdf/forearm_v0/forearm.transmission.xacro (robot description, xacro)
@@ -4,5 +4,5 @@
        xmlns:interface="http://playerstage.sourceforge.net/gazebo/xmlschema/#interface"
        xmlns:xacro="http://ros.org/wiki/xacro">
-  <xacro:macro name="pr2_forearm_transmission" params="side">
+  <xacro:macro name="pr2_forearm_transmission_v0" params="side">
     <!-- Wrist flex , Wrist roll -->
     <transmission type="WristTransmission" name="${side}_wrist_trans">

File: pr2_description/urdf/forearm_v0/forearm.urdf.xacro (robot description, xacro)
@@ -11,5 +11,5 @@
   <include filename="$(find pr2_description)/urdf/common.xacro" />
   <!-- ============================   Forearm   ============================ -->
-  <xacro:macro name="pr2_forearm" params="side parent reflect">
+  <xacro:macro name="pr2_forearm_v0" params="side parent reflect">
     <joint name="${side}_forearm_joint" type="fixed">
       <origin xyz="0 0 0" rpy="0 0 0" />
@@ -108,6 +108,6 @@
     </link>
     <!-- extensions-->
-    <xacro:pr2_forearm_gazebo side="${side}" />
-    <xacro:pr2_forearm_transmission side="${side}" />
+    <xacro:pr2_forearm_gazebo_v0 side="${side}" />
+    <xacro:pr2_forearm_transmission_v0 side="${side}" />
   </xacro:macro>
 </robot>

File: pr2_description/urdf/gripper_v0/gripper.gazebo.xacro (robot description, xacro)
@@ -16,5 +16,5 @@
   <property name="finger_tip_mu"              value="500.0" />
   <property name="finger_mu"                  value="500.0" />
-  <xacro:macro name="pr2_finger_gazebo" params="prefix">
+  <xacro:macro name="pr2_finger_gazebo_v0" params="prefix">
     <!-- Finger proximal digit -->
     <gazebo reference="${prefix}_l_finger_link">
@@ -140,5 +140,5 @@
     </gazebo>
   </xacro:macro>
-  <xacro:macro name="pr2_gripper_gazebo" params="side">
+  <xacro:macro name="pr2_gripper_gazebo_v0" params="side">
     <gazebo reference="${side}_gripper_palm_link">
       <turnGravityOff>true</turnGravityOff>

File: pr2_description/urdf/gripper_v0/gripper.transmission.xacro (robot description, xacro)
@@ -5,5 +5,5 @@
        xmlns:interface="http://playerstage.sourceforge.net/gazebo/xmlschema/#interface"
        xmlns:xacro="http://ros.org/wiki/xacro">
-  <xacro:macro name="pr2_gripper_transmission" params="side screw_reduction gear_ratio theta0 phi0 t0 L0 h a b r">
+  <xacro:macro name="pr2_gripper_transmission_v0" params="side screw_reduction gear_ratio theta0 phi0 t0 L0 h a b r">
     <!-- [lr]_gripper_joint is a fictitious joint, used by transmission for controller gap   -->
     <!-- [lr]_gripper_joint is not attached to any link                                      -->

File: pr2_description/urdf/gripper_v0/gripper.urdf.xacro (robot description, xacro)
@@ -13,5 +13,5 @@
   <property name="finger_tip_damping"         value="0.01" />
   <property name="finger_joint_effort_limit"  value="100.0" />
-  <xacro:macro name="pr2_finger_limits" params="reflect">
+  <xacro:macro name="pr2_finger_limits_v0" params="reflect">
     <limit effort="${finger_joint_effort_limit}" velocity="0.5"
            lower="${gripper_lower_angle}" upper="${gripper_upper_angle}" />
@@ -19,9 +19,9 @@
                        soft_lower_limit="${gripper_lower_angle+0.0}" soft_upper_limit="${gripper_upper_angle-0.0}" />
   </xacro:macro>
-  <xacro:macro name="pr2_finger" params="prefix parent">
+  <xacro:macro name="pr2_finger_v0" params="prefix parent">
     <!-- Finger proximal digit -->
     <joint name="${prefix}_l_finger_joint" type="revolute">
       <axis xyz="0 0 1" />
-      <xacro:pr2_finger_limits reflect="1" />
+      <xacro:pr2_finger_limits_v0 reflect="1" />
       <dynamics damping="${finger_damping}" />
       <origin xyz="0.07691 0.01 0" rpy="0 0 0" />
@@ -59,5 +59,5 @@
       <axis xyz="0 0 -1" />
       <origin xyz="0.07691 -0.01 0" rpy="0 0 0" />
-      <xacro:pr2_finger_limits reflect="1" />
+      <xacro:pr2_finger_limits_v0 reflect="1" />
       <dynamics damping="${finger_damping}" />
       <mimic joint="${prefix}_l_finger_joint" multiplier="1" offset="0"/>
@@ -95,5 +95,5 @@
       <axis xyz="0 0 -1" />
       <origin xyz="0.09137 0.00495 0" rpy="0 0 0" />
-      <xacro:pr2_finger_limits reflect="1" />
+      <xacro:pr2_finger_limits_v0 reflect="1" />
       <dynamics damping="${finger_tip_damping}" />
       <mimic joint="${prefix}_l_finger_joint" multiplier="1" offset="0"/>
@@ -128,5 +128,5 @@
       <axis xyz="0 0 1" />
       <origin xyz="${0.09137} ${-0.00495} 0" rpy="0 0 0" />
-      <xacro:pr2_finger_limits reflect="1" />
+      <xacro:pr2_finger_limits_v0 reflect="1" />
       <dynamics damping="${finger_tip_damping}" />
       <mimic joint="${prefix}_l_finger_joint" multiplier="1" offset="0"/>
@@ -158,7 +158,7 @@
     </link>
     <!-- extensions -->
-    <xacro:pr2_finger_gazebo prefix="${prefix}" />
+    <xacro:pr2_finger_gazebo_v0 prefix="${prefix}" />
   </xacro:macro>
-  <xacro:macro name="pr2_gripper" params="side parent *origin gear_ratio screw_reduction theta0 phi0 t0 L0 h a b r">
+  <xacro:macro name="pr2_gripper_v0" params="side parent *origin gear_ratio screw_reduction theta0 phi0 t0 L0 h a b r">
     <joint name="${side}_gripper_palm_joint" type="fixed">
       <insert_block name="origin"/>
@@ -275,5 +275,5 @@
     </link>
     <!-- pr2 fingers macro -->
-    <pr2_finger prefix="${side}_gripper" parent="${side}_gripper_palm_link" />
+    <xacro:pr2_finger_v0 prefix="${side}_gripper" parent="${side}_gripper_palm_link" />
     <!-- fictitous joint that represents the gripper gap -->
     <!-- effort is the linear force at the gripper gap
@@ -287,6 +287,6 @@
     </joint>
     <!-- extensions -->
-    <xacro:pr2_gripper_gazebo side="${side}" />
-    <xacro:pr2_gripper_transmission side="${side}"
+    <xacro:pr2_gripper_gazebo_v0 side="${side}" />
+    <xacro:pr2_gripper_transmission_v0 side="${side}"
         screw_reduction="${screw_reduction}"
         gear_ratio="${gear_ratio}"

File: pr2_description/urdf/head_v0/head.gazebo.xacro (robot description, xacro)
@@ -4,15 +4,15 @@
        xmlns:interface="http://playerstage.sourceforge.net/gazebo/xmlschema/#interface"
        xmlns:xacro="http://ros.org/wiki/xacro">
-  <xacro:macro name="pr2_head_pan_gazebo" params="name">
+  <xacro:macro name="pr2_head_pan_gazebo_v0" params="name">
     <gazebo reference="${name}_link">
       <material value="PR2/Blue" />
     </gazebo>
   </xacro:macro>
-  <xacro:macro name="pr2_head_tilt_gazebo" params="name">
+  <xacro:macro name="pr2_head_tilt_gazebo_v0" params="name">
     <gazebo reference="${name}_link">
       <material value="PR2/Green" />
     </gazebo>
   </xacro:macro>
-  <xacro:macro name="pr2_head_gazebo" params="name">
+  <xacro:macro name="pr2_head_gazebo_v0" params="name">
     <gazebo reference="${name}_plate_frame">
       <material value="PR2/Blue" />

File: pr2_description/urdf/head_v0/head.transmission.xacro (robot description, xacro)
@@ -4,5 +4,5 @@
        xmlns:interface="http://playerstage.sourceforge.net/gazebo/xmlschema/#interface"
        xmlns:xacro="http://ros.org/wiki/xacro">
-  <xacro:macro name="pr2_head_pan_transmission" params="name">
+  <xacro:macro name="pr2_head_pan_transmission_v0" params="name">
     <transmission type="SimpleTransmission" name="${name}_trans">
       <actuator name="${name}_motor" />
@@ -11,5 +11,5 @@
     </transmission>
   </xacro:macro>
-  <xacro:macro name="pr2_head_tilt_transmission" params="name">
+  <xacro:macro name="pr2_head_tilt_transmission_v0" params="name">
     <transmission type="SimpleTransmission" name="${name}_trans">
       <actuator name="${name}_motor" />

File: pr2_description/urdf/head_v0/head.urdf.xacro (robot description, xacro)
@@ -7,5 +7,5 @@
   <include filename="$(find pr2_description)/urdf/head_v0/head.transmission.xacro" />
   <property name="M_PI" value="3.1415926535897931" />
-  <xacro:macro name="pr2_head_pan" params="name parent *origin">
+  <xacro:macro name="pr2_head_pan_v0" params="name parent *origin">
     <joint name="${name}_joint" type="revolute">
       <axis xyz="0 0 1" />
@@ -40,8 +40,8 @@
     </link>
     <!-- extensions -->
-    <xacro:pr2_head_pan_gazebo name="${name}" />
-    <xacro:pr2_head_pan_transmission name="${name}" />
+    <xacro:pr2_head_pan_gazebo_v0 name="${name}" />
+    <xacro:pr2_head_pan_transmission_v0 name="${name}" />
   </xacro:macro>
-  <xacro:macro name="pr2_head_tilt" params="name parent *origin">
+  <xacro:macro name="pr2_head_tilt_v0" params="name parent *origin">
     <joint name="${name}_joint" type="revolute">
       <axis xyz="0 1 0" />
@@ -77,14 +77,14 @@
     </link>
     <!-- extensions -->
-    <xacro:pr2_head_tilt_gazebo name="${name}" />
-    <xacro:pr2_head_tilt_transmission name="${name}" />
+    <xacro:pr2_head_tilt_gazebo_v0 name="${name}" />
+    <xacro:pr2_head_tilt_transmission_v0 name="${name}" />
   </xacro:macro>
-  <xacro:macro name="pr2_head" params="name parent *origin">
-    <xacro:pr2_head_pan name="${name}_pan" parent="${parent}">
+  <xacro:macro name="pr2_head_v0" params="name parent *origin">
+    <xacro:pr2_head_pan_v0 name="${name}_pan" parent="${parent}">
       <insert_block name="origin" />
-    </xacro:pr2_head_pan>
-    <xacro:pr2_head_tilt name="${name}_tilt" parent="${name}_pan_link">
+    </xacro:pr2_head_pan_v0>
+    <xacro:pr2_head_tilt_v0 name="${name}_tilt" parent="${name}_pan_link">
       <origin xyz="0.058 0 0" rpy="0 0 0" />
-    </xacro:pr2_head_tilt>
+    </xacro:pr2_head_tilt_v0>
     <!-- Head plate frame -->
     <joint name="${name}_plate_frame_joint" type="fixed">
@@ -116,5 +116,5 @@
     </link>
     <!-- extensions -->
-    <xacro:pr2_head_gazebo name="${name}" />
+    <xacro:pr2_head_gazebo_v0 name="${name}" />
   </xacro:macro>
 </robot>

File: pr2_description/urdf/sensors/double_stereo_camera.gazebo.xacro (robot description, xacro)
@@ -6,5 +6,5 @@
   <!-- Made by Kevin for double stereo camera for PR-2 Beta. -->
   <!-- Needs calibration verification, and CAD check. -->
-  <xacro:macro name="double_stereo_camera_gazebo" params="name">
+  <xacro:macro name="double_stereo_camera_gazebo_v0" params="name">
     <!-- Define link to stereo cameras, set origin relative to that -->
     <gazebo reference="${name}_double_stereo_link">

File: pr2_description/urdf/sensors/double_stereo_camera.urdf.xacro (robot description, xacro)
@@ -8,5 +8,5 @@
   <!-- Made by Kevin for double stereo camera for PR-2 Beta. -->
   <!-- Needs calibration verification, and CAD check. -->
-  <macro name="double_stereo_camera" params="name parent *origin">
+  <xacro:macro name="double_stereo_camera_v0" params="name parent *origin">
     <!-- Define link to stereo cameras, set origin relative to that -->
     <joint name="${name}_frame_joint" type="fixed">
@@ -40,12 +40,12 @@
     <!-- Wide camera is on robot right (hca1), narrow on left (hca2)? -->
     <!-- 15mm offset from center needs check with CAD -->
-    <xacro:stereo_camera parent="${name}_link" name="wide_stereo" focal_length="320" hfov="90" >
+    <xacro:stereo_camera_v0 parent="${name}_link" name="wide_stereo" focal_length="320" hfov="90" >
       <origin xyz="0 -0.015 0" rpy="0 0 0" />
-    </xacro:stereo_camera>
-    <xacro:stereo_camera parent="${name}_link" name="narrow_stereo" focal_length="772.55" hfov="45" >
+    </xacro:stereo_camera_v0>
+    <xacro:stereo_camera_v0 parent="${name}_link" name="narrow_stereo" focal_length="772.55" hfov="45" >
       <origin xyz="0 0.015 0" rpy="0 0 0" />
-    </xacro:stereo_camera>
+    </xacro:stereo_camera_v0>
     <!-- extensions -->
-    <xacro:double_stereo_camera_gazebo name="${name}" />
-  </macro>
+    <xacro:double_stereo_camera_gazebo_v0 name="${name}" />
+  </xacro:macro>
 </robot>
