Commit message: * adding _v0 suffix to all macros.  * reuse wge100_camera macros for stereo camera.

File: pr2_description/urdf/sensors/head_sensor_package.gazebo.xacro (robot description, xacro)
@@ -8,8 +8,8 @@
   <!-- Origin is center mount screw on sensor plate mount -->
   <!-- When mounted properly, should have same origin as head plate frame -->
-  <macro name="pr2_head_sensor_package_gazebo" params="name">
+  <xacro:macro name="pr2_head_sensor_package_gazebo_v0" params="name">
     <gazebo reference="${name}_sensor_link">
       <material value="PR2/Blue" />
     </gazebo>
-  </macro>
+  </xacro:macro>
 </robot>

File: pr2_description/urdf/sensors/head_sensor_package.urdf.xacro (robot description, xacro)
@@ -14,5 +14,5 @@
   <!-- Origin is center mount screw on sensor plate mount -->
   <!-- When mounted properly, should have same origin as head plate frame -->
-  <xacro:macro name="pr2_head_sensor_package" params="name hd_name stereo_name parent *origin">
+  <xacro:macro name="pr2_head_sensor_package_v0" params="name hd_name stereo_name parent *origin">
     <joint name="${name}_frame_joint" type="fixed">
       <insert_block name="origin" />
@@ -44,15 +44,15 @@
     </link>
     <!-- Prosilica Camera -->
-    <xacro:prosilica_cam name="${hd_name}" parent="${name}_link" >
+    <xacro:prosilica_cam_v0 name="${hd_name}" parent="${name}_link" >
       <!-- Center of camera is 109mm right of center screw, 35mm up -->
       <!-- Camera is slightly recessed from front, where is camera origin? Lens? -->
       <origin xyz="0 -0.109 0.035" rpy="0 0 0" />
-    </xacro:prosilica_cam>
+    </xacro:prosilica_cam_v0>
     <!-- construct wide and narrow double stereo camera -->
-    <xacro:double_stereo_camera name="${stereo_name}" parent="${name}_link" >
+    <xacro:double_stereo_camera_v0 name="${stereo_name}" parent="${name}_link" >
       <origin xyz="0.0 0.0 0.003" rpy="0 0 0" />
-    </xacro:double_stereo_camera>
+    </xacro:double_stereo_camera_v0>
     <!-- extensions -->
-    <xacro:pr2_head_sensor_package_gazebo name="${name}" />
+    <xacro:pr2_head_sensor_package_gazebo_v0 name="${name}" />
   </xacro:macro>
 </robot>

File: pr2_description/urdf/sensors/hokuyo_lx30_laser.gazebo.xacro (robot description, xacro)
@@ -4,5 +4,5 @@
        xmlns:interface="http://playerstage.sourceforge.net/gazebo/xmlschema/#interface"
        xmlns:xacro="http://ros.org/wiki/xacro">
-  <xacro:macro name="hokuyo_lx30_laser_gazebo" params="name ros_topic">
+  <xacro:macro name="hokuyo_lx30_laser_gazebo_v0" params="name ros_topic">
     <gazebo reference="${name}_link">
       <sensor:ray name="${name}">

File: pr2_description/urdf/sensors/hokuyo_lx30_laser.urdf.xacro (robot description, xacro)
@@ -5,5 +5,5 @@
        xmlns:xacro="http://ros.org/wiki/xacro">
   <include filename="$(find pr2_description)/urdf/sensors/hokuyo_lx30_laser.gazebo.xacro" />
-  <xacro:macro name="hokuyo_lx30_laser" params="name parent *origin ros_topic">
+  <xacro:macro name="hokuyo_lx30_laser_v0" params="name parent *origin ros_topic">
     <joint name="${name}_joint" type="fixed">
       <axis xyz="0 1 0" />
@@ -33,5 +33,5 @@
     </link>
     <!-- gazebo extensions -->
-    <xacro:hokuyo_lx30_laser_gazebo name="${name}" ros_topic="${ros_topic}" />
+    <xacro:hokuyo_lx30_laser_gazebo_v0 name="${name}" ros_topic="${ros_topic}" />
   </xacro:macro>
 </robot>

File: pr2_description/urdf/sensors/prosilica_gc2450_camera.gazebo.xacro (robot description, xacro)
@@ -4,5 +4,5 @@
       xmlns:interface="http://playerstage.sourceforge.net/gazebo/xmlschema/#interface"
       xmlns:xacro="http://ros.org/wiki/xacro">
-<xacro:macro name="prosilica_cam_gazebo" params="name">
+<xacro:macro name="prosilica_cam_gazebo_v0" params="name">
   <gazebo reference="${name}_frame">
     <sensor:camera name="${name}_sensor">

Commit message: Fixes to URDF files for qualification

File: pr2_description/robots/pr2.urdf.xacro (robot description, xacro)
@@ -8,5 +8,5 @@
   <!-- misc common stuff? -->
   <include filename="$(find pr2_description)/urdf/common.xacro" />
-  <!-- PR2 gripper -->
+  <!-- PR2 Arm -->
   <include filename="$(find pr2_description)/urdf/shoulder_v0/shoulder.urdf.xacro" />
   <include filename="$(find pr2_description)/urdf/upper_arm_v0/upper_arm.urdf.xacro" />
@@ -45,5 +45,5 @@
   </xacro:pr2_torso_v0>
   <!-- The xacro preprocesser will replace the parameters below, such as ${cal_head_x}, with
-       numerical values that were specified in default_cal.xml which was included above -->
+       numerical values that were specified in common.xacro which was included above -->
   <xacro:pr2_head_v0 name="head" parent="torso_lift_link">
     <origin xyz="${cal_head_x}    ${cal_head_y}     ${0.3915+cal_head_z}"

File: pr2_description/urdf/base_v0/base.transmission.xacro (robot description, xacro)
@@ -7,5 +7,5 @@
   <!-- Alpha 2.0 hardware                                   -->
   <!--                                                      -->
-  <xacro:macro name="pr2_wheel_transmission" params="suffix parent reflect">
+  <xacro:macro name="pr2_wheel_transmission_v0" params="suffix parent reflect">
     <transmission type="SimpleTransmission" name="${parent}_${suffix}_wheel_trans">
       <actuator name="${parent}_${suffix}_wheel_motor" />
@@ -14,5 +14,5 @@
     </transmission>
   </xacro:macro>
-  <xacro:macro name="pr2_caster_transmission" params="suffix">
+  <xacro:macro name="pr2_caster_transmission_v0" params="suffix">
     <transmission type="SimpleTransmission" name="${suffix}_caster_rotation_trans">
       <actuator name="${suffix}_caster_rotation_motor" />

Commit message: * update ros_camera topic name from left_image/right_image to left/image_raw and right/image_raw  * add information of projection matrix for gazebo camera extensions

File: pr2_description/robots/pr2.urdf.xacro (robot description, xacro)
@@ -98,9 +98,11 @@
   <!-- Forearm Cam (Hand approximated values) -->
   <xacro:wge100_camera_v0 name="l_forearm_cam" topic_name="l_forearm_cam/image"
-                          parent="l_forearm_roll_link" hfov="90" focal_length="320">
+                          parent="l_forearm_roll_link" hfov="90" focal_length="320"
+                          image_width="640" image_height="480">
     <origin xyz=".15 0 .07" rpy="${ M_PI/2} ${-45*M_PI/180} 0" />
   </xacro:wge100_camera_v0>
   <xacro:wge100_camera_v0 name="r_forearm_cam" topic_name="r_forearm_cam/image"
-                          parent="r_forearm_roll_link" hfov="90" focal_length="320">
+                          parent="r_forearm_roll_link" hfov="90" focal_length="320"
+                          image_width="640" image_height="480">
     <origin xyz=".15 0 .07" rpy="${-M_PI/2} ${-45*M_PI/180} 0" />
   </xacro:wge100_camera_v0>

File: pr2_description/urdf/sensors/double_stereo_camera.urdf.xacro (robot description, xacro)
@@ -40,8 +40,8 @@
     <!-- Wide camera is on robot right (hca1), narrow on left (hca2)? -->
     <!-- 15mm offset from center needs check with CAD -->
-    <xacro:stereo_camera_v0 parent="${name}_link" name="wide_stereo" focal_length="320" hfov="90" >
+    <xacro:stereo_camera_v0 parent="${name}_link" name="wide_stereo" focal_length="320" hfov="90" image_width="640" image_height="480" >
       <origin xyz="0 -0.015 0" rpy="0 0 0" />
     </xacro:stereo_camera_v0>
-    <xacro:stereo_camera_v0 parent="${name}_link" name="narrow_stereo" focal_length="772.55" hfov="45" >
+    <xacro:stereo_camera_v0 parent="${name}_link" name="narrow_stereo" focal_length="772.55" hfov="45" image_width="640" image_height="480" >
       <origin xyz="0 0.015 0" rpy="0 0 0" />
     </xacro:stereo_camera_v0>

File: pr2_description/urdf/sensors/stereo_camera.gazebo.xacro (robot description, xacro)
@@ -5,5 +5,5 @@
        xmlns:xacro="http://ros.org/wiki/xacro">
   <!-- this macro is used for creating wide and narrow double stereo camera in simulation -->
-  <xacro:macro name="stereo_camera_gazebo_v0" params="name focal_length hfov">
+  <xacro:macro name="stereo_camera_gazebo_v0" params="name focal_length hfov image_width image_height">
     <gazebo reference="${name}_link">
       <material value="PR2/Blue" />
@@ -21,7 +21,7 @@
         <topicName>${name}/raw_stereo</topicName>
         <frameName>${name}_optical_frame</frameName>
-        <CxPrime>320</CxPrime>
-        <Cx>320</Cx>
-        <Cy>240</Cy>
+        <CxPrime>${(image_width+1)/2}</CxPrime>
+        <Cx>${(image_width+1)/2}</Cx>
+        <Cy>${(image_height+1)/2}</Cy>
         <!-- image_width / (2*tan(hfov_radian /2)) -->
         <!-- 320 for wide and 772.55 for narrow stereo camera -->

File: pr2_description/urdf/sensors/stereo_camera.urdf.xacro (robot description, xacro)
@@ -19,5 +19,5 @@
   <property name="stereo_rz" value="0.00" />
   <!-- this macro is used for creating wide and narrow double stereo camera links -->
-  <xacro:macro name="stereo_camera_v0" params="name parent focal_length hfov *origin">
+  <xacro:macro name="stereo_camera_v0" params="name parent focal_length hfov image_width image_height *origin">
     <joint name="${name}_frame_joint" type="fixed">
       <insert_block name="origin" />
@@ -74,17 +74,20 @@
     </link>
     <!-- stereo left camera -->
-    <xacro:wge100_camera_v0 name="${name}_l_stereo_camera" topic_name="${name}/left_image"
+    <xacro:wge100_camera_v0 name="${name}_l_stereo_camera" topic_name="${name}/left/image_raw"
                             parent="${name}_optical_frame"
-                            hfov="${hfov}" focal_length="${focal_length}">
+                            hfov="${hfov}" focal_length="${focal_length}"
+                            image_width="${image_width}" image_height="${image_height}">
       <origin xyz="0 0 0" rpy="0 ${-M_PI/2} ${M_PI/2}" />
     </xacro:wge100_camera_v0>
     <!-- stereo right camera -->
-    <xacro:wge100_camera_v0 name="${name}_r_stereo_camera" topic_name="${name}/right_image"
+    <xacro:wge100_camera_v0 name="${name}_r_stereo_camera" topic_name="${name}/right/image_raw"
                             parent="${name}_l_stereo_camera_frame"
-                            hfov="${hfov}" focal_length="${focal_length}">
+                            hfov="${hfov}" focal_length="${focal_length}"
+                            image_width="${image_width}" image_height="${image_height}">
       <origin xyz="${stereo_dx} ${stereo_dy} ${stereo_dz}" rpy="${stereo_rx} ${stereo_ry} ${stereo_rz}" />
     </xacro:wge100_camera_v0>
     <!-- extensions -->
-    <xacro:stereo_camera_gazebo_v0 name="${name}" focal_length="${focal_length}" hfov="${hfov}" />
+    <xacro:stereo_camera_gazebo_v0 name="${name}" focal_length="${focal_length}" hfov="${hfov}"
+                                   image_width="${image_width}" image_height="${image_height}"/>
   </xacro:macro>
 </robot>

File: pr2_description/urdf/sensors/wge100_camera.gazebo.xacro (robot description, xacro)
@@ -4,10 +4,8 @@
        xmlns:interface="http://playerstage.sourceforge.net/gazebo/xmlschema/#interface"
        xmlns:xacro="http://ros.org/wiki/xacro">
-  <xacro:macro name="wge100_camera_gazebo_v0" params="name topic_name hfov focal_length">
-    <!-- focal_length is not used at the moment, but will be needed for projection matrix
-         if we are to generate a camera projection matrix for CameraInfo message. -->
+  <xacro:macro name="wge100_camera_gazebo_v0" params="name topic_name hfov focal_length image_width image_height">
     <gazebo reference="${name}_frame">
       <sensor:camera name="${name}_sensor">
-        <imageSize>640 480</imageSize>
+        <imageSize>${image_width} ${image_height}</imageSize>
         <imageFormat>L8</imageFormat>
         <hfov>${hfov}</hfov>
@@ -20,4 +18,15 @@
           <topicName>${topic_name}</topicName>
           <frameName>${name}_frame</frameName>
+          <CxPrime>${(image_width+1)/2}</CxPrime>
+          <Cx>${(image_width+1)/2}</Cx>
+          <Cy>${(image_height+1)/2}</Cy>
+          <!-- image_width / (2*tan(hfov_radian /2)) -->
+          <!-- 320 for wide and 772.55 for narrow stereo camera -->
+          <focal_length>${focal_length}</focal_length>
+          <distortion_k1>0</distortion_k1>
+          <distortion_k2>0</distortion_k2>
+          <distortion_k3>0</distortion_k3>
+          <distortion_t1>0</distortion_t1>
+          <distortion_t2>0</distortion_t2>
           <interface:camera name="${name}_iface" />
         </controller:ros_camera>

File: pr2_description/urdf/sensors/wge100_camera.urdf.xacro (robot description, xacro)
@@ -6,5 +6,5 @@
        xmlns:xacro="http://ros.org/wiki/xacro">
   <include filename="$(find pr2_description)/urdf/sensors/wge100_camera.gazebo.xacro" />
-  <xacro:macro name="wge100_camera_v0" params="name topic_name parent hfov focal_length *origin">
+  <xacro:macro name="wge100_camera_v0" params="name topic_name parent hfov focal_length image_width image_height *origin">
     <joint name="${name}_frame_joint" type="fixed">
       <insert_block name="origin" />
@@ -61,5 +61,6 @@
     <!-- extensions -->
     <xacro:wge100_camera_gazebo_v0 name="${name}" topic_name="${topic_name}"
-                                   hfov="${hfov}" focal_length="${focal_length}"/>
+                                   hfov="${hfov}" focal_length="${focal_length}"
+                                   image_width="${image_width}" image_height="${image_height}"/>
   </xacro:macro>
 </robot>

Commit message: pr2_description urdf updates:  * tilt laser at 40Hz, base laser at 20Hz  * camera image topics --> image_raw

File: pr2_description/robots/pr2.urdf.xacro (robot description, xacro)
@@ -97,10 +97,12 @@
   </xacro:pr2_gripper_v0>
   <!-- Forearm Cam (Hand approximated values) -->
-  <xacro:wge100_camera_v0 name="l_forearm_cam" topic_name="l_forearm_cam/image"
+  <xacro:wge100_camera_v0 name="l_forearm_cam" image_topic_name="l_forearm_cam/image_raw"
+                          camera_info_topic_name="l_forearm_cam/camera_info"
                           parent="l_forearm_roll_link" hfov="90" focal_length="320"
                           image_width="640" image_height="480">
     <origin xyz=".15 0 .07" rpy="${ M_PI/2} ${-45*M_PI/180} 0" />
   </xacro:wge100_camera_v0>
-  <xacro:wge100_camera_v0 name="r_forearm_cam" topic_name="r_forearm_cam/image"
+  <xacro:wge100_camera_v0 name="r_forearm_cam" image_topic_name="r_forearm_cam/image_raw"
+                          camera_info_topic_name="r_forearm_cam/camera_info"
                           parent="r_forearm_roll_link" hfov="90" focal_length="320"
                           image_width="640" image_height="480">

File: pr2_description/urdf/base_v0/base.urdf.xacro (robot description, xacro)
@@ -141,5 +141,5 @@
     </link>
     <!-- base laser -->
-    <xacro:hokuyo_lx30_laser_v0 name="${name}_laser" parent="${name}" ros_topic="base_scan" >
+    <xacro:hokuyo_lx30_laser_v0 name="${name}_laser" parent="${name}" ros_topic="base_scan" update_rate="20" >
       <origin xyz="${base_laser_x} ${base_laser_y} ${base_laser_z}" rpy="0 0 0" />
     </xacro:hokuyo_lx30_laser_v0>

File: pr2_description/urdf/sensors/hokuyo_lx30_laser.gazebo.xacro (robot description, xacro)
@@ -4,5 +4,5 @@
        xmlns:interface="http://playerstage.sourceforge.net/gazebo/xmlschema/#interface"
        xmlns:xacro="http://ros.org/wiki/xacro">
-  <xacro:macro name="hokuyo_lx30_laser_gazebo_v0" params="name ros_topic">
+  <xacro:macro name="hokuyo_lx30_laser_gazebo_v0" params="name ros_topic update_rate">
     <gazebo reference="${name}_link">
       <sensor:ray name="${name}">
@@ -17,5 +17,5 @@
         <maxRange>10.0</maxRange>
         <resRange>0.01</resRange>
-        <updateRate>40.0</updateRate>
+        <updateRate>${update_rate}</updateRate>
         <controller:ros_laser name="ros_${name}_controller" plugin="libros_laser.so">
           <gaussianNoise>0.005</gaussianNoise>

File: pr2_description/urdf/sensors/hokuyo_lx30_laser.urdf.xacro (robot description, xacro)
@@ -5,5 +5,5 @@
        xmlns:xacro="http://ros.org/wiki/xacro">
   <include filename="$(find pr2_description)/urdf/sensors/hokuyo_lx30_laser.gazebo.xacro" />
-  <xacro:macro name="hokuyo_lx30_laser_v0" params="name parent *origin ros_topic">
+  <xacro:macro name="hokuyo_lx30_laser_v0" params="name parent *origin ros_topic update_rate">
     <joint name="${name}_joint" type="fixed">
       <axis xyz="0 1 0" />
@@ -33,5 +33,5 @@
     </link>
     <!-- gazebo extensions -->
-    <xacro:hokuyo_lx30_laser_gazebo_v0 name="${name}" ros_topic="${ros_topic}" />
+    <xacro:hokuyo_lx30_laser_gazebo_v0 name="${name}" ros_topic="${ros_topic}" update_rate="${update_rate}" />
   </xacro:macro>
 </robot>

File: pr2_description/urdf/sensors/stereo_camera.urdf.xacro (robot description, xacro)
@@ -74,6 +74,6 @@
     </link>
     <!-- stereo left camera -->
-    <xacro:wge100_camera_v0 name="${name}_l_stereo_camera" topic_name="${name}/left/image_raw"
-                            parent="${name}_optical_frame"
+    <xacro:wge100_camera_v0 name="${name}_l_stereo_camera" image_topic_name="${name}/left/image_raw"
+                            camera_info_topic_name="${name}/right/camera_info" parent="${name}_optical_frame"
                             hfov="${hfov}" focal_length="${focal_length}"
                             image_width="${image_width}" image_height="${image_height}">
@@ -81,6 +81,6 @@
     </xacro:wge100_camera_v0>
     <!-- stereo right camera -->
-    <xacro:wge100_camera_v0 name="${name}_r_stereo_camera" topic_name="${name}/right/image_raw"
-                            parent="${name}_l_stereo_camera_frame"
+    <xacro:wge100_camera_v0 name="${name}_r_stereo_camera" image_topic_name="${name}/right/image_raw"
+                            camera_info_topic_name="${name}/right/camera_info" parent="${name}_l_stereo_camera_frame"
                             hfov="${hfov}" focal_length="${focal_length}"
                             image_width="${image_width}" image_height="${image_height}">

File: pr2_description/urdf/sensors/wge100_camera.gazebo.xacro (robot description, xacro)
@@ -4,5 +4,5 @@
        xmlns:interface="http://playerstage.sourceforge.net/gazebo/xmlschema/#interface"
        xmlns:xacro="http://ros.org/wiki/xacro">
-  <xacro:macro name="wge100_camera_gazebo_v0" params="name topic_name hfov focal_length image_width image_height">
+  <xacro:macro name="wge100_camera_gazebo_v0" params="name image_topic_name camera_info_topic_name hfov focal_length image_width image_height">
     <gazebo reference="${name}_frame">
       <sensor:camera name="${name}_sensor">
@@ -16,5 +16,6 @@
           <alwaysOn>true</alwaysOn>
           <updateRate>20.0</updateRate>
-          <topicName>${topic_name}</topicName>
+          <imageTopicName>${image_topic_name}</imageTopicName>
+          <cameraInfoTopicName>${camera_info_topic_name}</cameraInfoTopicName>
           <frameName>${name}_frame</frameName>
           <CxPrime>${(image_width+1)/2}</CxPrime>

File: pr2_description/urdf/sensors/wge100_camera.urdf.xacro (robot description, xacro)
@@ -6,5 +6,5 @@
        xmlns:xacro="http://ros.org/wiki/xacro">
   <include filename="$(find pr2_description)/urdf/sensors/wge100_camera.gazebo.xacro" />
-  <xacro:macro name="wge100_camera_v0" params="name topic_name parent hfov focal_length image_width image_height *origin">
+  <xacro:macro name="wge100_camera_v0" params="name image_topic_name camera_info_topic_name parent hfov focal_length image_width image_height *origin">
     <joint name="${name}_frame_joint" type="fixed">
       <insert_block name="origin" />
@@ -60,5 +60,6 @@
     </link>
     <!-- extensions -->
-    <xacro:wge100_camera_gazebo_v0 name="${name}" topic_name="${topic_name}"
+    <xacro:wge100_camera_gazebo_v0 name="${name}" image_topic_name="${image_topic_name}"
+                                   camera_info_topic_name="${camera_info_topic_name}"
                                    hfov="${hfov}" focal_length="${focal_length}"
                                    image_width="${image_width}" image_height="${image_height}"/>

File: pr2_description/urdf/tilting_laser_v0/tilting_laser.urdf.xacro (robot description, xacro)
@@ -40,5 +40,5 @@
       </collision>
     </link>
-    <xacro:hokuyo_lx30_laser_v0 name="${name}" parent="${name}_mount" ros_topic="tilt_scan">
+    <xacro:hokuyo_lx30_laser_v0 name="${name}" parent="${name}_mount" ros_topic="tilt_scan" update_rate="40" >
       <origin xyz="0 0 0.03" rpy="0 0 0" />
     </xacro:hokuyo_lx30_laser_v0>
