Commit message: * create image_format parameter for wge100_camera.  * make wge100_cameras 25hz

File: pr2_description/robots/pr2.urdf.xacro (robot description, xacro)
@@ -97,5 +97,5 @@
   </xacro:pr2_gripper_v0>
   <!-- Forearm Cam (Hand approximated values) -->
-  <xacro:wge100_camera_v0 name="l_forearm_cam" image_topic_name="l_forearm_cam/image_raw"
+  <xacro:wge100_camera_v0 name="l_forearm_cam" image_format="L8" image_topic_name="l_forearm_cam/image_raw"
                           camera_info_topic_name="l_forearm_cam/camera_info"
                           parent="l_forearm_roll_link" hfov="90" focal_length="320"
@@ -103,5 +103,5 @@
     <origin xyz=".15 0 .07" rpy="${ M_PI/2} ${-45*M_PI/180} 0" />
   </xacro:wge100_camera_v0>
-  <xacro:wge100_camera_v0 name="r_forearm_cam" image_topic_name="r_forearm_cam/image_raw"
+  <xacro:wge100_camera_v0 name="r_forearm_cam" image_format="L8" image_topic_name="r_forearm_cam/image_raw"
                           camera_info_topic_name="r_forearm_cam/camera_info"
                           parent="r_forearm_roll_link" hfov="90" focal_length="320"

File: pr2_description/urdf/sensors/double_stereo_camera.urdf.xacro (robot description, xacro)
@@ -40,8 +40,8 @@
     <!-- Wide camera is on robot right (hca1), narrow on left (hca2)? -->
     <!-- 15mm offset from center needs check with CAD -->
-    <xacro:stereo_camera_v0 parent="${name}_link" name="wide_stereo" focal_length="320" hfov="90" image_width="640" image_height="480" >
+    <xacro:stereo_camera_v0 parent="${name}_link" name="wide_stereo" focal_length="320" hfov="90" image_format="B8G8R8" image_width="640" image_height="480" >
       <origin xyz="0 -0.015 0" rpy="0 0 0" />
     </xacro:stereo_camera_v0>
-    <xacro:stereo_camera_v0 parent="${name}_link" name="narrow_stereo" focal_length="772.55" hfov="45" image_width="640" image_height="480" >
+    <xacro:stereo_camera_v0 parent="${name}_link" name="narrow_stereo" focal_length="772.55" hfov="45" image_format="L8" image_width="640" image_height="480" >
       <origin xyz="0 0.015 0" rpy="0 0 0" />
     </xacro:stereo_camera_v0>

File: pr2_description/urdf/sensors/stereo_camera.urdf.xacro (robot description, xacro)
@@ -19,5 +19,5 @@
   <property name="stereo_rz" value="0.00" />
   <!-- this macro is used for creating wide and narrow double stereo camera links -->
-  <xacro:macro name="stereo_camera_v0" params="name parent focal_length hfov image_width image_height *origin">
+  <xacro:macro name="stereo_camera_v0" params="name parent focal_length hfov image_format image_width image_height *origin">
     <joint name="${name}_frame_joint" type="fixed">
       <insert_block name="origin" />
@@ -74,5 +74,5 @@
     </link>
     <!-- stereo left camera -->
-    <xacro:wge100_camera_v0 name="${name}_l_stereo_camera" image_topic_name="${name}/left/image_raw"
+    <xacro:wge100_camera_v0 name="${name}_l_stereo_camera" image_format="${image_format}" image_topic_name="${name}/left/image_raw"
                             camera_info_topic_name="${name}/left/camera_info" parent="${name}_optical_frame"
                             hfov="${hfov}" focal_length="${focal_length}"
@@ -81,5 +81,5 @@
     </xacro:wge100_camera_v0>
     <!-- stereo right camera -->
-    <xacro:wge100_camera_v0 name="${name}_r_stereo_camera" image_topic_name="${name}/right/image_raw"
+    <xacro:wge100_camera_v0 name="${name}_r_stereo_camera" image_format="${image_format}" image_topic_name="${name}/right/image_raw"
                             camera_info_topic_name="${name}/right/camera_info" parent="${name}_l_stereo_camera_frame"
                             hfov="${hfov}" focal_length="${focal_length}"

File: pr2_description/urdf/sensors/wge100_camera.gazebo.xacro (robot description, xacro)
@@ -4,9 +4,9 @@
        xmlns:interface="http://playerstage.sourceforge.net/gazebo/xmlschema/#interface"
        xmlns:xacro="http://ros.org/wiki/xacro">
-  <xacro:macro name="wge100_camera_gazebo_v0" params="name image_topic_name camera_info_topic_name hfov focal_length image_width image_height">
+  <xacro:macro name="wge100_camera_gazebo_v0" params="name image_format image_topic_name camera_info_topic_name hfov focal_length image_width image_height">
     <gazebo reference="${name}_frame">
       <sensor:camera name="${name}_sensor">
         <imageSize>${image_width} ${image_height}</imageSize>
-        <imageFormat>L8</imageFormat>
+        <imageFormat>${image_format}</imageFormat>
         <hfov>${hfov}</hfov>
         <nearClip>0.1</nearClip>
@@ -15,5 +15,5 @@
         <controller:ros_camera name="${name}_controller" plugin="libros_camera.so">
           <alwaysOn>true</alwaysOn>
-          <updateRate>20.0</updateRate>
+          <updateRate>25.0</updateRate>
           <imageTopicName>${image_topic_name}</imageTopicName>
           <cameraInfoTopicName>${camera_info_topic_name}</cameraInfoTopicName>

File: pr2_description/urdf/sensors/wge100_camera.urdf.xacro (robot description, xacro)
@@ -6,5 +6,5 @@
        xmlns:xacro="http://ros.org/wiki/xacro">
   <include filename="$(find pr2_description)/urdf/sensors/wge100_camera.gazebo.xacro" />
-  <xacro:macro name="wge100_camera_v0" params="name image_topic_name camera_info_topic_name parent hfov focal_length image_width image_height *origin">
+  <xacro:macro name="wge100_camera_v0" params="name image_format image_topic_name camera_info_topic_name parent hfov focal_length image_width image_height *origin">
     <joint name="${name}_frame_joint" type="fixed">
       <insert_block name="origin" />
@@ -60,5 +60,5 @@
     </link>
     <!-- extensions -->
-    <xacro:wge100_camera_gazebo_v0 name="${name}" image_topic_name="${image_topic_name}"
+    <xacro:wge100_camera_gazebo_v0 name="${name}" image_format="${image_format}" image_topic_name="${image_topic_name}"
                                    camera_info_topic_name="${camera_info_topic_name}"
                                    hfov="${hfov}" focal_length="${focal_length}"

Commit message: adding changes needed to specify stereo camera in sim

File: pr2_description/robots/pr2.urdf.xacro (robot description, xacro)
@@ -100,4 +100,5 @@
                           camera_info_topic_name="l_forearm_cam/camera_info"
                           parent="l_forearm_roll_link" hfov="90" focal_length="320"
+                          frame_id="l_forearm_cam_frame" hack_baseline="0"
                           image_width="640" image_height="480">
     <origin xyz=".15 0 .07" rpy="${ M_PI/2} ${-45*M_PI/180} 0" />
@@ -106,4 +107,5 @@
                           camera_info_topic_name="r_forearm_cam/camera_info"
                           parent="r_forearm_roll_link" hfov="90" focal_length="320"
+                          frame_id="r_forearm_cam_frame" hack_baseline="0"
                           image_width="640" image_height="480">
     <origin xyz=".15 0 .07" rpy="${-M_PI/2} ${-45*M_PI/180} 0" />

File: pr2_description/urdf/sensors/stereo_camera.urdf.xacro (robot description, xacro)
@@ -77,4 +77,5 @@
                             camera_info_topic_name="${name}/left/camera_info" parent="${name}_optical_frame"
                             hfov="${hfov}" focal_length="${focal_length}"
+                            frame_id="${name}_l_stereo_camera_frame" hack_baseline="0"
                             image_width="${image_width}" image_height="${image_height}">
       <origin xyz="0 0 0" rpy="0 ${-M_PI/2} ${M_PI/2}" />
@@ -84,4 +85,5 @@
                             camera_info_topic_name="${name}/right/camera_info" parent="${name}_l_stereo_camera_frame"
                             hfov="${hfov}" focal_length="${focal_length}"
+                            frame_id="${name}_l_stereo_camera_frame" hack_baseline="${stereo_dy}"
                             image_width="${image_width}" image_height="${image_height}">
       <origin xyz="${stereo_dx} ${stereo_dy} ${stereo_dz}" rpy="${stereo_rx} ${stereo_ry} ${stereo_rz}" />

File: pr2_description/urdf/sensors/wge100_camera.gazebo.xacro (robot description, xacro)
@@ -4,5 +4,5 @@
        xmlns:interface="http://playerstage.sourceforge.net/gazebo/xmlschema/#interface"
        xmlns:xacro="http://ros.org/wiki/xacro">
-  <xacro:macro name="wge100_camera_gazebo_v0" params="name image_format image_topic_name camera_info_topic_name hfov focal_length image_width image_height">
+  <xacro:macro name="wge100_camera_gazebo_v0" params="name image_format image_topic_name camera_info_topic_name hfov focal_length frame_id hack_baseline image_width image_height">
     <gazebo reference="${name}_frame">
       <sensor:camera name="${name}_sensor">
@@ -18,5 +18,6 @@
           <imageTopicName>${image_topic_name}</imageTopicName>
           <cameraInfoTopicName>${camera_info_topic_name}</cameraInfoTopicName>
-          <frameName>${name}_frame</frameName>
+          <frameName>${frame_id}</frameName>
+          <baseline>${hack_baseline}</baseline>
           <CxPrime>${(image_width+1)/2}</CxPrime>
           <Cx>${(image_width+1)/2}</Cx>

File: pr2_description/urdf/sensors/wge100_camera.urdf.xacro (robot description, xacro)
@@ -6,5 +6,7 @@
        xmlns:xacro="http://ros.org/wiki/xacro">
   <include filename="$(find pr2_description)/urdf/sensors/wge100_camera.gazebo.xacro" />
-  <xacro:macro name="wge100_camera_v0" params="name image_format image_topic_name camera_info_topic_name parent hfov focal_length image_width image_height *origin">
+  <!-- hack_baseline is used to simulate right stereo camera projection matrix translation to left stereo camera frame, currently on the hardware,
+       custom left stereo camera frame_id is passed to right stereo wge100 camera node at launch time, baseline is stored on the camera. -->
+  <xacro:macro name="wge100_camera_v0" params="name image_format image_topic_name camera_info_topic_name parent hfov focal_length frame_id hack_baseline image_width image_height *origin">
     <joint name="${name}_frame_joint" type="fixed">
       <insert_block name="origin" />
@@ -63,4 +65,5 @@
                                    camera_info_topic_name="${camera_info_topic_name}"
                                    hfov="${hfov}" focal_length="${focal_length}"
+                                   frame_id="${frame_id}" hack_baseline="${hack_baseline}"
                                    image_width="${image_width}" image_height="${image_height}"/>
   </xacro:macro>

Commit message: adding parameter to pr2_forearm_v0 for setting origin for forearm attachment (for qualification testing).

File: pr2_description/robots/pr2.urdf.xacro (robot description, xacro)
@@ -61,6 +61,10 @@
     <origin xyz="0.0 -0.188 0.0" rpy="0 0 0" />
   </xacro:pr2_shoulder_v0>
-  <xacro:pr2_upper_arm_v0 side="r" reflect="-1" parent="r_upper_arm_roll_link"/>
-  <xacro:pr2_forearm_v0 side="r" reflect="-1" parent="r_forearm_roll_link"/>
+  <xacro:pr2_upper_arm_v0 side="r" reflect="-1" parent="r_upper_arm_roll_link">
+    <origin xyz="0 0 0" rpy="0 0 0" />
+  </xacro:pr2_upper_arm_v0>
+  <xacro:pr2_forearm_v0 side="r" reflect="-1" parent="r_forearm_roll_link">
+    <origin xyz="0 0 0" rpy="0 0 0" />
+  </xacro:pr2_upper_arm_v0>
   <xacro:pr2_gripper_v0 side="r" parent="r_wrist_roll_link"
                screw_reduction="${4.0/1000.0}"

File: pr2_description/urdf/forearm_v0/forearm.urdf.xacro (robot description, xacro)
@@ -11,7 +11,7 @@
   <include filename="$(find pr2_description)/urdf/common.xacro" />
   <!-- ============================   Forearm   ============================ -->
-  <xacro:macro name="pr2_forearm_v0" params="side parent reflect">
+  <xacro:macro name="pr2_forearm_v0" params="side parent reflect *origin">
     <joint name="${side}_forearm_joint" type="fixed">
-      <origin xyz="0 0 0" rpy="0 0 0" />
+      <insert_block name="origin" /> <!-- transform from parent link to this joint frame -->
       <parent link="${parent}"/>
       <child link="${side}_forearm_link"/>

Commit message: fix urdf typo.

File: pr2_description/robots/pr2.urdf.xacro (robot description, xacro)
@@ -61,10 +61,8 @@
     <origin xyz="0.0 -0.188 0.0" rpy="0 0 0" />
   </xacro:pr2_shoulder_v0>
-  <xacro:pr2_upper_arm_v0 side="r" reflect="-1" parent="r_upper_arm_roll_link">
-    <origin xyz="0 0 0" rpy="0 0 0" />
-  </xacro:pr2_upper_arm_v0>
+  <xacro:pr2_upper_arm_v0 side="r" reflect="-1" parent="r_upper_arm_roll_link"/>
   <xacro:pr2_forearm_v0 side="r" reflect="-1" parent="r_forearm_roll_link">
     <origin xyz="0 0 0" rpy="0 0 0" />
-  </xacro:pr2_upper_arm_v0>
+  </xacro:pr2_forearm_v0>
   <xacro:pr2_gripper_v0 side="r" parent="r_wrist_roll_link"
                screw_reduction="${4.0/1000.0}"
@@ -84,5 +82,7 @@
   </xacro:pr2_shoulder_v0>
   <xacro:pr2_upper_arm_v0 side="l" reflect="1" parent="l_upper_arm_roll_link"/>
-  <xacro:pr2_forearm_v0 side="l" reflect="1" parent="l_forearm_roll_link"/>
+  <xacro:pr2_forearm_v0 side="l" reflect="1" parent="l_forearm_roll_link">
+    <origin xyz="0 0 0" rpy="0 0 0" />
+  </xacro:pr2_forearm_v0>
   <xacro:pr2_gripper_v0 side="l" parent="l_wrist_roll_link"
                screw_reduction="${4.0/1000.0}"

Commit message: Updating PR2 beta description as per mechanical drawings from Function. #3473

File: pr2_description/robots/pr2.urdf.xacro (robot description, xacro)
@@ -45,6 +45,6 @@
        numerical values that were specified in common.xacro which was included above -->
   <xacro:pr2_head_v0 name="head" parent="torso_lift_link">
-    <origin xyz="${cal_head_x}    ${cal_head_y}     ${0.3915+cal_head_z}"
-            rpy="${cal_head_roll} ${cal_head_pitch} ${cal_head_yaw}" />
+    <origin xyz="-0.01707 0.0 0.38145"
+            rpy="0.0 0.0 0.0" />
   </xacro:pr2_head_v0>
   <!-- Camera package: double stereo, prosilica -->
@@ -55,5 +55,5 @@
   </xacro:pr2_head_sensor_package_v0>
   <xacro:pr2_tilting_laser_v0 name="laser_tilt" parent="torso_lift_link" laser_calib_ref="0.0">
-    <origin xyz="0.1 0 0.235" rpy="0 0 0" />
+    <origin xyz="0.09893 0 0.227" rpy="0 0 0" />
   </xacro:pr2_tilting_laser_v0>
   <!-- This is a common convention, to use a reflect parameter that equals +-1 to distinguish left from right -->

File: pr2_description/urdf/head_v0/head.urdf.xacro (robot description, xacro)
@@ -13,5 +13,5 @@
       <safety_controller k_velocity="1.5" soft_lower_limit="${-3.007+0.15}" soft_upper_limit="${3.007-0.15}" k_position="100" />
       <!-- hold both reference_position and upper/lower for tick-tock, remove reference_positiion after verifying upper/lower works with calibration controllers.  if search velocity in pr2_calibration_controllers.yaml is +, the reference_position is rising, if - then it is falling -->
-      <calibration reference_position="${0.0+cal_head_pan_flag}" rising="${0.0+cal_head_pan_flag}" />
+      <calibration reference_position="0.0" rising="0.0" />
       <dynamics damping="1.0" />
       <insert_block name="origin" />
@@ -87,5 +87,5 @@
     </xacro:pr2_head_pan_v0>
     <xacro:pr2_head_tilt_v0 name="${name}_tilt" parent="${name}_pan_link">
-      <origin xyz="0.058 0 0" rpy="0 0 0" />
+      <origin xyz="0.068 0 0" rpy="0 0 0" />
     </xacro:pr2_head_tilt_v0>
     <!-- Head plate frame -->

Commit message: Changing forearm cam rotations in URDF

File: pr2_description/robots/pr2.urdf.xacro (robot description, xacro)
@@ -104,5 +104,5 @@
                           frame_id="l_forearm_cam_frame" hack_baseline="0"
                           image_width="640" image_height="480">
-    <origin xyz=".15 0 .07" rpy="${ M_PI/2} ${-45*M_PI/180} 0" />
+    <origin xyz=".15 0 .07" rpy="${-M_PI/2} ${-M_PI/4} 0" />
   </xacro:wge100_camera_v0>
   <xacro:wge100_camera_v0 name="r_forearm_cam" image_format="L8" image_topic_name="r_forearm_cam/image_raw"
@@ -111,5 +111,5 @@
                           frame_id="r_forearm_cam_frame" hack_baseline="0"
                           image_width="640" image_height="480">
-    <origin xyz=".15 0 .07" rpy="${-M_PI/2} ${-45*M_PI/180} 0" />
+    <origin xyz=".15 0 .07" rpy="${M_PI/2} ${-M_PI/4} 0" />
   </xacro:wge100_camera_v0>
 </robot>

Commit message: Updating forearm camera pose

File: pr2_description/robots/pr2.urdf.xacro (robot description, xacro)
@@ -98,5 +98,6 @@
     <origin xyz="0 0 0" rpy="0 0 0" />
   </xacro:pr2_gripper_v0>
-  <!-- Forearm Cam (Hand approximated values) -->
+  <!-- Forearm cam Position is a guess, based on full robot calibration -->
+  <!-- Forearm cam Orientation is from Function -->
   <xacro:wge100_camera_v0 name="l_forearm_cam" image_format="L8" image_topic_name="l_forearm_cam/image_raw"
                           camera_info_topic_name="l_forearm_cam/camera_info"
@@ -104,5 +105,5 @@
                           frame_id="l_forearm_cam_frame" hack_baseline="0"
                           image_width="640" image_height="480">
-    <origin xyz=".15 0 .07" rpy="${-M_PI/2} ${-M_PI/4} 0" />
+    <origin xyz=".135 0 .044" rpy="${-M_PI/2} ${-32.25*M_PI/180} 0" />
   </xacro:wge100_camera_v0>
   <xacro:wge100_camera_v0 name="r_forearm_cam" image_format="L8" image_topic_name="r_forearm_cam/image_raw"
@@ -111,5 +112,5 @@
                           frame_id="r_forearm_cam_frame" hack_baseline="0"
                           image_width="640" image_height="480">
-    <origin xyz=".15 0 .07" rpy="${M_PI/2} ${-M_PI/4} 0" />
+    <origin xyz=".135 0 .044" rpy="${M_PI/2} ${-32.25*M_PI/180} 0" />
   </xacro:wge100_camera_v0>
 </robot>
