Commit message: hiding parallel links into gazebo extensions

File: pr2_description/robots/pr2.urdf.xacro (robot description, xacro)
@@ -65,5 +65,5 @@
     <origin xyz="0 0 0" rpy="0 0 0" />
   </xacro:pr2_forearm_v0>
-  <xacro:pr2_gripper_v0 side="r" parent="r_wrist_roll_link"
+  <xacro:pr2_gripper_v0 reflect="-1.0" side="r" parent="r_wrist_roll_link"
                screw_reduction="${4.0/1000.0}"
                gear_ratio="${(729.0/25.0)*(22.0/16.0)}"
@@ -85,5 +85,5 @@
     <origin xyz="0 0 0" rpy="0 0 0" />
   </xacro:pr2_forearm_v0>
-  <xacro:pr2_gripper_v0 side="l" parent="l_wrist_roll_link"
+  <xacro:pr2_gripper_v0 reflect="1.0" side="l" parent="l_wrist_roll_link"
                screw_reduction="${4.0/1000.0}"
                gear_ratio="${(729.0/25.0)*(22.0/16.0)}"

File: pr2_description/urdf/gripper_v0/gripper.gazebo.xacro (robot description, xacro)
@@ -18,5 +18,7 @@
   <property name="finger_tip_mu"              value="500.0" />
   <property name="finger_mu"                  value="500.0" />
-  <xacro:macro name="pr2_finger_gazebo_v0" params="prefix parallel_link_x_offset parallel_link_y_offset">
+  <property name="parallel_link_x_offset"     value="-0.018" />
+  <property name="parallel_link_y_offset"     value="0.021" />
+  <xacro:macro name="pr2_finger_gazebo_v0" params="prefix reflect">
     <!-- Finger proximal digit -->
     <gazebo reference="${prefix}_l_finger_link">
@@ -139,4 +141,56 @@
     <!-- parallel link for simulating gripper constraints -->
     <gazebo>
+      <body:box name="${prefix}_l_parallel_link">
+          <massMatrix>true</massMatrix>
+          <mass>0.17126</mass>
+          <ixx>7.7562e-05</ixx>
+          <ixy>1.49095e-06</ixy>
+          <ixz>-9.83385e-06</ixz>
+          <iyy>0.000197083</iyy>
+          <iyz>-3.06125e-06</iyz>
+          <izz>0.000181054</izz>
+          <cx>0.03598</cx>
+          <cy>0.0173</cy>
+          <cz>-0.00164</cz>
+          <xyz>0.82991 ${0.188*reflect+0.031} 0.790675</xyz>
+          <rpy>0 -0 0</rpy>
+          <turnGravityOff>true</turnGravityOff>
+          <selfCollide>false</selfCollide>
+      </body:box>
+      <body:box name="${prefix}_r_parallel_link">
+          <massMatrix>true</massMatrix>
+          <mass>0.17389</mass>
+          <ixx>7.73841e-05</ixx>
+          <ixy>-2.09309e-06</ixy>
+          <ixz>-8.36228e-06</ixz>
+          <iyy>0.000198474</iyy>
+          <iyz>2.4611e-06</iyz>
+          <izz>0.00018107</izz>
+          <cx>0.03576</cx>
+          <cy>-0.01736</cy>
+          <cz>-0.00095</cz>
+          <xyz>0.82991 ${0.188*reflect-0.031} 0.790675</xyz>
+          <rpy>0 -0 0</rpy>
+          <turnGravityOff>true</turnGravityOff>
+          <selfCollide>false</selfCollide>
+      </body:box>
+    </gazebo>
+    <gazebo>
+      <joint:hinge name="${prefix}_r_parallel_root_joint">
+          <body1>${prefix}_r_parallel_link</body1>
+          <body2>${prefix}_palm_link</body2>
+          <anchor>${prefix}_palm_link</anchor>
+          <axis>0 0 -1</axis>
+          <damping>0.2</damping>
+          <anchorOffset>${0.07691+parallel_link_x_offset} ${-0.01-parallel_link_y_offset} 0</anchorOffset>
+      </joint:hinge>
+      <joint:hinge name="${prefix}_l_parallel_root_joint">
+          <body1>${prefix}_l_parallel_link</body1>
+          <body2>${prefix}_palm_link</body2>
+          <anchor>${prefix}_palm_link</anchor>
+          <axis>0 0 1</axis>
+          <damping>0.2</damping>
+          <anchorOffset>${0.07691+parallel_link_x_offset} ${0.01+parallel_link_y_offset} 0</anchorOffset>
+      </joint:hinge>
       <joint:hinge name="${prefix}_r_parallel_tip_joint">
           <body1>${prefix}_r_parallel_link</body1>

File: pr2_description/urdf/gripper_v0/gripper.transmission.xacro (robot description, xacro)
@@ -37,6 +37,4 @@
       <passive_joint  name="${side}_gripper_r_finger_tip_joint" />
       <passive_joint  name="${side}_gripper_l_finger_tip_joint" />
-      <passive_joint  name="${side}_gripper_r_parallel_root_joint" />
-      <passive_joint  name="${side}_gripper_l_parallel_root_joint" />
     </transmission>
   </xacro:macro>

File: pr2_description/urdf/gripper_v0/gripper.urdf.xacro (robot description, xacro)
@@ -13,8 +13,6 @@
   <property name="gripper_damping"            value="100.0" />
   <property name="finger_tip_damping"         value="0.01" />
-  <property name="parallel_link_x_offset"     value="-0.018" />
-  <property name="parallel_link_y_offset"     value="0.021" />
   <property name="finger_joint_effort_limit"  value="1000.0" />
-  <xacro:macro name="pr2_finger_limits_v0" params="reflect">
+  <xacro:macro name="pr2_finger_limits_v0">
     <!-- limits on passive finger and finger top joints without
          transmission are not enforced by safety controllers.
@@ -25,9 +23,9 @@
            lower="${gripper_lower_angle}" upper="${gripper_upper_angle}" />
   </xacro:macro>
-  <xacro:macro name="pr2_finger_v0" params="prefix parent">
+  <xacro:macro name="pr2_finger_v0" params="prefix parent reflect">
     <!-- Finger proximal digit -->
     <joint name="${prefix}_l_finger_joint" type="revolute">
       <axis xyz="0 0 1" />
-      <xacro:pr2_finger_limits_v0 reflect="1" />
+      <xacro:pr2_finger_limits_v0/>
       <dynamics damping="${finger_damping}" />
       <origin xyz="0.07691 0.01 0" rpy="0 0 0" />
@@ -65,5 +63,5 @@
       <axis xyz="0 0 -1" />
       <origin xyz="0.07691 -0.01 0" rpy="0 0 0" />
-      <xacro:pr2_finger_limits_v0 reflect="1" />
+      <xacro:pr2_finger_limits_v0/>
       <dynamics damping="${finger_damping}" />
       <mimic joint="${prefix}_l_finger_joint" multiplier="1" offset="0"/>
@@ -97,84 +95,9 @@
       </collision>
     </link>
-    <!-- Floating Link -->
-    <joint name="${prefix}_l_parallel_root_joint" type="revolute">
-      <axis xyz="0 0 1" />
-      <origin xyz="${0.07691+parallel_link_x_offset} ${+0.01+parallel_link_y_offset} 0" rpy="0 0 0" />
-      <dynamics damping="${finger_damping}" />
-      <mimic joint="${prefix}_l_finger_joint" multiplier="1" offset="0"/>
-      <parent link="${parent}"/>
-      <child link="${prefix}_l_parallel_link"/>
-      <xacro:pr2_finger_limits_v0 reflect="1" />
-    </joint>
-    <joint name="${prefix}_r_parallel_root_joint" type="revolute">
-      <axis xyz="0 0 -1" />
-      <origin xyz="${0.07691+parallel_link_x_offset} ${-0.01-parallel_link_y_offset} 0" rpy="0 0 0" />
-      <dynamics damping="${finger_damping}" />
-      <mimic joint="${prefix}_l_finger_joint" multiplier="-1" offset="0"/>
-      <parent link="${parent}"/>
-      <child link="${prefix}_r_parallel_link"/>
-      <xacro:pr2_finger_limits_v0 reflect="1" />
-    </joint>
-    <link name="${prefix}_l_parallel_link">
-      <inertial>
-        <mass value="0.17126" />
-        <origin xyz="${0.03598} 0.01730 -0.00164" rpy="0 0 0" />
-        <inertia  ixx= "0.00007756198"
-                  ixy= "0.00000149095"
-                  ixz="-0.00000983385"
-                  iyy= "0.00019708305"
-                  iyz="-0.00000306125"
-                  izz= "0.00018105446" />
-      </inertial>
-<!--
-      <visual>
-        <origin xyz="${0.0914942479/2.0} 0 0" rpy="0 0 0.0541224233" />
-        <geometry>
-          <box size="${0.0914942479} 0.005 0.005" />
-        </geometry>
-        <material name="Green" />
-      </visual>
--->
-      <collision>
-        <origin xyz="${0.0914942479/2.0} 0 0" rpy="0 0 0.0541224233" />
-        <geometry>
-          <box size="${0.0914942479} 0.005 0.005" />
-        </geometry>
-        <verbose value="Yes" />
-      </collision>
-    </link>
-    <link name="${prefix}_r_parallel_link">
-      <inertial>
-        <mass value="0.17389" />
-        <origin xyz="${0.03576} -0.01736 -0.00095" rpy="0 0 0" />
-        <inertia  ixx= "0.00007738410"
-                  ixy="-0.00000209309"
-                  ixz="-0.00000836228"
-                  iyy= "0.00019847383"
-                  iyz= "0.00000246110"
-                  izz= "0.00018106988" />
-      </inertial>
-<!--
-      <visual>
-        <origin xyz="${0.0914942479/2.0} 0 0" rpy="0 0 -0.0541224233" />
-        <geometry>
-          <box size="${0.0914942479} 0.005 0.005" />
-        </geometry>
-        <material name="Green" />
-      </visual>
--->
-      <collision>
-        <origin xyz="${0.0914942479/2.0} 0 0" rpy="0 0 -0.0541224233" />
-        <geometry>
-          <box size="${0.0914942479} 0.005 0.005" />
-        </geometry>
-        <verbose value="Yes" />
-      </collision>
-    </link>
     <!-- Finger tip -->
     <joint name="${prefix}_l_finger_tip_joint" type="revolute">
       <axis xyz="0 0 -1" />
       <origin xyz="0.09137 0.00495 0" rpy="0 0 0" />
-      <xacro:pr2_finger_limits_v0 reflect="1" />
+      <xacro:pr2_finger_limits_v0/>
       <dynamics damping="${finger_tip_damping}" />
       <mimic joint="${prefix}_l_finger_joint" multiplier="1" offset="0"/>
@@ -209,5 +132,5 @@
       <axis xyz="0 0 1" />
       <origin xyz="${0.09137} ${-0.00495} 0" rpy="0 0 0" />
-      <xacro:pr2_finger_limits_v0 reflect="1" />
+      <xacro:pr2_finger_limits_v0/>
       <dynamics damping="${finger_tip_damping}" />
       <mimic joint="${prefix}_l_finger_joint" multiplier="1" offset="0"/>
@@ -239,7 +162,7 @@
     </link>
     <!-- extensions -->
-    <xacro:pr2_finger_gazebo_v0 prefix="${prefix}" parallel_link_x_offset="${parallel_link_x_offset}" parallel_link_y_offset="${parallel_link_y_offset}" />
+    <xacro:pr2_finger_gazebo_v0 prefix="${prefix}" reflect="${reflect}" />
   </xacro:macro>
-  <xacro:macro name="pr2_gripper_v0" params="side parent *origin gear_ratio screw_reduction theta0 phi0 t0 L0 h a b r">
+  <xacro:macro name="pr2_gripper_v0" params="side reflect parent *origin gear_ratio screw_reduction theta0 phi0 t0 L0 h a b r">
     <joint name="${side}_gripper_palm_joint" type="fixed">
       <insert_block name="origin"/>
@@ -310,5 +233,5 @@
     <link name="${side}_gripper_tool_frame"/>
     <!-- pr2 fingers macro -->
-    <xacro:pr2_finger_v0 prefix="${side}_gripper" parent="${side}_gripper_palm_link" />
+    <xacro:pr2_finger_v0 prefix="${side}_gripper" reflect="${reflect}" parent="${side}_gripper_palm_link" />
     <!-- fictitous joint that represents the gripper gap -->
     <!-- effort is the linear force at the gripper gap

Commit message: cleanup projector urdf.  adding projector urdf to pr2 robot.

File: pr2_description/robots/pr2.urdf.xacro (robot description, xacro)
@@ -26,4 +26,6 @@
   <!-- Camera sensors -->
   <include filename="$(find pr2_description)/urdf/sensors/wge100_camera.urdf.xacro" />
+  <!-- Texture projector -->
+  <include filename="$(find pr2_description)/urdf/sensors/projector_wg6802418.urdf.xacro" />
   <!-- generic simulator_gazebo plugins for starting mechanism control, ros time, ros battery -->
   <include filename="$(find pr2_description)/gazebo/gazebo.urdf.xacro" />
@@ -54,4 +56,9 @@
     <origin xyz="0.0 0.0 0.0" rpy="0 0 0" />
   </xacro:pr2_head_sensor_package_v0>
+  <!-- Projector -->
+  <xacro:projector_wg6802418_v0 name="projector_wg6802418" parent="head_plate_frame" >
+    <!-- Camera is slightly recessed from front, where is camera origin? Lens? -->
+    <origin xyz="0 0.109 0.035" rpy="0 0 0" />
+  </xacro:projector_wg6802418_v0>
   <xacro:pr2_tilting_laser_v0 name="laser_tilt" parent="torso_lift_link" laser_calib_ref="0.0">
     <origin xyz="0.09893 0 0.227" rpy="0 0 0" />

File: pr2_description/robots/pr2_no_arms.urdf.xacro (robot description, xacro)
@@ -20,4 +20,6 @@
   <!-- Camera sensors -->
   <include filename="$(find pr2_description)/urdf/sensors/wge100_camera.urdf.xacro" />
+  <!-- Texture projector -->
+  <include filename="$(find pr2_description)/urdf/sensors/projector_wg6802418.urdf.xacro" />
   <!-- generic simulator_gazebo plugins for starting mechanism control, ros time, ros battery -->
   <include filename="$(find pr2_description)/gazebo/gazebo.urdf.xacro" />
@@ -42,4 +44,9 @@
             rpy="${cal_head_roll} ${cal_head_pitch} ${cal_head_yaw}" />
   </xacro:pr2_head_v0>
+  <!-- Projector -->
+  <xacro:projector_wg6802418_v0 name="projector_wg6802418" parent="head_plate_frame" >
+    <!-- Camera is slightly recessed from front, where is camera origin? Lens? -->
+    <origin xyz="0 0.109 0.035" rpy="0 0 0" />
+  </xacro:projector_wg6802418_v0>
   <!-- Camera package: double stereo, prosilica -->
   <xacro:pr2_head_sensor_package_v0 name="sensor_mount" hd_name="high_def"

File: pr2_description/urdf/sensors/projector_wg6802418.urdf.xacro (robot description, xacro)
@@ -60,34 +60,5 @@
         </geometry>
       </collision>
-    </link> -->
-<!--
-    <joint name="${name}_projector_wg6802418_frame_joint" type="fixed">
-      <origin xyz="${cal_high_def_x}            ${cal_high_def_y}         ${cal_high_def_z}"
-                rpy="${-M_PI/2+cal_high_def_roll} ${0.0+cal_high_def_pitch} ${-M_PI/2+cal_high_def_yaw}" />
-      <parent link="${name}_frame"/>
-      <child link="${name}_child_frame"/>
-    </joint>
-    <link name="${name}_child_frame">
-      <inertial>
-        <mass value="0.01" />
-        <origin xyz="0 0 0" rpy="0 0 0"/>
-        <inertia ixx="0.001"  ixy="0.0"  ixz="0.0"
-                 iyy="0.001"  iyz="0.0"
-                 izz="0.001" />
-      </inertial>
-      <visual>
-        <origin xyz="0 0 0" rpy="0 0 ${M_PI/2}" />
-        <geometry>
-          <cylinder radius="0.02" length="0.05" />
-        </geometry>
-        <material name="Blue" />
-      </visual>
-      <collision>
-        <origin xyz="0 0 0" rpy="0 0 0"/>
-        <geometry>
-          <box size="0.01 0.01 0.01" />
-        </geometry>
-      </collision>
-    </link> -->
+    </link>
     <!-- extensions -->
     <xacro:projector_wg6802418_gazebo_v0 name="${name}"/>

Commit message: !!!XACRO API BREAK!!! ====================================================================================================== To mimic wg100 cameras on the robot, "wge100_camera_gazebo_v0" xacro has a new parameter "camera_name"   which will deprecate/replace parameters "image_topic_name" and "camera_info_topic_name". Anyone using the "wge100_camera_v0" xacro should add a "camera_name" parameter to the xacro. Also refer to ticket #4871.

File: pr2_description/robots/pr2.urdf.xacro (robot description, xacro)
@@ -107,6 +107,6 @@
   <!-- Forearm cam Position is a guess, based on full robot calibration -->
   <!-- Forearm cam Orientation is from Function -->
-  <xacro:wge100_camera_v0 name="l_forearm_cam" image_format="L8" image_topic_name="l_forearm_cam/image_raw"
-                          camera_info_topic_name="l_forearm_cam/camera_info"
+  <xacro:wge100_camera_v0 name="l_forearm_cam" image_format="L8" camera_name="l_forearm_cam" image_topic_name="image_raw"
+                          camera_info_topic_name="camera_info"
                           parent="l_forearm_roll_link" hfov="90" focal_length="320"
                           frame_id="l_forearm_cam_optical_frame" hack_baseline="0"
@@ -114,6 +114,6 @@
     <origin xyz=".135 0 .044" rpy="${-M_PI/2} ${-32.25*M_PI/180} 0" />
   </xacro:wge100_camera_v0>
-  <xacro:wge100_camera_v0 name="r_forearm_cam" image_format="L8" image_topic_name="r_forearm_cam/image_raw"
-                          camera_info_topic_name="r_forearm_cam/camera_info"
+  <xacro:wge100_camera_v0 name="r_forearm_cam" image_format="L8" camera_name="r_forearm_cam" image_topic_name="image_raw"
+                          camera_info_topic_name="camera_info"
                           parent="r_forearm_roll_link" hfov="90" focal_length="320"
                           frame_id="r_forearm_cam_optical_frame" hack_baseline="0"

File: pr2_description/urdf/sensors/stereo_camera.urdf.xacro (robot description, xacro)
@@ -37,6 +37,6 @@
     <link name="${name}_optical_frame" type="camera"/>
     <!-- stereo left camera -->
-    <xacro:wge100_camera_v0 name="${name}_gazebo_l_stereo_camera" image_format="${image_format}" image_topic_name="${name}/left/image_raw"
-                            camera_info_topic_name="${name}/left/camera_info" parent="${name}_link"
+    <xacro:wge100_camera_v0 name="${name}_gazebo_l_stereo_camera" camera_name="${name}/left" image_format="${image_format}" image_topic_name="image_raw"
+                            camera_info_topic_name="camera_info" parent="${name}_link"
                             hfov="${hfov}" focal_length="${focal_length}"
                             frame_id="${name}_optical_frame" hack_baseline="0"
@@ -45,6 +45,6 @@
     </xacro:wge100_camera_v0>
     <!-- stereo right camera -->
-    <xacro:wge100_camera_v0 name="${name}_gazebo_r_stereo_camera" image_format="${image_format}" image_topic_name="${name}/right/image_raw"
-                            camera_info_topic_name="${name}/right/camera_info" parent="${name}_gazebo_l_stereo_camera_frame"
+    <xacro:wge100_camera_v0 name="${name}_gazebo_r_stereo_camera" camera_name="${name}/right" image_format="${image_format}" image_topic_name="image_raw"
+                            camera_info_topic_name="camera_info" parent="${name}_gazebo_l_stereo_camera_frame"
                             hfov="${hfov}" focal_length="${focal_length}"
                             frame_id="${name}_optical_frame" hack_baseline="${-stereo_dy}"

File: pr2_description/urdf/sensors/wge100_camera.gazebo.xacro (robot description, xacro)
@@ -4,5 +4,5 @@
        xmlns:interface="http://playerstage.sourceforge.net/gazebo/xmlschema/#interface"
        xmlns:xacro="http://ros.org/wiki/xacro">
-  <xacro:macro name="wge100_camera_gazebo_v0" params="name image_format image_topic_name camera_info_topic_name hfov focal_length frame_id hack_baseline image_width image_height">
+  <xacro:macro name="wge100_camera_gazebo_v0" params="name camera_name image_format image_topic_name camera_info_topic_name hfov focal_length frame_id hack_baseline image_width image_height">
     <gazebo reference="${name}_frame">
       <sensor:camera name="${name}_sensor">
@@ -16,4 +16,5 @@
           <alwaysOn>true</alwaysOn>
           <updateRate>25.0</updateRate>
+          <cameraName>${camera_name}</cameraName>
           <imageTopicName>${image_topic_name}</imageTopicName>
           <cameraInfoTopicName>${camera_info_topic_name}</cameraInfoTopicName>

File: pr2_description/urdf/sensors/wge100_camera.urdf.xacro (robot description, xacro)
@@ -8,5 +8,5 @@
   <!-- hack_baseline is used to simulate right stereo camera projection matrix translation to left stereo camera frame, currently on the hardware,
        custom left stereo camera frame_id is passed to right stereo wge100 camera node at launch time, baseline is stored on the camera. -->
-  <xacro:macro name="wge100_camera_v0" params="name image_format image_topic_name camera_info_topic_name parent hfov focal_length frame_id hack_baseline image_width image_height *origin">
+  <xacro:macro name="wge100_camera_v0" params="name camera_name image_format image_topic_name camera_info_topic_name parent hfov focal_length frame_id hack_baseline image_width image_height *origin">
     <joint name="${name}_frame_joint" type="fixed">
       <insert_block name="origin" />
@@ -30,5 +30,5 @@
     <link name="${name}_optical_frame"/>
     <!-- extensions -->
-    <xacro:wge100_camera_gazebo_v0 name="${name}" image_format="${image_format}" image_topic_name="${image_topic_name}"
+    <xacro:wge100_camera_gazebo_v0 name="${name}" camera_name="${camera_name}" image_format="${image_format}" image_topic_name="${image_topic_name}"
                                    camera_info_topic_name="${camera_info_topic_name}"
                                    hfov="${hfov}" focal_length="${focal_length}"
