Commit message: properly distinguishing between frame and camera name for prosilica model.

File: pr2_description/robots/pr2.urdf.xacro (robot description, xacro)
@@ -51,5 +51,6 @@
   </xacro:pr2_head_v0>
   <!-- Camera package: double stereo, prosilica -->
-  <xacro:pr2_head_sensor_package_v0 name="sensor_mount" hd_name="high_def"
+  <xacro:pr2_head_sensor_package_v0 name="sensor_mount" hd_frame_name="high_def"
+			   hd_camera_name="prosilica"
 			   stereo_name="double_stereo"
 			   parent="head_plate_frame">

File: pr2_description/urdf/sensors/head_sensor_package.urdf.xacro (robot description, xacro)
@@ -14,5 +14,5 @@
   <!-- Origin is center mount screw on sensor plate mount -->
   <!-- When mounted properly, should have same origin as head plate frame -->
-  <xacro:macro name="pr2_head_sensor_package_v0" params="name hd_name stereo_name parent *origin">
+  <xacro:macro name="pr2_head_sensor_package_v0" params="name hd_frame_name hd_camera_name stereo_name parent *origin">
     <joint name="${name}_frame_joint" type="fixed">
       <insert_block name="origin" />
@@ -38,5 +38,5 @@
     </link>
     <!-- Prosilica Camera -->
-    <xacro:prosilica_cam_v0 name="${hd_name}" parent="${name}_link" >
+    <xacro:prosilica_cam_v0 frame_name="${hd_frame_name}" camera_name="${hd_camera_name}" parent="${name}_link" >
       <!-- Center of camera is 109mm right of center screw, 35mm up -->
       <!-- Camera is slightly recessed from front, where is camera origin? Lens? -->

File: pr2_description/urdf/sensors/prosilica_gc2450_camera.gazebo.xacro (robot description, xacro)
@@ -4,7 +4,7 @@
       xmlns:interface="http://playerstage.sourceforge.net/gazebo/xmlschema/#interface"
       xmlns:xacro="http://ros.org/wiki/xacro">
-<xacro:macro name="prosilica_cam_gazebo_v0" params="name">
-  <gazebo reference="${name}_frame">
-    <sensor:camera name="${name}_sensor">
+<xacro:macro name="prosilica_cam_gazebo_v0" params="camera_name frame_name">
+  <gazebo reference="${frame_name}_frame">
+    <sensor:camera name="${frame_name}_sensor">
       <imageFormat>R8G8B8</imageFormat>
       <imageSize>2448 2050</imageSize>
@@ -13,11 +13,12 @@
       <farClip>100</farClip>
       <updateRate>20.0</updateRate>
-      <controller:gazebo_ros_prosilica name="${name}_controller" plugin="libgazebo_ros_prosilica.so">
+      <controller:gazebo_ros_prosilica name="${frame_name}_controller" plugin="libgazebo_ros_prosilica.so">
         <alwaysOn>true</alwaysOn>
         <updateRate>20.0</updateRate>
-        <imageTopicName>/prosilica/image_raw</imageTopicName>
-        <cameraInfoTopicName>/prosilica/camera_info</cameraInfoTopicName>
-        <pollServiceName>/prosilica/request_image</pollServiceName>
-        <frameName>${name}_frame</frameName>
+        <cameraName>${camera_name}</cameraName>
+        <imageTopicName>image_raw</imageTopicName>
+        <cameraInfoTopicName>camera_info</cameraInfoTopicName>
+        <pollServiceName>request_image</pollServiceName>
+        <frameName>${frame_name}_optical_frame</frameName>
         <CxPrime>1224.5</CxPrime>
         <Cx>1224.5</Cx>
@@ -29,5 +30,4 @@
         <distortion_t1>0.0</distortion_t1>
         <distortion_t2>0.0</distortion_t2>
-        <interface:camera name="${name}_iface" />
       </controller:gazebo_ros_prosilica>
     </sensor:camera>

File: pr2_description/urdf/sensors/prosilica_gc2450_camera.urdf.xacro (robot description, xacro)
@@ -5,11 +5,11 @@
       xmlns:xacro="http://ros.org/wiki/xacro">
   <include filename="$(find pr2_description)/urdf/sensors/prosilica_gc2450_camera.gazebo.xacro" />
-  <xacro:macro name="prosilica_cam_v0" params="name parent *origin">
-    <joint name="${name}_frame_joint" type="fixed">
+  <xacro:macro name="prosilica_cam_v0" params="frame_name parent *origin camera_name">
+    <joint name="${frame_name}_frame_joint" type="fixed">
       <insert_block name="origin" />
       <parent link="${parent}"/>
-      <child link="${name}_frame"/>
+      <child link="${frame_name}_frame"/>
     </joint>
-    <link name="${name}_frame">
+    <link name="${frame_name}_frame">
       <inertial>
         <mass value="0.01" />
@@ -28,11 +28,11 @@
       </visual>
     </link>
-    <joint name="${name}_optical_frame_joint" type="fixed">
+    <joint name="${frame_name}_optical_frame_joint" type="fixed">
       <origin xyz="${cal_high_def_x}            ${cal_high_def_y}         ${cal_high_def_z}"
                 rpy="${-M_PI/2+cal_high_def_roll} ${0.0+cal_high_def_pitch} ${-M_PI/2+cal_high_def_yaw}" />
-      <parent link="${name}_frame"/>
-      <child link="${name}_optical_frame"/>
+      <parent link="${frame_name}_frame"/>
+      <child link="${frame_name}_optical_frame"/>
     </joint>
-    <link name="${name}_optical_frame">
+    <link name="${frame_name}_optical_frame">
       <inertial>
         <mass value="0.01" />
@@ -52,5 +52,5 @@
     </link>
     <!-- extensions -->
-    <xacro:prosilica_cam_gazebo_v0 name="${name}"/>
+    <xacro:prosilica_cam_gazebo_v0 camera_name="${camera_name}" frame_name="${frame_name}" />
   </xacro:macro>
 </root>

Commit message: edits to robot urdf files

File: pr2_description/robots/pr2.urdf.xacro (robot description, xacro)
@@ -24,4 +24,5 @@
   <!-- Head sensors -->
   <include filename="$(find pr2_description)/urdf/sensors/head_sensor_package.urdf.xacro" />
+  <include filename="$(find pr2_description)/urdf/sensors/kinect_prosilica_camera.urdf.xacro" />
   <!-- Camera sensors -->
   <include filename="$(find pr2_description)/urdf/sensors/wge100_camera.urdf.xacro" />
@@ -62,4 +63,20 @@
     <origin xyz="0 0.109 0.035" rpy="0 0 0" />
   </xacro:projector_wg6802418_v0>
+  <!-- Base of Kinect/Prosilica Mount -->
+  <xacro:kinect_prosilica_camera_swept_back_v0 name="head_mount" parent="head_plate_frame" >
+    <origin xyz="-0.137376 0 0.091746" rpy="0 0 0" />
+    <!--
+          Was -0.1 0 0.09225, -0.138 0 0.09225 looks good front back and sheet metal on bolt pattern,
+          -0.138 0 0.06225 is where Prosilica FOV just clears the head.
+          This is 30 mm (!) below the position in SolidWorks.
+          Lowering the Prosilica by this amount in SW makes the FOV hit around the aluminum / plastic junction.
+          Turns out that head_plate_frame is in some random position in space.
+          It is [0.0232 0 0.0645 from its parent, head_tilt_link.
+          The distance from head_plate_frame to the head_kinect_prosilica is 137.376 mm X and 91.746 mm Z.
+          So the origin should in fact be -0.137376 0 0.091746.
+          John is changing the Prosilica FOV based on my numbers.
+          Just need to roscd and svn up.
+    -->
+  </xacro:kinect_prosilica_camera_swept_back_v0>
   <xacro:pr2_tilting_laser_v0 name="laser_tilt" parent="torso_lift_link" laser_calib_ref="0.0">
     <origin xyz="0.09893 0 0.227" rpy="0 0 0" />

File: pr2_description/robots/pr2_se.urdf.xacro (robot description, xacro)
@@ -24,5 +24,5 @@
   <!-- Head sensors -->
   <!-- kinect/prosilica model -->
-  <include filename="$(find pr2_kinect_test_description)/urdf/kinect_prosilica_camera.urdf.xacro" />
+  <include filename="$(find pr2_description)/urdf/sensors/kinect_prosilica_camera.urdf.xacro" />
   <!-- Camera sensors -->
   <include filename="$(find pr2_description)/urdf/sensors/wge100_camera.urdf.xacro" />
@@ -52,5 +52,5 @@
   </xacro:pr2_head_v0>
   <!-- Base of Kinect/Prosilica Mount -->
-  <xacro:kinect_prosilica_camera_swept_back_v0 name="head_sensors" parent="head_plate_frame" >
+  <xacro:kinect_prosilica_camera_swept_back_v0 name="head_mount" parent="head_plate_frame" >
     <origin xyz="-0.137376 0 0.091746" rpy="0 0 0" />
     <!--

File: pr2_description/urdf/sensors/kinect_prosilica_camera.urdf.xacro (robot description, xacro)
@@ -8,12 +8,12 @@
   <xacro:macro name="kinect_prosilica_camera_swept_back_v0" params="name parent *origin">
     <!-- stl contains structure + kinect + prosilica combo -->
-    <joint name="${name}_mount_joint" type="fixed">
+    <joint name="${name}_joint" type="fixed">
       <!-- <limit lower="0.1" upper="0.1" effort="10000" velocity="100.0"/> -->
       <!-- <insert_block name="origin" /> -->
       <origin xyz="-0.138 0 0.091" rpy="0 0 0"/>
       <parent link="${parent}"/>
-      <child link="${name}_mount_link"/>
+      <child link="${name}_link"/>
     </joint>
-    <link name="${name}_mount_link">
+    <link name="${name}_link">
       <inertial>
         <mass value="0.1" />
@@ -26,5 +26,5 @@
         <origin xyz="0.0 0.0 0" rpy="0 0 0"/>
         <geometry>
-          <mesh filename="package://pr2_kinect_test_description/meshes/115x100_swept_back--coarse.STL" scale="0.001 0.001 0.001" />
+          <mesh filename="package://pr2_description/meshes/sensors/kinect_prosilica_v0/115x100_swept_back--coarse.STL" scale="0.001 0.001 0.001" />
         </geometry>
         <material name="gray">
@@ -46,5 +46,5 @@
     <joint name="${name}_kinect_joint" type="fixed">
       <origin xyz="-0.032267 0.0125 0.136453" rpy="0 0 0"/>
-      <parent link="${name}_mount_link"/>
+      <parent link="${name}_link"/>
       <child link="${name}_kinect_frame"/>
     </joint>
@@ -125,5 +125,5 @@
     <joint name="${name}_prosilica_joint" type="fixed">
       <origin xyz="-0.046457 0.0125 0.088921" rpy="0 0 0"/>
-      <parent link="${name}_mount_link"/>
+      <parent link="${name}_link"/>
       <child link="${name}_prosilica_link"/>
     </joint>

Commit message: moving double stereo and projector center so they match with model (shift according to changes for prosilica in r52841)

File: pr2_description/robots/pr2.urdf.xacro (robot description, xacro)
@@ -60,5 +60,5 @@
   <xacro:projector_wg6802418_v0 name="projector_wg6802418" parent="head_plate_frame" >
     <!-- Camera is slightly recessed from front, where is camera origin? Lens? -->
-    <origin xyz="0 0.109 0.035" rpy="0 0 0" />
+    <origin xyz="0.046457 0.110 0.0546" rpy="0 0 0" />
   </xacro:projector_wg6802418_v0>
   <xacro:pr2_tilting_laser_v0 name="laser_tilt" parent="torso_lift_link" laser_calib_ref="0.0">

File: pr2_description/robots/pr2_kinect_swept_back.urdf.xacro (robot description, xacro)
@@ -61,5 +61,5 @@
   <xacro:projector_wg6802418_v0 name="projector_wg6802418" parent="head_plate_frame" >
     <!-- Camera is slightly recessed from front, where is camera origin? Lens? -->
-    <origin xyz="0 0.109 0.035" rpy="0 0 0" />
+    <origin xyz="0 0.110 0.0546" rpy="0 0 0" />
   </xacro:projector_wg6802418_v0>
   <!-- Base of Kinect/Prosilica Mount -->

File: pr2_description/robots/pr2_se.urdf.xacro (robot description, xacro)
@@ -69,5 +69,5 @@
   <!-- Projector
   <xacro:projector_wg6802418_v0 name="projector_wg6802418" parent="head_plate_frame" >
-    <origin xyz="0 0.109 0.035" rpy="0 0 0" />
+    <origin xyz="0 0.110 0.0546" rpy="0 0 0" />
   </xacro:projector_wg6802418_v0>
   -->

File: pr2_description/urdf/sensors/double_stereo_camera.urdf.xacro (robot description, xacro)
@@ -40,8 +40,8 @@
     <!-- 15mm offset from center needs check with CAD -->
     <xacro:stereo_camera_v0 parent="${name}_link" name="wide_stereo" focal_length="320" hfov="90" image_format="BAYER_BGGR8" image_width="640" image_height="480" >
-      <origin xyz="0.0 ${0.045-0.015} 0.0305" rpy="0.0   0.0   0.0" />
+      <origin xyz="0.045 ${0.045-0.015} 0.0501" rpy="0.0   0.0   0.0" />
     </xacro:stereo_camera_v0>
     <xacro:stereo_camera_v0 parent="${name}_link" name="narrow_stereo" focal_length="772.55" hfov="45" image_format="L8" image_width="640" image_height="480" >
-      <origin xyz="0.0 ${0.045+0.015} 0.0305" rpy="0.0   0.0   0.0" />
+      <origin xyz="0.045 ${0.045+0.015} 0.0501" rpy="0.0   0.0   0.0" />
     </xacro:stereo_camera_v0>
     <!-- extensions -->

File: pr2_description/urdf/sensors/head_sensor_package.urdf.xacro (robot description, xacro)
@@ -44,5 +44,5 @@
     <!-- construct wide and narrow double stereo camera -->
     <xacro:double_stereo_camera_v0 name="${stereo_name}" parent="${name}_link" >
-      <origin xyz="0.0 0.0 0.003" rpy="0 0 0" />
+      <origin xyz="0.0 0.0 0.0" rpy="0 0 0" />
     </xacro:double_stereo_camera_v0>
     <!-- extensions -->

Commit message: make kinect mount the standard pr2 urdf

File: pr2_description/robots/pr2.urdf.xacro (robot description, xacro)
@@ -24,4 +24,5 @@
   <!-- Head sensors -->
   <include filename="$(find pr2_description)/urdf/sensors/head_sensor_package.urdf.xacro" />
+  <include filename="$(find pr2_description)/urdf/sensors/kinect_prosilica_camera.urdf.xacro" />
   <!-- Camera sensors -->
   <include filename="$(find pr2_description)/urdf/sensors/wge100_camera.urdf.xacro" />
@@ -60,6 +61,22 @@
   <xacro:projector_wg6802418_v0 name="projector_wg6802418" parent="head_plate_frame" >
     <!-- Camera is slightly recessed from front, where is camera origin? Lens? -->
-    <origin xyz="0.046457 0.110 0.0546" rpy="0 0 0" />
+    <origin xyz="0 0.110 0.0546" rpy="0 0 0" />
   </xacro:projector_wg6802418_v0>
+  <!-- Base of Kinect/Prosilica Mount -->
+  <xacro:kinect_prosilica_camera_swept_back_v0 name="head_mount" parent="head_plate_frame" >
+    <origin xyz="-0.137376 0 0.091746" rpy="0 0 0" />
+    <!--
+          Was -0.1 0 0.09225, -0.138 0 0.09225 looks good front back and sheet metal on bolt pattern,
+          -0.138 0 0.06225 is where Prosilica FOV just clears the head.
+          This is 30 mm (!) below the position in SolidWorks.
+          Lowering the Prosilica by this amount in SW makes the FOV hit around the aluminum / plastic junction.
+          Turns out that head_plate_frame is in some random position in space.
+          It is [0.0232 0 0.0645 from its parent, head_tilt_link.
+          The distance from head_plate_frame to the head_kinect_prosilica is 137.376 mm X and 91.746 mm Z.
+          So the origin should in fact be -0.137376 0 0.091746.
+          John is changing the Prosilica FOV based on my numbers.
+          Just need to roscd and svn up.
+    -->
+  </xacro:kinect_prosilica_camera_swept_back_v0>
   <xacro:pr2_tilting_laser_v0 name="laser_tilt" parent="torso_lift_link" laser_calib_ref="0.0">
     <origin xyz="0.09893 0 0.227" rpy="0 0 0" />

File: pr2_description/robots/pr2_no_kinect.urdf.xacro (robot description, xacro)
@@ -24,5 +24,4 @@
   <!-- Head sensors -->
   <include filename="$(find pr2_description)/urdf/sensors/head_sensor_package.urdf.xacro" />
-  <include filename="$(find pr2_description)/urdf/sensors/kinect_prosilica_camera.urdf.xacro" />
   <!-- Camera sensors -->
   <include filename="$(find pr2_description)/urdf/sensors/wge100_camera.urdf.xacro" />
@@ -61,22 +60,6 @@
   <xacro:projector_wg6802418_v0 name="projector_wg6802418" parent="head_plate_frame" >
     <!-- Camera is slightly recessed from front, where is camera origin? Lens? -->
-    <origin xyz="0 0.110 0.0546" rpy="0 0 0" />
+    <origin xyz="0.046457 0.110 0.0546" rpy="0 0 0" />
   </xacro:projector_wg6802418_v0>
-  <!-- Base of Kinect/Prosilica Mount -->
-  <xacro:kinect_prosilica_camera_swept_back_v0 name="head_mount" parent="head_plate_frame" >
-    <origin xyz="-0.137376 0 0.091746" rpy="0 0 0" />
-    <!--
-          Was -0.1 0 0.09225, -0.138 0 0.09225 looks good front back and sheet metal on bolt pattern,
-          -0.138 0 0.06225 is where Prosilica FOV just clears the head.
-          This is 30 mm (!) below the position in SolidWorks.
-          Lowering the Prosilica by this amount in SW makes the FOV hit around the aluminum / plastic junction.
-          Turns out that head_plate_frame is in some random position in space.
-          It is [0.0232 0 0.0645 from its parent, head_tilt_link.
-          The distance from head_plate_frame to the head_kinect_prosilica is 137.376 mm X and 91.746 mm Z.
-          So the origin should in fact be -0.137376 0 0.091746.
-          John is changing the Prosilica FOV based on my numbers.
-          Just need to roscd and svn up.
-    -->
-  </xacro:kinect_prosilica_camera_swept_back_v0>
   <xacro:pr2_tilting_laser_v0 name="laser_tilt" parent="torso_lift_link" laser_calib_ref="0.0">
     <origin xyz="0.09893 0 0.227" rpy="0 0 0" />
