Commit message: Added kinect2 in place of kinect but need to add if to support both, fix camera frames, and fix tf linking. Minor changes to fix tags and new Gazebo requirements (less xmlns in robot tag).

File: pr2_description/robots/pr2.urdf.xacro (robot description, xacro)
@@ -1,8 +1,4 @@
 <?xml version="1.0"?>
-<robot xmlns:sensor="http://playerstage.sourceforge.net/gazebo/xmlschema/#sensor"
-       xmlns:controller="http://playerstage.sourceforge.net/gazebo/xmlschema/#controller"
-       xmlns:interface="http://playerstage.sourceforge.net/gazebo/xmlschema/#interface"
-       xmlns:xacro="http://playerstage.sourceforge.net/gazebo/xmlschema/#interface"
-       name="pr2" >
+<robot name="pr2" xmlns:xacro="http://ros.org/wiki/xacro">
   <!-- The following included files set up definitions of parts of the robot body -->
   <!-- misc common stuff? -->
@@ -79,4 +75,7 @@
     -->
   </xacro:kinect_prosilica_camera_swept_back_v0>
+  <xacro:kinect_mount_v0 name="kinect2_mount" parent="head_mount_link" >
+    <origin xyz="-0.137376 0 0.091746" rpy="0 0 0" />
+  </xacro:kinect_mount_v0>
   <xacro:pr2_tilting_laser_v0 name="laser_tilt" parent="torso_lift_link" laser_calib_ref="0.0">
     <origin xyz="0.09893 0 0.227" rpy="0 0 0" />

File: pr2_description/urdf/sensors/kinect_prosilica_camera.gazebo.xacro (robot description, xacro)
@@ -1,4 +1,4 @@
 <?xml version="1.0"?>
-<root xmlns:xacro="http://ros.org/wiki/xacro">
+<robot xmlns:xacro="http://ros.org/wiki/xacro">
 <xacro:macro name="kinect_ir_gazebo_v0" params="link_name frame_name camera_name">
   <gazebo reference="${link_name}">
@@ -185,3 +185,3 @@
   </gazebo>
 </xacro:macro>
-</root>
+</robot>

File: pr2_description/urdf/sensors/kinect_prosilica_camera.urdf.xacro (robot description, xacro)
@@ -1,16 +1,13 @@
 <?xml version="1.0"?>
-<root xmlns:sensor="http://playerstage.sourceforge.net/gazebo/xmlschema/#sensor"
-      xmlns:controller="http://playerstage.sourceforge.net/gazebo/xmlschema/#controller"
-      xmlns:interface="http://playerstage.sourceforge.net/gazebo/xmlschema/#interface"
-      xmlns:xacro="http://ros.org/wiki/xacro">
+<robot xmlns:xacro="http://ros.org/wiki/xacro">
   <xacro:include filename="$(find pr2_description)/urdf/sensors/kinect_prosilica_camera.gazebo.xacro" />
   <property name="ir_depth_rgb_offset_y" value="0.01"/> <!-- FIXME: what is this offset? -->
-  <!-- kinect and prosilica combo -->
+  <!-- kinect2 combo -->
   <xacro:macro name="kinect_prosilica_camera_swept_back_v0" params="name parent *origin">
-    <!-- stl contains structure + kinect + prosilica combo -->
+    <!-- stl contains structure + kinect2 bracket + kinect2 combo -->
     <joint name="${name}_joint" type="fixed">
       <!-- <limit lower="0.1" upper="0.1" effort="10000" velocity="100.0"/> -->
       <!-- <insert_block name="origin" /> -->
-      <origin xyz="-0.138 0 0.091" rpy="0 0 0"/>
+      <origin xyz="-0.228 -0.148 0.091" rpy="${M_PI/2} 0 ${M_PI/2}"/> <!-- 0.0905 -->
       <parent link="${parent}"/>
       <child link="${name}_link"/>
@@ -25,7 +22,7 @@
       </inertial>
       <visual>
-        <origin xyz="0.0 0.0 0" rpy="0 0 0"/>
+        <origin xyz="0 0 0" rpy="0 0 0"/>
         <geometry>
-          <mesh filename="package://pr2_description/meshes/sensors/kinect_prosilica_v0/115x100_swept_back--coarse.STL" scale="0.001 0.001 0.001" />
+          <mesh filename="package://pr2_description/meshes/sensors/kinect_prosilica_v0/kinect2_mount.STL" scale="0.001 0.001 0.001" />
         </geometry>
         <material name="gray">
@@ -34,7 +31,33 @@
       </visual>
       <collision>
-        <origin xyz="0.0 0.0 0" rpy="0 0 0"/>
+        <origin xyz="0 0 0" rpy="0 0 0"/>
         <geometry>
           <sphere radius="0.0005"/>
+        </geometry>
+      </collision>
+    </link>
+    <joint name="${name}_bracket_joint" type="fixed">
+      <origin xyz="0.148 0.128 0.0321" rpy="${M_PI} ${M_PI} ${M_PI}"/>
+      <parent link="${name}_link"/>
+      <child link="${name}_bracket_link"/>
+    </joint>
+    <link name="${name}_bracket_link">
+      <inertial>
+        <mass value="0.1" />
+        <origin xyz="0 0 0" rpy="0 0 0"/>
+        <inertia ixx="0.01"  ixy="0.0"  ixz="0.0"
+                 iyy="0.01"  iyz="0.0"
+                 izz="0.01" />
+      </inertial>
+      <visual>
+        <origin xyz="0 0 0" rpy="0 0 0"/>
+        <geometry>
+          <mesh filename="package://pr2_description/meshes/sensors/kinect_prosilica_v0/kinect2_bracket.STL" />
+        </geometry>
+      </visual>
+      <collision>
+        <origin xyz="0 0 0" rpy="0 0 0"/>
+        <geometry>
+          <box size="0.15 0.08 0.06" />
         </geometry>
       </collision>
@@ -45,5 +68,5 @@
     -->
     <!-- kinect ir sensor physical attachment -->
-    <joint name="${name}_kinect_ir_joint" type="fixed">
+<!--    <joint name="${name}_kinect_ir_joint" type="fixed">
       <origin xyz="-0.032267 0.0125 0.136453" rpy="0 0 0"/>
       <parent link="${name}_link"/>
@@ -70,7 +93,7 @@
         </geometry>
       </collision>
-    </link>
+    </link> -->
     <!-- kinect ir sensor frame -->
-    <joint name="${name}_kinect_ir_optical_frame_joint" type="fixed">
+<!--    <joint name="${name}_kinect_ir_optical_frame_joint" type="fixed">
       <origin xyz="${cal_kinect_x}            ${cal_kinect_y + ir_depth_rgb_offset_y}         ${cal_kinect_z}"
                 rpy="${-M_PI/2+cal_kinect_roll} ${0.0+cal_kinect_pitch} ${-M_PI/2+cal_kinect_yaw}" />
@@ -78,9 +101,11 @@
       <child link="${name}_kinect_ir_optical_frame"/>
     </joint>
-    <link name="${name}_kinect_ir_optical_frame"/>
+    <link name="${name}_kinect_ir_optical_frame"/> -->
     <!-- gazebo extensions -->
-    <xacro:kinect_ir_gazebo_v0 link_name="${name}_kinect_ir_link" frame_name="${name}_kinect_ir_optical_frame" camera_name="head_mount_kinect" />
+<!--     <xacro:kinect_ir_gazebo_v0 link_name="${name}_kinect_ir_link" frame_name="${name}_kinect_ir_optical_frame" camera_name="head_mount_kinect" />
+ -->
+<!-- kinect2 -->
     <!-- kinect rgb sensor physical attachment -->
-    <joint name="${name}_kinect_rgb_joint" type="fixed">
+<!--     <joint name="${name}_kinect_rgb_joint" type="fixed">
       <origin xyz="0 -0.03 0" rpy="0 0 0"/>
       <parent link="${name}_kinect_ir_link"/>
@@ -107,7 +132,7 @@
         </geometry>
       </collision>
-    </link>
+    </link> -->
     <!-- kinect rgb sensor frame -->
-    <joint name="${name}_kinect_rgb_optical_frame_joint" type="fixed">
+<!--    <joint name="${name}_kinect_rgb_optical_frame_joint" type="fixed">
       <origin xyz="${cal_kinect_x}            ${cal_kinect_y}         ${cal_kinect_z}"
                 rpy="${-M_PI/2+cal_kinect_roll} ${0.0+cal_kinect_pitch} ${-M_PI/2+cal_kinect_yaw}" />
@@ -115,14 +140,13 @@
       <child link="${name}_kinect_rgb_optical_frame"/>
     </joint>
-    <link name="${name}_kinect_rgb_optical_frame"/>
+    <link name="${name}_kinect_rgb_optical_frame"/> -->
     <!-- gazebo extensions -->
-    <xacro:kinect_rgb_gazebo_v0 link_name="${name}_kinect_rgb_link" frame_name="${name}_kinect_rgb_optical_frame" camera_name="head_mount_kinect" />
-    <!-- prosilica sensor physical attachment -->
-    <joint name="${name}_prosilica_joint" type="fixed">
-      <origin xyz="-0.046457 0.0125 0.088921" rpy="0 0 0"/>
-      <parent link="${name}_link"/>
-      <child link="${name}_prosilica_link"/>
+<!--     <xacro:kinect_rgb_gazebo_v0 link_name="${name}_kinect_rgb_link" frame_name="${name}_kinect_rgb_optical_frame" camera_name="head_mount_kinect" /> -->
+    <joint name="${name}_kinect2_joint" type="fixed">
+      <origin xyz="0 0.0255 0.01" rpy="0 0 0"/>
+      <parent link="${name}_bracket_link"/>
+      <child link="${name}_kinect2_link"/>
     </joint>
-    <link name="${name}_prosilica_link">
+    <link name="${name}_kinect2_link">
       <inertial>
         <mass value="0.1" />
@@ -133,26 +157,28 @@
       </inertial>
       <visual>
-        <origin xyz="0.0 0.0 0" rpy="0 0 0"/>
+        <origin xyz="0 0 0" rpy="0 0 0"/>
         <geometry>
-          <sphere radius="0.0005"/>
+          <box size="0.25 0.043 0.067"/>
+          <material name="black">
+            <color rgba="0.05 0.05 0.05 1"/>
+          </material>
         </geometry>
       </visual>
       <collision>
-        <origin xyz="0.0 0.0 0" rpy="0 0 0"/>
+        <origin xyz="0 0 0" rpy="0 0 0"/>
         <geometry>
-          <sphere radius="0.0005"/>
+          <box size="0.25 0.043 0.067"/>
         </geometry>
       </collision>
     </link>
-    <!-- prosilica sensor frame -->
-    <joint name="${name}_prosilica_optical_frame_joint" type="fixed">
-      <origin xyz="${cal_high_def_x}            ${cal_high_def_y}         ${cal_high_def_z}"
-                rpy="${-M_PI/2+cal_high_def_roll} ${0.0+cal_high_def_pitch} ${-M_PI/2+cal_high_def_yaw}" />
-      <parent link="${name}_prosilica_link"/>
-      <child link="${name}_prosilica_optical_frame"/>
+<!--
+    <joint name="${name}_optical_joint" type="fixed">
+      <origin xyz="${cal_kinect_x}            ${cal_kinect_y}         ${cal_kinect_z}"
+                rpy="${-M_PI/2+cal_kinect_roll} ${0.0+cal_kinect_pitch} ${-M_PI/2+cal_kinect_yaw}" />
+      <parent link="${name}_kinect_frame"/>
+      <child link="${name}_optical_frame"/>
     </joint>
-    <link name="${name}_prosilica_optical_frame"/>
-    <!-- gazebo extensions -->
-    <xacro:prosilica_cam_gazebo_v1 link_name="${name}_prosilica_link" camera_name="prosilica_camera" frame_name="${name}_prosilica_optical_frame" />
+    <link name="${name}_optical_frame"/>
+-->
   </xacro:macro>
-</root>
+</robot>

Commit message: Changed link organization and some dimensions.

File: pr2_description/robots/pr2.urdf.xacro (robot description, xacro)
@@ -75,7 +75,4 @@
     -->
   </xacro:kinect_prosilica_camera_swept_back_v0>
-  <xacro:kinect_mount_v0 name="kinect2_mount" parent="head_mount_link" >
-    <origin xyz="-0.137376 0 0.091746" rpy="0 0 0" />
-  </xacro:kinect_mount_v0>
   <xacro:pr2_tilting_laser_v0 name="laser_tilt" parent="torso_lift_link" laser_calib_ref="0.0">
     <origin xyz="0.09893 0 0.227" rpy="0 0 0" />

File: pr2_description/urdf/sensors/kinect_prosilica_camera.urdf.xacro (robot description, xacro)
@@ -8,6 +8,6 @@
     <joint name="${name}_joint" type="fixed">
       <!-- <limit lower="0.1" upper="0.1" effort="10000" velocity="100.0"/> -->
-      <!-- <insert_block name="origin" /> -->
-      <origin xyz="-0.228 -0.148 0.091" rpy="${M_PI/2} 0 ${M_PI/2}"/>
+      <insert_block name="origin" />
+      <!-- <origin xyz="-0.228 -0.148 0.091" rpy="${M_PI/2} 0 ${M_PI/2}"/> -->
       <parent link="${parent}"/>
       <child link="${name}_link"/>
@@ -15,5 +15,5 @@
     <link name="${name}_link">
       <inertial>
-        <mass value="0.1" />
+        <mass value="0.1"/>
         <origin xyz="0 0 0" rpy="0 0 0"/>
         <inertia ixx="0.01"  ixy="0.0"  ixz="0.0"
@@ -22,5 +22,5 @@
       </inertial>
       <visual>
-        <origin xyz="0 0 0" rpy="0 0 0"/>
+        <origin xyz="0 -0.138 0" rpy="${M_PI/2} 0 ${M_PI/2}"/>
         <geometry>
           <mesh filename="package://pr2_description/meshes/sensors/kinect_prosilica_v0/kinect2_mount.STL" scale="0.001 0.001 0.001" />
@@ -44,5 +44,5 @@
     <link name="${name}_bracket_link">
       <inertial>
-        <mass value="0.1" />
+        <mass value="0.1"/>
         <origin xyz="0 0 0" rpy="0 0 0"/>
         <inertia ixx="0.01"  ixy="0.0"  ixz="0.0"
@@ -150,9 +150,9 @@
     <link name="${name}_kinect2_link">
       <inertial>
-        <mass value="0.1" />
+        <mass value="0.1"/>
         <origin xyz="0 0 0" rpy="0 0 0"/>
         <inertia ixx="0.01"  ixy="0.0"  ixz="0.0"
                  iyy="0.01"  iyz="0.0"
-                 izz="0.01" />
+                 izz="0.01"/>
       </inertial>
       <visual>

Commit message: Added parameter passing

File: pr2_description/robots/pr2.urdf.xacro (robot description, xacro)
@@ -24,5 +24,4 @@
   <!-- Head sensors -->
   <xacro:include filename="$(find pr2_description)/urdf/sensors/head_sensor_package.urdf.xacro" />
-  <xacro:include filename="$(find pr2_description)/urdf/sensors/kinect_prosilica_camera.urdf.xacro" />
   <!-- Camera sensors -->
   <xacro:include filename="$(find pr2_description)/urdf/sensors/wge100_camera.urdf.xacro" />
@@ -63,20 +62,4 @@
     <origin xyz="0 0.110 0.0546" rpy="0 0 0" />
   </xacro:projector_wg6802418_v0>
-  <!-- Base of Kinect/Prosilica Mount -->
-  <xacro:kinect_prosilica_camera_swept_back_v0 name="head_mount" parent="head_plate_frame" >
-    <origin xyz="-0.137376 0 0.091746" rpy="0 0 0" />
-    <!--
-          Was -0.1 0 0.09225, -0.138 0 0.09225 looks good front back and sheet metal on bolt pattern,
-          -0.138 0 0.06225 is where Prosilica FOV just clears the head.
-          This is 30 mm (!) below the position in SolidWorks.
-          Lowering the Prosilica by this amount in SW makes the FOV hit around the aluminum / plastic junction.
-          Turns out that head_plate_frame is in some random position in space.
-          It is [0.0232 0 0.0645 from its parent, head_tilt_link.
-          The distance from head_plate_frame to the head_kinect_prosilica is 137.376 mm X and 91.746 mm Z.
-          So the origin should in fact be -0.137376 0 0.091746.
-          John is changing the Prosilica FOV based on my numbers.
-          Just need to roscd and svn up.
-    -->
-  </xacro:kinect_prosilica_camera_swept_back_v0>
   <xacro:pr2_tilting_laser_v0 name="laser_tilt" parent="torso_lift_link" laser_calib_ref="0.0">
     <origin xyz="0.09893 0 0.227" rpy="0 0 0" />
@@ -139,3 +122,32 @@
     <origin xyz=".135 0 .044" rpy="${M_PI/2} ${-32.25*M_PI/180} 0" />
   </xacro:wge100_camera_v0>
+  <!-- Kinect models -->
+  <xacro:arg name="kinect2" default="false"/>
+  <!-- Kinect1 xacro -->
+  <xacro:unless value="$(arg kinect2)">
+    <xacro:include filename="$(find pr2_description)/urdf/sensors/kinect_prosilica_camera.urdf.xacro" />
+    <!-- Base of Kinect/Prosilica Mount -->
+    <xacro:kinect_prosilica_camera_swept_back_v0 name="head_mount" parent="head_plate_frame" >
+      <origin xyz="-0.137376 0 0.091746" rpy="0 0 0" />
+      <!--
+            Was -0.1 0 0.09225, -0.138 0 0.09225 looks good front back and sheet metal on bolt pattern,
+            -0.138 0 0.06225 is where Prosilica FOV just clears the head.
+            This is 30 mm (!) below the position in SolidWorks.
+            Lowering the Prosilica by this amount in SW makes the FOV hit around the aluminum / plastic junction.
+            Turns out that head_plate_frame is in some random position in space.
+            It is [0.0232 0 0.0645 from its parent, head_tilt_link.
+            The distance from head_plate_frame to the head_kinect_prosilica is 137.376 mm X and 91.746 mm Z.
+            So the origin should in fact be -0.137376 0 0.091746.
+            John is changing the Prosilica FOV based on my numbers.
+            Just need to roscd and svn up.
+      -->
+    </xacro:kinect_prosilica_camera_swept_back_v0>
+  </xacro:unless>
+  <!-- Kinect2 xacro -->
+  <xacro:if value="$(arg kinect2)">
+    <xacro:include filename="$(find pr2_description)/urdf/sensors/kinect2.urdf.xacro" />
+    <xacro:kinect2_v0 name="head_mount" parent="head_plate_frame" >
+      <origin xyz="-0.137376 0 0.091746" rpy="0 0 0" />
+    </xacro:kinect2_v0>
+  </xacro:if>
 </robot>

File: pr2_description/test.urdf (robot description, URDF)
Before this commit: robot pr2, 93 links, 92 joints
Joints:
- joint head_mount_kinect2_ir_optical_frame_joint: origin (none) -> xyz=0.0                  0.01 0.0 rpy=-1.57079632679       0.0               -1.57079632679
- joint head_mount_kinect2_rgb_optical_frame_joint: origin (none) -> xyz=0.0            0.0                 0.0 rpy=-1.57079632679 0.0         -1.57079632679

File: pr2_description/urdf/sensors/kinect2.urdf.xacro (robot description, xacro)
@@ -3,5 +3,5 @@
   <xacro:include filename="$(find pr2_description)/urdf/sensors/kinect2.gazebo.xacro" />
   <property name="ir_depth_rgb_offset_y" value="0.01"/> <!-- FIXME: what is this offset? -->
-  <!-- frame + Kinect2 mount + Kinect2 combo -->
+  <!-- Kinect2 and mount assembly -->
   <xacro:macro name="kinect2_v0" params="name parent *origin">
     <joint name="${name}_joint" type="fixed">
@@ -63,6 +63,6 @@
     <!-- kinect2 ir sensor frame -->
     <joint name="${name}_kinect2_ir_optical_frame_joint" type="fixed">
-<!--       <origin xyz="${cal_kinect_x}                         ${cal_kinect_y + ir_depth_rgb_offset_y} {cal_kinect_z}"
-              rpy="${-M_PI/2+cal_kinect_roll}              ${0.0+cal_kinect_pitch}                 ${-M_PI/2+cal_kinect_yaw}" /> -->
+      <origin xyz="${cal_kinect_x}                  ${cal_kinect_y+ir_depth_rgb_offset_y} ${cal_kinect_z}"
+              rpy="${-M_PI/2+cal_kinect_roll}       ${0.0+cal_kinect_pitch}               ${-M_PI/2+cal_kinect_yaw}" />
       <parent link="${name}_kinect2_ir_link"/>
       <child link="${name}_kinect2_ir_optical_frame"/>
@@ -86,6 +86,6 @@
       </inertial>
       <visual>
-<!--         <origin xyz="${cal_kinect_x}            ${cal_kinect_y}            ${cal_kinect_z}"
-                rpy="${-M_PI/2+cal_kinect_roll} ${0.0+cal_kinect_pitch}    ${-M_PI/2+cal_kinect_yaw}" /> -->
+        <origin xyz="${cal_kinect_x}            ${cal_kinect_y}                 ${cal_kinect_z}"
+                rpy="${-M_PI/2+cal_kinect_roll} ${0.0+cal_kinect_pitch}         ${-M_PI/2+cal_kinect_yaw}" />
         <geometry>
           <sphere radius="0.0005"/>
@@ -101,6 +101,6 @@
     <!-- kinect2 rgb sensor frame -->
     <joint name="${name}_kinect2_rgb_optical_frame_joint" type="fixed">
-<!--       <origin xyz="${cal_kinect_x}            ${cal_kinect_y}            ${cal_kinect_z}"
-              rpy="${-M_PI/2+cal_kinect_roll} ${0.0+cal_kinect_pitch}    ${-M_PI/2+cal_kinect_yaw}" /> -->
+      <origin xyz="${cal_kinect_x}            ${cal_kinect_y}                 ${cal_kinect_z}"
+              rpy="${-M_PI/2+cal_kinect_roll} ${0.0+cal_kinect_pitch}         ${-M_PI/2+cal_kinect_yaw}" />
       <parent link="${name}_kinect2_rgb_link"/>
       <child link="${name}_kinect2_rgb_optical_frame"/>

Commit message: Added sanity checking in .xacro so no errors pop up if both KINECT2 and KINECT1 are set true

File: pr2_description/robots/pr2.urdf.xacro (robot description, xacro)
@@ -123,24 +123,4 @@
   </xacro:wge100_camera_v0>
   <!-- Kinect models -->
-  <!-- Kinect1 xacro -->
-  <xacro:if value="$(optenv KINECT1 false)">
-    <xacro:include filename="$(find pr2_description)/urdf/sensors/kinect_prosilica_camera.urdf.xacro" />
-    <!-- Base of Kinect/Prosilica Mount -->
-    <xacro:kinect_prosilica_camera_swept_back_v0 name="head_mount" parent="head_plate_frame" >
-      <origin xyz="-0.137376 0 0.091746" rpy="0 0 0" />
-      <!--
-            Was -0.1 0 0.09225, -0.138 0 0.09225 looks good front back and sheet metal on bolt pattern,
-            -0.138 0 0.06225 is where Prosilica FOV just clears the head.
-            This is 30 mm (!) below the position in SolidWorks.
-            Lowering the Prosilica by this amount in SW makes the FOV hit around the aluminum / plastic junction.
-            Turns out that head_plate_frame is in some random position in space.
-            It is [0.0232 0 0.0645 from its parent, head_tilt_link.
-            The distance from head_plate_frame to the head_kinect_prosilica is 137.376 mm X and 91.746 mm Z.
-            So the origin should in fact be -0.137376 0 0.091746.
-            John is changing the Prosilica FOV based on my numbers.
-            Just need to roscd and svn up.
-      -->
-    </xacro:kinect_prosilica_camera_swept_back_v0>
-  </xacro:if>
   <!-- Kinect2 xacro -->
   <xacro:if value="$(optenv KINECT2 false)">
@@ -150,3 +130,25 @@
     </xacro:kinect2_v0>
   </xacro:if>
+  <!-- Kinect1 xacro -->
+  <xacro:unless value="$(optenv KINECT2 false">
+    <xacro:if value="$(optenv KINECT1 false)">
+      <xacro:include filename="$(find pr2_description)/urdf/sensors/kinect_prosilica_camera.urdf.xacro" />
+      <!-- Base of Kinect/Prosilica Mount -->
+      <xacro:kinect_prosilica_camera_swept_back_v0 name="head_mount" parent="head_plate_frame" >
+        <origin xyz="-0.137376 0 0.091746" rpy="0 0 0" />
+        <!--
+              Was -0.1 0 0.09225, -0.138 0 0.09225 looks good front back and sheet metal on bolt pattern,
+              -0.138 0 0.06225 is where Prosilica FOV just clears the head.
+              This is 30 mm (!) below the position in SolidWorks.
+              Lowering the Prosilica by this amount in SW makes the FOV hit around the aluminum / plastic junction.
+              Turns out that head_plate_frame is in some random position in space.
+              It is [0.0232 0 0.0645 from its parent, head_tilt_link.
+              The distance from head_plate_frame to the head_kinect_prosilica is 137.376 mm X and 91.746 mm Z.
+              So the origin should in fact be -0.137376 0 0.091746.
+              John is changing the Prosilica FOV based on my numbers.
+              Just need to roscd and svn up.
+        -->
+      </xacro:kinect_prosilica_camera_swept_back_v0>
+    </xacro:if>
+  </xacro:unless>
 </robot>
