Commit message: allow pr2.urdf.xacro to accept customized calibration values
1. add calibration parameters in separate xacro files
2. in urdf/shoulder_v0/shoulder.urdf.xacro,
we detect if parameters shoulder_pan_calibi, upper_arm_roll_calib equal to 0.
If equal, use the default values.
If not equal, use the passing values.

File: pr2_description/robots/pr2.urdf.xacro (robot description, xacro)
@@ -58,5 +58,5 @@
     <origin xyz="0 0.110 0.0546" rpy="0 0 0" />
   </xacro:projector_wg6802418_v0>
-  <xacro:pr2_tilting_laser_v0 name="laser_tilt" parent="torso_lift_link" laser_calib_ref="0.0">
+  <xacro:pr2_tilting_laser_v0 name="laser_tilt" parent="torso_lift_link" laser_calib="0.0">
     <origin xyz="0.09893 0 0.227" rpy="0 0 0" />
   </xacro:pr2_tilting_laser_v0>

File: pr2_description/urdf/forearm_v0/forearm.urdf.xacro (robot description, xacro)
@@ -8,5 +8,7 @@
   <xacro:include filename="$(find pr2_description)/urdf/common.xacro" />
   <!-- ============================   Forearm   ============================ -->
-  <xacro:macro name="pr2_forearm_v0" params="side parent reflect *origin">
+  <xacro:macro name="pr2_forearm_v0" params="side parent reflect *origin
+    wrist_flex_calib:=${-0.5410521+cal_r_wrist_flex_flag}
+    wrist_roll_calib:=${-M_PI/2+cal_r_wrist_roll_flag}">
     <joint name="${side}_forearm_joint" type="fixed">
       <xacro:insert_block name="origin" /> <!-- transform from parent link to this joint frame -->
@@ -42,5 +44,5 @@
       <safety_controller k_position="20" k_velocity="4" soft_upper_limit="${0.0 - 0.10}" soft_lower_limit="${-2.18 + 0.18}" />
       <dynamics damping="0.1" />
-      <calibration falling="${-0.5410521 + cal_r_wrist_flex_flag}" />
+      <calibration falling="${wrist_flex_calib}" />
       <origin xyz="0.321 0 0" rpy="0 0 0" />
       <parent link="${side}_forearm_link"/>
@@ -75,5 +77,5 @@
       <safety_controller k_velocity="2" />
       <dynamics damping="0.1" />
-      <calibration rising="${-M_PI / 2 + cal_r_wrist_roll_flag}" />
+      <calibration rising="${wrist_roll_calib}" />
       <origin xyz="0 0 0" rpy="0 0 0" />
       <parent link="${side}_wrist_flex_link"/>

File: pr2_description/urdf/head_v0/head.urdf.xacro (robot description, xacro)
@@ -4,10 +4,10 @@
   <xacro:include filename="$(find pr2_description)/urdf/head_v0/head.transmission.xacro" />
   <xacro:property name="M_PI" value="3.1415926535897931" />
-  <xacro:macro name="pr2_head_pan_v0" params="name parent *origin">
+  <xacro:macro name="pr2_head_pan_v0" params="name parent *origin head_pan_calib">
     <joint name="${name}_joint" type="revolute">
       <axis xyz="0 0 1" />
       <limit lower="-3.007" upper="3.007" effort="2.645" velocity="6" /> <!-- alpha tested velocity and effort limits -->
       <safety_controller k_velocity="1.5" soft_lower_limit="${-3.007+0.15}" soft_upper_limit="${3.007-0.15}" k_position="100" />
-      <calibration rising="0.0" />
+      <calibration rising="${head_pan_calib}" />
       <dynamics damping="0.5" />
       <xacro:insert_block name="origin" />
@@ -38,10 +38,10 @@
     <xacro:pr2_head_pan_transmission_v0 name="${name}" />
   </xacro:macro>
-  <xacro:macro name="pr2_head_tilt_v0" params="name parent *origin">
+  <xacro:macro name="pr2_head_tilt_v0" params="name parent *origin head_tilt_calib">
     <joint name="${name}_joint" type="revolute">
       <axis xyz="0 1 0" />
       <limit lower="-0.471238" upper="1.39626" effort="18" velocity="5" /> <!-- alpha tested velocity and effort limits -->
       <safety_controller k_velocity="3.0" soft_lower_limit="${-0.4712 + 0.1}" soft_upper_limit="${1.39626 - 0.1}" k_position="100" />
-      <calibration falling="${0.0+cal_head_tilt_flag}" />
+      <calibration falling="${head_tilt_calib}" />
       <dynamics damping="10.0" />
       <xacro:insert_block name="origin" />
@@ -74,9 +74,9 @@
     <xacro:pr2_head_tilt_transmission_v0 name="${name}" />
   </xacro:macro>
-  <xacro:macro name="pr2_head_v0" params="name parent *origin">
-    <xacro:pr2_head_pan_v0 name="${name}_pan" parent="${parent}">
+  <xacro:macro name="pr2_head_v0" params="name parent *origin head_pan_calib:=0.0 head_tilt_calib:=${0.0+cal_head_tilt_flag}">
+    <xacro:pr2_head_pan_v0 name="${name}_pan" parent="${parent}" head_pan_calib="${head_pan_calib}">
       <xacro:insert_block name="origin" />
     </xacro:pr2_head_pan_v0>
-    <xacro:pr2_head_tilt_v0 name="${name}_tilt" parent="${name}_pan_link">
+    <xacro:pr2_head_tilt_v0 name="${name}_tilt" parent="${name}_pan_link" head_tilt_calib="${head_tilt_calib}">
       <origin xyz="0.068 0 0" rpy="0 0 0" />
     </xacro:pr2_head_tilt_v0>

File: pr2_description/urdf/shoulder_v0/shoulder.urdf.xacro (robot description, xacro)
@@ -10,5 +10,9 @@
   <xacro:property name="shoulder_lift_radius" value="0.12" />  <!--TODO Define and give source-->
  <!-- ============================   Shoulder   ============================ -->
-  <xacro:macro name="pr2_shoulder_v0" params="side parent reflect *origin">
+  <xacro:macro name="pr2_shoulder_v0" params="side parent reflect *origin
+   shoulder_pan_calib:=0.0
+   shoulder_lift_calib:=${cal_r_shoulder_lift_flag}
+   upper_arm_roll_calib:=0.0">
+    <xacro:property name="the_length" value="4.5" />
     <!-- Shoulder pan -->
     <joint name="${side}_shoulder_pan_joint" type="revolute">
@@ -24,5 +28,10 @@
                          soft_upper_limit="${reflect*M_PI/4+1.5-0.15}" />
       <!-- joint angle when the rising or the falling flag is activated on PR2 -->
-      <calibration  rising="${(reflect*M_PI/4)*cal_r_shoulder_pan_gearing+cal_r_shoulder_pan_flag}" />
+      <xacro:if value="${shoulder_pan_calib == '0.0'}">
+        <calibration  rising="${(reflect*M_PI/4)*cal_r_shoulder_pan_gearing+cal_r_shoulder_pan_flag}" />
+      </xacro:if>
+      <xacro:unless value="${shoulder_pan_calib == '0.0'}">
+        <calibration  rising="${shoulder_pan_calib}" />
+      </xacro:unless>
     </joint>
     <link name="${side}_shoulder_pan_link">
@@ -56,5 +65,5 @@
       <safety_controller k_position="100" k_velocity="10"
                          soft_lower_limit="${-0.5236+0.17}" soft_upper_limit="${1.3963-0.10}" />
-      <calibration falling="${cal_r_shoulder_lift_flag}" />
+      <calibration falling="${shoulder_lift_calib}" />
       <dynamics damping="10.0" />
       <origin xyz="0.1 0 0" rpy="0 0 0" />
@@ -85,5 +94,6 @@
     </link>
     <!-- Upper arm roll is separate macro -->
-    <xacro:pr2_upper_arm_roll_v0 side="${side}" parent="${side}_shoulder_lift_link" reflect="${reflect}" >
+    <xacro:pr2_upper_arm_roll_v0 side="${side}" parent="${side}_shoulder_lift_link" reflect="${reflect}"
+                                 upper_arm_roll_calib="${upper_arm_roll_calib}">
       <origin xyz="0 0 0" rpy="0 0 0" />
     </xacro:pr2_upper_arm_roll_v0>
@@ -93,6 +103,7 @@
   </xacro:macro>
   <!-- Upperarm roll: internal fixed attchment point for upper arm -->
-  <xacro:macro name="pr2_upper_arm_roll_v0" params="side parent reflect *origin">
-    <joint name="${side}_upper_arm_roll_joint" type="revolute">
+  <xacro:macro name="pr2_upper_arm_roll_v0" params="side parent reflect *origin
+    upper_arm_roll_calib">
+    <joint name="${side}_upper_arm_roll_joint" type="revolute" >
       <axis xyz="1 0 0" />
       <xacro:insert_block name="origin" />
@@ -101,5 +112,10 @@
       <limit lower="${reflect*1.55-2.35}" upper="${reflect*1.55+2.35}" effort="30" velocity="${VELOCITY_LIMIT_SCALE*5.45}" /> <!-- alpha tested velocity and effort limits -->
       <safety_controller k_position="100" k_velocity="2" soft_lower_limit="${reflect*1.55-2.35+0.15}" soft_upper_limit="${reflect*1.55+2.35-0.15}" />
-      <calibration rising="${(reflect*M_PI/2)*cal_r_upper_arm_roll_gearing + cal_r_upper_arm_roll_flag}" />
+      <xacro:if value="${upper_arm_roll_calib == '0.0'}">
+        <calibration  rising="${(reflect*M_PI/2)*cal_r_upper_arm_roll_gearing+cal_r_upper_arm_roll_flag}" />
+      </xacro:if>
+      <xacro:unless value="${upper_arm_roll_calib == '0.0'}">
+        <calibration  rising="${upper_arm_roll_calib}" />
+      </xacro:unless>
       <dynamics damping="0.1" />
     </joint>

File: pr2_description/urdf/tilting_laser_v0/tilting_laser.urdf.xacro (robot description, xacro)
@@ -4,10 +4,10 @@
   <xacro:include filename="$(find pr2_description)/urdf/tilting_laser_v0/tilting_laser.transmission.xacro" />
   <xacro:include filename="$(find pr2_description)/urdf/sensors/hokuyo_lx30_laser.urdf.xacro" />
-  <xacro:macro name="pr2_tilting_laser_v0" params="name parent laser_calib_ref *origin">
+  <xacro:macro name="pr2_tilting_laser_v0" params="name parent laser_calib *origin">
     <joint name="${name}_mount_joint" type="revolute">
       <axis xyz="0 1 0" />
       <limit lower="-0.7854" upper="1.48353" effort="0.65" velocity="10.0" /> <!-- alpha tested velocity and effort limits -->
       <safety_controller k_position="100" k_velocity="0.05" soft_lower_limit="${-0.7854+0.05}" soft_upper_limit="${1.48353-0.05}" />
-      <calibration falling="${laser_calib_ref}" />
+      <calibration falling="${laser_calib}" />
       <dynamics damping="0.008" />
       <xacro:insert_block name="origin" />

File: pr2_description/urdf/torso_v0/torso.urdf.xacro (robot description, xacro)
@@ -4,10 +4,10 @@
   <xacro:include filename="$(find pr2_description)/urdf/torso_v0/torso.transmission.xacro" />
   <xacro:include filename="$(find pr2_description)/urdf/sensors/microstrain_3dmgx2_imu.urdf.xacro" />
-  <xacro:macro name="pr2_torso_v0" params="name parent *origin">
+  <xacro:macro name="pr2_torso_v0" params="name parent *origin torso_calib:=0.00475">
     <joint name="${name}_joint" type="prismatic">
       <axis xyz="0 0 1" />
       <limit lower="0.0" upper="0.33" effort="10000" velocity="0.013"/> <!-- alpha tested velocity and effort limits -->
       <safety_controller  k_velocity="2000000" soft_lower_limit="${0.0+0.0115}" soft_upper_limit="${0.33-0.005}" k_position="100" />
-      <calibration falling="0.00475" />
+      <calibration falling="${torso_calib}" />
       <dynamics damping="20000.0" />
       <xacro:insert_block name="origin" />

File: pr2_description/urdf/upper_arm_v0/upper_arm.urdf.xacro (robot description, xacro)
@@ -28,5 +28,7 @@
   <!-- ============================   Upper Arm   ============================ -->
   <!-- Includes elbow flex, FA roll joints in macros below -->
-  <xacro:macro name="pr2_upper_arm_v0" params="side parent reflect">
+  <xacro:macro name="pr2_upper_arm_v0" params="side parent reflect
+   forearm_roll_calib:=${0.0+cal_r_forearm_roll_flag}
+   elbow_flex_calib:=${-1.1606+cal_r_elbow_flex_flag}">
     <joint name="${side}_upper_arm_joint" type="fixed">
       <origin xyz="0 0 0" rpy="0 0 0" />
@@ -64,8 +66,11 @@
     <!-- No transmission, since this a fixed joint w/o actuator -->
     <!-- Elbow flex, FA roll macros -->
-    <xacro:pr2_forearm_roll_v0 side="${side}" parent="${side}_elbow_flex_link" reflect="${reflect}" />
-    <xacro:pr2_elbow_flex_v0 side="${side}" parent="${side}_upper_arm_link" reflect="${reflect}" />
+    <xacro:pr2_forearm_roll_v0 side="${side}" parent="${side}_elbow_flex_link" reflect="${reflect}"
+                               forearm_roll_calib="${forearm_roll_calib}"/>
+    <xacro:pr2_elbow_flex_v0 side="${side}" parent="${side}_upper_arm_link" reflect="${reflect}"
+                             elbow_flex_calib="${elbow_flex_calib}"/>
   </xacro:macro>
-  <xacro:macro name="pr2_elbow_flex_v0" params="side parent reflect">
+  <xacro:macro name="pr2_elbow_flex_v0" params="side parent reflect
+   elbow_flex_calib">
     <!-- Elbow flex -->
     <joint name="${side}_elbow_flex_joint" type="revolute">
@@ -74,5 +79,5 @@
       <limit lower="-2.3213" upper="0.00" effort="30" velocity="${VELOCITY_LIMIT_SCALE*5.5}" /> <!-- alpha tested velocity and effort limits -->
       <safety_controller k_position="100" k_velocity="3" soft_lower_limit="${-2.3213+0.2}" soft_upper_limit="${0.00-0.15}" />
-      <calibration falling="${-1.1606 + cal_r_elbow_flex_flag}"/>
+      <calibration falling="${elbow_flex_calib}"/>
       <dynamics damping="1.0" />
       <origin xyz="0.4 0 0" rpy="0 0 0" />
@@ -106,5 +111,6 @@
   </xacro:macro>
   <!-- FA roll joint only -->
-  <xacro:macro name="pr2_forearm_roll_v0" params="side parent reflect">
+  <xacro:macro name="pr2_forearm_roll_v0" params="side parent reflect
+   forearm_roll_calib">
     <!-- forearm_roll_link is a fictitious link internal to elbow_flex_link, provides an attachment point for the actual forearm -->
     <joint name="${side}_forearm_roll_joint" type="continuous">
@@ -112,5 +118,5 @@
       <limit effort="30" velocity="${VELOCITY_LIMIT_SCALE*6}" /> <!-- alpha tested velocity and effort limits -->
       <safety_controller k_velocity="1" />
-      <calibration rising="${0.0 + cal_r_forearm_roll_flag}" />
+      <calibration rising="${forearm_roll_calib}" />
       <dynamics damping="0.1" />
       <origin xyz="0 0 0" rpy="0 0 0" />
