Commit message: make all calibration parameter name consistent

File: pr2_description/robots/pr2.urdf.xacro (robot description, xacro)
@@ -58,5 +58,5 @@
     <origin xyz="0 0.110 0.0546" rpy="0 0 0" />
   </xacro:projector_wg6802418_v0>
-  <xacro:pr2_tilting_laser_v0 name="laser_tilt" parent="torso_lift_link" laser_calib="0.0">
+  <xacro:pr2_tilting_laser_v0 name="laser_tilt" parent="torso_lift_link" laser_calib_ref="0.0">
     <origin xyz="0.09893 0 0.227" rpy="0 0 0" />
   </xacro:pr2_tilting_laser_v0>

File: pr2_description/robots/pr2_no_arms.urdf.xacro (robot description, xacro)
@@ -52,5 +52,5 @@
     <origin xyz="0.0 0.0 0.0" rpy="0 0 0" />
   </xacro:pr2_head_sensor_package_v0>
-  <xacro:pr2_tilting_laser_v0 name="laser_tilt" parent="torso_lift_link" laser_calib="0.0">
+  <xacro:pr2_tilting_laser_v0 name="laser_tilt" parent="torso_lift_link" laser_calib_ref="0.0">
     <origin xyz="0.1 0 0.235" rpy="0 0 0" />
   </xacro:pr2_tilting_laser_v0>

File: pr2_description/robots/pr2_no_kinect.urdf.xacro (robot description, xacro)
@@ -58,5 +58,5 @@
     <origin xyz="0.046457 0.110 0.0546" rpy="0 0 0" />
   </xacro:projector_wg6802418_v0>
-  <xacro:pr2_tilting_laser_v0 name="laser_tilt" parent="torso_lift_link" laser_calib="0.0">
+  <xacro:pr2_tilting_laser_v0 name="laser_tilt" parent="torso_lift_link" laser_calib_ref="0.0">
     <origin xyz="0.09893 0 0.227" rpy="0 0 0" />
   </xacro:pr2_tilting_laser_v0>

File: pr2_description/robots/pr2_se.urdf.xacro (robot description, xacro)
@@ -68,5 +68,5 @@
   </xacro:projector_wg6802418_v0>
   -->
-  <xacro:pr2_tilting_laser_v0 name="laser_tilt" parent="torso_lift_link" laser_calib="0.0">
+  <xacro:pr2_tilting_laser_v0 name="laser_tilt" parent="torso_lift_link" laser_calib_ref="0.0">
     <origin xyz="0.09893 0 0.227" rpy="0 0 0" />
   </xacro:pr2_tilting_laser_v0>

File: pr2_description/urdf/forearm_v0/forearm.urdf.xacro (robot description, xacro)
@@ -9,6 +9,6 @@
   <!-- ============================   Forearm   ============================ -->
   <xacro:macro name="pr2_forearm_v0" params="side parent reflect *origin
-    wrist_flex_calib:=${-0.5410521+cal_r_wrist_flex_flag}
-    wrist_roll_calib:=${-M_PI/2+cal_r_wrist_roll_flag}">
+    wrist_flex_calib_ref:=0.0
+    wrist_roll_calib_ref:=0.0">
     <joint name="${side}_forearm_joint" type="fixed">
       <xacro:insert_block name="origin" /> <!-- transform from parent link to this joint frame -->
@@ -44,5 +44,10 @@
       <safety_controller k_position="20" k_velocity="4" soft_upper_limit="${0.0 - 0.10}" soft_lower_limit="${-2.18 + 0.18}" />
       <dynamics damping="0.1" />
-      <calibration falling="${wrist_flex_calib}" />
+      <xacro:unless value="${wrist_flex_calib_ref}">
+        <calibration  falling="${-0.5410521+cal_r_wrist_flex_flag}" />
+      </xacro:unless>
+      <xacro:if value="${wrist_flex_calib_ref}">
+        <calibration  falling="${wrist_flex_calib_ref}" />
+      </xacro:if>
       <origin xyz="0.321 0 0" rpy="0 0 0" />
       <parent link="${side}_forearm_link"/>
@@ -77,5 +82,10 @@
       <safety_controller k_velocity="2" />
       <dynamics damping="0.1" />
-      <calibration rising="${wrist_roll_calib}" />
+      <xacro:unless value="${wrist_roll_calib_ref}">
+        <calibration rising="${-M_PI/2+cal_r_wrist_roll_flag}" />
+      </xacro:unless>
+      <xacro:if value="${wrist_roll_calib_ref}">
+        <calibration  rising="${wrist_roll_calib_ref}" />
+      </xacro:if>
       <origin xyz="0 0 0" rpy="0 0 0" />
       <parent link="${side}_wrist_flex_link"/>

File: pr2_description/urdf/head_v0/head.urdf.xacro (robot description, xacro)
@@ -4,10 +4,10 @@
   <xacro:include filename="$(find pr2_description)/urdf/head_v0/head.transmission.xacro" />
   <xacro:property name="M_PI" value="3.1415926535897931" />
-  <xacro:macro name="pr2_head_pan_v0" params="name parent *origin head_pan_calib">
+  <xacro:macro name="pr2_head_pan_v0" params="name parent *origin head_pan_calib_ref">
     <joint name="${name}_joint" type="revolute">
       <axis xyz="0 0 1" />
       <limit lower="-3.007" upper="3.007" effort="2.645" velocity="6" /> <!-- alpha tested velocity and effort limits -->
       <safety_controller k_velocity="1.5" soft_lower_limit="${-3.007+0.15}" soft_upper_limit="${3.007-0.15}" k_position="100" />
-      <calibration rising="${head_pan_calib}" />
+      <calibration rising="${head_pan_calib_ref}" />
       <dynamics damping="0.5" />
       <xacro:insert_block name="origin" />
@@ -38,10 +38,15 @@
     <xacro:pr2_head_pan_transmission_v0 name="${name}" />
   </xacro:macro>
-  <xacro:macro name="pr2_head_tilt_v0" params="name parent *origin head_tilt_calib">
+  <xacro:macro name="pr2_head_tilt_v0" params="name parent *origin head_tilt_calib_ref">
     <joint name="${name}_joint" type="revolute">
       <axis xyz="0 1 0" />
       <limit lower="-0.471238" upper="1.39626" effort="18" velocity="5" /> <!-- alpha tested velocity and effort limits -->
       <safety_controller k_velocity="3.0" soft_lower_limit="${-0.4712 + 0.1}" soft_upper_limit="${1.39626 - 0.1}" k_position="100" />
-      <calibration falling="${head_tilt_calib}" />
+      <xacro:unless value="${head_tilt_calib_ref}">
+        <calibration  falling="${0.0+cal_head_tilt_flag}" />
+      </xacro:unless>
+      <xacro:if value="${head_tilt_calib_ref}">
+        <calibration  falling="${head_tilt_calib_ref}" />
+      </xacro:if>
       <dynamics damping="10.0" />
       <xacro:insert_block name="origin" />
@@ -74,9 +79,11 @@
     <xacro:pr2_head_tilt_transmission_v0 name="${name}" />
   </xacro:macro>
-  <xacro:macro name="pr2_head_v0" params="name parent *origin head_pan_calib:=0.0 head_tilt_calib:=${0.0+cal_head_tilt_flag}">
-    <xacro:pr2_head_pan_v0 name="${name}_pan" parent="${parent}" head_pan_calib="${head_pan_calib}">
+  <xacro:macro name="pr2_head_v0" params="name parent *origin
+  head_pan_calib_ref:=0.0
+  head_tilt_calib_ref:=0.0 ">
+    <xacro:pr2_head_pan_v0 name="${name}_pan" parent="${parent}" head_pan_calib_ref="${head_pan_calib_ref}">
       <xacro:insert_block name="origin" />
     </xacro:pr2_head_pan_v0>
-    <xacro:pr2_head_tilt_v0 name="${name}_tilt" parent="${name}_pan_link" head_tilt_calib="${head_tilt_calib}">
+    <xacro:pr2_head_tilt_v0 name="${name}_tilt" parent="${name}_pan_link" head_tilt_calib_ref="${head_tilt_calib_ref}">
       <origin xyz="0.068 0 0" rpy="0 0 0" />
     </xacro:pr2_head_tilt_v0>

File: pr2_description/urdf/shoulder_v0/shoulder.urdf.xacro (robot description, xacro)
@@ -11,8 +11,7 @@
  <!-- ============================   Shoulder   ============================ -->
   <xacro:macro name="pr2_shoulder_v0" params="side parent reflect *origin
-   shoulder_pan_calib:=0.0
-   shoulder_lift_calib:=${cal_r_shoulder_lift_flag}
-   upper_arm_roll_calib:=0.0">
-    <xacro:property name="the_length" value="4.5" />
+   shoulder_pan_calib_ref:=0.0
+   shoulder_lift_calib_ref:=0.0
+   upper_arm_roll_calib_ref:=0.0">
     <!-- Shoulder pan -->
     <joint name="${side}_shoulder_pan_joint" type="revolute">
@@ -28,10 +27,10 @@
                          soft_upper_limit="${reflect*M_PI/4+1.5-0.15}" />
       <!-- joint angle when the rising or the falling flag is activated on PR2 -->
-      <xacro:if value="${shoulder_pan_calib == '0.0'}">
+      <xacro:unless value="${shoulder_pan_calib_ref}">
         <calibration  rising="${(reflect*M_PI/4)*cal_r_shoulder_pan_gearing+cal_r_shoulder_pan_flag}" />
+      </xacro:unless>
+      <xacro:if value="${shoulder_pan_calib_ref}">
+        <calibration  rising="${shoulder_pan_calib_ref}" />
       </xacro:if>
-      <xacro:unless value="${shoulder_pan_calib == '0.0'}">
-        <calibration  rising="${shoulder_pan_calib}" />
-      </xacro:unless>
     </joint>
     <link name="${side}_shoulder_pan_link">
@@ -65,5 +64,10 @@
       <safety_controller k_position="100" k_velocity="10"
                          soft_lower_limit="${-0.5236+0.17}" soft_upper_limit="${1.3963-0.10}" />
-      <calibration falling="${shoulder_lift_calib}" />
+      <xacro:unless value="${shoulder_lift_calib_ref}">
+        <calibration falling="${cal_r_shoulder_lift_flag}" />
+      </xacro:unless>
+      <xacro:if value="${shoulder_lift_calib_ref}">
+        <calibration falling="${shoulder_lift_calib_ref}" />
+      </xacro:if>
       <dynamics damping="10.0" />
       <origin xyz="0.1 0 0" rpy="0 0 0" />
@@ -95,5 +99,5 @@
     <!-- Upper arm roll is separate macro -->
     <xacro:pr2_upper_arm_roll_v0 side="${side}" parent="${side}_shoulder_lift_link" reflect="${reflect}"
-                                 upper_arm_roll_calib="${upper_arm_roll_calib}">
+                                 upper_arm_roll_calib_ref="${upper_arm_roll_calib_ref}">
       <origin xyz="0 0 0" rpy="0 0 0" />
     </xacro:pr2_upper_arm_roll_v0>
@@ -104,5 +108,5 @@
   <!-- Upperarm roll: internal fixed attchment point for upper arm -->
   <xacro:macro name="pr2_upper_arm_roll_v0" params="side parent reflect *origin
-    upper_arm_roll_calib">
+    upper_arm_roll_calib_ref">
     <joint name="${side}_upper_arm_roll_joint" type="revolute" >
       <axis xyz="1 0 0" />
@@ -112,10 +116,10 @@
       <limit lower="${reflect*1.55-2.35}" upper="${reflect*1.55+2.35}" effort="30" velocity="${VELOCITY_LIMIT_SCALE*5.45}" /> <!-- alpha tested velocity and effort limits -->
       <safety_controller k_position="100" k_velocity="2" soft_lower_limit="${reflect*1.55-2.35+0.15}" soft_upper_limit="${reflect*1.55+2.35-0.15}" />
-      <xacro:if value="${upper_arm_roll_calib == '0.0'}">
+      <xacro:unless value="${upper_arm_roll_calib_ref}">
         <calibration  rising="${(reflect*M_PI/2)*cal_r_upper_arm_roll_gearing+cal_r_upper_arm_roll_flag}" />
+      </xacro:unless>
+      <xacro:if value="${upper_arm_roll_calib_ref}">
+        <calibration  rising="${upper_arm_roll_calib_ref}" />
       </xacro:if>
-      <xacro:unless value="${upper_arm_roll_calib == '0.0'}">
-        <calibration  rising="${upper_arm_roll_calib}" />
-      </xacro:unless>
       <dynamics damping="0.1" />
     </joint>

File: pr2_description/urdf/tilting_laser_v0/tilting_laser.urdf.xacro (robot description, xacro)
@@ -4,10 +4,10 @@
   <xacro:include filename="$(find pr2_description)/urdf/tilting_laser_v0/tilting_laser.transmission.xacro" />
   <xacro:include filename="$(find pr2_description)/urdf/sensors/hokuyo_lx30_laser.urdf.xacro" />
-  <xacro:macro name="pr2_tilting_laser_v0" params="name parent laser_calib *origin">
+  <xacro:macro name="pr2_tilting_laser_v0" params="name parent laser_calib_ref *origin">
     <joint name="${name}_mount_joint" type="revolute">
       <axis xyz="0 1 0" />
       <limit lower="-0.7854" upper="1.48353" effort="0.65" velocity="10.0" /> <!-- alpha tested velocity and effort limits -->
       <safety_controller k_position="100" k_velocity="0.05" soft_lower_limit="${-0.7854+0.05}" soft_upper_limit="${1.48353-0.05}" />
-      <calibration falling="${laser_calib}" />
+      <calibration falling="${laser_calib_ref}" />
       <dynamics damping="0.008" />
       <xacro:insert_block name="origin" />

File: pr2_description/urdf/torso_v0/torso.urdf.xacro (robot description, xacro)
@@ -4,10 +4,15 @@
   <xacro:include filename="$(find pr2_description)/urdf/torso_v0/torso.transmission.xacro" />
   <xacro:include filename="$(find pr2_description)/urdf/sensors/microstrain_3dmgx2_imu.urdf.xacro" />
-  <xacro:macro name="pr2_torso_v0" params="name parent *origin torso_calib:=0.00475">
+  <xacro:macro name="pr2_torso_v0" params="name parent *origin torso_calib_ref:=0.0">
     <joint name="${name}_joint" type="prismatic">
       <axis xyz="0 0 1" />
       <limit lower="0.0" upper="0.33" effort="10000" velocity="0.013"/> <!-- alpha tested velocity and effort limits -->
       <safety_controller  k_velocity="2000000" soft_lower_limit="${0.0+0.0115}" soft_upper_limit="${0.33-0.005}" k_position="100" />
-      <calibration falling="${torso_calib}" />
+      <xacro:unless value="${torso_calib_ref}">
+        <calibration  falling="0.00475" />
+      </xacro:unless>
+      <xacro:if value="${torso_calib_ref}">
+        <calibration  falling="${torso_calib_ref}" />
+      </xacro:if>
       <dynamics damping="20000.0" />
       <xacro:insert_block name="origin" />

File: pr2_description/urdf/upper_arm_v0/upper_arm.urdf.xacro (robot description, xacro)
@@ -29,6 +29,6 @@
   <!-- Includes elbow flex, FA roll joints in macros below -->
   <xacro:macro name="pr2_upper_arm_v0" params="side parent reflect
-   forearm_roll_calib:=${0.0+cal_r_forearm_roll_flag}
-   elbow_flex_calib:=${-1.1606+cal_r_elbow_flex_flag}">
+   forearm_roll_calib_ref:=0.0
+   elbow_flex_calib_ref:=0.0 ">
     <joint name="${side}_upper_arm_joint" type="fixed">
       <origin xyz="0 0 0" rpy="0 0 0" />
@@ -67,10 +67,10 @@
     <!-- Elbow flex, FA roll macros -->
     <xacro:pr2_forearm_roll_v0 side="${side}" parent="${side}_elbow_flex_link" reflect="${reflect}"
-                               forearm_roll_calib="${forearm_roll_calib}"/>
+                               forearm_roll_calib_ref="${forearm_roll_calib_ref}"/>
     <xacro:pr2_elbow_flex_v0 side="${side}" parent="${side}_upper_arm_link" reflect="${reflect}"
-                             elbow_flex_calib="${elbow_flex_calib}"/>
+                             elbow_flex_calib_ref="${elbow_flex_calib_ref}"/>
   </xacro:macro>
   <xacro:macro name="pr2_elbow_flex_v0" params="side parent reflect
-   elbow_flex_calib">
+   elbow_flex_calib_ref">
     <!-- Elbow flex -->
     <joint name="${side}_elbow_flex_joint" type="revolute">
@@ -79,5 +79,10 @@
       <limit lower="-2.3213" upper="0.00" effort="30" velocity="${VELOCITY_LIMIT_SCALE*5.5}" /> <!-- alpha tested velocity and effort limits -->
       <safety_controller k_position="100" k_velocity="3" soft_lower_limit="${-2.3213+0.2}" soft_upper_limit="${0.00-0.15}" />
-      <calibration falling="${elbow_flex_calib}"/>
+      <xacro:unless value="${elbow_flex_calib_ref}">
+        <calibration falling="${-1.1606+cal_r_elbow_flex_flag}"/>
+      </xacro:unless>
+      <xacro:if value="${elbow_flex_calib_ref}">
+        <calibration falling="${elbow_flex_calib_ref}"/>
+      </xacro:if>
       <dynamics damping="1.0" />
       <origin xyz="0.4 0 0" rpy="0 0 0" />
@@ -112,5 +117,5 @@
   <!-- FA roll joint only -->
   <xacro:macro name="pr2_forearm_roll_v0" params="side parent reflect
-   forearm_roll_calib">
+   forearm_roll_calib_ref">
     <!-- forearm_roll_link is a fictitious link internal to elbow_flex_link, provides an attachment point for the actual forearm -->
     <joint name="${side}_forearm_roll_joint" type="continuous">
@@ -118,5 +123,10 @@
       <limit effort="30" velocity="${VELOCITY_LIMIT_SCALE*6}" /> <!-- alpha tested velocity and effort limits -->
       <safety_controller k_velocity="1" />
-      <calibration rising="${forearm_roll_calib}" />
+      <xacro:unless value="${forearm_roll_calib_ref}">
+      <calibration rising="${0.0+cal_r_forearm_roll_flag}" />
+      </xacro:unless>
+      <xacro:if value="${forearm_roll_calib_ref}">
+      <calibration rising="${forearm_roll_calib_ref}" />
+      </xacro:if>
       <dynamics damping="0.1" />
       <origin xyz="0 0 0" rpy="0 0 0" />
