Commit message: updates from (#3036)

File: pr2_defs/defs/gazebo/gazebo_defs.urdf.xacro (robot description, xacro)
@@ -4,18 +4,12 @@
        xmlns:interface="http://playerstage.sourceforge.net/gazebo/xmlschema/#interface">
   <gazebo>
-    <!-- distribute state for sensors -->
-    <controller:ros_pub_world_state name="ros_pub_world_state_controller" plugin="libros_pub_world_state.so">
+    <!-- PR2_ACTARRAY -->
+    <controller:ros_controller_manager name="ros_controller_manager" plugin="libros_controller_manager.so">
       <alwaysOn>true</alwaysOn>
       <updateRate>1000.0</updateRate>
-      <interface:audio name="gazebo_pub_world_state_control_dummy_iface" />
-    </controller:ros_pub_world_state>
-    <!-- PR2_ACTARRAY -->
-    <controller:gazebo_controller_manager name="gazebo_controller_manager" plugin="libgazebo_controller_manager.so">
-      <alwaysOn>true</alwaysOn>
-      <updateRate>1000.0</updateRate>
-      <interface:audio name="gazebo_controller_manager_dummy_iface" />
-    </controller:gazebo_controller_manager>
+      <interface:audio name="ros_controller_manager_dummy_iface" />
+    </controller:ros_controller_manager>
     <!-- battery controls -->
-    <controller:gazebo_battery name="gazebo_battery_controller" plugin="libgazebo_battery.so">
+    <controller:ros_battery name="ros_battery_controller" plugin="libros_battery.so">
       <alwaysOn>true</alwaysOn>
       <updateRate>1.0</updateRate>
@@ -29,5 +23,5 @@
       <selfTestServiceName>self_test</selfTestServiceName>
       <interface:audio name="battery_dummy_interface" />
-    </controller:gazebo_battery>
+    </controller:ros_battery>
     <controller:ros_time name="ros_time" plugin="libros_time.so">
       <alwaysOn>true</alwaysOn>

File: pr2_defs/robots/pr2_armless.urdf.xacro (robot description, xacro)
@@ -29,5 +29,5 @@
   </pr2_head_sensor_package>
   <pr2_tilting_laser name="laser_tilt" parent="torso_lift_link" laser_calib_ref="-0.35">
-    <origin xyz="0.1 0 0.235" rpy="0 0 0" />
+    <origin xyz="0.1 0 0.2275" rpy="0 0 0" /> <!-- from hand measurement by JH on PRE (was originally .235 from CAD: -->
   </pr2_tilting_laser>
 </robot>

File: pr2_description/gazebo/gazebo.urdf.xacro (robot description, xacro)
@@ -4,10 +4,10 @@
        xmlns:interface="http://playerstage.sourceforge.net/gazebo/xmlschema/#interface">
   <gazebo>
-    <controller:gazebo_controller_manager name="gazebo_controller_manager" plugin="libgazebo_controller_manager.so">
+    <controller:ros_controller_manager name="ros_controller_manager" plugin="libros_controller_manager.so">
       <alwaysOn>true</alwaysOn>
       <updateRate>1000.0</updateRate>
-      <interface:audio name="gazebo_controller_manager_dummy_iface" />
-    </controller:gazebo_controller_manager>
-    <controller:gazebo_battery name="gazebo_battery_controller" plugin="libgazebo_battery.so">
+      <interface:audio name="ros_controller_manager_dummy_iface" />
+    </controller:ros_controller_manager>
+    <controller:ros_battery name="ros_battery_controller" plugin="libros_battery.so">
       <alwaysOn>true</alwaysOn>
       <updateRate>1.0</updateRate>
@@ -21,5 +21,5 @@
       <dischargeVoltage>15.52</dischargeVoltage>
       <chargeVoltage>16.41</chargeVoltage>
-    </controller:gazebo_battery>
+    </controller:ros_battery>
     <controller:ros_time name="ros_time" plugin="libros_time.so">
       <alwaysOn>true</alwaysOn>
