Commit message: update test to include new urdf parser. fix some urdf errors.

File: pr2_defs/defs/gripper/gripper_defs.urdf.xacro (robot description, xacro)
@@ -190,5 +190,5 @@
     <!-- floating link for simulating gripper constraints -->
     <joint name="${side}_gripper_float_joint" type="prismatic">
-      <limit lower="-0.05" upper="0.001" effort="0" />
+      <limit lower="-0.05" upper="0.001" velocity="10" effort="10" />
       <safety_controller soft_lower_limit="${-0.05+0.0}" soft_upper_limit="${0.001-0.0}" />
       <axis xyz="1 0 0" />

File: pr2_defs/robots/laser_tilt.urdf.xacro (robot description, xacro)
@@ -1,3 +1,4 @@
  <robot name="laser_tilt_test">
+  <include filename="$(find pr2_defs)/defs/materials.urdf.xacro" />
   <include filename="$(find pr2_defs)/defs/head/head_defs.urdf.xacro" />
   <include filename="$(find pr2_defs)/defs/body/body_defs.urdf.xacro" />

Commit message: fix mesh name.

File: pr2_defs/defs/gripper/gripper_defs.urdf.xacro (robot description, xacro)
@@ -118,5 +118,5 @@
         <origin xyz="0 0 0" rpy="0 0 0" />
         <geometry name="${prefix}_l_finger_tip_collision_geom">
-          <mesh filename="package://pr2_defs/meshes/finger_tip_pad2_l.stlb" />
+          <mesh filename="package://pr2_defs/meshes/finger_tip_pad2_l.stl" />
         </geometry>
         <verbose value="Yes" />
@@ -151,5 +151,5 @@
         <origin xyz="0 0 0" rpy="0 0 0" />
         <geometry name="${prefix}_r_finger_tip_collision_geom">
-          <mesh filename="package://pr2_defs/meshes/finger_tip_pad2_r.stlb" />
+          <mesh filename="package://pr2_defs/meshes/finger_tip_pad2_r.stl" />
         </geometry>
         <verbose value="Yes" />

Commit message: adding [lr]_gripper_motor_accelerometer_link for gripper palm imu

File: pr2_defs/defs/gripper/gripper_defs.urdf.xacro (robot description, xacro)
@@ -188,4 +188,30 @@
       </collision>
     </link>
+    <joint name="${side}_gripper_motor_accelerometer_joint" type="fixed">
+      <origin xyz="0 0 0" rpy="0 0 0" />
+      <parent link="${side}_gripper_palm_link"/>
+      <child link="${side}_gripper_motor_accelerometer_link"/>
+    </joint>
+    <link name="${side}_gripper_motor_accelerometer_link">
+      <inertial>
+        <mass value="0.001" />
+        <origin xyz="0 0 0" rpy="0 0 0" />
+        <inertia  ixx="0.001" ixy="0.0" ixz="0.0"
+                  iyy="0.001" iyz="0.0"
+                  izz="0.001" />
+      </inertial>
+      <visual>
+        <origin xyz="0 0 0" rpy="0 0 0" />
+        <geometry>
+          <box size="0.001 0.001 0.001" />
+        </geometry>
+      </visual>
+      <collision>
+        <origin xyz="0 0 0" rpy="0 0 0" />
+        <geometry>
+          <box size="0.001 0.001 0.001" />
+        </geometry>
+      </collision>
+    </link>
     <!-- floating link for simulating gripper constraints -->
     <joint name="${side}_gripper_float_joint" type="prismatic">

Commit message: moving floating link for gripper simulation into gazebo extension.

File: pr2_defs/defs/gripper/gripper_defs.urdf.xacro (robot description, xacro)
@@ -215,37 +215,4 @@
       </collision>
     </link>
-    <!-- floating link for simulating gripper constraints -->
-    <joint name="${side}_gripper_float_joint" type="prismatic">
-      <limit lower="-0.05" upper="0.001" velocity="10" effort="10" />
-      <safety_controller soft_lower_limit="${-0.05+0.0}" soft_upper_limit="${0.001-0.0}" k_position="20" k_velocity="20" />
-      <axis xyz="1 0 0" />
-      <dynamics damping="10.0" />
-      <origin xyz="0.05 0 0" rpy="0 0 0" />
-      <parent link="${side}_gripper_palm_link"/>
-      <child link="${side}_gripper_float_link"/>
-    </joint>
-    <link name="${side}_gripper_float_link">
-      <inertial>
-        <mass value="0.01" />
-        <origin xyz="0 0 0" rpy="0 0 0" />
-        <inertia  ixx="0.0001" ixy="0" ixz="0"
-                  iyy="0.0001" iyz="0"
-                  izz="0.0001" />
-      </inertial>
-      <visual name="${side}_gripper_float_visual">
-        <origin xyz="0 0 0" rpy="0 0 0" />
-        <geometry name="${side}_gripper_float_visual_geom">
-          <box size="0.001 0.001 0.001" />
-        </geometry>
-        <material name="White" />
-      </visual>
-      <collision name="${side}_gripper_float_collision">
-        <origin xyz="0 0 0" rpy="0 0 0" />
-        <geometry name="${side}_gripper_float_collision_geom">
-          <box size="0.001 0.001 0.001" />
-        </geometry>
-        <verbose value="Yes" />
-      </collision>
-    </link>
     <joint name="${side}_gripper_tool_joint" type="fixed">
       <origin xyz="0.18 0 0" rpy="0 0 0" />

File: pr2_defs/defs/gripper/gripper_gazebo.xacro (robot description, xacro)
@@ -3,4 +3,6 @@
        xmlns:controller="http://playerstage.sourceforge.net/gazebo/xmlschema/#controller"
        xmlns:joint="http://playerstage.sourceforge.net/gazebo/xmlschema/#slider"
+       xmlns:body="http://playerstage.sourceforge.net/gazebo/xmlschema/#body"
+       xmlns:geom="http://playerstage.sourceforge.net/gazebo/xmlschema/#geom"
        xmlns:interface="http://playerstage.sourceforge.net/gazebo/xmlschema/#interface">
   <property name="finger_stop_kd"             value="1.0" />
@@ -158,4 +160,42 @@
     </gazebo>
     <gazebo>
+      <!-- floating link for enforcing gripper constraints -->
+      <body:box name="${side}_gripper_float_link">
+          <massMatrix>true</massMatrix>
+          <mass>0.01</mass>
+          <ixx>0.0001</ixx>
+          <ixy>0</ixy>
+          <ixz>0</ixz>
+          <iyy>0.0001</iyy>
+          <iyz>0</iyz>
+          <izz>0.0001</izz>
+          <cx>0</cx>
+          <cy>0</cy>
+          <cz>0</cz>
+          <xyz>0.82025 0.188 0.790675</xyz>
+          <rpy>0 -0 0</rpy>
+          <geom:box name="${side}_gripper_float_link_geom">
+              <xyz>0 0 0</xyz>
+              <rpy>0 -0 0</rpy>
+              <size>0.001 0.001 0.001</size>
+              <visual>
+                  <xyz>0 0 0</xyz>
+                  <rpy>0 -0 0</rpy>
+                  <scale>0.001 0.001 0.001</scale>
+                  <mesh>unit_box</mesh>
+                  <material>PR2/White</material>
+              </visual>
+          </geom:box>
+          <turnGravityOff>true</turnGravityOff>
+          <selfCollide>false</selfCollide>
+      </body:box>
+      <joint:slider name="${side}_gripper_float_joint">
+          <body1>${side}_gripper_float_link</body1>
+          <body2>${side}_gripper_palm_link</body2>
+          <anchor>${side}_gripper_float_link</anchor>
+          <axis>1 0 0</axis>
+          <lowStop>-0.05</lowStop>
+          <highStop>0.001</highStop>
+      </joint:slider>
       <joint:slider name="${side}_gripper_l_finger_tip_slider_joint">
           <body1>${side}_gripper_l_finger_tip_link</body1>

File: pr2_defs/defs/gripper_beta/gripper_defs.urdf.xacro (robot description, xacro)
@@ -214,37 +214,4 @@
       </collision>
     </link>
-    <!-- floating link for simulating gripper constraints -->
-    <joint name="${side}_gripper_float_joint" type="prismatic">
-      <limit lower="-0.05" upper="0.001" velocity="10" effort="10" />
-      <safety_controller soft_lower_limit="${-0.05+0.0}" soft_upper_limit="${0.001-0.0}" k_position="20" k_velocity="20" />
-      <axis xyz="1 0 0" />
-      <dynamics damping="10.0" />
-      <origin xyz="0.05 0 0" rpy="0 0 0" />
-      <parent link="${side}_gripper_palm_link"/>
-      <child link="${side}_gripper_float_link"/>
-    </joint>
-    <link name="${side}_gripper_float_link">
-      <inertial>
-        <mass value="0.01" />
-        <origin xyz="0 0 0" rpy="0 0 0" />
-        <inertia  ixx="0.0001" ixy="0" ixz="0"
-                  iyy="0.0001" iyz="0"
-                  izz="0.0001" />
-      </inertial>
-      <visual name="${side}_gripper_float_visual">
-        <origin xyz="0 0 0" rpy="0 0 0" />
-        <geometry name="${side}_gripper_float_visual_geom">
-          <box size="0.001 0.001 0.001" />
-        </geometry>
-        <material name="White" />
-      </visual>
-      <collision name="${side}_gripper_float_collision">
-        <origin xyz="0 0 0" rpy="0 0 0" />
-        <geometry name="${side}_gripper_float_collision_geom">
-          <box size="0.001 0.001 0.001" />
-        </geometry>
-        <verbose value="Yes" />
-      </collision>
-    </link>
     <joint name="${side}_gripper_tool_joint" type="fixed">
       <origin xyz="0.18 0 0" rpy="0 0 0" />

File: pr2_defs/defs/gripper_beta/gripper_gazebo.xacro (robot description, xacro)
@@ -3,4 +3,6 @@
        xmlns:controller="http://playerstage.sourceforge.net/gazebo/xmlschema/#controller"
        xmlns:joint="http://playerstage.sourceforge.net/gazebo/xmlschema/#slider"
+       xmlns:body="http://playerstage.sourceforge.net/gazebo/xmlschema/#body"
+       xmlns:geom="http://playerstage.sourceforge.net/gazebo/xmlschema/#geom"
        xmlns:interface="http://playerstage.sourceforge.net/gazebo/xmlschema/#interface">
   <property name="finger_stop_kd"             value="1.0" />
@@ -160,4 +162,42 @@
     </gazebo>
     <gazebo>
+      <!-- floating link for enforcing gripper constraints -->
+      <body:box name="${side}_gripper_float_link">
+          <massMatrix>true</massMatrix>
+          <mass>0.01</mass>
+          <ixx>0.0001</ixx>
+          <ixy>0</ixy>
+          <ixz>0</ixz>
+          <iyy>0.0001</iyy>
+          <iyz>0</iyz>
+          <izz>0.0001</izz>
+          <cx>0</cx>
+          <cy>0</cy>
+          <cz>0</cz>
+          <xyz>0.82025 0.188 0.790675</xyz>
+          <rpy>0 -0 0</rpy>
+          <geom:box name="${side}_gripper_float_link_geom">
+              <xyz>0 0 0</xyz>
+              <rpy>0 -0 0</rpy>
+              <size>0.001 0.001 0.001</size>
+              <visual>
+                  <xyz>0 0 0</xyz>
+                  <rpy>0 -0 0</rpy>
+                  <scale>0.001 0.001 0.001</scale>
+                  <mesh>unit_box</mesh>
+                  <material>PR2/White</material>
+              </visual>
+          </geom:box>
+          <turnGravityOff>true</turnGravityOff>
+          <selfCollide>false</selfCollide>
+      </body:box>
+      <joint:slider name="${side}_gripper_float_joint">
+          <body1>${side}_gripper_float_link</body1>
+          <body2>${side}_gripper_palm_link</body2>
+          <anchor>${side}_gripper_float_link</anchor>
+          <axis>1 0 0</axis>
+          <lowStop>-0.05</lowStop>
+          <highStop>0.001</highStop>
+      </joint:slider>
       <joint:slider name="${side}_gripper_l_finger_tip_slider_joint">
           <body1>${side}_gripper_l_finger_tip_link</body1>
