Commit message: fix per ticket #3148, setting gripper params explicitly for pr2_alpha2.

File: pr2_defs/defs/gripper/gripper_defs.urdf.xacro (robot description, xacro)
@@ -160,5 +160,5 @@
     <pr2_finger_gazebo prefix="${prefix}" />
   </macro>
-  <macro name="pr2_gripper" params="side parent *origin gear_ratio screw_reduction">
+  <macro name="pr2_gripper" params="side parent *origin gear_ratio screw_reduction theta0 phi0 t0 L0 h a b r">
     <joint name="${side}_gripper_palm_joint" type="fixed">
       <insert_block name="origin"/>
@@ -255,5 +255,15 @@
     <!-- extensions -->
     <pr2_gripper_gazebo side="${side}" />
-    <pr2_gripper_transmission side="${side}" />
+    <pr2_gripper_transmission side="${side}"
+        screw_reduction="${screw_reduction}"
+        gear_ratio="${gear_ratio}"
+        theta0="${theta0}"
+        phi0="${phi0}"
+        t0="${t0}"
+        L0="${L0}"
+        h="${h}"
+        a="${a}"
+        b="${b}"
+        r="${r}" />
   </macro>
 </robot>

File: pr2_defs/defs/gripper/gripper_transmission.xacro (robot description, xacro)
@@ -4,5 +4,5 @@
        xmlns:joint="http://playerstage.sourceforge.net/gazebo/xmlschema/#slider"
        xmlns:interface="http://playerstage.sourceforge.net/gazebo/xmlschema/#interface">
-  <macro name="pr2_gripper_transmission" params="side">
+  <macro name="pr2_gripper_transmission" params="side screw_reduction gear_ratio theta0 phi0 t0 L0 h a b r">
     <!-- [lr]_gripper_joint is a fictitious joint, used by transmission for controller gap   -->
     <!-- [lr]_gripper_joint is not attached to any link                                      -->
@@ -16,5 +16,16 @@
     <transmission type="PR2GripperTransmission" name="${side}_gripper_trans" >
       <actuator       name="${side}_gripper_motor" />
-      <gap_joint      name="${side}_gripper_joint" screw_reduction="${screw_reduction}" gear_ratio="${gear_ratio}" mechanical_reduction="1.0" />
+      <gap_joint      name="${side}_gripper_joint"
+                      mechanical_reduction="1.0"
+                      screw_reduction="${screw_reduction}"
+                      gear_ratio="${gear_ratio}"
+                      theta0="${theta0}"
+                      phi0="${phi0}"
+                      t0="${t0}"
+                      L0="${L0}"
+                      h="${h}"
+                      a="${a}"
+                      b="${b}"
+                      r="${r}" />
       <passive_joint  name="${side}_gripper_l_finger_joint"     />
       <passive_joint  name="${side}_gripper_r_finger_joint"     />

File: pr2_defs/robots/l_arm.urdf.xacro (robot description, xacro)
@@ -25,5 +25,14 @@
     <origin xyz="0.0 0.0 1.0" rpy="0 0 0" />
   </pr2_arm>
-  <pr2_gripper screw_reduction="${2.0/1000.0}" gear_ratio="${29.16}" side="l" parent="l_wrist_roll_link" >
+  <pr2_gripper side="l" parent="l_wrist_roll_link"
+               screw_reduction="${2.0/1000.0}" gear_ratio="${29.16}"
+               theta0="${2.97571*M_PI/180.0}"
+               phi0="${29.98717*M_PI/180.0}"
+               t0="${-0.19543/1000.0}"
+               L0="${34.70821/1000.0}"
+               h="${5.200/1000.0}"
+               a="${67.56801/1000.0}"
+               b="${48.97193/1000.0}"
+               r="${91.50000/1000.0}" >
     <origin xyz="0 0 0" rpy="0 0 0" />
   </pr2_gripper>

File: pr2_defs/robots/l_gripper.urdf.xacro (robot description, xacro)
@@ -20,5 +20,14 @@
   <include filename="$(find pr2_defs)/defs/materials.urdf.xacro" />
   <!-- for new gripper gear_ratio="29.16*22.0/16.0*0.9" screw_reduction="4.0/1000.0" -->
-  <pr2_gripper screw_reduction="${2.0/1000.0}" gear_ratio="${29.16}" side="l" parent="base_link" >
+  <pr2_gripper side="l" parent="base_link"
+               screw_reduction="${2.0/1000.0}" gear_ratio="${29.16}"
+               theta0="${2.97571*M_PI/180.0}"
+               phi0="${29.98717*M_PI/180.0}"
+               t0="${-0.19543/1000.0}"
+               L0="${34.70821/1000.0}"
+               h="${5.200/1000.0}"
+               a="${67.56801/1000.0}"
+               b="${48.97193/1000.0}"
+               r="${91.50000/1000.0}" >
     <origin xyz="0 0 1" rpy="0 0 0" />
   </pr2_gripper>

File: pr2_defs/robots/pr2.urdf.xacro (robot description, xacro)
@@ -47,5 +47,14 @@
     <origin xyz="0 -0.188 0.0" rpy="0 0 0" />
   </pr2_arm>
-  <pr2_gripper screw_reduction="${2.0/1000.0}" gear_ratio="${29.16}" side="r" parent="r_wrist_roll_link" >
+  <pr2_gripper side="r" parent="r_wrist_roll_link"
+               screw_reduction="${2.0/1000.0}" gear_ratio="${29.16}"
+               theta0="${2.97571*M_PI/180.0}"
+               phi0="${29.98717*M_PI/180.0}"
+               t0="${-0.19543/1000.0}"
+               L0="${34.70821/1000.0}"
+               h="${5.200/1000.0}"
+               a="${67.56801/1000.0}"
+               b="${48.97193/1000.0}"
+               r="${91.50000/1000.0}" >
     <origin xyz="0 0 0" rpy="0 0 0" />
   </pr2_gripper>
@@ -53,5 +62,14 @@
     <origin xyz="0.0 0.188 0.0" rpy="0 0 0" />
   </pr2_arm>
-  <pr2_gripper screw_reduction="${2.0/1000.0}" gear_ratio="${29.16}" side="l" parent="l_wrist_roll_link" >
+  <pr2_gripper side="l" parent="l_wrist_roll_link"
+               screw_reduction="${2.0/1000.0}" gear_ratio="${29.16}"
+               theta0="${2.97571*M_PI/180.0}"
+               phi0="${29.98717*M_PI/180.0}"
+               t0="${-0.19543/1000.0}"
+               L0="${34.70821/1000.0}"
+               h="${5.200/1000.0}"
+               a="${67.56801/1000.0}"
+               b="${48.97193/1000.0}"
+               r="${91.50000/1000.0}" >
     <origin xyz="0 0 0" rpy="0 0 0" />
   </pr2_gripper>

File: pr2_defs/robots/pre.urdf.xacro (robot description, xacro)
@@ -47,5 +47,14 @@
     <origin xyz="0 -0.188 0.0" rpy="0 0 0" />
   </pr2_arm>
-  <pr2_gripper screw_reduction="${2.0/1000.0}" gear_ratio="${29.16}" side="r" parent="r_wrist_roll_link" >
+  <pr2_gripper side="r" parent="r_wrist_roll_link"
+               screw_reduction="${2.0/1000.0}" gear_ratio="${29.16}"
+               theta0="${2.97571*M_PI/180.0}"
+               phi0="${29.98717*M_PI/180.0}"
+               t0="${-0.19543/1000.0}"
+               L0="${34.70821/1000.0}"
+               h="${5.200/1000.0}"
+               a="${67.56801/1000.0}"
+               b="${48.97193/1000.0}"
+               r="${91.50000/1000.0}" >
     <origin xyz="0 0 0" rpy="0 0 0" />
   </pr2_gripper>
@@ -53,5 +62,14 @@
     <origin xyz="0.0 0.188 0.0" rpy="0 0 0" />
   </pr2_arm>
-  <pr2_gripper screw_reduction="${2.0/1000.0}" gear_ratio="${29.16}" side="l" parent="l_wrist_roll_link" >
+  <pr2_gripper side="l" parent="l_wrist_roll_link"
+               screw_reduction="${2.0/1000.0}" gear_ratio="${29.16}"
+               theta0="${2.97571*M_PI/180.0}"
+               phi0="${29.98717*M_PI/180.0}"
+               t0="${-0.19543/1000.0}"
+               L0="${34.70821/1000.0}"
+               h="${5.200/1000.0}"
+               a="${67.56801/1000.0}"
+               b="${48.97193/1000.0}"
+               r="${91.50000/1000.0}" >
     <origin xyz="0 0 0" rpy="0 0 0" />
   </pr2_gripper>

File: pr2_defs/robots/prf.urdf.xacro (robot description, xacro)
@@ -39,15 +39,16 @@
     <origin xyz="0 -0.188 0.0" rpy="0 0 0" />
   </pr2_arm>
-  <pr2_gripper screw_reduction="${2.0/1000.0}" gear_ratio="${29.16}" side="r" parent="r_wrist_roll_link" >
+  <pr2_gripper side="r" parent="r_wrist_roll_link"
+               screw_reduction="${2.0/1000.0}" gear_ratio="${29.16}"
+               theta0="${2.97571*M_PI/180.0}"
+               phi0="${29.98717*M_PI/180.0}"
+               t0="${-0.19543/1000.0}"
+               L0="${34.70821/1000.0}"
+               h="${5.200/1000.0}"
+               a="${67.56801/1000.0}"
+               b="${48.97193/1000.0}"
+               r="${91.50000/1000.0}" >
     <origin xyz="0 0 0" rpy="0 0 0" />
   </pr2_gripper>
-  <!--
-  <pr2_arm side="l" reflect="1" parent="torso_lift_link">
-    <origin xyz="0.0 0.188 0.0" rpy="0 0 0" />
-  </pr2_arm>
-  <pr2_gripper screw_reduction="${2.0/1000.0}" gear_ratio="${29.16}" side="l" parent="l_wrist_roll_link" >
-    <origin xyz="0 0 0" rpy="0 0 0" />
-  </pr2_gripper>
-  -->
   <!-- Forearm Cam (Hand approximated values) -->
   <mono_cam name="r_forearm_cam" parent="r_forearm_roll_link">

File: pr2_defs/robots/prg.urdf.xacro (robot description, xacro)
@@ -39,15 +39,16 @@
     <origin xyz="0 -0.188 0.0" rpy="0 0 0" />
   </pr2_arm>
-  <pr2_gripper screw_reduction="${2.0/1000.0}" gear_ratio="${29.16}" side="r" parent="r_wrist_roll_link" >
+  <pr2_gripper side="r" parent="r_wrist_roll_link"
+               screw_reduction="${2.0/1000.0}" gear_ratio="${29.16}"
+               theta0="${2.97571*M_PI/180.0}"
+               phi0="${29.98717*M_PI/180.0}"
+               t0="${-0.19543/1000.0}"
+               L0="${34.70821/1000.0}"
+               h="${5.200/1000.0}"
+               a="${67.56801/1000.0}"
+               b="${48.97193/1000.0}"
+               r="${91.50000/1000.0}" >
     <origin xyz="0 0 0" rpy="0 0 0" />
   </pr2_gripper>
-  <!--
-  <pr2_arm side="l" reflect="1" parent="torso_lift_link">
-    <origin xyz="0.0 0.188 0.0" rpy="0 0 0" />
-  </pr2_arm>
-  <pr2_gripper screw_reduction="${2.0/1000.0}" gear_ratio="${29.16}" side="l" parent="l_wrist_roll_link" >
-    <origin xyz="0 0 0" rpy="0 0 0" />
-  </pr2_gripper>
-  -->
   <!-- Forearm Cam (Hand approximated values) -->
   <mono_cam name="r_forearm_cam" parent="r_forearm_roll_link">

File: pr2_defs/robots/r_arm.urdf.xacro (robot description, xacro)
@@ -25,5 +25,14 @@
     <origin xyz="0.0 0.0 1.0" rpy="0 0 0" />
   </pr2_arm>
-  <pr2_gripper screw_reduction="${2.0/1000.0}" gear_ratio="${29.16}" side="r" parent="r_wrist_roll_link" >
+  <pr2_gripper side="r" parent="r_wrist_roll_link"
+               screw_reduction="${2.0/1000.0}" gear_ratio="${29.16}"
+               theta0="${2.97571*M_PI/180.0}"
+               phi0="${29.98717*M_PI/180.0}"
+               t0="${-0.19543/1000.0}"
+               L0="${34.70821/1000.0}"
+               h="${5.200/1000.0}"
+               a="${67.56801/1000.0}"
+               b="${48.97193/1000.0}"
+               r="${91.50000/1000.0}" >
     <origin xyz="0 0 0" rpy="0 0 0" />
   </pr2_gripper>

File: pr2_defs/robots/r_forearm_gripper.urdf.xacro (robot description, xacro)
@@ -23,5 +23,14 @@
   <include filename="$(find pr2_defs)/defs/materials.urdf.xacro" />
   <pr2_forearm side="r" reflect="1" parent="base_link"/>
-  <pr2_gripper screw_reduction="${2.0/1000.0}" gear_ratio="${29.16}" side="r" parent="r_wrist_roll_link" >
+  <pr2_gripper side="r" parent="r_wrist_roll_link"
+               screw_reduction="${2.0/1000.0}" gear_ratio="${29.16}"
+               theta0="${2.97571*M_PI/180.0}"
+               phi0="${29.98717*M_PI/180.0}"
+               t0="${-0.19543/1000.0}"
+               L0="${34.70821/1000.0}"
+               h="${5.200/1000.0}"
+               a="${67.56801/1000.0}"
+               b="${48.97193/1000.0}"
+               r="${91.50000/1000.0}" >
     <origin xyz="0 0 0" rpy="0 0 0" />
   </pr2_gripper>

File: pr2_defs/robots/r_gripper.urdf.xacro (robot description, xacro)
@@ -20,5 +20,14 @@
   <include filename="$(find pr2_defs)/defs/materials.urdf.xacro" />
   <!-- for new gripper gear_ratio="29.16*22.0/16.0*0.9" screw_reduction="4.0/1000.0" -->
-  <pr2_gripper screw_reduction="${2.0/1000.0}" gear_ratio="${29.16}" side="r" parent="base_link" >
+  <pr2_gripper side="r" parent="base_link"
+               screw_reduction="${2.0/1000.0}" gear_ratio="${29.16}"
+               theta0="${2.97571*M_PI/180.0}"
+               phi0="${29.98717*M_PI/180.0}"
+               t0="${-0.19543/1000.0}"
+               L0="${34.70821/1000.0}"
+               h="${5.200/1000.0}"
+               a="${67.56801/1000.0}"
+               b="${48.97193/1000.0}"
+               r="${91.50000/1000.0}" >
     <origin xyz="0 0 1" rpy="0 0 0" />
   </pr2_gripper>

File: pr2_description/urdf/forearm_v0/forearm.urdf.xacro (robot description, xacro)
@@ -41,5 +41,5 @@
     <!-- Wrist flex -->
     <joint name="${side}_wrist_flex_joint" type="revolute">
-      <axis xyz="0 -1 0" />
+      <axis xyz="0 1 0" />
       <limit lower="0.0" upper="2.094" effort="10" velocity="${VELOCITY_LIMIT_SCALE*5.13}" />
       <safety_controller k_position="20" k_velocity="4" soft_lower_limit="${0.0 + 0.10}" soft_upper_limit="${2.094 - 0.10}" />

File: pr2_description/urdf/upper_arm_v0/upper_arm.urdf.xacro (robot description, xacro)
@@ -98,5 +98,5 @@
     <!-- forearm_roll_link is a fictitious link internal to elbow_flex_link, provides an attachment point for the actual forearm -->
     <joint name="${side}_forearm_roll_joint" type="continuous">
-      <axis xyz="-1 0 0" />
+      <axis xyz="1 0 0" />
       <limit effort="30" velocity="${VELOCITY_LIMIT_SCALE*6}" />
       <safety_controller k_velocity="1" />
