Commit message: Fixing Beta defs after #3123 cleanup. Wrist has positive axes, and is now tested on Beta HW

File: pr2_description/urdf/forearm_v0/forearm.transmission.xacro (robot description, xacro)
@@ -9,5 +9,5 @@
       <rightActuator name="${side}_wrist_r_motor" mechanicalReduction="${624/35*54/16}"/>
       <leftActuator name="${side}_wrist_l_motor"  mechanicalReduction="${624/35*54/16}"/>
-      <flexJoint name="${side}_wrist_flex_joint"  mechanicalReduction="1.0" />
+      <flexJoint name="${side}_wrist_flex_joint"  mechanicalReduction="-1.0" />
       <rollJoint name="${side}_wrist_roll_joint"  mechanicalReduction="1.0" />
     </transmission>

File: pr2_description/urdf/forearm_v0/forearm.urdf.xacro (robot description, xacro)
@@ -42,8 +42,8 @@
     <joint name="${side}_wrist_flex_joint" type="revolute">
       <axis xyz="0 1 0" />
-      <limit lower="0.0" upper="2.094" effort="10" velocity="${VELOCITY_LIMIT_SCALE*5.13}" />
-      <safety_controller k_position="20" k_velocity="4" soft_lower_limit="${0.0 + 0.10}" soft_upper_limit="${2.094 - 0.10}" />
+      <limit upper="0.0" lower="-2.094" effort="10" velocity="${VELOCITY_LIMIT_SCALE*5.13}" />
+      <safety_controller k_position="20" k_velocity="4" soft_upper_limit="${0.0 - 0.10}" soft_lower_limit="${-2.094 + 0.10}" />
       <dynamics damping="0.1" />
-      <calibration reference_position="${0.5410521 + cal_r_wrist_flex_flag}" />
+      <calibration reference_position="${-0.5410521 + cal_r_wrist_flex_flag}" />
       <origin xyz="0.32025 0 0" rpy="0 0 0" />
       <parent link="${side}_forearm_link"/>
