Commit message: adding upper arm and forearm sleeve 3D meshes in collada

File: pr2_description/urdf/forearm_v0/forearm.gazebo.xacro (robot description, xacro)
@@ -17,5 +17,4 @@
         </controller:gazebo_ros_bumper>
       </sensor:contact>
-      <material value="PR2/Grey" />
     </gazebo>
     <!-- Wrist flex -->

File: pr2_description/urdf/forearm_v0/forearm.urdf.xacro (robot description, xacro)
@@ -25,15 +25,39 @@
                  izz="0.01659310749" />
       </inertial>
-      <visual name="${side}_forearm_visual">
+      <visual>
         <origin xyz="0 0 0" rpy="0 0 0" />
-        <geometry name="${side}_forearm_visual_geom">
+        <geometry>
           <mesh filename="package://pr2_description/meshes/forearm_v0/forearm.stl" />
-        </geometry>
+       </geometry>
         <material name="Grey" />
       </visual>
-      <collision name="${side}_forearm_collision">
+      <collision>
         <origin xyz="0 0 0" rpy="0 0 0" />
-        <geometry name="${side}_forearm_collision_geom">
+        <geometry>
           <mesh filename="package://pr2_description/meshes/forearm_v0/convex/forearm_convex.stlb" />
+        </geometry>
+      </collision>
+    </link>
+    <joint name="${side}_forearm_sleeve_joint" type="fixed">
+      <insert_block name="origin" /> <!-- transform from parent link to this joint frame -->
+      <parent link="${parent}"/>
+      <child link="${side}_forearm_sleeve_link"/>
+    </joint>
+    <link name="${side}_forearm_sleeve_link">
+      <inertial>
+        <mass value="0.1" />
+        <origin xyz="0 0 0" />
+        <inertia ixx="0.01" ixy="0.00" ixz="0.00" iyy="0.01" iyz="0.00" izz="0.01" />
+      </inertial>
+      <visual>
+        <origin xyz="-0.02 0 0" rpy="0 ${M_PI/2} 0" />
+        <geometry>
+          <mesh filename="package://pr2_description/meshes/forearm_v0/forearm.dae" scale="0.001 0.001 0.001" />
+        </geometry>
+      </visual>
+      <collision>
+        <origin xyz="-0.02 0 0" rpy="0 ${M_PI/2} 0" />
+        <geometry>
+          <mesh filename="package://pr2_description/meshes/forearm_v0/forearm.dae" scale="0.001 0.001 0.001" />
         </geometry>
       </collision>

File: pr2_description/urdf/upper_arm_v0/upper_arm.gazebo.xacro (robot description, xacro)
@@ -17,5 +17,4 @@
       </sensor:contact>
       <turnGravityOff>true</turnGravityOff>
-      <material value="Gazebo/Grey" />
     </gazebo>
   </xacro:macro>

File: pr2_description/urdf/upper_arm_v0/upper_arm.urdf.xacro (robot description, xacro)
@@ -49,15 +49,41 @@
                   izz="${0.5*((reflect+1)*ual_izz+(1-reflect)*uar_izz)}" />
       </inertial>
-      <visual name="{side}_upper_arm_visual">
+      <visual>
         <origin xyz="0 0 0" rpy="0 0 0" />
-        <geometry name="${side}_upper_arm_visual_geom">
+        <geometry>
           <mesh filename="package://pr2_description/meshes/upper_arm_v0/upper_arm.stl" />
         </geometry>
         <material name="Green" />
       </visual>
-      <collision name="${side}_upper_arm_collision">
+      <collision>
         <origin xyz="0 0 0" rpy="0 0 0" />
-        <geometry name="${side}_upper_arm_collision_geom">
+        <geometry>
           <mesh filename="package://pr2_description/meshes/upper_arm_v0/convex/upper_arm_convex.stlb" />
+        </geometry>
+      </collision>
+    </link>
+    <joint name="${side}_upper_arm_sleeve_joint" type="fixed">
+      <origin xyz="0 0 0" rpy="0 0 0" />
+      <parent link="${parent}"/>
+      <child link="${side}_upper_arm_sleeve_link"/>
+    </joint>
+    <link name="${side}_upper_arm_sleeve_link">
+      <inertial>
+        <!-- NOTE:reflect==-1 for right side, reflect==1 for the left side -->
+        <mass value="0.1" />
+        <origin xyz="0 0 0" />
+        <inertia  ixx="0.01" ixy="0.00" ixz="0.00" iyy="0.01" iyz="0.00" izz="0.01" />
+      </inertial>
+      <visual>
+        <origin rpy="0 1.57079632679 0" xyz="-0.01 0 0"/>
+        <geometry>
+          <mesh filename="package://pr2_description/meshes/upper_arm_v0/upper_arm.dae" scale="0.001 0.001 0.001"/>
+        </geometry>
+        <material name="Green" />
+      </visual>
+      <collision>
+        <origin rpy="0 1.57079632679 0" xyz="-0.01 0 0"/>
+        <geometry>
+          <mesh filename="package://pr2_description/meshes/upper_arm_v0/upper_arm.dae" scale="0.001 0.001 0.001"/>
         </geometry>
       </collision>
