Commit message: Updating pr2 beta arm defs. Also adding gripper LED. Trac #3565

File: pr2_description/urdf/forearm_v0/forearm.urdf.xacro (robot description, xacro)
@@ -47,5 +47,5 @@
       <!-- hold both reference_position and upper/lower for tick-tock, remove reference_positiion after verifying upper/lower works with calibration controllers.  if search velocity in pr2_calibration_controllers.yaml is +, the reference_position is rising, if - then it is falling -->
       <calibration reference_position="${-0.5410521 + cal_r_wrist_flex_flag}" falling="${-0.5410521 + cal_r_wrist_flex_flag}" />
-      <origin xyz="0.32025 0 0" rpy="0 0 0" />
+      <origin xyz="0.321 0 0" rpy="0 0 0" />
       <parent link="${side}_forearm_link"/>
       <child link="${side}_wrist_flex_link"/>

File: pr2_description/urdf/gripper_v0/gripper.urdf.xacro (robot description, xacro)
@@ -192,4 +192,11 @@
       </collision>
     </link>
+    <joint name="${side}_gripper_led_joint" type="fixed">
+      <!--  Need to check if we need a positive or negative Z term -->
+      <origin xyz="0.0513 0.0 .0244"/>
+      <parent link="${side}_gripper_palm_link"/>
+      <child link="${side}_gripper_led_frame"/>
+    </joint>
+    <link name="${side}_gripper_led_frame" />
     <joint name="${side}_gripper_motor_accelerometer_joint" type="fixed">
       <origin xyz="0 0 0" rpy="0 0 0" />

Commit message: adjust sleeves

File: pr2_description/urdf/forearm_v0/forearm.urdf.xacro (robot description, xacro)
@@ -51,5 +51,5 @@
       </inertial>
       <visual>
-        <origin xyz="-0.02 0 0" rpy="0 ${M_PI/2} 0" />
+        <origin xyz="-0.03 0 0" rpy="0 ${M_PI/2} 0" />
         <geometry>
           <mesh filename="package://pr2_description/meshes/forearm_v0/forearm.dae" scale="0.001 0.001 0.001" />
@@ -57,5 +57,5 @@
       </visual>
       <collision>
-        <origin xyz="-0.02 0 0" rpy="0 ${M_PI/2} 0" />
+        <origin xyz="-0.03 0 0" rpy="0 ${M_PI/2} 0" />
         <geometry>
           <mesh filename="package://pr2_description/meshes/forearm_v0/forearm.dae" scale="0.001 0.001 0.001" />

File: pr2_description/urdf/upper_arm_v0/upper_arm.urdf.xacro (robot description, xacro)
@@ -52,5 +52,5 @@
         <origin xyz="0 0 0" rpy="0 0 0" />
         <geometry>
-          <mesh filename="package://pr2_description/meshes/upper_arm_v0/upper_arm.stl" />
+          <mesh filename="package://pr2_description/meshes/upper_arm_v0/upper_arm.stl" scale="0.98 0.98 0.98" />
         </geometry>
         <material name="Green" />
@@ -59,5 +59,5 @@
         <origin xyz="0 0 0" rpy="0 0 0" />
         <geometry>
-          <mesh filename="package://pr2_description/meshes/upper_arm_v0/convex/upper_arm_convex.stlb" />
+          <mesh filename="package://pr2_description/meshes/upper_arm_v0/convex/upper_arm_convex.stlb" scale="0.98 0.98 0.98" />
         </geometry>
       </collision>
@@ -76,5 +76,5 @@
       </inertial>
       <visual>
-        <origin rpy="0 1.57079632679 0" xyz="-0.01 0 0"/>
+        <origin rpy="0 1.59 0.02" xyz="-0.015 0 0"/>
         <geometry>
           <mesh filename="package://pr2_description/meshes/upper_arm_v0/upper_arm.dae" scale="0.001 0.001 0.001"/>
@@ -83,5 +83,5 @@
       </visual>
       <collision>
-        <origin rpy="0 1.57079632679 0" xyz="-0.01 0 0"/>
+        <origin rpy="0 1.59 0.02" xyz="-0.015 0 0"/>
         <geometry>
           <mesh filename="package://pr2_description/meshes/upper_arm_v0/upper_arm.dae" scale="0.001 0.001 0.001"/>

Commit message: slight touch up on sleeves

File: pr2_description/urdf/forearm_v0/forearm.urdf.xacro (robot description, xacro)
@@ -51,5 +51,5 @@
       </inertial>
       <visual>
-        <origin xyz="-0.03 0 0" rpy="0 ${M_PI/2} 0" />
+        <origin xyz="-0.03 0.009 0" rpy="0 1.5707 -0.04" />
         <geometry>
           <mesh filename="package://pr2_description/meshes/forearm_v0/forearm.dae" scale="0.001 0.001 0.001" />
@@ -57,5 +57,5 @@
       </visual>
       <collision>
-        <origin xyz="-0.03 0 0" rpy="0 ${M_PI/2} 0" />
+        <origin xyz="-0.03 0.009 0" rpy="0 1.5707 -0.04" />
         <geometry>
           <mesh filename="package://pr2_description/meshes/forearm_v0/forearm.dae" scale="0.001 0.001 0.001" />

Commit message: Wrist joint limits updated based on corrected datasheet. Safety limits unchanged. #4770

File: pr2_description/urdf/forearm_v0/forearm.urdf.xacro (robot description, xacro)
@@ -42,6 +42,6 @@
     <joint name="${side}_wrist_flex_joint" type="revolute">
       <axis xyz="0 1 0" />
-      <limit upper="0.0" lower="-2.094" effort="10" velocity="${VELOCITY_LIMIT_SCALE*5.13}" /> <!-- alpha tested velocity and effort limits -->
-      <safety_controller k_position="20" k_velocity="4" soft_upper_limit="${0.0 - 0.10}" soft_lower_limit="${-2.094 + 0.10}" />
+      <limit upper="0.0" lower="-2.18" effort="10" velocity="${VELOCITY_LIMIT_SCALE*5.13}" /> <!-- alpha tested velocity and effort limits -->
+      <safety_controller k_position="20" k_velocity="4" soft_upper_limit="${0.0 - 0.10}" soft_lower_limit="${-2.18 + 0.18}" />
       <dynamics damping="0.1" />
       <calibration falling="${-0.5410521 + cal_r_wrist_flex_flag}" />

Commit message: allow pr2.urdf.xacro to accept customized calibration values (#285)
If 0.0, use the default values. (This retains backward compatibility)
If not 0.0, use the passed values. (Enable custom calibration values for all macro instantiations

Using 0.0 to trigger the old defaults is necessary because some default values need to be computed from other parameters.

File: pr2_description/urdf/forearm_v0/forearm.urdf.xacro (robot description, xacro)
@@ -8,5 +8,7 @@
   <xacro:include filename="$(find pr2_description)/urdf/common.xacro" />
   <!-- ============================   Forearm   ============================ -->
-  <xacro:macro name="pr2_forearm_v0" params="side parent reflect *origin">
+  <xacro:macro name="pr2_forearm_v0" params="side parent reflect *origin
+    wrist_flex_calib_ref:=0.0
+    wrist_roll_calib_ref:=0.0">
     <joint name="${side}_forearm_joint" type="fixed">
       <xacro:insert_block name="origin" /> <!-- transform from parent link to this joint frame -->
@@ -42,5 +44,10 @@
       <safety_controller k_position="20" k_velocity="4" soft_upper_limit="${0.0 - 0.10}" soft_lower_limit="${-2.18 + 0.18}" />
       <dynamics damping="0.1" />
-      <calibration falling="${-0.5410521 + cal_r_wrist_flex_flag}" />
+      <xacro:unless value="${wrist_flex_calib_ref}">
+        <calibration  falling="${-0.5410521+cal_r_wrist_flex_flag}" />
+      </xacro:unless>
+      <xacro:if value="${wrist_flex_calib_ref}">
+        <calibration  falling="${wrist_flex_calib_ref}" />
+      </xacro:if>
       <origin xyz="0.321 0 0" rpy="0 0 0" />
       <parent link="${side}_forearm_link"/>
@@ -75,5 +82,10 @@
       <safety_controller k_velocity="2" />
       <dynamics damping="0.1" />
-      <calibration rising="${-M_PI / 2 + cal_r_wrist_roll_flag}" />
+      <xacro:unless value="${wrist_roll_calib_ref}">
+        <calibration rising="${-M_PI/2+cal_r_wrist_roll_flag}" />
+      </xacro:unless>
+      <xacro:if value="${wrist_roll_calib_ref}">
+        <calibration  rising="${wrist_roll_calib_ref}" />
+      </xacro:if>
       <origin xyz="0 0 0" rpy="0 0 0" />
       <parent link="${side}_wrist_flex_link"/>

File: pr2_description/urdf/head_v0/head.urdf.xacro (robot description, xacro)
@@ -4,10 +4,10 @@
   <xacro:include filename="$(find pr2_description)/urdf/head_v0/head.transmission.xacro" />
   <xacro:property name="M_PI" value="3.1415926535897931" />
-  <xacro:macro name="pr2_head_pan_v0" params="name parent *origin">
+  <xacro:macro name="pr2_head_pan_v0" params="name parent *origin head_pan_calib_ref:=0.0">
     <joint name="${name}_joint" type="revolute">
       <axis xyz="0 0 1" />
       <limit lower="-3.007" upper="3.007" effort="2.645" velocity="6" /> <!-- alpha tested velocity and effort limits -->
       <safety_controller k_velocity="1.5" soft_lower_limit="${-3.007+0.15}" soft_upper_limit="${3.007-0.15}" k_position="100" />
-      <calibration rising="0.0" />
+      <calibration rising="${head_pan_calib_ref}" />
       <dynamics damping="0.5" />
       <xacro:insert_block name="origin" />
@@ -38,10 +38,15 @@
     <xacro:pr2_head_pan_transmission_v0 name="${name}" />
   </xacro:macro>
-  <xacro:macro name="pr2_head_tilt_v0" params="name parent *origin">
+  <xacro:macro name="pr2_head_tilt_v0" params="name parent *origin head_tilt_calib_ref:=0.0">
     <joint name="${name}_joint" type="revolute">
       <axis xyz="0 1 0" />
       <limit lower="-0.471238" upper="1.39626" effort="18" velocity="5" /> <!-- alpha tested velocity and effort limits -->
       <safety_controller k_velocity="3.0" soft_lower_limit="${-0.4712 + 0.1}" soft_upper_limit="${1.39626 - 0.1}" k_position="100" />
-      <calibration falling="${0.0+cal_head_tilt_flag}" />
+      <xacro:unless value="${head_tilt_calib_ref}">
+        <calibration  falling="${0.0+cal_head_tilt_flag}" />
+      </xacro:unless>
+      <xacro:if value="${head_tilt_calib_ref}">
+        <calibration  falling="${head_tilt_calib_ref}" />
+      </xacro:if>
       <dynamics damping="10.0" />
       <xacro:insert_block name="origin" />
@@ -74,9 +79,11 @@
     <xacro:pr2_head_tilt_transmission_v0 name="${name}" />
   </xacro:macro>
-  <xacro:macro name="pr2_head_v0" params="name parent *origin">
-    <xacro:pr2_head_pan_v0 name="${name}_pan" parent="${parent}">
+  <xacro:macro name="pr2_head_v0" params="name parent *origin
+  head_pan_calib_ref:=0.0
+  head_tilt_calib_ref:=0.0 ">
+    <xacro:pr2_head_pan_v0 name="${name}_pan" parent="${parent}" head_pan_calib_ref="${head_pan_calib_ref}">
       <xacro:insert_block name="origin" />
     </xacro:pr2_head_pan_v0>
-    <xacro:pr2_head_tilt_v0 name="${name}_tilt" parent="${name}_pan_link">
+    <xacro:pr2_head_tilt_v0 name="${name}_tilt" parent="${name}_pan_link" head_tilt_calib_ref="${head_tilt_calib_ref}">
       <origin xyz="0.068 0 0" rpy="0 0 0" />
     </xacro:pr2_head_tilt_v0>

File: pr2_description/urdf/shoulder_v0/shoulder.urdf.xacro (robot description, xacro)
@@ -10,5 +10,8 @@
   <xacro:property name="shoulder_lift_radius" value="0.12" />  <!--TODO Define and give source-->
  <!-- ============================   Shoulder   ============================ -->
-  <xacro:macro name="pr2_shoulder_v0" params="side parent reflect *origin">
+  <xacro:macro name="pr2_shoulder_v0" params="side parent reflect *origin
+   shoulder_pan_calib_ref:=0.0
+   shoulder_lift_calib_ref:=0.0
+   upper_arm_roll_calib_ref:=0.0">
     <!-- Shoulder pan -->
     <joint name="${side}_shoulder_pan_joint" type="revolute">
@@ -24,5 +27,10 @@
                          soft_upper_limit="${reflect*M_PI/4+1.5-0.15}" />
       <!-- joint angle when the rising or the falling flag is activated on PR2 -->
-      <calibration  rising="${(reflect*M_PI/4)*cal_r_shoulder_pan_gearing+cal_r_shoulder_pan_flag}" />
+      <xacro:unless value="${shoulder_pan_calib_ref}">
+        <calibration  rising="${(reflect*M_PI/4)*cal_r_shoulder_pan_gearing+cal_r_shoulder_pan_flag}" />
+      </xacro:unless>
+      <xacro:if value="${shoulder_pan_calib_ref}">
+        <calibration  rising="${shoulder_pan_calib_ref}" />
+      </xacro:if>
     </joint>
     <link name="${side}_shoulder_pan_link">
@@ -56,5 +64,10 @@
       <safety_controller k_position="100" k_velocity="10"
                          soft_lower_limit="${-0.5236+0.17}" soft_upper_limit="${1.3963-0.10}" />
-      <calibration falling="${cal_r_shoulder_lift_flag}" />
+      <xacro:unless value="${shoulder_lift_calib_ref}">
+        <calibration falling="${cal_r_shoulder_lift_flag}" />
+      </xacro:unless>
+      <xacro:if value="${shoulder_lift_calib_ref}">
+        <calibration falling="${shoulder_lift_calib_ref}" />
+      </xacro:if>
       <dynamics damping="10.0" />
       <origin xyz="0.1 0 0" rpy="0 0 0" />
@@ -85,5 +98,6 @@
     </link>
     <!-- Upper arm roll is separate macro -->
-    <xacro:pr2_upper_arm_roll_v0 side="${side}" parent="${side}_shoulder_lift_link" reflect="${reflect}" >
+    <xacro:pr2_upper_arm_roll_v0 side="${side}" parent="${side}_shoulder_lift_link" reflect="${reflect}"
+                                 upper_arm_roll_calib_ref="${upper_arm_roll_calib_ref}">
       <origin xyz="0 0 0" rpy="0 0 0" />
     </xacro:pr2_upper_arm_roll_v0>
@@ -93,6 +107,7 @@
   </xacro:macro>
   <!-- Upperarm roll: internal fixed attchment point for upper arm -->
-  <xacro:macro name="pr2_upper_arm_roll_v0" params="side parent reflect *origin">
-    <joint name="${side}_upper_arm_roll_joint" type="revolute">
+  <xacro:macro name="pr2_upper_arm_roll_v0" params="side parent reflect *origin
+    upper_arm_roll_calib_ref:=0.0">
+    <joint name="${side}_upper_arm_roll_joint" type="revolute" >
       <axis xyz="1 0 0" />
       <xacro:insert_block name="origin" />
@@ -101,5 +116,10 @@
       <limit lower="${reflect*1.55-2.35}" upper="${reflect*1.55+2.35}" effort="30" velocity="${VELOCITY_LIMIT_SCALE*5.45}" /> <!-- alpha tested velocity and effort limits -->
       <safety_controller k_position="100" k_velocity="2" soft_lower_limit="${reflect*1.55-2.35+0.15}" soft_upper_limit="${reflect*1.55+2.35-0.15}" />
-      <calibration rising="${(reflect*M_PI/2)*cal_r_upper_arm_roll_gearing + cal_r_upper_arm_roll_flag}" />
+      <xacro:unless value="${upper_arm_roll_calib_ref}">
+        <calibration  rising="${(reflect*M_PI/2)*cal_r_upper_arm_roll_gearing+cal_r_upper_arm_roll_flag}" />
+      </xacro:unless>
+      <xacro:if value="${upper_arm_roll_calib_ref}">
+        <calibration  rising="${upper_arm_roll_calib_ref}" />
+      </xacro:if>
       <dynamics damping="0.1" />
     </joint>

File: pr2_description/urdf/torso_v0/torso.urdf.xacro (robot description, xacro)
@@ -4,10 +4,15 @@
   <xacro:include filename="$(find pr2_description)/urdf/torso_v0/torso.transmission.xacro" />
   <xacro:include filename="$(find pr2_description)/urdf/sensors/microstrain_3dmgx2_imu.urdf.xacro" />
-  <xacro:macro name="pr2_torso_v0" params="name parent *origin">
+  <xacro:macro name="pr2_torso_v0" params="name parent *origin torso_calib_ref:=0.0">
     <joint name="${name}_joint" type="prismatic">
       <axis xyz="0 0 1" />
       <limit lower="0.0" upper="0.33" effort="10000" velocity="0.013"/> <!-- alpha tested velocity and effort limits -->
       <safety_controller  k_velocity="2000000" soft_lower_limit="${0.0+0.0115}" soft_upper_limit="${0.33-0.005}" k_position="100" />
-      <calibration falling="0.00475" />
+      <xacro:unless value="${torso_calib_ref}">
+        <calibration  falling="0.00475" />
+      </xacro:unless>
+      <xacro:if value="${torso_calib_ref}">
+        <calibration  falling="${torso_calib_ref}" />
+      </xacro:if>
       <dynamics damping="20000.0" />
       <xacro:insert_block name="origin" />

File: pr2_description/urdf/upper_arm_v0/upper_arm.urdf.xacro (robot description, xacro)
@@ -28,5 +28,7 @@
   <!-- ============================   Upper Arm   ============================ -->
   <!-- Includes elbow flex, FA roll joints in macros below -->
-  <xacro:macro name="pr2_upper_arm_v0" params="side parent reflect">
+  <xacro:macro name="pr2_upper_arm_v0" params="side parent reflect
+   forearm_roll_calib_ref:=0.0
+   elbow_flex_calib_ref:=0.0 ">
     <joint name="${side}_upper_arm_joint" type="fixed">
       <origin xyz="0 0 0" rpy="0 0 0" />
@@ -64,8 +66,11 @@
     <!-- No transmission, since this a fixed joint w/o actuator -->
     <!-- Elbow flex, FA roll macros -->
-    <xacro:pr2_forearm_roll_v0 side="${side}" parent="${side}_elbow_flex_link" reflect="${reflect}" />
-    <xacro:pr2_elbow_flex_v0 side="${side}" parent="${side}_upper_arm_link" reflect="${reflect}" />
+    <xacro:pr2_forearm_roll_v0 side="${side}" parent="${side}_elbow_flex_link" reflect="${reflect}"
+                               forearm_roll_calib_ref="${forearm_roll_calib_ref}"/>
+    <xacro:pr2_elbow_flex_v0 side="${side}" parent="${side}_upper_arm_link" reflect="${reflect}"
+                             elbow_flex_calib_ref="${elbow_flex_calib_ref}"/>
   </xacro:macro>
-  <xacro:macro name="pr2_elbow_flex_v0" params="side parent reflect">
+  <xacro:macro name="pr2_elbow_flex_v0" params="side parent reflect
+   elbow_flex_calib_ref:=0.0">
     <!-- Elbow flex -->
     <joint name="${side}_elbow_flex_joint" type="revolute">
@@ -74,5 +79,10 @@
       <limit lower="-2.3213" upper="0.00" effort="30" velocity="${VELOCITY_LIMIT_SCALE*5.5}" /> <!-- alpha tested velocity and effort limits -->
       <safety_controller k_position="100" k_velocity="3" soft_lower_limit="${-2.3213+0.2}" soft_upper_limit="${0.00-0.15}" />
-      <calibration falling="${-1.1606 + cal_r_elbow_flex_flag}"/>
+      <xacro:unless value="${elbow_flex_calib_ref}">
+        <calibration falling="${-1.1606+cal_r_elbow_flex_flag}"/>
+      </xacro:unless>
+      <xacro:if value="${elbow_flex_calib_ref}">
+        <calibration falling="${elbow_flex_calib_ref}"/>
+      </xacro:if>
       <dynamics damping="1.0" />
       <origin xyz="0.4 0 0" rpy="0 0 0" />
@@ -106,5 +116,6 @@
   </xacro:macro>
   <!-- FA roll joint only -->
-  <xacro:macro name="pr2_forearm_roll_v0" params="side parent reflect">
+  <xacro:macro name="pr2_forearm_roll_v0" params="side parent reflect
+   forearm_roll_calib_ref:=0.0">
     <!-- forearm_roll_link is a fictitious link internal to elbow_flex_link, provides an attachment point for the actual forearm -->
     <joint name="${side}_forearm_roll_joint" type="continuous">
@@ -112,5 +123,10 @@
       <limit effort="30" velocity="${VELOCITY_LIMIT_SCALE*6}" /> <!-- alpha tested velocity and effort limits -->
       <safety_controller k_velocity="1" />
-      <calibration rising="${0.0 + cal_r_forearm_roll_flag}" />
+      <xacro:unless value="${forearm_roll_calib_ref}">
+      <calibration rising="${0.0+cal_r_forearm_roll_flag}" />
+      </xacro:unless>
+      <xacro:if value="${forearm_roll_calib_ref}">
+      <calibration rising="${forearm_roll_calib_ref}" />
+      </xacro:if>
       <dynamics damping="0.1" />
       <origin xyz="0 0 0" rpy="0 0 0" />
