Commit message: Moving forearm roll, elbow flex into sub macro of upperarm. Tested in gazebo, on beta unit. WG#3301

File: pr2_description/urdf/upper_arm_v0/upper_arm.gazebo.xacro (robot description, xacro)
@@ -19,5 +19,7 @@
       <material value="PR2/Green" />
     </gazebo>
-    <!-- Elbow flex -->
+  </xacro:macro>
+  <!-- Elbow flex -->
+  <xacro:macro name="pr2_elbow_flex_gazebo_v0" params="side">
     <!-- testing initial joint position, to be parsed at urdf2gazebo parse time -->
     <gazebo reference="${side}_elbow_flex_joint">
@@ -42,5 +44,7 @@
       <stopKp value="1000000.0" />
     </gazebo>
-    <!-- Forearm roll -->
+  </xacro:macro>
+  <!-- Forearm roll -->
+  <xacro:macro name="pr2_forearm_roll_gazebo_v0" params="side" >
     <gazebo reference="${side}_forearm_roll_link">
       <material value="PR2/RollLinks" />

File: pr2_description/urdf/upper_arm_v0/upper_arm.transmission.xacro (robot description, xacro)
@@ -5,5 +5,5 @@
        xmlns:xacro="http://ros.org/wiki/xacro">
   <!-- ============================   Upper Arm   ============================ -->
-  <xacro:macro name="pr2_upper_arm_transmission_v0" params="side">
+  <xacro:macro name="pr2_elbow_flex_transmission_v0" params="side">
     <!-- Elbow flex -->
     <transmission type="SimpleTransmission" name="${side}_elbow_flex_trans">
@@ -12,9 +12,11 @@
       <mechanicalReduction>${-13/3 * 127.532/15.28}</mechanicalReduction>
     </transmission>
-    <!-- Forearm roll -->
+  </xacro:macro>
+  <!-- Forearm roll -->
+  <xacro:macro name="pr2_forearm_roll_transmission_v0" params="side" >
     <transmission type="SimpleTransmission" name="${side}_forearm_roll_trans">
       <actuator name="${side}_forearm_roll_motor" />
       <joint name="${side}_forearm_roll_joint" />
-      <mechanicalReduction>-${576/25 * 55/14}</mechanicalReduction>
+      <mechanicalReduction>${-576/25 * 55/14}</mechanicalReduction>
     </transmission>
   </xacro:macro>

File: pr2_description/urdf/upper_arm_v0/upper_arm.urdf.xacro (robot description, xacro)
@@ -30,4 +30,5 @@
   <property name="ual_izz"  value= "0.07601594191" />
   <!-- ============================   Upper Arm   ============================ -->
+  <!-- Includes elbow flex, FA roll joints in macros below -->
   <xacro:macro name="pr2_upper_arm_v0" params="side parent reflect">
     <joint name="${side}_upper_arm_joint" type="fixed">
@@ -62,4 +63,12 @@
       </collision>
     </link>
+    <!-- extensions-->
+    <xacro:pr2_upper_arm_gazebo_v0 side="${side}" /> <!-- Has upperarm link -->
+    <!-- No transmission, since this a fixed joint w/o actuator -->
+    <!-- Elbow flex, FA roll macros -->
+    <xacro:pr2_forearm_roll_v0 side="${side}" parent="${side}_elbow_flex_link" reflect="${reflect}" />
+    <xacro:pr2_elbow_flex_v0 side="${side}" parent="${side}_upper_arm_link" reflect="${reflect}" />
+  </xacro:macro>
+  <xacro:macro name="pr2_elbow_flex_v0" params="side parent reflect">
     <!-- Elbow flex -->
     <joint name="${side}_elbow_flex_joint" type="revolute">
@@ -71,5 +80,5 @@
       <dynamics damping="1.0" />
       <origin xyz="0.4 0 0" rpy="0 0 0" />
-      <parent link="${side}_upper_arm_link"/>
+      <parent link="${parent}"/>
       <child link="${side}_elbow_flex_link"/>
     </joint>
@@ -96,4 +105,9 @@
       </collision>
     </link>
+    <xacro:pr2_elbow_flex_gazebo_v0 side="${side}" />
+    <xacro:pr2_elbow_flex_transmission_v0 side="${side}" />
+  </xacro:macro>
+  <!-- FA roll joint only -->
+  <xacro:macro name="pr2_forearm_roll_v0" params="side parent reflect">
     <!-- forearm_roll_link is a fictitious link internal to elbow_flex_link, provides an attachment point for the actual forearm -->
     <joint name="${side}_forearm_roll_joint" type="continuous">
@@ -104,5 +118,5 @@
       <dynamics damping="0.1" />
       <origin xyz="0 0 0" rpy="0 0 0" />
-      <parent link="${side}_elbow_flex_link"/>
+      <parent link="${parent}"/>
       <child link="${side}_forearm_roll_link"/>
     </joint>
@@ -133,7 +147,6 @@
       </collision>
     </link>
-    <!-- extensions-->
-    <xacro:pr2_upper_arm_gazebo_v0 side="${side}" />
-    <xacro:pr2_upper_arm_transmission_v0 side="${side}" />
+    <xacro:pr2_forearm_roll_gazebo_v0 side="${side}" />
+    <xacro:pr2_forearm_roll_transmission_v0 side="${side}" />
   </xacro:macro>
 </robot>
