Commit message: Making separate upperarm roll URDF for UA roll only test. #3422

File: pr2_description/urdf/shoulder_v0/shoulder.gazebo.xacro (robot description, xacro)
@@ -42,5 +42,7 @@
       <stopKp value="1000000.0" />
     </gazebo>
-    <!-- Upperarm roll: internal fixed attchment point for upper arm -->
+  </xacro:macro>
+  <!-- Upperarm roll: internal fixed attchment point for upper arm -->
+  <xacro:macro name="pr2_upper_arm_roll_gazebo_v0" params="side" >
     <gazebo reference="${side}_upper_arm_roll_link">
       <material value="PR2/RollLinks" />

File: pr2_description/urdf/shoulder_v0/shoulder.transmission.xacro (robot description, xacro)
@@ -17,5 +17,7 @@
       <mechanicalReduction>${13/3 * 245.532/17.19 / cal_r_shoulder_lift_gearing}</mechanicalReduction>
     </transmission>
-    <!-- Upperarm roll: internal fixed attchment point for upper arm -->
+  </xacro:macro>
+  <xacro:macro name="pr2_upper_arm_roll_transmission_v0" params="side" >
+        <!-- Upperarm roll: internal fixed attchment point for upper arm -->
     <transmission type="SimpleTransmission" name="${side}_upper_arm_roll_trans">
       <actuator name="${side}_upper_arm_roll_motor" />

File: pr2_description/urdf/shoulder_v0/shoulder.urdf.xacro (robot description, xacro)
@@ -87,9 +87,18 @@
       </collision>
     </link>
-    <!-- Upperarm roll: internal fixed attchment point for upper arm -->
+    <!-- Upper arm roll is separate macro -->
+    <xacro:pr2_upper_arm_roll_v0 side="${side}" parent="${side}_shoulder_lift_link" reflect="${reflect}" >
+      <origin xyz="0 0 0" rpy="0 0 0" />
+    </xacro:pr2_upper_arm_roll_v0>
+    <!-- extensions -->
+    <xacro:pr2_shoulder_gazebo_v0 side="${side}" />
+    <xacro:pr2_shoulder_transmission_v0 side="${side}" />
+  </xacro:macro>
+  <!-- Upperarm roll: internal fixed attchment point for upper arm -->
+  <xacro:macro name="pr2_upper_arm_roll_v0" params="side parent reflect *origin">
     <joint name="${side}_upper_arm_roll_joint" type="revolute">
       <axis xyz="1 0 0" />
-      <origin xyz="0 0 0" rpy="0 0 0" />
-      <parent link="${side}_shoulder_lift_link" />
+      <insert_block name="origin" />
+      <parent link="${parent}" />
       <child link="${side}_upper_arm_roll_link"/>
       <limit lower="${reflect*1.55-2.35}" upper="${reflect*1.55+2.35}" effort="30" velocity="${VELOCITY_LIMIT_SCALE*5.45}" /> <!-- alpha tested velocity and effort limits -->
@@ -124,6 +133,6 @@
     </link>
     <!-- extensions -->
-    <xacro:pr2_shoulder_gazebo_v0 side="${side}" />
-    <xacro:pr2_shoulder_transmission_v0 side="${side}" />
+    <xacro:pr2_upper_arm_roll_gazebo_v0 side="${side}" />
+    <xacro:pr2_upper_arm_roll_transmission_v0 side="${side}" />
   </xacro:macro>
 </robot>
