Commit message: fix typo.

File: pr2_description/urdf/shoulder_v0/shoulder.urdf.xacro (robot description, xacro)
@@ -111,5 +111,5 @@
         <origin xyz="0 0 0" rpy="0 0 0" />
         <geometry name="${side}_upper_arm_roll_visual_geom">
-          <mesh filename="package://pr2_description/shoulder_v0/meshes/upper_arm_roll.stl" />
+          <mesh filename="package://pr2_description/meshes/shoulder_v0/upper_arm_roll.stl" />
         </geometry>
         <material name="RollLinks" />

Commit message: update damping values

File: pr2_description/urdf/shoulder_v0/shoulder.urdf.xacro (robot description, xacro)
@@ -22,5 +22,5 @@
       <limit lower="${reflect*M_PI/4-1.5}"  upper="${reflect*M_PI/4+1.5}"
              effort="30" velocity="${VELOCITY_LIMIT_SCALE*3.48}" /> <!-- alpha tested velocity and effort limits -->
-      <dynamics damping="10.0" />
+      <dynamics damping="100.0" />
       <safety_controller k_position="100" k_velocity="10"
                          soft_lower_limit="${reflect*M_PI/4-1.5+0.15}"
@@ -62,5 +62,5 @@
       <!-- hold both reference_position and upper/lower for tick-tock, remove reference_positiion after verifying upper/lower works with calibration controllers.  if search velocity in pr2_calibration_controllers.yaml is +, the reference_position is rising, if - then it is falling -->
       <calibration reference_position="${cal_r_shoulder_lift_flag}" falling="${cal_r_shoulder_lift_flag}" />
-      <dynamics damping="10.0" />
+      <dynamics damping="100.0" />
       <origin xyz="0.1 0 0" rpy="0 0 0" />
       <parent link="${side}_shoulder_pan_link"/>
@@ -108,5 +108,5 @@
       <!-- hold both reference_position and upper/lower for tick-tock, remove reference_positiion after verifying upper/lower works with calibration controllers.  if search velocity in pr2_calibration_controllers.yaml is +, the reference_position is rising, if - then it is falling -->
       <calibration reference_position="${(reflect*M_PI/2)*cal_r_upper_arm_roll_gearing + cal_r_upper_arm_roll_flag}" rising="${(reflect*M_PI/2)*cal_r_upper_arm_roll_gearing + cal_r_upper_arm_roll_flag}" />
-      <dynamics damping="0.1" />
+      <dynamics damping="10.0" />
     </joint>
     <link name="${side}_upper_arm_roll_link">

Commit message: update damping.

File: pr2_description/urdf/shoulder_v0/shoulder.urdf.xacro (robot description, xacro)
@@ -62,5 +62,5 @@
       <!-- hold both reference_position and upper/lower for tick-tock, remove reference_positiion after verifying upper/lower works with calibration controllers.  if search velocity in pr2_calibration_controllers.yaml is +, the reference_position is rising, if - then it is falling -->
       <calibration reference_position="${cal_r_shoulder_lift_flag}" falling="${cal_r_shoulder_lift_flag}" />
-      <dynamics damping="100.0" />
+      <dynamics damping="50.0" />
       <origin xyz="0.1 0 0" rpy="0 0 0" />
       <parent link="${side}_shoulder_pan_link"/>
@@ -108,5 +108,5 @@
       <!-- hold both reference_position and upper/lower for tick-tock, remove reference_positiion after verifying upper/lower works with calibration controllers.  if search velocity in pr2_calibration_controllers.yaml is +, the reference_position is rising, if - then it is falling -->
       <calibration reference_position="${(reflect*M_PI/2)*cal_r_upper_arm_roll_gearing + cal_r_upper_arm_roll_flag}" rising="${(reflect*M_PI/2)*cal_r_upper_arm_roll_gearing + cal_r_upper_arm_roll_flag}" />
-      <dynamics damping="10.0" />
+      <dynamics damping="5.0" />
     </joint>
     <link name="${side}_upper_arm_roll_link">

Commit message: update damping

File: pr2_description/urdf/shoulder_v0/shoulder.urdf.xacro (robot description, xacro)
@@ -108,5 +108,5 @@
       <!-- hold both reference_position and upper/lower for tick-tock, remove reference_positiion after verifying upper/lower works with calibration controllers.  if search velocity in pr2_calibration_controllers.yaml is +, the reference_position is rising, if - then it is falling -->
       <calibration reference_position="${(reflect*M_PI/2)*cal_r_upper_arm_roll_gearing + cal_r_upper_arm_roll_flag}" rising="${(reflect*M_PI/2)*cal_r_upper_arm_roll_gearing + cal_r_upper_arm_roll_flag}" />
-      <dynamics damping="5.0" />
+      <dynamics damping="20.0" />
     </joint>
     <link name="${side}_upper_arm_roll_link">

File: pr2_description/urdf/upper_arm_v0/upper_arm.urdf.xacro (robot description, xacro)
@@ -79,5 +79,5 @@
       <!-- hold both reference_position and upper/lower for tick-tock, remove reference_positiion after verifying upper/lower works with calibration controllers.  if search velocity in pr2_calibration_controllers.yaml is +, the reference_position is rising, if - then it is falling -->
       <calibration reference_position="${-1.1606 + cal_r_elbow_flex_flag}" falling="${-1.1606 + cal_r_elbow_flex_flag}"/>
-      <dynamics damping="1.0" />
+      <dynamics damping="10.0" />
       <origin xyz="0.4 0 0" rpy="0 0 0" />
       <parent link="${parent}"/>

Commit message: turns out actions are failing due to damping being too large whcih prolonged settling time in sim.

File: pr2_description/urdf/shoulder_v0/shoulder.urdf.xacro (robot description, xacro)
@@ -22,5 +22,5 @@
       <limit lower="${reflect*M_PI/4-1.5}"  upper="${reflect*M_PI/4+1.5}"
              effort="30" velocity="${VELOCITY_LIMIT_SCALE*3.48}" /> <!-- alpha tested velocity and effort limits -->
-      <dynamics damping="100.0" />
+      <dynamics damping="10.0" />
       <safety_controller k_position="100" k_velocity="10"
                          soft_lower_limit="${reflect*M_PI/4-1.5+0.15}"
@@ -62,5 +62,5 @@
       <!-- hold both reference_position and upper/lower for tick-tock, remove reference_positiion after verifying upper/lower works with calibration controllers.  if search velocity in pr2_calibration_controllers.yaml is +, the reference_position is rising, if - then it is falling -->
       <calibration reference_position="${cal_r_shoulder_lift_flag}" falling="${cal_r_shoulder_lift_flag}" />
-      <dynamics damping="50.0" />
+      <dynamics damping="10.0" />
       <origin xyz="0.1 0 0" rpy="0 0 0" />
       <parent link="${side}_shoulder_pan_link"/>

Commit message: update damping

File: pr2_description/urdf/shoulder_v0/shoulder.urdf.xacro (robot description, xacro)
@@ -22,5 +22,5 @@
       <limit lower="${reflect*M_PI/4-1.5}"  upper="${reflect*M_PI/4+1.5}"
              effort="30" velocity="${VELOCITY_LIMIT_SCALE*3.48}" /> <!-- alpha tested velocity and effort limits -->
-      <dynamics damping="10.0" />
+      <dynamics damping="80.0" />
       <safety_controller k_position="100" k_velocity="10"
                          soft_lower_limit="${reflect*M_PI/4-1.5+0.15}"

Commit message: copy damping from boxturtle, result of MW tuning for plugging-in

File: pr2_description/urdf/shoulder_v0/shoulder.urdf.xacro (robot description, xacro)
@@ -22,5 +22,5 @@
       <limit lower="${reflect*M_PI/4-1.5}"  upper="${reflect*M_PI/4+1.5}"
              effort="30" velocity="${VELOCITY_LIMIT_SCALE*3.48}" /> <!-- alpha tested velocity and effort limits -->
-      <dynamics damping="80.0" />
+      <dynamics damping="10.0" />
       <safety_controller k_position="100" k_velocity="10"
                          soft_lower_limit="${reflect*M_PI/4-1.5+0.15}"
@@ -108,5 +108,5 @@
       <!-- hold both reference_position and upper/lower for tick-tock, remove reference_positiion after verifying upper/lower works with calibration controllers.  if search velocity in pr2_calibration_controllers.yaml is +, the reference_position is rising, if - then it is falling -->
       <calibration reference_position="${(reflect*M_PI/2)*cal_r_upper_arm_roll_gearing + cal_r_upper_arm_roll_flag}" rising="${(reflect*M_PI/2)*cal_r_upper_arm_roll_gearing + cal_r_upper_arm_roll_flag}" />
-      <dynamics damping="20.0" />
+      <dynamics damping="0.1" />
     </joint>
     <link name="${side}_upper_arm_roll_link">

File: pr2_description/urdf/upper_arm_v0/upper_arm.urdf.xacro (robot description, xacro)
@@ -79,5 +79,5 @@
       <!-- hold both reference_position and upper/lower for tick-tock, remove reference_positiion after verifying upper/lower works with calibration controllers.  if search velocity in pr2_calibration_controllers.yaml is +, the reference_position is rising, if - then it is falling -->
       <calibration reference_position="${-1.1606 + cal_r_elbow_flex_flag}" falling="${-1.1606 + cal_r_elbow_flex_flag}"/>
-      <dynamics damping="10.0" />
+      <dynamics damping="1.0" />
       <origin xyz="0.4 0 0" rpy="0 0 0" />
       <parent link="${parent}"/>
