Commit message: adding LightGrey material

File: pr2_description/urdf/materials.urdf.xacro (robot description, xacro)
@@ -19,4 +19,7 @@
     <color rgba="1.0 1.0 1.0 1.0"/>
   </material>
+  <material name="LightGrey">
+    <color rgba="0.6 0.6 0.6 1.0"/>
+  </material>
   <material name="Caster">
     <texture filename="package://pr2_ogre/Media/materials/textures/pr2_caster_texture.png" />

Commit message: adding black color for bellow

File: pr2_description/urdf/materials.urdf.xacro (robot description, xacro)
@@ -19,4 +19,7 @@
     <color rgba="1.0 1.0 1.0 1.0"/>
   </material>
+  <material name="Black">
+    <color rgba="0.1 0.1 0.1 1.0"/>
+  </material>
   <material name="LightGrey">
     <color rgba="0.6 0.6 0.6 1.0"/>
