Commit message: remove simulated joint from urdf #4233

File: pr2_description/urdf/gripper_v0/gripper.transmission.xacro (robot description, xacro)
@@ -30,5 +30,4 @@
                       r="${r}"
                       />
-      <simulated_gripper_joint name="${side}_gripper_simulated_joint" />
       <passive_joint  name="${side}_gripper_l_finger_joint"     />
       <passive_joint  name="${side}_gripper_r_finger_joint"     />

File: pr2_description/urdf/gripper_v0/gripper.urdf.xacro (robot description, xacro)
@@ -321,11 +321,4 @@
       <safety_controller k_velocity="5000.0" k_position="20.0" soft_lower_limit="${0.0-0.01}" soft_upper_limit="${0.09-0.002}" />
     </joint>
-    <!-- simulated gripper joint between gripper tips -->
-    <joint name="${side}_gripper_simulated_joint" type="prismatic">
-      <axis xyz="0 1 0" />
-      <dynamics damping="${gripper_damping}" />
-      <limit effort="1000.0" velocity="0.2" lower="0.0" upper="0.09" />
-      <safety_controller k_velocity="5000.0" k_position="20.0" soft_lower_limit="${0.0-0.01}" soft_upper_limit="${0.09-0.002}" />
-    </joint>
     <!-- extensions -->
     <xacro:pr2_gripper_gazebo_v0 side="${side}" />

Commit message: * removing visual for parallel links to prevent rviz error report for missing transforms  * adding transmissions for parallel links so every non-fixed link has a published joint state

File: pr2_description/urdf/gripper_v0/gripper.transmission.xacro (robot description, xacro)
@@ -38,4 +38,15 @@
       <passive_joint  name="${side}_gripper_l_finger_tip_joint" />
     </transmission>
+    <!-- parallel links -->
+    <transmission type="SimpleTransmission" name="${side}_gripper_l_parallel_trans">
+      <actuator name="${side}_gripper_l_parallel_motor" />
+      <joint name="${side}_gripper_l_parallel_joint" />
+      <mechanicalReduction>1</mechanicalReduction>
+    </transmission>
+    <transmission type="SimpleTransmission" name="${side}_gripper_r_parallel_trans">
+      <actuator name="${side}_gripper_r_parallel_motor" />
+      <joint name="${side}_gripper_r_parallel_joint" />
+      <mechanicalReduction>1</mechanicalReduction>
+    </transmission>
   </xacro:macro>
 </robot>

File: pr2_description/urdf/gripper_v0/gripper.urdf.xacro (robot description, xacro)
@@ -127,4 +127,5 @@
                   izz= "0.00018105446" />
       </inertial>
+<!--
       <visual>
         <origin xyz="${0.0914942479/2.0} 0 0" rpy="0 0 0.0541224233" />
@@ -134,4 +135,5 @@
         <material name="Green" />
       </visual>
+-->
       <collision>
         <origin xyz="${0.0914942479/2.0} 0 0" rpy="0 0 0.0541224233" />
@@ -153,4 +155,5 @@
                   izz= "0.00018106988" />
       </inertial>
+<!--
       <visual>
         <origin xyz="${0.0914942479/2.0} 0 0" rpy="0 0 -0.0541224233" />
@@ -160,4 +163,5 @@
         <material name="Green" />
       </visual>
+-->
       <collision>
         <origin xyz="${0.0914942479/2.0} 0 0" rpy="0 0 -0.0541224233" />

Commit message: bug fix, update joint name

File: pr2_description/urdf/gripper_v0/gripper.transmission.xacro (robot description, xacro)
@@ -39,12 +39,12 @@
     </transmission>
     <!-- parallel links -->
-    <transmission type="SimpleTransmission" name="${side}_gripper_l_parallel_trans">
-      <actuator name="${side}_gripper_l_parallel_motor" />
-      <joint name="${side}_gripper_l_parallel_joint" />
+    <transmission type="SimpleTransmission" name="${side}_gripper_l_parallel_root_trans">
+      <actuator name="${side}_gripper_l_parallel_root_motor" />
+      <joint name="${side}_gripper_l_parallel_root_joint" />
       <mechanicalReduction>1</mechanicalReduction>
     </transmission>
-    <transmission type="SimpleTransmission" name="${side}_gripper_r_parallel_trans">
-      <actuator name="${side}_gripper_r_parallel_motor" />
-      <joint name="${side}_gripper_r_parallel_joint" />
+    <transmission type="SimpleTransmission" name="${side}_gripper_r_parallel_root_trans">
+      <actuator name="${side}_gripper_r_parallel_root_motor" />
+      <joint name="${side}_gripper_r_parallel_root_joint" />
       <mechanicalReduction>1</mechanicalReduction>
     </transmission>

Commit message: move parallel links root joints into gripper transmission as passive joints

File: pr2_description/urdf/gripper_v0/gripper.transmission.xacro (robot description, xacro)
@@ -37,15 +37,6 @@
       <passive_joint  name="${side}_gripper_r_finger_tip_joint" />
       <passive_joint  name="${side}_gripper_l_finger_tip_joint" />
-    </transmission>
-    <!-- parallel links -->
-    <transmission type="SimpleTransmission" name="${side}_gripper_l_parallel_root_trans">
-      <actuator name="${side}_gripper_l_parallel_root_motor" />
-      <joint name="${side}_gripper_l_parallel_root_joint" />
-      <mechanicalReduction>1</mechanicalReduction>
-    </transmission>
-    <transmission type="SimpleTransmission" name="${side}_gripper_r_parallel_root_trans">
-      <actuator name="${side}_gripper_r_parallel_root_motor" />
-      <joint name="${side}_gripper_r_parallel_root_joint" />
-      <mechanicalReduction>1</mechanicalReduction>
+      <passive_joint  name="${side}_gripper_r_parallel_root_joint" />
+      <passive_joint  name="${side}_gripper_l_parallel_root_joint" />
     </transmission>
   </xacro:macro>

Commit message: renaming screw_joint to simulated_actuated_joint in transmission.  added screw constraint for torso as well.

File: pr2_description/urdf/gripper_v0/gripper.transmission.xacro (robot description, xacro)
@@ -40,6 +40,6 @@
       <passive_joint  name="${side}_gripper_l_finger_tip_joint" />
       <!-- screw joint to capture gripper "dynamics" -->
-      <screw_joint    name="${side}_gripper_motor_screw_joint"
-                      simulated_thread_pitch="3141.6"   />
+      <simulated_actuated_joint name="${side}_gripper_motor_screw_joint"
+                                simulated_reduction="3141.6"   />
     </transmission>
   </xacro:macro>

File: pr2_description/urdf/gripper_v0/gripper.urdf.xacro (robot description, xacro)
@@ -243,5 +243,5 @@
                   izz="0.001" />
       </inertial>
-      <!--
+      <!-- for debugging only
       <visual>
         <origin xyz="0 0 0" rpy="0 0 0" />
@@ -272,5 +272,5 @@
                   izz="0.0001" />
       </inertial>
-      <!--
+      <!-- for debugging only
       <visual>
         <origin xyz="0 0 0" rpy="0 0 0" />

File: pr2_description/urdf/torso_v0/torso.gazebo.xacro (robot description, xacro)
@@ -3,4 +3,5 @@
        xmlns:controller="http://playerstage.sourceforge.net/gazebo/xmlschema/#controller"
        xmlns:interface="http://playerstage.sourceforge.net/gazebo/xmlschema/#interface"
+       xmlns:joint="http://playerstage.sourceforge.net/gazebo/xmlschema/#joint"
        xmlns:xacro="http://ros.org/wiki/xacro">
   <xacro:macro name="pr2_torso_gazebo_v0" params="name">
@@ -17,4 +18,15 @@
       </sensor:contact>
     </gazebo>
+    <gazebo>
+      <joint:screw name="${name}_screw_torso_lift_joint">
+          <body1>${name}_motor_screw_link</body1>
+          <body2>${name}_link</body2>
+          <anchor>${name}_motor_screw_link</anchor>
+          <anchorOffset>0 0 0</anchorOffset>
+          <axis>0 0 1</axis>
+          <threadPitch>3141.6</threadPitch>
+          <damping>1000.0</damping>
+      </joint:screw>
+    </gazebo>
   </xacro:macro>
 </robot>

File: pr2_description/urdf/torso_v0/torso.transmission.xacro (robot description, xacro)
@@ -9,4 +9,6 @@
       <joint name="${name}_joint" />
       <mechanicalReduction>-52143.33</mechanicalReduction>
+      <simulated_actuated_joint name="${name}_motor_screw_joint"
+                                simulated_reduction="3141.6" />
     </transmission>
   </xacro:macro>

File: pr2_description/urdf/torso_v0/torso.urdf.xacro (robot description, xacro)
@@ -13,5 +13,5 @@
       <safety_controller  k_velocity="2000000" soft_lower_limit="${0.0+0.0115}" soft_upper_limit="${0.31-0.005}" k_position="100" />
       <calibration falling="0.00536" />
-      <dynamics damping="20000.0" /> <!-- strictly tuned for sim only right now -->
+      <dynamics damping="100.0" />
       <insert_block name="origin" />
       <parent link="${parent}"/>
@@ -67,4 +67,34 @@
       </inertial>
     </link>
+    <!-- actuated motor screw joint -->
+    <link name="${name}_motor_screw_link">
+      <inertial>
+        <mass value="1.0" />
+        <origin xyz="0 0 0" rpy="0 0 0" />
+        <inertia  ixx="0.001" ixy="0.0" ixz="0.0"
+                  iyy="0.001" iyz="0.0"
+                  izz="0.001" />
+      </inertial>
+      <!-- for debugging only
+      <visual>
+        <origin xyz="0 0 0" rpy="0 0 0" />
+        <geometry>
+          <box size="0.5 0.7 0.01" />
+        </geometry>
+      </visual>
+      <collision>
+        <origin xyz="0 0 0" rpy="0 0 0" />
+        <geometry>
+          <box size="0.5 0.7 0.01" />
+        </geometry>
+      </collision>
+      -->
+    </link>
+    <joint name="${name}_motor_screw_joint" type="continuous">
+      <origin xyz="-0.15 0.0 0.7"/>
+      <axis xyz="0 0 1"/>
+      <parent link="${parent}"/>
+      <child link="${name}_motor_screw_link"/>
+    </joint>
     <!-- extensions -->
     <xacro:pr2_torso_gazebo_v0 name="${name}" />
