Commit message: remove mesh dependency on pr2_defs per ticket #3529

File: pr2_description/urdf/gripper_v0/gripper.urdf.xacro (robot description, xacro)
@@ -46,5 +46,5 @@
         <origin xyz="0 0 0" rpy="0 0 0" />
         <geometry name="${prefix}_l_finger_visual_geom">
-          <mesh filename="package://pr2_defs/meshes/upper_finger_l.stl" />
+          <mesh filename="package://pr2_description/meshes/gripper_v0/upper_finger_l.stl" />
         </geometry>
         <material name="Grey" />
@@ -53,5 +53,5 @@
         <origin xyz="0 0 0" rpy="0 0 0" />
         <geometry name="${prefix}_l_finger_collision_geom">
-          <mesh filename="package://pr2_defs/meshes/convex/upper_finger_l_convex.stlb" />
+          <mesh filename="package://pr2_description/meshes/gripper_v0/convex/upper_finger_l_convex.stlb" />
         </geometry>
         <verbose value="Yes" />
@@ -82,5 +82,5 @@
         <origin xyz="0 0 0" rpy="0 0 0" />
         <geometry name="${prefix}_r_finger_visual_geom">
-          <mesh filename="package://pr2_defs/meshes/upper_finger_r.stl" />
+          <mesh filename="package://pr2_description/meshes/gripper_v0/upper_finger_r.stl" />
         </geometry>
         <material name="Grey" />
@@ -89,5 +89,5 @@
         <origin xyz="0 0 0" rpy="0 0 0" />
         <geometry name="${prefix}_r_finger_collision_geom">
-          <mesh filename="package://pr2_defs/meshes/convex/upper_finger_r_convex.stlb" />
+          <mesh filename="package://pr2_description/meshes/gripper_v0/convex/upper_finger_r_convex.stlb" />
         </geometry>
         <verbose value="Yes" />
@@ -115,5 +115,5 @@
         <origin xyz="0 0 0" rpy="0 0 0" />
         <geometry name="${prefix}_l_finger_tip_visual_geom">
-          <mesh filename="package://pr2_defs/meshes/finger_tip_l.stl" />
+          <mesh filename="package://pr2_description/meshes/gripper_v0/finger_tip_l.stl" />
         </geometry>
         <material name="Green" />
@@ -122,5 +122,5 @@
         <origin xyz="0 0 0" rpy="0 0 0" />
         <geometry name="${prefix}_l_finger_tip_collision_geom">
-          <mesh filename="package://pr2_defs/meshes/finger_tip_pad2_l.stl" />
+          <mesh filename="package://pr2_description/meshes/gripper_v0/finger_tip_pad2_l.stl" />
         </geometry>
         <verbose value="Yes" />
@@ -148,5 +148,5 @@
         <origin xyz="0 0 0" rpy="0 0 0" />
         <geometry name="${prefix}_r_finger_tip_visual_geom">
-          <mesh filename="package://pr2_defs/meshes/finger_tip_r.stl" />
+          <mesh filename="package://pr2_description/meshes/gripper_v0/finger_tip_r.stl" />
         </geometry>
         <material name="Green" />
@@ -155,5 +155,5 @@
         <origin xyz="0 0 0" rpy="0 0 0" />
         <geometry name="${prefix}_r_finger_tip_collision_geom">
-          <mesh filename="package://pr2_defs/meshes/finger_tip_pad2_r.stl" />
+          <mesh filename="package://pr2_description/meshes/gripper_v0/finger_tip_pad2_r.stl" />
         </geometry>
         <verbose value="Yes" />
@@ -180,5 +180,5 @@
         <origin xyz="0 0 0" rpy="0 0 0" />
         <geometry name="${side}_gripper_palm_visual_geom">
-          <mesh filename="package://pr2_defs/meshes/gripper_palm.stl" />
+          <mesh filename="package://pr2_description/meshes/gripper_v0/gripper_palm.stl" />
         </geometry>
         <material name="Red" />
@@ -187,5 +187,5 @@
         <origin xyz="0 0 0" rpy="0 0 0" />
         <geometry name="${side}_gripper_palm_collision_geom">
-          <mesh filename="package://pr2_defs/meshes/convex/gripper_palm_convex.stlb" />
+          <mesh filename="package://pr2_description/meshes/gripper_v0/convex/gripper_palm_convex.stlb" />
         </geometry>
         <verbose value="Yes" />

Commit message: switching gripper palm and uppper finger collision model to the same as visual.  tested in sim to have minimal performance impact when not grasping objects.

File: pr2_description/urdf/gripper_v0/gripper.urdf.xacro (robot description, xacro)
@@ -53,5 +53,5 @@
         <origin xyz="0 0 0" rpy="0 0 0" />
         <geometry name="${prefix}_l_finger_collision_geom">
-          <mesh filename="package://pr2_description/meshes/gripper_v0/convex/upper_finger_l_convex.stlb" />
+          <mesh filename="package://pr2_description/meshes/gripper_v0/upper_finger_l.stl" />
         </geometry>
         <verbose value="Yes" />
@@ -89,5 +89,5 @@
         <origin xyz="0 0 0" rpy="0 0 0" />
         <geometry name="${prefix}_r_finger_collision_geom">
-          <mesh filename="package://pr2_description/meshes/gripper_v0/convex/upper_finger_r_convex.stlb" />
+          <mesh filename="package://pr2_description/meshes/gripper_v0/upper_finger_r.stl" />
         </geometry>
         <verbose value="Yes" />
@@ -187,5 +187,5 @@
         <origin xyz="0 0 0" rpy="0 0 0" />
         <geometry name="${side}_gripper_palm_collision_geom">
-          <mesh filename="package://pr2_description/meshes/gripper_v0/convex/gripper_palm_convex.stlb" />
+          <mesh filename="package://pr2_description/meshes/gripper_v0/gripper_palm.stl" />
         </geometry>
         <verbose value="Yes" />

Commit message: Upped gripper effort limits to 1000.0

File: pr2_description/urdf/gripper_v0/gripper.urdf.xacro (robot description, xacro)
@@ -12,5 +12,5 @@
   <property name="finger_damping"             value="0.2" />
   <property name="finger_tip_damping"         value="0.01" />
-  <property name="finger_joint_effort_limit"  value="100.0" />
+  <property name="finger_joint_effort_limit"  value="1000.0" />
   <xacro:macro name="pr2_finger_limits_v0" params="reflect">
     <!-- limits on passive finger and finger top joints without
@@ -261,5 +261,5 @@
     <joint name="${side}_gripper_joint" type="prismatic">
       <axis xyz="0 0 1" />
-      <limit effort="100.0" velocity="0.2" lower="0.0" upper="0.09" />
+      <limit effort="1000.0" velocity="0.2" lower="0.0" upper="0.09" />
       <safety_controller k_velocity="500.0" k_position="20.0" soft_lower_limit="${0.0-0.01}" soft_upper_limit="${0.09-0.002}" />
     </joint>

Commit message: minor fix: clean up <collision name="..." > to simply <collision> as name tag for collision is not used.

File: pr2_description/urdf/gripper_v0/gripper.urdf.xacro (robot description, xacro)
@@ -53,5 +53,5 @@
         <material name="Grey" />
       </visual>
-      <collision name="${prefix}_l_finger_collision">
+      <collision>
         <origin xyz="0 0 0" rpy="0 0 0" />
         <geometry>
@@ -89,5 +89,5 @@
         <material name="Grey" />
       </visual>
-      <collision name="${prefix}_r_finger_collision">
+      <collision>
         <origin xyz="0 0 0" rpy="${M_PI} 0 0" />
         <geometry>
@@ -197,5 +197,5 @@
         <material name="Green" />
       </visual>
-      <collision name="${prefix}_l_finger_tip_collision">
+      <collision>
         <origin xyz="0 0 0" rpy="0 0 0" />
         <geometry>
@@ -230,5 +230,5 @@
         <material name="Green" />
       </visual>
-      <collision name="${prefix}_r_finger_tip_collision">
+      <collision>
         <origin xyz="0 0 0" rpy="${M_PI} 0 0" />
         <geometry>
@@ -262,5 +262,5 @@
         <material name="Red" />
       </visual>
-      <collision name="${side}_gripper_palm_collision">
+      <collision>
         <origin xyz="0 0 0" rpy="0 0 0" />
         <geometry>

Commit message: attach gripper joint to finger tips, ticket 4448

File: pr2_description/urdf/gripper_v0/gripper.urdf.xacro (robot description, xacro)
@@ -320,4 +320,6 @@
     -->
     <joint name="${side}_gripper_joint" type="prismatic">
+      <parent link="${side}_gripper_r_finger_tip_link"/>
+      <child link="${side}_gripper_l_finger_tip_frame"/>
       <axis xyz="0 1 0" />
       <dynamics damping="${gripper_damping}" />
@@ -325,4 +327,8 @@
       <safety_controller k_velocity="5000.0" k_position="20.0" soft_lower_limit="${0.0-0.01}" soft_upper_limit="${0.09-0.002}" />
     </joint>
+    <!-- This link is the same as the l_finger_tip_link,
+	 but because the urdf does not support graph structures,
+	 this link exists twice -->
+    <link name="${side}_gripper_l_finger_tip_frame" />
     <!-- extensions -->
     <xacro:pr2_gripper_gazebo_v0 side="${side}" />

Commit message: added limits to new simulation prismatic joint

File: pr2_description/urdf/gripper_v0/gripper.urdf.xacro (robot description, xacro)
@@ -263,4 +263,5 @@
       <parent link="${side}_gripper_palm_link"/>
       <child link="${side}_gripper_motor_slider_link"/>
+      <limit effort="1000.0" velocity="0.2" lower="-0.1" upper="0.1" />
     </joint>
     <link name="${side}_gripper_motor_screw_link">
