Commit message: moving gripper floating link into gazebo extension. this link is only used to enforce gripper parallelness in simulation.

File: pr2_description/urdf/gripper_v0/gripper.gazebo.xacro (robot description, xacro)
@@ -4,4 +4,6 @@
        xmlns:joint="http://playerstage.sourceforge.net/gazebo/xmlschema/#slider"
        xmlns:interface="http://playerstage.sourceforge.net/gazebo/xmlschema/#interface"
+       xmlns:body="http://playerstage.sourceforge.net/gazebo/xmlschema/#body"
+       xmlns:geom="http://playerstage.sourceforge.net/gazebo/xmlschema/#geom"
        xmlns:xacro="http://ros.org/wiki/xacro">
   <property name="finger_stop_kd"             value="1.0" />
@@ -161,4 +163,42 @@
     </gazebo>
     <gazebo>
+      <!-- floating link for enforcing gripper constraints -->
+      <body:box name="${side}_gripper_float_link">
+          <massMatrix>true</massMatrix>
+          <mass>0.01</mass>
+          <ixx>0.0001</ixx>
+          <ixy>0</ixy>
+          <ixz>0</ixz>
+          <iyy>0.0001</iyy>
+          <iyz>0</iyz>
+          <izz>0.0001</izz>
+          <cx>0</cx>
+          <cy>0</cy>
+          <cz>0</cz>
+          <xyz>0.82025 0.188 0.790675</xyz>
+          <rpy>0 -0 0</rpy>
+          <geom:box name="${side}_gripper_float_link_geom">
+              <xyz>0 0 0</xyz>
+              <rpy>0 -0 0</rpy>
+              <size>0.001 0.001 0.001</size>
+              <visual>
+                  <xyz>0 0 0</xyz>
+                  <rpy>0 -0 0</rpy>
+                  <scale>0.001 0.001 0.001</scale>
+                  <mesh>unit_box</mesh>
+                  <material>PR2/White</material>
+              </visual>
+          </geom:box>
+          <turnGravityOff>true</turnGravityOff>
+          <selfCollide>false</selfCollide>
+      </body:box>
+      <joint:slider name="${side}_gripper_float_joint">
+          <body1>${side}_gripper_float_link</body1>
+          <body2>${side}_gripper_palm_link</body2>
+          <anchor>${side}_gripper_float_link</anchor>
+          <axis>1 0 0</axis>
+          <lowStop>-0.05</lowStop>
+          <highStop>0.001</highStop>
+      </joint:slider>
       <joint:slider name="${side}_gripper_l_finger_tip_slider_joint">
           <body1>${side}_gripper_l_finger_tip_link</body1>

File: pr2_description/urdf/gripper_v0/gripper.urdf.xacro (robot description, xacro)
@@ -215,36 +215,4 @@
       </collision>
     </link>
-    <!-- floating link for simulating gripper constraints -->
-    <joint name="${side}_gripper_float_joint" type="prismatic">
-      <limit lower="-0.05" upper="0.001" velocity="10" effort="10" />
-      <axis xyz="1 0 0" />
-      <dynamics damping="10.0" />
-      <origin xyz="0.05 0 0" rpy="0 0 0" />
-      <parent link="${side}_gripper_palm_link"/>
-      <child link="${side}_gripper_float_link"/>
-    </joint>
-    <link name="${side}_gripper_float_link">
-      <inertial>
-        <mass value="0.01" />
-        <origin xyz="0 0 0" rpy="0 0 0" />
-        <inertia  ixx="0.0001" ixy="0" ixz="0"
-                  iyy="0.0001" iyz="0"
-                  izz="0.0001" />
-      </inertial>
-      <visual name="${side}_gripper_float_visual">
-        <origin xyz="0 0 0" rpy="0 0 0" />
-        <geometry name="${side}_gripper_float_visual_geom">
-          <box size="0.001 0.001 0.001" />
-        </geometry>
-        <material name="White" />
-      </visual>
-      <collision name="${side}_gripper_float_collision">
-        <origin xyz="0 0 0" rpy="0 0 0" />
-        <geometry name="${side}_gripper_float_collision_geom">
-          <box size="0.001 0.001 0.001" />
-        </geometry>
-        <verbose value="Yes" />
-      </collision>
-    </link>
     <joint name="${side}_gripper_tool_joint" type="fixed">
       <origin xyz="0.18 0 0" rpy="0 0 0" />

Commit message: removing gripper tool frame #3408

File: pr2_description/urdf/gripper_v0/gripper.gazebo.xacro (robot description, xacro)
@@ -227,32 +227,4 @@
       -->
     </gazebo>
-    <gazebo>
-      <controller:gazebo_ros_p3d name="p3d_${side}_gripper_palm_controller" plugin="libgazebo_ros_p3d.so">
-        <alwaysOn>true</alwaysOn>
-        <updateRate>100.0</updateRate>
-        <bodyName>${side}_gripper_palm_link</bodyName>
-        <topicName>${side}_gripper_palm_pose_ground_truth</topicName>
-        <xyzOffsets>0 0 0</xyzOffsets>
-        <rpyOffsets>0 0 0</rpyOffsets>
-        <gaussianNoise>0.0</gaussianNoise>
-        <frameName>base_link</frameName>
-        <interface:position name="p3d_${side}_gripper_palm_position_iface" />
-      </controller:gazebo_ros_p3d>
-      <controller:gazebo_ros_p3d name="p3d_${side}_gripper_tool_frame" plugin="libgazebo_ros_p3d.so">
-        <alwaysOn>true</alwaysOn>
-        <updateRate>100.0</updateRate>
-        <bodyName>${side}_gripper_tool_frame</bodyName>
-        <topicName>${side}_gripper_tool_frame_pose_ground_truth</topicName>
-        <xyzOffsets>0 0 0</xyzOffsets>
-        <rpyOffsets>0 0 0</rpyOffsets>
-        <gaussianNoise>0.0</gaussianNoise>
-        <frameName>base_link</frameName>
-        <interface:position name="p3d_${side}_gripper_tool_frame_position_iface" />
-      </controller:gazebo_ros_p3d>
-    </gazebo>
-    <gazebo reference="${side}_gripper_tool_frame">
-      <turnGravityOff>true</turnGravityOff>
-      <material value="PR2/Grey" />
-    </gazebo>
   </xacro:macro>
 </robot>

File: pr2_description/urdf/gripper_v0/gripper.urdf.xacro (robot description, xacro)
@@ -230,25 +230,5 @@
       <child link="${side}_gripper_tool_frame"/>
     </joint>
-    <link name="${side}_gripper_tool_frame">
-      <!-- TODO: all that follows is made-up and useless, but the old parser crashes without it -->
-      <inertial>
-        <mass value="0.01" />
-        <origin xyz="0 0 0" rpy="0 0 0" />
-        <inertia ixx="0.001" ixy="0" ixz="0" iyy="0.001" iyz="0" izz="0.001" />
-      </inertial>
-      <visual>
-        <origin xyz="0 0 0" rpy="0 0 0" />
-        <geometry name="${side}_gripper_tool_visual_geom">
-          <box size="0.001 0.001 0.001" />
-        </geometry>
-        <material name="Grey" />
-      </visual>
-      <collision>
-        <origin xyz="-0.1 0 0" rpy="0 0 0" /> <!-- move it out of the way -->
-        <geometry name="${side}_gripper_tool_collision_geom">
-          <box size="0.001 0.001 0.001" />
-        </geometry>
-      </collision>
-    </link>
+    <link name="${side}_gripper_tool_frame"/>
     <!-- pr2 fingers macro -->
     <xacro:pr2_finger_v0 prefix="${side}_gripper" parent="${side}_gripper_palm_link" />

Commit message: merging from trunk:  *removing gripper tool frame #3408

File: pr2_description/urdf/gripper_v0/gripper.gazebo.xacro (robot description, xacro)
@@ -251,8 +251,4 @@
       </controller:gazebo_ros_p3d>
     </gazebo>
-    <gazebo reference="${side}_gripper_tool_frame">
-      <turnGravityOff>true</turnGravityOff>
-      <material value="PR2/Grey" />
-    </gazebo>
   </xacro:macro>
 </robot>

Commit message: update simulation gripper joint:  * removed old slider "floating link".  * added parallel links to enforce tips stay parallel.  * added slider between finger tips.  * added slider to gripper transmission.  this will be used by updated pr2 gripper transmission.

File: pr2_description/urdf/gripper_v0/gripper.gazebo.xacro (robot description, xacro)
@@ -18,5 +18,5 @@
   <property name="finger_tip_mu"              value="500.0" />
   <property name="finger_mu"                  value="500.0" />
-  <xacro:macro name="pr2_finger_gazebo_v0" params="prefix">
+  <xacro:macro name="pr2_finger_gazebo_v0" params="prefix parallel_link_x_offset parallel_link_y_offset">
     <!-- Finger proximal digit -->
     <gazebo reference="${prefix}_l_finger_link">
@@ -141,4 +141,35 @@
       <provideFeedback value="true"/>
     </gazebo>
+    <!-- parallel link for simulating gripper constraints -->
+    <gazebo>
+      <joint:hinge name="${prefix}_r_parallel_tip_joint">
+          <body1>${prefix}_r_parallel_link</body1>
+          <body2>${prefix}_r_finger_tip_link</body2>
+          <anchor>${prefix}_r_finger_tip_link</anchor>
+          <axis>0 0 1</axis>
+          <anchorOffset>${parallel_link_x_offset} ${-parallel_link_y_offset} 0</anchorOffset>
+      </joint:hinge>
+      <joint:hinge name="${prefix}_l_parallel_tip_joint">
+          <body1>${prefix}_l_parallel_link</body1>
+          <body2>${prefix}_l_finger_tip_link</body2>
+          <anchor>${prefix}_l_finger_tip_link</anchor>
+          <axis>0 0 1</axis>
+          <anchorOffset>${parallel_link_x_offset} ${parallel_link_y_offset} 0</anchorOffset>
+      </joint:hinge>
+      <joint:slider name="${prefix}_simulated_joint">
+          <body1>${prefix}_l_finger_tip_link</body1>
+          <body2>${prefix}_r_finger_tip_link</body2>
+          <anchor>${prefix}_r_finger_tip_link</anchor>
+          <axis>0 1 0</axis>
+      </joint:slider>
+    </gazebo>
+    <gazebo reference="${prefix}_l_parallel_link">
+      <turnGravityOff>true</turnGravityOff>
+      <material value="PR2/Red" />
+    </gazebo>
+    <gazebo reference="${prefix}_r_parallel_link">
+      <turnGravityOff>true</turnGravityOff>
+      <material value="PR2/Red" />
+    </gazebo>
   </xacro:macro>
   <xacro:macro name="pr2_gripper_gazebo_v0" params="side">
@@ -156,74 +187,4 @@
       </sensor:contact>
       <material value="PR2/Red" />
-    </gazebo>
-    <!-- floating link for simulating gripper constraints -->
-    <gazebo reference="${side}_gripper_float_link">
-      <turnGravityOff>true</turnGravityOff>
-      <material value="PR2/White" />
-    </gazebo>
-    <gazebo>
-      <!-- floating link for enforcing gripper constraints -->
-      <body:box name="${side}_gripper_float_link">
-          <massMatrix>true</massMatrix>
-          <mass>0.01</mass>
-          <ixx>0.0001</ixx>
-          <ixy>0</ixy>
-          <ixz>0</ixz>
-          <iyy>0.0001</iyy>
-          <iyz>0</iyz>
-          <izz>0.0001</izz>
-          <cx>0</cx>
-          <cy>0</cy>
-          <cz>0</cz>
-          <xyz>0.82025 0.188 0.790675</xyz>
-          <rpy>0 -0 0</rpy>
-          <geom:box name="${side}_gripper_float_link_geom">
-              <xyz>0 0 0</xyz>
-              <rpy>0 -0 0</rpy>
-              <size>0.0 0.0 0.0</size>
-              <visual>
-                  <xyz>0 0 0</xyz>
-                  <rpy>0 -0 0</rpy>
-                  <scale>0.0 0.0 0.0</scale>
-                  <mesh>unit_box</mesh>
-                  <material>PR2/White</material>
-              </visual>
-          </geom:box>
-          <turnGravityOff>true</turnGravityOff>
-          <selfCollide>false</selfCollide>
-      </body:box>
-      <joint:slider name="${side}_gripper_float_joint">
-          <body1>${side}_gripper_float_link</body1>
-          <body2>${side}_gripper_palm_link</body2>
-          <anchor>${side}_gripper_float_link</anchor>
-          <axis>1 0 0</axis>
-          <lowStop>-0.05</lowStop>
-          <highStop>0.001</highStop>
-      </joint:slider>
-      <joint:slider name="${side}_gripper_l_finger_tip_slider_joint">
-          <body1>${side}_gripper_l_finger_tip_link</body1>
-          <body2>${side}_gripper_float_link</body2>
-          <anchor>${side}_gripper_l_finger_tip_link</anchor>
-          <axis>0 1 0</axis>
-          <anchorOffset>0 0 0</anchorOffset>
-      </joint:slider>
-      <joint:slider name="${side}_gripper_r_finger_tip_slider_joint">
-          <body1>${side}_gripper_r_finger_tip_link</body1>
-          <body2>${side}_gripper_float_link</body2>
-          <anchor>${side}_gripper_r_finger_tip_link</anchor>
-          <axis>0 1 0</axis>
-          <anchorOffset>0 0 0</anchorOffset>
-      </joint:slider>
-      <!--
-      <joint:slider name="${side}_gripper_finger_tip_slider_joint">
-          <body1>${side}_gripper_l_finger_tip_link</body1>
-          <body2>${side}_gripper_r_finger_tip_link</body2>
-          <anchor>${side}_gripper_l_finger_tip_link</anchor>
-          <axis>0 1 0</axis>
-          <anchorOffset>0 0 0</anchorOffset>
-          <lowStop>0.0</lowStop>
-          <highStop>0.08</highStop>
-      </joint:slider>
-      -->
     </gazebo>
     <gazebo>

File: pr2_description/urdf/gripper_v0/gripper.transmission.xacro (robot description, xacro)
@@ -30,4 +30,5 @@
                       r="${r}"
                       />
+      <simulated_gripper_joint name="${side}_gripper_simulated_joint" />
       <passive_joint  name="${side}_gripper_l_finger_joint"     />
       <passive_joint  name="${side}_gripper_r_finger_joint"     />

File: pr2_description/urdf/gripper_v0/gripper.urdf.xacro (robot description, xacro)
@@ -11,5 +11,8 @@
   <property name="gripper_lower_angle" value="0.00" />
   <property name="finger_damping"             value="0.2" />
+  <property name="gripper_damping"            value="100.0" />
   <property name="finger_tip_damping"         value="0.01" />
+  <property name="parallel_link_x_offset"     value="-0.018" />
+  <property name="parallel_link_y_offset"     value="0.021" />
   <property name="finger_joint_effort_limit"  value="1000.0" />
   <xacro:macro name="pr2_finger_limits_v0" params="reflect">
@@ -94,4 +97,75 @@
       </collision>
     </link>
+    <!-- Floating Link -->
+    <joint name="${prefix}_l_parallel_root_joint" type="revolute">
+      <axis xyz="0 0 1" />
+      <origin xyz="${0.07691+parallel_link_x_offset} ${+0.01+parallel_link_y_offset} 0" rpy="0 0 0" />
+      <dynamics damping="${finger_damping}" />
+      <mimic joint="${prefix}_l_finger_joint" multiplier="1" offset="0"/>
+      <parent link="${parent}"/>
+      <child link="${prefix}_l_parallel_link"/>
+      <xacro:pr2_finger_limits_v0 reflect="1" />
+    </joint>
+    <joint name="${prefix}_r_parallel_root_joint" type="revolute">
+      <axis xyz="0 0 -1" />
+      <origin xyz="${0.07691+parallel_link_x_offset} ${-0.01-parallel_link_y_offset} 0" rpy="0 0 0" />
+      <dynamics damping="${finger_damping}" />
+      <mimic joint="${prefix}_l_finger_joint" multiplier="-1" offset="0"/>
+      <parent link="${parent}"/>
+      <child link="${prefix}_r_parallel_link"/>
+      <xacro:pr2_finger_limits_v0 reflect="1" />
+    </joint>
+    <link name="${prefix}_l_parallel_link">
+      <inertial>
+        <mass value="0.17126" />
+        <origin xyz="${0.03598} 0.01730 -0.00164" rpy="0 0 0" />
+        <inertia  ixx= "0.00007756198"
+                  ixy= "0.00000149095"
+                  ixz="-0.00000983385"
+                  iyy= "0.00019708305"
+                  iyz="-0.00000306125"
+                  izz= "0.00018105446" />
+      </inertial>
+      <visual>
+        <origin xyz="${0.0914942479/2.0} 0 0" rpy="0 0 0.0541224233" />
+        <geometry>
+          <box size="${0.0914942479} 0.005 0.005" />
+        </geometry>
+        <material name="Green" />
+      </visual>
+      <collision>
+        <origin xyz="${0.0914942479/2.0} 0 0" rpy="0 0 0.0541224233" />
+        <geometry>
+          <box size="${0.0914942479} 0.005 0.005" />
+        </geometry>
+        <verbose value="Yes" />
+      </collision>
+    </link>
+    <link name="${prefix}_r_parallel_link">
+      <inertial>
+        <mass value="0.17389" />
+        <origin xyz="${0.03576} -0.01736 -0.00095" rpy="0 0 0" />
+        <inertia  ixx= "0.00007738410"
+                  ixy="-0.00000209309"
+                  ixz="-0.00000836228"
+                  iyy= "0.00019847383"
+                  iyz= "0.00000246110"
+                  izz= "0.00018106988" />
+      </inertial>
+      <visual>
+        <origin xyz="${0.0914942479/2.0} 0 0" rpy="0 0 -0.0541224233" />
+        <geometry>
+          <box size="${0.0914942479} 0.005 0.005" />
+        </geometry>
+        <material name="Green" />
+      </visual>
+      <collision>
+        <origin xyz="${0.0914942479/2.0} 0 0" rpy="0 0 -0.0541224233" />
+        <geometry>
+          <box size="${0.0914942479} 0.005 0.005" />
+        </geometry>
+        <verbose value="Yes" />
+      </collision>
+    </link>
     <!-- Finger tip -->
     <joint name="${prefix}_l_finger_tip_joint" type="revolute">
@@ -161,5 +235,5 @@
     </link>
     <!-- extensions -->
-    <xacro:pr2_finger_gazebo_v0 prefix="${prefix}" />
+    <xacro:pr2_finger_gazebo_v0 prefix="${prefix}" parallel_link_x_offset="${parallel_link_x_offset}" parallel_link_y_offset="${parallel_link_y_offset}" />
   </xacro:macro>
   <xacro:macro name="pr2_gripper_v0" params="side parent *origin gear_ratio screw_reduction theta0 phi0 t0 L0 h a b r">
@@ -242,5 +316,13 @@
     -->
     <joint name="${side}_gripper_joint" type="prismatic">
-      <axis xyz="0 0 1" />
+      <axis xyz="0 1 0" />
+      <dynamics damping="${gripper_damping}" />
+      <limit effort="1000.0" velocity="0.2" lower="0.0" upper="0.09" />
+      <safety_controller k_velocity="5000.0" k_position="20.0" soft_lower_limit="${0.0-0.01}" soft_upper_limit="${0.09-0.002}" />
+    </joint>
+    <!-- simulated gripper joint between gripper tips -->
+    <joint name="${side}_gripper_simulated_joint" type="prismatic">
+      <axis xyz="0 1 0" />
+      <dynamics damping="${gripper_damping}" />
       <limit effort="1000.0" velocity="0.2" lower="0.0" upper="0.09" />
       <safety_controller k_velocity="5000.0" k_position="20.0" soft_lower_limit="${0.0-0.01}" soft_upper_limit="${0.09-0.002}" />

Commit message: simulated gripper joint is named after urdf joint

File: pr2_description/urdf/gripper_v0/gripper.gazebo.xacro (robot description, xacro)
@@ -157,5 +157,5 @@
           <anchorOffset>${parallel_link_x_offset} ${parallel_link_y_offset} 0</anchorOffset>
       </joint:hinge>
-      <joint:slider name="${prefix}_simulated_joint">
+      <joint:slider name="${prefix}_joint">
           <body1>${prefix}_l_finger_tip_link</body1>
           <body2>${prefix}_r_finger_tip_link</body2>

File: pr2_description/urdf/gripper_v0/gripper.transmission.xacro (robot description, xacro)
@@ -30,5 +30,5 @@
                       r="${r}"
                       />
-      <simulated_gripper_joint name="${side}_gripper_simulated_joint" />
+      <use_simulated_gripper_joint/>
       <passive_joint  name="${side}_gripper_l_finger_joint"     />
       <passive_joint  name="${side}_gripper_r_finger_joint"     />
