Commit message: reduced finger damping and adding a screw joint for gazebo. still need to limit gripper slider / screw limits in case ode/gazebo does not support screw joints yet

File: pr2_description/urdf/gripper_v0/gripper.gazebo.xacro (robot description, xacro)
@@ -159,4 +159,24 @@
     </gazebo>
     <gazebo>
+      <joint:screw name="${prefix}_r_screw_screw_joint">
+          <body1>${prefix}_motor_screw_link</body1>
+          <body2>${prefix}_r_finger_tip_link</body2>
+          <anchor>${prefix}_r_finger_tip_link</anchor>
+          <anchorOffset>0 0 0</anchorOffset>
+          <axis>0 1 0</axis>
+          <threadPitch>-3141.6</threadPitch>
+          <damping>100.0</damping>
+      </joint:screw>
+      <joint:screw name="${prefix}_l_screw_screw_joint">
+          <body1>${prefix}_motor_screw_link</body1>
+          <body2>${prefix}_l_finger_tip_link</body2>
+          <anchor>${prefix}_l_finger_tip_link</anchor>
+          <anchorOffset>0 0 0</anchorOffset>
+          <axis>0 1 0</axis>
+          <threadPitch>3141.6</threadPitch>
+          <damping>10.0</damping>
+      </joint:screw>
+    </gazebo>
+    <gazebo>
       <joint:hinge name="${prefix}_r_parallel_root_joint">
           <body1>${prefix}_r_parallel_link</body1>

File: pr2_description/urdf/gripper_v0/gripper.transmission.xacro (robot description, xacro)
@@ -31,10 +31,15 @@
                       />
       <!-- if a gazebo joint exists as [l|r]_gripper_joint, use this tag to have
-           gripper transmission apply torque directly to prismatic joint -->
+           gripper transmission apply torque directly to prismatic joint
+           this should be the default behavior in diamondback, deprecating this flag -->
       <use_simulated_gripper_joint/>
+      <!-- set passive joint angles so things look nice in rviz -->
       <passive_joint  name="${side}_gripper_l_finger_joint"     />
       <passive_joint  name="${side}_gripper_r_finger_joint"     />
       <passive_joint  name="${side}_gripper_r_finger_tip_joint" />
       <passive_joint  name="${side}_gripper_l_finger_tip_joint" />
+      <!-- screw joint to capture gripper "dynamics" -->
+      <screw_joint    name="${side}_gripper_motor_screw_joint"
+                      simulated_thread_pitch="3141.6"   />
     </transmission>
   </xacro:macro>

File: pr2_description/urdf/gripper_v0/gripper.urdf.xacro (robot description, xacro)
@@ -10,8 +10,10 @@
   <property name="gripper_upper_angle" value="0.548" />
   <property name="gripper_lower_angle" value="0.00" />
-  <property name="finger_damping"             value="0.2" />
-  <property name="gripper_damping"            value="100.0" />
-  <property name="finger_tip_damping"         value="0.01" />
+  <property name="finger_damping"             value="0.02" />
+  <property name="gripper_damping"            value="10.0" />
+  <property name="finger_tip_damping"         value="0.001" />
   <property name="finger_joint_effort_limit"  value="1000.0" />
+  <property name="finger_to_finger_tip_x"     value="0.09137" />
+  <property name="palm_to_finger_x"           value="0.07691" />
   <xacro:macro name="pr2_finger_limits_v0">
     <!-- limits on passive finger and finger top joints without
@@ -62,5 +64,5 @@
     <joint name="${prefix}_r_finger_joint" type="revolute">
       <axis xyz="0 0 -1" />
-      <origin xyz="0.07691 -0.01 0" rpy="0 0 0" />
+      <origin xyz="${palm_to_finger_x} -0.01 0" rpy="0 0 0" />
       <xacro:pr2_finger_limits_v0/>
       <dynamics damping="${finger_damping}" />
@@ -98,5 +100,5 @@
     <joint name="${prefix}_l_finger_tip_joint" type="revolute">
       <axis xyz="0 0 -1" />
-      <origin xyz="0.09137 0.00495 0" rpy="0 0 0" />
+      <origin xyz="${finger_to_finger_tip_x} 0.00495 0" rpy="0 0 0" />
       <xacro:pr2_finger_limits_v0/>
       <dynamics damping="${finger_tip_damping}" />
@@ -232,4 +234,63 @@
     </joint>
     <link name="${side}_gripper_tool_frame"/>
+    <!-- actuated motor screw joint -->
+    <link name="${side}_gripper_motor_slider_link">
+      <inertial>
+        <mass value="0.01" />
+        <origin xyz="0 0 0" rpy="0 0 0" />
+        <inertia  ixx="0.001" ixy="0.0" ixz="0.0"
+                  iyy="0.001" iyz="0.0"
+                  izz="0.001" />
+      </inertial>
+      <!--
+      <visual>
+        <origin xyz="0 0 0" rpy="0 0 0" />
+        <geometry>
+          <box size="0.05 0.01 0.05" />
+        </geometry>
+      </visual>
+      <collision>
+        <origin xyz="0 0 0" rpy="0 0 0" />
+        <geometry>
+          <box size="0.05 0.01 0.05" />
+        </geometry>
+      </collision>
+      -->
+    </link>
+    <joint name="${side}_gripper_motor_slider_joint" type="prismatic">
+      <origin xyz="${finger_to_finger_tip_x+palm_to_finger_x} 0 0" rpy="0 0 0" />
+      <axis xyz="1 0 0"/>
+      <parent link="${side}_gripper_palm_link"/>
+      <child link="${side}_gripper_motor_slider_link"/>
+    </joint>
+    <link name="${side}_gripper_motor_screw_link">
+      <inertial>
+        <mass value="0.01" />
+        <origin xyz="0 0 0" rpy="0 0 0" />
+        <inertia  ixx="0.0001" ixy="0.0" ixz="0.0"
+                  iyy="0.0001" iyz="0.0"
+                  izz="0.0001" />
+      </inertial>
+      <!--
+      <visual>
+        <origin xyz="0 0 0" rpy="0 0 0" />
+        <geometry>
+          <box size="0.05 0.01 0.05" />
+        </geometry>
+      </visual>
+      <collision>
+        <origin xyz="0 0 0" rpy="0 0 0" />
+        <geometry>
+          <box size="0.05 0.01 0.05" />
+        </geometry>
+      </collision>
+      -->
+    </link>
+    <joint name="${side}_gripper_motor_screw_joint" type="continuous">
+      <origin xyz="0.0 0 0" rpy="0 0 0" />
+      <axis xyz="0 1 0"/>
+      <parent link="${side}_gripper_motor_slider_link"/>
+      <child link="${side}_gripper_motor_screw_link"/>
+    </joint>
     <!-- pr2 fingers macro -->
     <xacro:pr2_finger_v0 prefix="${side}_gripper" reflect="${reflect}" parent="${side}_gripper_palm_link" />

Commit message: moving damping to the right place.

File: pr2_description/urdf/gripper_v0/gripper.gazebo.xacro (robot description, xacro)
@@ -166,5 +166,4 @@
           <axis>0 1 0</axis>
           <threadPitch>-3141.6</threadPitch>
-          <damping>0.0001</damping>
       </joint:screw>
       <joint:screw name="${prefix}_l_screw_screw_joint">
@@ -175,5 +174,4 @@
           <axis>0 1 0</axis>
           <threadPitch>3141.6</threadPitch>
-          <damping>0.0001</damping>
       </joint:screw>
     </gazebo>

File: pr2_description/urdf/gripper_v0/gripper.urdf.xacro (robot description, xacro)
@@ -293,4 +293,5 @@
       <parent link="${side}_gripper_motor_slider_link"/>
       <child link="${side}_gripper_motor_screw_link"/>
+      <dynamics damping="0.0001" />
     </joint>
     <!-- pr2 fingers macro -->

File: pr2_description/urdf/torso_v0/torso.gazebo.xacro (robot description, xacro)
@@ -26,5 +26,4 @@
           <axis>0 0 1</axis>
           <threadPitch>3141.6</threadPitch>
-          <damping>0.01</damping>
       </joint:screw>
     </gazebo>

File: pr2_description/urdf/torso_v0/torso.urdf.xacro (robot description, xacro)
@@ -96,4 +96,5 @@
       <parent link="${parent}"/>
       <child link="${name}_motor_screw_link"/>
+      <dynamics damping="0.0001" />
     </joint>
     <!-- extensions -->

Commit message: fix gazebo gripper simulation

File: pr2_description/urdf/gripper_v0/gripper.gazebo.xacro (robot description, xacro)
@@ -162,5 +162,5 @@
           <body1>${prefix}_motor_screw_link</body1>
           <body2>${prefix}_r_finger_tip_link</body2>
-          <anchor>${prefix}_r_finger_tip_link</anchor>
+          <anchor>${prefix}_motor_screw_link</anchor>
           <anchorOffset>0 0 0</anchorOffset>
           <axis>0 1 0</axis>
@@ -170,5 +170,5 @@
           <body1>${prefix}_motor_screw_link</body1>
           <body2>${prefix}_l_finger_tip_link</body2>
-          <anchor>${prefix}_l_finger_tip_link</anchor>
+          <anchor>${prefix}_motor_screw_link</anchor>
           <anchorOffset>0 0 0</anchorOffset>
           <axis>0 1 0</axis>
@@ -213,4 +213,12 @@
           <axis>0 1 0</axis>
       </joint:slider>
+    </gazebo>
+    <gazebo reference="${prefix}_motor_slider_link">
+      <turnGravityOff>true</turnGravityOff>
+      <material value="PR2/Red" />
+    </gazebo>
+    <gazebo reference="${prefix}_motor_screw_link">
+      <turnGravityOff>true</turnGravityOff>
+      <material value="PR2/Red" />
     </gazebo>
     <gazebo reference="${prefix}_l_parallel_link">

File: pr2_description/urdf/gripper_v0/gripper.urdf.xacro (robot description, xacro)
@@ -240,13 +240,13 @@
       <!-- for debugging only
       <visual>
-        <origin xyz="0 0 0" rpy="0 0 0" />
-        <geometry>
-          <box size="0.05 0.01 0.05" />
-        </geometry>
-      </visual>
-      <collision>
-        <origin xyz="0 0 0" rpy="0 0 0" />
-        <geometry>
-          <box size="0.05 0.01 0.05" />
+        <origin xyz="0 0 0" rpy="1.5708 0 0" />
+        <geometry>
+          <cylinder length="0.002" radius="0.025"/>
+        </geometry>
+      </visual>
+      <collision>
+        <origin xyz="0 0 0" rpy="1.5708 0 0" />
+        <geometry>
+          <cylinder length="0.002" radius="0.025"/>
         </geometry>
       </collision>
@@ -272,11 +272,11 @@
         <origin xyz="0 0 0" rpy="0 0 0" />
         <geometry>
-          <box size="0.05 0.01 0.05" />
-        </geometry>
-      </visual>
-      <collision>
-        <origin xyz="0 0 0" rpy="0 0 0" />
-        <geometry>
-          <box size="0.05 0.01 0.05" />
+          <box size="0.05 0.001 0.05" />
+        </geometry>
+      </visual>
+      <collision>
+        <origin xyz="0 0 0" rpy="0 0 0" />
+        <geometry>
+          <box size="0.05 0.001 0.05" />
         </geometry>
       </collision>

Commit message: fix camera type (to depth for openni/prosilica plugins)

File: pr2_description/urdf/gripper_v0/gripper.gazebo.xacro (robot description, xacro)
@@ -179,5 +179,5 @@
     </gazebo>
     <gazebo>
-      <joint type="hinge" name="${prefix}_r_parallel_root_joint">
+      <joint type="revolute" name="${prefix}_r_parallel_root_joint">
           <child>${prefix}_r_parallel_link</child>
           <parent>${prefix}_palm_link</parent>
@@ -190,5 +190,5 @@
           <pose>${0.07691+parallel_link_x_offset} ${-0.01-parallel_link_y_offset} 0 0 0 0</pose>
       </joint>
-      <joint type="hinge" name="${prefix}_l_parallel_root_joint">
+      <joint type="revolute" name="${prefix}_l_parallel_root_joint">
           <child>${prefix}_l_parallel_link</child>
           <parent>${prefix}_palm_link</parent>
@@ -201,5 +201,5 @@
           <pose>${0.07691+parallel_link_x_offset} ${0.01+parallel_link_y_offset} 0 0 0 0</pose>
       </joint>
-      <joint type="hinge" name="${prefix}_r_parallel_tip_joint">
+      <joint type="revolute" name="${prefix}_r_parallel_tip_joint">
           <child>${prefix}_r_parallel_link</child>
           <parent>${prefix}_r_finger_tip_link</parent>
@@ -209,5 +209,5 @@
           <pose>${parallel_link_x_offset} ${-parallel_link_y_offset} 0 0 0 0</pose>
       </joint>
-      <joint type="hinge" name="${prefix}_l_parallel_tip_joint">
+      <joint type="revolute" name="${prefix}_l_parallel_tip_joint">
           <child>${prefix}_l_parallel_link</child>
           <parent>${prefix}_l_finger_tip_link</parent>
@@ -217,5 +217,5 @@
           <pose>${parallel_link_x_offset} ${parallel_link_y_offset} 0 0 0 0</pose>
       </joint>
-      <joint type="slider" name="${prefix}_joint">
+      <joint type="prismatic" name="${prefix}_joint">
           <parent>${prefix}_l_finger_tip_link</parent>
           <child>${prefix}_r_finger_tip_link</child>

File: pr2_description/urdf/sensors/kinect_camera.gazebo.xacro (robot description, xacro)
@@ -6,5 +6,5 @@
 <xacro:macro name="kinect_camera_gazebo_v0" params="name">
   <gazebo reference="${name}_frame">
-    <sensor type="camera" name="${name}_frame_sensor">
+    <sensor type="depth" name="${name}_frame_sensor">
       <update_rate>20.0</update_rate>
       <camera>
@@ -38,5 +38,5 @@
       </plugin>
     </sensor>
-    <sensor type="camera" name="${name}_frame_sensor">
+    <sensor type="depth" name="${name}_frame_sensor">
       <update_rate>20.0</update_rate>
       <camera>

File: pr2_description/urdf/sensors/kinect_prosilica_camera.gazebo.xacro (robot description, xacro)
@@ -6,5 +6,5 @@
 <xacro:macro name="kinect_ir_gazebo_v0" params="link_name frame_name camera_name">
   <gazebo reference="${link_name}">
-    <sensor type="camera" name="${name}_ir_sensor">
+    <sensor type="depth" name="${name}_ir_sensor">
       <update_rate>1.0</update_rate>
       <camera>
@@ -43,5 +43,5 @@
 <xacro:macro name="kinect_rgb_gazebo_v0" params="link_name frame_name camera_name">
   <gazebo reference="${link_name}">
-    <sensor type="camera" name="${name}_rgb_sensor">
+    <sensor type="depth" name="${name}_rgb_sensor">
       <update_rate>1.0</update_rate>
       <camera>
@@ -94,5 +94,5 @@
 <xacro:macro name="prosilica_cam_gazebo_v1" params="link_name frame_name camera_name ">
   <gazebo reference="${link_name}">
-    <sensor type="camera" name="${link_name}_sensor">
+    <sensor type="depth" name="${link_name}_sensor">
       <update_rate>1.0</update_rate>
       <camera>
@@ -123,5 +123,5 @@
       </plugin>
     </sensor>
-    <sensor type="camera" name="${link_name}_sim_pcd_sensor">
+    <sensor type="depth" name="${link_name}_sim_pcd_sensor">
       <update_rate>1.0</update_rate>
       <camera>

File: pr2_description/urdf/sensors/prosilica_gc2450_camera.gazebo.xacro (robot description, xacro)
@@ -6,5 +6,5 @@
 <xacro:macro name="prosilica_cam_gazebo_v0" params="camera_name frame_name">
   <gazebo reference="${frame_name}_frame">
-    <sensor type="camera" name="${frame_name}_sensor">
+    <sensor type="depth" name="${frame_name}_sensor">
       <update_rate>20.0</update_rate>
       <camera>

File: pr2_description/urdf/sensors/wge100_camera.gazebo.xacro (robot description, xacro)
@@ -20,5 +20,5 @@
           </clip>
         </camera>
-        <plugin name="${name}_controller" filename="libgazebo_ros_depth_camera.so">
+        <plugin name="${name}_controller" filename="libgazebo_ros_camera.so">
           <alwaysOn>true</alwaysOn>
           <updateRate>25.0</updateRate>
