Commit message: converting old gazebo xml to sdf

File: pr2_description/urdf/gripper_v0/gripper.gazebo.xacro (robot description, xacro)
@@ -1,9 +1,5 @@
 <?xml version="1.0"?>
-<robot xmlns:sensor="http://playerstage.sourceforge.net/gazebo/xmlschema/#sensor"
-       xmlns:controller="http://playerstage.sourceforge.net/gazebo/xmlschema/#controller"
-       xmlns:joint="http://playerstage.sourceforge.net/gazebo/xmlschema/#slider"
-       xmlns:interface="http://playerstage.sourceforge.net/gazebo/xmlschema/#interface"
+<robot xmlns:joint="http://playerstage.sourceforge.net/gazebo/xmlschema/#slider"
        xmlns:body="http://playerstage.sourceforge.net/gazebo/xmlschema/#body"
-       xmlns:geom="http://playerstage.sourceforge.net/gazebo/xmlschema/#geom"
        xmlns:xacro="http://ros.org/wiki/xacro">
   <property name="finger_stop_kd"             value="1.0" />
@@ -54,15 +50,16 @@
       <turnGravityOff>true</turnGravityOff>
       <selfCollide>false</selfCollide>
-      <sensor:contact name="${prefix}_l_finger_tip_contact_sensor">
-        <geom>${prefix}_l_finger_tip_link_geom</geom>
-        <updateRate>100.0</updateRate>
-        <controller:gazebo_ros_bumper name="${prefix}_l_finger_tip_gazebo_ros_bumper_controller" plugin="libgazebo_ros_bumper.so">
+      <sensor type="contact" name="${prefix}_l_finger_tip_contact_sensor">
+        <update_rate>100.0</update_rate>
+        <contact>
+          <collision>${prefix}_l_finger_tip_link_geom</collision>
+        </contact>
+        <plugin name="${prefix}_l_finger_tip_gazebo_ros_bumper_controller" filename="libgazebo_ros_bumper.so">
           <alwaysOn>true</alwaysOn>
           <frameName>${prefix}_l_finger_tip_link</frameName>
           <updateRate>100.0</updateRate>
           <bumperTopicName>${prefix}_l_finger_tip_bumper</bumperTopicName>
-          <interface:bumper name="${prefix}_l_finger_tip_gazebo_ros_bumper_iface" />
-        </controller:gazebo_ros_bumper>
-      </sensor:contact>
+        </plugin>
+      </sensor>
       <mu1 value="${finger_tip_mu}" />
       <mu2 value="${finger_tip_mu}" />
@@ -80,15 +77,16 @@
       <turnGravityOff>true</turnGravityOff>
       <selfCollide>false</selfCollide>
-      <sensor:contact name="${prefix}_r_finger_tip_contact_sensor">
-        <geom>${prefix}_r_finger_tip_link_geom</geom>
-        <updateRate>100.0</updateRate>
-        <controller:gazebo_ros_bumper name="${prefix}_r_finger_tip_gazebo_ros_bumper_controller" plugin="libgazebo_ros_bumper.so">
+      <sensor type="contact" name="${prefix}_r_finger_tip_contact_sensor">
+        <update_rate>100.0</update_rate>
+        <contact>
+          <collision>${prefix}_r_finger_tip_link_geom</collision>
+        </contact>
+        <plugin name="${prefix}_r_finger_tip_gazebo_ros_bumper_controller" filename="libgazebo_ros_bumper.so">
           <alwaysOn>true</alwaysOn>
           <frameName>${prefix}_r_finger_tip_link</frameName>
           <updateRate>100.0</updateRate>
           <bumperTopicName>${prefix}_r_finger_tip_bumper</bumperTopicName>
-          <interface:bumper name="${prefix}_r_finger_tip_gazebo_ros_bumper_iface" />
-        </controller:gazebo_ros_bumper>
-      </sensor:contact>
+        </plugin>
+      </sensor>
       <mu1 value="${finger_tip_mu}" />
       <mu2 value="${finger_tip_mu}" />
@@ -97,5 +95,5 @@
     </gazebo>
     <gazebo>
-      <controller:gazebo_ros_p3d name="p3d_${prefix}_l_finger_controller" plugin="libgazebo_ros_p3d.so">
+      <plugin name="p3d_${prefix}_l_finger_controller" filename="libgazebo_ros_p3d.so">
         <alwaysOn>true</alwaysOn>
         <updateRate>100.0</updateRate>
@@ -104,7 +102,6 @@
         <gaussianNoise>0.0</gaussianNoise>
         <frameName>base_link</frameName>
-        <interface:position name="p3d_${prefix}_l_finger_position_iface" />
-      </controller:gazebo_ros_p3d>
-      <controller:gazebo_ros_f3d name="f3d_${prefix}_l_finger_controller" plugin="libgazebo_ros_f3d.so">
+      </plugin>
+      <plugin name="f3d_${prefix}_l_finger_controller" filename="libgazebo_ros_f3d.so">
         <alwaysOn>true</alwaysOn>
         <updateRate>100.0</updateRate>
@@ -112,6 +109,5 @@
         <topicName>${prefix}_l_finger_force_ground_truth</topicName>
         <frameName>${prefix}_l_finger_link</frameName>
-        <interface:position name="f3d_${prefix}_l_finger_force_iface" />
-      </controller:gazebo_ros_f3d>
+      </plugin>
     </gazebo>
     <gazebo reference="${prefix}_r_finger_tip_joint">
@@ -236,5 +232,5 @@
     </gazebo>
     <gazebo>
-      <controller:gazebo_ros_p3d name="p3d_${side}_gripper_palm_controller" plugin="libgazebo_ros_p3d.so">
+      <plugin name="p3d_${side}_gripper_palm_controller" filename="libgazebo_ros_p3d.so">
         <alwaysOn>true</alwaysOn>
         <updateRate>100.0</updateRate>
@@ -245,6 +241,5 @@
         <gaussianNoise>0.0</gaussianNoise>
         <frameName>map</frameName>
-        <interface:position name="p3d_${side}_gripper_palm_position_iface" />
-      </controller:gazebo_ros_p3d>
+      </plugin>
       <!-- a formal implementation of grasp hack in gazebo with fixed joint -->
       <gripper name="${side}_grasp_hack">

File: pr2_description/urdf/sensors/hokuyo_lx30_laser.gazebo.xacro (robot description, xacro)
@@ -1,22 +1,27 @@
 <?xml version="1.0"?>
-<robot xmlns:sensor="http://playerstage.sourceforge.net/gazebo/xmlschema/#sensor"
-       xmlns:controller="http://playerstage.sourceforge.net/gazebo/xmlschema/#controller"
-       xmlns:interface="http://playerstage.sourceforge.net/gazebo/xmlschema/#interface"
-       xmlns:xacro="http://ros.org/wiki/xacro">
+<robot xmlns:xacro="http://ros.org/wiki/xacro">
   <xacro:macro name="hokuyo_lx30_laser_gazebo_v0" params="name ros_topic update_rate min_angle max_angle">
     <gazebo reference="${name}_link">
-      <sensor:ray name="${name}">
-        <rayCount>640</rayCount>
-        <rangeCount>640</rangeCount>
-        <laserCount>1</laserCount>
-        <origin>0.0 0.0 0.0</origin>
-        <displayRays>false</displayRays>
-        <minAngle>${min_angle*180.0/M_PI}</minAngle>
-        <maxAngle>${max_angle*180.0/M_PI}</maxAngle>
-        <minRange>0.08</minRange>
-        <maxRange>10.0</maxRange>
-        <resRange>0.01</resRange>
-        <updateRate>${update_rate}</updateRate>
-        <controller:gazebo_ros_laser name="gazebo_ros_${name}_controller" plugin="libgazebo_ros_laser.so">
+      <sensor type="ray" name="${name}">
+        <always_on>true</always_on>
+        <update_rate>${update_rate}</update_rate>
+        <pose>0 0 0 0 0 0</pose>
+        <visualize>false</visualize>
+        <ray>
+          <scan>
+            <horizontal>
+              <samples>640</samples>
+              <resolution>1</resolution>
+              <min_angle>${min_angle}</min_angle>
+              <max_angle>${max_angle}</max_angle>
+            </horizontal>
+          </scan>
+          <range>
+            <min>0.08</min>
+            <max>10.0</max>
+            <resolution>0.01</resolution>
+          </range>
+        </ray>
+        <plugin name="gazebo_ros_${name}_controller" filename="libgazebo_ros_laser.so">
           <gaussianNoise>0.005</gaussianNoise>
           <alwaysOn>true</alwaysOn>
@@ -24,7 +29,6 @@
           <topicName>${ros_topic}</topicName>
           <frameName>${name}_link</frameName>
-          <interface:laser name="gazebo_ros_${name}_iface" />
-        </controller:gazebo_ros_laser>
-      </sensor:ray>
+        </plugin>
+      </sensor>
     </gazebo>
   </xacro:macro>

File: pr2_description/urdf/sensors/kinect_camera.gazebo.xacro (robot description, xacro)
@@ -1,18 +1,22 @@
 <?xml version="1.0"?>
-<root xmlns:sensor="http://playerstage.sourceforge.net/gazebo/xmlschema/#sensor"
-      xmlns:controller="http://playerstage.sourceforge.net/gazebo/xmlschema/#controller"
-      xmlns:interface="http://playerstage.sourceforge.net/gazebo/xmlschema/#interface"
-      xmlns:xacro="http://ros.org/wiki/xacro">
+<root xmlns:xacro="http://ros.org/wiki/xacro">
 <xacro:macro name="kinect_camera_gazebo_v0" params="name">
   <gazebo reference="${name}_frame">
-    <sensor:camera name="${name}_frame_sensor">
-      <imageFormat>R8G8B8</imageFormat>
-      <imageSize>640 480</imageSize>
-      <hfov>57</hfov>
-      <nearClip>0.01</nearClip>
-      <farClip>5</farClip>
-      <updateRate>20.0</updateRate>
-      <baseline>0.2</baseline>
-      <controller:gazebo_ros_openni_kinect name="${name}_frame_controller" plugin="libgazebo_ros_openni_kinect.so">
+    <sensor type="depth" name="${name}_frame_sensor">
+      <always_on>true</always_on>
+      <update_rate>20.0</update_rate>
+      <camera>
+        <horizontal_fov>${57.0*M_PI/180.0}</horizontal_fov>
+        <image>
+          <format>R8G8B8</format>
+          <width>640</width>
+          <height>480</height>
+        </image>
+        <clip>
+          <near>0.01</near>
+          <far>5</far>
+        </clip>
+      </camera>
+      <plugin name="${name}_frame_controller" filename="libgazebo_ros_openni_kinect.so">
         <alwaysOn>true</alwaysOn>
         <updateRate>20.0</updateRate>
@@ -30,15 +34,22 @@
         <distortionT1>0.00000001</distortionT1>
         <distortionT2>0.00000001</distortionT2>
-      </controller:gazebo_ros_openni_kinect>
-    </sensor:camera>
-    <sensor:camera name="${name}_frame_sensor">
-      <imageFormat>R8G8B8</imageFormat>
-      <imageSize>640 480</imageSize>
-      <hfov>57</hfov>
-      <nearClip>0.01</nearClip>
-      <farClip>5</farClip>
-      <updateRate>20.0</updateRate>
-      <baseline>0.2</baseline>
-      <controller:gazebo_ros_openni_kinect name="${name}_frame_controller" plugin="libgazebo_ros_openni_kinect.so">
+      </plugin>
+    </sensor>
+    <sensor type="depth" name="${name}_frame_sensor">
+      <always_on>true</always_on>
+      <update_rate>20.0</update_rate>
+      <camera>
+        <horizontal_fov>${57.0*M_PI/180.0}</horizontal_fov>
+        <image>
+          <format>R8G8B8</format>
+          <width>640</width>
+          <height>480</height>
+        </image>
+        <clip>
+          <near>0.01</near>
+          <far>5</far>
+        </clip>
+      </camera>
+      <plugin name="${name}_frame_controller" filename="libgazebo_ros_openni_kinect.so">
         <alwaysOn>true</alwaysOn>
         <updateRate>20.0</updateRate>
@@ -54,6 +65,6 @@
         <distortionT1>0.00000001</distortionT1>
         <distortionT2>0.00000001</distortionT2>
-      </controller:gazebo_ros_openni_kinect>
-    </sensor:camera>
+      </plugin>
+    </sensor>
   </gazebo>
 </xacro:macro>

File: pr2_description/urdf/sensors/kinect_prosilica_camera.gazebo.xacro (robot description, xacro)
@@ -1,18 +1,23 @@
 <?xml version="1.0"?>
-<root xmlns:sensor="http://playerstage.sourceforge.net/gazebo/xmlschema/#sensor"
-      xmlns:controller="http://playerstage.sourceforge.net/gazebo/xmlschema/#controller"
-      xmlns:interface="http://playerstage.sourceforge.net/gazebo/xmlschema/#interface"
-      xmlns:xacro="http://ros.org/wiki/xacro">
+<root xmlns:xacro="http://ros.org/wiki/xacro">
 <xacro:macro name="kinect_ir_gazebo_v0" params="link_name frame_name camera_name">
   <gazebo reference="${link_name}">
-    <sensor:camera name="${name}_ir_sensor">
-      <imageFormat>L8</imageFormat>
-      <imageSize>640 480</imageSize>
-      <hfov>57</hfov>
-      <nearClip>0.01</nearClip>
-      <farClip>5</farClip>
-      <updateRate>1.0</updateRate>
-      <baseline>0.2</baseline>
-      <controller:gazebo_ros_openni_kinect name="${link_name}_controller" plugin="libgazebo_ros_openni_kinect.so">
+    <sensor type="depth" name="${name}_ir_sensor">
+      <always_on>true</always_on>
+      <update_rate>1.0</update_rate>
+      <camera>
+        <horizontal_fov>${57.0*M_PI/180.0}</horizontal_fov>
+        <image>
+          <format>L8</format>
+          <width>640</width>
+          <height>480</height>
+        </image>
+        <clip>
+          <near>0.01</near>
+          <far>5</far>
+        </clip>
+      </camera>
+      <plugin name="${link_name}_controller" filename="libgazebo_ros_openni_kinect.so">
+        <baseline>0.2</baseline>
         <alwaysOn>true</alwaysOn>
         <updateRate>1.0</updateRate>
@@ -30,6 +35,6 @@
         <distortionT1>0.00000001</distortionT1>
         <distortionT2>0.00000001</distortionT2>
-      </controller:gazebo_ros_openni_kinect>
-    </sensor:camera>
+      </plugin>
+    </sensor>
     <material value="Gazebo/Red" />
   </gazebo>
@@ -37,13 +42,20 @@
 <xacro:macro name="kinect_rgb_gazebo_v0" params="link_name frame_name camera_name">
   <gazebo reference="${link_name}">
-    <sensor:camera name="${name}_rgb_sensor">
-      <imageFormat>R8G8B8</imageFormat>
-      <imageSize>640 480</imageSize>
-      <hfov>57</hfov>
-      <nearClip>0.01</nearClip>
-      <farClip>5</farClip>
-      <updateRate>1.0</updateRate>
-      <baseline>0.2</baseline>
-      <controller:gazebo_ros_openni_kinect name="${link_name}_controller" plugin="libgazebo_ros_openni_kinect.so">
+    <sensor type="depth" name="${name}_rgb_sensor">
+      <always_on>true</always_on>
+      <update_rate>1.0</update_rate>
+      <camera>
+        <horizontal_fov>${57.0*M_PI/180.0}</horizontal_fov>
+        <image>
+          <format>R8G8B8</format>
+          <width>640</width>
+          <height>480</height>
+        </image>
+        <clip>
+          <near>0.01</near>
+          <far>5</far>
+        </clip>
+      </camera>
+      <plugin name="${link_name}_controller" filename="libgazebo_ros_openni_kinect.so">
         <alwaysOn>true</alwaysOn>
         <updateRate>1.0</updateRate>
@@ -59,6 +71,6 @@
         <distortionT1>0.00000001</distortionT1>
         <distortionT2>0.00000001</distortionT2>
-      </controller:gazebo_ros_openni_kinect>
-    </sensor:camera>
+      </plugin>
+    </sensor>
     <material value="Gazebo/Red" />
   </gazebo>
@@ -66,27 +78,35 @@
 <xacro:macro name="kinect_prosilica_gazebo" params="joint_name link_name">
   <gazebo>
-    <controller:gazebo_ros_srp name="${link_name}_srp_controller" plugin="libgazebo_ros_srp.so">
+    <plugin name="${link_name}_srp_controller" filename="libgazebo_ros_srp.so">
       <bodyName>${link_name}</bodyName>
       <jointName>${joint_name}</jointName>
       <topicName>${link_name}</topicName>
-    </controller:gazebo_ros_srp>
+    </plugin>
   </gazebo>
   <!-- also add transmission for this sliding joint -->
-      <transmission type="pr2_mechanism_model/SimpleTransmission" name="${joint_name}_trans">
-      <actuator name="${joint_name}_motor" />
-      <joint name="${joint_name}" />
-      <mechanicalReduction>1</mechanicalReduction>
-    </transmission>
+  <transmission type="pr2_mechanism_model/SimpleTransmission" name="${joint_name}_trans">
+    <actuator name="${joint_name}_motor" />
+    <joint name="${joint_name}" />
+    <mechanicalReduction>1</mechanicalReduction>
+  </transmission>
 </xacro:macro>
 <xacro:macro name="prosilica_cam_gazebo_v1" params="link_name frame_name camera_name ">
   <gazebo reference="${link_name}">
-    <sensor:camera name="${link_name}_sensor">
-      <imageFormat>R8G8B8</imageFormat>
-      <imageSize>320 240</imageSize>
-      <hfov>64.2</hfov>
-      <nearClip>0.1</nearClip>
-      <farClip>100</farClip>
-      <updateRate>1.0</updateRate>
-      <controller:gazebo_ros_prosilica name="${link_name}_controller" plugin="libgazebo_ros_prosilica.so">
+    <sensor type="depth" name="${link_name}_sensor">
+      <always_on>true</always_on>
+      <update_rate>1.0</update_rate>
+      <camera>
+        <horizontal_fov>${64.2*M_PI/180.0}</horizontal_fov>
+        <image>
+          <format>R8G8B8</format>
+          <width>320</width>
+          <height>240</height>
+        </image>
+        <clip>
+          <near>0.1</near>
+          <far>100</far>
+        </clip>
+      </camera>
+      <plugin name="${link_name}_controller" filename="libgazebo_ros_prosilica.so">
         <alwaysOn>true</alwaysOn>
         <updateRate>1.0</updateRate>
@@ -101,14 +121,22 @@
         <distortionT1>0.0</distortionT1>
         <distortionT2>0.0</distortionT2>
-      </controller:gazebo_ros_prosilica>
-    </sensor:camera>
-    <sensor:camera name="${link_name}_sim_pcd_sensor">
-      <imageFormat>R8G8B8</imageFormat>
-      <imageSize>320 240</imageSize>
-      <hfov>64.2</hfov>
-      <nearClip>0.1</nearClip>
-      <farClip>100</farClip>
-      <updateRate>1.0</updateRate>
-      <controller:gazebo_ros_openni_kinect name="${link_name}_sim_pcd_controller" plugin="libgazebo_ros_openni_kinect.so">
+      </plugin>
+    </sensor>
+    <sensor type="depth" name="${link_name}_sim_pcd_sensor">
+      <always_on>true</always_on>
+      <update_rate>1.0</update_rate>
+      <camera>
+        <horizontal_fov>${64.2*M_PI/180.0}</horizontal_fov>
+        <image>
+          <format>R8G8B8</format>
+          <width>320</width>
+          <height>240</height>
+        </image>
+        <clip>
+          <near>0.1</near>
+          <far>100</far>
+        </clip>
+      </camera>
+      <plugin name="${link_name}_sim_pcd_controller" filename="libgazebo_ros_openni_kinect.so">
         <alwaysOn>true</alwaysOn>
         <updateRate>1.0</updateRate>
@@ -117,6 +145,6 @@
         <cameraInfoTopicName>camera_info</cameraInfoTopicName>
         <frameName>${frame_name}</frameName>
-      </controller:gazebo_ros_openni_kinect>
-    </sensor:camera>
+      </plugin>
+    </sensor>
     <material value="Gazebo/Red" />
   </gazebo>

File: pr2_description/urdf/sensors/microstrain_3dmgx2_imu.gazebo.xacro (robot description, xacro)
@@ -1,9 +1,7 @@
 <?xml version="1.0"?>
-<robot xmlns:controller="http://playerstage.sourceforge.net/gazebo/xmlschema/#controller"
-       xmlns:interface="http://playerstage.sourceforge.net/gazebo/xmlschema/#interface"
-       xmlns:xacro="http://ros.org/wiki/xacro">
+<robot xmlns:xacro="http://ros.org/wiki/xacro">
   <xacro:macro name="microstrain_3dmgx2_imu_gazebo_v0" params="name imu_topic update_rate stdev">
     <gazebo>
-      <controller:gazebo_ros_imu name="imu_controller" plugin="libgazebo_ros_imu.so">
+      <plugin name="imu_controller" filename="libgazebo_ros_imu.so">
         <alwaysOn>true</alwaysOn>
         <updateRate>${update_rate}</updateRate>
@@ -13,6 +11,5 @@
         <xyzOffset>0 0 0</xyzOffset>
         <rpyOffset>0 -180.0 0</rpyOffset>
-        <interface:position name="imu_position"/>
-      </controller:gazebo_ros_imu>
+      </plugin>
     </gazebo>
   </xacro:macro>

File: pr2_description/urdf/sensors/projector_wg6802418.gazebo.xacro (robot description, xacro)
@@ -1,7 +1,4 @@
 <?xml version="1.0"?>
-<root xmlns:sensor="http://playerstage.sourceforge.net/gazebo/xmlschema/#sensor"
-      xmlns:controller="http://playerstage.sourceforge.net/gazebo/xmlschema/#controller"
-      xmlns:interface="http://playerstage.sourceforge.net/gazebo/xmlschema/#interface"
-      xmlns:xacro="http://ros.org/wiki/xacro">
+<root xmlns:xacro="http://ros.org/wiki/xacro">
 <!-- this controller is pushed into a body scope (previously model scope)
      this will only work with added r36415 patch in simulator_gazebo stack
@@ -18,5 +15,5 @@
   </gazebo>
   <gazebo>
-    <controller:gazebo_ros_projector name="${name}_controller" plugin="libgazebo_ros_projector.so">
+    <plugin name="${name}_controller" filename="libgazebo_ros_projector.so">
       <projector>${name}_child_frame/${name}_projector_wg6802418</projector>
       <alwaysOn>true</alwaysOn>
@@ -26,5 +23,5 @@
       <textureTopicName>${name}_controller/image</textureTopicName>
       <projectorTopicName>${name}_controller/projector</projectorTopicName>
-    </controller:gazebo_ros_projector>
+    </plugin>
   </gazebo>
 </xacro:macro>

File: pr2_description/urdf/sensors/prosilica_gc2450_camera.gazebo.xacro (robot description, xacro)
@@ -1,18 +1,22 @@
 <?xml version="1.0"?>
-<root xmlns:sensor="http://playerstage.sourceforge.net/gazebo/xmlschema/#sensor"
-      xmlns:controller="http://playerstage.sourceforge.net/gazebo/xmlschema/#controller"
-      xmlns:interface="http://playerstage.sourceforge.net/gazebo/xmlschema/#interface"
-      xmlns:xacro="http://ros.org/wiki/xacro">
+<root xmlns:xacro="http://ros.org/wiki/xacro">
 <xacro:macro name="prosilica_cam_gazebo_v0" params="camera_name frame_name">
   <gazebo reference="${frame_name}_frame">
-    <sensor:camera name="${frame_name}_sensor">
-      <imageFormat>R8G8B8</imageFormat>
-      <imageSize>2448 2050</imageSize>
-      <hfov>45</hfov>
-      <nearClip>0.1</nearClip>
-      <farClip>100</farClip>
-      <updateRate>20.0</updateRate>
-      <controller:gazebo_ros_prosilica name="${frame_name}_controller" plugin="libgazebo_ros_prosilica.so">
-        <alwaysOn>true</alwaysOn>
+    <sensor type="depth" name="${frame_name}_sensor">
+      <always_on>true</always_on>
+      <update_rate>20.0</update_rate>
+      <camera>
+        <horizontal_fov>${M_PI/4}</horizontal_fov>
+        <image>
+          <format>R8G8B8</format>
+          <width>2448</width>
+          <height>2050</height>
+        </image>
+        <clip>
+          <near>0.1</near>
+          <far>100</far>
+        </clip>
+      </camera>
+      <plugin name="${frame_name}_controller" filename="libgazebo_ros_prosilica.so">
         <updateRate>20.0</updateRate>
         <cameraName>${camera_name}</cameraName>
@@ -24,5 +28,5 @@
         <Cx>1224.5</Cx>
         <Cy>1025.5</Cy>
-        <focalLength>2955</focalLength> <!-- image_width / (2*tan(hfov_radian /2)) -->
+        <focalLength>2955</focalLength>
         <distortionK1>0.0</distortionK1>
         <distortionK2>0.0</distortionK2>
@@ -30,6 +34,6 @@
         <distortionT1>0.0</distortionT1>
         <distortionT2>0.0</distortionT2>
-      </controller:gazebo_ros_prosilica>
-    </sensor:camera>
+      </plugin>
+    </sensor>
     <material value="Gazebo/Black" />
   </gazebo>
