Commit message: converting old gazebo xml to sdf

File: pr2_description/urdf/sensors/wge100_camera.gazebo.xacro (robot description, xacro)
@@ -1,17 +1,22 @@
 <?xml version="1.0"?>
-<robot xmlns:sensor="http://playerstage.sourceforge.net/gazebo/xmlschema/#sensor"
-       xmlns:controller="http://playerstage.sourceforge.net/gazebo/xmlschema/#controller"
-       xmlns:interface="http://playerstage.sourceforge.net/gazebo/xmlschema/#interface"
-       xmlns:xacro="http://ros.org/wiki/xacro">
+<robot xmlns:xacro="http://ros.org/wiki/xacro">
   <xacro:macro name="wge100_camera_gazebo_v0" params="name camera_name image_format image_topic_name camera_info_topic_name hfov focal_length frame_id hack_baseline image_width image_height">
     <gazebo reference="${name}_frame">
-      <sensor:camera name="${name}_sensor">
-        <imageSize>${image_width} ${image_height}</imageSize>
-        <imageFormat>${image_format}</imageFormat>
-        <hfov>${hfov}</hfov>
-        <nearClip>0.1</nearClip>
-        <farClip>100</farClip>
-        <updateRate>25.0</updateRate>
-        <controller:gazebo_ros_depth_camera name="${name}_controller" plugin="libgazebo_ros_depth_camera.so">
+      <sensor type="depth" name="${name}_sensor">
+        <always_on>true</always_on>
+        <update_rate>25.0</update_rate>
+        <camera>
+          <horizontal_fov>${hfov}</horizontal_fov>
+          <image>
+            <format>${image_format}</format>
+            <width>${image_width}</width>
+            <height>${image_height}</height>
+          </image>
+          <clip>
+            <near>0.1</near>
+            <far>100</far>
+          </clip>
+        </camera>
+        <plugin name="${name}_controller" filename="libgazebo_ros_depth_camera.so">
           <alwaysOn>true</alwaysOn>
           <updateRate>25.0</updateRate>
@@ -32,7 +37,6 @@
           <distortionT1>0.0</distortionT1>
           <distortionT2>0.0</distortionT2>
-          <interface:camera name="${name}_iface" />
-        </controller:gazebo_ros_depth_camera>
-      </sensor:camera>
+        </plugin>
+      </sensor>
       <turnGravityOff>true</turnGravityOff>
       <material>PR2/Blue</material>

File: pr2_description/urdf/torso_v0/torso.gazebo.xacro (robot description, xacro)
@@ -2,5 +2,4 @@
 <robot xmlns:sensor="http://playerstage.sourceforge.net/gazebo/xmlschema/#sensor"
        xmlns:controller="http://playerstage.sourceforge.net/gazebo/xmlschema/#controller"
-       xmlns:interface="http://playerstage.sourceforge.net/gazebo/xmlschema/#interface"
        xmlns:joint="http://playerstage.sourceforge.net/gazebo/xmlschema/#joint"
        xmlns:xacro="http://ros.org/wiki/xacro">
@@ -14,5 +13,4 @@
           <updateRate>100.0</updateRate>
           <bumperTopicName>${name}_bumper</bumperTopicName>
-          <interface:bumper name="${name}_gazebo_ros_bumper_iface" />
         </controller:gazebo_ros_bumper>
       </sensor:contact>

Commit message: changed old gazebo xml to sdf

File: pr2_description/urdf/gripper_v0/gripper.gazebo.xacro (robot description, xacro)
@@ -1,6 +1,4 @@
 <?xml version="1.0"?>
-<robot xmlns:joint="http://playerstage.sourceforge.net/gazebo/xmlschema/#slider"
-       xmlns:body="http://playerstage.sourceforge.net/gazebo/xmlschema/#body"
-       xmlns:xacro="http://ros.org/wiki/xacro">
+<robot xmlns:xacro="http://ros.org/wiki/xacro">
   <property name="finger_stop_kd"             value="1.0" />
   <property name="finger_stop_kp"             value="10000000.0" />
@@ -119,94 +117,101 @@
     <!-- parallel link for simulating gripper constraints -->
     <gazebo>
-      <body:box name="${prefix}_l_parallel_link">
-          <massMatrix>true</massMatrix>
-          <mass>0.17126</mass>
-          <ixx>7.7562e-05</ixx>
-          <ixy>1.49095e-06</ixy>
-          <ixz>-9.83385e-06</ixz>
-          <iyy>0.000197083</iyy>
-          <iyz>-3.06125e-06</iyz>
-          <izz>0.000181054</izz>
-          <cx>0.03598</cx>
-          <cy>0.0173</cy>
-          <cz>-0.00164</cz>
-          <xyz>0.82991 ${0.188*reflect+0.031} 0.790675</xyz>
-          <rpy>0 -0 0</rpy>
-          <turnGravityOff>true</turnGravityOff>
-          <selfCollide>false</selfCollide>
-      </body:box>
-      <body:box name="${prefix}_r_parallel_link">
-          <massMatrix>true</massMatrix>
-          <mass>0.17389</mass>
-          <ixx>7.73841e-05</ixx>
-          <ixy>-2.09309e-06</ixy>
-          <ixz>-8.36228e-06</ixz>
-          <iyy>0.000198474</iyy>
-          <iyz>2.4611e-06</iyz>
-          <izz>0.00018107</izz>
-          <cx>0.03576</cx>
-          <cy>-0.01736</cy>
-          <cz>-0.00095</cz>
-          <xyz>0.82991 ${0.188*reflect-0.031} 0.790675</xyz>
-          <rpy>0 -0 0</rpy>
-          <turnGravityOff>true</turnGravityOff>
-          <selfCollide>false</selfCollide>
-      </body:box>
-    </gazebo>
-    <gazebo>
-      <joint:screw name="${prefix}_r_screw_screw_joint">
-          <body1>${prefix}_motor_screw_link</body1>
-          <body2>${prefix}_r_finger_tip_link</body2>
-          <anchor>${prefix}_motor_screw_link</anchor>
-          <anchorOffset>0 0 0</anchorOffset>
-          <axis>0 1 0</axis>
-          <threadPitch>-3141.6</threadPitch>
-      </joint:screw>
-      <joint:screw name="${prefix}_l_screw_screw_joint">
-          <body1>${prefix}_motor_screw_link</body1>
-          <body2>${prefix}_l_finger_tip_link</body2>
-          <anchor>${prefix}_motor_screw_link</anchor>
-          <anchorOffset>0 0 0</anchorOffset>
-          <axis>0 1 0</axis>
-          <threadPitch>3141.6</threadPitch>
-      </joint:screw>
-    </gazebo>
-    <gazebo>
-      <joint:hinge name="${prefix}_r_parallel_root_joint">
-          <body1>${prefix}_r_parallel_link</body1>
-          <body2>${prefix}_palm_link</body2>
-          <anchor>${prefix}_palm_link</anchor>
-          <axis>0 0 -1</axis>
-          <damping>0.2</damping>
-          <anchorOffset>${0.07691+parallel_link_x_offset} ${-0.01-parallel_link_y_offset} 0</anchorOffset>
-      </joint:hinge>
-      <joint:hinge name="${prefix}_l_parallel_root_joint">
-          <body1>${prefix}_l_parallel_link</body1>
-          <body2>${prefix}_palm_link</body2>
-          <anchor>${prefix}_palm_link</anchor>
-          <axis>0 0 1</axis>
-          <damping>0.2</damping>
-          <anchorOffset>${0.07691+parallel_link_x_offset} ${0.01+parallel_link_y_offset} 0</anchorOffset>
-      </joint:hinge>
-      <joint:hinge name="${prefix}_r_parallel_tip_joint">
-          <body1>${prefix}_r_parallel_link</body1>
-          <body2>${prefix}_r_finger_tip_link</body2>
-          <anchor>${prefix}_r_finger_tip_link</anchor>
-          <axis>0 0 1</axis>
-          <anchorOffset>${parallel_link_x_offset} ${-parallel_link_y_offset} 0</anchorOffset>
-      </joint:hinge>
-      <joint:hinge name="${prefix}_l_parallel_tip_joint">
-          <body1>${prefix}_l_parallel_link</body1>
-          <body2>${prefix}_l_finger_tip_link</body2>
-          <anchor>${prefix}_l_finger_tip_link</anchor>
-          <axis>0 0 1</axis>
-          <anchorOffset>${parallel_link_x_offset} ${parallel_link_y_offset} 0</anchorOffset>
-      </joint:hinge>
-      <joint:slider name="${prefix}_joint">
-          <body1>${prefix}_l_finger_tip_link</body1>
-          <body2>${prefix}_r_finger_tip_link</body2>
-          <anchor>${prefix}_l_finger_tip_link</anchor>
-          <axis>0 1 0</axis>
-      </joint:slider>
+      <link name="${prefix}_l_parallel_link">
+          <inertial>
+            <mass>0.17126</mass>
+            <inertia>
+              <ixx>7.7562e-05</ixx>
+              <ixy>1.49095e-06</ixy>
+              <ixz>-9.83385e-06</ixz>
+              <iyy>0.000197083</iyy>
+              <iyz>-3.06125e-06</iyz>
+              <izz>0.000181054</izz>
+            </inertia>
+            <pose>0.03598 0.0173 -0.00164 0 0 0</pose>
+          </inertial>
+          <pose>0.82991 ${0.188*reflect+0.031} 0.790675 0 -0 0</pose>
+          <gravity>false</gravity>
+      </link>
+      <link name="${prefix}_r_parallel_link">
+          <inertial>
+            <mass>0.17389</mass>
+            <inertia>
+              <ixx>7.73841e-05</ixx>
+              <ixy>-2.09309e-06</ixy>
+              <ixz>-8.36228e-06</ixz>
+              <iyy>0.000198474</iyy>
+              <iyz>2.4611e-06</iyz>
+              <izz>0.00018107</izz>
+            </inertia>
+            <pose>0.03576 -0.01736 -0.00095 0 0 0</pose>
+          </inertial>
+          <pose>0.82991 ${0.188*reflect-0.031} 0.790675 0 0 0</pose>
+          <gravity>false</gravity>
+      </link>
+    </gazebo>
+    <gazebo>
+      <joint type="screw" name="${prefix}_r_screw_screw_joint">
+          <child>${prefix}_motor_screw_link</child>
+          <parent>${prefix}_r_finger_tip_link</parent>
+          <thread_pitch>-3141.6</thread_pitch>
+          <axis>
+            <xyz>0 1 0</xyz>
+          </axis>
+      </joint>
+      <joint type="screw" name="${prefix}_l_screw_screw_joint">
+          <parent>${prefix}_l_finger_tip_link</parent>
+          <child>${prefix}_motor_screw_link</child>
+          <thread_pitch>3141.6</thread_pitch>
+          <axis>
+            <xyz>0 1 0</xyz>
+          </axis>
+      </joint>
+    </gazebo>
+    <gazebo>
+      <joint type="revolute" name="${prefix}_r_parallel_root_joint">
+          <parent>${prefix}_r_parallel_link</parent>
+          <child>${prefix}_palm_link</child>
+          <axis>
+            <xyz>0 0 -1</xyz>
+            <dynamics>
+              <damping>0.2</damping>
+            </dynamics>
+          </axis>
+          <pose>${0.07691+parallel_link_x_offset} ${-0.01-parallel_link_y_offset} 0 0 0 0</pose>
+      </joint>
+      <joint type="revolute" name="${prefix}_l_parallel_root_joint">
+          <parent>${prefix}_l_parallel_link</parent>
+          <child>${prefix}_palm_link</child>
+          <axis>
+            <xyz>0 0 1</xyz>
+            <dynamics>
+              <damping>0.2</damping>
+            </dynamics>
+          </axis>
+          <pose>${0.07691+parallel_link_x_offset} ${0.01+parallel_link_y_offset} 0 0 0 0</pose>
+      </joint>
+      <joint type="revolute" name="${prefix}_r_parallel_tip_joint">
+          <parent>${prefix}_r_parallel_link</parent>
+          <child>${prefix}_r_finger_tip_link</child>
+          <axis>
+            <xyz>0 0 1</xyz>
+          </axis>
+          <pose>${parallel_link_x_offset} ${-parallel_link_y_offset} 0 0 0 0</pose>
+      </joint>
+      <joint type="revolute" name="${prefix}_l_parallel_tip_joint">
+          <parent>${prefix}_l_parallel_link</parent>
+          <child>${prefix}_l_finger_tip_link</child>
+          <axis>
+            <xyz>0 0 1</xyz>
+          </axis>
+          <pose>${parallel_link_x_offset} ${parallel_link_y_offset} 0 0 0 0</pose>
+      </joint>
+      <joint type="prismatic" name="${prefix}_joint">
+          <parent>${prefix}_r_finger_tip_link</parent>
+          <child>${prefix}_l_finger_tip_link</child>
+          <axis>
+            <xyz>0 1 0</xyz>
+          </axis>
+      </joint>
     </gazebo>
     <gazebo reference="${prefix}_motor_slider_link">

File: pr2_description/urdf/sensors/wge100_camera.gazebo.xacro (robot description, xacro)
@@ -7,5 +7,5 @@
         <update_rate>25.0</update_rate>
         <camera>
-          <horizontal_fov>${hfov}</horizontal_fov>
+          <horizontal_fov>${hfov*M_PI/180.0}</horizontal_fov>
           <image>
             <format>${image_format}</format>

File: pr2_description/urdf/torso_v0/torso.gazebo.xacro (robot description, xacro)
@@ -1,28 +1,27 @@
 <?xml version="1.0"?>
-<robot xmlns:sensor="http://playerstage.sourceforge.net/gazebo/xmlschema/#sensor"
-       xmlns:controller="http://playerstage.sourceforge.net/gazebo/xmlschema/#controller"
-       xmlns:joint="http://playerstage.sourceforge.net/gazebo/xmlschema/#joint"
-       xmlns:xacro="http://ros.org/wiki/xacro">
+<robot xmlns:xacro="http://ros.org/wiki/xacro">
   <xacro:macro name="pr2_torso_gazebo_v0" params="name">
     <gazebo reference="${name}_link">
-      <sensor:contact name="${name}_contact_sensor">
-        <geom>${name}_link_geom</geom>
-        <updateRate>100.0</updateRate>
-        <controller:gazebo_ros_bumper name="${name}_gazebo_ros_bumper_controller" plugin="libgazebo_ros_bumper.so">
+      <sensor type="contact" name="${name}_contact_sensor">
+        <contact>
+          <collision>${name}_link_geom</collision>
+        </contact>
+        <update_rate>100.0</update_rate>
+        <plugin name="${name}_gazebo_ros_bumper_controller" filename="libgazebo_ros_bumper.so">
           <alwaysOn>true</alwaysOn>
           <updateRate>100.0</updateRate>
           <bumperTopicName>${name}_bumper</bumperTopicName>
-        </controller:gazebo_ros_bumper>
-      </sensor:contact>
+        </plugin>
+      </sensor>
     </gazebo>
     <gazebo>
-      <joint:screw name="${name}_screw_torso_lift_joint">
-          <body1>${name}_motor_screw_link</body1>
-          <body2>${name}_link</body2>
-          <anchor>${name}_motor_screw_link</anchor>
-          <anchorOffset>0 0 0</anchorOffset>
-          <axis>0 0 1</axis>
-          <threadPitch>3141.6</threadPitch>
-      </joint:screw>
+      <joint type="screw" name="${name}_screw_torso_lift_joint">
+          <parent>${name}_link</parent>
+          <child>${name}_motor_screw_link</child>
+          <axis>
+            <xyz>0 0 1</xyz>
+          </axis>
+          <thread_pitch>3141.6</thread_pitch>
+      </joint>
     </gazebo>
   </xacro:macro>
