Commit message: Lowering torso velocity safety limit to 0.013 m/s after reviewing data from Fx

File: pr2_description/urdf/torso_v0/torso.urdf.xacro (robot description, xacro)
@@ -9,8 +9,6 @@
     <joint name="${name}_joint" type="prismatic">
       <axis xyz="0 0 1" />
-      <!-- KWatts: Max should be 0.31, changed to 0.20 to prevent jamming -->
-      <!-- HW ticket 481, will examine spine to determine failures -->
-      <limit lower="0.0" upper="0.20" effort="10000" velocity="0.015"/>
-      <safety_controller  k_velocity="400000" soft_lower_limit="${0.0+0.005}" soft_upper_limit="${0.20-0.005}" k_position="1000" />
+      <limit lower="0.0" upper="0.31" effort="10000" velocity="0.013"/>
+      <safety_controller  k_velocity="400000" soft_lower_limit="${0.0+0.003}" soft_upper_limit="${0.31-0.005}" k_position="1000" />
       <calibration reference_position="0.00536" />
       <dynamics damping="10.0" />

Commit message: Updating IMU coordinates in pr2_torso macro WG#3286

File: pr2_description/urdf/torso_v0/torso.urdf.xacro (robot description, xacro)
@@ -45,5 +45,5 @@
     <!-- imu -->
     <xacro:microstrain_3dmgx2_imu_v0 name="imu" parent="${name}" ros_topic="imu_data" update_rate="100.0">
-        <origin xyz="0 0 0" rpy="0 0 0" />
+        <origin xyz="-0.02977 -0.1497 0.164" rpy="0 0 0" />
     </xacro:microstrain_3dmgx2_imu_v0>
   </xacro:macro>

Commit message: uppping simulation damping for torso_lift due to increased k_velocity to 2e6 (#3450).

File: pr2_description/urdf/torso_v0/torso.urdf.xacro (robot description, xacro)
@@ -14,5 +14,5 @@
       <!-- hold both reference_position and upper/lower for tick-tock, remove reference_positiion after verifying upper/lower works with calibration controllers.  if search velocity in pr2_calibration_controllers.yaml is +, the reference_position is rising, if - then it is falling -->
       <calibration reference_position="0.00536" falling="0.00536" />
-      <dynamics damping="5000.0" /> <!-- strictly tuned for sim only right now -->
+      <dynamics damping="20000.0" /> <!-- strictly tuned for sim only right now -->
       <insert_block name="origin" />
       <parent link="${parent}"/>

Commit message: #4932 initial draft for new torso side plate frames. slight mismatch with existing visual mesh, pending further verification.

File: pr2_description/urdf/torso_v0/torso.urdf.xacro (robot description, xacro)
@@ -39,4 +39,32 @@
       </collision>
     </link>
+    <joint name="l_${name}_side_plate_joint" type="fixed">
+      <origin xyz="0.0535 -0.209285 0.176625" /> <!-- location of bottom front bolt hole location -->
+      <parent link="${name}_link"/>
+      <child link="l_${name}_side_plate_link"/>
+    </joint>
+    <link name="l_${name}_side_plate_link">
+      <inertial>
+        <mass value="0.1" />
+        <origin xyz="-0.0625 0.0 0.05" />  <!-- center of the 12.5cm by 10cm bolt hole pattern -->
+        <inertia ixx="0.001" ixy="0.0" ixz="0.0"
+                 iyy="0.001" iyz="0.0"
+                 izz="0.001" />
+      </inertial>
+    </link>
+    <joint name="r_${name}_side_plate_joint" type="fixed">
+      <origin xyz="0.0535  0.209285 0.176625" /> <!-- location of bottom front bolt hole location -->
+      <parent link="${name}_link"/>
+      <child link="r_${name}_side_plate_link"/>
+    </joint>
+    <link name="r_${name}_side_plate_link">
+      <inertial>
+        <mass value="0.1" />
+        <origin xyz="-0.0625 0.0 0.05" />  <!-- center of the 12.5cm by 10cm bolt hole pattern -->
+        <inertia ixx="0.001" ixy="0.0" ixz="0.0"
+                 iyy="0.001" iyz="0.0"
+                 izz="0.001" />
+      </inertial>
+    </link>
     <!-- extensions -->
     <xacro:pr2_torso_gazebo_v0 name="${name}" />

Commit message: fix left and right torso side plate link

File: pr2_description/urdf/torso_v0/torso.urdf.xacro (robot description, xacro)
@@ -40,5 +40,5 @@
     </link>
     <joint name="l_${name}_side_plate_joint" type="fixed">
-      <origin xyz="0.0535 -0.209285 0.176625" /> <!-- location of bottom front bolt hole location -->
+      <origin xyz="0.0535 0.209285 0.176625" /> <!-- location of bottom front bolt hole location -->
       <parent link="${name}_link"/>
       <child link="l_${name}_side_plate_link"/>
@@ -54,5 +54,5 @@
     </link>
     <joint name="r_${name}_side_plate_joint" type="fixed">
-      <origin xyz="0.0535  0.209285 0.176625" /> <!-- location of bottom front bolt hole location -->
+      <origin xyz="0.0535  -0.209285 0.176625" /> <!-- location of bottom front bolt hole location -->
       <parent link="${name}_link"/>
       <child link="r_${name}_side_plate_link"/>

Commit message: revert damping value for torso lift

File: pr2_description/urdf/torso_v0/torso.urdf.xacro (robot description, xacro)
@@ -13,5 +13,5 @@
       <safety_controller  k_velocity="2000000" soft_lower_limit="${0.0+0.0115}" soft_upper_limit="${0.31-0.005}" k_position="100" />
       <calibration falling="0.00536" />
-      <dynamics damping="100.0" />
+      <dynamics damping="20000.0" />
       <insert_block name="origin" />
       <parent link="${parent}"/>
