Commit message: Updating PR2 torso transmission limits as specified in PR2 SCDS ticket 1999

File: pr2_description/urdf/torso_v0/torso.transmission.xacro (robot description, xacro)
@@ -8,5 +8,5 @@
       <actuator name="${name}_motor" />
       <joint name="${name}_joint" />
-      <mechanicalReduction>-47275.06</mechanicalReduction>
+      <mechanicalReduction>-47641.53</mechanicalReduction>
       <simulated_actuated_joint name="${name}_motor_screw_joint"
                                 simulated_reduction="3141.6" />

File: pr2_description/urdf/torso_v0/torso.urdf.xacro (robot description, xacro)
@@ -10,7 +10,7 @@
     <joint name="${name}_joint" type="prismatic">
       <axis xyz="0 0 1" />
-      <limit lower="0.0" upper="0.31" effort="10000" velocity="0.013"/> <!-- alpha tested velocity and effort limits -->
-      <safety_controller  k_velocity="2000000" soft_lower_limit="${0.0+0.0115}" soft_upper_limit="${0.31-0.005}" k_position="100" />
-      <calibration falling="0.00536" />
+      <limit lower="0.0" upper="0.33" effort="10000" velocity="0.013"/> <!-- alpha tested velocity and effort limits -->
+      <safety_controller  k_velocity="2000000" soft_lower_limit="${0.0+0.0115}" soft_upper_limit="${0.33-0.005}" k_position="100" />
+      <calibration falling="0.00475" />
       <dynamics damping="20000.0" />
       <insert_block name="origin" />
