Commit message: Added rgb and ir frames.

File: pr2_description/test.urdf (robot description, URDF)
Before this commit: robot pr2, 91 links, 90 joints
Links:
- added link head_mount_kinect2_ir_optical_frame
- added link head_mount_kinect2_rgb_optical_frame
Joints:
- added joint head_mount_kinect2_ir_optical_frame_joint: type fixed, parent head_mount_kinect2_ir_link, child head_mount_kinect2_ir_optical_frame
- added joint head_mount_kinect2_rgb_optical_frame_joint: type fixed, parent head_mount_kinect2_rgb_link, child head_mount_kinect2_rgb_optical_frame
- joint head_mount_kinect2_rgb_joint: origin xyz=0 -0.052 0 rpy=0 0 0 -> xyz=0 -0.05175 0 rpy=0 0 0

File: pr2_description/urdf/sensors/kinect2.gazebo.xacro (robot description, xacro)
@@ -88,18 +88,3 @@
   </gazebo>
 </xacro:macro>
-<xacro:macro name="kinect2_prosilica_gazebo" params="joint_name link_name">
-  <gazebo>
-    <plugin name="${link_name}_srp_controller" filename="libgazebo_ros_srp.so">
-      <bodyName>${link_name}</bodyName>
-      <jointName>${joint_name}</jointName>
-      <topicName>${link_name}</topicName>
-    </plugin>
-  </gazebo>
-  <!-- also add transmission for this sliding joint -->
-  <transmission type="pr2_mechanism_model/SimpleTransmission" name="${joint_name}_trans">
-    <actuator name="${joint_name}_motor" />
-    <joint name="${joint_name}" />
-    <mechanicalReduction>1</mechanicalReduction>
-  </transmission>
-</xacro:macro>
 </robot>

File: pr2_description/urdf/sensors/kinect2.urdf.xacro (robot description, xacro)
@@ -1,7 +1,4 @@
 <?xml version="1.0"?>
 <robot xmlns:xacro="http://ros.org/wiki/xacro">
-  <!-- Instead of making a xacro for each individual component, create one .STL for the frame, mount and the Kinect2 -->
-  <!-- Multiple components is also likely the cause of the tf linking problem -->
-  <!-- Depending on where origin is for the mesh, a joint and link may be needed for the camera/ir sensor -->
   <xacro:include filename="$(find pr2_description)/urdf/sensors/kinect2.gazebo.xacro" />
   <property name="ir_depth_rgb_offset_y" value="0.01"/> <!-- FIXME: what is this offset? -->
@@ -65,16 +62,16 @@
     </link>
     <!-- kinect2 ir sensor frame -->
-<!--     <joint name="${name}_kinect2_ir_optical_frame_joint" type="fixed">
-      <origin xyz="${cal_kinect_x}            ${cal_kinect_y + ir_depth_rgb_offset_y}         ${cal_kinect_z}"
-                rpy="${-M_PI/2+cal_kinect_roll} ${0.0+cal_kinect_pitch} ${-M_PI/2+cal_kinect_yaw}" />
+    <joint name="${name}_kinect2_ir_optical_frame_joint" type="fixed">
+<!--       <origin xyz="${cal_kinect_x}                         ${cal_kinect_y + ir_depth_rgb_offset_y} {cal_kinect_z}"
+              rpy="${-M_PI/2+cal_kinect_roll}              ${0.0+cal_kinect_pitch}                 ${-M_PI/2+cal_kinect_yaw}" /> -->
       <parent link="${name}_kinect2_ir_link"/>
       <child link="${name}_kinect2_ir_optical_frame"/>
     </joint>
-    <link name="${name}_kinect2_ir_optical_frame"/> -->
+    <link name="${name}_kinect2_ir_optical_frame"/>
     <!-- gazebo extensions -->
-<!--     <xacro:kinect2_ir_gazebo_v0 link_name="${name}_kinect2_ir_link" frame_name="${name}_kinect2_ir_optical_frame" camera_name="head_mount_kinect2" /> -->
+    <xacro:kinect2_ir_gazebo_v0 link_name="${name}_kinect2_ir_link" frame_name="${name}_kinect2_ir_optical_frame" camera_name="head_mount_kinect2" />
     <!-- kinect2 rgb sensor physical attachment -->
     <joint name="${name}_kinect2_rgb_joint" type="fixed">
-      <origin xyz="0 -0.052 0" rpy="0 0 0"/>
+      <origin xyz="0 -0.05175 0" rpy="0 0 0"/>
       <parent link="${name}_kinect2_ir_link"/>
       <child link="${name}_kinect2_rgb_link"/>
@@ -89,5 +86,6 @@
       </inertial>
       <visual>
-        <origin xyz="0.0 0.0 0" rpy="0 0 0"/>
+<!--         <origin xyz="${cal_kinect_x}            ${cal_kinect_y}            ${cal_kinect_z}"
+                rpy="${-M_PI/2+cal_kinect_roll} ${0.0+cal_kinect_pitch}    ${-M_PI/2+cal_kinect_yaw}" /> -->
         <geometry>
           <sphere radius="0.0005"/>
@@ -102,13 +100,13 @@
     </link>
     <!-- kinect2 rgb sensor frame -->
-<!--     <joint name="${name}_kinect2_rgb_optical_frame_joint" type="fixed">
-      <origin xyz="${cal_kinect_x}            ${cal_kinect_y}         ${cal_kinect_z}"
-                rpy="${-M_PI/2+cal_kinect_roll} ${0.0+cal_kinect_pitch} ${-M_PI/2+cal_kinect_yaw}" />
+    <joint name="${name}_kinect2_rgb_optical_frame_joint" type="fixed">
+<!--       <origin xyz="${cal_kinect_x}            ${cal_kinect_y}            ${cal_kinect_z}"
+              rpy="${-M_PI/2+cal_kinect_roll} ${0.0+cal_kinect_pitch}    ${-M_PI/2+cal_kinect_yaw}" /> -->
       <parent link="${name}_kinect2_rgb_link"/>
       <child link="${name}_kinect2_rgb_optical_frame"/>
     </joint>
-    <link name="${name}_kinect2_rgb_optical_frame"/> -->
+    <link name="${name}_kinect2_rgb_optical_frame"/>
     <!-- gazebo extensions -->
-<!--     <xacro:kinect2_rgb_gazebo_v0 link_name="${name}_kinect2_rgb_link" frame_name="${name}_kinect2_rgb_optical_frame" camera_name="head_mount_kinect2" /> -->
+    <xacro:kinect2_rgb_gazebo_v0 link_name="${name}_kinect2_rgb_link" frame_name="${name}_kinect2_rgb_optical_frame" camera_name="head_mount_kinect2" />
   </xacro:macro>
 </robot>
