Commit message: Setting head limits to values given by Fx-Fong 10/23/09

File: pr2_description/urdf/head_v0/head.urdf.xacro (robot description, xacro)
@@ -10,7 +10,7 @@
     <joint name="${name}_joint" type="revolute">
       <axis xyz="0 0 1" />
-      <limit lower="-2.92" upper="2.92" effort="2.645" velocity="6" />
-      <safety_controller k_velocity="1.5" soft_lower_limit="${-2.92+0.15}" soft_upper_limit="${2.92-0.15}" k_position="100" />
-      <calibration reference_position="${-2.79+cal_head_pan_flag}" />
+      <limit lower="-3.038729" upper="3.0368729" effort="2.645" velocity="6" />
+      <safety_controller k_velocity="1.5" soft_lower_limit="${-3.038729+0.20}" soft_upper_limit="${3.0368729-0.20}" k_position="100" />
+      <calibration reference_position="${0.0+cal_head_pan_flag}" />
       <dynamics damping="1.0" />
       <insert_block name="origin" />
@@ -28,5 +28,5 @@
         <origin xyz="0 0 0.0" rpy="0 0 0 " />
         <geometry name="${name}_visual_geom">
-          <mesh filename="package://pr2_description/head_v0/meshes/head_pan.stl" />
+          <mesh filename="package://pr2_description/meshes/head_v0/head_pan.stl" />
         </geometry>
         <material name="Blue" />
@@ -46,7 +46,7 @@
     <joint name="${name}_joint" type="revolute">
       <axis xyz="0 1 0" />
-      <limit lower="-0.55" upper="1.047" effort="12.21" velocity="100" />
+      <limit lower="-0.471238" upper="1.39626" effort="12.21" velocity="100" />
       <safety_controller k_velocity="1.5" soft_lower_limit="${-0.55+0.02}" soft_upper_limit="${1.047-0.002}" k_position="100" />
-      <calibration reference_position="${-0.195+cal_head_tilt_flag}" />
+      <calibration reference_position="${0.0+cal_head_tilt_flag}" />
       <dynamics damping="20.0" />
       <insert_block name="origin" />
@@ -65,5 +65,5 @@
         <origin xyz="0 0 0" rpy="0.0 0.0 0.0 " />
         <geometry name="${name}_visual_geom">
-          <mesh filename="package://pr2_description/head_v0/meshes/head_tilt.stl" />
+          <mesh filename="package://pr2_description/meshes/head_v0/head_tilt.stl" />
         </geometry>
         <material name="Green" />

File: pr2_description/urdf/tilting_laser_v0/tilting_laser.urdf.xacro (robot description, xacro)
@@ -10,5 +10,5 @@
     <joint name="${name}_mount_joint" type="revolute">
       <axis xyz="0 1 0" />
-      <limit lower="-0.785" upper="1.57" effort="0.5292" velocity="10.0" />
+      <limit lower="-0.7854" upper="1.48353" effort="0.5292" velocity="10.0" />
       <safety_controller k_position="100" k_velocity="0.05" soft_lower_limit="${-0.785+0.0}" soft_upper_limit="${1.57-0.0}" />
       <calibration reference_position="${laser_calib_ref}" />

Commit message: Head URDF fixes to joint limits for Beta head

File: pr2_description/urdf/head_v0/head.urdf.xacro (robot description, xacro)
@@ -10,6 +10,6 @@
     <joint name="${name}_joint" type="revolute">
       <axis xyz="0 0 1" />
-      <limit lower="-3.038729" upper="3.0368729" effort="2.645" velocity="6" />
-      <safety_controller k_velocity="1.5" soft_lower_limit="${-3.038729+0.20}" soft_upper_limit="${3.0368729-0.20}" k_position="100" />
+      <limit lower="-3.007" upper="3.007" effort="2.645" velocity="6" />
+      <safety_controller k_velocity="1.5" soft_lower_limit="${-3.007+0.10}" soft_upper_limit="${3.007-0.10}" k_position="100" />
       <calibration reference_position="${0.0+cal_head_pan_flag}" />
       <dynamics damping="1.0" />
@@ -46,6 +46,6 @@
     <joint name="${name}_joint" type="revolute">
       <axis xyz="0 1 0" />
-      <limit lower="-0.471238" upper="1.39626" effort="12.21" velocity="100" />
-      <safety_controller k_velocity="1.5" soft_lower_limit="${-0.55+0.02}" soft_upper_limit="${1.047-0.002}" k_position="100" />
+      <limit lower="-0.471238" upper="1.39626" effort="15" velocity="100" />
+      <safety_controller k_velocity="1.5" soft_lower_limit="${-0.4712 + 0.05}" soft_upper_limit="${1.39626 - 0.05}" k_position="100" />
       <calibration reference_position="${0.0+cal_head_tilt_flag}" />
       <dynamics damping="20.0" />

Commit message: Changing Beta head pan/tilt joint safety limits to prevent damage in life test

File: pr2_description/urdf/head_v0/head.urdf.xacro (robot description, xacro)
@@ -11,5 +11,5 @@
       <axis xyz="0 0 1" />
       <limit lower="-3.007" upper="3.007" effort="2.645" velocity="6" />
-      <safety_controller k_velocity="1.5" soft_lower_limit="${-3.007+0.10}" soft_upper_limit="${3.007-0.10}" k_position="100" />
+      <safety_controller k_velocity="1.5" soft_lower_limit="${-3.007+0.15}" soft_upper_limit="${3.007-0.15}" k_position="100" />
       <calibration reference_position="${0.0+cal_head_pan_flag}" />
       <dynamics damping="1.0" />
@@ -46,6 +46,6 @@
     <joint name="${name}_joint" type="revolute">
       <axis xyz="0 1 0" />
-      <limit lower="-0.471238" upper="1.39626" effort="15" velocity="100" />
-      <safety_controller k_velocity="1.5" soft_lower_limit="${-0.4712 + 0.05}" soft_upper_limit="${1.39626 - 0.05}" k_position="100" />
+      <limit lower="-0.471238" upper="1.39626" effort="15" velocity="5" />
+      <safety_controller k_velocity="1.5" soft_lower_limit="${-0.4712 + 0.1}" soft_upper_limit="${1.39626 - 0.1}" k_position="100" />
       <calibration reference_position="${0.0+cal_head_tilt_flag}" />
       <dynamics damping="20.0" />

Commit message: Lowering head tilt damping for gazebo

File: pr2_description/urdf/head_v0/head.urdf.xacro (robot description, xacro)
@@ -49,5 +49,5 @@
       <safety_controller k_velocity="1.5" soft_lower_limit="${-0.4712 + 0.1}" soft_upper_limit="${1.39626 - 0.1}" k_position="100" />
       <calibration reference_position="${0.0+cal_head_tilt_flag}" />
-      <dynamics damping="20.0" />
+      <dynamics damping="1.0" />
       <insert_block name="origin" />
       <parent link="${parent}"/>

Commit message: remove name tag for visual, collision, geometry (not used by urdf)

File: pr2_description/urdf/head_v0/head.urdf.xacro (robot description, xacro)
@@ -25,14 +25,14 @@
                  iyy="0.005218991412"  iyz="-0.000314239509"  izz="0.008618784925" />
       </inertial>
-      <visual name="${name}_visual">
+      <visual>
         <origin xyz="0 0 0.0" rpy="0 0 0 " />
-        <geometry name="${name}_visual_geom">
+        <geometry>
           <mesh filename="package://pr2_description/meshes/head_v0/head_pan.stl" />
         </geometry>
         <material name="Blue" />
       </visual>
-      <collision name="${name}_collision">
+      <collision>
         <origin xyz="-0.005717  0.010312 -0.029649" rpy="0.0 0.0 0.0 " />
-        <geometry name="${name}_collision_geom">
+        <geometry>
           <box size="0.188 0.219 0.137" />
         </geometry>
@@ -62,14 +62,14 @@
                  izz="0.005516790626" />
       </inertial>
-      <visual name="${name}_visual">
-        <origin xyz="0 0 0" rpy="0.0 0.0 0.0 " />
-        <geometry name="${name}_visual_geom">
+      <visual>
+        <origin xyz="0 0 0" rpy="0.0 0.0 0.0" />
+        <geometry>
           <mesh filename="package://pr2_description/meshes/head_v0/head_tilt.stl" />
         </geometry>
         <material name="Green" />
       </visual>
-      <collision name="${name}_collision">
+      <collision>
         <origin xyz="0.041935 0.003569 0.028143" rpy="0 0 0" />
-        <geometry name="${name}_collision_geom">
+        <geometry>
           <box size="0.064 0.253 0.181" />
         </geometry>
@@ -101,14 +101,14 @@
                  izz="0.001" />
       </inertial>
-      <visual name="${name}_plate_frame_visual">
+      <visual>
         <origin xyz="0 0 0" rpy="0 0 0" />
-        <geometry name="${name}_plate_frame_visual_geom">
+        <geometry>
           <box size="0.01 0.01 0.01" />
         </geometry>
         <material name="Blue" />
       </visual>
-      <collision name="${name}_plate_frame_collision">
+      <collision>
         <origin xyz="0 0 0" rpy="0 0 0" />
-        <geometry name="${name}_plate_frame_collision_geom">
+        <geometry>
           <box size="0.01 0.01 0.01" />
         </geometry>

Commit message: #4296, updated head pan and head tilt masses per spreadsheet 100505_link_data.xls

File: pr2_description/urdf/head_v0/head.urdf.xacro (robot description, xacro)
@@ -20,8 +20,8 @@
     <link name="${name}_link">
       <inertial>
-        <mass value="1.611118" />
-        <origin xyz="-0.005717  0.010312 -0.029649" rpy="0 0 0" />
-        <inertia ixx="0.00482611007"  ixy="-0.000144683999"  ixz="0.000110076136"
-                 iyy="0.005218991412"  iyz="-0.000314239509"  izz="0.008618784925" />
+        <mass value="6.339" /> <!-- mass/cog/moi updated per 100505_link_data.xls -->
+        <origin xyz="0.010907 0.031693 0.090507" rpy="0 0 0" />
+        <inertia ixx="0.032497592"  ixy="0.00063604088"  ixz="0.0025851534"
+                 iyy="0.046545627"  iyz="-0.0024534295"  izz="0.057652724" />
       </inertial>
       <visual>
@@ -55,9 +55,9 @@
     <link name="${name}_link">
       <inertial>
-        <mass value="1.749727" />
-        <origin xyz="0.041935 0.003569 0.028143" rpy="0 0 0" />
-        <inertia ixx="0.010602303435"  ixy="-0.000408814235"  ixz="0.00198303894"
-                 iyy="0.011874383747"  iyz="0.000197908779"
-                 izz="0.005516790626" />
+        <mass value="4.479" /> <!-- mass/cog/moi updated per 100505_link_data.xls -->
+        <origin xyz="0.001716 -0.019556 0.055002" rpy="0 0 0" />
+        <inertia ixx="0.024223222"  ixy="0.00062063507"  ixz="-0.000096909696"
+                 iyy="0.054723086"  iyz="0.00279702400"
+                 izz="0.067306377" />
       </inertial>
       <visual>

Commit message: Increasing max effort of head tilt joint, #5141

File: pr2_description/urdf/head_v0/head.urdf.xacro (robot description, xacro)
@@ -44,5 +44,5 @@
     <joint name="${name}_joint" type="revolute">
       <axis xyz="0 1 0" />
-      <limit lower="-0.471238" upper="1.39626" effort="15" velocity="5" /> <!-- alpha tested velocity and effort limits -->
+      <limit lower="-0.471238" upper="1.39626" effort="18" velocity="5" /> <!-- alpha tested velocity and effort limits -->
       <safety_controller k_velocity="3.0" soft_lower_limit="${-0.4712 + 0.1}" soft_upper_limit="${1.39626 - 0.1}" k_position="100" />
       <calibration falling="${0.0+cal_head_tilt_flag}" />

Commit message: change head pan/tilt damping (too low from sushi runs)

File: pr2_description/urdf/head_v0/head.urdf.xacro (robot description, xacro)
@@ -13,5 +13,5 @@
       <safety_controller k_velocity="1.5" soft_lower_limit="${-3.007+0.15}" soft_upper_limit="${3.007-0.15}" k_position="100" />
       <calibration rising="0.0" />
-      <dynamics damping="1.0" />
+      <dynamics damping="2.0" />
       <insert_block name="origin" />
       <parent link="${parent}"/>
@@ -47,5 +47,5 @@
       <safety_controller k_velocity="3.0" soft_lower_limit="${-0.4712 + 0.1}" soft_upper_limit="${1.39626 - 0.1}" k_position="100" />
       <calibration falling="${0.0+cal_head_tilt_flag}" />
-      <dynamics damping="1.0" />
+      <dynamics damping="10.0" />
       <insert_block name="origin" />
       <parent link="${parent}"/>

Commit message: test reduce head pan damping as the head pan is much slower than real life

File: pr2_description/urdf/head_v0/head.urdf.xacro (robot description, xacro)
@@ -13,5 +13,5 @@
       <safety_controller k_velocity="1.5" soft_lower_limit="${-3.007+0.15}" soft_upper_limit="${3.007-0.15}" k_position="100" />
       <calibration rising="0.0" />
-      <dynamics damping="2.0" />
+      <dynamics damping="0.5" />
       <insert_block name="origin" />
       <parent link="${parent}"/>

Commit message: set default values of calib parameters in each property block

File: pr2_description/urdf/head_v0/head.urdf.xacro (robot description, xacro)
@@ -4,5 +4,5 @@
   <xacro:include filename="$(find pr2_description)/urdf/head_v0/head.transmission.xacro" />
   <xacro:property name="M_PI" value="3.1415926535897931" />
-  <xacro:macro name="pr2_head_pan_v0" params="name parent *origin head_pan_calib_ref">
+  <xacro:macro name="pr2_head_pan_v0" params="name parent *origin head_pan_calib_ref:=0.0">
     <joint name="${name}_joint" type="revolute">
       <axis xyz="0 0 1" />
@@ -38,5 +38,5 @@
     <xacro:pr2_head_pan_transmission_v0 name="${name}" />
   </xacro:macro>
-  <xacro:macro name="pr2_head_tilt_v0" params="name parent *origin head_tilt_calib_ref">
+  <xacro:macro name="pr2_head_tilt_v0" params="name parent *origin head_tilt_calib_ref:=0.0">
     <joint name="${name}_joint" type="revolute">
       <axis xyz="0 1 0" />

File: pr2_description/urdf/shoulder_v0/shoulder.urdf.xacro (robot description, xacro)
@@ -108,5 +108,5 @@
   <!-- Upperarm roll: internal fixed attchment point for upper arm -->
   <xacro:macro name="pr2_upper_arm_roll_v0" params="side parent reflect *origin
-    upper_arm_roll_calib_ref">
+    upper_arm_roll_calib_ref:=0.0">
     <joint name="${side}_upper_arm_roll_joint" type="revolute" >
       <axis xyz="1 0 0" />

File: pr2_description/urdf/tilting_laser_v0/tilting_laser.urdf.xacro (robot description, xacro)
@@ -4,5 +4,5 @@
   <xacro:include filename="$(find pr2_description)/urdf/tilting_laser_v0/tilting_laser.transmission.xacro" />
   <xacro:include filename="$(find pr2_description)/urdf/sensors/hokuyo_lx30_laser.urdf.xacro" />
-  <xacro:macro name="pr2_tilting_laser_v0" params="name parent laser_calib_ref *origin">
+  <xacro:macro name="pr2_tilting_laser_v0" params="name parent laser_calib_ref:=0.0 *origin">
     <joint name="${name}_mount_joint" type="revolute">
       <axis xyz="0 1 0" />

File: pr2_description/urdf/upper_arm_v0/upper_arm.urdf.xacro (robot description, xacro)
@@ -72,5 +72,5 @@
   </xacro:macro>
   <xacro:macro name="pr2_elbow_flex_v0" params="side parent reflect
-   elbow_flex_calib_ref">
+   elbow_flex_calib_ref:=0.0">
     <!-- Elbow flex -->
     <joint name="${side}_elbow_flex_joint" type="revolute">
@@ -117,5 +117,5 @@
   <!-- FA roll joint only -->
   <xacro:macro name="pr2_forearm_roll_v0" params="side parent reflect
-   forearm_roll_calib_ref">
+   forearm_roll_calib_ref:=0.0">
     <!-- forearm_roll_link is a fictitious link internal to elbow_flex_link, provides an attachment point for the actual forearm -->
     <joint name="${side}_forearm_roll_joint" type="continuous">
